Commit message: Update folder structure and kinematics tree visualization

File: toddleroid/robot_descriptions/sustaina_op/sustaina_op.urdf (robot description, URDF)
Before this commit: robot SUSTAINA-OP, 35 links, 34 joints
Links:
- link body_link: geometry collision mesh filename=package:///meshes/body.stl; visual mesh filename=package:///meshes/body.stl
- link head_yaw_link: geometry collision mesh filename=package:///meshes/head.stl; visual mesh filename=package:///meshes/head.stl
- link left_ankle_pitch_link: geometry collision mesh filename=package:///meshes/ankle_pitch.stl; visual mesh filename=package:///meshes/ankle_pitch.stl
- link left_ankle_roll_link: geometry collision mesh filename=package:///meshes/ankle_roll_left.stl; visual mesh filename=package:///meshes/ankle_roll_left.stl
- link left_independent_pitch_link: geometry collision mesh filename=package:///meshes/independent_pitch.stl; visual mesh filename=package:///meshes/independent_pitch.stl
- link left_knee_pitch_link: geometry collision mesh filename=package:///meshes/knee_pitch.stl; visual mesh filename=package:///meshes/knee_pitch.stl
- link left_lower_arm_link: geometry collision mesh filename=package:///meshes/hand.stl; visual mesh filename=package:///meshes/hand.stl
- link left_shin_pitch_link: geometry collision mesh filename=package:///meshes/waist_pitch.stl; visual mesh filename=package:///meshes/waist_pitch.stl
- link left_shin_pitch_mimic_link: geometry collision mesh filename=package:///meshes/waist_pitch_mimic.stl; visual mesh filename=package:///meshes/waist_pitch_mimic.stl
- link left_shoulder_link: geometry collision mesh filename=package:///meshes/shoulder.stl; visual mesh filename=package:///meshes/shoulder.stl
- link left_slider_crank_link: geometry collision mesh filename=package:///meshes/slider_crank.stl; visual mesh filename=package:///meshes/slider_crank.stl
- link left_upper_arm_link: geometry collision mesh filename=package:///meshes/arm.stl; visual mesh filename=package:///meshes/arm.stl
- link left_waist_pitch_link: geometry collision mesh filename=package:///meshes/waist_pitch.stl; visual mesh filename=package:///meshes/waist_pitch.stl
- link left_waist_pitch_mimic_link: geometry collision mesh filename=package:///meshes/waist_pitch_mimic.stl; visual mesh filename=package:///meshes/waist_pitch_mimic.stl
- link left_waist_roll_link: geometry collision mesh filename=package:///meshes/waist_roll.stl; visual mesh filename=package:///meshes/waist_roll.stl
- link left_waist_yaw_link: geometry collision mesh filename=package:///meshes/waist_yaw.stl; visual mesh filename=package:///meshes/waist_yaw.stl
- link right_ankle_pitch_link: geometry collision mesh filename=package:///meshes/ankle_pitch.stl; visual mesh filename=package:///meshes/ankle_pitch.stl
- link right_ankle_roll_link: geometry collision mesh filename=package:///meshes/ankle_roll_right.stl; visual mesh filename=package:///meshes/ankle_roll_right.stl
- link right_independent_pitch_link: geometry collision mesh filename=package:///meshes/independent_pitch.stl; visual mesh filename=package:///meshes/independent_pitch.stl
- link right_knee_pitch_link: geometry collision mesh filename=package:///meshes/knee_pitch.stl; visual mesh filename=package:///meshes/knee_pitch.stl
- link right_lower_arm_link: geometry collision mesh filename=package:///meshes/hand.stl; visual mesh filename=package:///meshes/hand.stl
- link right_shin_pitch_link: geometry collision mesh filename=package:///meshes/waist_pitch.stl; visual mesh filename=package:///meshes/waist_pitch.stl
- link right_shin_pitch_mimic_link: geometry collision mesh filename=package:///meshes/waist_pitch_mimic.stl; visual mesh filename=package:///meshes/waist_pitch_mimic.stl
- link right_shoulder_link: geometry collision mesh filename=package:///meshes/shoulder.stl; visual mesh filename=package:///meshes/shoulder.stl
- link right_slider_crank_link: geometry collision mesh filename=package:///meshes/slider_crank.stl; visual mesh filename=package:///meshes/slider_crank.stl
- link right_upper_arm_link: geometry collision mesh filename=package:///meshes/arm.stl; visual mesh filename=package:///meshes/arm.stl
- link right_waist_pitch_link: geometry collision mesh filename=package:///meshes/waist_pitch.stl; visual mesh filename=package:///meshes/waist_pitch.stl
- link right_waist_pitch_mimic_link: geometry collision mesh filename=package:///meshes/waist_pitch_mimic.stl; visual mesh filename=package:///meshes/waist_pitch_mimic.stl
- link right_waist_roll_link: geometry collision mesh filename=package:///meshes/waist_roll.stl; visual mesh filename=package:///meshes/waist_roll.stl
- link right_waist_yaw_link: geometry collision mesh filename=package:///meshes/waist_yaw.stl; visual mesh filename=package:///meshes/waist_yaw.stl
