Commit message: Streamline the mujoco test of urdf

File: toddleroid/robot_descriptions/base/base.urdf (robot description, URDF)
Before this commit: robot base, 22 links, 21 joints
Links:
- removed link closing_ank_act1_1
- removed link closing_ank_act1_2
- removed link closing_ank_act2_1
- removed link closing_ank_act2_2
- link ank_act_link: mass 0.014875829689094588817 -> 0.044782197696050358993
- link ank_act_link_2: mass 0.014875829689094592287 -> 0.044782197696050352054
- link ank_act_link_head: mass 0.001013742855626921513 -> 0.0030517714925792842166
- link ank_act_link_head_2: mass 0.001013742855626921513 -> 0.0030517714925792842166
- link ank_act_rod: mass 0.00089508237670679559241 -> 0.0026945559868381376359
- link ank_act_rod_2: mass 0.00089508237670679559241 -> 0.0026945559868381376359
- link ank_act_rod_head: mass 0.00021950575367189157174 -> 0.00066080012085386230676
- link ank_act_rod_head_2: mass 0.00021950575367189157174 -> 0.00066080012085386230676
- link ank_b_link: mass 0.0018061238347465617769 -> 0.00089583742203429468642
- link ank_b_link_2: mass 0.0018061238347465617769 -> 0.00089583742203429468642
- link ank_base_link: mass 0.028754206043588168701 -> 0.014262086197619731551
- link ank_pitch_link: mass 0.0030690306166371106658 -> 0.0041366725921694342399
- link ank_rigid_foot_link: mass 0.016563983404687340067 -> 0.0082157357687249205763
- link ank_roll_link: mass 0.01093507166678692015 -> 0.0054237955467263095424
- link ank_rr_link: mass 0.00095937776863479966132 -> 0.00047585137324286067191
- link ank_rr_link_2: mass 0.00095937776863479966132 -> 0.00047585137324286067191
- link hip_pitch_link: mass 0.032344925814368437333 -> 0.016043083203926743197
- link knee_link: mass 0.0088445512816305894843 -> 0.0043868974356887704968
Joints:
- removed joint ank_B11_passive
- removed joint ank_B12_passive
- removed joint ank_B21_passive
- removed joint ank_B22_passive
- removed joint ank_B31_passive
- removed joint ank_B32_passive
- removed joint ank_R11_passive
- removed joint ank_R12_passive
- removed joint ank_R21_passive
- removed joint ank_R22_passive
- removed joint ank_act1_passive
- removed joint ank_act2_passive
- removed joint closing_ank_act1_1_frame
- removed joint closing_ank_act1_2_frame
- removed joint closing_ank_act2_1_frame
- removed joint closing_ank_act2_2_frame
- added joint ank_B11: type revolute, parent ank_base_link, child ank_b_link, origin xyz=0.018680019623524654615 0.010000000000000702771 0.023399999999999573919 rpy=-1.5707963267948796826 -1.5053435939903385687 1.5707963267951574604, axis 0 0 1, limit lower=-3.141592653589793116 upper=0 effort=1 velocity=20
- added joint ank_B12: type revolute, parent ank_base_link, child ank_b_link_2, origin xyz=0.019999999999999386324 0.010000000000000314193 -0.011499999999999789904 rpy=1.5707963267948996666 1.4913243300613441278 1.5707963267949569541, axis 0 0 1, limit lower=-1.570796326794896558 upper=1.570796326794896558 effort=1 velocity=20
- added joint ank_B21: type revolute, parent ank_b_link, child ank_act_link_head, origin xyz=-0.0045000000000000126704 0 -0.016999999999999990813 rpy=1.570796326794891451 1.5534345204864312695 -1.5707963267939346608, axis 0 0 1, limit lower=-1.570796326794896558 upper=1.570796326794896558 effort=1 velocity=20
- added joint ank_B22: type revolute, parent ank_b_link_2, child ank_act_link_head_2, origin xyz=0.0044999999999999987926 -5.5511151231257827021e-17 0.016999999999999983874 rpy=-1.5707963267945563857 -1.5676670190976655928 -1.5707963267937707919, axis 0 0 1, limit lower=-1.570796326794896558 upper=1.570796326794896558 effort=1 velocity=20
- added joint ank_B31: type revolute, parent ank_act_link_head, child ank_act_link, origin xyz=-6.9388939039072283776e-18 -0.0060499999999999998224 -0.0043000000000000104111 rpy=1.5707963267948956698 5.4574690063281408408e-06 -3.1415926535897900074, axis 0 0 1, limit lower=-1.570796326794896558 upper=1.570796326794896558 effort=1 velocity=20
- added joint ank_B32: type revolute, parent ank_act_link_head_2, child ank_act_link_2, origin xyz=-4.1633363423443370266e-17 -0.0060499999999999720668 -0.0042999999999999635736 rpy=1.5707963267948958919 5.4574691649268270539e-06 3.1415926535897900074, axis 0 0 1, limit lower=-1.570796326794896558 upper=1.570796326794896558 effort=1 velocity=20
- added joint ank_R11: type revolute, parent ank_roll_link, child ank_rr_link, origin xyz=0.009999999999999995004 -0.01250000000000002498 0.040599999999999976386 rpy=4.5538414498539748188e-14 8.2432841012071876929e-15 3.0761399207850028681, axis 0 0 1, limit lower=-1.570796326794896558 upper=1.570796326794896558 effort=1 velocity=20
- added joint ank_R12: type revolute, parent ank_roll_link, child ank_rr_link_2, origin xyz=-0.0099999999999999845957 -0.012500000000000052736 0.040599999999999969447 rpy=-4.7709545858758676013e-14 1.2384261596296442717e-14 0.079471996733595215434, axis 0 0 1, limit lower=-1.570796326794896558 upper=1.570796326794896558 effort=1 velocity=20
- added joint ank_R21: type revolute, parent ank_rr_link, child ank_act_rod_head, origin xyz=0.001999999999999990067 -0.0099999999999999672484 -0.0019000000000000058509 rpy=-1.5707963267948636954 -1.5534345204865058765 -1.5707963267948001906, axis 0 0 1, limit lower=-1.570796326794896558 upper=1.570796326794896558 effort=1 velocity=20
- added joint ank_R22: type revolute, parent ank_rr_link_2, child ank_act_rod_head_2, origin xyz=0.0020000000000000139194 0.010000000000000050515 -0.0019000000000000127898 rpy=-1.5707963267951321473 1.5676670190976929042 -1.5707963267984343947, axis 0 0 1, limit lower=-1.570796326794896558 upper=1.570796326794896558 effort=1 velocity=20
- added joint ank_act1: type prismatic, parent ank_act_link, child ank_act_rod, origin xyz=2.2722093444352275959e-06 -2.0041477158394549463e-15 -0.059207313423200264024 rpy=3.141592653589793116 -7.1063902759635634618e-15 -0.636713564420013034, axis 0 0 1, limit lower=-0.017000000000000001221 upper=0.017000000000000001221 effort=1 velocity=20
- added joint ank_act2: type prismatic, parent ank_act_link_2, child ank_act_rod_2, origin xyz=2.2722093450874836229e-06 -8.5521867365656589755e-16 -0.059245886443141021482 rpy=-3.141592653589793116 7.4572825813947619791e-15 -0.63671356442005910825, axis 0 0 1, limit lower=-0.017000000000000001221 upper=0.017000000000000001221 effort=1 velocity=20
