Commit message: Import the humanoid urdf

File: toddleroid/robot_descriptions/base/base.urdf (robot description, URDF)
Before this commit: robot base, 18 links, 17 joints
Links:
- removed link ank_base_link
- added link ank_act_link_3, mass 0.044782197696050352054; collision mesh filename=package:///meshes/ank_act_link_3_collision.stl; visual mesh filename=package:///meshes/ank_act_link_3_visual.stl
- added link ank_act_link_4, mass 0.044782197696050352054; collision mesh filename=package:///meshes/ank_act_link_4_collision.stl; visual mesh filename=package:///meshes/ank_act_link_4_visual.stl
- added link ank_act_link_head_3, mass 0.0030517714925792842166; collision mesh filename=package:///meshes/ank_act_link_head_3_collision.stl; visual mesh filename=package:///meshes/ank_act_link_head_3_visual.stl
- added link ank_act_link_head_4, mass 0.0030517714925792842166; collision mesh filename=package:///meshes/ank_act_link_head_4_collision.stl; visual mesh filename=package:///meshes/ank_act_link_head_4_visual.stl
- added link ank_act_rod_3, mass 0.0026945559868381376359; collision mesh filename=package:///meshes/ank_act_rod_3_collision.stl; visual mesh filename=package:///meshes/ank_act_rod_3_visual.stl
- added link ank_act_rod_4, mass 0.0026945559868381376359; collision mesh filename=package:///meshes/ank_act_rod_4_collision.stl; visual mesh filename=package:///meshes/ank_act_rod_4_visual.stl
- added link ank_act_rod_head_3, mass 0.00066080012085386230676; collision mesh filename=package:///meshes/ank_act_rod_head_3_collision.stl; visual mesh filename=package:///meshes/ank_act_rod_head_3_visual.stl
- added link ank_act_rod_head_4, mass 0.00066080012085386230676; collision mesh filename=package:///meshes/ank_act_rod_head_4_collision.stl; visual mesh filename=package:///meshes/ank_act_rod_head_4_visual.stl
- added link ank_b_link_3, mass 0.00089583742203429468642; collision mesh filename=package:///meshes/ank_b_link_3_collision.stl; visual mesh filename=package:///meshes/ank_b_link_3_visual.stl
- added link ank_b_link_4, mass 0.00089583742203429468642; collision mesh filename=package:///meshes/ank_b_link_4_collision.stl; visual mesh filename=package:///meshes/ank_b_link_4_visual.stl
- added link ank_pitch_link_2, mass 0.0041366725921694342399; collision mesh filename=package:///meshes/ank_pitch_link_2_collision.stl; visual mesh filename=package:///meshes/ank_pitch_link_2_visual.stl
- added link ank_rigid_foot_link_2, mass 0.0082157357687249205763; collision mesh filename=package:///meshes/ank_rigid_foot_link_2_collision.stl; visual mesh filename=package:///meshes/ank_rigid_foot_link_2_visual.stl
- added link ank_roll_link_2, mass 0.0054237955467263104098; collision mesh filename=package:///meshes/ank_roll_link_2_collision.stl; visual mesh filename=package:///meshes/ank_roll_link_2_visual.stl
- added link ank_rr_link_3, mass 0.00047585137324286056349; collision mesh filename=package:///meshes/ank_rr_link_3_collision.stl; visual mesh filename=package:///meshes/ank_rr_link_3_visual.stl
- added link ank_rr_link_4, mass 0.00047585137324286056349; collision mesh filename=package:///meshes/ank_rr_link_4_collision.stl; visual mesh filename=package:///meshes/ank_rr_link_4_visual.stl
- added link base_link
- added link body_link, mass 0.47165072969679472381; collision mesh filename=package:///meshes/body_link_collision.stl; visual mesh filename=package:///meshes/body_link_visual.stl
- added link elb_link, mass 0.011587175244532090662; collision mesh filename=package:///meshes/elb_link_collision.stl; visual mesh filename=package:///meshes/elb_link_visual.stl
- added link elb_link_2, mass 0.011587175244532090662; collision mesh filename=package:///meshes/elb_link_2_collision.stl; visual mesh filename=package:///meshes/elb_link_2_visual.stl
- added link head_link, mass 0.33570139948734667446; collision mesh filename=package:///meshes/head_link_collision.stl; visual mesh filename=package:///meshes/head_link_visual.stl
- added link hip_pitch_link_2, mass 0.075144662701080264244; collision mesh filename=package:///meshes/hip_pitch_link_2_collision.stl; visual mesh filename=package:///meshes/hip_pitch_link_2_visual.stl
- added link hip_roll_link, mass 0.09801239148352869357; collision mesh filename=package:///meshes/hip_roll_link_collision.stl; visual mesh filename=package:///meshes/hip_roll_link_visual.stl
- added link hip_roll_link_2, mass 0.09801239148352869357; collision mesh filename=package:///meshes/hip_roll_link_2_collision.stl; visual mesh filename=package:///meshes/hip_roll_link_2_visual.stl
- added link hip_yaw_link, mass 0.0052740645607467504311; collision mesh filename=package:///meshes/hip_yaw_link_collision.stl; visual mesh filename=package:///meshes/hip_yaw_link_visual.stl
- added link hip_yaw_link_2, mass 0.0052740645607467504311; collision mesh filename=package:///meshes/hip_yaw_link_2_collision.stl; visual mesh filename=package:///meshes/hip_yaw_link_2_visual.stl
- added link knee_link_2, mass 0.0043868974356887713642; collision mesh filename=package:///meshes/knee_link_2_collision.stl; visual mesh filename=package:///meshes/knee_link_2_visual.stl
- added link left_ank_base_link, mass 0.014262086197619733285; collision mesh filename=package:///meshes/left_ank_base_link_collision.stl; visual mesh filename=package:///meshes/left_ank_base_link_visual.stl
- added link neck_link, mass 0.038955748904513441688; collision mesh filename=package:///meshes/neck_link_collision.stl; visual mesh filename=package:///meshes/neck_link_visual.stl
- added link right_ank_base_link, mass 0.014262085602793538042; collision mesh filename=package:///meshes/right_ank_base_link_collision.stl; visual mesh filename=package:///meshes/right_ank_base_link_visual.stl
- added link sho_pitch_link, mass 0.0050714799847967799787; collision mesh filename=package:///meshes/sho_pitch_link_collision.stl; visual mesh filename=package:///meshes/sho_pitch_link_visual.stl
- added link sho_pitch_link_2, mass 0.0050714799847967799787; collision mesh filename=package:///meshes/sho_pitch_link_2_collision.stl; visual mesh filename=package:///meshes/sho_pitch_link_2_visual.stl
- added link sho_roll_link, mass 0.14053933881247798743; collision mesh filename=package:///meshes/sho_roll_link_collision.stl; visual mesh filename=package:///meshes/sho_roll_link_visual.stl
- added link sho_roll_link_2, mass 0.14053933881247798743; collision mesh filename=package:///meshes/sho_roll_link_2_collision.stl; visual mesh filename=package:///meshes/sho_roll_link_2_visual.stl
- link ank_act_link: mass 0.044782197696050358993 -> 0.044782197696050345115
- link ank_pitch_link: mass 0.0041366725921694342399 -> 0.0041366725921694333726
- link ank_roll_link: mass 0.0054237955467263095424 -> 0.0054237955467263104098
- link ank_rr_link: mass 0.00047585137324286067191 -> 0.00047585137324286056349
- link ank_rr_link_2: mass 0.00047585137324286067191 -> 0.00047585137324286056349
- link hip_pitch_link: mass 0.016043083203926743197 -> 0.075144662701080264244
- link knee_link: mass 0.0043868974356887704968 -> 0.0043868974356887713642
Joints:
- removed joint ank_B11
- removed joint ank_B12
- removed joint ank_B21
- removed joint ank_B22
- removed joint ank_B31
- removed joint ank_B32
- removed joint ank_R11
- removed joint ank_R12
- removed joint ank_R21
- removed joint ank_R22
- removed joint ank_act1
- removed joint ank_act2
- removed joint ank_base
- removed joint ank_foot
- removed joint ank_pitch
- removed joint ank_roll
- removed joint knee
- added joint base_link_to_base: type fixed, parent base_link, child body_link, origin xyz=0 0 0 rpy=0.0 0 0
- added joint head: type fixed, parent neck_link, child head_link, origin xyz=-8.1185058675714572018e-16 0.025000000000000202616 -0.049999999999999877875 rpy=1.1627977162610714148e-16 3.9441543390747586137e-31 -3.4420113463443417279e-33, axis 0 0 1, limit effort=1 velocity=20
- added joint left_ank_B11: type revolute, parent left_ank_base_link, child ank_b_link, origin xyz=0.018680019623525515038 0.010000000000000258682 0.023399999999999653716 rpy=-1.570796326794896558 -1.5053435939902863883 1.5707963267948972241, axis 0 0 1, limit lower=-1.570796326794896558 upper=1.570796326794896558 effort=1 velocity=20
- added joint left_ank_B12: type revolute, parent left_ank_base_link, child ank_b_link_2, origin xyz=0.020000000000000000416 0.010000000000000008882 -0.011499999999999996336 rpy=1.570796326794896558 1.4952155260088482169 1.5707963267948961139, axis 0 0 1, limit lower=-1.570796326794896558 upper=1.570796326794896558 effort=1 velocity=20
- added joint left_ank_B21: type revolute, parent ank_b_link, child ank_act_link_head, origin xyz=-0.0044999999999999970579 0 -0.016999999999999997752 rpy=1.5707963267948970021 1.553434520486443482 -1.5707963267948976682, axis 0 0 1, limit lower=-1.570796326794896558 upper=1.570796326794896558 effort=1 velocity=20
- added joint left_ank_B22: type revolute, parent ank_b_link_2, child ank_act_link_head_2, origin xyz=-0.0045000000000000039968 2.7755575615628913511e-17 0.016999999999999997752 rpy=1.5707963267948976682 -1.5676670403455870151 -1.5707963267941265073, axis 0 0 1, limit lower=-1.570796326794896558 upper=1.570796326794896558 effort=1 velocity=20
- added joint left_ank_B31: type revolute, parent ank_act_link_head, child ank_act_link, origin xyz=-4.336808689942017736e-19 -0.0060499999999999720668 -0.0043000000000000017375 rpy=1.570796326794896558 5.4574690063457464206e-06 3.1415926535897917837, axis 0 0 1, limit lower=-1.570796326794896558 upper=1.570796326794896558 effort=1 velocity=20
- added joint left_ank_B32: type revolute, parent ank_act_link_head_2, child ank_act_link_2, origin xyz=-1.7347234759768070944e-18 0.0060499999999999998224 -0.0043000000000000190847 rpy=-1.5707963267948970021 -5.4574692695236841152e-06 3.1415926535897900074, axis 0 0 1, limit lower=-1.570796326794896558 upper=1.570796326794896558 effort=1 velocity=20
- added joint left_ank_R11: type revolute, parent ank_roll_link, child ank_rr_link, origin xyz=0.010000000000000001943 -0.012500000000000004163 0.040599999999999997202 rpy=-1.2787963292933377177e-17 -1.8228899889648075415e-17 3.0761399207850530502, axis 0 0 1, limit lower=-1.570796326794896558 upper=1.570796326794896558 effort=1 velocity=20
- added joint left_ank_R12: type revolute, parent ank_roll_link, child ank_rr_link_2, origin xyz=-0.0099999999999999741873 -0.012499999999999997224 0.040599999999999997202 rpy=-7.7301105620767295759e-15 2.7427633691344020646e-15 0.075580800785947366283, axis 0 0 1, limit lower=-1.570796326794896558 upper=1.570796326794896558 effort=1 velocity=20
- added joint left_ank_R21: type revolute, parent ank_rr_link, child ank_act_rod_head, origin xyz=0.0020000000000000087153 -0.010000000000000008882 -0.0018999999999999995625 rpy=-1.57079632679489678 -1.5534345204865469547 -1.5707963267964526466, axis 0 0 1, limit lower=-1.570796326794896558 upper=1.570796326794896558 effort=1 velocity=20
- added joint left_ank_R22: type revolute, parent ank_rr_link_2, child ank_act_rod_head_2, origin xyz=0.0019999999999999948375 0.010000000000000015821 -0.0018999999999999999962 rpy=-1.5707963267948945596 1.5676670403457815262 -1.5707963267949440755, axis 0 0 1, limit lower=-1.570796326794896558 upper=1.570796326794896558 effort=1 velocity=20
- added joint left_ank_act1: type prismatic, parent ank_act_link, child ank_act_rod, origin xyz=2.2722093439889699817e-06 -2.3175905639050142781e-15 -0.059207313423199875446 rpy=3.141592653589793116 6.878790537704591275e-16 -0.63671356442007176479, axis 0 0 1, limit lower=-0.017000000000000001221 upper=0.017000000000000001221 effort=1 velocity=20
- added joint left_ank_act2: type prismatic, parent ank_act_link_2, child ank_act_rod_2, origin xyz=2.2722093437109805447e-06 2.2204460492503130808e-16 -0.059246516530140014289 rpy=-3.141592653589793116 -3.3046120317952816603e-15 -0.6367135644200548894, axis 0 0 1, limit lower=-0.017000000000000001221 upper=0.017000000000000001221 effort=1 velocity=20
- added joint left_ank_base: type fixed, parent knee_link, child left_ank_base_link, origin xyz=-2.7755575615628913511e-17 -2.7755575615628913511e-17 -0.0065000000000000404676 rpy=-2.5778424446483550449e-15 -5.8771504303585622093e-17 -2.0891591146372152643, axis 0 0 1, limit effort=1 velocity=20
- added joint left_ank_foot: type fixed, parent ank_roll_link, child ank_rigid_foot_link, origin xyz=0 -0.022499999999999999167 0.025599999999999994288 rpy=-1.570796326794896558 -1.570796326794896558 0, axis 0 0 1, limit effort=1 velocity=20
- added joint left_ank_pitch: type revolute, parent left_ank_base_link, child ank_pitch_link, origin xyz=2.2898349882893853646e-16 0.099999999999999186762 0.020899999999999321898 rpy=-3.9765493497921600178e-15 1.6032661971899303447e-14 1.5707963267949018871, axis 0 0 1, limit lower=-1.570796326794896558 upper=1.570796326794896558 effort=1 velocity=20
- added joint left_ank_roll: type revolute, parent ank_pitch_link, child ank_roll_link, origin xyz=1.3877787807814456755e-17 0.0014999999999999805156 -0.014600000000000008804 rpy=1.5707963267948836794 -1.5707963267948876762 0, axis 0 0 1, limit lower=-1.570796326794896558 upper=1.570796326794896558 effort=1 velocity=20
- added joint left_elb: type revolute, parent sho_roll_link, child elb_link, origin xyz=-0.089500000000000148881 0 5.5511151231257827021e-17 rpy=-3.141592653589793116 -8.8760630082751599313e-15 -1.570796326794896558, axis 0 0 1, limit lower=-1.570796326794896558 upper=1.570796326794896558 effort=1 velocity=20
- added joint left_hip_pitch: type revolute, parent hip_roll_link, child hip_pitch_link, origin xyz=-0.024000000716140057477 -0.019000000152448709434 -0.019000000152448379837 rpy=-1.5707963267948990005 1.5707963267948346076 0, axis 0 0 1, limit lower=-1.570796326794896558 upper=1.570796326794896558 effort=1 velocity=20
- added joint left_hip_roll: type revolute, parent hip_yaw_link, child hip_roll_link, origin xyz=0.01899999999999998912 -6.9388939039072283776e-18 -0.027499999999999968914 rpy=3.1415926535897926719 -1.5707963267948950037 0, axis 0 0 1, limit lower=-1.570796326794896558 upper=1.570796326794896558 effort=1 velocity=20
- added joint left_hip_yaw: type revolute, parent body_link, child hip_yaw_link, origin xyz=0.034999999999999989453 -0.039999999999999993894 0.32359999999999999876 rpy=8.2736565350258079362e-17 -1.1884745520697063838e-16 1.570796326794742015, axis 0 0 1, limit lower=-1.570796326794896558 upper=1.570796326794896558 effort=1 velocity=20
- added joint left_knee: type revolute, parent hip_pitch_link, child knee_link, origin xyz=-7.6327832942979512154e-17 0.10750000000000065059 0.021499999999999946237 rpy=-3.141592653589793116 1.6520983539851397786e-15 1.0471975511966311601, axis 0 0 1, limit lower=-1.0471975511965976313 upper=2.0943951023931952626 effort=1 velocity=20
- added joint left_sho_pitch: type revolute, parent body_link, child sho_pitch_link, origin xyz=0.060499999999999609646 -0.044999999999999804046 0.45499999999999990452 rpy=-1.5707963267948705788 3.7242253603279489435e-14 1.5707963267949578423, axis 0 0 1, limit lower=-1.570796326794896558 upper=1.570796326794896558 effort=1 velocity=20
- added joint left_sho_roll: type revolute, parent sho_pitch_link, child sho_roll_link, origin xyz=-0.019000000000000009936 0.0090000000000000079936 -0.027499999999999982792 rpy=-0 -1.5707963267948894526 0, axis 0 0 1, limit lower=-1.570796326794896558 upper=1.570796326794896558 effort=1 velocity=20
- added joint neck: type fixed, parent body_link, child neck_link, origin xyz=-2.8389897409080418735e-95 -0.040000000000000007772 0.47500000000000003331 rpy=-3.141592653589793116 1.4194948704540149157e-93 -2.3182110490017671006e-77, axis 0 0 1, limit effort=1 velocity=20
- added joint right_ank_B11: type revolute, parent right_ank_base_link, child ank_b_link_3, origin xyz=0.020000000000000010825 -0.010000000000000008882 -0.011499999999999996336 rpy=-1.570796326794896558 -1.4985484105593720461 1.5707963267948759079, axis 0 0 1, limit lower=-1.570796326794896558 upper=1.570796326794896558 effort=1 velocity=20
- added joint right_ank_B12: type revolute, parent right_ank_base_link, child ank_b_link_4, origin xyz=0.018680019623525549732 -0.0099999999999999811262 0.023400000000000007599 rpy=1.5707963267949001107 1.502009063389788901 1.5707963267948978903, axis 0 0 1, limit lower=-1.570796326794896558 upper=1.570796326794896558 effort=1 velocity=20
- added joint right_ank_B21: type revolute, parent ank_b_link_3, child ank_act_link_head_3, origin xyz=0.0045000000000000039968 0 -0.016999999999999994282 rpy=-1.57079632679489678 -1.5353521467806920953 -1.5707963267954754283, axis 0 0 1, limit lower=-1.570796326794896558 upper=1.570796326794896558 effort=1 velocity=20
- added joint right_ank_B22: type revolute, parent ank_b_link_4, child ank_act_link_head_4, origin xyz=0.004499999999999990119 2.7755575615628913511e-17 0.016999999999999997752 rpy=-1.57079632679489678 1.5211261901953414544 -1.5707963267943136909, axis 0 0 1, limit lower=-1.570796326794896558 upper=1.570796326794896558 effort=1 velocity=20
- added joint right_ank_B31: type revolute, parent ank_act_link_head_3, child ank_act_link_3, origin xyz=8.6736173798840354721e-19 0.0060500000000000275779 -0.0042999999999999982681 rpy=1.57079632679489678 5.4574690011256526203e-06 5.2875499908971443947e-15, axis 0 0 1, limit lower=-1.570796326794896558 upper=1.570796326794896558 effort=1 velocity=20
- added joint right_ank_B32: type revolute, parent ank_act_link_head_4, child ank_act_link_4, origin xyz=-8.6736173798840354721e-19 -0.0060499999999999720668 -0.0042999999999999982681 rpy=-1.570796326794896558 -5.4574693955425126324e-06 3.8245928442555554852e-15, axis 0 0 1, limit lower=-1.570796326794896558 upper=1.570796326794896558 effort=1 velocity=20
- added joint right_ank_R11: type revolute, parent ank_roll_link_2, child ank_rr_link_3, origin xyz=0.010000000000000008882 -0.012500000000000018041 0.040600000000000004141 rpy=2.5313865286216826369e-15 1.7810538515162586169e-15 3.0693447373541720147, axis 0 0 1, limit lower=-1.570796326794896558 upper=1.570796326794896558 effort=1 velocity=20
- added joint right_ank_R12: type revolute, parent ank_roll_link_2, child ank_rr_link_4, origin xyz=-0.010000000000000005412 -0.012500000000000018041 0.04060000000000001108 rpy=-2.1857493624022859542e-15 -1.8666708694869886266e-15 0.068787263405216209078, axis 0 0 1, limit lower=-1.570796326794896558 upper=1.570796326794896558 effort=1 velocity=20
- added joint right_ank_R21: type revolute, parent ank_rr_link_3, child ank_act_rod_head_3, origin xyz=0.0019999999999999878986 -0.009999999999999995004 -0.0018999999999999991288 rpy=-1.5707963267948961139 -1.5353521467807458301 -1.5707963267947508967, axis 0 0 1, limit lower=-1.570796326794896558 upper=1.570796326794896558 effort=1 velocity=20
- added joint right_ank_R22: type revolute, parent ank_rr_link_4, child ank_act_rod_head_4, origin xyz=0.0020000000000000017764 0.009999999999999995004 -0.0018999999999999999962 rpy=-1.57079632679489678 1.5211261901953123665 -1.570796326794951181, axis 0 0 1, limit lower=-1.570796326794896558 upper=1.570796326794896558 effort=1 velocity=20
- added joint right_ank_act1: type prismatic, parent ank_act_link_3, child ank_act_rod_3, origin xyz=2.2722093423522583822e-06 -2.9004576518332214619e-15 -0.059300761807581189866 rpy=3.141592653589793116 4.3394957676616399489e-15 -0.63671356442003834708, axis 0 0 1, limit lower=-0.017000000000000001221 upper=0.017000000000000001221 effort=1 velocity=20
- added joint right_ank_act2: type prismatic, parent ank_act_link_4, child ank_act_rod_4, origin xyz=2.2722093449703897883e-06 1.8110513089197866066e-15 -0.059305633004860927593 rpy=-3.1415926535897846783 -1.11945757313106456e-14 -0.63671356441985949015, axis 0 0 1, limit lower=-0.017000000000000001221 upper=0.017000000000000001221 effort=1 velocity=20
- added joint right_ank_base: type fixed, parent knee_link_2, child right_ank_base_link, origin xyz=2.7755575615628913511e-17 0 -0.0065000000000000057732 rpy=5.6993076818632995017e-17 -9.6318510415490070481e-17 1.0524335389525802942, axis 0 0 1, limit effort=1 velocity=20
- added joint right_ank_foot: type fixed, parent ank_roll_link_2, child ank_rigid_foot_link_2, origin xyz=0 -0.022500000000000019984 0.025600000000000001227 rpy=-1.570796326794896558 -1.570796326794896336 0, axis 0 0 1, limit effort=1 velocity=20
- added joint right_ank_pitch: type revolute, parent right_ank_base_link, child ank_pitch_link_2, origin xyz=6.9388939039072283776e-18 -0.10000000000000000555 0.02089999999999999844 rpy=-1.2383945132469940545e-15 -9.5544025531341604884e-15 -1.5707963267949187625, axis 0 0 1, limit lower=-1.570796326794896558 upper=1.570796326794896558 effort=1 velocity=20
- added joint right_ank_roll: type revolute, parent ank_pitch_link_2, child ank_roll_link_2, origin xyz=-1.3877787807814456755e-17 0.0014999999999999805156 -0.01459999999999984574 rpy=-1.5707963267948943376 1.5707963267947937513 0, axis 0 0 1, limit lower=-1.570796326794896558 upper=1.570796326794896558 effort=1 velocity=20
- added joint right_elb: type revolute, parent sho_roll_link_2, child elb_link_2, origin xyz=-0.089500000000000051736 0 1.3877787807814456755e-17 rpy=-3.141592653589793116 -3.3306690738761288132e-16 1.5707963267948976682, axis 0 0 1, limit lower=-1.570796326794896558 upper=1.570796326794896558 effort=1 velocity=20
- added joint right_hip_pitch: type revolute, parent hip_roll_link_2, child hip_pitch_link_2, origin xyz=-0.02400000071614161179 -0.019000000152454406266 -0.019000000152450496199 rpy=-1.5707963267946469799 -1.5707963267948819031 0, axis 0 0 1, limit lower=-1.570796326794896558 upper=1.570796326794896558 effort=1 velocity=20
- added joint right_hip_roll: type revolute, parent hip_yaw_link_2, child hip_roll_link_2, origin xyz=0.018999999999999992589 -1.3877787807814456755e-17 -0.027500000000000024425 rpy=-3.141592653589793116 -1.5707963267946309927 0, axis 0 0 1, limit lower=-1.570796326794896558 upper=1.570796326794896558 effort=1 velocity=20
- added joint right_hip_yaw: type revolute, parent body_link, child hip_yaw_link_2, origin xyz=-0.035000000000000003331 -0.040000000000000007772 0.32359999999999999876 rpy=1.1485706107586878963e-15 -6.1238048206303817597e-17 1.5707963267948590325, axis 0 0 1, limit lower=-1.570796326794896558 upper=1.570796326794896558 effort=1 velocity=20
- added joint right_knee: type revolute, parent hip_pitch_link_2, child knee_link_2, origin xyz=-4.1633363423443370266e-17 -0.10749999999999990119 0.016499999999997842781 rpy=3.4590285370200512466e-17 -1.0374608420584268216e-16 -1.0471975511965516681, axis 0 0 1, limit lower=-1.0471975511965976313 upper=2.0943951023931952626 effort=1 velocity=20
- added joint right_sho_pitch: type revolute, parent body_link, child sho_pitch_link_2, origin xyz=-0.060500000000000005163 -0.044999999999999991396 0.45499999999999996003 rpy=-1.570796326794896558 7.2736973397141567712e-16 -1.570796326794896558, axis 0 0 1, limit lower=-1.570796326794896558 upper=1.570796326794896558 effort=1 velocity=20
- added joint right_sho_roll: type revolute, parent sho_pitch_link_2, child sho_roll_link_2, origin xyz=0.019000000000000009936 0.0090000000000000079936 -0.027500000000000003608 rpy=-3.141592653589793116 -1.570796326794896558 0, axis 0 0 1, limit lower=-1.570796326794896558 upper=1.570796326794896558 effort=1 velocity=20
