Commit message: Load base in mujoco

File: toddleroid/robot_descriptions/base/base.urdf (robot description, URDF)
Before this commit: robot base, 50 links, 49 joints
Links:
- link ank_act_link: mass 0.044782197696050345115 -> 0.044782197696050352054
- link ank_act_link_2: mass 0.044782197696050352054 -> 0.044782197696050358993
- link ank_act_link_3: mass 0.044782197696050352054 -> 0.044782197696050358993
- link ank_act_link_4: mass 0.044782197696050352054 -> 0.044782197696050358993
- link ank_rr_link: mass 0.00047585137324286056349 -> 0.0004758513732428606177
- link ank_rr_link_2: mass 0.00047585137324286056349 -> 0.0004758513732428606177
- link ank_rr_link_3: mass 0.00047585137324286056349 -> 0.0004758513732428606177
- link ank_rr_link_4: mass 0.00047585137324286056349 -> 0.0004758513732428606177
- link body_link: mass 0.47165072969679472381 -> 0.4716507296967951679
- link elb_link: mass 0.011587175244532090662 -> 0.011587175244532088927
- link elb_link_2: mass 0.011587175244532090662 -> 0.011587175244532088927
- link head_link: mass 0.33570139948734667446 -> 0.15100469056885920671
- link hip_pitch_link: mass 0.075144662701080264244 -> 0.075144662701080278122
- link hip_pitch_link_2: mass 0.075144662701080264244 -> 0.075144662701080278122
- link hip_roll_link: mass 0.09801239148352869357 -> 0.098012391483528735203
- link hip_roll_link_2: mass 0.09801239148352869357 -> 0.098012391483528735203
- link knee_link: mass 0.0043868974356887713642 -> 0.0043868974356887722316
- link knee_link_2: mass 0.0043868974356887713642 -> 0.0043868974356887722316
- link neck_link: mass 0.038955748904513441688 -> 0.017530087007031042168
- link right_ank_base_link: mass 0.014262085602793538042 -> 0.014262085602793541511
Joints:
- joint head: origin xyz=-8.1185058675714572018e-16 0.025000000000000202616 -0.049999999999999877875 rpy=1.1627977162610714148e-16 3.9441543390747586137e-31 -3.4420113463443417279e-33 -> xyz=4.6467068165737631661e-19 0 -0.040000000000000035527 rpy=-1.232595164407830946e-32 2.9519052500171698995e-47 3.141592653589793116
- joint left_ank_B11: origin xyz=0.018680019623525515038 0.010000000000000258682 0.023399999999999653716 rpy=-1.570796326794896558 -1.5053435939902863883 1.5707963267948972241 -> xyz=0.018680019623525546263 0.010000000000000064393 0.02340000000000000413 rpy=-1.570796326794896558 -1.5053435939903097029 1.5707963267948918951
- joint left_ank_B12: origin xyz=0.020000000000000000416 0.010000000000000008882 -0.011499999999999996336 rpy=1.570796326794896558 1.4952155260088482169 1.5707963267948961139 -> xyz=0.020000000000000007355 0.0099999999999999811262 -0.011500000000000003275 rpy=1.570796326794896558 1.4952155260088222377 1.5707963267949036634
- joint left_ank_B21: origin xyz=-0.0044999999999999970579 0 -0.016999999999999997752 rpy=1.5707963267948970021 1.553434520486443482 -1.5707963267948976682 -> xyz=-0.0045000000000000074662 0 -0.016999999999999997752 rpy=1.570796326794896336 1.5534345204864428158 -1.570796326794806852
- joint left_ank_B22: origin xyz=-0.0045000000000000039968 2.7755575615628913511e-17 0.016999999999999997752 rpy=1.5707963267948976682 -1.5676670403455870151 -1.5707963267941265073 -> xyz=-0.0044999999999999970579 -2.7755575615628913511e-17 0.016999999999999997752 rpy=1.570796326794896558 -1.5676670403455679192 -1.5707963267926954298
- joint left_ank_B31: origin xyz=-4.336808689942017736e-19 -0.0060499999999999720668 -0.0043000000000000017375 rpy=1.570796326794896558 5.4574690063457464206e-06 3.1415926535897917837 -> xyz=-8.6736173798840354721e-19 -0.0060500000000000275779 -0.0043000000000000121458 rpy=1.570796326794896558 5.4574690878165813072e-06 3.1415926535897908956
- joint left_ank_B32: origin xyz=-1.7347234759768070944e-18 0.0060499999999999998224 -0.0043000000000000190847 rpy=-1.5707963267948970021 -5.4574692695236841152e-06 3.1415926535897900074 -> xyz=-8.6736173798840354721e-19 0.0060500000000000553335 -0.0042999999999999913292 rpy=-1.570796326794896558 -5.4574693029296022226e-06 -3.141592653589793116
- joint left_ank_R11: origin xyz=0.010000000000000001943 -0.012500000000000004163 0.040599999999999997202 rpy=-1.2787963292933377177e-17 -1.8228899889648075415e-17 3.0761399207850530502 -> xyz=0.010000000000000001943 -0.012500000000000007633 0.040599999999999990263 rpy=5.5133286511563240655e-17 -1.424248725567722883e-16 3.0761399207850415038
- joint left_ank_R12: origin xyz=-0.0099999999999999741873 -0.012499999999999997224 0.040599999999999997202 rpy=-7.7301105620767295759e-15 2.7427633691344020646e-15 0.075580800785947366283 -> xyz=-0.010000000000000008882 -0.012500000000000000694 0.040599999999999997202 rpy=-1.0021582319192169566e-15 1.9109166915830268034e-16 0.075580800785917862106
- joint left_ank_R21: origin xyz=0.0020000000000000087153 -0.010000000000000008882 -0.0018999999999999995625 rpy=-1.57079632679489678 -1.5534345204865469547 -1.5707963267964526466 -> xyz=0.0020000000000000087153 -0.010000000000000001943 -0.0019000000000000004299 rpy=-1.5707963267948961139 -1.553434520486503656 -1.5707963267948825692
- joint left_ank_R22: origin xyz=0.0019999999999999948375 0.010000000000000015821 -0.0018999999999999999962 rpy=-1.5707963267948945596 1.5676670403457815262 -1.5707963267949440755 -> xyz=0.0020000000000000017764 0.010000000000000001943 -0.0018999999999999995625 rpy=-1.5707963267949007768 1.5676670403457919623 -1.5707963267947144814
- joint left_ank_act1: origin xyz=2.2722093439889699817e-06 -2.3175905639050142781e-15 -0.059207313423199875446 rpy=3.141592653589793116 6.878790537704591275e-16 -0.63671356442007176479 -> xyz=2.2722093435375081971e-06 -2.3071822230491534356e-15 -0.059207313423202775904 rpy=3.141592653589793116 4.2775187765792706995e-15 -0.63671356442004245491
- joint left_ank_act2: origin xyz=2.2722093437109805447e-06 2.2204460492503130808e-16 -0.059246516530140014289 rpy=-3.141592653589793116 -3.3046120317952816603e-15 -0.6367135644200548894 -> xyz=2.2722093432694934201e-06 -4.024558464266192459e-16 -0.059246516530146259294 rpy=-3.141592653589793116 -1.9929871652631197461e-17 -0.63671356442003623766
- joint left_ank_base: origin xyz=-2.7755575615628913511e-17 -2.7755575615628913511e-17 -0.0065000000000000404676 rpy=-2.5778424446483550449e-15 -5.8771504303585622093e-17 -2.0891591146372152643 -> xyz=-2.6367796834847467835e-16 -9.7144514654701197287e-17 -0.0065000000000002416956 rpy=-3.3438186186406859098e-14 -6.9220172543623322901e-15 -2.0891591146372241461
- joint left_ank_foot: origin xyz=0 -0.022499999999999999167 0.025599999999999994288 rpy=-1.570796326794896558 -1.570796326794896558 0 -> xyz=0 -0.022500000000000006106 0.025599999999999990818 rpy=-1.570796326794896558 -1.570796326794896558 0
- joint left_ank_pitch: origin xyz=2.2898349882893853646e-16 0.099999999999999186762 0.020899999999999321898 rpy=-3.9765493497921600178e-15 1.6032661971899303447e-14 1.5707963267949018871 -> xyz=0 0.10000000000000003331 0.020899999999999988032 rpy=7.807247938257453967e-15 5.4959122264044313487e-15 1.5707963267949247577
- joint left_ank_roll: origin xyz=1.3877787807814456755e-17 0.0014999999999999805156 -0.014600000000000008804 rpy=1.5707963267948836794 -1.5707963267948876762 0 -> xyz=0 0.0014999999999999943934 -0.014599999999999994926 rpy=1.5707963267948952257 -1.5707963267948858999 0
- joint left_elb: origin xyz=-0.089500000000000148881 0 5.5511151231257827021e-17 rpy=-3.141592653589793116 -8.8760630082751599313e-15 -1.570796326794896558 -> xyz=-0.089500000000000121125 0 5.5511151231257827021e-17 rpy=-3.141592653589793116 -8.8760630082751599313e-15 -1.570796326794896558
- joint left_hip_pitch: origin xyz=-0.024000000716140057477 -0.019000000152448709434 -0.019000000152448379837 rpy=-1.5707963267948990005 1.5707963267948346076 0 -> xyz=-0.024000000716140224011 -0.019000000152450662733 -0.019000000152448726781 rpy=-1.5707963267948796826 1.5707963267948239494 0
- joint left_hip_roll: origin xyz=0.01899999999999998912 -6.9388939039072283776e-18 -0.027499999999999968914 rpy=3.1415926535897926719 -1.5707963267948950037 0 -> xyz=0.018999999999999992589 -6.9388939039072283776e-18 -0.027499999999999968914 rpy=3.141592653589793116 -1.5707963267948794606 0
- joint left_hip_yaw: origin xyz=0.034999999999999989453 -0.039999999999999993894 0.32359999999999999876 rpy=8.2736565350258079362e-17 -1.1884745520697063838e-16 1.570796326794742015 -> xyz=0.034999999999999989453 -0.039999999999999993894 0.29868541999999997927 rpy=4.1258627841574100087e-29 -6.1232339957431151336e-17 1.5707963267949682784
- joint left_knee: origin xyz=-7.6327832942979512154e-17 0.10750000000000065059 0.021499999999999946237 rpy=-3.141592653589793116 1.6520983539851397786e-15 1.0471975511966311601 -> xyz=-4.1633363423443370266e-17 0.10750000000000001221 0.02149999999999999481 rpy=3.1415926535897895633 2.6314965551403718944e-14 1.047197551196626053
- joint left_sho_pitch: origin xyz=0.060499999999999609646 -0.044999999999999804046 0.45499999999999990452 rpy=-1.5707963267948705788 3.7242253603279489435e-14 1.5707963267949578423 -> xyz=0.06049999999999895739 -0.044999999999999804046 0.43008541999999988503 rpy=-1.5707963267948705788 3.7242253603279489435e-14 1.5707963267949578423
- joint left_sho_roll: origin xyz=-0.019000000000000009936 0.0090000000000000079936 -0.027499999999999982792 rpy=-0 -1.5707963267948894526 0 -> xyz=-0.018999999999999996059 0.0090000000000000079936 -0.02749999999999998973 rpy=-0 -1.5707963267948894526 0
- joint neck: origin xyz=-2.8389897409080418735e-95 -0.040000000000000007772 0.47500000000000003331 rpy=-3.141592653589793116 1.4194948704540149157e-93 -2.3182110490017671006e-77 -> xyz=-1.0873011537518218883e-17 -0.040000000000000007772 0.45008542000000001382 rpy=-3.141592653589793116 7.7518614875493756421e-90 -1.2659750538598650252e-73
- joint right_ank_B11: origin xyz=0.020000000000000010825 -0.010000000000000008882 -0.011499999999999996336 rpy=-1.570796326794896558 -1.4985484105593720461 1.5707963267948759079 -> xyz=0.019999999999999996947 -0.0099999999999999811262 -0.011499999999999982458 rpy=-1.570796326794896558 -1.4985484105593833704 1.5707963267948970021
- joint right_ank_B12: origin xyz=0.018680019623525549732 -0.0099999999999999811262 0.023400000000000007599 rpy=1.5707963267949001107 1.502009063389788901 1.5707963267948978903 -> xyz=0.01868001962352556708 -0.0099999999999999811262 0.023399999999999976374 rpy=1.57079632679490655 1.5020090633897773547 1.5707963267949058839
- joint right_ank_B21: origin xyz=0.0045000000000000039968 0 -0.016999999999999994282 rpy=-1.57079632679489678 -1.5353521467806920953 -1.5707963267954754283 -> xyz=0.0044999999999999762412 2.7755575615628913511e-17 -0.017000000000000004691 rpy=-1.5707963267948961139 -1.5676670168131927596 -1.5707963267948830133
- joint right_ank_B22: origin xyz=0.004499999999999990119 2.7755575615628913511e-17 0.016999999999999997752 rpy=-1.57079632679489678 1.5211261901953414544 -1.5707963267943136909 -> xyz=0.0044999999999999970579 0 0.017000000000000001221 rpy=-1.57079632679489678 1.55343465115961199 -1.5707963267948699126
- joint right_ank_B31: origin xyz=8.6736173798840354721e-19 0.0060500000000000275779 -0.0042999999999999982681 rpy=1.57079632679489678 5.4574690011256526203e-06 5.2875499908971443947e-15 -> xyz=2.168404344971008868e-19 0.0060500000000000553335 -0.0043000000000000052069 rpy=1.570796326794896558 5.4574690704063518601e-06 1.7018354478117103418e-17
- joint right_ank_B32: origin xyz=-8.6736173798840354721e-19 -0.0060499999999999720668 -0.0042999999999999982681 rpy=-1.570796326794896558 -5.4574693955425126324e-06 3.8245928442555554852e-15 -> xyz=2.8189256484623115284e-18 -0.0060500000000000275779 -0.0042999999999999947986 rpy=-1.570796326794896558 -5.4574694521280218192e-06 -1.2970245616443644851e-17
- joint right_ank_R11: origin xyz=0.010000000000000008882 -0.012500000000000018041 0.040600000000000004141 rpy=2.5313865286216826369e-15 1.7810538515162586169e-15 3.0693447373541720147 -> xyz=0.0099999999999999880651 -0.012499999999999993755 0.040600000000000004141 rpy=1.838132558719167337e-14 -1.968550043761323508e-15 3.0693447373542399603
- joint right_ank_R12: origin xyz=-0.010000000000000005412 -0.012500000000000018041 0.04060000000000001108 rpy=-2.1857493624022859542e-15 -1.8666708694869886266e-15 0.068787263405216209078 -> xyz=-0.010000000000000005412 -0.012499999999999993755 0.040600000000000004141 rpy=-5.4208100503948111158e-17 1.2515168021403654183e-16 0.068787263405284487794
- joint right_ank_R21: origin xyz=0.0019999999999999878986 -0.009999999999999995004 -0.0018999999999999991288 rpy=-1.5707963267948961139 -1.5353521467807458301 -1.5707963267947508967 -> xyz=0.0019999999999999948375 -0.009999999999999995004 -0.001900000000000000213 rpy=-1.5707963267948972241 -1.5676670168132933458 -1.570796326795488973
- joint right_ank_R22: origin xyz=0.0020000000000000017764 0.009999999999999995004 -0.0018999999999999999962 rpy=-1.57079632679489678 1.5211261901953123665 -1.570796326794951181 -> xyz=0.0020000000000000052458 0.0099999999999999984734 -0.0019000000000000006467 rpy=-1.57079632679489678 1.5534346511596015539 -1.5707963267942353092
- joint right_ank_act1: origin xyz=2.2722093423522583822e-06 -2.9004576518332214619e-15 -0.059300761807581189866 rpy=3.141592653589793116 4.3394957676616399489e-15 -0.63671356442003834708 -> xyz=2.2722093422193351958e-06 -3.0045410603918298875e-15 -0.059245818700239413768 rpy=3.141592653589793116 2.3300461121301510461e-18 -0.63671356442004811704
- joint right_ank_act2: origin xyz=2.2722093449703897883e-06 1.8110513089197866066e-15 -0.059305633004860927593 rpy=-3.1415926535897846783 -1.11945757313106456e-14 -0.63671356441985949015 -> xyz=2.2722093449636677348e-06 1.7694179454963432363e-15 -0.059208011505606339409 rpy=-3.1415926535897860106 -1.9568267140524259683e-14 -0.636713564419863709
- joint right_ank_base: origin xyz=2.7755575615628913511e-17 0 -0.0065000000000000057732 rpy=5.6993076818632995017e-17 -9.6318510415490070481e-17 1.0524335389525802942 -> xyz=0 2.0816681711721685133e-17 -0.0064999999999999918954 rpy=-2.3897681857549792405e-16 -1.6802318149906911049e-16 1.0524335389525802942
- joint right_ank_foot: origin xyz=0 -0.022500000000000019984 0.025600000000000001227 rpy=-1.570796326794896558 -1.570796326794896336 0 -> xyz=6.9388939039072283776e-18 -0.022499999999999999167 0.025600000000000018574 rpy=-1.5707963267949041075 -1.570796326794896558 0
- joint right_ank_pitch: origin xyz=6.9388939039072283776e-18 -0.10000000000000000555 0.02089999999999999844 rpy=-1.2383945132469940545e-15 -9.5544025531341604884e-15 -1.5707963267949187625 -> xyz=1.0408340855860842566e-16 -0.10000000000000013045 0.020900000000000147626 rpy=-7.5018482240547858138e-15 2.5176249968740924777e-16 1.5707963267948918951
- joint right_ank_roll: origin xyz=-1.3877787807814456755e-17 0.0014999999999999805156 -0.01459999999999984574 rpy=-1.5707963267948943376 1.5707963267947937513 0 -> xyz=-1.3877787807814456755e-17 0.0015000000000000013323 -0.014600000000000012274 rpy=1.570796326794896558 1.570796326794707154 0
- joint right_elb: origin xyz=-0.089500000000000051736 0 1.3877787807814456755e-17 rpy=-3.141592653589793116 -3.3306690738761288132e-16 1.5707963267948976682 -> xyz=-0.089500000000000065614 0 1.3877787807814456755e-17 rpy=-3.141592653589793116 -3.3306690738761288132e-16 1.5707963267948976682
- joint right_hip_pitch: origin xyz=-0.02400000071614161179 -0.019000000152454406266 -0.019000000152450496199 rpy=-1.5707963267946469799 -1.5707963267948819031 0 -> xyz=-0.02400000071614186159 -0.019000000152455120972 -0.019000000152451717444 rpy=-1.5707963267946463137 -1.5707963267948112929 0
- joint right_hip_roll: origin xyz=0.018999999999999992589 -1.3877787807814456755e-17 -0.027500000000000024425 rpy=-3.141592653589793116 -1.5707963267946309927 0 -> xyz=0.018999999999999999528 -6.9388939039072283776e-18 -0.027499999999999913403 rpy=3.141592653589793116 -1.5707963267948641395 0
- joint right_hip_yaw: origin xyz=-0.035000000000000003331 -0.040000000000000007772 0.32359999999999999876 rpy=1.1485706107586878963e-15 -6.1238048206303817597e-17 1.5707963267948590325 -> xyz=-0.035000000000000003331 -0.039999999999999993894 0.29868541999999997927 rpy=-6.3173742254660021089e-26 -6.1232339666714670147e-17 1.5707963267947904207
- joint right_knee: origin xyz=-4.1633363423443370266e-17 -0.10749999999999990119 0.016499999999997842781 rpy=3.4590285370200512466e-17 -1.0374608420584268216e-16 -1.0471975511965516681 -> xyz=-4.1633363423443370266e-17 -0.10749999999999998446 0.016499999999999986899 rpy=-7.9136240096094387749e-16 -6.4063376207831640667e-16 -1.0471975511964932704
- joint right_sho_pitch: origin xyz=-0.060500000000000005163 -0.044999999999999991396 0.45499999999999996003 rpy=-1.570796326794896558 7.2736973397141567712e-16 -1.570796326794896558 -> xyz=-0.060500000000000005163 -0.044999999999999977518 0.43008541999999994054 rpy=-1.570796326794896558 7.2736973397141567712e-16 -1.570796326794896558
- joint right_sho_roll: origin xyz=0.019000000000000009936 0.0090000000000000079936 -0.027500000000000003608 rpy=-3.141592653589793116 -1.570796326794896558 0 -> xyz=0.019000000000000002998 0.0090000000000000079936 -0.02749999999999998973 rpy=-3.141592653589793116 -1.570796326794896558 0
