Commit message: Enable base to walk one step

File: toddleroid/robot_descriptions/base/base.urdf (robot description, URDF)
Before this commit: robot base, 50 links, 49 joints
Links:
- link ank_act_link_2: mass 0.044782197696050358993 -> 0.044782197696050365932
- link ank_roll_link: mass 0.0054237955467263104098 -> 0.0054237955467263112772
- link ank_roll_link_2: mass 0.0054237955467263104098 -> 0.0054237955467263112772
- link body_link: mass 0.4716507296967951679 -> 0.67608257475273081383
- link elb_link: mass 0.011587175244532088927 -> 0.011587175244532094132
- link elb_link_2: mass 0.011587175244532088927 -> 0.011587175244532094132
- link head_link: mass 0.15100469056885920671 -> 0.075015538754886992856
- link hip_pitch_link: mass 0.075144662701080278122 -> 0.075144662701080264244
- link hip_pitch_link_2: mass 0.075144662701080278122 -> 0.075144662701080264244
- link hip_roll_link: mass 0.098012391483528735203 -> 0.098012391483528707448
- link hip_roll_link_2: mass 0.098012391483528735203 -> 0.098012391483528707448
- link knee_link: mass 0.0043868974356887722316 -> 0.0043868974356887730989
- link knee_link_2: mass 0.0043868974356887722316 -> 0.0043868974356887730989
- link sho_pitch_link: mass 0.0050714799847967799787 -> 0.005071479984796780846
- link sho_pitch_link_2: mass 0.0050714799847967799787 -> 0.005071479984796780846
- link sho_roll_link: mass 0.14053933881247798743 -> 0.14053933881247801518
Joints:
- joint head: origin xyz=4.6467068165737631661e-19 0 -0.040000000000000035527 rpy=-1.232595164407830946e-32 2.9519052500171698995e-47 3.141592653589793116 -> xyz=0 1.7347234759768070944e-18 -0.039999999999999980016 rpy=0 -1.0509729472670562853e-99 -4.1486002514987779604e-69
- joint left_ank_B11: origin xyz=0.018680019623525546263 0.010000000000000064393 0.02340000000000000413 rpy=-1.570796326794896558 -1.5053435939903097029 1.5707963267948918951 -> xyz=0.018680019623525362382 0.009999999999999731326 0.023399999999999900047 rpy=-1.5707963267948952257 -1.505343593990304818 1.5707963267948974462
- joint left_ank_B12: origin xyz=0.020000000000000007355 0.0099999999999999811262 -0.011500000000000003275 rpy=1.570796326794896558 1.4952155260088222377 1.5707963267949036634 -> xyz=0.019999999999999996947 0.010000000000000008882 -0.011499999999999996336 rpy=1.570796326794896558 1.4952155260088879629 1.57079632679525516
- joint left_ank_B21: origin xyz=-0.0045000000000000074662 0 -0.016999999999999997752 rpy=1.570796326794896336 1.5534345204864428158 -1.570796326794806852 -> xyz=-0.0044999999999999970579 2.7755575615628913511e-17 -0.016999999999999997752 rpy=1.57079632679489678 1.5534345204864243861 -1.5707963267948996666
- joint left_ank_B22: origin xyz=-0.0044999999999999970579 -2.7755575615628913511e-17 0.016999999999999997752 rpy=1.570796326794896558 -1.5676670403455679192 -1.5707963267926954298 -> xyz=-0.0044999999999999970579 0 0.016999999999999994282 rpy=1.5707963267990325829 -1.567667040345596563 -1.5707963267904616611
- joint left_ank_B31: origin xyz=-8.6736173798840354721e-19 -0.0060500000000000275779 -0.0043000000000000121458 rpy=1.570796326794896558 5.4574690878165813072e-06 3.1415926535897908956 -> xyz=-1.3877787807814456755e-17 -0.0060500000000000830891 -0.0043000000000000086764 rpy=1.570796326794896558 5.4574690367119021436e-06 -3.141592653589793116
- joint left_ank_B32: origin xyz=-8.6736173798840354721e-19 0.0060500000000000553335 -0.0042999999999999913292 rpy=-1.570796326794896558 -5.4574693029296022226e-06 -3.141592653589793116 -> xyz=0 0.0060499999999999998224 -0.0042999999999999913292 rpy=-1.570796326794896558 -5.4574692127553140676e-06 3.1415926535897922278
- joint left_ank_R11: origin xyz=0.010000000000000001943 -0.012500000000000007633 0.040599999999999990263 rpy=5.5133286511563240655e-17 -1.424248725567722883e-16 3.0761399207850415038 -> xyz=0.010000000000000001943 -0.012500000000000007633 0.040599999999999997202 rpy=-2.3809415734231673378e-15 -2.8771866469601532264e-15 3.0761399207850583792
- joint left_ank_R12: origin xyz=-0.010000000000000008882 -0.012500000000000000694 0.040599999999999997202 rpy=-1.0021582319192169566e-15 1.9109166915830268034e-16 0.075580800785917862106 -> xyz=-0.009999999999999995004 -0.012500000000000011102 0.040599999999999997202 rpy=-1.3103682910477166415e-14 1.457398994851742625e-15 0.075580800785893090254
- joint left_ank_R21: origin xyz=0.0020000000000000087153 -0.010000000000000001943 -0.0019000000000000004299 rpy=-1.5707963267948961139 -1.553434520486503656 -1.5707963267948825692 -> xyz=0.0020000000000000017764 -0.0099999999999999984734 -0.001899999999999998912 rpy=-1.570796326794896558 -1.5534345204864692391 -1.5707963267950264541
- joint left_ank_R22: origin xyz=0.0020000000000000017764 0.010000000000000001943 -0.0018999999999999995625 rpy=-1.5707963267949007768 1.5676670403457919623 -1.5707963267947144814 -> xyz=0.0020000000000000087153 0.0099999999999999984734 -0.0019000000000000058509 rpy=-1.57079632679489678 1.567667040345726015 -1.5707963267956523978
- joint left_ank_act1: origin xyz=2.2722093435375081971e-06 -2.3071822230491534356e-15 -0.059207313423202775904 rpy=3.141592653589793116 4.2775187765792706995e-15 -0.63671356442004245491 -> xyz=2.2722093436094992214e-06 -2.5604518505417672714e-15 -0.059207313423198439095 rpy=-3.141592653589793116 1.328302970873878818e-14 -0.6367135644199727329
- joint left_ank_act2: origin xyz=2.2722093432694934201e-06 -4.024558464266192459e-16 -0.059246516530146259294 rpy=-3.141592653589793116 -1.9929871652631197461e-17 -0.63671356442003623766 -> xyz=2.2722093434603130024e-06 -2.8449465006019636348e-16 -0.059246516530142220858 rpy=3.141592653589793116 1.5679305736050431748e-15 -0.63671356442004867215
- joint left_ank_base: origin xyz=-2.6367796834847467835e-16 -9.7144514654701197287e-17 -0.0065000000000002416956 rpy=-3.3438186186406859098e-14 -6.9220172543623322901e-15 -2.0891591146372241461 -> xyz=-3.0253577421035515727e-15 -3.2196467714129539672e-15 -0.0064999999999985694221 rpy=-9.7170810831163359999e-14 1.1559030630111302718e-13 -2.0943951023931739464
- joint left_ank_foot: origin xyz=0 -0.022500000000000006106 0.025599999999999990818 rpy=-1.570796326794896558 -1.570796326794896558 0 -> xyz=-6.9388939039072283776e-18 -0.022500000000000009576 0.025600000000000004696 rpy=-1.570796326794896558 -1.5707963267948956698 0
- joint left_ank_pitch: origin xyz=0 0.10000000000000003331 0.020899999999999988032 rpy=7.807247938257453967e-15 5.4959122264044313487e-15 1.5707963267949247577 -> xyz=-5.7245874707234634116e-17 0.10000000000000028311 0.020900000000000012318 rpy=-8.6690501906182033625e-15 2.4133613739470252907e-15 1.5707963267949272002
- joint left_ank_roll: origin xyz=0 0.0014999999999999943934 -0.014599999999999994926 rpy=1.5707963267948952257 -1.5707963267948858999 0 -> xyz=-6.9388939039072283776e-18 0.0014999999999998920447 -0.014600000000000140643 rpy=1.5707963267949041075 -1.570796326794886788 0
- joint left_elb: origin xyz=-0.089500000000000121125 0 5.5511151231257827021e-17 rpy=-3.141592653589793116 -8.8760630082751599313e-15 -1.570796326794896558 -> xyz=-0.089499999999999607647 -6.6613381477509392425e-16 6.1860239153332940987e-15 rpy=3.1415926535897122918 4.7267745273418620861e-14 -1.5707963267948943376
- joint left_hip_pitch: origin xyz=-0.024000000716140224011 -0.019000000152450662733 -0.019000000152448726781 rpy=-1.5707963267948796826 1.5707963267948239494 0 -> xyz=-0.02400000071614330488 -0.019000000152458163677 -0.019000000152447526353 rpy=-1.5707963267950237896 1.5707963267946956076 0
- joint left_hip_roll: origin xyz=0.018999999999999992589 -6.9388939039072283776e-18 -0.027499999999999968914 rpy=3.141592653589793116 -1.5707963267948794606 0 -> xyz=0.018999999999999999528 -1.3877787807814456755e-17 -0.027499999999999968914 rpy=3.141592653589793116 -1.5707963267944953234 0
- joint left_hip_yaw: origin xyz=0.034999999999999989453 -0.039999999999999993894 0.29868541999999997927 rpy=4.1258627841574100087e-29 -6.1232339957431151336e-17 1.5707963267949682784 -> xyz=0.0099999999999999915345 0.034999999999999913125 0.29868541999999997927 rpy=-1.8067035244472241688e-16 8.4612053737384914357e-16 -3.1415926535895151162
- joint left_knee: limit lower=-1.0471975511965976313 upper=2.0943951023931952626 effort=1 velocity=20 -> lower=-1.570796326794896558 upper=1.570796326794896558 effort=1 velocity=20; origin xyz=-4.1633363423443370266e-17 0.10750000000000001221 0.02149999999999999481 rpy=3.1415926535897895633 2.6314965551403718944e-14 1.047197551196626053 -> xyz=-3.9898639947466563171e-17 0.10750000000000001221 0.021499999999999998279 rpy=-3.141592653589793116 6.738865135048413848e-16 1.047197551196626053
- joint left_sho_pitch: origin xyz=0.06049999999999895739 -0.044999999999999804046 0.43008541999999988503 rpy=-1.5707963267948705788 3.7242253603279489435e-14 1.5707963267949578423 -> xyz=0.009999999999999812858 0.060500000000000025979 0.43008541999999988503 rpy=-1.5707963267948708008 3.5465916442993729594e-14 -3.1415926535897371608
- joint left_sho_roll: origin xyz=-0.018999999999999996059 0.0090000000000000079936 -0.02749999999999998973 rpy=-0 -1.5707963267948894526 0 -> xyz=-0.018999999999999996059 0.0090000000000000079936 -0.027500000000000003608 rpy=-8.3871691443097975151e-27 -1.570796326794896558 0
- joint neck: origin xyz=-1.0873011537518218883e-17 -0.040000000000000007772 0.45008542000000001382 rpy=-3.141592653589793116 7.7518614875493756421e-90 -1.2659750538598650252e-73 -> xyz=0.010000000000000005412 -7.4035645855646046943e-18 0.45008542000000001382 rpy=-3.141592653589793116 2.5403140807248779693e-85 1.570796326794896558
- joint right_ank_B11: origin xyz=0.019999999999999996947 -0.0099999999999999811262 -0.011499999999999982458 rpy=-1.570796326794896558 -1.4985484105593833704 1.5707963267948970021 -> xyz=0.020000000000000003886 -0.010000000000000008882 -0.011499999999999996336 rpy=-1.570796326794896558 -1.4985484105593944726 1.5707963267948243935
- joint right_ank_B12: origin xyz=0.01868001962352556708 -0.0099999999999999811262 0.023399999999999976374 rpy=1.57079632679490655 1.5020090633897773547 1.5707963267949058839 -> xyz=0.018680019623525320749 -0.010000000000000230926 0.023400000000000087397 rpy=1.5707963267948670261 1.5020090633897098531 1.5707963267948634734
- joint right_ank_B21: origin xyz=0.0044999999999999762412 2.7755575615628913511e-17 -0.017000000000000004691 rpy=-1.5707963267948961139 -1.5676670168131927596 -1.5707963267948830133 -> xyz=0.0044999999999999970579 -2.7755575615628913511e-17 -0.016999999999999987343 rpy=-1.5707963267948970021 -1.5676670168131963123 -1.5707963267930378226
- joint right_ank_B22: origin xyz=0.0044999999999999970579 0 0.017000000000000001221 rpy=-1.57079632679489678 1.55343465115961199 -1.5707963267948699126 -> xyz=0.0045000000000000074662 2.7755575615628913511e-17 0.016999999999999990813 rpy=-1.570796326794896558 1.5534346511595640283 -1.5707963267948497066
- joint right_ank_B31: origin xyz=2.168404344971008868e-19 0.0060500000000000553335 -0.0043000000000000052069 rpy=1.570796326794896558 5.4574690704063518601e-06 1.7018354478117103418e-17 -> xyz=3.4694469519536141888e-18 0.0060499999999999998224 -0.0042999999999999982681 rpy=1.570796326794896558 5.4574690872732503291e-06 -6.982789409669460301e-15
- joint right_ank_B32: origin xyz=2.8189256484623115284e-18 -0.0060500000000000275779 -0.0042999999999999947986 rpy=-1.570796326794896558 -5.4574694521280218192e-06 -1.2970245616443644851e-17 -> xyz=0 -0.0060499999999999998224 -0.0043000000000000052069 rpy=-1.570796326794896558 -5.4574696104194713947e-06 3.4815685893995744447e-15
- joint right_ank_R11: origin xyz=0.0099999999999999880651 -0.012499999999999993755 0.040600000000000004141 rpy=1.838132558719167337e-14 -1.968550043761323508e-15 3.0693447373542399603 -> xyz=0.010000000000000008882 -0.012499999999999986816 0.040599999999999997202 rpy=-1.2738457375408576304e-15 -4.0550136926307496733e-16 3.0693447373542608325
- joint right_ank_R12: origin xyz=-0.010000000000000005412 -0.012499999999999993755 0.040600000000000004141 rpy=-5.4208100503948111158e-17 1.2515168021403654183e-16 0.068787263405284487794 -> xyz=-0.009999999999999995004 -0.012499999999999997224 0.040600000000000004141 rpy=-1.4195250767777299134e-15 -8.2011968504619910654e-16 0.068787263405297796592
- joint right_ank_R21: origin xyz=0.0019999999999999948375 -0.009999999999999995004 -0.001900000000000000213 rpy=-1.5707963267948972241 -1.5676670168132933458 -1.570796326795488973 -> xyz=0.0020000000000000087153 -0.0099999999999999880651 -0.0018999999999999954425 rpy=-1.57079632679489678 -1.5676670168133319816 -1.5707963267950320052
- joint right_ank_R22: origin xyz=0.0020000000000000052458 0.0099999999999999984734 -0.0019000000000000006467 rpy=-1.57079632679489678 1.5534346511596015539 -1.5707963267942353092 -> xyz=0.0019999999999999983069 0.010000000000000008882 -0.0018999999999999919731 rpy=-1.570796326794896558 1.5534346511597014739 -1.5707963267948095165
- joint right_ank_act1: origin xyz=2.2722093422193351958e-06 -3.0045410603918298875e-15 -0.059245818700239413768 rpy=3.141592653589793116 2.3300461121301510461e-18 -0.63671356442004811704 -> xyz=2.2722093397584131047e-06 -2.7686186676589841227e-15 -0.059245818700240301946 rpy=-3.141592653589793116 7.3578695758415008682e-17 -0.63671356442004967136
- joint right_ank_act2: origin xyz=2.2722093449636677348e-06 1.7694179454963432363e-15 -0.059208011505606339409 rpy=-3.1415926535897860106 -1.9568267140524259683e-14 -0.636713564419863709 -> xyz=2.272209344501147088e-06 1.4641066137244251877e-15 -0.059208011505609073333 rpy=-3.1415926535897842342 -1.2265099222370623061e-14 -0.63671356441985804686
- joint right_ank_base: origin xyz=0 2.0816681711721685133e-17 -0.0064999999999999918954 rpy=-2.3897681857549792405e-16 -1.6802318149906911049e-16 1.0524335389525802942 -> xyz=3.9968028886505635455e-15 4.8572257327350598644e-16 -0.0064999999999950860974 rpy=1.27734443221197649e-13 -6.3880475103413010967e-14 1.0471975511965967431
- joint right_ank_foot: origin xyz=6.9388939039072283776e-18 -0.022499999999999999167 0.025600000000000018574 rpy=-1.5707963267949041075 -1.570796326794896558 0 -> xyz=0 -0.022499999999999995698 0.025600000000000008166 rpy=-1.570796326794896558 -1.570796326794896558 0
- joint right_ank_pitch: origin xyz=1.0408340855860842566e-16 -0.10000000000000013045 0.020900000000000147626 rpy=-7.5018482240547858138e-15 2.5176249968740924777e-16 1.5707963267948918951 -> xyz=-6.9388939039072283776e-18 -0.10000000000000000555 0.020899999999999994971 rpy=3.6059393234140185209e-15 -3.7146934833685194718e-15 1.570796326794886788
- joint right_ank_roll: origin xyz=-1.3877787807814456755e-17 0.0015000000000000013323 -0.014600000000000012274 rpy=1.570796326794896558 1.570796326794707154 0 -> xyz=6.9388939039072283776e-18 0.001500000000000034292 -0.014600000000000123296 rpy=1.5707963267948956698 1.5707963267946689623 0
- joint right_elb: origin xyz=-0.089500000000000065614 0 1.3877787807814456755e-17 rpy=-3.141592653589793116 -3.3306690738761288132e-16 1.5707963267948976682 -> xyz=-0.08950000000000021827 3.3306690738754696213e-16 9.3675067702747583098e-16 rpy=3.1415926535897562566 1.9686607660635860793e-14 1.5707963267949027752
- joint right_hip_pitch: origin xyz=-0.02400000071614186159 -0.019000000152455120972 -0.019000000152451717444 rpy=-1.5707963267946463137 -1.5707963267948112929 0 -> xyz=-0.024000000716142805279 -0.019000000152457847957 -0.019000000152452387048 rpy=-1.5707963267945825869 -1.5707963267948072961 0
- joint right_hip_roll: origin xyz=0.018999999999999999528 -6.9388939039072283776e-18 -0.027499999999999913403 rpy=3.141592653589793116 -1.5707963267948641395 0 -> xyz=0.018999999999999999528 -6.9388939039072283776e-18 -0.027499999999999968914 rpy=3.141592653589793116 -1.5707963267948796826 0
- joint right_hip_yaw: origin xyz=-0.035000000000000003331 -0.039999999999999993894 0.29868541999999997927 rpy=-6.3173742254660021089e-26 -6.1232339666714670147e-17 1.5707963267947904207 -> xyz=0.0099999999999999811262 -0.035000000000001744993 0.29868542000000003478 rpy=-5.1216840438065031123e-28 -6.1232339957451267289e-17 3.1415926535897638061
- joint right_knee: limit lower=-1.0471975511965976313 upper=2.0943951023931952626 effort=1 velocity=20 -> lower=-1.570796326794896558 upper=1.570796326794896558 effort=1 velocity=20; origin xyz=-4.1633363423443370266e-17 -0.10749999999999998446 0.016499999999999986899 rpy=-7.9136240096094387749e-16 -6.4063376207831640667e-16 -1.0471975511964932704 -> xyz=-5.0306980803327405738e-17 -0.10750000000000056732 0.016500000000000014655 rpy=-7.8824308298556449856e-16 -7.8500864033074576926e-16 -1.0471975511964610739
- joint right_sho_pitch: origin xyz=-0.060500000000000005163 -0.044999999999999977518 0.43008541999999994054 rpy=-1.570796326794896558 7.2736973397141567712e-16 -1.570796326794896558 -> xyz=0.010000000000000000208 -0.060499999999999568012 0.43008541999999994054 rpy=-1.570796326794896336 -2.036000207561118885e-14 3.7865323450622927166e-29
- joint right_sho_roll: origin xyz=0.019000000000000002998 0.0090000000000000079936 -0.02749999999999998973 rpy=-3.141592653589793116 -1.570796326794896558 0 -> xyz=0.018999999999999996059 0.0089999999999999524825 -0.027499999999999996669 rpy=-3.141592653589793116 -1.570796326794896558 0
