Commit message: Make the urdf modular

File: toddlerbot/robot_descriptions/base/base.urdf (robot description, URDF)
Before this commit: robot base, 50 links, 49 joints
Links:
- link ank_act_link: mass 0.044782197696050352054 -> 0.044782197690790455369; geometry collision mesh filename=../assemblies/left_3R+RH5_leg/meshes/left_ank_act_link_coll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; visual mesh filename=../assemblies/left_3R+RH5_leg/meshes/left_ank_act_link_visu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
- link ank_act_link_2: mass 0.044782197696050365932 -> 0.04478219769079044843; geometry collision mesh filename=../assemblies/left_3R+RH5_leg/meshes/left_ank_act_link_2_co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; visual mesh filename=../assemblies/left_3R+RH5_leg/meshes/left_ank_act_link_2_vi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
- link ank_act_link_3: mass 0.044782197696050358993 -> 0.044782197690790462308; geometry collision mesh filename=../assemblies/right_3R+RH5_leg/meshes/right_ank_act_link_co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; visual mesh filename=../assemblies/right_3R+RH5_leg/meshes/right_ank_act_link_vi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
- link ank_act_link_4: mass 0.044782197696050358993 -> 0.044782197690790455369; geometry collision mesh filename=../assemblies/right_3R+RH5_leg/meshes/right_ank_act_link_2_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; visual mesh filename=../assemblies/right_3R+RH5_leg/meshes/right_ank_act_link_2_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
- link ank_act_link_head: mass 0.0030517714925792842166 -> 0.003051771492579283783; geometry collision mesh filename=../assemblies/left_3R+RH5_leg/meshes/left_ank_act_link_head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; visual mesh filename=../assemblies/left_3R+RH5_leg/meshes/left_ank_act_link_head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
- link ank_act_link_head_2: mass 0.0030517714925792842166 -> 0.003051771492579283783; geometry collision mesh filename=../assemblies/left_3R+RH5_leg/meshes/left_ank_act_link_head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; visual mesh filename=../assemblies/left_3R+RH5_leg/meshes/left_ank_act_link_head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
- link ank_act_link_head_3: mass 0.0030517714925792842166 -> 0.003051771492579283783; geometry collision mesh filename=../assemblies/right_3R+RH5_leg/meshes/right_ank_act_link_he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; visual mesh filename=../assemblies/right_3R+RH5_leg/meshes/right_ank_act_link_he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
- link ank_act_link_head_4: mass 0.0030517714925792842166 -> 0.003051771492579283783; geometry collision mesh filename=../assemblies/right_3R+RH5_leg/meshes/right_ank_act_link_he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; visual mesh filename=../assemblies/right_3R+RH5_leg/meshes/right_ank_act_link_he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
- link ank_act_rod: geometry collision mesh filename=../assemblies/left_3R+RH5_leg/meshes/left_ank_act_rod_colli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; visual mesh filename=../assemblies/left_3R+RH5_leg/meshes/left_ank_act_rod_visua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
- link ank_act_rod_2: geometry collision mesh filename=../assemblies/left_3R+RH5_leg/meshes/left_ank_act_rod_2_col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; visual mesh filename=../assemblies/left_3R+RH5_leg/meshes/left_ank_act_rod_2_vis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
- link ank_act_rod_3: geometry collision mesh filename=../assemblies/right_3R+RH5_leg/meshes/right_ank_act_rod_col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; visual mesh filename=../assemblies/right_3R+RH5_leg/meshes/right_ank_act_rod_vis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
- link ank_act_rod_4: geometry collision mesh filename=../assemblies/right_3R+RH5_leg/meshes/right_ank_act_rod_2_c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; visual mesh filename=../assemblies/right_3R+RH5_leg/meshes/right_ank_act_rod_2_v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
- link ank_act_rod_head: geometry collision mesh filename=../assemblies/left_3R+RH5_leg/meshes/left_ank_act_rod_head_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; visual mesh filename=../assemblies/left_3R+RH5_leg/meshes/left_ank_act_rod_head_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
- link ank_act_rod_head_2: geometry collision mesh filename=../assemblies/left_3R+RH5_leg/meshes/left_ank_act_rod_head_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; visual mesh filename=../assemblies/left_3R+RH5_leg/meshes/left_ank_act_rod_head_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
- link ank_act_rod_head_3: geometry collision mesh filename=../assemblies/right_3R+RH5_leg/meshes/right_ank_act_rod_hea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; visual mesh filename=../assemblies/right_3R+RH5_leg/meshes/right_ank_act_rod_hea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
- link ank_act_rod_head_4: geometry collision mesh filename=../assemblies/right_3R+RH5_leg/meshes/right_ank_act_rod_hea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; visual mesh filename=../assemblies/right_3R+RH5_leg/meshes/right_ank_act_rod_hea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
- link ank_b_link: geometry collision mesh filename=../assemblies/left_3R+RH5_leg/meshes/left_ank_b_link_collis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; visual mesh filename=../assemblies/left_3R+RH5_leg/meshes/left_ank_b_link_visual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
- link ank_b_link_2: geometry collision mesh filename=../assemblies/left_3R+RH5_leg/meshes/left_ank_b_link_2_coll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; visual mesh filename=../assemblies/left_3R+RH5_leg/meshes/left_ank_b_link_2_visu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
- link ank_b_link_3: geometry collision mesh filename=../assemblies/right_3R+RH5_leg/meshes/right_ank_b_link_coll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; visual mesh filename=../assemblies/right_3R+RH5_leg/meshes/right_ank_b_link_visu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
- link ank_b_link_4: geometry collision mesh filename=../assemblies/right_3R+RH5_leg/meshes/right_ank_b_link_2_co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; visual mesh filename=../assemblies/right_3R+RH5_leg/meshes/right_ank_b_link_2_vi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
- link ank_pitch_link: geometry collision mesh filename=../assemblies/left_3R+RH5_leg/meshes/left_ank_pitch_link_co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; visual mesh filename=../assemblies/left_3R+RH5_leg/meshes/left_ank_pitch_link_vi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
- link ank_pitch_link_2: mass 0.0041366725921694342399 -> 0.0041366725921694333726; geometry collision mesh filename=../assemblies/right_3R+RH5_leg/meshes/right_ank_pitch_link_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; visual mesh filename=../assemblies/right_3R+RH5_leg/meshes/right_ank_pitch_link_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
- link ank_rigid_foot_link: geometry collision mesh filename=../assemblies/left_3R+RH5_leg/meshes/left_ank_rigid_foot_li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; visual mesh filename=../assemblies/left_3R+RH5_leg/meshes/left_ank_rigid_foot_li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
- link ank_rigid_foot_link_2: geometry collision mesh filename=../assemblies/right_3R+RH5_leg/meshes/right_ank_rigid_foot_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; visual mesh filename=../assemblies/right_3R+RH5_leg/meshes/right_ank_rigid_foot_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
- link ank_roll_link: geometry collision mesh filename=../assemblies/left_3R+RH5_leg/meshes/left_ank_roll_link_col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; visual mesh filename=../assemblies/left_3R+RH5_leg/meshes/left_ank_roll_link_vis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
- link ank_roll_link_2: geometry collision mesh filename=../assemblies/right_3R+RH5_leg/meshes/right_ank_roll_link_c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; visual mesh filename=../assemblies/right_3R+RH5_leg/meshes/right_ank_roll_link_v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
- link ank_rr_link: mass 0.0004758513732428606177 -> 0.00047585137324286072612; geometry collision mesh filename=../assemblies/left_3R+RH5_leg/meshes/left_ank_rr_link_colli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; visual mesh filename=../assemblies/left_3R+RH5_leg/meshes/left_ank_rr_link_visua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
- link ank_rr_link_2: mass 0.0004758513732428606177 -> 0.00047585137324286072612; geometry collision mesh filename=../assemblies/left_3R+RH5_leg/meshes/left_ank_rr_link_2_col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; visual mesh filename=../assemblies/left_3R+RH5_leg/meshes/left_ank_rr_link_2_vis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
- link ank_rr_link_3: mass 0.0004758513732428606177 -> 0.00047585137324286072612; geometry collision mesh filename=../assemblies/right_3R+RH5_leg/meshes/right_ank_rr_link_col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; visual mesh filename=../assemblies/right_3R+RH5_leg/meshes/right_ank_rr_link_vis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
- link ank_rr_link_4: mass 0.0004758513732428606177 -> 0.00047585137324286072612; geometry collision mesh filename=../assemblies/right_3R+RH5_leg/meshes/right_ank_rr_link_2_c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; visual mesh filename=../assemblies/right_3R+RH5_leg/meshes/right_ank_rr_link_2_v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
- link body_link: geometry collision mesh filename=../assemblies/4R_body/meshes/body_link_collision.stl; visual mesh filename=../assemblies/4R_body/meshes/body_link_visual.stl
- link elb_link: mass 0.011587175244532094132 -> 0.011587175244532097601; geometry collision mesh filename=../assemblies/left_OP3_arm/meshes/left_elb_link_collision.s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; visual mesh filename=../assemblies/left_OP3_arm/meshes/left_elb_link_visual.stl
- link elb_link_2: mass 0.011587175244532094132 -> 0.011587175244532097601; geometry collision mesh filename=../assemblies/right_OP3_arm/meshes/right_elb_link_collision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; visual mesh filename=../assemblies/right_OP3_arm/meshes/right_elb_link_visual.stl
- link head_link: geometry collision mesh filename=../assemblies/4R_body/meshes/head_link_collision.stl; visual mesh filename=../assemblies/4R_body/meshes/head_link_visual.stl
- link hip_pitch_link: mass 0.075144662701080264244 -> 0.075144662701080278122; geometry collision mesh filename=../assemblies/left_3R+RH5_leg/meshes/left_hip_pitch_link_co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; visual mesh filename=../assemblies/left_3R+RH5_leg/meshes/left_hip_pitch_link_vi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
- link hip_pitch_link_2: mass 0.075144662701080264244 -> 0.075144662701080278122; geometry collision mesh filename=../assemblies/right_3R+RH5_leg/meshes/right_hip_pitch_link_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; visual mesh filename=../assemblies/right_3R+RH5_leg/meshes/right_hip_pitch_link_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
- link hip_roll_link: mass 0.098012391483528707448 -> 0.098012391483528665814; geometry collision mesh filename=../assemblies/left_3R+RH5_leg/meshes/left_hip_roll_link_col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; visual mesh filename=../assemblies/left_3R+RH5_leg/meshes/left_hip_roll_link_vis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
- link hip_roll_link_2: mass 0.098012391483528707448 -> 0.098012391483528665814; geometry collision mesh filename=../assemblies/right_3R+RH5_leg/meshes/right_hip_roll_link_c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; visual mesh filename=../assemblies/right_3R+RH5_leg/meshes/right_hip_roll_link_v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
- link hip_yaw_link: mass 0.0052740645607467504311 -> 0.0052740645607467486963; geometry collision mesh filename=../assemblies/left_3R+RH5_leg/meshes/left_hip_yaw_link_coll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; visual mesh filename=../assemblies/left_3R+RH5_leg/meshes/left_hip_yaw_link_visu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
- link hip_yaw_link_2: mass 0.0052740645607467504311 -> 0.0052740645607467486963; geometry collision mesh filename=../assemblies/right_3R+RH5_leg/meshes/right_hip_yaw_link_co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; visual mesh filename=../assemblies/right_3R+RH5_leg/meshes/right_hip_yaw_link_vi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
- link knee_link: mass 0.0043868974356887730989 -> 0.0043868974356887722316; geometry collision mesh filename=../assemblies/left_3R+RH5_leg/meshes/left_knee_link_collisi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; visual mesh filename=../assemblies/left_3R+RH5_leg/meshes/left_knee_link_visual.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
- link knee_link_2: mass 0.0043868974356887730989 -> 0.0043868974356887722316; geometry collision mesh filename=../assemblies/right_3R+RH5_leg/meshes/right_knee_link_colli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; visual mesh filename=../assemblies/right_3R+RH5_leg/meshes/right_knee_link_visua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
- link left_ank_base_link: mass 0.014262086197619733285 -> 0.014262086197619729816; geometry collision mesh filename=../assemblies/left_3R+RH5_leg/meshes/left_ank_base_link_col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; visual mesh filename=../assemblies/left_3R+RH5_leg/meshes/left_ank_base_link_vis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
- link neck_link: geometry collision mesh filename=../assemblies/4R_body/meshes/neck_link_collision.stl; visual mesh filename=../assemblies/4R_body/meshes/neck_link_visual.stl
- link right_ank_base_link: mass 0.014262085602793541511 -> 0.014262085602793538042; geometry collision mesh filename=../assemblies/right_3R+RH5_leg/meshes/right_ank_base_link_c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; visual mesh filename=../assemblies/right_3R+RH5_leg/meshes/right_ank_base_link_v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
- link sho_pitch_link: geometry collision mesh filename=../assemblies/left_OP3_arm/meshes/left_sho_pitch_link_colli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; visual mesh filename=../assemblies/left_OP3_arm/meshes/left_sho_pitch_link_visua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
- link sho_pitch_link_2: geometry collision mesh filename=../assemblies/right_OP3_arm/meshes/right_sho_pitch_link_col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; visual mesh filename=../assemblies/right_OP3_arm/meshes/right_sho_pitch_link_vis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
- link sho_roll_link: mass 0.14053933881247801518 -> 0.14053933881247793192; geometry collision mesh filename=../assemblies/left_OP3_arm/meshes/left_sho_roll_link_collis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; visual mesh filename=../assemblies/left_OP3_arm/meshes/left_sho_roll_link_visual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
- link sho_roll_link_2: mass 0.14053933881247798743 -> 0.14053933881247795967; geometry collision mesh filename=../assemblies/right_OP3_arm/meshes/right_sho_roll_link_coll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; visual mesh filename=../assemblies/right_OP3_arm/meshes/right_sho_roll_link_visu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
Joints:
- joint left_ank_B11: origin xyz=0.018680019623525362382 0.009999999999999731326 0.023399999999999900047 rpy=-1.5707963267948952257 -1.505343593990304818 1.5707963267948974462 -> xyz=0.018680019623525050132 0.0099999999999995092814 0.023399999999999601674 rpy=-1.570796326794896558 -1.5053435939902766183 1.5707963267949058839
- joint left_ank_B12: origin xyz=0.019999999999999996947 0.010000000000000008882 -0.011499999999999996336 rpy=1.570796326794896558 1.4952155260088879629 1.57079632679525516 -> xyz=0.020000000000000007355 0.010000000000000064393 -0.011499999999999999806 rpy=1.570796326794896558 1.4952155260088901834 1.5707963267949052177
- joint left_ank_B21: origin xyz=-0.0044999999999999970579 2.7755575615628913511e-17 -0.016999999999999997752 rpy=1.57079632679489678 1.5534345204864243861 -1.5707963267948996666 -> xyz=-0.0045000000000000005274 0 -0.016999999999999994282 rpy=1.57079632679489678 1.5534345204863466705 -1.5707963267948821251
- joint left_ank_B22: origin xyz=-0.0044999999999999970579 0 0.016999999999999994282 rpy=1.5707963267990325829 -1.567667040345596563 -1.5707963267904616611 -> xyz=-0.0045000000000000005274 -2.7755575615628913511e-17 0.016999999999999997752 rpy=1.57079632679489678 -1.5676670403455787994 -1.5707963267950848518
- joint left_ank_B31: origin xyz=-1.3877787807814456755e-17 -0.0060500000000000830891 -0.0043000000000000086764 rpy=1.570796326794896558 5.4574690367119021436e-06 -3.141592653589793116 -> xyz=0 -0.0060500000000000275779 -0.0042999999999999947986 rpy=1.570796326794896558 5.4574690924646923929e-06 3.1415926535897926719
- joint left_ank_B32: origin xyz=0 0.0060499999999999998224 -0.0042999999999999913292 rpy=-1.570796326794896558 -5.4574692127553140676e-06 3.1415926535897922278 -> xyz=1.3877787807814456755e-17 0.0060500000000000275779 -0.0043000000000000017375 rpy=-1.570796326794896558 -5.4574692361237511426e-06 3.1415926535897891192
- joint left_ank_R11: origin xyz=0.010000000000000001943 -0.012500000000000007633 0.040599999999999997202 rpy=-2.3809415734231673378e-15 -2.8771866469601532264e-15 3.0761399207850583792 -> xyz=0.010000000000000000208 -0.012499999999999955591 0.040599999999999990263 rpy=-7.1428247202731315625e-15 -8.6315599408597654911e-15 3.0761399207850761428
- joint left_ank_R12: origin xyz=-0.009999999999999995004 -0.012500000000000011102 0.040599999999999997202 rpy=-1.3103682910477166415e-14 1.457398994851742625e-15 0.075580800785893090254 -> xyz=-0.0099999999999999984734 -0.012500000000000011102 0.040600000000000004141 rpy=-5.5307227023405179375e-16 7.5341850347009380651e-16 0.075580800785909410533
- joint left_ank_R21: origin xyz=0.0020000000000000017764 -0.0099999999999999984734 -0.001899999999999998912 rpy=-1.570796326794896558 -1.5534345204864692391 -1.5707963267950264541 -> xyz=0.0019999999999999983069 -0.010000000000000008882 -0.0018999999999999919731 rpy=-1.57079632679489678 -1.5534345204864852263 -1.5707963267953415354
- joint left_ank_R22: origin xyz=0.0020000000000000087153 0.0099999999999999984734 -0.0019000000000000058509 rpy=-1.57079632679489678 1.567667040345726015 -1.5707963267956523978 -> xyz=0.0019999999999999878986 0.0099999999999998978595 -0.0019000000000000058509 rpy=-1.5707963267948954478 1.5676670403457018121 -1.5707963267948694686
- joint left_ank_act1: origin xyz=2.2722093436094992214e-06 -2.5604518505417672714e-15 -0.059207313423198439095 rpy=-3.141592653589793116 1.328302970873878818e-14 -0.6367135644199727329 -> xyz=2.2722093436094992214e-06 -2.5673907444456744997e-15 -0.059207313423197016622 rpy=-3.141592653589793116 2.2049374431327776337e-15 -0.63671356442004234388
- joint left_ank_act2: origin xyz=2.2722093434603130024e-06 -2.8449465006019636348e-16 -0.059246516530142220858 rpy=3.141592653589793116 1.5679305736050431748e-15 -0.63671356442004867215 -> xyz=2.272209343491538025e-06 -2.8449465006019636348e-16 -0.059246516530139459178 rpy=3.141592653589793116 6.3943189148119461475e-15 -0.63671356442004400922
- joint left_ank_base: origin xyz=-3.0253577421035515727e-15 -3.2196467714129539672e-15 -0.0064999999999985694221 rpy=-9.7170810831163359999e-14 1.1559030630111302718e-13 -2.0943951023931739464 -> xyz=-2.9698465908722937456e-15 -3.233524559220768424e-15 -0.0064999999999985815652 rpy=-1.0661697646906630524e-13 1.1573381888160480481e-13 -2.0943951023931757227
- joint left_ank_foot: origin xyz=-6.9388939039072283776e-18 -0.022500000000000009576 0.025600000000000004696 rpy=-1.570796326794896558 -1.5707963267948956698 0 -> xyz=2.6020852139652106416e-18 -0.022499999999999964473 0.025600000000000008166 rpy=-1.5707963267948961139 -1.5707963267948961139 0
- joint left_ank_pitch: origin xyz=-5.7245874707234634116e-17 0.10000000000000028311 0.020900000000000012318 rpy=-8.6690501906182033625e-15 2.4133613739470252907e-15 1.5707963267949272002 -> xyz=-1.6741183324487654366e-16 0.10000000000000086597 0.020900000000000071299 rpy=-3.0159878742287526962e-14 3.8772695991165318582e-15 1.5707963267949285324
- joint left_ank_roll: origin xyz=-6.9388939039072283776e-18 0.0014999999999998920447 -0.014600000000000140643 rpy=1.5707963267949041075 -1.570796326794886788 0 -> xyz=-5.5511151231257827021e-17 0.0014999999999999904902 -0.01460000000000040779 rpy=1.5707963267949189845 -1.5707963267948734654 0
- joint left_elb: origin xyz=-0.089499999999999607647 -6.6613381477509392425e-16 6.1860239153332940987e-15 rpy=3.1415926535897122918 4.7267745273418620861e-14 -1.5707963267948943376 -> xyz=-0.089499999999999663158 -3.2265856653168611956e-16 5.9049987122250513494e-15 rpy=3.1415926535897367167 2.2793048768987009608e-14 -1.5707963267948858999
- joint left_hip_pitch: origin xyz=-0.02400000071614330488 -0.019000000152458163677 -0.019000000152447526353 rpy=-1.5707963267950237896 1.5707963267946956076 0 -> xyz=-0.024000000716143325696 -0.019000000152458135921 -0.019000000152447495128 rpy=-1.5707963267950240116 1.5707963267946891683 0
- joint left_hip_roll: origin xyz=0.018999999999999999528 -1.3877787807814456755e-17 -0.027499999999999968914 rpy=3.141592653589793116 -1.5707963267944953234 0 -> xyz=0.01900000000000030137 -8.4257398398633673697e-18 -0.027500000000000288103 rpy=3.141592653589793116 -1.5707963267948705788 0
- joint left_hip_yaw: origin xyz=0.0099999999999999915345 0.034999999999999913125 0.29868541999999997927 rpy=-1.8067035244472241688e-16 8.4612053737384914357e-16 -3.1415926535895151162 -> xyz=0.0099999999999999915345 0.034999999999999982514 0.29868541999999997927 rpy=-1.2830740121451429552e-26 -6.1232339959922830135e-17 3.1415926535897598093
- joint left_knee: origin xyz=-3.9898639947466563171e-17 0.10750000000000001221 0.021499999999999998279 rpy=-3.141592653589793116 6.738865135048413848e-16 1.047197551196626053 -> xyz=7.9552488872441493797e-18 0.10749999999999991507 0.021500000000001306261 rpy=-3.141592653589793116 1.8251939963481432238e-15 1.0471975511966649108
- joint left_sho_roll: origin xyz=-0.018999999999999996059 0.0090000000000000079936 -0.027500000000000003608 rpy=-8.3871691443097975151e-27 -1.570796326794896558 0 -> xyz=-0.018999999999999999528 0.0089999999999999646255 -0.027499999999999986261 rpy=-6.3254956828146051492e-14 -1.5707963267948947816 0
- joint right_ank_B11: origin xyz=0.020000000000000003886 -0.010000000000000008882 -0.011499999999999996336 rpy=-1.570796326794896558 -1.4985484105593944726 1.5707963267948243935 -> xyz=0.019999999999999990008 -0.010000000000000064393 -0.011500000000000110828 rpy=-1.5707963267949649477 -1.498548410559401356 1.570796326794752229
- joint right_ank_B12: origin xyz=0.018680019623525320749 -0.010000000000000230926 0.023400000000000087397 rpy=1.5707963267948670261 1.5020090633897098531 1.5707963267948634734 -> xyz=0.018680019623525341566 -0.010000000000000314193 0.023400000000000680672 rpy=1.5707963267949003328 1.5020090633896872045 1.5707963267948876762
- joint right_ank_B21: origin xyz=0.0044999999999999970579 -2.7755575615628913511e-17 -0.016999999999999987343 rpy=-1.5707963267948970021 -1.5676670168131963123 -1.5707963267930378226 -> xyz=0.00450000000000061115 -5.5511151231257827021e-17 -0.016999999999999966527 rpy=-1.5707963267952360642 -1.567667016813194536 -1.5707963267890037162
- joint right_ank_B22: origin xyz=0.0045000000000000074662 2.7755575615628913511e-17 0.016999999999999990813 rpy=-1.570796326794896558 1.5534346511595640283 -1.5707963267948497066 -> xyz=0.0045000000000000144051 8.3266726846886740532e-17 0.01700000000000001163 rpy=-1.5707963267949425212 1.5534346511595631402 -1.5707963267948024111
- joint right_ank_B31: origin xyz=3.4694469519536141888e-18 0.0060499999999999998224 -0.0042999999999999982681 rpy=1.570796326794896558 5.4574690872732503291e-06 -6.982789409669460301e-15 -> xyz=-4.1633363423443370266e-17 0.0060499999999999998224 -0.0043000000000000086764 rpy=1.5707963267948934494 5.4574690957684207369e-06 -1.3977638364514914411e-14
- joint right_ank_B32: origin xyz=0 -0.0060499999999999998224 -0.0043000000000000052069 rpy=-1.570796326794896558 -5.4574696104194713947e-06 3.4815685893995744447e-15 -> xyz=1.3877787807814456755e-17 -0.0060499999999998332889 -0.0043000000000000607181 rpy=-1.5707963267948961139 -5.45746960946283069e-06 6.9689783799507381887e-15
- joint right_ank_R11: origin xyz=0.010000000000000008882 -0.012499999999999986816 0.040599999999999997202 rpy=-1.2738457375408576304e-15 -4.0550136926307496733e-16 3.0693447373542608325 -> xyz=0.0099999999999999429623 -0.012500000000000066613 0.040600000000000337208 rpy=-2.5476914750798164726e-15 -8.1100273852236014827e-16 3.0693447373540605483
- joint right_ank_R12: origin xyz=-0.009999999999999995004 -0.012499999999999997224 0.040600000000000004141 rpy=-1.4195250767777299134e-15 -8.2011968504619910654e-16 0.068787263405297796592 -> xyz=-0.0099999999999999516359 -0.012499999999999955591 0.040600000000000358025 rpy=-1.2454338751916450574e-14 5.795879650126974938e-15 0.068787263405096929492
- joint right_ank_R21: origin xyz=0.0020000000000000087153 -0.0099999999999999880651 -0.0018999999999999954425 rpy=-1.57079632679489678 -1.5676670168133319816 -1.5707963267950320052 -> xyz=0.001999999999999991368 -0.010000000000000008882 -0.0019000000000000336065 rpy=-1.5707963267950324493 -1.5676670168133113314 -1.5707963267951672304
- joint right_ank_R22: origin xyz=0.0019999999999999983069 0.010000000000000008882 -0.0018999999999999919731 rpy=-1.570796326794896558 1.5534346511597014739 -1.5707963267948095165 -> xyz=0.0019999999999999844291 0.0099999999999997868372 -0.0019000000000000058509 rpy=-1.5707963267949827113 1.5534346511596899276 -1.570796326794722253
- joint right_ank_act1: origin xyz=2.2722093397584131047e-06 -2.7686186676589841227e-15 -0.059245818700240301946 rpy=-3.141592653589793116 7.3578695758415008682e-17 -0.63671356442004967136 -> xyz=2.2722093397584131047e-06 -2.7616797737550768943e-15 -0.059245818700238817023 rpy=-3.141592653589793116 7.8730370890791872833e-17 -0.63671356442004978238
- joint right_ank_act2: origin xyz=2.272209344501147088e-06 1.4641066137244251877e-15 -0.059208011505609073333 rpy=-3.1415926535897842342 -1.2265099222370623061e-14 -0.63671356441985804686 -> xyz=2.2722093444768609594e-06 1.4190038033490282032e-15 -0.059208011505612251346 rpy=-3.1415926535897846783 -1.2262068103869690541e-14 -0.6367135644198562705
- joint right_ank_base: origin xyz=3.9968028886505635455e-15 4.8572257327350598644e-16 -0.0064999999999950860974 rpy=1.27734443221197649e-13 -6.3880475103413010967e-14 1.0471975511965967431 -> xyz=3.9968028886505635455e-15 5.1347814888913489995e-16 -0.0064999999999950722196 rpy=1.2818767136087556972e-13 -6.6450035636680710077e-14 1.0471975511965969652
- joint right_ank_foot: origin xyz=0 -0.022499999999999995698 0.025600000000000008166 rpy=-1.570796326794896558 -1.570796326794896558 0 -> xyz=1.3877787807814456755e-17 -0.022500000000000131006 0.025600000000000136535 rpy=-1.570796326794896558 -1.570796326794896558 0
- joint right_ank_pitch: origin xyz=-6.9388939039072283776e-18 -0.10000000000000000555 0.020899999999999994971 rpy=3.6059393234140185209e-15 -3.7146934833685194718e-15 1.570796326794886788 -> xyz=-1.357934238180394094e-16 -0.10000000000000008882 0.020900000000000668043 rpy=7.2118786468278761141e-15 -7.4293869667367865081e-15 1.5707963267948599206
- joint right_ank_roll: origin xyz=6.9388939039072283776e-18 0.001500000000000034292 -0.014600000000000123296 rpy=1.5707963267948956698 1.5707963267946689623 0 -> xyz=5.5511151231257827021e-17 0.0014999999999999475558 -0.014600000000000026151 rpy=1.5707963267948925612 1.5707963267948934494 0
- joint right_elb: origin xyz=-0.08950000000000021827 3.3306690738754696213e-16 9.3675067702747583098e-16 rpy=3.1415926535897562566 1.9686607660635860793e-14 1.5707963267949027752 -> xyz=-0.08949999999999827538 -7.2650219173908681114e-15 1.0956513474269513608e-14 rpy=-3.1415926535897145122 9.187667647645342109e-14 1.5707963267949796027
- joint right_hip_pitch: origin xyz=-0.024000000716142805279 -0.019000000152457847957 -0.019000000152452387048 rpy=-1.5707963267945825869 -1.5707963267948072961 0 -> xyz=-0.024000000716142506907 -0.019000000152458108166 -0.019000000152452390517 rpy=-1.5707963267945823649 -1.570796326794816844 0
- joint right_hip_roll: origin xyz=0.018999999999999999528 -6.9388939039072283776e-18 -0.027499999999999968914 rpy=3.141592653589793116 -1.5707963267948796826 0 -> xyz=0.018999999999999829525 -1.2563796310537849955e-17 -0.027499999999999951567 rpy=3.1415926535897926719 -1.570796326794896558 0
- joint right_hip_yaw: origin xyz=0.0099999999999999811262 -0.035000000000001744993 0.29868542000000003478 rpy=-5.1216840438065031123e-28 -6.1232339957451267289e-17 3.1415926535897638061 -> xyz=0.0099999999999999897998 -0.034999999999999989453 0.29868541999999997927 rpy=-2.8487879681803368219e-27 -6.1232339957719874427e-17 -3.1415926535897793492
- joint right_knee: origin xyz=-5.0306980803327405738e-17 -0.10750000000000056732 0.016500000000000014655 rpy=-7.8824308298556449856e-16 -7.8500864033074576926e-16 -1.0471975511964610739 -> xyz=-1.5911557041301218853e-16 -0.10750000000000003997 0.016499999999999702405 rpy=-1.7587631597966056551e-15 -9.4692391792157564628e-16 -1.0471975511964521921
- joint right_sho_pitch: origin xyz=0.010000000000000000208 -0.060499999999999568012 0.43008541999999994054 rpy=-1.570796326794896336 -2.036000207561118885e-14 3.7865323450622927166e-29 -> xyz=0.0099999999999999932693 -0.06050000000000008149 0.43008541999999999605 rpy=-1.570796326794896336 6.9606380272961593273e-16 1.3836137928249486855e-31
- joint right_sho_roll: origin xyz=0.018999999999999996059 0.0089999999999999524825 -0.027499999999999996669 rpy=-3.141592653589793116 -1.570796326794896558 0 -> xyz=0.018999999999999954425 0.0089999999999999576866 -0.027499999999999899525 rpy=-3.1415926535896976368 -1.5707963267948958919 0
