Commit message: Fix the collision meshes

File: toddlerbot/robot_descriptions/base/base.urdf (robot description, URDF)
Before this commit: robot base, 45 links, 44 joints
Links:
- link 12lf: geometry visual mesh filename=../assemblies/left_3R+RH5_leg/meshes/left_12lf_visual.stl
- link 12lf_2: geometry visual mesh filename=../assemblies/left_3R+RH5_leg/meshes/left_12lf_2_visual.stl
- link 12lf_3: geometry visual mesh filename=../assemblies/right_3R+RH5_leg/meshes/right_12lf_visual.stl
- link 12lf_4: geometry visual mesh filename=../assemblies/right_3R+RH5_leg/meshes/right_12lf_2_visual.s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
- link 12lf_rod: geometry visual mesh filename=../assemblies/left_3R+RH5_leg/meshes/left_12lf_rod_visual.s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
- link 12lf_rod_2: geometry visual mesh filename=../assemblies/left_3R+RH5_leg/meshes/left_12lf_rod_2_visual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
- link 12lf_rod_3: geometry visual mesh filename=../assemblies/right_3R+RH5_leg/meshes/right_12lf_rod_visual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
- link 12lf_rod_4: geometry visual mesh filename=../assemblies/right_3R+RH5_leg/meshes/right_12lf_rod_2_visu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
- link 12lf_rod_end: geometry visual mesh filename=../assemblies/left_3R+RH5_leg/meshes/left_12lf_rod_end_visu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
- link 12lf_rod_end_2: geometry visual mesh filename=../assemblies/left_3R+RH5_leg/meshes/left_12lf_rod_end_2_vi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
- link 12lf_rod_end_3: geometry visual mesh filename=../assemblies/right_3R+RH5_leg/meshes/right_12lf_rod_end_vi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
- link 12lf_rod_end_4: geometry visual mesh filename=../assemblies/right_3R+RH5_leg/meshes/right_12lf_rod_end_2_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
- link ank_pitch_link: geometry visual mesh filename=../assemblies/left_3R+RH5_leg/meshes/left_ank_pitch_link_vi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
- link ank_pitch_link_2: geometry visual mesh filename=../assemblies/right_3R+RH5_leg/meshes/right_ank_pitch_link_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
- link ank_roll_link: geometry collision mesh filename=collisions/left_ank_roll_link_collision.stl; visual mesh filename=../assemblies/left_3R+RH5_leg/meshes/left_ank_roll_link_vis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
- link ank_roll_link_2: geometry collision mesh filename=collisions/right_ank_roll_link_collision.stl; visual mesh filename=../assemblies/right_3R+RH5_leg/meshes/right_ank_roll_link_v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
- link ank_rr_link: geometry visual mesh filename=../assemblies/left_3R+RH5_leg/meshes/left_ank_rr_link_visua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
- link ank_rr_link_2: geometry visual mesh filename=../assemblies/left_3R+RH5_leg/meshes/left_ank_rr_link_2_vis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
- link ank_rr_link_3: geometry visual mesh filename=../assemblies/right_3R+RH5_leg/meshes/right_ank_rr_link_vis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
- link ank_rr_link_4: geometry visual mesh filename=../assemblies/right_3R+RH5_leg/meshes/right_ank_rr_link_2_v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
- link ball_joint_ball: geometry visual mesh filename=../assemblies/left_3R+RH5_leg/meshes/left_ball_joint_ball_v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
- link ball_joint_ball_2: geometry visual mesh filename=../assemblies/left_3R+RH5_leg/meshes/left_ball_joint_ball_2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
- link ball_joint_ball_3: geometry visual mesh filename=../assemblies/right_3R+RH5_leg/meshes/right_ball_joint_ball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
- link ball_joint_ball_4: geometry visual mesh filename=../assemblies/right_3R+RH5_leg/meshes/right_ball_joint_ball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
- link ball_joint_container: geometry visual mesh filename=../assemblies/left_3R+RH5_leg/meshes/left_ball_joint_contai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
- link ball_joint_container_2: geometry visual mesh filename=../assemblies/left_3R+RH5_leg/meshes/left_ball_joint_contai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
- link ball_joint_container_3: geometry visual mesh filename=../assemblies/right_3R+RH5_leg/meshes/right_ball_joint_cont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
- link ball_joint_container_4: geometry visual mesh filename=../assemblies/right_3R+RH5_leg/meshes/right_ball_joint_cont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
- link body_link: geometry collision mesh filename=collisions/body_link_collision.stl; visual mesh filename=../assemblies/4R_body/meshes/body_link_visual.stl
- link elb_link: geometry collision mesh filename=collisions/left_elb_link_collision.stl; visual mesh filename=../assemblies/left_OP3_arm/meshes/left_elb_link_visual.stl
- link elb_link_2: geometry collision mesh filename=collisions/right_elb_link_collision.stl; visual mesh filename=../assemblies/right_OP3_arm/meshes/right_elb_link_visual.stl
- link head_link: geometry collision mesh filename=collisions/head_link_collision.stl; visual mesh filename=../assemblies/4R_body/meshes/head_link_visual.stl
- link hip_roll_link: geometry collision mesh filename=collisions/left_hip_roll_link_collision.stl; visual mesh filename=../assemblies/left_3R+RH5_leg/meshes/left_hip_roll_link_vis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
- link hip_roll_link_2: geometry collision mesh filename=collisions/right_hip_roll_link_collision.stl; visual mesh filename=../assemblies/right_3R+RH5_leg/meshes/right_hip_roll_link_v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
- link hip_yaw_link: geometry visual mesh filename=../assemblies/left_3R+RH5_leg/meshes/left_hip_yaw_link_visu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
- link hip_yaw_link_2: geometry visual mesh filename=../assemblies/right_3R+RH5_leg/meshes/right_hip_yaw_link_vi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
- link left_calf_link: geometry collision mesh filename=collisions/left_calf_link_collision.stl; visual mesh filename=../assemblies/left_3R+RH5_leg/meshes/left_calf_link_visual.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
- link left_hip_pitch_link: geometry collision mesh filename=collisions/left_hip_pitch_link_collision.stl; visual mesh filename=../assemblies/left_3R+RH5_leg/meshes/left_hip_pitch_link_vi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
- link neck_link: geometry collision mesh filename=collisions/neck_link_collision.stl; visual mesh filename=../assemblies/4R_body/meshes/neck_link_visual.stl
- link right_calf_link: geometry collision mesh filename=collisions/right_calf_link_collision.stl; visual mesh filename=../assemblies/right_3R+RH5_leg/meshes/right_calf_link_visua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
- link right_hip_pitch_link: geometry collision mesh filename=collisions/right_hip_pitch_link_collision.stl; visual mesh filename=../assemblies/right_3R+RH5_leg/meshes/right_hip_pitch_link_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
- link sho_pitch_link: geometry visual mesh filename=../assemblies/left_OP3_arm/meshes/left_sho_pitch_link_visua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
- link sho_pitch_link_2: geometry visual mesh filename=../assemblies/right_OP3_arm/meshes/right_sho_pitch_link_vis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
- link sho_roll_link: geometry collision mesh filename=collisions/left_sho_roll_link_collision.stl; visual mesh filename=../assemblies/left_OP3_arm/meshes/left_sho_roll_link_visual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
- link sho_roll_link_2: geometry collision mesh filename=collisions/right_sho_roll_link_collision.stl; visual mesh filename=../assemblies/right_OP3_arm/meshes/right_sho_roll_link_visu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
