Commit message: Refactor the walking task
- Include history error into zmp preview control
- Update the planner to plan a hermite spline path
- Remove redundant configs
- Add vis functions

File: toddlerbot/robot_descriptions/assemblies/4R_body/4R_body.urdf (robot description, URDF)
Before this commit: robot 4R_body, 8 links, 7 joints
Links:
- link body_link: mass 0.67608257475273081383 -> 0.67608257475273170201
- link left_3r+rh5_leg: mass 0.31997833445896267657 -> 0.3199783344694824283
- link right_3r+rh5_leg: mass 0.31997833386413643275 -> 0.31997833387465629551
- link right_op3_arm: mass 0.15719799404180678781 -> 0.15719799404180676006
Joints:
- joint head: origin xyz=0 1.7347234759768070944e-18 -0.039999999999999980016 rpy=0 -1.0509729472670562853e-99 -4.1486002514987779604e-69 -> xyz=0 8.6736173798840354721e-19 -0.039999999999999980016 rpy=0 -1.0509729472670562853e-99 -4.1486002514987779604e-69
- joint left_hip_yaw: origin xyz=0.0099999999999999915345 0.034999999999999982514 0.29868541999999997927 rpy=-1.2830740121451429552e-26 -6.1232339959922830135e-17 3.1415926535897598093 -> xyz=-0.0064000000000000055109 0.034999999999999982514 0.29859999999999997655 rpy=2.5294987785272742576e-29 -6.1232339957503159545e-17 3.1415926535897900074
- joint left_sho_pitch: origin xyz=0.009999999999999812858 0.060500000000000025979 0.43008541999999988503 rpy=-1.5707963267948708008 3.5465916442993729594e-14 -3.1415926535897371608 -> xyz=-0.0064000000000001572992 0.060499999999999110045 0.42999999999999988232 rpy=-1.5707963267948708008 3.5465916442993729594e-14 -3.1415926535897371608
- joint neck: origin xyz=0.010000000000000005412 -7.4035645855646046943e-18 0.45008542000000001382 rpy=-3.141592653589793116 2.5403140807248779693e-85 1.570796326794896558 -> xyz=-0.0063999999999999925004 -7.4035645855646046943e-18 0.4500000000000000111 rpy=-3.141592653589793116 2.5403140807248779693e-85 1.570796326794896558
- joint right_hip_yaw: origin xyz=0.0099999999999999897998 -0.034999999999999989453 0.29868541999999997927 rpy=-2.8487879681803368219e-27 -6.1232339957719874427e-17 -3.1415926535897793492 -> xyz=-0.0064000000000000063782 -0.034999999999999996392 0.29859999999999997655 rpy=-4.0795765885139752246e-16 -1.4246408104590497614e-16 -3.1415926535897877869
- joint right_sho_pitch: origin xyz=0.0099999999999999932693 -0.06050000000000008149 0.43008541999999999605 rpy=-1.570796326794896336 6.9606380272961593273e-16 1.3836137928249486855e-31 -> xyz=-0.0064000000000000063782 -0.06050000000000008149 0.42999999999999993783 rpy=-1.570796326794896336 6.9606380272961593273e-16 1.3836137928249486855e-31

File: toddlerbot/robot_descriptions/base/base.urdf (robot description, URDF)
Before this commit: robot base, 50 links, 49 joints
Links:
- link body_link: mass 0.67608257475273081383 -> 0.67608257475273170201
Joints:
- joint head: origin xyz=0 1.7347234759768070944e-18 -0.039999999999999980016 rpy=0 -1.0509729472670562853e-99 -4.1486002514987779604e-69 -> xyz=0 8.6736173798840354721e-19 -0.039999999999999980016 rpy=0 -1.0509729472670562853e-99 -4.1486002514987779604e-69
- joint left_hip_yaw: origin xyz=0.0099999999999999915345 0.034999999999999982514 0.29868541999999997927 rpy=-1.2830740121451429552e-26 -6.1232339959922830135e-17 3.1415926535897598093 -> xyz=-0.0064000000000000055109 0.034999999999999982514 0.29859999999999997655 rpy=2.5294987785272742576e-29 -6.1232339957503159545e-17 3.1415926535897900074
- joint left_sho_pitch: origin xyz=0.009999999999999812858 0.060500000000000025979 0.43008541999999988503 rpy=-1.5707963267948708008 3.5465916442993729594e-14 -3.1415926535897371608 -> xyz=-0.0064000000000001572992 0.060499999999999110045 0.42999999999999988232 rpy=-1.5707963267948708008 3.5465916442993729594e-14 -3.1415926535897371608
- joint neck: origin xyz=0.010000000000000005412 -7.4035645855646046943e-18 0.45008542000000001382 rpy=-3.141592653589793116 2.5403140807248779693e-85 1.570796326794896558 -> xyz=-0.0063999999999999925004 -7.4035645855646046943e-18 0.4500000000000000111 rpy=-3.141592653589793116 2.5403140807248779693e-85 1.570796326794896558
- joint right_hip_yaw: origin xyz=0.0099999999999999897998 -0.034999999999999989453 0.29868541999999997927 rpy=-2.8487879681803368219e-27 -6.1232339957719874427e-17 -3.1415926535897793492 -> xyz=-0.0064000000000000063782 -0.034999999999999996392 0.29859999999999997655 rpy=-4.0795765885139752246e-16 -1.4246408104590497614e-16 -3.1415926535897877869
- joint right_sho_pitch: origin xyz=0.0099999999999999932693 -0.06050000000000008149 0.43008541999999999605 rpy=-1.570796326794896336 6.9606380272961593273e-16 1.3836137928249486855e-31 -> xyz=-0.0064000000000000063782 -0.06050000000000008149 0.42999999999999993783 rpy=-1.570796326794896336 6.9606380272961593273e-16 1.3836137928249486855e-31
