Commit message: Update CoM

File: toddlerbot/robot_descriptions/assemblies/4R_body/4R_body.urdf (robot description, URDF)
Before this commit: robot 4R_body, 8 links, 7 joints
Links:
- link body_link: mass 0.67608257475273170201 -> 0.67608257475273103587
- link right_3r+rh5_leg: mass 0.31997833387465629551 -> 0.31997833387465624
Joints:
- joint left_hip_yaw: origin xyz=-0.0064000000000000055109 0.034999999999999982514 0.29859999999999997655 rpy=2.5294987785272742576e-29 -6.1232339957503159545e-17 3.1415926535897900074 -> xyz=-0.0064000000000000063782 0.034999999999999989453 0.29849999999999998757 rpy=3.2485353740361531821e-29 -6.1232339957386420457e-17 3.1415926535897265026
- joint left_sho_pitch: origin xyz=-0.0064000000000001572992 0.060499999999999110045 0.42999999999999988232 rpy=-1.5707963267948708008 3.5465916442993729594e-14 -3.1415926535897371608 -> xyz=-0.0064000000000001572992 0.060499999999999103106 0.42989999999999989333 rpy=-1.5707963267948708008 3.5465916442993729594e-14 -3.1415926535897371608
- joint neck: origin xyz=-0.0063999999999999925004 -7.4035645855646046943e-18 0.4500000000000000111 rpy=-3.141592653589793116 2.5403140807248779693e-85 1.570796326794896558 -> xyz=-0.0063999999999999925004 -7.4035645855646046943e-18 0.44990000000000002212 rpy=-3.141592653589793116 2.5403140807248779693e-85 1.570796326794896558
- joint right_hip_yaw: origin xyz=-0.0064000000000000063782 -0.034999999999999996392 0.29859999999999997655 rpy=-4.0795765885139752246e-16 -1.4246408104590497614e-16 -3.1415926535897877869 -> xyz=-0.0064000000000000063782 -0.035000000000000003331 0.29849999999999998757 rpy=2.7148356055467616192e-15 4.7934048230446615859e-16 3.1415926535897602534
- joint right_sho_pitch: origin xyz=-0.0064000000000000063782 -0.06050000000000008149 0.42999999999999993783 rpy=-1.570796326794896336 6.9606380272961593273e-16 1.3836137928249486855e-31 -> xyz=-0.0064000000000000063782 -0.06050000000000008149 0.42989999999999994884 rpy=-1.570796326794896336 6.9606380272961593273e-16 1.3836137928249486855e-31

File: toddlerbot/robot_descriptions/assemblies/left_3R+RH5_leg/left_3R+RH5_leg.urdf (robot description, URDF)
Before this commit: robot left_3R+RH5_leg, 20 links, 19 joints
Links:
- link ank_act_link: mass 0.044782197690790455369 -> 0.044782197696050352054
- link ank_act_link_2: mass 0.04478219769079044843 -> 0.044782197696050345115
- link ank_act_link_head: mass 0.003051771492579283783 -> 0.0030517714925792842166
- link ank_act_link_head_2: mass 0.003051771492579283783 -> 0.0030517714925792842166
- link ank_act_rod: mass 0.0026945559868381376359 -> 0.0026945559868381372022
- link ank_act_rod_2: mass 0.0026945559868381376359 -> 0.0026945559868381372022
- link ank_roll_link: mass 0.0054237955467263112772 -> 0.0054237955467263104098
- link ank_rr_link: mass 0.00047585137324286072612 -> 0.0004758513732428606177
- link ank_rr_link_2: mass 0.00047585137324286072612 -> 0.0004758513732428606177
- link hip_yaw_link: mass 0.0052740645607467486963 -> 0.0052740645607467495637
- link knee_link: mass 0.0043868974356887722316 -> 0.0043868974356887713642
- link left_ank_base_link: mass 0.014262086197619729816 -> 0.014262086197619733285

File: toddlerbot/robot_descriptions/assemblies/right_3R+RH5_leg/right_3R+RH5_leg.urdf (robot description, URDF)
Before this commit: robot right_3R+RH5_leg, 20 links, 19 joints
Links:
- link ank_act_link: mass 0.044782197690790462308 -> 0.044782197696050365932
- link ank_act_link_2: mass 0.044782197690790455369 -> 0.044782197696050352054
- link ank_act_link_head: mass 0.003051771492579283783 -> 0.0030517714925792842166
- link ank_act_link_head_2: mass 0.003051771492579283783 -> 0.0030517714925792842166
- link ank_act_rod: mass 0.0026945559868381376359 -> 0.0026945559868381372022
- link ank_act_rod_2: mass 0.0026945559868381376359 -> 0.0026945559868381372022
- link ank_roll_link: mass 0.0054237955467263112772 -> 0.0054237955467263104098
- link ank_rr_link: mass 0.00047585137324286072612 -> 0.0004758513732428606177
- link ank_rr_link_2: mass 0.00047585137324286072612 -> 0.0004758513732428606177
- link hip_yaw_link: mass 0.0052740645607467486963 -> 0.0052740645607467495637
- link knee_link: mass 0.0043868974356887722316 -> 0.0043868974356887713642
- link right_ank_base_link: mass 0.014262085602793538042 -> 0.014262085602793541511
Joints:
- joint right_ank_B11: origin xyz=0.019999999999999990008 -0.010000000000000064393 -0.011500000000000110828 rpy=-1.5707963267949649477 -1.498548410559401356 1.570796326794752229 -> xyz=0.020000000000000000416 -0.0099999999999999811262 -0.011499999999999996336 rpy=-1.570796326794896558 -1.4985484105594246707 1.5707963267948987784
- joint right_ank_B12: origin xyz=0.018680019623525341566 -0.010000000000000314193 0.023400000000000680672 rpy=1.5707963267949003328 1.5020090633896872045 1.5707963267948876762 -> xyz=0.018680019623525345035 -0.010000000000000203171 0.023400000000000038824 rpy=1.570796326794896558 1.5020090633896898691 1.5707963267948452657
- joint right_ank_B21: origin xyz=0.00450000000000061115 -5.5511151231257827021e-17 -0.016999999999999966527 rpy=-1.5707963267952360642 -1.567667016813194536 -1.5707963267890037162 -> xyz=0.0045000000000000005274 -2.7755575615628913511e-17 -0.017000000000000001221 rpy=-1.5707963267940137086 -1.5676670168132000871 -1.5707963267958193754
- joint right_ank_B22: origin xyz=0.0045000000000000144051 8.3266726846886740532e-17 0.01700000000000001163 rpy=-1.5707963267949425212 1.5534346511595631402 -1.5707963267948024111 -> xyz=0.0045000000000000005274 0 0.017000000000000001221 rpy=-1.5707963267948961139 1.5534346511595535922 -1.5707963267945059815
- joint right_ank_B31: origin xyz=-4.1633363423443370266e-17 0.0060499999999999998224 -0.0043000000000000086764 rpy=1.5707963267948934494 5.4574690957684207369e-06 -1.3977638364514914411e-14 -> xyz=6.9388939039072283776e-18 0.0060499999999999998224 -0.0043000000000000052069 rpy=1.570796326794896558 5.4574690831719151044e-06 -5.3684158344603204677e-16
- joint right_ank_B32: origin xyz=1.3877787807814456755e-17 -0.0060499999999998332889 -0.0043000000000000607181 rpy=-1.5707963267948961139 -5.45746960946283069e-06 6.9689783799507381887e-15 -> xyz=1.3877787807814456755e-17 -0.0060499999999999998224 -0.0043000000000000017375 rpy=-1.5707963267948992225 -5.457469620238887183e-06 7.9371251948125348319e-15
- joint right_ank_R11: origin xyz=0.0099999999999999429623 -0.012500000000000066613 0.040600000000000337208 rpy=-2.5476914750798164726e-15 -8.1100273852236014827e-16 3.0693447373540605483 -> xyz=0.010000000000000001943 -0.012500000000000011102 0.040600000000000004141 rpy=-1.6768084170781386496e-16 1.6793651800265835693e-16 3.0693447373540627687
- joint right_ank_R12: origin xyz=-0.0099999999999999516359 -0.012499999999999955591 0.040600000000000358025 rpy=-1.2454338751916450574e-14 5.795879650126974938e-15 0.068787263405096929492 -> xyz=-0.0099999999999999967387 -0.012500000000000066613 0.040600000000000004141 rpy=9.9988103143397809154e-17 -2.0967218556959505843e-16 0.068787263405097776037
- joint right_ank_R21: origin xyz=0.001999999999999991368 -0.010000000000000008882 -0.0019000000000000336065 rpy=-1.5707963267950324493 -1.5676670168133113314 -1.5707963267951672304 -> xyz=0.0019999999999999948375 -0.010000000000000008882 -0.001899999999999998912 rpy=-1.5707963267948978903 -1.5676670168133413075 -1.5707963267948421571
- joint right_ank_R22: origin xyz=0.0019999999999999844291 0.0099999999999997868372 -0.0019000000000000058509 rpy=-1.5707963267949827113 1.5534346511596899276 -1.570796326794722253 -> xyz=0.0019999999999999983069 0.010000000000000008882 -0.0018999999999999919731 rpy=-1.57079632679489678 1.5534346511597141305 -1.5707963267948845676
- joint right_ank_act1: origin xyz=2.2722093397584131047e-06 -2.7616797737550768943e-15 -0.059245818700238817023 rpy=-3.141592653589793116 7.8730370890791872833e-17 -0.63671356442004978238 -> xyz=2.272209339737596423e-06 -2.7408630920433552092e-15 -0.0592458187002377068 rpy=-3.141592653589793116 1.1304262253414882217e-15 -0.63671356442004933829
- joint right_ank_act2: origin xyz=2.2722093444768609594e-06 1.4190038033490282032e-15 -0.059208011505612251346 rpy=-3.1415926535897846783 -1.2262068103869690541e-14 -0.6367135644198562705 -> xyz=2.2722093445462498984e-06 1.4675760606763788019e-15 -0.059208011505609670078 rpy=-3.1415926535897837901 -1.2381997508906741431e-14 -0.63671356441984272578
- joint right_ank_base: origin xyz=3.9968028886505635455e-15 5.1347814888913489995e-16 -0.0064999999999950722196 rpy=1.2818767136087556972e-13 -6.6450035636680710077e-14 1.0471975511965969652 -> xyz=3.9968028886505635455e-15 4.9960036108132044319e-16 -0.0064999999999950843627 rpy=1.318134964783001977e-13 -6.6907839384880761199e-14 1.0471975511965974093
- joint right_ank_foot: origin xyz=1.3877787807814456755e-17 -0.022500000000000131006 0.025600000000000136535 rpy=-1.570796326794896558 -1.570796326794896558 0 -> xyz=2.6020852139652106416e-18 -0.022500000000000019984 0.025600000000000008166 rpy=-1.5707963267948936714 -1.570796326794896558 0
- joint right_ank_pitch: origin xyz=-1.357934238180394094e-16 -0.10000000000000008882 0.020900000000000668043 rpy=7.2118786468278761141e-15 -7.4293869667367865081e-15 1.5707963267948599206 -> xyz=6.1700474640187238976e-18 -0.10000000000000003331 0.020900000000000050482 rpy=2.1524613638062562596e-14 -2.3065317017433820093e-14 1.570796326794886566
- joint right_ank_roll: origin xyz=5.5511151231257827021e-17 0.0014999999999999475558 -0.014600000000000026151 rpy=1.5707963267948925612 1.5707963267948934494 0 -> xyz=-5.5511151231257827021e-17 0.0014999999999999768293 -0.014599999999999951558 rpy=1.5707963267948819031 1.5707963267948903408 0
- joint right_hip_pitch: origin xyz=-0.024000000716142506907 -0.019000000152458108166 -0.019000000152452390517 rpy=-1.5707963267945823649 -1.570796326794816844 0 -> xyz=-0.024000000716144390817 -0.019000000152457414276 -0.019000000152450624569 rpy=-1.5707963267951599029 1.570796326794861697 0
- joint right_hip_roll: origin xyz=0.018999999999999829525 -1.2563796310537849955e-17 -0.027499999999999951567 rpy=3.1415926535897926719 -1.570796326794896558 0 -> xyz=-0.018999999999999881567 -8.4133799350138936069e-18 -0.0274999999999999932 rpy=7.2939485982875388073e-31 -1.5707963267948756858 0
- joint right_knee: origin xyz=-1.5911557041301218853e-16 -0.10750000000000003997 0.016499999999999702405 rpy=-1.7587631597966056551e-15 -9.4692391792157564628e-16 -1.0471975511964521921 -> xyz=-7.1206608387014969571e-17 0.10750000000000017875 0.021499999999999321737 rpy=3.141592653589788231 2.2515415620049152478e-15 1.0471975511964732863

File: toddlerbot/robot_descriptions/base/base.urdf (robot description, URDF)
Before this commit: robot base, 50 links, 49 joints
Links:
- link ank_act_link: mass 0.044782197690790455369 -> 0.044782197696050352054
- link ank_act_link_2: mass 0.04478219769079044843 -> 0.044782197696050345115
- link ank_act_link_3: mass 0.044782197690790462308 -> 0.044782197696050365932
- link ank_act_link_4: mass 0.044782197690790455369 -> 0.044782197696050352054
- link ank_act_link_head: mass 0.003051771492579283783 -> 0.0030517714925792842166
- link ank_act_link_head_2: mass 0.003051771492579283783 -> 0.0030517714925792842166
- link ank_act_link_head_3: mass 0.003051771492579283783 -> 0.0030517714925792842166
- link ank_act_link_head_4: mass 0.003051771492579283783 -> 0.0030517714925792842166
- link ank_act_rod: mass 0.0026945559868381376359 -> 0.0026945559868381372022
- link ank_act_rod_2: mass 0.0026945559868381376359 -> 0.0026945559868381372022
- link ank_act_rod_3: mass 0.0026945559868381376359 -> 0.0026945559868381372022
- link ank_act_rod_4: mass 0.0026945559868381376359 -> 0.0026945559868381372022
- link ank_roll_link: mass 0.0054237955467263112772 -> 0.0054237955467263104098
- link ank_roll_link_2: mass 0.0054237955467263112772 -> 0.0054237955467263104098
- link ank_rr_link: mass 0.00047585137324286072612 -> 0.0004758513732428606177
- link ank_rr_link_2: mass 0.00047585137324286072612 -> 0.0004758513732428606177
- link ank_rr_link_3: mass 0.00047585137324286072612 -> 0.0004758513732428606177
- link ank_rr_link_4: mass 0.00047585137324286072612 -> 0.0004758513732428606177
- link body_link: mass 0.67608257475273170201 -> 0.67608257475273103587
- link hip_yaw_link: mass 0.0052740645607467486963 -> 0.0052740645607467495637
- link hip_yaw_link_2: mass 0.0052740645607467486963 -> 0.0052740645607467495637
- link knee_link: mass 0.0043868974356887722316 -> 0.0043868974356887713642
- link knee_link_2: mass 0.0043868974356887722316 -> 0.0043868974356887713642
- link left_ank_base_link: mass 0.014262086197619729816 -> 0.014262086197619733285
- link right_ank_base_link: mass 0.014262085602793538042 -> 0.014262085602793541511
Joints:
- joint left_hip_yaw: origin xyz=-0.0064000000000000055109 0.034999999999999982514 0.29859999999999997655 rpy=2.5294987785272742576e-29 -6.1232339957503159545e-17 3.1415926535897900074 -> xyz=-0.0064000000000000063782 0.034999999999999989453 0.29849999999999998757 rpy=3.2485353740361531821e-29 -6.1232339957386420457e-17 3.1415926535897265026
- joint left_sho_pitch: origin xyz=-0.0064000000000001572992 0.060499999999999110045 0.42999999999999988232 rpy=-1.5707963267948708008 3.5465916442993729594e-14 -3.1415926535897371608 -> xyz=-0.0064000000000001572992 0.060499999999999103106 0.42989999999999989333 rpy=-1.5707963267948708008 3.5465916442993729594e-14 -3.1415926535897371608
- joint neck: origin xyz=-0.0063999999999999925004 -7.4035645855646046943e-18 0.4500000000000000111 rpy=-3.141592653589793116 2.5403140807248779693e-85 1.570796326794896558 -> xyz=-0.0063999999999999925004 -7.4035645855646046943e-18 0.44990000000000002212 rpy=-3.141592653589793116 2.5403140807248779693e-85 1.570796326794896558
- joint right_ank_B11: origin xyz=0.019999999999999990008 -0.010000000000000064393 -0.011500000000000110828 rpy=-1.5707963267949649477 -1.498548410559401356 1.570796326794752229 -> xyz=0.020000000000000000416 -0.0099999999999999811262 -0.011499999999999996336 rpy=-1.570796326794896558 -1.4985484105594246707 1.5707963267948987784
- joint right_ank_B12: origin xyz=0.018680019623525341566 -0.010000000000000314193 0.023400000000000680672 rpy=1.5707963267949003328 1.5020090633896872045 1.5707963267948876762 -> xyz=0.018680019623525345035 -0.010000000000000203171 0.023400000000000038824 rpy=1.570796326794896558 1.5020090633896898691 1.5707963267948452657
- joint right_ank_B21: origin xyz=0.00450000000000061115 -5.5511151231257827021e-17 -0.016999999999999966527 rpy=-1.5707963267952360642 -1.567667016813194536 -1.5707963267890037162 -> xyz=0.0045000000000000005274 -2.7755575615628913511e-17 -0.017000000000000001221 rpy=-1.5707963267940137086 -1.5676670168132000871 -1.5707963267958193754
- joint right_ank_B22: origin xyz=0.0045000000000000144051 8.3266726846886740532e-17 0.01700000000000001163 rpy=-1.5707963267949425212 1.5534346511595631402 -1.5707963267948024111 -> xyz=0.0045000000000000005274 0 0.017000000000000001221 rpy=-1.5707963267948961139 1.5534346511595535922 -1.5707963267945059815
- joint right_ank_B31: origin xyz=-4.1633363423443370266e-17 0.0060499999999999998224 -0.0043000000000000086764 rpy=1.5707963267948934494 5.4574690957684207369e-06 -1.3977638364514914411e-14 -> xyz=6.9388939039072283776e-18 0.0060499999999999998224 -0.0043000000000000052069 rpy=1.570796326794896558 5.4574690831719151044e-06 -5.3684158344603204677e-16
- joint right_ank_B32: origin xyz=1.3877787807814456755e-17 -0.0060499999999998332889 -0.0043000000000000607181 rpy=-1.5707963267948961139 -5.45746960946283069e-06 6.9689783799507381887e-15 -> xyz=1.3877787807814456755e-17 -0.0060499999999999998224 -0.0043000000000000017375 rpy=-1.5707963267948992225 -5.457469620238887183e-06 7.9371251948125348319e-15
- joint right_ank_R11: origin xyz=0.0099999999999999429623 -0.012500000000000066613 0.040600000000000337208 rpy=-2.5476914750798164726e-15 -8.1100273852236014827e-16 3.0693447373540605483 -> xyz=0.010000000000000001943 -0.012500000000000011102 0.040600000000000004141 rpy=-1.6768084170781386496e-16 1.6793651800265835693e-16 3.0693447373540627687
- joint right_ank_R12: origin xyz=-0.0099999999999999516359 -0.012499999999999955591 0.040600000000000358025 rpy=-1.2454338751916450574e-14 5.795879650126974938e-15 0.068787263405096929492 -> xyz=-0.0099999999999999967387 -0.012500000000000066613 0.040600000000000004141 rpy=9.9988103143397809154e-17 -2.0967218556959505843e-16 0.068787263405097776037
- joint right_ank_R21: origin xyz=0.001999999999999991368 -0.010000000000000008882 -0.0019000000000000336065 rpy=-1.5707963267950324493 -1.5676670168133113314 -1.5707963267951672304 -> xyz=0.0019999999999999948375 -0.010000000000000008882 -0.001899999999999998912 rpy=-1.5707963267948978903 -1.5676670168133413075 -1.5707963267948421571
- joint right_ank_R22: origin xyz=0.0019999999999999844291 0.0099999999999997868372 -0.0019000000000000058509 rpy=-1.5707963267949827113 1.5534346511596899276 -1.570796326794722253 -> xyz=0.0019999999999999983069 0.010000000000000008882 -0.0018999999999999919731 rpy=-1.57079632679489678 1.5534346511597141305 -1.5707963267948845676
- joint right_ank_act1: origin xyz=2.2722093397584131047e-06 -2.7616797737550768943e-15 -0.059245818700238817023 rpy=-3.141592653589793116 7.8730370890791872833e-17 -0.63671356442004978238 -> xyz=2.272209339737596423e-06 -2.7408630920433552092e-15 -0.0592458187002377068 rpy=-3.141592653589793116 1.1304262253414882217e-15 -0.63671356442004933829
- joint right_ank_act2: origin xyz=2.2722093444768609594e-06 1.4190038033490282032e-15 -0.059208011505612251346 rpy=-3.1415926535897846783 -1.2262068103869690541e-14 -0.6367135644198562705 -> xyz=2.2722093445462498984e-06 1.4675760606763788019e-15 -0.059208011505609670078 rpy=-3.1415926535897837901 -1.2381997508906741431e-14 -0.63671356441984272578
- joint right_ank_base: origin xyz=3.9968028886505635455e-15 5.1347814888913489995e-16 -0.0064999999999950722196 rpy=1.2818767136087556972e-13 -6.6450035636680710077e-14 1.0471975511965969652 -> xyz=3.9968028886505635455e-15 4.9960036108132044319e-16 -0.0064999999999950843627 rpy=1.318134964783001977e-13 -6.6907839384880761199e-14 1.0471975511965974093
- joint right_ank_foot: origin xyz=1.3877787807814456755e-17 -0.022500000000000131006 0.025600000000000136535 rpy=-1.570796326794896558 -1.570796326794896558 0 -> xyz=2.6020852139652106416e-18 -0.022500000000000019984 0.025600000000000008166 rpy=-1.5707963267948936714 -1.570796326794896558 0
- joint right_ank_pitch: origin xyz=-1.357934238180394094e-16 -0.10000000000000008882 0.020900000000000668043 rpy=7.2118786468278761141e-15 -7.4293869667367865081e-15 1.5707963267948599206 -> xyz=6.1700474640187238976e-18 -0.10000000000000003331 0.020900000000000050482 rpy=2.1524613638062562596e-14 -2.3065317017433820093e-14 1.570796326794886566
- joint right_ank_roll: origin xyz=5.5511151231257827021e-17 0.0014999999999999475558 -0.014600000000000026151 rpy=1.5707963267948925612 1.5707963267948934494 0 -> xyz=-5.5511151231257827021e-17 0.0014999999999999768293 -0.014599999999999951558 rpy=1.5707963267948819031 1.5707963267948903408 0
- joint right_hip_pitch: origin xyz=-0.024000000716142506907 -0.019000000152458108166 -0.019000000152452390517 rpy=-1.5707963267945823649 -1.570796326794816844 0 -> xyz=-0.024000000716144390817 -0.019000000152457414276 -0.019000000152450624569 rpy=-1.5707963267951599029 1.570796326794861697 0
- joint right_hip_roll: origin xyz=0.018999999999999829525 -1.2563796310537849955e-17 -0.027499999999999951567 rpy=3.1415926535897926719 -1.570796326794896558 0 -> xyz=-0.018999999999999881567 -8.4133799350138936069e-18 -0.0274999999999999932 rpy=7.2939485982875388073e-31 -1.5707963267948756858 0
- joint right_hip_yaw: origin xyz=-0.0064000000000000063782 -0.034999999999999996392 0.29859999999999997655 rpy=-4.0795765885139752246e-16 -1.4246408104590497614e-16 -3.1415926535897877869 -> xyz=-0.0064000000000000063782 -0.035000000000000003331 0.29849999999999998757 rpy=2.7148356055467616192e-15 4.7934048230446615859e-16 3.1415926535897602534
- joint right_knee: origin xyz=-1.5911557041301218853e-16 -0.10750000000000003997 0.016499999999999702405 rpy=-1.7587631597966056551e-15 -9.4692391792157564628e-16 -1.0471975511964521921 -> xyz=-7.1206608387014969571e-17 0.10750000000000017875 0.021499999999999321737 rpy=3.141592653589788231 2.2515415620049152478e-15 1.0471975511964732863
- joint right_sho_pitch: origin xyz=-0.0064000000000000063782 -0.06050000000000008149 0.42999999999999993783 rpy=-1.570796326794896336 6.9606380272961593273e-16 1.3836137928249486855e-31 -> xyz=-0.0064000000000000063782 -0.06050000000000008149 0.42989999999999994884 rpy=-1.570796326794896336 6.9606380272961593273e-16 1.3836137928249486855e-31
