Commit message: Update base urdf

File: toddlerbot/robot_descriptions/assemblies/4R_body/4R_body.urdf (robot description, URDF)
Before this commit: robot 4R_body, 8 links, 7 joints
Links:
- link body_link: mass 1.2686663072771011684 -> 1.2686663072771013905
- link neck_link: mass 0.018378317023500283234 -> 0.018378317023500286703
Joints:
- joint left_hip_yaw: origin xyz=-0.0064000000000000124498 0.034999999999999982514 0.28649999999999997691 rpy=-8.5053965662328550408e-17 1.6935781366831981742e-17 -8.5937010830259145108e-14 -> xyz=-0.0064000000000000115824 0.034999999999999524547 0.28649999999999997691 rpy=-8.5053965663345416767e-17 1.6935781366380737897e-17 -6.7749854439787420343e-14
- joint right_hip_yaw: origin xyz=-0.006400000000000010715 -0.035000000000000031086 0.28649999999999997691 rpy=-8.1389120013700943975e-15 -2.6723536065549819767e-15 1.5242755372383673833e-15 -> xyz=-0.0064000000000000115824 -0.035000000000000017208 0.28649999999999997691 rpy=-1.3903812075106529584e-14 -4.1920818891027382935e-15 -1.1753904145936466635e-14

File: toddlerbot/robot_descriptions/assemblies/left_3R+RH5_leg/left_3R+RH5_leg.urdf (robot description, URDF)
Before this commit: robot left_3R+RH5_leg, 18 links, 17 joints
Links:
- link 12lf: mass 0.044782197696050345115 -> 0.044782197696050352054
- link 12lf_2: mass 0.044782197696050352054 -> 0.044782197696050345115
- link ank_rr_link: mass 0.00044289790445047673732 -> 0.00044289790445047684574
- link ank_rr_link_2: mass 0.00044289790445047673732 -> 0.00044289790445047684574
Joints:
- joint left_ank_B11: origin xyz=0.018000000000001722955 -0.010000000000000813793 -0.011500000000001694631 rpy=-1.5707963267952262942 -1.4752931174793157965 1.5707963267952236297 -> xyz=0.017999999999999957007 -0.01000000000000014766 0.028300000000000765515 rpy=-1.5707963267948972241 1.4719660848801743303 1.570796326794891451
- joint left_ank_B12: origin xyz=0.017999999999999995171 -0.0099999999999999811262 0.028299999999999998768 rpy=-1.5707963267948974462 1.4719660848801816577 1.570796326794891451 -> xyz=0.018000000000000002109 -0.010000000000000008882 -0.011499999999999999806 rpy=-1.570796326794896558 -1.4752931174793231239 1.5707963267948954478
- joint left_ank_B21: origin xyz=1.4085954624931673607e-15 6.9388939039072283776e-16 -0.011499999999998275491 rpy=1.5707963267945219688 -1.4871998384670930271 -1.5707963267945244112 -> xyz=7.8409501114151680667e-16 -1.1102230246251565404e-16 -0.011500000000000044909 rpy=1.5707963267948958919 -1.4871995686196806119 1.5707963267948610309
- joint left_ank_B22: origin xyz=0 0 -0.011500000000000003275 rpy=1.5707963267948958919 -1.4871995686196834985 1.5707963267948610309 -> xyz=-6.9388939039072283776e-18 -2.7755575615628913511e-17 -0.011499999999999999806 rpy=1.5707963267948872321 -1.4871998384670954696 -1.5707963267948854558
- joint left_ank_B31: origin xyz=3.4694469519536141888e-18 -0.0064387505004004919051 0 rpy=-1.5707963267948961139 -5.4574687307084241751e-06 -1.3272186503056431179e-15 -> xyz=-3.4694469519536141888e-18 -0.0064387505004004086384 0 rpy=-1.570796326794896558 -5.457469122271992718e-06 -4.1571660558495781323e-16
- joint left_ank_B32: origin xyz=6.9388939039072283776e-18 -0.006438750500400436394 -1.3877787807814456755e-17 rpy=-1.570796326794896558 -5.4574691333731972074e-06 -4.2441869528092810053e-16 -> xyz=3.4694469519536141888e-18 -0.0064387505004004641496 -1.3877787807814456755e-17 rpy=-1.5707963267948961139 -5.457468730707960001e-06 -1.2951865632219856922e-15
- joint left_ank_R11: origin xyz=0.010000000000000001943 0.012500000000000011102 -0.033000000000000015432 rpy=-3.141592653589793116 3.1995102797262784517e-17 -3.0460894442741315302 -> xyz=-0.0099999999999999984734 0.012500000000000011102 -0.033000000000000008493 rpy=3.1415926535897908956 7.3034946203131872804e-17 -0.098830241914560454375
- joint left_ank_R12: origin xyz=-0.010000000000000000208 0.012499999999999955591 -0.033000000000000008493 rpy=3.1415926535897908956 8.7615180526966664581e-17 -0.098830241914561453576 -> xyz=0.010000000000000003678 0.012500000000000066613 -0.033000000000000008493 rpy=-3.141592653589793116 4.6545838516711603543e-17 -3.0460894442741315302
- joint left_ank_R21: origin xyz=0.0021000000000000115796 -0.010000000000000064393 -0.0019000000000000058509 rpy=-1.570796326794896558 -1.4871998384676154981 -1.5707963267949049957 -> xyz=0.0021000000000002752576 0.010000000000000036637 -0.0019000000000000058509 rpy=-1.570796326794896558 1.4871995686199779296 -1.5707963267949018871
- joint left_ank_R22: origin xyz=0.0020999999999999977018 0.010000000000000008882 -0.0019000000000000058509 rpy=-1.570796326794896558 1.4871995686199819264 -1.5707963267949018871 -> xyz=0.0021000000000000115796 -0.010000000000000036637 -0.001899999999999998912 rpy=-1.5707963267950195707 -1.4871998384676159422 -1.5707963267947853137
- joint left_ank_act1: origin xyz=2.2722093409276167275e-06 -1.7208456881689926377e-15 -0.059356459443564629774 rpy=3.141592653589793116 2.4817422405761382149e-15 -0.63671356442004534149 -> xyz=2.272209342117637032e-06 -2.1996293675385913957e-15 -0.059356158967298844331 rpy=-3.141592653589793116 -9.2921664633026457838e-16 -0.63671356442004722886
- joint left_ank_act2: origin xyz=2.2722093421072286912e-06 -2.1926904736346841673e-15 -0.059356158967298594531 rpy=-3.141592653589793116 -1.0178228435009863141e-15 -0.63671356442004711784 -> xyz=2.2722093409414945153e-06 -1.7347234759768070944e-15 -0.05935645944356465753 rpy=3.141592653589793116 2.5208502705617295898e-15 -0.63671356442004545251
- joint left_ank_pitch: origin xyz=3.4706895064806395478e-18 -0.09999999999999995004 -0.0062000000000000006495 rpy=3.141592653589718509 -7.4989609117638464726e-14 -1.5707963267948470421 -> xyz=4.2143614023597344721e-19 -0.09999999999999995004 -0.0062000000000000023842 rpy=3.1415926535897074068 -7.168818208916126976e-14 -1.5707963267948470421
- joint left_ank_roll: origin xyz=3.6082248300317587564e-16 -0.0061000000000003698833 -0.014600000000000702693 rpy=-1.5707963267949007768 -1.5707963267947899766 0 -> xyz=3.3306690738754696213e-16 -0.0061000000000003698833 -0.014600000000000704428 rpy=-1.5707963267949007768 -1.5707963267947875341 0
- joint left_hip_pitch: origin xyz=-0.024000000716140685447 -0.01900000015244484447 -0.019000000152450791102 rpy=-1.5707963267948210628 1.5707963267948126251 0 -> xyz=-0.024000000716140678508 -0.019000000152444841001 -0.019000000152450791102 rpy=-1.5707963267948210628 1.5707963267948126251 0
- joint left_hip_roll: origin xyz=0.019000000000000343003 5.6514465577048143112e-16 -0.02500000000000024078 rpy=3.141592653589793116 -1.5707963267948910069 0 -> xyz=0.019000000000000304839 -5.0328333128562291641e-18 -0.025000000000000268535 rpy=3.141592653589793116 -1.5707963267948947816 0
- joint left_knee: origin xyz=-4.6852077649545464941e-15 0.098000000000000059286 0.02740000000000222119 rpy=-3.1415926535897620298 -6.1069889650930221337e-15 -6.2009129724835898343e-14 -> xyz=-4.686453338044572818e-15 0.097999999999999976019 0.027400000000003393863 rpy=-3.1415926535897620298 -6.106988965093026078e-15 -6.2039230811899877997e-14

File: toddlerbot/robot_descriptions/assemblies/right_3R+RH5_leg/right_3R+RH5_leg.urdf (robot description, URDF)
Before this commit: robot right_3R+RH5_leg, 18 links, 17 joints
Links:
- link ank_rr_link: mass 0.00044289790445047673732 -> 0.00044289790445047684574
- link ank_rr_link_2: mass 0.00044289790445047673732 -> 0.00044289790445047684574
- link right_calf_link: mass 0.016572091442033143327 -> 0.016572091442033146796

File: toddlerbot/robot_descriptions/base/base.urdf (robot description, URDF)
Before this commit: robot base, 46 links, 45 joints
Links:
- link 12lf: mass 0.044782197696050345115 -> 0.044782197696050352054
- link 12lf_2: mass 0.044782197696050352054 -> 0.044782197696050345115
- link ank_rr_link: mass 0.00044289790445047673732 -> 0.00044289790445047684574
- link ank_rr_link_2: mass 0.00044289790445047673732 -> 0.00044289790445047684574
- link ank_rr_link_3: mass 0.00044289790445047673732 -> 0.00044289790445047684574
- link ank_rr_link_4: mass 0.00044289790445047673732 -> 0.00044289790445047684574
- link body_link: mass 1.2686663072771011684 -> 1.2686663072771013905
- link neck_link: mass 0.018378317023500283234 -> 0.018378317023500286703
- link right_calf_link: mass 0.016572091442033143327 -> 0.016572091442033146796
Joints:
- joint left_ank_B11: origin xyz=0.018000000000001722955 -0.010000000000000813793 -0.011500000000001694631 rpy=-1.5707963267952262942 -1.4752931174793157965 1.5707963267952236297 -> xyz=0.017999999999999957007 -0.01000000000000014766 0.028300000000000765515 rpy=-1.5707963267948972241 1.4719660848801743303 1.570796326794891451
- joint left_ank_B12: origin xyz=0.017999999999999995171 -0.0099999999999999811262 0.028299999999999998768 rpy=-1.5707963267948974462 1.4719660848801816577 1.570796326794891451 -> xyz=0.018000000000000002109 -0.010000000000000008882 -0.011499999999999999806 rpy=-1.570796326794896558 -1.4752931174793231239 1.5707963267948954478
- joint left_ank_B21: origin xyz=1.4085954624931673607e-15 6.9388939039072283776e-16 -0.011499999999998275491 rpy=1.5707963267945219688 -1.4871998384670930271 -1.5707963267945244112 -> xyz=7.8409501114151680667e-16 -1.1102230246251565404e-16 -0.011500000000000044909 rpy=1.5707963267948958919 -1.4871995686196806119 1.5707963267948610309
- joint left_ank_B22: origin xyz=0 0 -0.011500000000000003275 rpy=1.5707963267948958919 -1.4871995686196834985 1.5707963267948610309 -> xyz=-6.9388939039072283776e-18 -2.7755575615628913511e-17 -0.011499999999999999806 rpy=1.5707963267948872321 -1.4871998384670954696 -1.5707963267948854558
- joint left_ank_B31: origin xyz=3.4694469519536141888e-18 -0.0064387505004004919051 0 rpy=-1.5707963267948961139 -5.4574687307084241751e-06 -1.3272186503056431179e-15 -> xyz=-3.4694469519536141888e-18 -0.0064387505004004086384 0 rpy=-1.570796326794896558 -5.457469122271992718e-06 -4.1571660558495781323e-16
- joint left_ank_B32: origin xyz=6.9388939039072283776e-18 -0.006438750500400436394 -1.3877787807814456755e-17 rpy=-1.570796326794896558 -5.4574691333731972074e-06 -4.2441869528092810053e-16 -> xyz=3.4694469519536141888e-18 -0.0064387505004004641496 -1.3877787807814456755e-17 rpy=-1.5707963267948961139 -5.457468730707960001e-06 -1.2951865632219856922e-15
- joint left_ank_R11: origin xyz=0.010000000000000001943 0.012500000000000011102 -0.033000000000000015432 rpy=-3.141592653589793116 3.1995102797262784517e-17 -3.0460894442741315302 -> xyz=-0.0099999999999999984734 0.012500000000000011102 -0.033000000000000008493 rpy=3.1415926535897908956 7.3034946203131872804e-17 -0.098830241914560454375
- joint left_ank_R12: origin xyz=-0.010000000000000000208 0.012499999999999955591 -0.033000000000000008493 rpy=3.1415926535897908956 8.7615180526966664581e-17 -0.098830241914561453576 -> xyz=0.010000000000000003678 0.012500000000000066613 -0.033000000000000008493 rpy=-3.141592653589793116 4.6545838516711603543e-17 -3.0460894442741315302
- joint left_ank_R21: origin xyz=0.0021000000000000115796 -0.010000000000000064393 -0.0019000000000000058509 rpy=-1.570796326794896558 -1.4871998384676154981 -1.5707963267949049957 -> xyz=0.0021000000000002752576 0.010000000000000036637 -0.0019000000000000058509 rpy=-1.570796326794896558 1.4871995686199779296 -1.5707963267949018871
- joint left_ank_R22: origin xyz=0.0020999999999999977018 0.010000000000000008882 -0.0019000000000000058509 rpy=-1.570796326794896558 1.4871995686199819264 -1.5707963267949018871 -> xyz=0.0021000000000000115796 -0.010000000000000036637 -0.001899999999999998912 rpy=-1.5707963267950195707 -1.4871998384676159422 -1.5707963267947853137
- joint left_ank_act1: origin xyz=2.2722093409276167275e-06 -1.7208456881689926377e-15 -0.059356459443564629774 rpy=3.141592653589793116 2.4817422405761382149e-15 -0.63671356442004534149 -> xyz=2.272209342117637032e-06 -2.1996293675385913957e-15 -0.059356158967298844331 rpy=-3.141592653589793116 -9.2921664633026457838e-16 -0.63671356442004722886
- joint left_ank_act2: origin xyz=2.2722093421072286912e-06 -2.1926904736346841673e-15 -0.059356158967298594531 rpy=-3.141592653589793116 -1.0178228435009863141e-15 -0.63671356442004711784 -> xyz=2.2722093409414945153e-06 -1.7347234759768070944e-15 -0.05935645944356465753 rpy=3.141592653589793116 2.5208502705617295898e-15 -0.63671356442004545251
- joint left_ank_pitch: origin xyz=3.4706895064806395478e-18 -0.09999999999999995004 -0.0062000000000000006495 rpy=3.141592653589718509 -7.4989609117638464726e-14 -1.5707963267948470421 -> xyz=4.2143614023597344721e-19 -0.09999999999999995004 -0.0062000000000000023842 rpy=3.1415926535897074068 -7.168818208916126976e-14 -1.5707963267948470421
- joint left_ank_roll: origin xyz=3.6082248300317587564e-16 -0.0061000000000003698833 -0.014600000000000702693 rpy=-1.5707963267949007768 -1.5707963267947899766 0 -> xyz=3.3306690738754696213e-16 -0.0061000000000003698833 -0.014600000000000704428 rpy=-1.5707963267949007768 -1.5707963267947875341 0
- joint left_hip_pitch: origin xyz=-0.024000000716140685447 -0.01900000015244484447 -0.019000000152450791102 rpy=-1.5707963267948210628 1.5707963267948126251 0 -> xyz=-0.024000000716140678508 -0.019000000152444841001 -0.019000000152450791102 rpy=-1.5707963267948210628 1.5707963267948126251 0
- joint left_hip_roll: origin xyz=0.019000000000000343003 5.6514465577048143112e-16 -0.02500000000000024078 rpy=3.141592653589793116 -1.5707963267948910069 0 -> xyz=0.019000000000000304839 -5.0328333128562291641e-18 -0.025000000000000268535 rpy=3.141592653589793116 -1.5707963267948947816 0
- joint left_hip_yaw: origin xyz=-0.0064000000000000124498 0.034999999999999982514 0.28649999999999997691 rpy=-8.5053965662328550408e-17 1.6935781366831981742e-17 -8.5937010830259145108e-14 -> xyz=-0.0064000000000000115824 0.034999999999999524547 0.28649999999999997691 rpy=-8.5053965663345416767e-17 1.6935781366380737897e-17 -6.7749854439787420343e-14
- joint left_knee: origin xyz=-4.6852077649545464941e-15 0.098000000000000059286 0.02740000000000222119 rpy=-3.1415926535897620298 -6.1069889650930221337e-15 -6.2009129724835898343e-14 -> xyz=-4.686453338044572818e-15 0.097999999999999976019 0.027400000000003393863 rpy=-3.1415926535897620298 -6.106988965093026078e-15 -6.2039230811899877997e-14
- joint right_hip_yaw: origin xyz=-0.006400000000000010715 -0.035000000000000031086 0.28649999999999997691 rpy=-8.1389120013700943975e-15 -2.6723536065549819767e-15 1.5242755372383673833e-15 -> xyz=-0.0064000000000000115824 -0.035000000000000017208 0.28649999999999997691 rpy=-1.3903812075106529584e-14 -4.1920818891027382935e-15 -1.1753904145936466635e-14
