Commit message: Update the base robot

File: toddlerbot/robot_descriptions/assemblies/4R_body/4R_body.urdf (robot description, URDF)
Before this commit: robot 4R_body, 8 links, 7 joints
Links:
- link body_link: mass 1.2686663072771013905 -> 1.3010345634555096073
- link left_3r+rh5_leg: mass 0.32496567630925582426 -> 0.33313077160322585035
- link right_3r+rh5_leg: mass 0.32496567358416811322 -> 0.33284223245696664684
Joints:
- joint left_hip_yaw: origin xyz=-0.0064000000000000115824 0.034999999999999524547 0.28649999999999997691 rpy=-8.5053965663345416767e-17 1.6935781366380737897e-17 -6.7749854439787420343e-14 -> xyz=-0.011900000000000068509 0.033999999999999967748 0.27720000000000005747 rpy=-2.2204460494576350945e-16 2.2204460491537123791e-16 -1.0069344447037368454e-13
- joint right_hip_yaw: origin xyz=-0.0064000000000000115824 -0.035000000000000017208 0.28649999999999997691 rpy=-1.3903812075106529584e-14 -4.1920818891027382935e-15 -1.1753904145936466635e-14 -> xyz=-0.011900000000000259329 -0.033999999999999974687 0.27720000000000000195 rpy=-2.2204460561717224569e-16 2.2204460926237942003e-16 -6.0840221749459209504e-14
- joint right_sho_pitch: origin xyz=-0.0064000000000000167866 -0.057999999999999982125 0.4124999999999999778 rpy=-1.570796326794896558 1.3877787807814444922e-15 8.1990370565314014207e-16 -> xyz=-0.0063999999999999916331 -0.057999999999999989064 0.4124999999999999778 rpy=-1.5707963267948972241 1.3877787807856806753e-15 6.3545304591998415249e-17

File: toddlerbot/robot_descriptions/assemblies/left_3R+RH5_leg/left_3R+RH5_leg.urdf (robot description, URDF)
Before this commit: robot left_3R+RH5_leg, 18 links, 17 joints
Links:
- link ank_roll_link: mass 0.013844478784760253648 -> 0.013844478784760250178
- link ank_rr_link: mass 0.00044289790445047673732 -> 0.00044289790445047668311
- link ank_rr_link_2: mass 0.00044289790445047673732 -> 0.00044289790445047668311
- link hip_yaw_link: mass 0.009025883737097921064 -> 0.0090258837370979193293
- link left_calf_link: mass 0.016616268752102307527 -> 0.016579149141633314074
Joints:
- joint left_ank_B11: origin xyz=0.0079999999999999966971 -0.015000000000000179856 0.028300000000000005707 rpy=-1.570796326794896558 1.4686290291020840382 1.5707963267948819031 -> xyz=0.008000000000000053943 -0.014999999999999985567 0.028299999999999915501 rpy=-1.57079632679489678 1.4696360140379260972 1.5707963267948892305
- joint left_ank_B12: origin xyz=0.008000000000000003636 -0.015000000000000124345 -0.01149999999999918622 rpy=-1.570796326794896558 -1.4687304067506412597 1.5707963267949098807 -> xyz=0.0080000000000000504735 -0.014999999999999930056 -0.011500000000000076134 rpy=-1.5707963267948958919 -1.4697566621822790722 1.5707963267948983344
- joint left_ank_B21: origin xyz=6.9388939039072283776e-18 -2.7755575615628913511e-17 -0.011499999999999994602 rpy=1.57079632679489678 -1.4274634743672511838 1.570796326794916542 -> xyz=0 0 -0.011499999999999996336 rpy=1.570796326794896558 -1.4285697747625092369 1.5707963267948912289
- joint left_ank_B22: origin xyz=-1.3877787807814456755e-17 8.3266726846886740532e-17 -0.011500000000000011949 rpy=1.570796326794896558 -1.4274430275990750427 -1.570796326794906328 -> xyz=-6.9388939039072283776e-18 -8.3266726846886740532e-17 -0.011499999999999996336 rpy=1.5707963267948961139 -1.4285463212680367118 -1.5707963267948970021
- joint left_ank_B31: origin xyz=-1.4831885719601700657e-16 -0.0064387505004003253717 -6.9388939039072283776e-18 rpy=-1.570796326794896558 0.16912328473440299548 -4.2800865129067981483e-15 -> xyz=-3.4694469519536141888e-18 -0.0064387505004004086384 -6.9388939039072283776e-18 rpy=-1.570796326794896558 0.16913440034103149889 1.5363542389808260585e-15
- joint left_ank_B32: origin xyz=1.7347234759768070944e-17 -0.0064387505004004641496 1.3877787807814456755e-17 rpy=-1.5707963267948836794 -0.17992034540981183266 -3.9922693705457534994e-15 -> xyz=1.9949319973733281586e-17 -0.0064387505004002698605 1.3877787807814456755e-17 rpy=-1.5707963267948970021 -0.17993145005780439294 -1.804382386805444098e-17
- joint left_ank_R11: origin xyz=-0.010000000000000000208 0.012499999999999955591 -0.028000000000000004052 rpy=3.1415926535897775729 -1.1742161333363301013e-15 -0.10225158937860563679 -> xyz=-0.01000000000000001929 0.012500000000000011102 -0.027899999999999692407 rpy=-3.141592653589793116 3.5006616330671580104e-18 -0.10116031275702692949
- joint left_ank_R12: origin xyz=0.010000000000000001943 0.01249999999999990008 -0.027999999999999948541 rpy=3.1415926535897895633 4.4319359555376638558e-15 -3.0396078498296592585 -> xyz=0.0099999999999999932693 0.012500000000000066613 -0.027900000000000039352 rpy=3.1415926535897904515 2.6926878995557896255e-15 -3.0405529889787885622
- joint left_ank_R21: origin xyz=0.0021000000000000115796 0.010000000000000064393 -0.0018999999999999919731 rpy=-1.570796326794896558 1.4273561685593663118 -1.5707963267949194286 -> xyz=0 0.010000000000000036637 -0.001899999999999998912 rpy=1.570796326794896558 1.428569774762729061 -1.570796326794896558
- joint left_ank_R22: origin xyz=0.0021000000000000115796 -0.010000000000000092149 -0.001899999999999929523 rpy=-1.5707963267948974462 -1.4273357206756709381 -1.5707963267949238695 -> xyz=1.3877787807814456755e-17 -0.010000000000000036637 -0.0019000000000000058509 rpy=1.5707963267949061059 -1.4285463212675062472 -1.5707963267949052177
- joint left_ank_act1: origin xyz=2.272209354975407436e-06 9.4368957093138305936e-16 -0.072676675805820711851 rpy=-3.1415926535896590011 9.257153768608790258e-14 -2.2021168238262611716 -> xyz=2.2722093542849874925e-06 9.5062846483529028774e-16 -0.072660031604104974301 rpy=-3.1415926535896594451 8.6956799327801851499e-14 -2.2021168238262722738
- joint left_ank_act2: origin xyz=2.2722093495249062745e-06 -6.7446048745978259831e-15 -0.072678522047017385388 rpy=-3.1415926535895004612 6.2111251208581937571e-14 -2.2021168238262802674 -> xyz=2.2722093491103073637e-06 -6.5433769513845163601e-15 -0.072660030478827297706 rpy=-3.1415926535895009053 6.1538805987964111831e-14 -2.2021168238262798234
- joint left_ank_pitch: origin xyz=1.6466858937503582328e-18 -0.099999999999999922284 -0.0062000000000000058537 rpy=-3.1415926535897842342 8.6597368124280298137e-15 -1.5709041950953850364 -> xyz=1.0842022241842927186e-18 -0.10000000000000006106 -0.0061999999999999867717 rpy=-3.141592653589793116 -1.9981846038921943663e-15 -1.570796326794896558
- joint left_ank_roll: origin xyz=3.3306690738754696213e-16 -0.0060999999999999726316 -0.014599999999999384304 rpy=-1.5707963257530275225 -1.5707136234809810915 -1.1504969698363094907e-09 -> xyz=1.193489751472043281e-15 -0.00610000000000079836 -0.014600000000000288095 rpy=-1.5707963267948288344 -1.5707963267944542451 0
- joint left_hip_pitch: origin xyz=-0.024000000716150875213 -0.01900000015244158319 -0.019000000152448091872 rpy=-1.5707963267945472818 1.5707963267948001906 0 -> xyz=-0.02400000071615384506 -0.019000000152441031548 -0.019000000152448098811 rpy=-1.570796326794478226 1.5707963267948008568 0
- joint left_hip_roll: origin xyz=0.019000000000000304839 -3.3605706708588417072e-18 -0.026000000000000279832 rpy=1.5707963267908973126 -1.5707806634981131833 1.5707963268130720191 -> xyz=0.019000000000000273614 -2.891526265917987331e-16 -0.026000000000000279832 rpy=-3.141592653589793116 -1.5707963267945983521 0
- joint left_knee: origin xyz=-3.1366467205128203278e-15 0.095999999999999752198 0.027400000000000007683 rpy=-3.1415926535897926719 -2.5420496490693392505e-17 -8.4866560936749634e-15 -> xyz=-6.5714384231211065113e-15 0.09599999999999973832 0.027400000000000167277 rpy=-3.1415926535897891192 1.5325113271907731669e-16 -5.5621661637730288381e-17

File: toddlerbot/robot_descriptions/assemblies/left_OP3_arm/left_OP3_arm.urdf (robot description, URDF)
Before this commit: robot left_OP3_arm, 3 links, 2 joints
Links:
- link elb_link: mass 0.012147845014428806237 -> 0.012147845014428809707
- link sho_pitch_link: mass 0.0053168741776095278587 -> 0.0053168741776095304608

File: toddlerbot/robot_descriptions/assemblies/right_3R+RH5_leg/right_3R+RH5_leg.urdf (robot description, URDF)
Before this commit: robot right_3R+RH5_leg, 18 links, 17 joints
Links:
- link ank_roll_link: mass 0.013844478784760253648 -> 0.013844478784760250178
- link ank_rr_link: mass 0.00044289790445047673732 -> 0.00044289790445047668311
- link ank_rr_link_2: mass 0.00044289790445047673732 -> 0.00044289790445047668311
- link hip_yaw_link: mass 0.009025883737097921064 -> 0.0090258837370979193293
- link right_calf_link: mass 0.016616299594005391055 -> 0.016290630569901022595
Joints:
- joint right_ank_B11: origin xyz=0.007999999999999972411 0.014999999999999957812 -0.011500000000000010214 rpy=1.5707963267948978903 -1.4686162729650020786 -1.5707963267948970021 -> xyz=0.0080000000000000001665 0.015000000000000041078 -0.011499999999999994602 rpy=1.570796326794896558 -1.469636014037949634 -1.5707963267948781283
- joint right_ank_B12: origin xyz=0.0079999999999997000594 0.015000000000000290878 0.02830000000000029714 rpy=-1.5707963267948978903 -1.468735614201923223 1.5707963267949029973 -> xyz=0.0080000000000000088402 0.015000000000000068834 0.02829999999999998489 rpy=-1.5707963267948383823 -1.4697566621827073963 1.5707963267948992225
- joint right_ank_B21: origin xyz=-2.0816681711721685133e-17 1.1102230246251565404e-16 -0.011499999999999998071 rpy=1.570796326794896558 -1.4274562579810237128 1.5707963267948950037 -> xyz=-6.9388939039072283776e-18 0 -0.011500000000000006745 rpy=1.570796326794896558 -1.4285697747625620835 1.5707963267948821251
- joint right_ank_B22: origin xyz=-1.3877787807814456755e-17 -8.3266726846886740532e-17 -0.011499999999999991132 rpy=1.57079632679489678 -1.4274330297239778975 1.5707963267949012209 -> xyz=-6.9388939039072283776e-18 -2.7755575615628913511e-17 -0.011499999999999999806 rpy=1.570796326794896558 -1.4285463212677993461 1.5707963267949389685
- joint right_ank_B31: origin xyz=-1.3010426069826053208e-18 -0.0064387505004002698605 6.9388939039072283776e-18 rpy=-1.570796326794896558 0.16913440034154619829 2.2885625266571218396e-16 -> xyz=1.4745149545802860303e-17 -0.006438750500400436394 0 rpy=-1.5707963267948961139 0.16913440034159002434 1.9223858256087746368e-15
- joint right_ank_B32: origin xyz=-1.5178830414797062076e-17 -0.006438750500400436394 1.3877787807814456755e-17 rpy=-1.5707963267948854558 -0.17993145005756266963 -2.2505490007573420062e-15 -> xyz=5.6378512969246230568e-18 -0.006438750500400436394 0 rpy=-1.570796326794896336 -0.17993145005752267385 1.8689858510975082391e-15
- joint right_ank_R11: origin xyz=-0.0099999999999999932693 0.012500000000000038858 -0.02800000000000008038 rpy=-3.1415926535897926719 -7.9041717877712374794e-16 -0.10218566393336031561 -> xyz=-0.0099999999999999984734 0.012500000000000066613 -0.027900000000000015066 rpy=-3.1415926535897860106 -4.3778626236368231385e-15 -0.10116031275681484913
- joint right_ank_R12: origin xyz=0.0099999999999999967387 0.012499999999999761302 -0.02800000000000008038 rpy=-3.141592653589793116 2.6793361964555018776e-16 -3.0395375511005577884 -> xyz=0.010000000000000000208 0.012500000000000011102 -0.027900000000000001188 rpy=-3.1415926535897829019 -8.8337259752553850467e-15 -3.040552988977761828
- joint right_ank_R21: origin xyz=0.0021000000000000254574 0.010000000000000092149 -0.0018999999999999919731 rpy=-1.57079632679489678 1.4274562579811747032 -1.570796326794901665 -> xyz=0 0.010000000000000092149 -0.0019000000000000058509 rpy=1.570796326794896558 1.4285697747627268406 -1.5707963267948945596
- joint right_ank_R22: origin xyz=0.0021000000000000185185 -0.010000000000000203171 -0.0019000000000000336065 rpy=-1.5707963267948961139 -1.4274330297240631626 -1.5707963267948974462 -> xyz=6.9388939039072283776e-18 -0.010000000000000064393 -0.001899999999999998912 rpy=1.570796326794896558 -1.4285463212679276879 -1.5707963267948938935
- joint right_ank_act1: origin xyz=2.2722093427785666764e-06 1.2698175844150227931e-15 -0.072674150483189009497 rpy=-3.1415926535897811256 9.814572829871540247e-15 -2.2021168238260906413 -> xyz=2.2722093427473416538e-06 1.2559397966072083364e-15 -0.07266003160412204398 rpy=-3.1415926535897895633 9.1629640935489764995e-15 -2.2021168238260711014
- joint right_ank_act2: origin xyz=2.2722093417776312307e-06 -2.3800406090401793335e-15 -0.072674285805652133474 rpy=3.141592653589793116 -4.1997988128928857096e-16 -2.2021168238262838202 -> xyz=2.2722093417394673143e-06 -2.3939183968479937903e-15 -0.072660030478831599821 rpy=3.141592653589793116 -2.0657592427741678223e-15 -2.2021168238262744943
- joint right_ank_pitch: origin xyz=1.1774009739933720541e-18 0.099999999999999922284 -0.0061999999999999937106 rpy=-3.141592653589793116 3.885801455584734555e-16 -1.5707963267948825692 -> xyz=7.5714896865366240827e-19 0.10000000000000003331 -0.00619999999999999718 rpy=-3.141592653589793116 1.998618284759728781e-15 -1.57079632679489678
- joint right_ank_roll: origin xyz=1.7763568394002504647e-15 -0.0061000000000006751946 -0.014600000000001986389 rpy=1.5707963281806591738 1.5707907166914047981 -3.1415926522336965476 -> xyz=2.1926904736346841673e-15 -0.0061000000000001799311 -0.014600000000002237924 rpy=-1.5707963267949249797 1.5707963267947928632 0
- joint right_hip_pitch: origin xyz=-0.024000000716145986762 -0.019000000152457990205 -0.019000000152453774827 rpy=-1.5707963267951818853 1.5707963267947633312 0 -> xyz=-0.024000000716146760449 -0.019000000152456297114 -0.019000000152450020885 rpy=-1.5707963267951789987 1.5707963267947411268 0
- joint right_hip_roll: origin xyz=-0.018999999999999885036 -3.3499987806511678644e-18 -0.026000000000000002276 rpy=-1.5707963266839728433 -1.5707907166912637997 1.5707963266641831179 -> xyz=-0.018999999999999881567 -3.3500438889867783387e-18 -0.026000000000000002276 rpy=3.0518439807331778725e-31 -1.5707963267948181763 0
- joint right_knee: origin xyz=-2.4109230505694711738e-15 0.095999999999999821587 0.027399999999999948702 rpy=3.141592653589793116 -1.6870185802395130185e-16 3.1415926535897922278 -> xyz=-1.8821214288092669642e-15 0.096000000000001001199 0.027399999999998970318 rpy=3.1415926535897220617 -3.0356441407590551802e-14 3.1415926535897846783

File: toddlerbot/robot_descriptions/assemblies/right_OP3_arm/right_OP3_arm.urdf (robot description, URDF)
Before this commit: robot right_OP3_arm, 3 links, 2 joints
Links:
- link elb_link: mass 0.012147845014428806237 -> 0.012147845014428809707
- link sho_pitch_link: mass 0.0053168741776095278587 -> 0.0053168741776095304608
