Commit message: Update the base robot

File: toddlerbot/robot_descriptions/base/base.urdf (robot description, URDF)
Before this commit: robot base, 46 links, 45 joints
Links:
- removed link hip_pitch_link
- removed link hip_pitch_link_2
- added link left_hip_pitch_link, mass 0.094084588454108858402; collision mesh filename=../assemblies/left_3R+RH5_leg/meshes/left_hip_pitch_link_co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; visual mesh filename=../assemblies/left_3R+RH5_leg/meshes/left_hip_pitch_link_vi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
- added link right_hip_pitch_link, mass 0.094084567879581956773; collision mesh filename=../assemblies/right_3R+RH5_leg/meshes/right_hip_pitch_link_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; visual mesh filename=../assemblies/right_3R+RH5_leg/meshes/right_hip_pitch_link_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
- link 12lf_2: mass 0.044782197696050345115 -> 0.044782197696050352054
- link 12lf_3: mass 0.044782197696050345115 -> 0.044782197696050352054
- link 12lf_4: mass 0.044782197696050365932 -> 0.044782197696050358993
- link 12lf_rod: mass 0.0026945559868381376359 -> 0.0025088292483592140175
- link 12lf_rod_2: mass 0.0026945559868381376359 -> 0.0025088292483592140175
- link 12lf_rod_3: mass 0.0026945559868381376359 -> 0.0025088292483592140175
- link 12lf_rod_4: mass 0.0026945559868381376359 -> 0.0025088292483592140175
- link 12lf_rod_end: mass 0.00066080012085386230676 -> 0.00085420491177815905965
- link 12lf_rod_end_2: mass 0.00066080012085386230676 -> 0.00085420491177815905965
- link 12lf_rod_end_3: mass 0.00066080012085386230676 -> 0.00085420491177815905965
- link 12lf_rod_end_4: mass 0.00066080012085386230676 -> 0.00085420491177815905965
- link ank_pitch_link: mass 0.0042238381753791614387 -> 0.0042238381753791605713
- link ank_pitch_link_2: mass 0.0042238381753791614387 -> 0.0042238381753791605713
- link ank_roll_link: mass 0.014299508637166613578 -> 0.013844478784760250178
- link ank_roll_link_2: mass 0.014299508637166613578 -> 0.013844478784760250178
- link ank_rr_link: mass 0.00044289790445047684574 -> 0.00044289790445047668311
- link ank_rr_link_2: mass 0.00044289790445047684574 -> 0.00044289790445047668311
- link ank_rr_link_3: mass 0.00044289790445047684574 -> 0.00044289790445047668311
- link ank_rr_link_4: mass 0.00044289790445047684574 -> 0.00044289790445047668311
- link ball_joint_ball: mass 4.4053796295264623832e-05 -> 4.4053796295264630609e-05
- link ball_joint_ball_2: mass 4.4053796295264623832e-05 -> 4.4053796295264630609e-05
- link ball_joint_ball_3: mass 4.4053796295264623832e-05 -> 4.4053796295264630609e-05
- link ball_joint_ball_4: mass 4.4053796295264623832e-05 -> 4.4053796295264630609e-05
- link body_link: mass 1.2686663072771013905 -> 1.3010345634555096073
- link elb_link: mass 0.012147845014428806237 -> 0.012147845014428809707
- link elb_link_2: mass 0.012147845014428806237 -> 0.012147845014428809707
- link hip_yaw_link: mass 0.0081617461226117064832 -> 0.0090258837370979193293
- link hip_yaw_link_2: mass 0.0081617461226117064832 -> 0.0090258837370979193293
- link left_calf_link: mass 0.016572094167120694774 -> 0.016579149141633314074
- link right_calf_link: mass 0.016572091442033146796 -> 0.016290630569901022595
- link sho_pitch_link: mass 0.0053168741776095278587 -> 0.0053168741776095304608
- link sho_pitch_link_2: mass 0.0053168741776095278587 -> 0.0053168741776095304608
Joints:
- joint left_ank_B11: origin xyz=0.017999999999999957007 -0.01000000000000014766 0.028300000000000765515 rpy=-1.5707963267948972241 1.4719660848801743303 1.570796326794891451 -> xyz=0.008000000000000053943 -0.014999999999999985567 0.028299999999999915501 rpy=-1.57079632679489678 1.4696360140379260972 1.5707963267948892305
- joint left_ank_B12: origin xyz=0.018000000000000002109 -0.010000000000000008882 -0.011499999999999999806 rpy=-1.570796326794896558 -1.4752931174793231239 1.5707963267948954478 -> xyz=0.0080000000000000504735 -0.014999999999999930056 -0.011500000000000076134 rpy=-1.5707963267948958919 -1.4697566621822790722 1.5707963267948983344
- joint left_ank_B21: origin xyz=7.8409501114151680667e-16 -1.1102230246251565404e-16 -0.011500000000000044909 rpy=1.5707963267948958919 -1.4871995686196806119 1.5707963267948610309 -> xyz=0 0 -0.011499999999999996336 rpy=1.570796326794896558 -1.4285697747625092369 1.5707963267948912289
- joint left_ank_B22: origin xyz=-6.9388939039072283776e-18 -2.7755575615628913511e-17 -0.011499999999999999806 rpy=1.5707963267948872321 -1.4871998384670954696 -1.5707963267948854558 -> xyz=-6.9388939039072283776e-18 -8.3266726846886740532e-17 -0.011499999999999996336 rpy=1.5707963267948961139 -1.4285463212680367118 -1.5707963267948970021
- joint left_ank_B31: origin xyz=-3.4694469519536141888e-18 -0.0064387505004004086384 0 rpy=-1.570796326794896558 -5.457469122271992718e-06 -4.1571660558495781323e-16 -> xyz=-3.4694469519536141888e-18 -0.0064387505004004086384 -6.9388939039072283776e-18 rpy=-1.570796326794896558 0.16913440034103149889 1.5363542389808260585e-15
- joint left_ank_B32: origin xyz=3.4694469519536141888e-18 -0.0064387505004004641496 -1.3877787807814456755e-17 rpy=-1.5707963267948961139 -5.457468730707960001e-06 -1.2951865632219856922e-15 -> xyz=1.9949319973733281586e-17 -0.0064387505004002698605 1.3877787807814456755e-17 rpy=-1.5707963267948970021 -0.17993145005780439294 -1.804382386805444098e-17
- joint left_ank_R11: origin xyz=-0.0099999999999999984734 0.012500000000000011102 -0.033000000000000008493 rpy=3.1415926535897908956 7.3034946203131872804e-17 -0.098830241914560454375 -> xyz=-0.01000000000000001929 0.012500000000000011102 -0.027899999999999692407 rpy=-3.141592653589793116 3.5006616330671580104e-18 -0.10116031275702692949
- joint left_ank_R12: origin xyz=0.010000000000000003678 0.012500000000000066613 -0.033000000000000008493 rpy=-3.141592653589793116 4.6545838516711603543e-17 -3.0460894442741315302 -> xyz=0.0099999999999999932693 0.012500000000000066613 -0.027900000000000039352 rpy=3.1415926535897904515 2.6926878995557896255e-15 -3.0405529889787885622
- joint left_ank_R21: origin xyz=0.0021000000000002752576 0.010000000000000036637 -0.0019000000000000058509 rpy=-1.570796326794896558 1.4871995686199779296 -1.5707963267949018871 -> xyz=0 0.010000000000000036637 -0.001899999999999998912 rpy=1.570796326794896558 1.428569774762729061 -1.570796326794896558
- joint left_ank_R22: origin xyz=0.0021000000000000115796 -0.010000000000000036637 -0.001899999999999998912 rpy=-1.5707963267950195707 -1.4871998384676159422 -1.5707963267947853137 -> xyz=1.3877787807814456755e-17 -0.010000000000000036637 -0.0019000000000000058509 rpy=1.5707963267949061059 -1.4285463212675062472 -1.5707963267949052177
- joint left_ank_act1: limit lower=-0.01799999999999999864 upper=0.01799999999999999864 effort=1 velocity=20 -> lower=0 upper=0.040000000000000000833 effort=1 velocity=20; origin xyz=2.272209342117637032e-06 -2.1996293675385913957e-15 -0.059356158967298844331 rpy=-3.141592653589793116 -9.2921664633026457838e-16 -0.63671356442004722886 -> xyz=2.2722093542849874925e-06 9.5062846483529028774e-16 -0.072660031604104974301 rpy=-3.1415926535896594451 8.6956799327801851499e-14 -2.2021168238262722738
- joint left_ank_act2: limit lower=-0.01799999999999999864 upper=0.01799999999999999864 effort=1 velocity=20 -> lower=0 upper=0.040000000000000000833 effort=1 velocity=20; origin xyz=2.2722093409414945153e-06 -1.7347234759768070944e-15 -0.05935645944356465753 rpy=3.141592653589793116 2.5208502705617295898e-15 -0.63671356442004545251 -> xyz=2.2722093491103073637e-06 -6.5433769513845163601e-15 -0.072660030478827297706 rpy=-3.1415926535895009053 6.1538805987964111831e-14 -2.2021168238262798234
- joint left_ank_pitch: origin xyz=4.2143614023597344721e-19 -0.09999999999999995004 -0.0062000000000000023842 rpy=3.1415926535897074068 -7.168818208916126976e-14 -1.5707963267948470421 -> xyz=1.0842022241842927186e-18 -0.10000000000000006106 -0.0061999999999999867717 rpy=-3.141592653589793116 -1.9981846038921943663e-15 -1.570796326794896558
- joint left_ank_roll: origin xyz=3.3306690738754696213e-16 -0.0061000000000003698833 -0.014600000000000704428 rpy=-1.5707963267949007768 -1.5707963267947875341 0 -> xyz=1.193489751472043281e-15 -0.00610000000000079836 -0.014600000000000288095 rpy=-1.5707963267948288344 -1.5707963267944542451 0
- joint left_hip_pitch: child hip_pitch_link -> left_hip_pitch_link; origin xyz=-0.024000000716140678508 -0.019000000152444841001 -0.019000000152450791102 rpy=-1.5707963267948210628 1.5707963267948126251 0 -> xyz=-0.02400000071615384506 -0.019000000152441031548 -0.019000000152448098811 rpy=-1.570796326794478226 1.5707963267948008568 0
- joint left_hip_roll: origin xyz=0.019000000000000304839 -5.0328333128562291641e-18 -0.025000000000000268535 rpy=3.141592653589793116 -1.5707963267948947816 0 -> xyz=0.019000000000000273614 -2.891526265917987331e-16 -0.026000000000000279832 rpy=-3.141592653589793116 -1.5707963267945983521 0
- joint left_hip_yaw: origin xyz=-0.0064000000000000115824 0.034999999999999524547 0.28649999999999997691 rpy=-8.5053965663345416767e-17 1.6935781366380737897e-17 -6.7749854439787420343e-14 -> xyz=-0.011900000000000068509 0.033999999999999967748 0.27720000000000005747 rpy=-2.2204460494576350945e-16 2.2204460491537123791e-16 -1.0069344447037368454e-13
- joint left_knee: limit lower=-1.570796326794896558 upper=1.570796326794896558 effort=1 velocity=20 -> lower=-1.570796326794896558 upper=2.2689280275926284602 effort=1 velocity=20; origin xyz=-4.686453338044572818e-15 0.097999999999999976019 0.027400000000003393863 rpy=-3.1415926535897620298 -6.106988965093026078e-15 -6.2039230811899877997e-14 -> xyz=-6.5714384231211065113e-15 0.09599999999999973832 0.027400000000000167277 rpy=-3.1415926535897891192 1.5325113271907731669e-16 -5.5621661637730288381e-17; parent hip_pitch_link -> left_hip_pitch_link
- joint right_ank_B11: origin xyz=0.018000000000000015987 0.010000000000000036637 -0.011499999999999994602 rpy=1.5707963267948974462 -1.4719660848800855124 -1.570796326794896336 -> xyz=0.0080000000000000001665 0.015000000000000041078 -0.011499999999999994602 rpy=1.570796326794896558 -1.469636014037949634 -1.5707963267948781283
- joint right_ank_B12: origin xyz=0.018000000000000002109 0.010000000000000036637 0.028300000000000012645 rpy=-1.5707963267948974462 -1.4752931174794650104 1.5707963267948936714 -> xyz=0.0080000000000000088402 0.015000000000000068834 0.02829999999999998489 rpy=-1.5707963267948383823 -1.4697566621827073963 1.5707963267948992225
- joint right_ank_B21: origin xyz=-6.9388939039072283776e-18 0 -0.011499999999999992867 rpy=1.570796326794896558 -1.4871995686197141406 1.5707963267948958919 -> xyz=-6.9388939039072283776e-18 0 -0.011500000000000006745 rpy=1.570796326794896558 -1.4285697747625620835 1.5707963267948821251
- joint right_ank_B22: origin xyz=0 -2.7755575615628913511e-17 -0.011500000000000003275 rpy=1.570796326794896558 -1.4871998384672124871 1.5707963267948923392 -> xyz=-6.9388939039072283776e-18 -2.7755575615628913511e-17 -0.011499999999999999806 rpy=1.570796326794896558 -1.4285463212677993461 1.5707963267949389685
- joint right_ank_B31: origin xyz=0 -0.0064387505004004086384 6.9388939039072283776e-18 rpy=-1.570796326794896558 -5.4574696529115381853e-06 -1.2331483706146518492e-15 -> xyz=1.4745149545802860303e-17 -0.006438750500400436394 0 rpy=-1.5707963267948961139 0.16913440034159002434 1.9223858256087746368e-15
- joint right_ank_B32: origin xyz=0 -0.0064387505004004086384 0 rpy=-1.570796326794896558 -5.4574689504429525655e-06 -5.0339227696192602828e-16 -> xyz=5.6378512969246230568e-18 -0.006438750500400436394 0 rpy=-1.570796326794896336 -0.17993145005752267385 1.8689858510975082391e-15
- joint right_ank_R11: origin xyz=-0.010000000000000112965 0.012500000000000233147 -0.032999999999998946842 rpy=3.1415926535897922278 -2.5232420665482256888e-16 -0.098830241914703576001 -> xyz=-0.0099999999999999984734 0.012500000000000066613 -0.027900000000000015066 rpy=-3.1415926535897860106 -4.3778626236368231385e-15 -0.10116031275681484913
- joint right_ank_R12: origin xyz=0.0099999999999998891859 0.012500000000000066613 -0.032999999999998946842 rpy=-3.141592653589793116 -1.1886010661269619878e-15 -3.0460894442739978594 -> xyz=0.010000000000000000208 0.012500000000000011102 -0.027900000000000001188 rpy=-3.1415926535897829019 -8.8337259752553850467e-15 -3.040552988977761828
- joint right_ank_R21: origin xyz=0.0021000000000001434186 0.010000000000000230926 -0.0018999999999989442001 rpy=-1.5707963267948970021 1.4871995686198307141 -1.5707963267948983344 -> xyz=0 0.010000000000000092149 -0.0019000000000000058509 rpy=1.570796326794896558 1.4285697747627268406 -1.5707963267948945596
- joint right_ank_R22: origin xyz=0.0020999999999999074962 -0.010000000000000119904 -0.0018999999999989372612 rpy=-1.5707963267948956698 -1.487199838467331281 -1.5707963267948870101 -> xyz=6.9388939039072283776e-18 -0.010000000000000064393 -0.001899999999999998912 rpy=1.570796326794896558 -1.4285463212679276879 -1.5707963267948938935
- joint right_ank_act1: limit lower=-0.01799999999999999864 upper=0.01799999999999999864 effort=1 velocity=20 -> lower=0 upper=0.040000000000000000833 effort=1 velocity=20; origin xyz=2.2722093427941791877e-06 9.92261828258733658e-16 -0.059356158967292543815 rpy=-3.1415926535897837901 -1.2238359105881652741e-14 -0.63671356441985882402 -> xyz=2.2722093427473416538e-06 1.2559397966072083364e-15 -0.07266003160412204398 rpy=-3.1415926535897895633 9.1629640935489764995e-15 -2.2021168238260711014
- joint right_ank_act2: limit lower=-0.01799999999999999864 upper=0.01799999999999999864 effort=1 velocity=20 -> lower=0 upper=0.040000000000000000833 effort=1 velocity=20; origin xyz=2.2722093411253752038e-06 -2.4008572907519010187e-15 -0.059356459443579534518 rpy=-3.1415926535897926719 9.0510831053370240348e-16 -0.63671356442005022647 -> xyz=2.2722093417394673143e-06 -2.3939183968479937903e-15 -0.072660030478831599821 rpy=3.141592653589793116 -2.0657592427741678223e-15 -2.2021168238262744943
- joint right_ank_pitch: origin xyz=-1.0422817820682455029e-15 0.10000000000000003331 -0.0062000000000001706524 rpy=-3.1415926535897900074 3.0234911913779407472e-15 -1.5707963267948836794 -> xyz=7.5714896865366240827e-19 0.10000000000000003331 -0.00619999999999999718 rpy=-3.141592653589793116 1.998618284759728781e-15 -1.57079632679489678
- joint right_ank_roll: origin xyz=1.1102230246251565404e-15 -0.006100000000001146172 -0.014600000000001599545 rpy=-1.5707963267948990005 1.5707963267948332753 0 -> xyz=2.1926904736346841673e-15 -0.0061000000000001799311 -0.014600000000002237924 rpy=-1.5707963267949249797 1.5707963267947928632 0
- joint right_hip_pitch: child hip_pitch_link_2 -> right_hip_pitch_link; origin xyz=-0.024000000716145990232 -0.019000000152457986735 -0.019000000152453767888 rpy=-1.5707963267951823294 1.5707963267947557817 0 -> xyz=-0.024000000716146760449 -0.019000000152456297114 -0.019000000152450020885 rpy=-1.5707963267951789987 1.5707963267947411268 0
- joint right_hip_roll: origin xyz=-0.018999999999999885036 -5.020473408011439263e-18 -0.025000000000000001388 rpy=1.4827462901121851002e-29 -1.5707963267947766539 0 -> xyz=-0.018999999999999881567 -3.3500438889867783387e-18 -0.026000000000000002276 rpy=3.0518439807331778725e-31 -1.5707963267948181763 0
- joint right_hip_yaw: origin xyz=-0.0064000000000000115824 -0.035000000000000017208 0.28649999999999997691 rpy=-1.3903812075106529584e-14 -4.1920818891027382935e-15 -1.1753904145936466635e-14 -> xyz=-0.011900000000000259329 -0.033999999999999974687 0.27720000000000000195 rpy=-2.2204460561717224569e-16 2.2204460926237942003e-16 -6.0840221749459209504e-14
- joint right_knee: origin xyz=-2.5483606178382506831e-15 0.097999999999999684586 0.027399999999999827272 rpy=3.1415926535897926719 -1.2487298519101510075e-16 -3.141592653589788231 -> xyz=-1.8821214288092669642e-15 0.096000000000001001199 0.027399999999998970318 rpy=3.1415926535897220617 -3.0356441407590551802e-14 3.1415926535897846783; parent hip_pitch_link_2 -> right_hip_pitch_link
- joint right_sho_pitch: origin xyz=-0.0064000000000000167866 -0.057999999999999982125 0.4124999999999999778 rpy=-1.570796326794896558 1.3877787807814444922e-15 8.1990370565314014207e-16 -> xyz=-0.0063999999999999916331 -0.057999999999999989064 0.4124999999999999778 rpy=-1.5707963267948972241 1.3877787807856806753e-15 6.3545304591998415249e-17
