Commit message: Update the base robot

File: toddlerbot/robot_descriptions/assemblies/4R_body/4R_body.urdf (robot description, URDF)
Before this commit: robot 4R_body, 8 links, 7 joints
Links:
- link body_link: mass 1.3010345634555096073 -> 1.3010345634555104954
- link left_3r+rh5_leg: mass 0.33313077160322585035 -> 0.33284223932564410697
Joints:
- joint left_hip_yaw: origin xyz=-0.011900000000000068509 0.033999999999999967748 0.27720000000000005747 rpy=-2.2204460494576350945e-16 2.2204460491537123791e-16 -1.0069344447037368454e-13 -> xyz=-0.011900000000000070244 0.033999999999999974687 0.27720000000000011298 rpy=-2.2204460494577687078e-16 2.2204460491536837829e-16 -1.0069344447037764778e-13
- joint right_hip_yaw: origin xyz=-0.011900000000000259329 -0.033999999999999974687 0.27720000000000000195 rpy=-2.2204460561717224569e-16 2.2204460926237942003e-16 -6.0840221749459209504e-14 -> xyz=-0.011900000000000259329 -0.033999999999999981626 0.27720000000000000195 rpy=-2.2204460717259335277e-16 2.2204461793479381443e-16 -6.6849266279598662255e-15

File: toddlerbot/robot_descriptions/assemblies/left_3R+RH5_leg/left_3R+RH5_leg.urdf (robot description, URDF)
Before this commit: robot left_3R+RH5_leg, 18 links, 17 joints
Links:
- link ank_roll_link: mass 0.013844478784760250178 -> 0.013844478784760251913
- link ank_rr_link: mass 0.00044289790445047668311 -> 0.00044289790445047673732
- link ank_rr_link_2: mass 0.00044289790445047668311 -> 0.00044289790445047673732
- link left_calf_link: mass 0.016579149141633314074 -> 0.016290616864051549878
Joints:
- joint left_ank_B11: origin xyz=0.008000000000000053943 -0.014999999999999985567 0.028299999999999915501 rpy=-1.57079632679489678 1.4696360140379260972 1.5707963267948892305 -> xyz=0.0079999999999999880235 -0.015000000000000041078 0.028300000000000005707 rpy=-1.570796326794896558 1.469636014037934757 1.5707963267948754638
- joint left_ank_B12: origin xyz=0.0080000000000000504735 -0.014999999999999930056 -0.011500000000000076134 rpy=-1.5707963267948958919 -1.4697566621822790722 1.5707963267948983344 -> xyz=0.0080000000000001268013 -0.014999999999999791278 -0.011499999999999987663 rpy=-1.570796326794896558 -1.4697566621822597543 1.5707963267949038855
- joint left_ank_B21: origin xyz=0 0 -0.011499999999999996336 rpy=1.570796326794896558 -1.4285697747625092369 1.5707963267948912289 -> xyz=0 2.7755575615628913511e-17 -0.011499999999999999806 rpy=1.570796326794896558 -1.4285697747625467624 1.5707963267948807928
- joint left_ank_B22: origin xyz=-6.9388939039072283776e-18 -8.3266726846886740532e-17 -0.011499999999999996336 rpy=1.5707963267948961139 -1.4285463212680367118 -1.5707963267948970021 -> xyz=-3.4694469519536141888e-17 -2.7755575615628913511e-16 -0.01149999999999988011 rpy=1.570796326794896558 -1.4285463212680655776 -1.5707963267948985564
- joint left_ank_B31: origin xyz=-3.4694469519536141888e-18 -0.0064387505004004086384 -6.9388939039072283776e-18 rpy=-1.570796326794896558 0.16913440034103149889 1.5363542389808260585e-15 -> xyz=4.336808689942017736e-19 -0.0064387505004004641496 6.9388939039072283776e-18 rpy=-1.57079632679489678 0.16913440034102095177 4.5559338426713504067e-15
- joint left_ank_B32: origin xyz=1.9949319973733281586e-17 -0.0064387505004002698605 1.3877787807814456755e-17 rpy=-1.5707963267948970021 -0.17993145005780439294 -1.804382386805444098e-17 -> xyz=1.4311468676808658529e-17 -0.0064387505004005751719 6.9388939039072283776e-18 rpy=-1.5707963267948972241 -0.17993145005787733459 6.7429791500468328215e-16
- joint left_ank_R11: origin xyz=-0.01000000000000001929 0.012500000000000011102 -0.027899999999999692407 rpy=-3.141592653589793116 3.5006616330671580104e-18 -0.10116031275702692949 -> xyz=-0.0099999999999999915345 0.012499999999999872324 -0.033600000000000004863 rpy=1.6323812772036896109e-17 1.4002646486553138019e-17 -0.10116031275705798798
- joint left_ank_R12: origin xyz=0.0099999999999999932693 0.012500000000000066613 -0.027900000000000039352 rpy=3.1415926535897904515 2.6926878995557896255e-15 -3.0405529889787885622 -> xyz=0.0099999999999999984734 0.012499999999999761302 -0.033599999999999997924 rpy=3.1415926535897824579 9.4861357133311978266e-15 -3.0405529889788134312
- joint left_ank_R21: origin xyz=0 0.010000000000000036637 -0.001899999999999998912 rpy=1.570796326794896558 1.428569774762729061 -1.570796326794896558 -> xyz=0 -0.010000000000000036637 -2.0816681711721685133e-17 rpy=-1.5707963267949025532 -1.4285697747629921839 1.5707963267949025532
- joint left_ank_R22: origin xyz=1.3877787807814456755e-17 -0.010000000000000036637 -0.0019000000000000058509 rpy=1.5707963267949061059 -1.4285463212675062472 -1.5707963267949052177 -> xyz=-6.9388939039072283776e-18 -0.010000000000000008882 0 rpy=1.570796326794896558 -1.4285463212677487199 -1.5707963267948970021
- joint left_ank_act1: origin xyz=2.2722093542849874925e-06 9.5062846483529028774e-16 -0.072660031604104974301 rpy=-3.1415926535896594451 8.6956799327801851499e-14 -2.2021168238262722738 -> xyz=2.2722093543023347273e-06 9.5756735873919751612e-16 -0.072660031604096092517 rpy=-3.1415926535896594451 8.5062006308179150635e-14 -2.2021168238262847083
- joint left_ank_act2: origin xyz=2.2722093491103073637e-06 -6.5433769513845163601e-15 -0.072660030478827297706 rpy=-3.1415926535895009053 6.1538805987964111831e-14 -2.2021168238262798234 -> xyz=2.2722093491519407271e-06 -6.5988881026157741871e-15 -0.072660030478819720434 rpy=-3.1415926535895000171 5.9263713871214940499e-14 -2.2021168238262815997
- joint left_ank_pitch: origin xyz=1.0842022241842927186e-18 -0.10000000000000006106 -0.0061999999999999867717 rpy=-3.141592653589793116 -1.9981846038921943663e-15 -1.570796326794896558 -> xyz=9.1534583908775112557e-19 -0.10000000000000003331 -0.0061999999999999989148 rpy=3.1415926535897926719 -8.7927079361011792447e-15 -1.5707963267948961139
- joint left_ank_roll: origin xyz=1.193489751472043281e-15 -0.00610000000000079836 -0.014600000000000288095 rpy=-1.5707963267948288344 -1.5707963267944542451 0 -> xyz=2.2759572004815709079e-15 0.0015000000000041896053 -0.014599999999999611552 rpy=-1.570796326795051101 -1.5707963267944144992 0
- joint left_hip_pitch: origin xyz=-0.02400000071615384506 -0.019000000152441031548 -0.019000000152448098811 rpy=-1.570796326794478226 1.5707963267948008568 0 -> xyz=-0.024000000716153851998 -0.019000000152441028078 -0.019000000152448098811 rpy=-1.570796326794478226 1.5707963267948015229 0
- joint left_hip_roll: origin xyz=0.019000000000000273614 -2.891526265917987331e-16 -0.026000000000000279832 rpy=-3.141592653589793116 -1.5707963267945983521 0 -> xyz=0.019000000000000284023 -8.3919669538584410836e-16 -0.026000000000000463712 rpy=-3.1415926535897922278 -1.5707963267945732611 0
- joint left_knee: origin xyz=-6.5714384231211065113e-15 0.09599999999999973832 0.027400000000000167277 rpy=-3.1415926535897891192 1.5325113271907731669e-16 -5.5621661637730288381e-17 -> xyz=-6.5356617016366259295e-15 0.095999999999999696687 0.027400000000000260952 rpy=-3.1415926535897842342 1.6653345304510526278e-16 2.2176671495670943584e-16

File: toddlerbot/robot_descriptions/assemblies/right_3R+RH5_leg/right_3R+RH5_leg.urdf (robot description, URDF)
Before this commit: robot right_3R+RH5_leg, 18 links, 17 joints
Links:
- link ank_roll_link: mass 0.013844478784760250178 -> 0.013844478784760251913
- link ank_rr_link: mass 0.00044289790445047668311 -> 0.00044289790445047673732
- link ank_rr_link_2: mass 0.00044289790445047668311 -> 0.00044289790445047673732
- link right_hip_pitch_link: mass 0.094084567879581956773 -> 0.094084567879581970651
Joints:
- joint right_ank_B11: origin xyz=0.0080000000000000001665 0.015000000000000041078 -0.011499999999999994602 rpy=1.570796326794896558 -1.469636014037949634 -1.5707963267948781283 -> xyz=0.0079999999999999689415 0.015000000000000124345 -0.011500000000000058786 rpy=1.5707963267948932273 -1.4696360140379622905 -1.5707963267948383823
- joint right_ank_B12: origin xyz=0.0080000000000000088402 0.015000000000000068834 0.02829999999999998489 rpy=-1.5707963267948383823 -1.4697566621827073963 1.5707963267948992225 -> xyz=0.0080000000000000730249 0.015000000000000263123 0.028299999999999901623 rpy=-1.5707963267948388264 -1.4697566621826396727 1.5707963267950122432
- joint right_ank_B21: origin xyz=-6.9388939039072283776e-18 0 -0.011500000000000006745 rpy=1.570796326794896558 -1.4285697747625620835 1.5707963267948821251 -> xyz=0 5.5511151231257827021e-17 -0.011499999999999998071 rpy=1.570796326794896558 -1.4285697747625634157 1.5707963267948530373
- joint right_ank_B22: origin xyz=-6.9388939039072283776e-18 -2.7755575615628913511e-17 -0.011499999999999999806 rpy=1.570796326794896558 -1.4285463212677993461 1.5707963267949389685 -> xyz=0 0 -0.011499999999999992867 rpy=1.5707963267949405228 -1.4285463212677880218 1.5707963267949816011
- joint right_ank_B31: origin xyz=1.4745149545802860303e-17 -0.006438750500400436394 0 rpy=-1.5707963267948961139 0.16913440034159002434 1.9223858256087746368e-15 -> xyz=-7.3725747729014301513e-18 -0.006438750500400436394 -1.3877787807814456755e-17 rpy=-1.5707963267948954478 0.16913440034160504011 5.0191724325132069355e-15
- joint right_ank_B32: origin xyz=5.6378512969246230568e-18 -0.006438750500400436394 0 rpy=-1.570796326794896336 -0.17993145005752267385 1.8689858510975082391e-15 -> xyz=-1.6913553890773869171e-17 -0.0064387505004003531273 -1.3877787807814456755e-17 rpy=-1.5707963267948952257 -0.17993145005754265786 3.2634092460731900895e-15
- joint right_ank_R11: origin xyz=-0.0099999999999999984734 0.012500000000000066613 -0.027900000000000015066 rpy=-3.1415926535897860106 -4.3778626236368231385e-15 -0.10116031275681484913 -> xyz=-0.0099999999999999707179 0.012500000000000066613 -0.033600000000000039557 rpy=2.8867109174417181635e-14 -3.1302655555270997905e-14 -0.10116031275652562216
- joint right_ank_R12: origin xyz=0.010000000000000000208 0.012500000000000011102 -0.027900000000000001188 rpy=-3.1415926535897829019 -8.8337259752553850467e-15 -3.040552988977761828 -> xyz=0.010000000000000003678 0.012500000000000011102 -0.033600000000000004863 rpy=-3.1415926535897917837 -1.5904604637588844751e-15 -3.0405529889774984831
- joint right_ank_R21: origin xyz=0 0.010000000000000092149 -0.0019000000000000058509 rpy=1.570796326794896558 1.4285697747627268406 -1.5707963267948945596 -> xyz=1.3877787807814456755e-17 -0.010000000000000008882 1.3877787807814456755e-17 rpy=-1.570796326794896558 -1.4285697747627732479 1.5707963267950297848
- joint right_ank_R22: origin xyz=6.9388939039072283776e-18 -0.010000000000000064393 -0.001899999999999998912 rpy=1.570796326794896558 -1.4285463212679276879 -1.5707963267948938935 -> xyz=-1.3877787807814456755e-17 -0.010000000000000008882 2.7755575615628913511e-17 rpy=1.570796326794921649 -1.4285463212679851974 -1.5707963267949038855
- joint right_ank_act1: origin xyz=2.2722093427473416538e-06 1.2559397966072083364e-15 -0.07266003160412204398 rpy=-3.1415926535897895633 9.1629640935489764995e-15 -2.2021168238260711014 -> xyz=2.2722093427438722069e-06 1.6375789613221058971e-15 -0.072660031604109970305 rpy=-3.1415926535897806815 7.845419351877858644e-15 -2.2021168238260604433
- joint right_ank_act2: origin xyz=2.2722093417394673143e-06 -2.3939183968479937903e-15 -0.072660030478831599821 rpy=3.141592653589793116 -2.0657592427741678223e-15 -2.2021168238262744943 -> xyz=2.2722093418418159994e-06 -2.3939183968479937903e-15 -0.072660030478818443678 rpy=-3.1415926535897926719 -5.822843740105227622e-15 -2.202116823826253178
- joint right_ank_pitch: origin xyz=7.5714896865366240827e-19 0.10000000000000003331 -0.00619999999999999718 rpy=-3.141592653589793116 1.998618284759728781e-15 -1.57079632679489678 -> xyz=-7.3090839045994630973e-18 0.099999999999999839018 -0.006199999999999821973 rpy=-3.1415926535897926719 3.8309199562601306947e-15 -1.57079632679489678
- joint right_ank_roll: origin xyz=2.1926904736346841673e-15 -0.0061000000000001799311 -0.014600000000002237924 rpy=-1.5707963267949249797 1.5707963267947928632 0 -> xyz=1.1018963519404678664e-14 0.0015000000000008478773 -0.014599999999995005862 rpy=-1.5707963267950115771 1.5707963267945974639 0
- joint right_hip_pitch: origin xyz=-0.024000000716146760449 -0.019000000152456297114 -0.019000000152450020885 rpy=-1.5707963267951789987 1.5707963267947411268 0 -> xyz=-0.024000000716146767388 -0.019000000152456290176 -0.019000000152450020885 rpy=-1.5707963267951789987 1.5707963267947586683 0
- joint right_hip_roll: origin xyz=-0.018999999999999881567 -3.3500438889867783387e-18 -0.026000000000000002276 rpy=3.0518439807331778725e-31 -1.5707963267948181763 0 -> xyz=-0.018999999999999891975 2.3744804088669454642e-18 -0.025999999999999984929 rpy=-3.3306690738820289997e-16 -1.570796326794896558 0
- joint right_knee: origin xyz=-1.8821214288092669642e-15 0.096000000000001001199 0.027399999999998970318 rpy=3.1415926535897220617 -3.0356441407590551802e-14 3.1415926535897846783 -> xyz=-1.8318267252532356178e-15 0.095999999999998836264 0.027400000000000895861 rpy=3.1415926535897895633 -1.5829351718147190682e-16 -3.141592653589793116
