Commit message: Automate computing offsets and collision mesh

File: toddlerbot/robot_descriptions/assemblies/4R_body/4R_body.urdf (robot description, URDF)
Before this commit: robot 4R_body, 8 links, 7 joints
Links:
- removed link base_link
- link body_link: mass 1.3010345634555104954 -> 1.3010345634555091632
- link head_link: mass 0.075015538754887006734 -> 0.075015538754886992856
- link left_3r+rh5_leg: mass 0.33284223932564410697 -> 0.33284223931512424421
- link left_op3_arm: mass 0.15851190405198536948 -> 0.15851190405198534172
- link neck_link: mass 0.018378317023500286703 -> 0.018378317023500283234
- link right_3r+rh5_leg: mass 0.33284223245696664684 -> 0.33284223244644678408
Joints:
- removed joint base_link_to_base
- joint head: origin xyz=-4.1826855620466421722e-19 -2.6020852139652106416e-18 -0.039999999999999980016 rpy=-3.6199375412562401434e-16 -2.4218742848029192401e-16 -5.5511151231257722251e-17 -> xyz=0 0 -0.039999999999999980016 rpy=-3.6199375412562401434e-16 -2.4218742848029192401e-16 -5.5511151231257722251e-17
- joint left_hip_yaw: origin xyz=-0.011900000000000070244 0.033999999999999974687 0.27720000000000011298 rpy=-2.2204460494577687078e-16 2.2204460491536837829e-16 -1.0069344447037764778e-13 -> xyz=-0.011900000000000070244 0.033999999999999967748 0.28550000000000003153 rpy=-2.2204460494577687078e-16 2.2204460491536837829e-16 -1.0069344447037764778e-13
- joint left_sho_pitch: origin xyz=-0.0064000000000001278089 0.057999999999999600486 0.41249999999999986677 rpy=-1.570796326794871911 3.5360603334311235812e-14 -3.1415926535897371608 -> xyz=-0.0064000000000001781159 0.057999999999999808653 0.42079999999999984084 rpy=-1.570796326794871911 3.5360603334311235812e-14 -3.1415926535897371608
- joint neck: origin xyz=-0.0063999999999999838268 -5.2372852656669075105e-18 0.43249999999999999556 rpy=-3.141592653589793116 8.5053965662326763145e-17 1.57079632679489678 -> xyz=-0.0063999999999999820921 -4.4507968385753129991e-18 0.44079999999999996962 rpy=-3.141592653589793116 8.5053965662326763145e-17 1.57079632679489678
- joint right_hip_yaw: origin xyz=-0.011900000000000259329 -0.033999999999999981626 0.27720000000000000195 rpy=-2.2204460717259335277e-16 2.2204461793479381443e-16 -6.6849266279598662255e-15 -> xyz=-0.011900000000000261063 -0.033999999999999974687 0.28549999999999997602 rpy=-2.2204460717259335277e-16 2.2204461793479381443e-16 -6.6849266279598654366e-15
- joint right_sho_pitch: origin xyz=-0.0063999999999999916331 -0.057999999999999989064 0.4124999999999999778 rpy=-1.5707963267948972241 1.3877787807856806753e-15 6.3545304591998415249e-17 -> xyz=-0.006399999999999998572 -0.057999999999999982125 0.42079999999999995186 rpy=-1.5707963267948972241 1.3877787807856806753e-15 6.3545304591998415249e-17

File: toddlerbot/robot_descriptions/assemblies/left_3R+RH5_leg/left_3R+RH5_leg.urdf (robot description, URDF)
Before this commit: robot left_3R+RH5_leg, 18 links, 17 joints
Links:
- link 12lf: mass 0.044782197696050352054 -> 0.044782197690790462308
- link 12lf_2: mass 0.044782197696050352054 -> 0.044782197690790462308
- link 12lf_rod: mass 0.0025088292483592140175 -> 0.0025088292483592144512
- link 12lf_rod_2: mass 0.0025088292483592140175 -> 0.0025088292483592144512
- link 12lf_rod_end: mass 0.00085420491177815905965 -> 0.00085420491177815895123
- link 12lf_rod_end_2: mass 0.00085420491177815905965 -> 0.00085420491177815895123
- link ank_pitch_link: mass 0.0042238381753791605713 -> 0.0042238381753791614387
- link ank_roll_link: mass 0.013844478784760251913 -> 0.013844478784760248444
- link ball_joint_ball: mass 4.4053796295264630609e-05 -> 4.4053796295264623832e-05
- link ball_joint_ball_2: mass 4.4053796295264630609e-05 -> 4.4053796295264623832e-05
- link ball_joint_container: mass 4.803735642533054869e-05 -> 4.8037356425330562243e-05
- link ball_joint_container_2: mass 4.803735642533054869e-05 -> 4.8037356425330562243e-05
- link hip_roll_link: mass 0.098012391483528679692 -> 0.098012391483528651936
- link left_hip_pitch_link: mass 0.094084588454108858402 -> 0.094084588454108844524
Joints:
- joint left_ank_B21: origin xyz=0 2.7755575615628913511e-17 -0.011499999999999999806 rpy=1.570796326794896558 -1.4285697747625467624 1.5707963267948807928 -> xyz=-6.9388939039072283776e-18 2.7755575615628913511e-17 -0.011499999999999999806 rpy=1.570796326794896558 -1.4285697747625467624 1.5707963267948807928
- joint left_ank_B31: origin xyz=4.336808689942017736e-19 -0.0064387505004004641496 6.9388939039072283776e-18 rpy=-1.57079632679489678 0.16913440034102095177 4.5559338426713504067e-15 -> xyz=1.7347234759768070944e-18 -0.0064387505004004641496 1.3877787807814456755e-17 rpy=-1.57079632679489678 0.16913440034102092402 4.5559338426713504067e-15
- joint left_ank_B32: origin xyz=1.4311468676808658529e-17 -0.0064387505004005751719 6.9388939039072283776e-18 rpy=-1.5707963267948972241 -0.17993145005787733459 6.7429791500468328215e-16 -> xyz=8.6736173798840354721e-18 -0.0064387505004005751719 6.9388939039072283776e-18 rpy=-1.5707963267948972241 -0.17993145005787733459 6.7429791500468328215e-16
- joint left_ank_act2: origin xyz=2.2722093491519407271e-06 -6.5988881026157741871e-15 -0.072660030478819720434 rpy=-3.1415926535895000171 5.9263713871214940499e-14 -2.2021168238262815997 -> xyz=2.2722093491484712802e-06 -6.5988881026157741871e-15 -0.07266003047881974819 rpy=-3.1415926535895000171 5.9280886354915822063e-14 -2.2021168238262815997

File: toddlerbot/robot_descriptions/assemblies/left_OP3_arm/left_OP3_arm.urdf (robot description, URDF)
Before this commit: robot left_OP3_arm, 3 links, 2 joints
Links:
- link elb_link: mass 0.012147845014428809707 -> 0.012147845014428806237
- link sho_pitch_link: mass 0.0053168741776095304608 -> 0.0053168741776095261239

File: toddlerbot/robot_descriptions/assemblies/right_3R+RH5_leg/right_3R+RH5_leg.urdf (robot description, URDF)
Before this commit: robot right_3R+RH5_leg, 18 links, 17 joints
Links:
- link 12lf: mass 0.044782197696050352054 -> 0.044782197690790462308
- link 12lf_2: mass 0.044782197696050358993 -> 0.044782197690790476186
- link 12lf_rod: mass 0.0025088292483592140175 -> 0.0025088292483592144512
- link 12lf_rod_2: mass 0.0025088292483592140175 -> 0.0025088292483592144512
- link 12lf_rod_end: mass 0.00085420491177815905965 -> 0.00085420491177815895123
- link 12lf_rod_end_2: mass 0.00085420491177815905965 -> 0.00085420491177815895123
- link ank_pitch_link: mass 0.0042238381753791605713 -> 0.0042238381753791614387
- link ank_roll_link: mass 0.013844478784760251913 -> 0.013844478784760248444
- link ball_joint_ball: mass 4.4053796295264630609e-05 -> 4.4053796295264623832e-05
- link ball_joint_ball_2: mass 4.4053796295264630609e-05 -> 4.4053796295264623832e-05
- link ball_joint_container: mass 4.803735642533054869e-05 -> 4.8037356425330562243e-05
- link ball_joint_container_2: mass 4.803735642533054869e-05 -> 4.8037356425330562243e-05
- link hip_roll_link: mass 0.09801239148352869357 -> 0.098012391483528665814
- link right_hip_pitch_link: mass 0.094084567879581970651 -> 0.094084567879581942895
Joints:
- joint right_ank_B31: origin xyz=-7.3725747729014301513e-18 -0.006438750500400436394 -1.3877787807814456755e-17 rpy=-1.5707963267948954478 0.16913440034160504011 5.0191724325132069355e-15 -> xyz=-6.0715321659188248304e-18 -0.006438750500400436394 -1.3877787807814456755e-17 rpy=-1.5707963267948954478 0.16913440034160504011 5.0191724325132069355e-15
- joint right_ank_B32: origin xyz=-1.6913553890773869171e-17 -0.0064387505004003531273 -1.3877787807814456755e-17 rpy=-1.5707963267948952257 -0.17993145005754265786 3.2634092460731900895e-15 -> xyz=-1.561251128379126385e-17 -0.0064387505004003531273 -1.3877787807814456755e-17 rpy=-1.5707963267948952257 -0.17993145005754265786 3.2634092460731900895e-15
- joint right_ank_act1: origin xyz=2.2722093427438722069e-06 1.6375789613221058971e-15 -0.072660031604109970305 rpy=-3.1415926535897806815 7.845419351877858644e-15 -2.2021168238260604433 -> xyz=2.2722093427421374834e-06 1.6375789613221058971e-15 -0.072660031604109970305 rpy=-3.1415926535897806815 7.845419351877858644e-15 -2.2021168238260604433

File: toddlerbot/robot_descriptions/assemblies/right_OP3_arm/right_OP3_arm.urdf (robot description, URDF)
Before this commit: robot right_OP3_arm, 3 links, 2 joints
Links:
- link elb_link: mass 0.012147845014428809707 -> 0.012147845014428806237
- link sho_pitch_link: mass 0.0053168741776095304608 -> 0.0053168741776095261239
- link sho_roll_link: mass 0.1410471848599471334 -> 0.14104718485994710564

File: toddlerbot/robot_descriptions/base/base.urdf (robot description, URDF)
Before this commit: robot base, 46 links, 45 joints
Links:
- removed link base_link
- link 12lf: mass 0.044782197696050352054 -> 0.044782197690790462308
- link 12lf_2: mass 0.044782197696050352054 -> 0.044782197690790462308
- link 12lf_3: mass 0.044782197696050352054 -> 0.044782197690790462308
- link 12lf_4: mass 0.044782197696050358993 -> 0.044782197690790476186
- link 12lf_rod: mass 0.0025088292483592140175 -> 0.0025088292483592144512
- link 12lf_rod_2: mass 0.0025088292483592140175 -> 0.0025088292483592144512
- link 12lf_rod_3: mass 0.0025088292483592140175 -> 0.0025088292483592144512
- link 12lf_rod_4: mass 0.0025088292483592140175 -> 0.0025088292483592144512
- link 12lf_rod_end: mass 0.00085420491177815905965 -> 0.00085420491177815895123
- link 12lf_rod_end_2: mass 0.00085420491177815905965 -> 0.00085420491177815895123
- link 12lf_rod_end_3: mass 0.00085420491177815905965 -> 0.00085420491177815895123
- link 12lf_rod_end_4: mass 0.00085420491177815905965 -> 0.00085420491177815895123
- link ank_pitch_link: mass 0.0042238381753791605713 -> 0.0042238381753791614387
- link ank_pitch_link_2: mass 0.0042238381753791605713 -> 0.0042238381753791614387
- link ank_roll_link: mass 0.013844478784760251913 -> 0.013844478784760248444
- link ank_roll_link_2: mass 0.013844478784760251913 -> 0.013844478784760248444
- link ball_joint_ball: mass 4.4053796295264630609e-05 -> 4.4053796295264623832e-05
- link ball_joint_ball_2: mass 4.4053796295264630609e-05 -> 4.4053796295264623832e-05
- link ball_joint_ball_3: mass 4.4053796295264630609e-05 -> 4.4053796295264623832e-05
- link ball_joint_ball_4: mass 4.4053796295264630609e-05 -> 4.4053796295264623832e-05
- link ball_joint_container: mass 4.803735642533054869e-05 -> 4.8037356425330562243e-05
- link ball_joint_container_2: mass 4.803735642533054869e-05 -> 4.8037356425330562243e-05
- link ball_joint_container_3: mass 4.803735642533054869e-05 -> 4.8037356425330562243e-05
- link ball_joint_container_4: mass 4.803735642533054869e-05 -> 4.8037356425330562243e-05
- link body_link: mass 1.3010345634555104954 -> 1.3010345634555091632
- link elb_link: mass 0.012147845014428809707 -> 0.012147845014428806237
- link elb_link_2: mass 0.012147845014428809707 -> 0.012147845014428806237
- link head_link: mass 0.075015538754887006734 -> 0.075015538754886992856
- link hip_roll_link: mass 0.098012391483528679692 -> 0.098012391483528651936
- link hip_roll_link_2: mass 0.09801239148352869357 -> 0.098012391483528665814
- link left_hip_pitch_link: mass 0.094084588454108858402 -> 0.094084588454108844524
- link neck_link: mass 0.018378317023500286703 -> 0.018378317023500283234
- link right_hip_pitch_link: mass 0.094084567879581970651 -> 0.094084567879581942895
- link sho_pitch_link: mass 0.0053168741776095304608 -> 0.0053168741776095261239
- link sho_pitch_link_2: mass 0.0053168741776095304608 -> 0.0053168741776095261239
- link sho_roll_link_2: mass 0.1410471848599471334 -> 0.14104718485994710564
Joints:
- removed joint base_link_to_base
- joint head: origin xyz=-4.1826855620466421722e-19 -2.6020852139652106416e-18 -0.039999999999999980016 rpy=-3.6199375412562401434e-16 -2.4218742848029192401e-16 -5.5511151231257722251e-17 -> xyz=0 0 -0.039999999999999980016 rpy=-3.6199375412562401434e-16 -2.4218742848029192401e-16 -5.5511151231257722251e-17
- joint left_ank_B21: origin xyz=0 2.7755575615628913511e-17 -0.011499999999999999806 rpy=1.570796326794896558 -1.4285697747625467624 1.5707963267948807928 -> xyz=-6.9388939039072283776e-18 2.7755575615628913511e-17 -0.011499999999999999806 rpy=1.570796326794896558 -1.4285697747625467624 1.5707963267948807928
- joint left_ank_B31: origin xyz=4.336808689942017736e-19 -0.0064387505004004641496 6.9388939039072283776e-18 rpy=-1.57079632679489678 0.16913440034102095177 4.5559338426713504067e-15 -> xyz=1.7347234759768070944e-18 -0.0064387505004004641496 1.3877787807814456755e-17 rpy=-1.57079632679489678 0.16913440034102092402 4.5559338426713504067e-15
- joint left_ank_B32: origin xyz=1.4311468676808658529e-17 -0.0064387505004005751719 6.9388939039072283776e-18 rpy=-1.5707963267948972241 -0.17993145005787733459 6.7429791500468328215e-16 -> xyz=8.6736173798840354721e-18 -0.0064387505004005751719 6.9388939039072283776e-18 rpy=-1.5707963267948972241 -0.17993145005787733459 6.7429791500468328215e-16
- joint left_ank_act2: origin xyz=2.2722093491519407271e-06 -6.5988881026157741871e-15 -0.072660030478819720434 rpy=-3.1415926535895000171 5.9263713871214940499e-14 -2.2021168238262815997 -> xyz=2.2722093491484712802e-06 -6.5988881026157741871e-15 -0.07266003047881974819 rpy=-3.1415926535895000171 5.9280886354915822063e-14 -2.2021168238262815997
- joint left_hip_yaw: origin xyz=-0.011900000000000070244 0.033999999999999974687 0.27720000000000011298 rpy=-2.2204460494577687078e-16 2.2204460491536837829e-16 -1.0069344447037764778e-13 -> xyz=-0.011900000000000070244 0.033999999999999967748 0.28550000000000003153 rpy=-2.2204460494577687078e-16 2.2204460491536837829e-16 -1.0069344447037764778e-13
- joint left_sho_pitch: origin xyz=-0.0064000000000001278089 0.057999999999999600486 0.41249999999999986677 rpy=-1.570796326794871911 3.5360603334311235812e-14 -3.1415926535897371608 -> xyz=-0.0064000000000001781159 0.057999999999999808653 0.42079999999999984084 rpy=-1.570796326794871911 3.5360603334311235812e-14 -3.1415926535897371608
- joint neck: origin xyz=-0.0063999999999999838268 -5.2372852656669075105e-18 0.43249999999999999556 rpy=-3.141592653589793116 8.5053965662326763145e-17 1.57079632679489678 -> xyz=-0.0063999999999999820921 -4.4507968385753129991e-18 0.44079999999999996962 rpy=-3.141592653589793116 8.5053965662326763145e-17 1.57079632679489678
- joint right_ank_B31: origin xyz=-7.3725747729014301513e-18 -0.006438750500400436394 -1.3877787807814456755e-17 rpy=-1.5707963267948954478 0.16913440034160504011 5.0191724325132069355e-15 -> xyz=-6.0715321659188248304e-18 -0.006438750500400436394 -1.3877787807814456755e-17 rpy=-1.5707963267948954478 0.16913440034160504011 5.0191724325132069355e-15
- joint right_ank_B32: origin xyz=-1.6913553890773869171e-17 -0.0064387505004003531273 -1.3877787807814456755e-17 rpy=-1.5707963267948952257 -0.17993145005754265786 3.2634092460731900895e-15 -> xyz=-1.561251128379126385e-17 -0.0064387505004003531273 -1.3877787807814456755e-17 rpy=-1.5707963267948952257 -0.17993145005754265786 3.2634092460731900895e-15
- joint right_ank_act1: origin xyz=2.2722093427438722069e-06 1.6375789613221058971e-15 -0.072660031604109970305 rpy=-3.1415926535897806815 7.845419351877858644e-15 -2.2021168238260604433 -> xyz=2.2722093427421374834e-06 1.6375789613221058971e-15 -0.072660031604109970305 rpy=-3.1415926535897806815 7.845419351877858644e-15 -2.2021168238260604433
- joint right_hip_yaw: origin xyz=-0.011900000000000259329 -0.033999999999999981626 0.27720000000000000195 rpy=-2.2204460717259335277e-16 2.2204461793479381443e-16 -6.6849266279598662255e-15 -> xyz=-0.011900000000000261063 -0.033999999999999974687 0.28549999999999997602 rpy=-2.2204460717259335277e-16 2.2204461793479381443e-16 -6.6849266279598654366e-15
- joint right_sho_pitch: origin xyz=-0.0063999999999999916331 -0.057999999999999989064 0.4124999999999999778 rpy=-1.5707963267948972241 1.3877787807856806753e-15 6.3545304591998415249e-17 -> xyz=-0.006399999999999998572 -0.057999999999999982125 0.42079999999999995186 rpy=-1.5707963267948972241 1.3877787807856806753e-15 6.3545304591998415249e-17

Commit message: Fix the base walking

File: toddlerbot/robot_descriptions/assemblies/4R_body/4R_body.urdf (robot description, URDF)
Before this commit: robot 4R_body, 7 links, 6 joints
Links:
- link body_link: mass 1.3010345634555091632 -> 1.3010345634555100514
- link neck_link: mass 0.018378317023500283234 -> 0.018378317023500286703
Joints:
- joint head: origin xyz=0 0 -0.039999999999999980016 rpy=-3.6199375412562401434e-16 -2.4218742848029192401e-16 -5.5511151231257722251e-17 -> xyz=0 -6.505213034913026604e-19 -0.039999999999999980016 rpy=-3.6199375412562401434e-16 -2.4218742848029192401e-16 -5.5511151231257722251e-17
- joint left_hip_yaw: origin xyz=-0.011900000000000070244 0.033999999999999967748 0.28550000000000003153 rpy=-2.2204460494577687078e-16 2.2204460491536837829e-16 -1.0069344447037764778e-13 -> xyz=-0.006400000000000070563 0.033999999999999967748 0.28550000000000003153 rpy=-1.0062408617649953783e-14 -1.7373496713084857328e-15 -1.0702550091647256269e-13
- joint left_sho_pitch: origin xyz=-0.0064000000000001781159 0.057999999999999808653 0.42079999999999984084 rpy=-1.570796326794871911 3.5360603334311235812e-14 -3.1415926535897371608 -> xyz=-0.00090000000000018190449 0.058000000000000113964 0.42079999999999984084 rpy=-1.570796326794871911 3.5360603334311235812e-14 -3.1415926535897371608
- joint neck: origin xyz=-0.0063999999999999820921 -4.4507968385753129991e-18 0.44079999999999996962 rpy=-3.141592653589793116 8.5053965662326763145e-17 1.57079632679489678 -> xyz=-0.00089999999999998414602 -4.4507968385753129991e-18 0.44079999999999996962 rpy=-3.141592653589793116 8.5053965662326763145e-17 1.57079632679489678
- joint right_hip_yaw: origin xyz=-0.011900000000000261063 -0.033999999999999974687 0.28549999999999997602 rpy=-2.2204460717259335277e-16 2.2204461793479381443e-16 -6.6849266279598654366e-15 -> xyz=-0.0064000000000002613826 -0.033999999999999974687 0.28549999999999997602 rpy=-2.4175737836120826254e-16 2.1811947592303793928e-16 -1.3443908046660001512e-14
- joint right_sho_pitch: origin xyz=-0.006399999999999998572 -0.057999999999999982125 0.42079999999999995186 rpy=-1.5707963267948972241 1.3877787807856806753e-15 6.3545304591998415249e-17 -> xyz=-0.00090000000000000062589 -0.057999999999999982125 0.42079999999999995186 rpy=-1.5707963267948972241 1.3877787807856806753e-15 6.3545304591998415249e-17

File: toddlerbot/robot_descriptions/base/base.urdf (robot description, URDF)
Before this commit: robot base, 45 links, 44 joints
Links:
- link body_link: mass 1.3010345634555091632 -> 1.3010345634555100514
- link neck_link: mass 0.018378317023500283234 -> 0.018378317023500286703
Joints:
- joint head: origin xyz=0 0 -0.039999999999999980016 rpy=-3.6199375412562401434e-16 -2.4218742848029192401e-16 -5.5511151231257722251e-17 -> xyz=0 -6.505213034913026604e-19 -0.039999999999999980016 rpy=-3.6199375412562401434e-16 -2.4218742848029192401e-16 -5.5511151231257722251e-17
- joint left_hip_yaw: origin xyz=-0.011900000000000070244 0.033999999999999967748 0.28550000000000003153 rpy=-2.2204460494577687078e-16 2.2204460491536837829e-16 -1.0069344447037764778e-13 -> xyz=-0.006400000000000070563 0.033999999999999967748 0.28550000000000003153 rpy=-1.0062408617649953783e-14 -1.7373496713084857328e-15 -1.0702550091647256269e-13
- joint left_sho_pitch: origin xyz=-0.0064000000000001781159 0.057999999999999808653 0.42079999999999984084 rpy=-1.570796326794871911 3.5360603334311235812e-14 -3.1415926535897371608 -> xyz=-0.00090000000000018190449 0.058000000000000113964 0.42079999999999984084 rpy=-1.570796326794871911 3.5360603334311235812e-14 -3.1415926535897371608
- joint neck: origin xyz=-0.0063999999999999820921 -4.4507968385753129991e-18 0.44079999999999996962 rpy=-3.141592653589793116 8.5053965662326763145e-17 1.57079632679489678 -> xyz=-0.00089999999999998414602 -4.4507968385753129991e-18 0.44079999999999996962 rpy=-3.141592653589793116 8.5053965662326763145e-17 1.57079632679489678
- joint right_hip_yaw: origin xyz=-0.011900000000000261063 -0.033999999999999974687 0.28549999999999997602 rpy=-2.2204460717259335277e-16 2.2204461793479381443e-16 -6.6849266279598654366e-15 -> xyz=-0.0064000000000002613826 -0.033999999999999974687 0.28549999999999997602 rpy=-2.4175737836120826254e-16 2.1811947592303793928e-16 -1.3443908046660001512e-14
- joint right_sho_pitch: origin xyz=-0.006399999999999998572 -0.057999999999999982125 0.42079999999999995186 rpy=-1.5707963267948972241 1.3877787807856806753e-15 6.3545304591998415249e-17 -> xyz=-0.00090000000000000062589 -0.057999999999999982125 0.42079999999999995186 rpy=-1.5707963267948972241 1.3877787807856806753e-15 6.3545304591998415249e-17
