Commit message: Update humanoid gym

File: toddlerbot/robot_descriptions/toddlerbot_legs/toddlerbot_legs_isaac.urdf (robot description, URDF)
Before this commit: robot toddlerbot_legs, 37 links, 36 joints
Links:
- link 12lf: mass 0.044782197696050352054 -> 0.044782197690790462308
- link 12lf_2: mass 0.044782197696050352054 -> 0.044782197690790462308
- link 12lf_3: mass 0.044782197696050352054 -> 0.044782197690790462308
- link 12lf_4: mass 0.044782197696050358993 -> 0.044782197690790476186
- link 12lf_rod: mass 0.0025088292483592140175 -> 0.0025088292483592144512
- link 12lf_rod_2: mass 0.0025088292483592140175 -> 0.0025088292483592144512
- link 12lf_rod_3: mass 0.0025088292483592140175 -> 0.0025088292483592144512
- link 12lf_rod_4: mass 0.0025088292483592140175 -> 0.0025088292483592144512
- link 12lf_rod_end: mass 0.00085420491177815905965 -> 0.00085420491177815895123
- link 12lf_rod_end_2: mass 0.00085420491177815905965 -> 0.00085420491177815895123
- link 12lf_rod_end_3: mass 0.00085420491177815905965 -> 0.00085420491177815895123
- link 12lf_rod_end_4: mass 0.00085420491177815905965 -> 0.00085420491177815895123
- link ank_pitch_link: mass 0.0042238381753791605713 -> 0.0042238381753791614387
- link ank_pitch_link_2: mass 0.0042238381753791605713 -> 0.0042238381753791614387
- link ank_roll_link: mass 0.013844478784760248444 -> 0.020312412324461778801
- link ank_roll_link_2: mass 0.013844478784760248444 -> 0.020312412236862385784
- link ank_rr_link: mass 0.00044289790445047673732 -> 0.00042507093693768156772
- link ank_rr_link_2: mass 0.00044289790445047673732 -> 0.00042507093693768156772
- link ank_rr_link_3: mass 0.00044289790445047673732 -> 0.00042507093693768156772
- link ank_rr_link_4: mass 0.00044289790445047673732 -> 0.00042507093693768156772
- link ball_joint_ball: mass 4.4053796295264630609e-05 -> 4.4053796295264623832e-05
- link ball_joint_ball_2: mass 4.4053796295264630609e-05 -> 4.4053796295264623832e-05
- link ball_joint_ball_3: mass 4.4053796295264630609e-05 -> 4.4053796295264623832e-05
- link ball_joint_ball_4: mass 4.4053796295264630609e-05 -> 4.4053796295264623832e-05
- link ball_joint_container: mass 4.803735642533054869e-05 -> 4.8037356425330562243e-05
- link ball_joint_container_2: mass 4.803735642533054869e-05 -> 4.8037356425330562243e-05
- link ball_joint_container_3: mass 4.803735642533054869e-05 -> 4.8037356425330562243e-05
- link ball_joint_container_4: mass 4.803735642533054869e-05 -> 4.8037356425330562243e-05
- link hip_roll_link: mass 0.098012391483528679692 -> 0.098012391483528651936
- link hip_roll_link_2: mass 0.09801239148352869357 -> 0.098012391483528665814
- link hip_yaw_link: mass 0.0090258837370979193293 -> 0.009025883737097921064
- link hip_yaw_link_2: mass 0.0090258837370979193293 -> 0.009025883737097921064
- link left_calf_link: mass 0.016290616864051549878 -> 0.015782434194230747504
- link left_hip_pitch_link: mass 0.093882153942003054858 -> 0.093539065135968837983
- link right_calf_link: mass 0.016290630569901022595 -> 0.015779725212993943317
- link right_hip_pitch_link: mass 0.093882153558663708481 -> 0.09353906475262946385
Joints:
- joint left_ank_B11: origin xyz=0.0080000000000000123096 -0.014999999999999985567 0.028299999999999790601 rpy=-1.5707963267948918951 1.4696360140379163273 1.570796326794891673 -> xyz=0.0079999999999999949624 -0.015000000000000096589 0.028299999999999991829 rpy=-1.570796326794896558 1.5520170643097057628 1.5707963267950826314
- joint left_ank_B12: origin xyz=0.0080000000000000001665 -0.014999999999999985567 -0.011500000000000003275 rpy=-1.5707963267949205388 -1.469756662182277962 1.5707963267949025532 -> xyz=0.0080000000000000019013 -0.015000000000000041078 -0.011499999999999999806 rpy=-1.570796326794896558 -1.5521341097218244176 1.5707963267948896746
- joint left_ank_B21: origin xyz=6.9388939039072283776e-18 -2.7755575615628913511e-17 -0.01150000000000000154 rpy=1.570796326794896558 -1.4285697747625525356 1.5707963267948994446 -> xyz=-3.4694469519536141888e-18 -2.7755575615628913511e-17 -0.011499999999999999806 rpy=-1.570796326794896558 -1.5664147454872627829 -1.5707963267957041342
- joint left_ank_B22: origin xyz=0 0 -0.01150000000000000154 rpy=1.5707963267949021091 -1.4285463212680715728 -1.5707963267948938935 -> xyz=3.4694469519536141888e-18 0 -0.01150000000000000154 rpy=-1.570796326794896336 -1.5664376509754431854 1.570796326794866582
- joint left_ank_B31: origin xyz=4.336808689942017736e-19 -0.0064387505004003808828 0 rpy=-1.5707963267948970021 0.1691344003409792629 1.2463746926904215167e-14 -> xyz=0 -0.0064387505004003531273 -3.4694469519536141888e-18 rpy=-1.57079632679489678 0.16913440034090146402 5.8375589418798256921e-16
- joint left_ank_B32: origin xyz=-2.4286128663675299322e-17 -0.0064387505004003808828 0 rpy=-1.570796326794896558 -0.17993145005786467805 5.6818279199863494045e-15 -> xyz=2.498001805406602216e-16 -0.0064387505004004919051 -3.4694469519536141888e-18 rpy=-1.570796326794896558 -0.17993145005756983057 3.0408221168269646133e-14
- joint left_ank_R11: origin xyz=-0.0099999999999999967387 0.012500000000000011102 -0.033600000000000011802 rpy=-3.5821358734369027029e-16 -2.0703583441380111793e-15 -0.1011603127571137628 -> xyz=-0.018000000000000009048 0.016000000000000014211 -0.020599999999999996786 rpy=-4.1594268726375658989e-17 6.5315524930102152625e-16 -0.01877926248499593373
- joint left_ank_R12: origin xyz=0.010000000000000003678 0.012499999999999955591 -0.033600000000000004863 rpy=3.1415926535897606975 1.5562027335348888578e-14 -3.0405529889788582842 -> xyz=0.017999999999999995171 0.016000000000000014211 -0.020600000000000000255 rpy=3.1415926535897922278 7.4438972302667006905e-16 -3.1229304365180685643
- joint left_ank_R21: origin xyz=-6.9388939039072283776e-18 -0.0099999999999999533706 0 rpy=-1.570796326794896558 -1.4285697747629988452 1.5707963267949092145 -> xyz=0 -0.0099999999999999533706 0 rpy=1.570796326794896558 -1.5664147454868542209 -1.5707963267948135133
- joint left_ank_R22: origin xyz=6.9388939039072283776e-18 -0.010000000000000036637 6.9388939039072283776e-18 rpy=1.5707963267949194286 -1.4285463212677806943 -1.5707963267950313391 -> xyz=0 -0.0099999999999999533706 0 rpy=-1.570796326794896558 -1.5664376509758224376 1.570796326795195208
- joint left_ank_act1: origin xyz=2.2722093540906984632e-06 7.7021722333370234992e-16 -0.072660031604095037805 rpy=-3.1415926535896590011 8.173835939810196213e-14 -2.2021168238262767147 -> xyz=2.2722093531019060819e-06 5.1000870193718128576e-16 -0.074779998095377359091 rpy=-3.1415926535896590011 8.6569212672158331644e-14 -2.2021168238262673889
- joint left_ank_act2: origin xyz=2.2722093490027545082e-06 -7.7229889150487451843e-15 -0.07266003047881974819 rpy=-3.1415926535895000171 4.7493922909940523358e-14 -2.2021168238262776029 -> xyz=2.2722093474362992094e-06 -8.9372953482325101504e-15 -0.074779996992751340823 rpy=-3.1415926535895000171 6.172537580306697636e-14 -2.2021168238262789352
- joint left_ank_pitch: limit lower=-0.785398163397448279 upper=0.785398163397448279 effort=1 velocity=20 -> lower=-0.785398163397448279 upper=0.95993108859688125456 effort=1 velocity=20; origin xyz=7.2631635415802528961e-19 -0.099999999999999977796 -0.0061999999999999989148 rpy=-3.1415926535897922278 -4.216693940517171266e-15 -1.5707963267948972241 -> xyz=5.9135023084202893979e-19 -0.10000000000000006106 -0.0061999999999999989148 rpy=3.141592653589793116 3.3306690738944506007e-16 -1.5707963267948974462
- joint left_ank_roll: origin xyz=1.9984014443252817728e-15 0.0015000000000042093377 -0.014599999999997269676 rpy=-1.5707963267950535435 -1.5707963267944073937 0 -> xyz=3.0531133177191804862e-15 0.001500000000004121951 -0.014599999999997613151 rpy=-1.5707963267949702768 -1.5707963267946758457 0
- joint left_hip_pitch: origin xyz=-0.024000000716154958752 -0.019000000152441291756 -0.019000000152448955765 rpy=-1.5707963267944653474 1.5707963267948226171 0 -> xyz=-0.024000000716155274472 -0.019000000152442689944 -0.019000000152446339802 rpy=-1.5707963267945199703 1.5707963267948246155 0
- joint left_hip_roll: origin xyz=0.01900000000000030137 -3.3624037938346747648e-18 -0.026000000000000279832 rpy=3.141592653589793116 -1.570796326794573039 0 -> xyz=0.01900000000000030137 5.3821911112507180559e-16 -0.026000000000000168809 rpy=3.141592653589793116 -1.5707963267936781993 0
- joint left_hip_yaw: origin xyz=-0.0063999999999966045855 0.03399999999999939182 0.28550000000000008704 rpy=2.327572832560927136e-16 4.9789962508008699149e-17 -1.0650377544034614197e-13 -> xyz=-0.0063999999999966063202 0.033999999999999308553 0.28550000000000003153 rpy=2.3275728331677864905e-16 1.1102230242191363653e-16 -1.222458086656465435e-13
- joint left_knee: origin xyz=-6.5473275179360459098e-15 0.096000000000000071387 0.027400000000000535039 rpy=-3.141592653589783346 1.4838131564395688657e-16 6.5779908238917364858e-16 -> xyz=-8.1569325594195215653e-15 0.095999999999999391376 0.027400000000002110168 rpy=3.1415926535897917837 1.6653345451476814222e-16 -5.2069203968451419987e-17
- joint right_ank_B11: origin xyz=0.008000000000000003636 0.015000000000000013323 -0.011499999999999998071 rpy=1.570796326794896558 -1.469636014037899896 -1.5707963267948905628 -> xyz=0.0079999999999999984318 0.015000000000000041078 -0.01150000000000000154 rpy=1.570796326794896558 -1.5520170643097170871 -1.5707963267946734032
- joint right_ank_B12: origin xyz=0.0080000000000000365957 0.014999999999999985567 0.028300000000000158362 rpy=-1.570796326794896558 -1.469756662182680973 1.570796326794891451 -> xyz=0.008000000000000003636 0.015000000000000041078 0.028300000000000019584 rpy=-1.570796326794896558 -1.5521341097221632577 1.5707963267948059638
- joint right_ank_B21: origin xyz=6.9388939039072283776e-18 0 -0.01150000000000000154 rpy=1.570796326794896558 -1.4285697747626475707 1.5707963267948843455 -> xyz=0 -2.7755575615628913511e-17 -0.011500000000000006745 rpy=-1.570796326794896558 -1.5664147454871475418 -1.5707963267939402119
- joint right_ank_B22: origin xyz=0 0 -0.011499999999999999806 rpy=1.57079632679489678 -1.4285463212679265776 1.5707963267948943376 -> xyz=3.4694469519536141888e-18 0 -0.011499999999999998071 rpy=-1.57079632679489678 -1.5664376509754476263 -1.5707963267945079799
- joint right_ank_B31: origin xyz=9.1072982488782372457e-18 -0.0064387505004003808828 0 rpy=-1.5707963267948961139 0.16913440034171131621 -1.7599215475487529123e-15 -> xyz=6.9388939039072283776e-18 -0.0064387505004004086384 6.9388939039072283776e-18 rpy=-1.5707963267948970021 0.1691344003416279107 3.6048302674885136887e-16
- joint right_ank_B32: origin xyz=-8.6736173798840354721e-18 -0.0064387505004003531273 -1.3877787807814456755e-17 rpy=-1.5707963267948854558 -0.17993145005747521181 -6.9806032607149013267e-15 -> xyz=3.4694469519536141888e-18 -0.0064387505004004086384 -6.9388939039072283776e-18 rpy=-1.570796326794896558 -0.17993145005738314657 -8.7569826039094258121e-17
- joint right_ank_R11: origin xyz=-0.0099999999999999984734 0.012500000000000011102 -0.033599999999999997924 rpy=-2.3897964054427488116e-14 -3.8273675914490832965e-16 -0.10116031275657462463 -> xyz=-0.018000000000000005579 0.016000000000000014211 -0.020599999999999996786 rpy=-3.5360359477892277706e-16 8.2839943819914169726e-16 -0.018779262484754637164
- joint right_ank_R12: origin xyz=0.010000000000000003678 0.012499999999999955591 -0.033600000000000004863 rpy=-3.1415926535897709115 -4.1620274661327994973e-15 -3.0405529889776490293 -> xyz=0.01799999999999999864 0.016000000000000069722 -0.020600000000000003725 rpy=3.1415926535897922278 1.1785067659504147721e-15 -3.1229304365172114721
- joint right_ank_R21: origin xyz=0 -0.010000000000000008882 1.3877787807814456755e-17 rpy=-1.570796326794896558 -1.4285697747630956567 1.5707963267948958919 -> xyz=3.4694469519536141888e-18 -0.010000000000000008882 0 rpy=1.57079632679489678 -1.5664147454870704923 -1.5707963267947753216
- joint right_ank_R22: origin xyz=-6.9388939039072283776e-18 -0.0099999999999999811262 1.3877787807814456755e-17 rpy=1.570796326794896558 -1.428546321268451269 -1.570796326794896558 -> xyz=-3.4694469519536141888e-18 -0.0099999999999999533706 -3.4694469519536141888e-18 rpy=-1.570796326794896336 -1.5664376509754269762 1.5707963267952340658
- joint right_ank_act1: origin xyz=2.2722093427646888886e-06 1.7902346272080649214e-15 -0.072660031604104419189 rpy=-3.1415926535897806815 9.7899118131350707255e-15 -2.2021168238260933059 -> xyz=2.2722093412017030367e-06 1.8804402479588588903e-15 -0.074779998095388988677 rpy=-3.1415926535897829019 8.526808676235474948e-15 -2.2021168238260906413
- joint right_ank_act2: origin xyz=2.2722093383654301535e-06 -2.5118795932144166727e-15 -0.07266003047881591792 rpy=3.1415926535897926719 5.7157557368585280826e-16 -2.2021168238262842642 -> xyz=2.2722093371875529133e-06 -2.8553548414578244774e-15 -0.074779996992751840423 rpy=3.1415926535897922278 3.3072658899692120884e-15 -2.2021168238262864847
- joint right_ank_pitch: limit lower=-0.785398163397448279 upper=0.785398163397448279 effort=1 velocity=20 -> lower=-0.785398163397448279 upper=0.95993108859688125456 effort=1 velocity=20; origin xyz=1.0774845611827788694e-18 0.10000000000000003331 -0.0062000000000000006495 rpy=3.141592653589783346 -6.5431213406603904361e-15 -1.57079632679491632 -> xyz=5.0979769291920753058e-19 0.099999999999999977796 -0.0062000000000000023842 rpy=-3.1415926535897926719 5.5511151131695266928e-17 -1.5707963267946121189
- joint right_ank_roll: origin xyz=1.7486012637846215512e-15 0.001500000000009214015 -0.014599999999994360544 rpy=-1.5707963267952413933 1.570796326794632769 0 -> xyz=2.0816681711721685133e-15 0.0015000000000089284361 -0.014599999999994599936 rpy=-1.5707963267951812192 1.5707963267946736252 0
- joint right_hip_pitch: origin xyz=0.024000000358073002305 -0.019000000000011920548 -0.018999999847560570393 rpy=-1.5707963267950890707 -1.5707963267946420949 0 -> xyz=0.024000000358075784801 -0.019000000000012132184 -0.01899999984755619542 rpy=-1.5707963267951119413 -1.5707963267945823649 0
- joint right_hip_roll: origin xyz=0.018999999999999881567 -3.3500438889873688288e-18 -0.026000000000000002276 rpy=1.4130847605241333966e-30 1.5707963267948645836 0 -> xyz=0.018999999999999881567 -3.350043888987566044e-18 -0.026000000000000002276 rpy=2.9582283942363596652e-30 1.5707963267948799047 0
- joint right_hip_yaw: origin xyz=-0.0063999999999967962724 -0.034000000000000661637 0.28549999999999992051 rpy=1.2173498094910643509e-16 -6.1232339957301087894e-17 -5.033057304260250785e-13 -> xyz=-0.0063999999999967980072 -0.034000000000000668576 0.28549999999999992051 rpy=1.2173498094825229595e-16 9.8900267199457111713e-23 -3.0336177719551955022e-13
- joint right_knee: origin xyz=-2.892603788276459435e-15 0.095999999999999294231 0.027400000000000382383 rpy=-3.141592653589788231 -2.6961419186663855904e-16 -3.141592653589793116 -> xyz=-8.4133172564547814973e-15 0.095999999999998697486 0.027400000000003574274 rpy=3.1415926535897926719 9.3467860356166481656e-14 -3.1415926535895137839

Commit message: Update the config generation script

File: toddlerbot/robot_descriptions/toddlerbot_legs/toddlerbot_legs_isaac.urdf (robot description, URDF)
Before this commit: robot toddlerbot_legs, 37 links, 36 joints
Joints:
- joint left_ank_B11: limit lower=-0.785398163397448279 upper=0.785398163397448279 effort=1 velocity=20 -> lower=-0.785398163397448279 upper=0.785398163397448279 effort=10 velocity=20
- joint left_ank_B12: limit lower=-0.785398163397448279 upper=0.785398163397448279 effort=1 velocity=20 -> lower=-0.785398163397448279 upper=0.785398163397448279 effort=10 velocity=20
- joint left_ank_B21: limit lower=-0.785398163397448279 upper=0.785398163397448279 effort=1 velocity=20 -> lower=-0.785398163397448279 upper=0.785398163397448279 effort=10 velocity=20
- joint left_ank_B22: limit lower=-0.785398163397448279 upper=0.785398163397448279 effort=1 velocity=20 -> lower=-0.785398163397448279 upper=0.785398163397448279 effort=10 velocity=20
- joint left_ank_B31: limit lower=-0.785398163397448279 upper=0.785398163397448279 effort=1 velocity=20 -> lower=-0.785398163397448279 upper=0.785398163397448279 effort=10 velocity=20
- joint left_ank_B32: limit lower=-0.785398163397448279 upper=0.785398163397448279 effort=1 velocity=20 -> lower=-0.785398163397448279 upper=0.785398163397448279 effort=10 velocity=20
- joint left_ank_R11: limit lower=-1.570796326794896558 upper=1.570796326794896558 effort=1 velocity=20 -> lower=-1.570796326794896558 upper=1.570796326794896558 effort=10 velocity=20
- joint left_ank_R12: limit lower=-1.570796326794896558 upper=1.570796326794896558 effort=1 velocity=20 -> lower=-1.570796326794896558 upper=1.570796326794896558 effort=10 velocity=20
- joint left_ank_R21: limit lower=-1.570796326794896558 upper=1.570796326794896558 effort=1 velocity=20 -> lower=-1.570796326794896558 upper=1.570796326794896558 effort=10 velocity=20
- joint left_ank_R22: limit lower=-1.570796326794896558 upper=1.570796326794896558 effort=1 velocity=20 -> lower=-1.570796326794896558 upper=1.570796326794896558 effort=10 velocity=20
- joint left_ank_act1: limit lower=0 upper=0.040000000000000000833 effort=1 velocity=20 -> lower=0 upper=0.040000000000000000833 effort=10 velocity=20
- joint left_ank_act2: limit lower=0 upper=0.040000000000000000833 effort=1 velocity=20 -> lower=0 upper=0.040000000000000000833 effort=10 velocity=20
- joint left_ank_pitch: limit lower=-0.785398163397448279 upper=0.95993108859688125456 effort=1 velocity=20 -> lower=-0.785398163397448279 upper=0.95993108859688125456 effort=10 velocity=20
- joint left_ank_roll: limit lower=-0.785398163397448279 upper=0.785398163397448279 effort=1 velocity=20 -> lower=-0.785398163397448279 upper=0.785398163397448279 effort=10 velocity=20
- joint left_hip_pitch: limit lower=-1.570796326794896558 upper=1.570796326794896558 effort=1 velocity=20 -> lower=-1.570796326794896558 upper=1.570796326794896558 effort=10 velocity=20
- joint left_hip_roll: limit lower=-0.785398163397448279 upper=1.570796326794896558 effort=1 velocity=20 -> lower=-0.785398163397448279 upper=1.570796326794896558 effort=10 velocity=20
- joint left_hip_yaw: limit lower=-0.785398163397448279 upper=0.785398163397448279 effort=1 velocity=20 -> lower=-0.785398163397448279 upper=0.785398163397448279 effort=10 velocity=20
- joint left_knee: limit lower=0 upper=1.570796326794896558 effort=1 velocity=20 -> lower=0 upper=1.570796326794896558 effort=10 velocity=20
- joint right_ank_B11: limit lower=-0.785398163397448279 upper=0.785398163397448279 effort=1 velocity=20 -> lower=-0.785398163397448279 upper=0.785398163397448279 effort=10 velocity=20
- joint right_ank_B12: limit lower=-0.785398163397448279 upper=0.785398163397448279 effort=1 velocity=20 -> lower=-0.785398163397448279 upper=0.785398163397448279 effort=10 velocity=20
- joint right_ank_B21: limit lower=-0.785398163397448279 upper=0.785398163397448279 effort=1 velocity=20 -> lower=-0.785398163397448279 upper=0.785398163397448279 effort=10 velocity=20
- joint right_ank_B22: limit lower=-0.785398163397448279 upper=0.785398163397448279 effort=1 velocity=20 -> lower=-0.785398163397448279 upper=0.785398163397448279 effort=10 velocity=20
- joint right_ank_B31: limit lower=-0.785398163397448279 upper=0.785398163397448279 effort=1 velocity=20 -> lower=-0.785398163397448279 upper=0.785398163397448279 effort=10 velocity=20
- joint right_ank_B32: limit lower=-0.785398163397448279 upper=0.785398163397448279 effort=1 velocity=20 -> lower=-0.785398163397448279 upper=0.785398163397448279 effort=10 velocity=20
- joint right_ank_R11: limit lower=-1.570796326794896558 upper=1.570796326794896558 effort=1 velocity=20 -> lower=-1.570796326794896558 upper=1.570796326794896558 effort=10 velocity=20
- joint right_ank_R12: limit lower=-1.570796326794896558 upper=1.570796326794896558 effort=1 velocity=20 -> lower=-1.570796326794896558 upper=1.570796326794896558 effort=10 velocity=20
- joint right_ank_R21: limit lower=-1.570796326794896558 upper=1.570796326794896558 effort=1 velocity=20 -> lower=-1.570796326794896558 upper=1.570796326794896558 effort=10 velocity=20
- joint right_ank_R22: limit lower=-1.570796326794896558 upper=1.570796326794896558 effort=1 velocity=20 -> lower=-1.570796326794896558 upper=1.570796326794896558 effort=10 velocity=20
- joint right_ank_act1: limit lower=0 upper=0.040000000000000000833 effort=1 velocity=20 -> lower=0 upper=0.040000000000000000833 effort=10 velocity=20
- joint right_ank_act2: limit lower=0 upper=0.040000000000000000833 effort=1 velocity=20 -> lower=0 upper=0.040000000000000000833 effort=10 velocity=20
- joint right_ank_pitch: limit lower=-0.785398163397448279 upper=0.95993108859688125456 effort=1 velocity=20 -> lower=-0.785398163397448279 upper=0.95993108859688125456 effort=10 velocity=20
- joint right_ank_roll: limit lower=-0.785398163397448279 upper=0.785398163397448279 effort=1 velocity=20 -> lower=-0.785398163397448279 upper=0.785398163397448279 effort=10 velocity=20
- joint right_hip_pitch: limit lower=-1.570796326794896558 upper=1.570796326794896558 effort=1 velocity=20 -> lower=-1.570796326794896558 upper=1.570796326794896558 effort=10 velocity=20
- joint right_hip_roll: limit lower=-1.570796326794896558 upper=0.785398163397448279 effort=1 velocity=20 -> lower=-1.570796326794896558 upper=0.785398163397448279 effort=10 velocity=20
- joint right_hip_yaw: limit lower=-0.785398163397448279 upper=0.785398163397448279 effort=1 velocity=20 -> lower=-0.785398163397448279 upper=0.785398163397448279 effort=10 velocity=20
- joint right_knee: limit lower=-1.570796326794896558 upper=0 effort=1 velocity=20 -> lower=-1.570796326794896558 upper=0 effort=10 velocity=20
