Commit message: Add the base_legs robot

File: toddlerbot/robot_descriptions/assemblies/left_3R+RH5_leg/left_3R+RH5_leg.urdf (robot description, URDF)
Before this commit: robot left_3R+RH5_leg, 18 links, 17 joints
Links:
- removed link hip_pitch_link
- added link left_hip_pitch_link, mass 0.094115707917386950965; collision mesh filename=package:///meshes/left_hip_pitch_link_collision.stl; visual mesh filename=package:///meshes/left_hip_pitch_link_visual.stl
- link 12lf_2: mass 0.044782197696050345115 -> 0.044782197696050352054
- link 12lf_rod: mass 0.0026945559868381376359 -> 0.0025088292483592140175
- link 12lf_rod_2: mass 0.0026945559868381376359 -> 0.0025088292483592140175
- link 12lf_rod_end: mass 0.00066080012085386230676 -> 0.00085420491177815905965
- link 12lf_rod_end_2: mass 0.00066080012085386230676 -> 0.00085420491177815905965
- link ank_pitch_link: mass 0.0042238381753791614387 -> 0.0042238381753791605713
- link ank_roll_link: mass 0.014299508637166613578 -> 0.013844478784760248444
- link ank_rr_link: mass 0.00044289790445047684574 -> 0.00044289790445047673732
- link ank_rr_link_2: mass 0.00044289790445047684574 -> 0.00044289790445047673732
- link ball_joint_ball: mass 4.4053796295264623832e-05 -> 4.4053796295264630609e-05
- link ball_joint_ball_2: mass 4.4053796295264623832e-05 -> 4.4053796295264630609e-05
- link hip_yaw_link: mass 0.0081617461226117064832 -> 0.0090258837370979175946
- link left_calf_link: mass 0.016572094167120694774 -> 0.016616268752102307527
Joints:
- joint left_ank_B11: origin xyz=0.017999999999999957007 -0.01000000000000014766 0.028300000000000765515 rpy=-1.5707963267948972241 1.4719660848801743303 1.570796326794891451 -> xyz=0.0079999999999999966971 -0.015000000000000068834 0.028299999999999995298 rpy=-1.5707963267948998887 1.4686187149912932615 1.5707963267948792385
- joint left_ank_B12: origin xyz=0.018000000000000002109 -0.010000000000000008882 -0.011499999999999999806 rpy=-1.570796326794896558 -1.4752931174793231239 1.5707963267948954478 -> xyz=0.0080000000000000019013 -0.015000000000000013323 -0.011499999999999996336 rpy=-1.570796326794896558 -1.4687412243796080791 1.5707963267949098807
- joint left_ank_B21: origin xyz=7.8409501114151680667e-16 -1.1102230246251565404e-16 -0.011500000000000044909 rpy=1.5707963267948958919 -1.4871995686196806119 1.5707963267948610309 -> xyz=0 2.7755575615628913511e-17 -0.01150000000000000154 rpy=1.570796326794896558 -1.4274442472644790492 1.5707963267949169861
- joint left_ank_B22: origin xyz=-6.9388939039072283776e-18 -2.7755575615628913511e-17 -0.011499999999999999806 rpy=1.5707963267948872321 -1.4871998384670954696 -1.5707963267948854558 -> xyz=6.9388939039072283776e-18 0 -0.011500000000000003275 rpy=1.570796326794896558 -1.4274442651030925244 -1.5707963267949058839
- joint left_ank_B31: origin xyz=-3.4694469519536141888e-18 -0.0064387505004004086384 0 rpy=-1.570796326794896558 -5.457469122271992718e-06 -4.1571660558495781323e-16 -> xyz=-8.0794745893619790422e-16 -0.0064387505004003531273 0 rpy=-1.5707963267948918951 -0.0053985248584601302699 -5.6469137085305582343e-15
- joint left_ank_B32: origin xyz=3.4694469519536141888e-18 -0.0064387505004004641496 -1.3877787807814456755e-17 rpy=-1.5707963267948961139 -5.457468730707960001e-06 -1.2951865632219856922e-15 -> xyz=-1.8214596497756474491e-17 -0.0064387505004002976161 0 rpy=-1.570796326794896558 -0.0053985248584149493969 -1.0409444774216770496e-15
- joint left_ank_R11: origin xyz=-0.0099999999999999984734 0.012500000000000011102 -0.033000000000000008493 rpy=3.1415926535897908956 7.3034946203131872804e-17 -0.098830241914560454375 -> xyz=-0.010000000000000000208 0.01249999999999990008 -0.028000000000000010991 rpy=3.1415926535897775729 -1.2028245921984228645e-15 -0.10217761180348046424
- joint left_ank_R12: origin xyz=0.010000000000000003678 0.012500000000000066613 -0.033000000000000008493 rpy=-3.141592653589793116 4.6545838516711603543e-17 -3.0460894442741315302 -> xyz=0.010000000000000001943 0.012499999999999955591 -0.028000000000000004052 rpy=3.1415926535897895633 4.4869794467973275651e-15 -3.0395375511758455644
- joint left_ank_R21: origin xyz=0.0021000000000002752576 0.010000000000000036637 -0.0019000000000000058509 rpy=-1.570796326794896558 1.4871995686199779296 -1.5707963267949018871 -> xyz=0.0020999999999999977018 0.0099999999999998978595 -0.0018999999999999919731 rpy=-1.570796326794896558 1.427444247264781696 -1.5707963267949185404
- joint left_ank_R22: origin xyz=0.0021000000000000115796 -0.010000000000000036637 -0.001899999999999998912 rpy=-1.5707963267950195707 -1.4871998384676159422 -1.5707963267947853137 -> xyz=0.0020999999999999977018 -0.0099999999999999811262 -0.0018999999999999919731 rpy=-1.570796326794896558 -1.4274442651028091955 -1.5707963267949247577
- joint left_ank_act1: limit lower=-0.01799999999999999864 upper=0.01799999999999999864 effort=1 velocity=20 -> lower=0 upper=0.040000000000000000833 effort=1 velocity=20; origin xyz=2.272209342117637032e-06 -2.1996293675385913957e-15 -0.059356158967298844331 rpy=-3.141592653589793116 -9.2921664633026457838e-16 -0.63671356442004722886 -> xyz=2.2722093549316056682e-06 9.9920072216264088638e-16 -0.072674213012071053885 rpy=-3.1415926535896594451 9.2998178113314070509e-14 -2.2021168238262620598
- joint left_ank_act2: limit lower=-0.01799999999999999864 upper=0.01799999999999999864 effort=1 velocity=20 -> lower=0 upper=0.040000000000000000833 effort=1 velocity=20; origin xyz=2.2722093409414945153e-06 -1.7347234759768070944e-15 -0.05935645944356465753 rpy=3.141592653589793116 2.5208502705617295898e-15 -0.63671356442004545251 -> xyz=2.2722093494268943981e-06 -6.6960326172704753844e-15 -0.072674224000365938991 rpy=-3.1415926535895000171 6.1912461081019981423e-14 -2.2021168238262793793
- joint left_ank_pitch: origin xyz=4.2143614023597344721e-19 -0.09999999999999995004 -0.0062000000000000023842 rpy=3.1415926535897074068 -7.168818208916126976e-14 -1.5707963267948470421 -> xyz=1.423878333410664658e-18 -0.10000000000000000555 -0.0061999999999999989148 rpy=-3.1415926535897842342 8.6597395925459892621e-15 -1.5707963267949183184
- joint left_ank_roll: origin xyz=3.3306690738754696213e-16 -0.0061000000000003698833 -0.014600000000000704428 rpy=-1.5707963267949007768 -1.5707963267947875341 0 -> xyz=3.8857805861880478915e-16 -0.0060999999999999795705 -0.014599999999999386038 rpy=-1.5707963267948443775 -1.5707963267947531172 0
- joint left_hip_pitch: child hip_pitch_link -> left_hip_pitch_link; origin xyz=-0.024000000716140678508 -0.019000000152444841001 -0.019000000152450791102 rpy=-1.5707963267948210628 1.5707963267948126251 0 -> xyz=-0.024000000716150882152 -0.019000000152441572782 -0.019000000152448091872 rpy=-1.5707963267945472818 1.5707963267948001906 0
- joint left_hip_roll: origin xyz=0.019000000000000304839 -5.0328333128562291641e-18 -0.025000000000000268535 rpy=3.141592653589793116 -1.5707963267948947816 0 -> xyz=0.019000000000000304839 -3.3624037938353715663e-18 -0.026000000000000279832 rpy=3.141592653589793116 -1.5707963267948512609 0
- joint left_knee: limit lower=-1.570796326794896558 upper=1.570796326794896558 effort=1 velocity=20 -> lower=-1.570796326794896558 upper=2.2689280275926284602 effort=1 velocity=20; origin xyz=-4.686453338044572818e-15 0.097999999999999976019 0.027400000000003393863 rpy=-3.1415926535897620298 -6.106988965093026078e-15 -6.2039230811899877997e-14 -> xyz=-3.1353220349901300315e-15 0.095999999999999724443 0.027399999999999993805 rpy=-3.1415926535897926719 -2.5420496495350503733e-17 4.2811095712787448488e-16; parent hip_pitch_link -> left_hip_pitch_link

File: toddlerbot/robot_descriptions/assemblies/right_3R+RH5_leg/right_3R+RH5_leg.urdf (robot description, URDF)
Before this commit: robot right_3R+RH5_leg, 18 links, 17 joints
Links:
- removed link hip_pitch_link
- added link right_hip_pitch_link, mass 0.094115687342860077091; collision mesh filename=package:///meshes/right_hip_pitch_link_collision.stl; visual mesh filename=package:///meshes/right_hip_pitch_link_visual.stl
- link 12lf: mass 0.044782197696050345115 -> 0.044782197696050352054
- link 12lf_2: mass 0.044782197696050365932 -> 0.044782197696050358993
- link 12lf_rod: mass 0.0026945559868381376359 -> 0.0025088292483592140175
- link 12lf_rod_2: mass 0.0026945559868381376359 -> 0.0025088292483592140175
- link 12lf_rod_end: mass 0.00066080012085386230676 -> 0.00085420491177815905965
- link 12lf_rod_end_2: mass 0.00066080012085386230676 -> 0.00085420491177815905965
- link ank_pitch_link: mass 0.0042238381753791614387 -> 0.0042238381753791605713
- link ank_roll_link: mass 0.014299508637166613578 -> 0.013844478784760248444
- link ank_rr_link: mass 0.00044289790445047684574 -> 0.00044289790445047673732
- link ank_rr_link_2: mass 0.00044289790445047684574 -> 0.00044289790445047673732
- link ball_joint_ball: mass 4.4053796295264623832e-05 -> 4.4053796295264630609e-05
- link ball_joint_ball_2: mass 4.4053796295264623832e-05 -> 4.4053796295264630609e-05
- link hip_yaw_link: mass 0.0081617461226117064832 -> 0.0090258837370979175946
- link right_calf_link: mass 0.016572091442033146796 -> 0.016616299594005391055
Joints:
- joint right_ank_B11: origin xyz=0.018000000000000015987 0.010000000000000036637 -0.011499999999999994602 rpy=1.5707963267948974462 -1.4719660848800855124 -1.570796326794896336 -> xyz=0.008000000000000003636 0.015000000000000013323 -0.01150000000000000501 rpy=1.57079632679489678 -1.4686187149913361161 -1.5707963267948945596
- joint right_ank_B12: origin xyz=0.018000000000000002109 0.010000000000000036637 0.028300000000000012645 rpy=-1.5707963267948974462 -1.4752931174794650104 1.5707963267948936714 -> xyz=0.0079999999999990304561 0.015000000000000374145 0.028300000000000304079 rpy=-1.570796326794896558 -1.4687412243800435085 1.5707963267949029973
- joint right_ank_B21: origin xyz=-6.9388939039072283776e-18 0 -0.011499999999999992867 rpy=1.570796326794896558 -1.4871995686197141406 1.5707963267948958919 -> xyz=0 0 -0.011499999999999996336 rpy=1.570796326794896558 -1.4274442472645434421 1.5707963267948954478
- joint right_ank_B22: origin xyz=0 -2.7755575615628913511e-17 -0.011500000000000003275 rpy=1.570796326794896558 -1.4871998384672124871 1.5707963267948923392 -> xyz=-9.0205620750793968909e-17 -5.5511151231257827021e-16 -0.011500000000000809922 rpy=1.5707963267949021091 -1.4274442651029393136 1.5707963267948958919
- joint right_ank_B31: origin xyz=0 -0.0064387505004004086384 6.9388939039072283776e-18 rpy=-1.570796326794896558 -5.4574696529115381853e-06 -1.2331483706146518492e-15 -> xyz=8.2399365108898336985e-18 -0.006438750500400436394 2.5673907444456744997e-16 rpy=-1.570796326794896558 -0.0053985248578861414967 1.6676878818581557235e-16
- joint right_ank_B32: origin xyz=0 -0.0064387505004004086384 0 rpy=-1.570796326794896558 -5.4574689504429525655e-06 -5.0339227696192602828e-16 -> xyz=1.0408340855860842566e-17 -0.006438750500400436394 0 rpy=-1.57079632679489678 -0.0053985248581224047626 2.4993140229822924443e-16
- joint right_ank_R11: origin xyz=-0.010000000000000112965 0.012500000000000233147 -0.032999999999998946842 rpy=3.1415926535897922278 -2.5232420665482256888e-16 -0.098830241914703576001 -> xyz=-0.010000000000000165007 0.012500000000000260902 -0.027999999999999313632 rpy=-3.1415926535897926719 -6.3673174173468030794e-17 -0.102177611803432003
- joint right_ank_R12: origin xyz=0.0099999999999998891859 0.012500000000000066613 -0.032999999999998946842 rpy=-3.141592653589793116 -1.1886010661269619878e-15 -3.0460894442739978594 -> xyz=0.010000000000000003678 0.012499999999999983347 -0.028000000000000014461 rpy=3.141592653589793116 1.4948154307943495876e-16 -3.0395375511749724851
- joint right_ank_R21: origin xyz=0.0021000000000001434186 0.010000000000000230926 -0.0018999999999989442001 rpy=-1.5707963267948970021 1.4871995686198307141 -1.5707963267948983344 -> xyz=0.0020999999999992344235 0.010000000000000036637 -0.0019000000000000127898 rpy=-1.570796326794896558 1.4274442472646977631 -1.570796326794901665
- joint right_ank_R22: origin xyz=0.0020999999999999074962 -0.010000000000000119904 -0.0018999999999989372612 rpy=-1.5707963267948956698 -1.487199838467331281 -1.5707963267948870101 -> xyz=0.0021000000000000115796 -0.010000000000000008882 -0.001899999999999998912 rpy=-1.57079632679489678 -1.4274442651030334606 -1.5707963267948972241
- joint right_ank_act1: limit lower=-0.01799999999999999864 upper=0.01799999999999999864 effort=1 velocity=20 -> lower=0 upper=0.040000000000000000833 effort=1 velocity=20; origin xyz=2.2722093427941791877e-06 9.92261828258733658e-16 -0.059356158967292543815 rpy=-3.1415926535897837901 -1.2238359105881652741e-14 -0.63671356441985882402 -> xyz=2.2722093427881076555e-06 1.3183898417423733918e-15 -0.072674213012081267937 rpy=-3.1415926535897806815 9.5856772270727916853e-15 -2.2021168238260924177
- joint right_ank_act2: limit lower=-0.01799999999999999864 upper=0.01799999999999999864 effort=1 velocity=20 -> lower=0 upper=0.040000000000000000833 effort=1 velocity=20; origin xyz=2.2722093411253752038e-06 -2.4008572907519010187e-15 -0.059356459443579534518 rpy=-3.1415926535897926719 9.0510831053370240348e-16 -0.63671356442005022647 -> xyz=2.2722093417481409316e-06 -2.4008572907519010187e-15 -0.072674224000375264865 rpy=3.1415926535897922278 -4.7750794099672222252e-16 -2.2021168238262847083
- joint right_ank_pitch: origin xyz=-1.0422817820682455029e-15 0.10000000000000003331 -0.0062000000000001706524 rpy=-3.1415926535897900074 3.0234911913779407472e-15 -1.5707963267948836794 -> xyz=6.9626594985130732316e-16 0.099999999999999644729 -0.006199999999999853198 rpy=-3.1415926535897891192 -1.0660034804367828672e-14 -1.5707963267948825692
- joint right_ank_roll: origin xyz=1.1102230246251565404e-15 -0.006100000000001146172 -0.014600000000001599545 rpy=-1.5707963267948990005 1.5707963267948332753 0 -> xyz=1.7763568394002504647e-15 -0.0061000000000006751946 -0.014600000000001986389 rpy=-1.5707963267949152097 1.5707963267947568919 0
- joint right_hip_pitch: child hip_pitch_link -> right_hip_pitch_link; origin xyz=-0.024000000716145990232 -0.019000000152457986735 -0.019000000152453767888 rpy=-1.5707963267951823294 1.5707963267947557817 0 -> xyz=-0.024000000716145983293 -0.019000000152457983266 -0.019000000152453771357 rpy=-1.5707963267951818853 1.5707963267947633312 0
- joint right_hip_roll: origin xyz=-0.018999999999999885036 -5.020473408011439263e-18 -0.025000000000000001388 rpy=1.4827462901121851002e-29 -1.5707963267947766539 0 -> xyz=-0.018999999999999881567 -3.3500438889881561489e-18 -0.026000000000000002276 rpy=-4.6567077935502810538e-31 -1.5707963267948825692 0
- joint right_knee: origin xyz=-2.5483606178382506831e-15 0.097999999999999684586 0.027399999999999827272 rpy=3.1415926535897926719 -1.2487298519101510075e-16 -3.141592653589788231 -> xyz=-2.4092426568589641265e-15 0.095999999999999835465 0.027399999999999306854 rpy=3.1415926535897913396 -1.687018580240030462e-16 3.1415926535897922278; parent hip_pitch_link -> right_hip_pitch_link
