Commit message: Update the base_legs robot

File: toddlerbot/robot_descriptions/assemblies/left_3R+RH5_leg/left_3R+RH5_leg.urdf (robot description, URDF)
Before this commit: robot left_3R+RH5_leg, 18 links, 17 joints
Links:
- link ank_roll_link: mass 0.013844478784760248444 -> 0.013844478784760253648
- link hip_yaw_link: mass 0.0090258837370979175946 -> 0.009025883737097921064
- link left_hip_pitch_link: mass 0.094115707917386950965 -> 0.094084588454108858402
Joints:
- joint left_ank_B11: origin xyz=0.0079999999999999966971 -0.015000000000000068834 0.028299999999999995298 rpy=-1.5707963267948998887 1.4686187149912932615 1.5707963267948792385 -> xyz=0.0079999999999999966971 -0.015000000000000179856 0.028300000000000005707 rpy=-1.570796326794896558 1.4686290291020840382 1.5707963267948819031
- joint left_ank_B12: origin xyz=0.0080000000000000019013 -0.015000000000000013323 -0.011499999999999996336 rpy=-1.570796326794896558 -1.4687412243796080791 1.5707963267949098807 -> xyz=0.008000000000000003636 -0.015000000000000124345 -0.01149999999999918622 rpy=-1.570796326794896558 -1.4687304067506412597 1.5707963267949098807
- joint left_ank_B21: origin xyz=0 2.7755575615628913511e-17 -0.01150000000000000154 rpy=1.570796326794896558 -1.4274442472644790492 1.5707963267949169861 -> xyz=6.9388939039072283776e-18 -2.7755575615628913511e-17 -0.011499999999999994602 rpy=1.57079632679489678 -1.4274634743672511838 1.570796326794916542
- joint left_ank_B22: origin xyz=6.9388939039072283776e-18 0 -0.011500000000000003275 rpy=1.570796326794896558 -1.4274442651030925244 -1.5707963267949058839 -> xyz=-1.3877787807814456755e-17 8.3266726846886740532e-17 -0.011500000000000011949 rpy=1.570796326794896558 -1.4274430275990750427 -1.570796326794906328
- joint left_ank_B31: origin xyz=-8.0794745893619790422e-16 -0.0064387505004003531273 0 rpy=-1.5707963267948918951 -0.0053985248584601302699 -5.6469137085305582343e-15 -> xyz=-1.4831885719601700657e-16 -0.0064387505004003253717 -6.9388939039072283776e-18 rpy=-1.570796326794896558 0.16912328473440299548 -4.2800865129067981483e-15
- joint left_ank_B32: origin xyz=-1.8214596497756474491e-17 -0.0064387505004002976161 0 rpy=-1.570796326794896558 -0.0053985248584149493969 -1.0409444774216770496e-15 -> xyz=1.7347234759768070944e-17 -0.0064387505004004641496 1.3877787807814456755e-17 rpy=-1.5707963267948836794 -0.17992034540981183266 -3.9922693705457534994e-15
- joint left_ank_R11: origin xyz=-0.010000000000000000208 0.01249999999999990008 -0.028000000000000010991 rpy=3.1415926535897775729 -1.2028245921984228645e-15 -0.10217761180348046424 -> xyz=-0.010000000000000000208 0.012499999999999955591 -0.028000000000000004052 rpy=3.1415926535897775729 -1.1742161333363301013e-15 -0.10225158937860563679
- joint left_ank_R12: origin xyz=0.010000000000000001943 0.012499999999999955591 -0.028000000000000004052 rpy=3.1415926535897895633 4.4869794467973275651e-15 -3.0395375511758455644 -> xyz=0.010000000000000001943 0.01249999999999990008 -0.027999999999999948541 rpy=3.1415926535897895633 4.4319359555376638558e-15 -3.0396078498296592585
- joint left_ank_R21: origin xyz=0.0020999999999999977018 0.0099999999999998978595 -0.0018999999999999919731 rpy=-1.570796326794896558 1.427444247264781696 -1.5707963267949185404 -> xyz=0.0021000000000000115796 0.010000000000000064393 -0.0018999999999999919731 rpy=-1.570796326794896558 1.4273561685593663118 -1.5707963267949194286
- joint left_ank_R22: origin xyz=0.0020999999999999977018 -0.0099999999999999811262 -0.0018999999999999919731 rpy=-1.570796326794896558 -1.4274442651028091955 -1.5707963267949247577 -> xyz=0.0021000000000000115796 -0.010000000000000092149 -0.001899999999999929523 rpy=-1.5707963267948974462 -1.4273357206756709381 -1.5707963267949238695
- joint left_ank_act1: origin xyz=2.2722093549316056682e-06 9.9920072216264088638e-16 -0.072674213012071053885 rpy=-3.1415926535896594451 9.2998178113314070509e-14 -2.2021168238262620598 -> xyz=2.272209354975407436e-06 9.4368957093138305936e-16 -0.072676675805820711851 rpy=-3.1415926535896590011 9.257153768608790258e-14 -2.2021168238262611716
- joint left_ank_act2: origin xyz=2.2722093494268943981e-06 -6.6960326172704753844e-15 -0.072674224000365938991 rpy=-3.1415926535895000171 6.1912461081019981423e-14 -2.2021168238262793793 -> xyz=2.2722093495249062745e-06 -6.7446048745978259831e-15 -0.072678522047017385388 rpy=-3.1415926535895004612 6.2111251208581937571e-14 -2.2021168238262802674
- joint left_ank_pitch: origin xyz=1.423878333410664658e-18 -0.10000000000000000555 -0.0061999999999999989148 rpy=-3.1415926535897842342 8.6597395925459892621e-15 -1.5707963267949183184 -> xyz=1.6466858937503582328e-18 -0.099999999999999922284 -0.0062000000000000058537 rpy=-3.1415926535897842342 8.6597368124280298137e-15 -1.5709041950953850364
- joint left_ank_roll: origin xyz=3.8857805861880478915e-16 -0.0060999999999999795705 -0.014599999999999386038 rpy=-1.5707963267948443775 -1.5707963267947531172 0 -> xyz=3.3306690738754696213e-16 -0.0060999999999999726316 -0.014599999999999384304 rpy=-1.5707963257530275225 -1.5707136234809810915 -1.1504969698363094907e-09
- joint left_hip_pitch: origin xyz=-0.024000000716150882152 -0.019000000152441572782 -0.019000000152448091872 rpy=-1.5707963267945472818 1.5707963267948001906 0 -> xyz=-0.024000000716150875213 -0.01900000015244158319 -0.019000000152448091872 rpy=-1.5707963267945472818 1.5707963267948001906 0
- joint left_hip_roll: origin xyz=0.019000000000000304839 -3.3624037938353715663e-18 -0.026000000000000279832 rpy=3.141592653589793116 -1.5707963267948512609 0 -> xyz=0.019000000000000304839 -3.3605706708588417072e-18 -0.026000000000000279832 rpy=1.5707963267908973126 -1.5707806634981131833 1.5707963268130720191
- joint left_knee: origin xyz=-3.1353220349901300315e-15 0.095999999999999724443 0.027399999999999993805 rpy=-3.1415926535897926719 -2.5420496495350503733e-17 4.2811095712787448488e-16 -> xyz=-3.1366467205128203278e-15 0.095999999999999752198 0.027400000000000007683 rpy=-3.1415926535897926719 -2.5420496490693392505e-17 -8.4866560936749634e-15

File: toddlerbot/robot_descriptions/assemblies/no_body/no_body.urdf (robot description, URDF)
Before this commit: robot no_body, 4 links, 3 joints
Links:
- link left_3r+rh5_leg: mass 0.33319901067697282881 -> 0.33316789121369472237
- link right_3r+rh5_leg: mass 0.33319902094434905582 -> 0.33316790148107094938
Joints:
- joint left_hip_yaw: origin xyz=-0.0063999999999997730579 0.033999999999999780398 0.28550000000000019806 rpy=1.2173498077223837207e-16 -0 1.3877787807345010561e-17 -> xyz=-0.0063999999999966028508 0.033999999999999308553 0.28550000000000008704 rpy=1.2173498077216098975e-16 -2.7428229896967586736e-14 -8.3846071870935304412e-14
- joint right_hip_yaw: origin xyz=-0.0063999999999996715766 -0.034000000000000092648 0.28550000000000014255 rpy=1.2173498077030393722e-16 -4.683327753701002654e-30 2.5887568767631957634e-14 -> xyz=-0.006399999999996792803 -0.034000000000000661637 0.28549999999999997602 rpy=1.2173498094410956825e-16 -2.7428229798067236768e-14 -5.0714987764877150767e-13

File: toddlerbot/robot_descriptions/assemblies/right_3R+RH5_leg/right_3R+RH5_leg.urdf (robot description, URDF)
Before this commit: robot right_3R+RH5_leg, 18 links, 17 joints
Links:
- link ank_roll_link: mass 0.013844478784760248444 -> 0.013844478784760253648
- link hip_yaw_link: mass 0.0090258837370979175946 -> 0.009025883737097921064
- link right_hip_pitch_link: mass 0.094115687342860077091 -> 0.094084567879581956773
Joints:
- joint right_ank_B11: origin xyz=0.008000000000000003636 0.015000000000000013323 -0.01150000000000000501 rpy=1.57079632679489678 -1.4686187149913361161 -1.5707963267948945596 -> xyz=0.007999999999999972411 0.014999999999999957812 -0.011500000000000010214 rpy=1.5707963267948978903 -1.4686162729650020786 -1.5707963267948970021
- joint right_ank_B12: origin xyz=0.0079999999999990304561 0.015000000000000374145 0.028300000000000304079 rpy=-1.570796326794896558 -1.4687412243800435085 1.5707963267949029973 -> xyz=0.0079999999999997000594 0.015000000000000290878 0.02830000000000029714 rpy=-1.5707963267948978903 -1.468735614201923223 1.5707963267949029973
- joint right_ank_B21: origin xyz=0 0 -0.011499999999999996336 rpy=1.570796326794896558 -1.4274442472645434421 1.5707963267948954478 -> xyz=-2.0816681711721685133e-17 1.1102230246251565404e-16 -0.011499999999999998071 rpy=1.570796326794896558 -1.4274562579810237128 1.5707963267948950037
- joint right_ank_B22: origin xyz=-9.0205620750793968909e-17 -5.5511151231257827021e-16 -0.011500000000000809922 rpy=1.5707963267949021091 -1.4274442651029393136 1.5707963267948958919 -> xyz=-1.3877787807814456755e-17 -8.3266726846886740532e-17 -0.011499999999999991132 rpy=1.57079632679489678 -1.4274330297239778975 1.5707963267949012209
- joint right_ank_B31: origin xyz=8.2399365108898336985e-18 -0.006438750500400436394 2.5673907444456744997e-16 rpy=-1.570796326794896558 -0.0053985248578861414967 1.6676878818581557235e-16 -> xyz=-1.3010426069826053208e-18 -0.0064387505004002698605 6.9388939039072283776e-18 rpy=-1.570796326794896558 0.16913440034154619829 2.2885625266571218396e-16
- joint right_ank_B32: origin xyz=1.0408340855860842566e-17 -0.006438750500400436394 0 rpy=-1.57079632679489678 -0.0053985248581224047626 2.4993140229822924443e-16 -> xyz=-1.5178830414797062076e-17 -0.006438750500400436394 1.3877787807814456755e-17 rpy=-1.5707963267948854558 -0.17993145005756266963 -2.2505490007573420062e-15
- joint right_ank_R11: origin xyz=-0.010000000000000165007 0.012500000000000260902 -0.027999999999999313632 rpy=-3.1415926535897926719 -6.3673174173468030794e-17 -0.102177611803432003 -> xyz=-0.0099999999999999932693 0.012500000000000038858 -0.02800000000000008038 rpy=-3.1415926535897926719 -7.9041717877712374794e-16 -0.10218566393336031561
- joint right_ank_R12: origin xyz=0.010000000000000003678 0.012499999999999983347 -0.028000000000000014461 rpy=3.141592653589793116 1.4948154307943495876e-16 -3.0395375511749724851 -> xyz=0.0099999999999999967387 0.012499999999999761302 -0.02800000000000008038 rpy=-3.141592653589793116 2.6793361964555018776e-16 -3.0395375511005577884
- joint right_ank_R21: origin xyz=0.0020999999999992344235 0.010000000000000036637 -0.0019000000000000127898 rpy=-1.570796326794896558 1.4274442472646977631 -1.570796326794901665 -> xyz=0.0021000000000000254574 0.010000000000000092149 -0.0018999999999999919731 rpy=-1.57079632679489678 1.4274562579811747032 -1.570796326794901665
- joint right_ank_R22: origin xyz=0.0021000000000000115796 -0.010000000000000008882 -0.001899999999999998912 rpy=-1.57079632679489678 -1.4274442651030334606 -1.5707963267948972241 -> xyz=0.0021000000000000185185 -0.010000000000000203171 -0.0019000000000000336065 rpy=-1.5707963267948961139 -1.4274330297240631626 -1.5707963267948974462
- joint right_ank_act1: origin xyz=2.2722093427881076555e-06 1.3183898417423733918e-15 -0.072674213012081267937 rpy=-3.1415926535897806815 9.5856772270727916853e-15 -2.2021168238260924177 -> xyz=2.2722093427785666764e-06 1.2698175844150227931e-15 -0.072674150483189009497 rpy=-3.1415926535897811256 9.814572829871540247e-15 -2.2021168238260906413
- joint right_ank_act2: origin xyz=2.2722093417481409316e-06 -2.4008572907519010187e-15 -0.072674224000375264865 rpy=3.1415926535897922278 -4.7750794099672222252e-16 -2.2021168238262847083 -> xyz=2.2722093417776312307e-06 -2.3800406090401793335e-15 -0.072674285805652133474 rpy=3.141592653589793116 -4.1997988128928857096e-16 -2.2021168238262838202
- joint right_ank_pitch: origin xyz=6.9626594985130732316e-16 0.099999999999999644729 -0.006199999999999853198 rpy=-3.1415926535897891192 -1.0660034804367828672e-14 -1.5707963267948825692 -> xyz=1.1774009739933720541e-18 0.099999999999999922284 -0.0061999999999999937106 rpy=-3.141592653589793116 3.885801455584734555e-16 -1.5707963267948825692
- joint right_ank_roll: origin xyz=1.7763568394002504647e-15 -0.0061000000000006751946 -0.014600000000001986389 rpy=-1.5707963267949152097 1.5707963267947568919 0 -> xyz=1.7763568394002504647e-15 -0.0061000000000006751946 -0.014600000000001986389 rpy=1.5707963281806591738 1.5707907166914047981 -3.1415926522336965476
- joint right_hip_pitch: origin xyz=-0.024000000716145983293 -0.019000000152457983266 -0.019000000152453771357 rpy=-1.5707963267951818853 1.5707963267947633312 0 -> xyz=-0.024000000716145986762 -0.019000000152457990205 -0.019000000152453774827 rpy=-1.5707963267951818853 1.5707963267947633312 0
- joint right_hip_roll: origin xyz=-0.018999999999999881567 -3.3500438889881561489e-18 -0.026000000000000002276 rpy=-4.6567077935502810538e-31 -1.5707963267948825692 0 -> xyz=-0.018999999999999885036 -3.3499987806511678644e-18 -0.026000000000000002276 rpy=-1.5707963266839728433 -1.5707907166912637997 1.5707963266641831179
- joint right_knee: origin xyz=-2.4092426568589641265e-15 0.095999999999999835465 0.027399999999999306854 rpy=3.1415926535897913396 -1.687018580240030462e-16 3.1415926535897922278 -> xyz=-2.4109230505694711738e-15 0.095999999999999821587 0.027399999999999948702 rpy=3.141592653589793116 -1.6870185802395130185e-16 3.1415926535897922278
