Commit message: Update sysID for the ankle

File: toddlerbot/robot_descriptions/assemblies/left_3R+RH5_leg/left_3R+RH5_leg.urdf (robot description, URDF)
Before this commit: robot left_3R+RH5_leg, 18 links, 17 joints
Links:
- link 12lf: mass 0.044782197696050352054 -> 0.044782197690790462308
- link 12lf_2: mass 0.044782197696050352054 -> 0.044782197690790462308
- link 12lf_rod: mass 0.0025088292483592140175 -> 0.0025088292483592144512
- link 12lf_rod_2: mass 0.0025088292483592140175 -> 0.0025088292483592144512
- link 12lf_rod_end: mass 0.00085420491177815905965 -> 0.00085420491177815895123
- link 12lf_rod_end_2: mass 0.00085420491177815905965 -> 0.00085420491177815895123
- link ank_pitch_link: mass 0.0042238381753791605713 -> 0.0042238381753791614387
- link ank_roll_link: mass 0.013844478784760248444 -> 0.021210605042023062544
- link ank_rr_link: mass 0.00044289790445047673732 -> 0.00042507093693768156772
- link ank_rr_link_2: mass 0.00044289790445047673732 -> 0.00042507093693768156772
- link ball_joint_ball: mass 4.4053796295264630609e-05 -> 4.4053796295264623832e-05
- link ball_joint_ball_2: mass 4.4053796295264630609e-05 -> 4.4053796295264623832e-05
- link ball_joint_container: mass 4.803735642533054869e-05 -> 4.8037356425330562243e-05
- link ball_joint_container_2: mass 4.803735642533054869e-05 -> 4.8037356425330562243e-05
- link hip_roll_link: mass 0.098012391483528679692 -> 0.098012391483528651936
- link hip_yaw_link: mass 0.0090258837370979193293 -> 0.009025883737097921064
- link left_hip_pitch_link: mass 0.093882153942003054858 -> 0.093539065135968851861
Joints:
- joint left_ank_B11: origin xyz=0.0080000000000000123096 -0.014999999999999985567 0.028299999999999790601 rpy=-1.5707963267948918951 1.4696360140379163273 1.570796326794891673 -> xyz=0.0080000000000000643513 -0.015000000000000235367 0.028299999999999957134 rpy=-1.570796326794896558 1.4696360140379425285 1.5707963267949005548
- joint left_ank_B12: origin xyz=0.0080000000000000001665 -0.014999999999999985567 -0.011500000000000003275 rpy=-1.5707963267949205388 -1.469756662182277962 1.5707963267949025532 -> xyz=0.008000000000000003636 -0.015000000000000013323 -0.011500000000000003275 rpy=-1.5707963267949294206 -1.4697566621822577559 1.5707963267949305308
- joint left_ank_B21: origin xyz=6.9388939039072283776e-18 -2.7755575615628913511e-17 -0.01150000000000000154 rpy=1.570796326794896558 -1.4285697747625525356 1.5707963267948994446 -> xyz=0 0 -0.011499999999999996336 rpy=1.570796326794896558 -1.4285697747625691889 1.5707963267948952257
- joint left_ank_B22: origin xyz=0 0 -0.01150000000000000154 rpy=1.5707963267949021091 -1.4285463212680715728 -1.5707963267948938935 -> xyz=0 0 -0.011499999999999998071 rpy=1.570796326794896558 -1.4285463212681039913 -1.5707963267948852337
- joint left_ank_B31: origin xyz=4.336808689942017736e-19 -0.0064387505004003808828 0 rpy=-1.5707963267948970021 0.1691344003409792629 1.2463746926904215167e-14 -> xyz=1.3010426069826053208e-18 -0.006438750500400436394 0 rpy=-1.57079632679489678 0.16913440034098886633 2.9529351978209400659e-15
- joint left_ank_B32: origin xyz=-2.4286128663675299322e-17 -0.0064387505004003808828 0 rpy=-1.570796326794896558 -0.17993145005786467805 5.6818279199863494045e-15 -> xyz=1.7347234759768070944e-17 -0.006438750500400436394 0 rpy=-1.570796326794896336 -0.17993145005780261658 1.3200513083700388182e-15
- joint left_ank_R11: origin xyz=-0.0099999999999999967387 0.012500000000000011102 -0.033600000000000011802 rpy=-3.5821358734369027029e-16 -2.0703583441380111793e-15 -0.1011603127571137628 -> xyz=-0.0099999999999999967387 0.012500000000000038858 -0.033600000000000004863 rpy=-1.3295317856339465751e-14 8.7994714049036524006e-15 -0.1011603127570600974
- joint left_ank_R12: origin xyz=0.010000000000000003678 0.012499999999999955591 -0.033600000000000004863 rpy=3.1415926535897606975 1.5562027335348888578e-14 -3.0405529889788582842 -> xyz=0.010000000000000003678 0.012500000000000038858 -0.033600000000000004863 rpy=3.1415926535897802374 2.5015582227113039382e-14 -3.0405529889788152076
- joint left_ank_R21: origin xyz=-6.9388939039072283776e-18 -0.0099999999999999533706 0 rpy=-1.570796326794896558 -1.4285697747629988452 1.5707963267949092145 -> xyz=-6.9388939039072283776e-18 -0.0099999999999999533706 6.9388939039072283776e-18 rpy=-1.570796326794896558 -1.4285697747629295673 1.5707963267948288344
- joint left_ank_R22: origin xyz=6.9388939039072283776e-18 -0.010000000000000036637 6.9388939039072283776e-18 rpy=1.5707963267949194286 -1.4285463212677806943 -1.5707963267950313391 -> xyz=-6.9388939039072283776e-18 -0.0099999999999999811262 6.9388939039072283776e-18 rpy=1.570796326794896558 -1.4285463212677005362 -1.5707963267950528774
- joint left_ank_act1: origin xyz=2.2722093540906984632e-06 7.7021722333370234992e-16 -0.072660031604095037805 rpy=-3.1415926535896590011 8.173835939810196213e-14 -2.2021168238262767147 -> xyz=2.2722093528972087118e-06 4.2327252813834093104e-16 -0.072660031604101171787 rpy=-3.1415926535896590011 1.0257376628608333772e-13 -2.2021168238262784911
- joint left_ank_act2: origin xyz=2.2722093490027545082e-06 -7.7229889150487451843e-15 -0.07266003047881974819 rpy=-3.1415926535895000171 4.7493922909940523358e-14 -2.2021168238262776029 -> xyz=2.2722093472333365627e-06 -8.396061623727746337e-15 -0.072660030478823994793 rpy=-3.1415926535895000171 4.7380615214810755067e-14 -2.2021168238262500694
- joint left_ank_pitch: limit lower=-0.785398163397448279 upper=0.785398163397448279 effort=1 velocity=20 -> lower=-0.52359877559829881566 upper=0.52359877559829881566 effort=1 velocity=20; origin xyz=7.2631635415802528961e-19 -0.099999999999999977796 -0.0061999999999999989148 rpy=-3.1415926535897922278 -4.216693940517171266e-15 -1.5707963267948972241 -> xyz=1.1074470850715867721e-18 -0.10000000000000006106 -0.0062000000000000023842 rpy=3.141592653589793116 1.7874590696523099396e-14 -1.5707963267948983344
- joint left_ank_roll: origin xyz=1.9984014443252817728e-15 0.0015000000000042093377 -0.014599999999997269676 rpy=-1.5707963267950535435 -1.5707963267944073937 0 -> xyz=2.9976021664879226591e-15 0.0015000000000041202163 -0.014599999999997613151 rpy=-1.5707963267949680564 -1.5707963267944098362 0
- joint left_hip_pitch: origin xyz=-0.024000000716154958752 -0.019000000152441291756 -0.019000000152448955765 rpy=-1.5707963267944653474 1.5707963267948226171 0 -> xyz=-0.024000000716157210423 -0.019000000152441316043 -0.019000000152448022483 rpy=-1.5707963267944322627 1.570796326794811959 0
- joint left_hip_roll: origin xyz=0.01900000000000030137 -3.3624037938346747648e-18 -0.026000000000000279832 rpy=3.141592653589793116 -1.570796326794573039 0 -> xyz=0.019000000000000304839 -3.362403793834428631e-18 -0.026000000000000279832 rpy=3.141592653589793116 -1.5707963267945577179 0
- joint left_knee: origin xyz=-6.5473275179360459098e-15 0.096000000000000071387 0.027400000000000535039 rpy=-3.141592653589783346 1.4838131564395688657e-16 6.5779908238917364858e-16 -> xyz=-8.1704984642832938552e-15 0.095999999999999391376 0.027400000000000819533 rpy=3.1415926535897753524 1.6653345376122616675e-16 -1.6536824015790017811e-15

File: toddlerbot/robot_descriptions/assemblies/no_body/no_body.urdf (robot description, URDF)
Before this commit: robot no_body, 3 links, 2 joints
Links:
- link left_3r+rh5_leg: mass 0.3326398048030183574 -> 0.33962718831922139584
- link right_3r+rh5_leg: mass 0.33263981812552856354 -> 0.33962720155413217427
Joints:
- joint left_hip_yaw: origin xyz=-0.0063999999999966045855 0.03399999999999939182 0.28550000000000008704 rpy=2.327572832560927136e-16 4.9789962508008699149e-17 -1.0650377544034614197e-13 -> xyz=-0.0063999999999966063202 0.033999999999999308553 0.28550000000000003153 rpy=2.3275728331677864905e-16 1.1102230242191183694e-16 -1.1455751422015388711e-13
- joint right_hip_yaw: origin xyz=-0.0063999999999967962724 -0.034000000000000661637 0.28549999999999992051 rpy=1.2173498094910643509e-16 -6.1232339957301087894e-17 -5.033057304260250785e-13 -> xyz=-0.0063999999999967980072 -0.034000000000000668576 0.28549999999999992051 rpy=1.2173498094825229595e-16 9.8900267199457111713e-23 -3.0336177719551955022e-13

File: toddlerbot/robot_descriptions/assemblies/right_3R+RH5_leg/right_3R+RH5_leg.urdf (robot description, URDF)
Before this commit: robot right_3R+RH5_leg, 18 links, 17 joints
Links:
- link 12lf: mass 0.044782197696050352054 -> 0.044782197690790462308
- link 12lf_2: mass 0.044782197696050358993 -> 0.044782197690790476186
- link 12lf_rod: mass 0.0025088292483592140175 -> 0.0025088292483592144512
- link 12lf_rod_2: mass 0.0025088292483592140175 -> 0.0025088292483592144512
- link 12lf_rod_end: mass 0.00085420491177815905965 -> 0.00085420491177815895123
- link 12lf_rod_end_2: mass 0.00085420491177815905965 -> 0.00085420491177815895123
- link ank_pitch_link: mass 0.0042238381753791605713 -> 0.0042238381753791614387
- link ank_roll_link: mass 0.013844478784760248444 -> 0.021210604954423659119
- link ank_rr_link: mass 0.00044289790445047673732 -> 0.00042507093693768156772
- link ank_rr_link_2: mass 0.00044289790445047673732 -> 0.00042507093693768156772
- link ball_joint_ball: mass 4.4053796295264630609e-05 -> 4.4053796295264623832e-05
- link ball_joint_ball_2: mass 4.4053796295264630609e-05 -> 4.4053796295264623832e-05
- link ball_joint_container: mass 4.803735642533054869e-05 -> 4.8037356425330562243e-05
- link ball_joint_container_2: mass 4.803735642533054869e-05 -> 4.8037356425330562243e-05
- link hip_roll_link: mass 0.09801239148352869357 -> 0.098012391483528665814
- link hip_yaw_link: mass 0.0090258837370979193293 -> 0.009025883737097921064
- link right_hip_pitch_link: mass 0.093882153558663708481 -> 0.09353906475262946385
Joints:
- joint right_ank_B11: origin xyz=0.008000000000000003636 0.015000000000000013323 -0.011499999999999998071 rpy=1.570796326794896558 -1.469636014037899896 -1.5707963267948905628 -> xyz=0.0079999999999999238387 0.015000000000000124345 -0.01150000000000006746 rpy=1.5707963267949047736 -1.4696360140379067794 -1.5707963267948874542
- joint right_ank_B12: origin xyz=0.0080000000000000365957 0.014999999999999985567 0.028300000000000158362 rpy=-1.570796326794896558 -1.469756662182680973 1.570796326794891451 -> xyz=0.0080000000000000192485 0.015000000000000068834 0.028300000000000900824 rpy=-1.5707963267949041075 -1.469756662182670981 1.5707963267948925612
- joint right_ank_B21: origin xyz=6.9388939039072283776e-18 0 -0.01150000000000000154 rpy=1.570796326794896558 -1.4285697747626475707 1.5707963267948843455 -> xyz=0 0 -0.011500000000000022357 rpy=1.5707963267948794606 -1.4285697747626477927 1.5707963267948803487
- joint right_ank_B22: origin xyz=0 0 -0.011499999999999999806 rpy=1.57079632679489678 -1.4285463212679265776 1.5707963267948943376 -> xyz=0 -5.5511151231257827021e-17 -0.01150000000000000501 rpy=1.5707963267948947816 -1.4285463212679219147 1.5707963267948921171
- joint right_ank_B31: origin xyz=9.1072982488782372457e-18 -0.0064387505004003808828 0 rpy=-1.5707963267948961139 0.16913440034171131621 -1.7599215475487529123e-15 -> xyz=9.5409791178724390193e-17 -0.0064387505004002698605 -5.5511151231257827021e-17 rpy=-1.5707963267948954478 0.16913440034172153026 -1.8050260774851149667e-15
- joint right_ank_B32: origin xyz=-8.6736173798840354721e-18 -0.0064387505004003531273 -1.3877787807814456755e-17 rpy=-1.5707963267948854558 -0.17993145005747521181 -6.9806032607149013267e-15 -> xyz=-7.3725747729014301513e-18 -0.0064387505004002698605 6.9388939039072283776e-18 rpy=-1.5707963267948981123 -0.17993145005746249976 -8.7955855822383372175e-16
- joint right_ank_R11: origin xyz=-0.0099999999999999984734 0.012500000000000011102 -0.033599999999999997924 rpy=-2.3897964054427488116e-14 -3.8273675914490832965e-16 -0.10116031275657462463 -> xyz=-0.0099999999999998423483 0.012499999999999733546 -0.033599999999999782818 rpy=-1.4093527784308163928e-14 -9.1905749868284128401e-17 -0.10116031275663164846
- joint right_ank_R12: origin xyz=0.010000000000000003678 0.012499999999999955591 -0.033600000000000004863 rpy=-3.1415926535897709115 -4.1620274661327994973e-15 -3.0405529889776490293 -> xyz=0.0099999999999997174482 0.012499999999999733546 -0.03359999999999976894 rpy=-3.1415926535897820138 -2.2156165769524474289e-15 -3.0405529889777027641
- joint right_ank_R21: origin xyz=0 -0.010000000000000008882 1.3877787807814456755e-17 rpy=-1.570796326794896558 -1.4285697747630956567 1.5707963267948958919 -> xyz=4.1633363423443370266e-17 -0.010000000000000119904 -2.7755575615628913511e-17 rpy=-1.5707963267949331954 -1.4285697747630743404 1.5707963267949289765
- joint right_ank_R22: origin xyz=-6.9388939039072283776e-18 -0.0099999999999999811262 1.3877787807814456755e-17 rpy=1.570796326794896558 -1.428546321268451269 -1.570796326794896558 -> xyz=-5.5511151231257827021e-17 -0.0099999999999999811262 -1.3877787807814456755e-17 rpy=1.5707963267948956698 -1.4285463212684392786 -1.570796326794886566
- joint right_ank_act1: origin xyz=2.2722093427646888886e-06 1.7902346272080649214e-15 -0.072660031604104419189 rpy=-3.1415926535897806815 9.7899118131350707255e-15 -2.2021168238260933059 -> xyz=2.2722093427577499947e-06 1.727784582072899866e-15 -0.0726600316041042249 rpy=-3.1415926535897815697 1.0092007725908475977e-14 -2.2021168238260941941
- joint right_ank_act2: origin xyz=2.2722093383654301535e-06 -2.5118795932144166727e-15 -0.07266003047881591792 rpy=3.1415926535897926719 5.7157557368585280826e-16 -2.2021168238262842642 -> xyz=2.2722093383550218126e-06 -2.4633073358870660741e-15 -0.07266003047881686161 rpy=3.141592653589793116 2.7467349934334640921e-15 -2.2021168238262860406
- joint right_ank_pitch: limit lower=-0.785398163397448279 upper=0.785398163397448279 effort=1 velocity=20 -> lower=-0.52359877559829881566 upper=0.52359877559829881566 effort=1 velocity=20; origin xyz=1.0774845611827788694e-18 0.10000000000000003331 -0.0062000000000000006495 rpy=3.141592653589783346 -6.5431213406603904361e-15 -1.57079632679491632 -> xyz=-2.423086741528762234e-18 0.10000000000000014433 -0.006200000000000555761 rpy=-3.1415926535897922278 -1.0275284166593592938e-14 -1.570796326794896558
- joint right_ank_roll: origin xyz=1.7486012637846215512e-15 0.001500000000009214015 -0.014599999999994360544 rpy=-1.5707963267952413933 1.570796326794632769 0 -> xyz=1.8041124150158793782e-15 0.0015000000000095273494 -0.014599999999994438607 rpy=-1.5707963267952527175 1.5707963267946807306 0
- joint right_hip_pitch: origin xyz=0.024000000358073002305 -0.019000000000011920548 -0.018999999847560570393 rpy=-1.5707963267950890707 -1.5707963267946420949 0 -> xyz=0.024000000358073016182 -0.019000000000011917078 -0.018999999847560563454 rpy=-1.5707963267950879604 -1.5707963267946316588 0
- joint right_hip_roll: origin xyz=0.018999999999999881567 -3.3500438889873688288e-18 -0.026000000000000002276 rpy=1.4130847605241333966e-30 1.5707963267948645836 0 -> xyz=0.018999999999999874628 7.643544883287250703e-16 -0.025999999999999960643 rpy=-1.300781512818313455e-27 1.5707963267948954478 0
- joint right_knee: origin xyz=-2.892603788276459435e-15 0.095999999999999294231 0.027400000000000382383 rpy=-3.141592653589788231 -2.6961419186663855904e-16 -3.141592653589793116 -> xyz=-2.8905460953097867777e-15 0.095999999999999252598 0.027400000000001673017 rpy=-3.1415926535897824579 4.9746286444423846074e-17 -3.1415926535897891192
