Commit message: Update toddlerbot legs

File: toddlerbot/robot_descriptions/assemblies/left_3R+RH5_leg/left_3R+RH5_leg.urdf (robot description, URDF)
Before this commit: robot left_3R+RH5_leg, 18 links, 17 joints
Links:
- link ank_roll_link: mass 0.021210605042023062544 -> 0.020312412324461778801
- link left_calf_link: mass 0.016290616864051549878 -> 0.015782434194230747504
- link left_hip_pitch_link: mass 0.093539065135968851861 -> 0.093539065135968837983
Joints:
- joint left_ank_B11: origin xyz=0.0080000000000000643513 -0.015000000000000235367 0.028299999999999957134 rpy=-1.570796326794896558 1.4696360140379425285 1.5707963267949005548 -> xyz=0.0079999999999999949624 -0.015000000000000096589 0.028299999999999991829 rpy=-1.570796326794896558 1.5520170643097057628 1.5707963267950826314
- joint left_ank_B12: origin xyz=0.008000000000000003636 -0.015000000000000013323 -0.011500000000000003275 rpy=-1.5707963267949294206 -1.4697566621822577559 1.5707963267949305308 -> xyz=0.0080000000000000019013 -0.015000000000000041078 -0.011499999999999999806 rpy=-1.570796326794896558 -1.5521341097218244176 1.5707963267948896746
- joint left_ank_B21: origin xyz=0 0 -0.011499999999999996336 rpy=1.570796326794896558 -1.4285697747625691889 1.5707963267948952257 -> xyz=-3.4694469519536141888e-18 -2.7755575615628913511e-17 -0.011499999999999999806 rpy=-1.570796326794896558 -1.5664147454872627829 -1.5707963267957041342
- joint left_ank_B22: origin xyz=0 0 -0.011499999999999998071 rpy=1.570796326794896558 -1.4285463212681039913 -1.5707963267948852337 -> xyz=3.4694469519536141888e-18 0 -0.01150000000000000154 rpy=-1.570796326794896336 -1.5664376509754431854 1.570796326794866582
- joint left_ank_B31: origin xyz=1.3010426069826053208e-18 -0.006438750500400436394 0 rpy=-1.57079632679489678 0.16913440034098886633 2.9529351978209400659e-15 -> xyz=0 -0.0064387505004003531273 -3.4694469519536141888e-18 rpy=-1.57079632679489678 0.16913440034090146402 5.8375589418798256921e-16
- joint left_ank_B32: origin xyz=1.7347234759768070944e-17 -0.006438750500400436394 0 rpy=-1.570796326794896336 -0.17993145005780261658 1.3200513083700388182e-15 -> xyz=2.498001805406602216e-16 -0.0064387505004004919051 -3.4694469519536141888e-18 rpy=-1.570796326794896558 -0.17993145005756983057 3.0408221168269646133e-14
- joint left_ank_R11: origin xyz=-0.0099999999999999967387 0.012500000000000038858 -0.033600000000000004863 rpy=-1.3295317856339465751e-14 8.7994714049036524006e-15 -0.1011603127570600974 -> xyz=-0.018000000000000009048 0.016000000000000014211 -0.020599999999999996786 rpy=-4.1594268726375658989e-17 6.5315524930102152625e-16 -0.01877926248499593373
- joint left_ank_R12: origin xyz=0.010000000000000003678 0.012500000000000038858 -0.033600000000000004863 rpy=3.1415926535897802374 2.5015582227113039382e-14 -3.0405529889788152076 -> xyz=0.017999999999999995171 0.016000000000000014211 -0.020600000000000000255 rpy=3.1415926535897922278 7.4438972302667006905e-16 -3.1229304365180685643
- joint left_ank_R21: origin xyz=-6.9388939039072283776e-18 -0.0099999999999999533706 6.9388939039072283776e-18 rpy=-1.570796326794896558 -1.4285697747629295673 1.5707963267948288344 -> xyz=0 -0.0099999999999999533706 0 rpy=1.570796326794896558 -1.5664147454868542209 -1.5707963267948135133
- joint left_ank_R22: origin xyz=-6.9388939039072283776e-18 -0.0099999999999999811262 6.9388939039072283776e-18 rpy=1.570796326794896558 -1.4285463212677005362 -1.5707963267950528774 -> xyz=0 -0.0099999999999999533706 0 rpy=-1.570796326794896558 -1.5664376509758224376 1.570796326795195208
- joint left_ank_act1: origin xyz=2.2722093528972087118e-06 4.2327252813834093104e-16 -0.072660031604101171787 rpy=-3.1415926535896590011 1.0257376628608333772e-13 -2.2021168238262784911 -> xyz=2.2722093531019060819e-06 5.1000870193718128576e-16 -0.074779998095377359091 rpy=-3.1415926535896590011 8.6569212672158331644e-14 -2.2021168238262673889
- joint left_ank_act2: origin xyz=2.2722093472333365627e-06 -8.396061623727746337e-15 -0.072660030478823994793 rpy=-3.1415926535895000171 4.7380615214810755067e-14 -2.2021168238262500694 -> xyz=2.2722093474362992094e-06 -8.9372953482325101504e-15 -0.074779996992751340823 rpy=-3.1415926535895000171 6.172537580306697636e-14 -2.2021168238262789352
- joint left_ank_pitch: limit lower=-0.52359877559829881566 upper=0.52359877559829881566 effort=1 velocity=20 -> lower=-0.785398163397448279 upper=0.95993108859688125456 effort=1 velocity=20; origin xyz=1.1074470850715867721e-18 -0.10000000000000006106 -0.0062000000000000023842 rpy=3.141592653589793116 1.7874590696523099396e-14 -1.5707963267948983344 -> xyz=5.9135023084202893979e-19 -0.10000000000000006106 -0.0061999999999999989148 rpy=3.141592653589793116 3.3306690738944506007e-16 -1.5707963267948974462
- joint left_ank_roll: origin xyz=2.9976021664879226591e-15 0.0015000000000041202163 -0.014599999999997613151 rpy=-1.5707963267949680564 -1.5707963267944098362 0 -> xyz=3.0531133177191804862e-15 0.001500000000004121951 -0.014599999999997613151 rpy=-1.5707963267949702768 -1.5707963267946758457 0
- joint left_hip_pitch: origin xyz=-0.024000000716157210423 -0.019000000152441316043 -0.019000000152448022483 rpy=-1.5707963267944322627 1.570796326794811959 0 -> xyz=-0.024000000716155274472 -0.019000000152442689944 -0.019000000152446339802 rpy=-1.5707963267945199703 1.5707963267948246155 0
- joint left_hip_roll: origin xyz=0.019000000000000304839 -3.362403793834428631e-18 -0.026000000000000279832 rpy=3.141592653589793116 -1.5707963267945577179 0 -> xyz=0.01900000000000030137 5.3821911112507180559e-16 -0.026000000000000168809 rpy=3.141592653589793116 -1.5707963267936781993 0
- joint left_knee: origin xyz=-8.1704984642832938552e-15 0.095999999999999391376 0.027400000000000819533 rpy=3.1415926535897753524 1.6653345376122616675e-16 -1.6536824015790017811e-15 -> xyz=-8.1569325594195215653e-15 0.095999999999999391376 0.027400000000002110168 rpy=3.1415926535897917837 1.6653345451476814222e-16 -5.2069203968451419987e-17

File: toddlerbot/robot_descriptions/assemblies/no_body/no_body.urdf (robot description, URDF)
Before this commit: robot no_body, 3 links, 2 joints
Links:
- link left_3r+rh5_leg: mass 0.33962718831922139584 -> 0.33822081293183930972
- link right_3r+rh5_leg: mass 0.33962720155413217427 -> 0.33821810347966374533
Joints:
- joint left_hip_yaw: origin xyz=-0.0063999999999966063202 0.033999999999999308553 0.28550000000000003153 rpy=2.3275728331677864905e-16 1.1102230242191183694e-16 -1.1455751422015388711e-13 -> xyz=-0.0063999999999966063202 0.033999999999999308553 0.28550000000000003153 rpy=2.3275728331677864905e-16 1.1102230242191363653e-16 -1.222458086656465435e-13

File: toddlerbot/robot_descriptions/assemblies/right_3R+RH5_leg/right_3R+RH5_leg.urdf (robot description, URDF)
Before this commit: robot right_3R+RH5_leg, 18 links, 17 joints
Links:
- link ank_roll_link: mass 0.021210604954423659119 -> 0.020312412236862385784
- link right_calf_link: mass 0.016290630569901022595 -> 0.015779725212993943317
Joints:
- joint right_ank_B11: origin xyz=0.0079999999999999238387 0.015000000000000124345 -0.01150000000000006746 rpy=1.5707963267949047736 -1.4696360140379067794 -1.5707963267948874542 -> xyz=0.0079999999999999984318 0.015000000000000041078 -0.01150000000000000154 rpy=1.570796326794896558 -1.5520170643097170871 -1.5707963267946734032
- joint right_ank_B12: origin xyz=0.0080000000000000192485 0.015000000000000068834 0.028300000000000900824 rpy=-1.5707963267949041075 -1.469756662182670981 1.5707963267948925612 -> xyz=0.008000000000000003636 0.015000000000000041078 0.028300000000000019584 rpy=-1.570796326794896558 -1.5521341097221632577 1.5707963267948059638
- joint right_ank_B21: origin xyz=0 0 -0.011500000000000022357 rpy=1.5707963267948794606 -1.4285697747626477927 1.5707963267948803487 -> xyz=0 -2.7755575615628913511e-17 -0.011500000000000006745 rpy=-1.570796326794896558 -1.5664147454871475418 -1.5707963267939402119
- joint right_ank_B22: origin xyz=0 -5.5511151231257827021e-17 -0.01150000000000000501 rpy=1.5707963267948947816 -1.4285463212679219147 1.5707963267948921171 -> xyz=3.4694469519536141888e-18 0 -0.011499999999999998071 rpy=-1.57079632679489678 -1.5664376509754476263 -1.5707963267945079799
- joint right_ank_B31: origin xyz=9.5409791178724390193e-17 -0.0064387505004002698605 -5.5511151231257827021e-17 rpy=-1.5707963267948954478 0.16913440034172153026 -1.8050260774851149667e-15 -> xyz=6.9388939039072283776e-18 -0.0064387505004004086384 6.9388939039072283776e-18 rpy=-1.5707963267948970021 0.1691344003416279107 3.6048302674885136887e-16
- joint right_ank_B32: origin xyz=-7.3725747729014301513e-18 -0.0064387505004002698605 6.9388939039072283776e-18 rpy=-1.5707963267948981123 -0.17993145005746249976 -8.7955855822383372175e-16 -> xyz=3.4694469519536141888e-18 -0.0064387505004004086384 -6.9388939039072283776e-18 rpy=-1.570796326794896558 -0.17993145005738314657 -8.7569826039094258121e-17
- joint right_ank_R11: origin xyz=-0.0099999999999998423483 0.012499999999999733546 -0.033599999999999782818 rpy=-1.4093527784308163928e-14 -9.1905749868284128401e-17 -0.10116031275663164846 -> xyz=-0.018000000000000005579 0.016000000000000014211 -0.020599999999999996786 rpy=-3.5360359477892277706e-16 8.2839943819914169726e-16 -0.018779262484754637164
- joint right_ank_R12: origin xyz=0.0099999999999997174482 0.012499999999999733546 -0.03359999999999976894 rpy=-3.1415926535897820138 -2.2156165769524474289e-15 -3.0405529889777027641 -> xyz=0.01799999999999999864 0.016000000000000069722 -0.020600000000000003725 rpy=3.1415926535897922278 1.1785067659504147721e-15 -3.1229304365172114721
- joint right_ank_R21: origin xyz=4.1633363423443370266e-17 -0.010000000000000119904 -2.7755575615628913511e-17 rpy=-1.5707963267949331954 -1.4285697747630743404 1.5707963267949289765 -> xyz=3.4694469519536141888e-18 -0.010000000000000008882 0 rpy=1.57079632679489678 -1.5664147454870704923 -1.5707963267947753216
- joint right_ank_R22: origin xyz=-5.5511151231257827021e-17 -0.0099999999999999811262 -1.3877787807814456755e-17 rpy=1.5707963267948956698 -1.4285463212684392786 -1.570796326794886566 -> xyz=-3.4694469519536141888e-18 -0.0099999999999999533706 -3.4694469519536141888e-18 rpy=-1.570796326794896336 -1.5664376509754269762 1.5707963267952340658
- joint right_ank_act1: origin xyz=2.2722093427577499947e-06 1.727784582072899866e-15 -0.0726600316041042249 rpy=-3.1415926535897815697 1.0092007725908475977e-14 -2.2021168238260941941 -> xyz=2.2722093412017030367e-06 1.8804402479588588903e-15 -0.074779998095388988677 rpy=-3.1415926535897829019 8.526808676235474948e-15 -2.2021168238260906413
- joint right_ank_act2: origin xyz=2.2722093383550218126e-06 -2.4633073358870660741e-15 -0.07266003047881686161 rpy=3.141592653589793116 2.7467349934334640921e-15 -2.2021168238262860406 -> xyz=2.2722093371875529133e-06 -2.8553548414578244774e-15 -0.074779996992751840423 rpy=3.1415926535897922278 3.3072658899692120884e-15 -2.2021168238262864847
- joint right_ank_pitch: limit lower=-0.52359877559829881566 upper=0.52359877559829881566 effort=1 velocity=20 -> lower=-0.785398163397448279 upper=0.95993108859688125456 effort=1 velocity=20; origin xyz=-2.423086741528762234e-18 0.10000000000000014433 -0.006200000000000555761 rpy=-3.1415926535897922278 -1.0275284166593592938e-14 -1.570796326794896558 -> xyz=5.0979769291920753058e-19 0.099999999999999977796 -0.0062000000000000023842 rpy=-3.1415926535897926719 5.5511151131695266928e-17 -1.5707963267946121189
- joint right_ank_roll: origin xyz=1.8041124150158793782e-15 0.0015000000000095273494 -0.014599999999994438607 rpy=-1.5707963267952527175 1.5707963267946807306 0 -> xyz=2.0816681711721685133e-15 0.0015000000000089284361 -0.014599999999994599936 rpy=-1.5707963267951812192 1.5707963267946736252 0
- joint right_hip_pitch: origin xyz=0.024000000358073016182 -0.019000000000011917078 -0.018999999847560563454 rpy=-1.5707963267950879604 -1.5707963267946316588 0 -> xyz=0.024000000358075784801 -0.019000000000012132184 -0.01899999984755619542 rpy=-1.5707963267951119413 -1.5707963267945823649 0
- joint right_hip_roll: origin xyz=0.018999999999999874628 7.643544883287250703e-16 -0.025999999999999960643 rpy=-1.300781512818313455e-27 1.5707963267948954478 0 -> xyz=0.018999999999999881567 -3.350043888987566044e-18 -0.026000000000000002276 rpy=2.9582283942363596652e-30 1.5707963267948799047 0
- joint right_knee: origin xyz=-2.8905460953097867777e-15 0.095999999999999252598 0.027400000000001673017 rpy=-3.1415926535897824579 4.9746286444423846074e-17 -3.1415926535897891192 -> xyz=-8.4133172564547814973e-15 0.095999999999998697486 0.027400000000003574274 rpy=3.1415926535897926719 9.3467860356166481656e-14 -3.1415926535895137839
