Commit message: Update the toddlerbot_legs

File: toddlerbot/robot_descriptions/assemblies/left_3R+RH5_leg/left_3R+RH5_leg.urdf (robot description, URDF)
Before this commit: robot left_3R+RH5_leg, 18 links, 17 joints
Links:
- link 12lf: mass 0.044782197690790462308 -> 0.044782197696050358993
- link 12lf_2: mass 0.044782197690790462308 -> 0.044782197696050358993
- link 12lf_rod_end: mass 0.00085420491177815895123 -> 0.00085420491177815905965
- link 12lf_rod_end_2: mass 0.00085420491177815895123 -> 0.00085420491177815905965
- link ank_pitch_link: mass 0.0042238381753791614387 -> 0.0042238381753791605713
- link ank_roll_link: mass 0.020312412324461778801 -> 0.02031241232446178227
- link ank_rr_link: mass 0.00042507093693768156772 -> 0.00042507093693768162193
- link ank_rr_link_2: mass 0.00042507093693768156772 -> 0.00042507093693768162193
- link ball_joint_ball: mass 4.4053796295264623832e-05 -> 4.4053796295264630609e-05
- link ball_joint_ball_2: mass 4.4053796295264623832e-05 -> 4.4053796295264630609e-05
- link hip_yaw_link: mass 0.009025883737097921064 -> 0.0090258837370979175946
- link left_hip_pitch_link: mass 0.093539065135968837983 -> 0.093611654200831340145
Joints:
- joint left_ank_B11: origin xyz=0.0079999999999999949624 -0.015000000000000096589 0.028299999999999991829 rpy=-1.570796326794896558 1.5520170643097057628 1.5707963267950826314 -> xyz=0.0080000000000000123096 -0.015000000000000041078 0.028299999999999991829 rpy=-1.570796326794896558 1.5520170643096702356 1.5707963267949236474
- joint left_ank_B12: origin xyz=0.0080000000000000019013 -0.015000000000000041078 -0.011499999999999999806 rpy=-1.570796326794896558 -1.5521341097218244176 1.5707963267948896746 -> xyz=0.008000000000000003636 -0.014999999999999985567 -0.011499999999999998071 rpy=-1.570796326794896558 -1.5521341097218652738 1.5707963267948228392
- joint left_ank_B21: origin xyz=-3.4694469519536141888e-18 -2.7755575615628913511e-17 -0.011499999999999999806 rpy=-1.570796326794896558 -1.5664147454872627829 -1.5707963267957041342 -> xyz=-2.3245294578089215065e-16 0 -0.011500000000000003275 rpy=-1.5707963267921956074 -1.5664147454872743292 -1.5707963267976534638
- joint left_ank_B22: origin xyz=3.4694469519536141888e-18 0 -0.01150000000000000154 rpy=-1.570796326794896336 -1.5664376509754431854 1.570796326794866582 -> xyz=0 -8.3266726846886740532e-17 -0.011499999999999996336 rpy=-1.570796326794896558 -1.5664376509753994426 1.5707963267946438712
- joint left_ank_B31: origin xyz=0 -0.0064387505004003531273 -3.4694469519536141888e-18 rpy=-1.57079632679489678 0.16913440034090146402 5.8375589418798256921e-16 -> xyz=6.9388939039072283776e-18 -0.0064387505004001865938 -2.0816681711721685133e-17 rpy=-1.5707963267948947816 0.16913440034089716191 -5.6247294630893699029e-16
- joint left_ank_B32: origin xyz=2.498001805406602216e-16 -0.0064387505004004919051 -3.4694469519536141888e-18 rpy=-1.570796326794896558 -0.17993145005756983057 3.0408221168269646133e-14 -> xyz=-3.4694469519536141888e-18 -0.0064387505004003808828 -3.4694469519536141888e-18 rpy=-1.570796326794896558 -0.17993145005761934652 -1.3040300712961991222e-18
- joint left_ank_R11: origin xyz=-0.018000000000000009048 0.016000000000000014211 -0.020599999999999996786 rpy=-4.1594268726375658989e-17 6.5315524930102152625e-16 -0.01877926248499593373 -> xyz=-0.018000000000000005579 0.015999999999999986455 -0.020599999999999993316 rpy=7.372266899210394361e-15 1.2457991987000010843e-14 -0.018779262484739548539
- joint left_ank_R12: origin xyz=0.017999999999999995171 0.016000000000000014211 -0.020600000000000000255 rpy=3.1415926535897922278 7.4438972302667006905e-16 -3.1229304365180685643 -> xyz=0.017999999999999995171 0.015999999999999986455 -0.020600000000000007194 rpy=3.1415926535897837901 5.7200784449866287445e-15 -3.1229304365178514047
- joint left_ank_R21: origin xyz=0 -0.0099999999999999533706 0 rpy=1.570796326794896558 -1.5664147454868542209 -1.5707963267948135133 -> xyz=-3.4694469519536141888e-18 -0.0099999999999999533706 3.4694469519536141888e-18 rpy=1.5707963267999907053 -1.5664147454868477816 -1.5707963267999944801
- joint left_ank_R22: origin xyz=0 -0.0099999999999999533706 0 rpy=-1.570796326794896558 -1.5664376509758224376 1.570796326795195208 -> xyz=0 -0.010000000000000008882 0 rpy=-1.570796326795200093 -1.5664376509758415335 1.5707963267972691046
- joint left_ank_act1: origin xyz=2.2722093531019060819e-06 5.1000870193718128576e-16 -0.074779998095377359091 rpy=-3.1415926535896590011 8.6569212672158331644e-14 -2.2021168238262673889 -> xyz=2.272209352376791669e-06 3.5735303605122226145e-16 -0.074779998095385435963 rpy=-3.1415926535896594451 8.8365826112773068852e-14 -2.2021168238262687211
- joint left_ank_act2: origin xyz=2.2722093474362992094e-06 -8.9372953482325101504e-15 -0.074779996992751340823 rpy=-3.1415926535895000171 6.172537580306697636e-14 -2.2021168238262789352 -> xyz=2.2722093472662963087e-06 -8.4619811158148650065e-15 -0.074779996992748620777 rpy=-3.1415926535895000171 6.2188672547836847539e-14 -2.2021168238262793793
- joint left_ank_pitch: origin xyz=5.9135023084202893979e-19 -0.10000000000000006106 -0.0061999999999999989148 rpy=3.141592653589793116 3.3306690738944506007e-16 -1.5707963267948974462 -> xyz=9.1041832417877273971e-19 -0.099999999999999977796 -0.0062000000000000006495 rpy=3.1415926535897913396 3.2973623831365823964e-14 -1.5707963267949118791
- joint left_ank_roll: origin xyz=3.0531133177191804862e-15 0.001500000000004121951 -0.014599999999997613151 rpy=-1.5707963267949702768 -1.5707963267946758457 0 -> xyz=3.1086244689504383132e-15 0.00150000000000412065 -0.014599999999997594069 rpy=-1.5707963267949904829 -1.5707963267947890884 0
- joint left_hip_pitch: origin xyz=-0.024000000716155274472 -0.019000000152442689944 -0.019000000152446339802 rpy=-1.5707963267945199703 1.5707963267948246155 0 -> xyz=-0.024000000716140019313 -0.019000000152447758806 -0.019000000152447786561 rpy=-1.570796326794896336 1.5707963267947404606 0
- joint left_hip_roll: origin xyz=0.01900000000000030137 5.3821911112507180559e-16 -0.026000000000000168809 rpy=3.141592653589793116 -1.5707963267936781993 0 -> xyz=0.019000000000000304839 -3.362403793834026882e-18 -0.026000000000000279832 rpy=3.141592653589793116 -1.5707963267948437114 0
- joint left_knee: origin xyz=-8.1569325594195215653e-15 0.095999999999999391376 0.027400000000002110168 rpy=3.1415926535897917837 1.6653345451476814222e-16 -5.2069203968451419987e-17 -> xyz=-9.0379327827951061674e-15 0.095999999999999793832 0.027400000000001221989 rpy=3.1415926535896172567 6.1949089521373328246e-14 -1.573475576806645783e-15

File: toddlerbot/robot_descriptions/assemblies/no_body/no_body.urdf (robot description, URDF)
Before this commit: robot no_body, 3 links, 2 joints
Links:
- link body_link: mass 0.1326329205818372603 -> 0.4585959758251314522
- link left_3r+rh5_leg: mass 0.33822081293183930972 -> 0.33829340200722179954
- link right_3r+rh5_leg: mass 0.33821810347966374533 -> 0.33829069255504623515
Joints:
- joint left_hip_yaw: origin xyz=-0.0063999999999966063202 0.033999999999999308553 0.28550000000000003153 rpy=2.3275728331677864905e-16 1.1102230242191363653e-16 -1.222458086656465435e-13 -> xyz=-0.0093999999999961978553 0.033999999999999419575 0.28500000000000003109 rpy=9.2483505067470270586e-14 -1.7702340883530983486e-14 -6.9407309914055112031e-15
- joint right_hip_yaw: origin xyz=-0.0063999999999967980072 -0.034000000000000668576 0.28549999999999992051 rpy=1.2173498094825229595e-16 9.8900267199457111713e-23 -3.0336177719551955022e-13 -> xyz=-0.009399999999996381736 -0.03400000000000077266 0.28499999999999969802 rpy=8.8930762143875021541e-14 -1.7702340883511041083e-14 -2.3118089975893051414e-13

File: toddlerbot/robot_descriptions/assemblies/right_3R+RH5_leg/right_3R+RH5_leg.urdf (robot description, URDF)
Before this commit: robot right_3R+RH5_leg, 18 links, 17 joints
Links:
- link 12lf: mass 0.044782197690790462308 -> 0.044782197696050358993
- link 12lf_2: mass 0.044782197690790476186 -> 0.044782197696050358993
- link 12lf_rod_end: mass 0.00085420491177815895123 -> 0.00085420491177815905965
- link 12lf_rod_end_2: mass 0.00085420491177815895123 -> 0.00085420491177815905965
- link ank_pitch_link: mass 0.0042238381753791614387 -> 0.0042238381753791605713
- link ank_rr_link: mass 0.00042507093693768156772 -> 0.00042507093693768162193
- link ank_rr_link_2: mass 0.00042507093693768156772 -> 0.00042507093693768162193
- link ball_joint_ball: mass 4.4053796295264623832e-05 -> 4.4053796295264630609e-05
- link ball_joint_ball_2: mass 4.4053796295264623832e-05 -> 4.4053796295264630609e-05
- link hip_roll_link: mass 0.098012391483528665814 -> 0.098012391483528651936
- link hip_yaw_link: mass 0.009025883737097921064 -> 0.0090258837370979175946
- link right_hip_pitch_link: mass 0.09353906475262946385 -> 0.09361165381749210479
Joints:
- joint right_ank_B11: origin xyz=0.0079999999999999984318 0.015000000000000041078 -0.01150000000000000154 rpy=1.570796326794896558 -1.5520170643097170871 -1.5707963267946734032 -> xyz=0.0080000000000000019013 0.014999999999999985567 -0.011500000000000003275 rpy=1.5707963267948470421 -1.5520170643097048746 -1.570796326794996034
- joint right_ank_B12: origin xyz=0.008000000000000003636 0.015000000000000041078 0.028300000000000019584 rpy=-1.570796326794896558 -1.5521341097221632577 1.5707963267948059638 -> xyz=0.007999999999999972411 0.015000000000000041078 0.028299999999999964073 rpy=-1.570796326794911435 -1.5521341097221474925 1.5707963267949895947
- joint right_ank_B21: origin xyz=0 -2.7755575615628913511e-17 -0.011500000000000006745 rpy=-1.570796326794896558 -1.5664147454871475418 -1.5707963267939402119 -> xyz=-3.4694469519536141888e-18 0 -0.011499999999999996336 rpy=-1.5707963267952478326 -1.5664147454871724108 -1.5707963267955875608
- joint right_ank_B22: origin xyz=3.4694469519536141888e-18 0 -0.011499999999999998071 rpy=-1.57079632679489678 -1.5664376509754476263 -1.5707963267945079799 -> xyz=-3.4694469519536141888e-18 0 -0.01150000000000000154 rpy=-1.5707963267948972241 -1.5664376509754736055 -1.5707963267954201392
- joint right_ank_B31: origin xyz=6.9388939039072283776e-18 -0.0064387505004004086384 6.9388939039072283776e-18 rpy=-1.5707963267948970021 0.1691344003416279107 3.6048302674885136887e-16 -> xyz=-3.4694469519536141888e-18 -0.0064387505004003808828 0 rpy=-1.570796326794896558 0.16913440034157123382 1.0478833061949341326e-15
- joint right_ank_B32: origin xyz=3.4694469519536141888e-18 -0.0064387505004004086384 -6.9388939039072283776e-18 rpy=-1.570796326794896558 -0.17993145005738314657 -8.7569826039094258121e-17 -> xyz=-1.3877787807814456755e-17 -0.0064387505004004919051 3.4694469519536141888e-18 rpy=-1.57079632679489678 -0.17993145005742655629 -9.5188382896695163748e-16
- joint right_ank_R11: origin xyz=-0.018000000000000005579 0.016000000000000014211 -0.020599999999999996786 rpy=-3.5360359477892277706e-16 8.2839943819914169726e-16 -0.018779262484754637164 -> xyz=-0.018000000000000009048 0.015999999999999986455 -0.020599999999999996786 rpy=2.1199056220120536536e-16 1.7337184392140691041e-15 -0.018779262484772244607
- joint right_ank_R12: origin xyz=0.01799999999999999864 0.016000000000000069722 -0.020600000000000003725 rpy=3.1415926535897922278 1.1785067659504147721e-15 -3.1229304365172114721 -> xyz=0.017999999999999995171 0.015999999999999930944 -0.020600000000000003725 rpy=-3.1415926535897855665 2.3670754779580369231e-15 -3.1229304365172758651
- joint right_ank_R21: origin xyz=3.4694469519536141888e-18 -0.010000000000000008882 0 rpy=1.57079632679489678 -1.5664147454870704923 -1.5707963267947753216 -> xyz=-3.4694469519536141888e-18 -0.010000000000000008882 1.0408340855860842566e-17 rpy=1.5707963267949234254 -1.5664147454868782017 -1.5707963267941609242
- joint right_ank_R22: origin xyz=-3.4694469519536141888e-18 -0.0099999999999999533706 -3.4694469519536141888e-18 rpy=-1.570796326794896336 -1.5664376509754269762 1.5707963267952340658 -> xyz=-3.4694469519536141888e-18 -0.0099999999999998978595 1.0408340855860842566e-17 rpy=-1.570796326794896336 -1.5664376509751398725 1.5707963267966709164
- joint right_ank_act1: origin xyz=2.2722093412017030367e-06 1.8804402479588588903e-15 -0.074779998095388988677 rpy=-3.1415926535897829019 8.526808676235474948e-15 -2.2021168238260906413 -> xyz=2.2722093416596700344e-06 1.9567680809018384025e-15 -0.074779998095380800782 rpy=-3.1415926535897811256 5.9900329378763890994e-15 -2.2021168238260777628
- joint right_ank_act2: origin xyz=2.2722093371875529133e-06 -2.8553548414578244774e-15 -0.074779996992751840423 rpy=3.1415926535897922278 3.3072658899692120884e-15 -2.2021168238262864847 -> xyz=2.2722093354597683312e-06 -2.3106516700011070498e-15 -0.074779996992745872975 rpy=3.1415926535897926719 1.5779374385287525465e-15 -2.2021168238262811556
- joint right_ank_pitch: origin xyz=5.0979769291920753058e-19 0.099999999999999977796 -0.0062000000000000023842 rpy=-3.1415926535897926719 5.5511151131695266928e-17 -1.5707963267946121189 -> xyz=1.3701363056155178809e-18 0.10000000000000000555 -0.0061999999999999243216 rpy=-3.1415926535897917837 8.3351550965154899867e-16 -1.5707963267948104047
- joint right_ank_roll: origin xyz=2.0816681711721685133e-15 0.0015000000000089284361 -0.014599999999994599936 rpy=-1.5707963267951812192 1.5707963267946736252 0 -> xyz=3.3584246494910985348e-15 0.0015000000000102613543 -0.014599999999994976371 rpy=-1.5707963267951949859 1.5707963267946882802 0
- joint right_hip_pitch: origin xyz=0.024000000358075784801 -0.019000000000012132184 -0.01899999984755619542 rpy=-1.5707963267951119413 -1.5707963267945823649 0 -> xyz=-0.024000000716139988088 -0.01900000015244911189 -0.019000000152447529822 rpy=-1.5707963267949285324 -1.5707963267948303887 0
- joint right_hip_roll: origin xyz=0.018999999999999881567 -3.350043888987566044e-18 -0.026000000000000002276 rpy=2.9582283942363596652e-30 1.5707963267948799047 0 -> xyz=0.018999999999999881567 -3.6837601416870012287e-18 -0.026000000000000002276 rpy=3.141592653589793116 -1.570796326794896336 0
- joint right_knee: origin xyz=-8.4133172564547814973e-15 0.095999999999998697486 0.027400000000003574274 rpy=3.1415926535897926719 9.3467860356166481656e-14 -3.1415926535895137839 -> xyz=-8.6240005279115787276e-15 -0.096000000000003332667 0.0105999999999985689 rpy=-1.540481569708491688e-15 6.7185500345545200678e-16 3.1415926535894529437
