Commit message: Make the legs_only version walk

File: toddlerbot/robot_descriptions/assemblies/no_body/no_body.urdf (robot description, URDF)
Before this commit: robot no_body, 4 links, 3 joints
Links:
- removed link base_link
- removed link hip_link
- added link body_link, mass 0.1326329205818372603; collision mesh filename=package:///meshes/body_link_collision.stl; visual mesh filename=package:///meshes/body_link_visual.stl
- link left_3r+rh5_leg: mass 0.33316789121369472237 -> 0.33284223931512413319
- link right_3r+rh5_leg: mass 0.33316790148107094938 -> 0.33284223244644683959
Joints:
- removed joint base_link_to_base
- joint left_hip_yaw: origin xyz=-0.0063999999999966028508 0.033999999999999308553 0.28550000000000008704 rpy=1.2173498077216098975e-16 -2.7428229896967586736e-14 -8.3846071870935304412e-14 -> xyz=-0.0063999999999966045855 0.033999999999999447331 0.28550000000000008704 rpy=1.2173498077257119742e-16 -2.7439672175516685782e-14 -9.8815480994853422476e-14; parent hip_link -> body_link
- joint right_hip_yaw: parent hip_link -> body_link

File: toddlerbot/robot_descriptions/base_legs/base_legs.urdf (robot description, URDF)
Before this commit: robot base_legs, 38 links, 37 joints
Links:
- removed link base_link
- removed link hip_link
- added link body_link, mass 0.1326329205818372603; collision mesh filename=collisions/body_link_collision.stl; visual mesh filename=../assemblies/no_body/meshes/body_link_visual.stl
- link 12lf: mass 0.044782197696050352054 -> 0.044782197690790462308; geometry visual mesh filename=../assemblies/left_3R+RH5_leg/meshes/left_12lf_visual.stl
- link 12lf_2: mass 0.044782197696050352054 -> 0.044782197690790462308; geometry visual mesh filename=../assemblies/left_3R+RH5_leg/meshes/left_12lf_2_visual.stl
- link 12lf_3: mass 0.044782197696050352054 -> 0.044782197690790462308; geometry visual mesh filename=../assemblies/right_3R+RH5_leg/meshes/right_12lf_visual.stl
- link 12lf_4: mass 0.044782197696050358993 -> 0.044782197690790476186; geometry visual mesh filename=../assemblies/right_3R+RH5_leg/meshes/right_12lf_2_visual.s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
- link 12lf_rod: mass 0.0025088292483592140175 -> 0.0025088292483592144512; geometry visual mesh filename=../assemblies/left_3R+RH5_leg/meshes/left_12lf_rod_visual.s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
- link 12lf_rod_2: mass 0.0025088292483592140175 -> 0.0025088292483592144512; geometry visual mesh filename=../assemblies/left_3R+RH5_leg/meshes/left_12lf_rod_2_visual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
- link 12lf_rod_3: mass 0.0025088292483592140175 -> 0.0025088292483592144512; geometry visual mesh filename=../assemblies/right_3R+RH5_leg/meshes/right_12lf_rod_visual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
- link 12lf_rod_4: mass 0.0025088292483592140175 -> 0.0025088292483592144512; geometry visual mesh filename=../assemblies/right_3R+RH5_leg/meshes/right_12lf_rod_2_visu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
- link 12lf_rod_end: mass 0.00085420491177815905965 -> 0.00085420491177815895123; geometry visual mesh filename=../assemblies/left_3R+RH5_leg/meshes/left_12lf_rod_end_visu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
- link 12lf_rod_end_2: mass 0.00085420491177815905965 -> 0.00085420491177815895123; geometry visual mesh filename=../assemblies/left_3R+RH5_leg/meshes/left_12lf_rod_end_2_vi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
- link 12lf_rod_end_3: mass 0.00085420491177815905965 -> 0.00085420491177815895123; geometry visual mesh filename=../assemblies/right_3R+RH5_leg/meshes/right_12lf_rod_end_vi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
- link 12lf_rod_end_4: mass 0.00085420491177815905965 -> 0.00085420491177815895123; geometry visual mesh filename=../assemblies/right_3R+RH5_leg/meshes/right_12lf_rod_end_2_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
- link ank_pitch_link: mass 0.0042238381753791605713 -> 0.0042238381753791614387; geometry visual mesh filename=../assemblies/left_3R+RH5_leg/meshes/left_ank_pitch_link_vi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
- link ank_pitch_link_2: mass 0.0042238381753791605713 -> 0.0042238381753791614387; geometry visual mesh filename=../assemblies/right_3R+RH5_leg/meshes/right_ank_pitch_link_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
- link ank_roll_link: mass 0.013844478784760253648 -> 0.013844478784760248444; geometry collision mesh filename=collisions/left_ank_roll_link_collision.stl; visual mesh filename=../assemblies/left_3R+RH5_leg/meshes/left_ank_roll_link_vis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
- link ank_roll_link_2: mass 0.013844478784760253648 -> 0.013844478784760248444; geometry collision mesh filename=collisions/right_ank_roll_link_collision.stl; visual mesh filename=../assemblies/right_3R+RH5_leg/meshes/right_ank_roll_link_v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
- link ank_rr_link: geometry visual mesh filename=../assemblies/left_3R+RH5_leg/meshes/left_ank_rr_link_visua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
- link ank_rr_link_2: geometry visual mesh filename=../assemblies/left_3R+RH5_leg/meshes/left_ank_rr_link_2_vis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
- link ank_rr_link_3: geometry visual mesh filename=../assemblies/right_3R+RH5_leg/meshes/right_ank_rr_link_vis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
- link ank_rr_link_4: geometry visual mesh filename=../assemblies/right_3R+RH5_leg/meshes/right_ank_rr_link_2_v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
- link ball_joint_ball: mass 4.4053796295264630609e-05 -> 4.4053796295264623832e-05; geometry visual mesh filename=../assemblies/left_3R+RH5_leg/meshes/left_ball_joint_ball_v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
- link ball_joint_ball_2: mass 4.4053796295264630609e-05 -> 4.4053796295264623832e-05; geometry visual mesh filename=../assemblies/left_3R+RH5_leg/meshes/left_ball_joint_ball_2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
- link ball_joint_ball_3: mass 4.4053796295264630609e-05 -> 4.4053796295264623832e-05; geometry visual mesh filename=../assemblies/right_3R+RH5_leg/meshes/right_ball_joint_ball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
- link ball_joint_ball_4: mass 4.4053796295264630609e-05 -> 4.4053796295264623832e-05; geometry visual mesh filename=../assemblies/right_3R+RH5_leg/meshes/right_ball_joint_ball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
- link ball_joint_container: mass 4.803735642533054869e-05 -> 4.8037356425330562243e-05; geometry visual mesh filename=../assemblies/left_3R+RH5_leg/meshes/left_ball_joint_contai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
- link ball_joint_container_2: mass 4.803735642533054869e-05 -> 4.8037356425330562243e-05; geometry visual mesh filename=../assemblies/left_3R+RH5_leg/meshes/left_ball_joint_contai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
- link ball_joint_container_3: mass 4.803735642533054869e-05 -> 4.8037356425330562243e-05; geometry visual mesh filename=../assemblies/right_3R+RH5_leg/meshes/right_ball_joint_cont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
- link ball_joint_container_4: mass 4.803735642533054869e-05 -> 4.8037356425330562243e-05; geometry visual mesh filename=../assemblies/right_3R+RH5_leg/meshes/right_ball_joint_cont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
- link hip_roll_link: mass 0.098012391483528679692 -> 0.098012391483528651936; geometry collision mesh filename=collisions/left_hip_roll_link_collision.stl; visual mesh filename=../assemblies/left_3R+RH5_leg/meshes/left_hip_roll_link_vis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
- link hip_roll_link_2: mass 0.09801239148352869357 -> 0.098012391483528665814; geometry collision mesh filename=collisions/right_hip_roll_link_collision.stl; visual mesh filename=../assemblies/right_3R+RH5_leg/meshes/right_hip_roll_link_v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
- link hip_yaw_link: mass 0.009025883737097921064 -> 0.0090258837370979193293; geometry visual mesh filename=../assemblies/left_3R+RH5_leg/meshes/left_hip_yaw_link_visu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
- link hip_yaw_link_2: mass 0.009025883737097921064 -> 0.0090258837370979193293; geometry visual mesh filename=../assemblies/right_3R+RH5_leg/meshes/right_hip_yaw_link_vi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
- link left_calf_link: mass 0.016616268752102307527 -> 0.016290616864051549878; geometry collision mesh filename=collisions/left_calf_link_collision.stl; visual mesh filename=../assemblies/left_3R+RH5_leg/meshes/left_calf_link_visual.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
- link left_hip_pitch_link: mass 0.094084588454108858402 -> 0.094084588454108844524; geometry collision mesh filename=collisions/left_hip_pitch_link_collision.stl; visual mesh filename=../assemblies/left_3R+RH5_leg/meshes/left_hip_pitch_link_vi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
- link right_calf_link: mass 0.016616299594005391055 -> 0.016290630569901022595; geometry collision mesh filename=collisions/right_calf_link_collision.stl; visual mesh filename=../assemblies/right_3R+RH5_leg/meshes/right_calf_link_visua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
- link right_hip_pitch_link: mass 0.094084567879581956773 -> 0.094084567879581942895; geometry collision mesh filename=collisions/right_hip_pitch_link_collision.stl; visual mesh filename=../assemblies/right_3R+RH5_leg/meshes/right_hip_pitch_link_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
Joints:
- removed joint base_link_to_base
- joint left_ank_B11: origin xyz=0.0079999999999999966971 -0.015000000000000179856 0.028300000000000005707 rpy=-1.570796326794896558 1.4686290291020840382 1.5707963267948819031 -> xyz=0.0079999999999999880235 -0.015000000000000041078 0.028300000000000005707 rpy=-1.570796326794896558 1.469636014037934757 1.5707963267948754638
- joint left_ank_B12: origin xyz=0.008000000000000003636 -0.015000000000000124345 -0.01149999999999918622 rpy=-1.570796326794896558 -1.4687304067506412597 1.5707963267949098807 -> xyz=0.0080000000000001268013 -0.014999999999999791278 -0.011499999999999987663 rpy=-1.570796326794896558 -1.4697566621822597543 1.5707963267949038855
- joint left_ank_B21: origin xyz=6.9388939039072283776e-18 -2.7755575615628913511e-17 -0.011499999999999994602 rpy=1.57079632679489678 -1.4274634743672511838 1.570796326794916542 -> xyz=-6.9388939039072283776e-18 2.7755575615628913511e-17 -0.011499999999999999806 rpy=1.570796326794896558 -1.4285697747625467624 1.5707963267948807928
- joint left_ank_B22: origin xyz=-1.3877787807814456755e-17 8.3266726846886740532e-17 -0.011500000000000011949 rpy=1.570796326794896558 -1.4274430275990750427 -1.570796326794906328 -> xyz=-3.4694469519536141888e-17 -2.7755575615628913511e-16 -0.01149999999999988011 rpy=1.570796326794896558 -1.4285463212680655776 -1.5707963267948985564
- joint left_ank_B31: origin xyz=-1.4831885719601700657e-16 -0.0064387505004003253717 -6.9388939039072283776e-18 rpy=-1.570796326794896558 0.16912328473440299548 -4.2800865129067981483e-15 -> xyz=1.7347234759768070944e-18 -0.0064387505004004641496 1.3877787807814456755e-17 rpy=-1.57079632679489678 0.16913440034102092402 4.5559338426713504067e-15
- joint left_ank_B32: origin xyz=1.7347234759768070944e-17 -0.0064387505004004641496 1.3877787807814456755e-17 rpy=-1.5707963267948836794 -0.17992034540981183266 -3.9922693705457534994e-15 -> xyz=8.6736173798840354721e-18 -0.0064387505004005751719 6.9388939039072283776e-18 rpy=-1.5707963267948972241 -0.17993145005787733459 6.7429791500468328215e-16
- joint left_ank_R11: origin xyz=-0.010000000000000000208 0.012499999999999955591 -0.028000000000000004052 rpy=3.1415926535897775729 -1.1742161333363301013e-15 -0.10225158937860563679 -> xyz=-0.0099999999999999915345 0.012499999999999872324 -0.033600000000000004863 rpy=1.6323812772036896109e-17 1.4002646486553138019e-17 -0.10116031275705798798
- joint left_ank_R12: origin xyz=0.010000000000000001943 0.01249999999999990008 -0.027999999999999948541 rpy=3.1415926535897895633 4.4319359555376638558e-15 -3.0396078498296592585 -> xyz=0.0099999999999999984734 0.012499999999999761302 -0.033599999999999997924 rpy=3.1415926535897824579 9.4861357133311978266e-15 -3.0405529889788134312
- joint left_ank_R21: origin xyz=0.0021000000000000115796 0.010000000000000064393 -0.0018999999999999919731 rpy=-1.570796326794896558 1.4273561685593663118 -1.5707963267949194286 -> xyz=0 -0.010000000000000036637 -2.0816681711721685133e-17 rpy=-1.5707963267949025532 -1.4285697747629921839 1.5707963267949025532
- joint left_ank_R22: origin xyz=0.0021000000000000115796 -0.010000000000000092149 -0.001899999999999929523 rpy=-1.5707963267948974462 -1.4273357206756709381 -1.5707963267949238695 -> xyz=-6.9388939039072283776e-18 -0.010000000000000008882 0 rpy=1.570796326794896558 -1.4285463212677487199 -1.5707963267948970021
- joint left_ank_act1: origin xyz=2.272209354975407436e-06 9.4368957093138305936e-16 -0.072676675805820711851 rpy=-3.1415926535896590011 9.257153768608790258e-14 -2.2021168238262611716 -> xyz=2.2722093543023347273e-06 9.5756735873919751612e-16 -0.072660031604096092517 rpy=-3.1415926535896594451 8.5062006308179150635e-14 -2.2021168238262847083
- joint left_ank_act2: origin xyz=2.2722093495249062745e-06 -6.7446048745978259831e-15 -0.072678522047017385388 rpy=-3.1415926535895004612 6.2111251208581937571e-14 -2.2021168238262802674 -> xyz=2.2722093491484712802e-06 -6.5988881026157741871e-15 -0.07266003047881974819 rpy=-3.1415926535895000171 5.9280886354915822063e-14 -2.2021168238262815997
- joint left_ank_pitch: origin xyz=1.6466858937503582328e-18 -0.099999999999999922284 -0.0062000000000000058537 rpy=-3.1415926535897842342 8.6597368124280298137e-15 -1.5709041950953850364 -> xyz=9.1534583908775112557e-19 -0.10000000000000003331 -0.0061999999999999989148 rpy=3.1415926535897926719 -8.7927079361011792447e-15 -1.5707963267948961139
- joint left_ank_roll: origin xyz=3.3306690738754696213e-16 -0.0060999999999999726316 -0.014599999999999384304 rpy=-1.5707963257530275225 -1.5707136234809810915 -1.1504969698363094907e-09 -> xyz=2.2759572004815709079e-15 0.0015000000000041896053 -0.014599999999999611552 rpy=-1.570796326795051101 -1.5707963267944144992 0
- joint left_hip_pitch: origin xyz=-0.024000000716150875213 -0.01900000015244158319 -0.019000000152448091872 rpy=-1.5707963267945472818 1.5707963267948001906 0 -> xyz=-0.024000000716153851998 -0.019000000152441028078 -0.019000000152448098811 rpy=-1.570796326794478226 1.5707963267948015229 0
- joint left_hip_roll: origin xyz=0.019000000000000304839 -3.3605706708588417072e-18 -0.026000000000000279832 rpy=1.5707963267908973126 -1.5707806634981131833 1.5707963268130720191 -> xyz=0.019000000000000284023 -8.3919669538584410836e-16 -0.026000000000000463712 rpy=-3.1415926535897922278 -1.5707963267945732611 0
- joint left_hip_yaw: origin xyz=-0.0063999999999966028508 0.033999999999999308553 0.28550000000000008704 rpy=1.2173498077216098975e-16 -2.7428229896967586736e-14 -8.3846071870935304412e-14 -> xyz=-0.0063999999999966045855 0.033999999999999447331 0.28550000000000008704 rpy=1.2173498077257119742e-16 -2.7439672175516685782e-14 -9.8815480994853422476e-14; parent hip_link -> body_link
- joint left_knee: origin xyz=-3.1366467205128203278e-15 0.095999999999999752198 0.027400000000000007683 rpy=-3.1415926535897926719 -2.5420496490693392505e-17 -8.4866560936749634e-15 -> xyz=-6.5356617016366259295e-15 0.095999999999999696687 0.027400000000000260952 rpy=-3.1415926535897842342 1.6653345304510526278e-16 2.2176671495670943584e-16
- joint right_ank_B11: origin xyz=0.007999999999999972411 0.014999999999999957812 -0.011500000000000010214 rpy=1.5707963267948978903 -1.4686162729650020786 -1.5707963267948970021 -> xyz=0.0079999999999999689415 0.015000000000000124345 -0.011500000000000058786 rpy=1.5707963267948932273 -1.4696360140379622905 -1.5707963267948383823
- joint right_ank_B12: origin xyz=0.0079999999999997000594 0.015000000000000290878 0.02830000000000029714 rpy=-1.5707963267948978903 -1.468735614201923223 1.5707963267949029973 -> xyz=0.0080000000000000730249 0.015000000000000263123 0.028299999999999901623 rpy=-1.5707963267948388264 -1.4697566621826396727 1.5707963267950122432
- joint right_ank_B21: origin xyz=-2.0816681711721685133e-17 1.1102230246251565404e-16 -0.011499999999999998071 rpy=1.570796326794896558 -1.4274562579810237128 1.5707963267948950037 -> xyz=0 5.5511151231257827021e-17 -0.011499999999999998071 rpy=1.570796326794896558 -1.4285697747625634157 1.5707963267948530373
- joint right_ank_B22: origin xyz=-1.3877787807814456755e-17 -8.3266726846886740532e-17 -0.011499999999999991132 rpy=1.57079632679489678 -1.4274330297239778975 1.5707963267949012209 -> xyz=0 0 -0.011499999999999992867 rpy=1.5707963267949405228 -1.4285463212677880218 1.5707963267949816011
- joint right_ank_B31: origin xyz=-1.3010426069826053208e-18 -0.0064387505004002698605 6.9388939039072283776e-18 rpy=-1.570796326794896558 0.16913440034154619829 2.2885625266571218396e-16 -> xyz=-6.0715321659188248304e-18 -0.006438750500400436394 -1.3877787807814456755e-17 rpy=-1.5707963267948954478 0.16913440034160504011 5.0191724325132069355e-15
- joint right_ank_B32: origin xyz=-1.5178830414797062076e-17 -0.006438750500400436394 1.3877787807814456755e-17 rpy=-1.5707963267948854558 -0.17993145005756266963 -2.2505490007573420062e-15 -> xyz=-1.561251128379126385e-17 -0.0064387505004003531273 -1.3877787807814456755e-17 rpy=-1.5707963267948952257 -0.17993145005754265786 3.2634092460731900895e-15
- joint right_ank_R11: origin xyz=-0.0099999999999999932693 0.012500000000000038858 -0.02800000000000008038 rpy=-3.1415926535897926719 -7.9041717877712374794e-16 -0.10218566393336031561 -> xyz=-0.0099999999999999707179 0.012500000000000066613 -0.033600000000000039557 rpy=2.8867109174417181635e-14 -3.1302655555270997905e-14 -0.10116031275652562216
- joint right_ank_R12: origin xyz=0.0099999999999999967387 0.012499999999999761302 -0.02800000000000008038 rpy=-3.141592653589793116 2.6793361964555018776e-16 -3.0395375511005577884 -> xyz=0.010000000000000003678 0.012500000000000011102 -0.033600000000000004863 rpy=-3.1415926535897917837 -1.5904604637588844751e-15 -3.0405529889774984831
- joint right_ank_R21: origin xyz=0.0021000000000000254574 0.010000000000000092149 -0.0018999999999999919731 rpy=-1.57079632679489678 1.4274562579811747032 -1.570796326794901665 -> xyz=1.3877787807814456755e-17 -0.010000000000000008882 1.3877787807814456755e-17 rpy=-1.570796326794896558 -1.4285697747627732479 1.5707963267950297848
- joint right_ank_R22: origin xyz=0.0021000000000000185185 -0.010000000000000203171 -0.0019000000000000336065 rpy=-1.5707963267948961139 -1.4274330297240631626 -1.5707963267948974462 -> xyz=-1.3877787807814456755e-17 -0.010000000000000008882 2.7755575615628913511e-17 rpy=1.570796326794921649 -1.4285463212679851974 -1.5707963267949038855
- joint right_ank_act1: origin xyz=2.2722093427785666764e-06 1.2698175844150227931e-15 -0.072674150483189009497 rpy=-3.1415926535897811256 9.814572829871540247e-15 -2.2021168238260906413 -> xyz=2.2722093427421374834e-06 1.6375789613221058971e-15 -0.072660031604109970305 rpy=-3.1415926535897806815 7.845419351877858644e-15 -2.2021168238260604433
- joint right_ank_act2: origin xyz=2.2722093417776312307e-06 -2.3800406090401793335e-15 -0.072674285805652133474 rpy=3.141592653589793116 -4.1997988128928857096e-16 -2.2021168238262838202 -> xyz=2.2722093418418159994e-06 -2.3939183968479937903e-15 -0.072660030478818443678 rpy=-3.1415926535897926719 -5.822843740105227622e-15 -2.202116823826253178
- joint right_ank_pitch: origin xyz=1.1774009739933720541e-18 0.099999999999999922284 -0.0061999999999999937106 rpy=-3.141592653589793116 3.885801455584734555e-16 -1.5707963267948825692 -> xyz=-7.3090839045994630973e-18 0.099999999999999839018 -0.006199999999999821973 rpy=-3.1415926535897926719 3.8309199562601306947e-15 -1.57079632679489678
- joint right_ank_roll: origin xyz=1.7763568394002504647e-15 -0.0061000000000006751946 -0.014600000000001986389 rpy=1.5707963281806591738 1.5707907166914047981 -3.1415926522336965476 -> xyz=1.1018963519404678664e-14 0.0015000000000008478773 -0.014599999999995005862 rpy=-1.5707963267950115771 1.5707963267945974639 0
- joint right_hip_pitch: origin xyz=-0.024000000716145986762 -0.019000000152457990205 -0.019000000152453774827 rpy=-1.5707963267951818853 1.5707963267947633312 0 -> xyz=-0.024000000716146767388 -0.019000000152456290176 -0.019000000152450020885 rpy=-1.5707963267951789987 1.5707963267947586683 0
- joint right_hip_roll: origin xyz=-0.018999999999999885036 -3.3499987806511678644e-18 -0.026000000000000002276 rpy=-1.5707963266839728433 -1.5707907166912637997 1.5707963266641831179 -> xyz=-0.018999999999999891975 2.3744804088669454642e-18 -0.025999999999999984929 rpy=-3.3306690738820289997e-16 -1.570796326794896558 0
- joint right_hip_yaw: parent hip_link -> body_link
- joint right_knee: origin xyz=-2.4109230505694711738e-15 0.095999999999999821587 0.027399999999999948702 rpy=3.141592653589793116 -1.6870185802395130185e-16 3.1415926535897922278 -> xyz=-1.8318267252532356178e-15 0.095999999999998836264 0.027400000000000895861 rpy=3.1415926535897895633 -1.5829351718147190682e-16 -3.141592653589793116

Commit message: Update the real-world controller

File: toddlerbot/robot_descriptions/assemblies/no_body/no_body.urdf (robot description, URDF)
Before this commit: robot no_body, 3 links, 2 joints
Links:
- link left_3r+rh5_leg: mass 0.33284223931512413319 -> 0.3326398048030183574
- link right_3r+rh5_leg: mass 0.33284223244644683959 -> 0.33263981812552856354
Joints:
- joint left_hip_yaw: limit lower=-1.570796326794896558 upper=1.570796326794896558 effort=1 velocity=20 -> lower=-0.785398163397448279 upper=0.785398163397448279 effort=1 velocity=20; origin xyz=-0.0063999999999966045855 0.033999999999999447331 0.28550000000000008704 rpy=1.2173498077257119742e-16 -2.7439672175516685782e-14 -9.8815480994853422476e-14 -> xyz=-0.0063999999999966045855 0.03399999999999939182 0.28550000000000008704 rpy=2.327572832560927136e-16 4.9789962508008699149e-17 -1.0650377544034614197e-13
- joint right_hip_yaw: limit lower=-1.570796326794896558 upper=1.570796326794896558 effort=1 velocity=20 -> lower=-0.785398163397448279 upper=0.785398163397448279 effort=1 velocity=20; origin xyz=-0.006399999999996792803 -0.034000000000000661637 0.28549999999999997602 rpy=1.2173498094410956825e-16 -2.7428229798067236768e-14 -5.0714987764877150767e-13 -> xyz=-0.0063999999999967962724 -0.034000000000000661637 0.28549999999999992051 rpy=1.2173498094910643509e-16 -6.1232339957301087894e-17 -5.033057304260250785e-13

File: toddlerbot/robot_descriptions/toddlerbot_legs/toddlerbot_legs_isaac.urdf (robot description, URDF)
Before this commit: robot toddlerbot_legs, 37 links, 36 joints
Joints:
- joint left_ank_B11: type revolute -> fixed
- joint left_ank_B12: type revolute -> fixed
- joint left_ank_B21: type revolute -> fixed
- joint left_ank_B22: type revolute -> fixed
- joint left_ank_B31: type revolute -> fixed
- joint left_ank_B32: type revolute -> fixed
- joint left_ank_R11: type revolute -> fixed
- joint left_ank_R12: type revolute -> fixed
- joint left_ank_R21: type revolute -> fixed
- joint left_ank_R22: type revolute -> fixed
- joint left_ank_act1: type prismatic -> fixed
- joint left_ank_act2: type prismatic -> fixed
- joint right_ank_B11: type revolute -> fixed
- joint right_ank_B12: type revolute -> fixed
- joint right_ank_B21: type revolute -> fixed
- joint right_ank_B22: type revolute -> fixed
- joint right_ank_B31: type revolute -> fixed
- joint right_ank_B32: type revolute -> fixed
- joint right_ank_R11: type revolute -> fixed
- joint right_ank_R12: type revolute -> fixed
- joint right_ank_R21: type revolute -> fixed
- joint right_ank_R22: type revolute -> fixed
- joint right_ank_act1: type prismatic -> fixed
- joint right_ank_act2: type prismatic -> fixed
