Commit message: Update the body weight

File: toddlerbot/robot_descriptions/assemblies/no_body/no_body.urdf (robot description, URDF)
Before this commit: robot no_body, 3 links, 2 joints
Links:
- link body_link: mass 0.45859597582513078606 -> 1.0086534506317459403
Joints:
- joint left_hip_yaw: origin xyz=-0.0093999999999960781594 0.033999999999999308553 0.2850000000000000866 rpy=9.5014891068789895479e-14 -1.3383908635459135619e-14 -4.8061927846509854508e-15 -> xyz=-0.0093999999999961926511 0.033999999999999301614 0.28500000000000003109 rpy=9.5014891068790173158e-14 -1.7824800733959379972e-14 -7.7962407392327512346e-15
- joint right_hip_yaw: origin xyz=-0.0093999999999962672442 -0.034000000000000779599 0.28499999999999980904 rpy=9.1462148145193586205e-14 -1.3383908635439859014e-14 -2.1556636800468298824e-13 -> xyz=-0.009399999999996381736 -0.034000000000000807354 0.28499999999999969802 rpy=9.1462148145194911492e-14 -1.7824800733940560906e-14 -2.1356041234847096424e-13

File: toddlerbot/robot_descriptions/toddlerbot_legs/toddlerbot_legs.urdf (robot description, URDF)
Before this commit: robot toddlerbot_legs, 37 links, 36 joints
Links:
- link body_link: mass 0.45859597582513078606 -> 1.0086534506317459403
Joints:
- joint left_hip_yaw: origin xyz=-0.0093999999999960781594 0.033999999999999308553 0.2850000000000000866 rpy=9.5014891068789895479e-14 -1.3383908635459135619e-14 -4.8061927846509854508e-15 -> xyz=-0.0093999999999961926511 0.033999999999999301614 0.28500000000000003109 rpy=9.5014891068790173158e-14 -1.7824800733959379972e-14 -7.7962407392327512346e-15
- joint right_hip_yaw: origin xyz=-0.0093999999999962672442 -0.034000000000000779599 0.28499999999999980904 rpy=9.1462148145193586205e-14 -1.3383908635439859014e-14 -2.1556636800468298824e-13 -> xyz=-0.009399999999996381736 -0.034000000000000807354 0.28499999999999969802 rpy=9.1462148145194911492e-14 -1.7824800733940560906e-14 -2.1356041234847096424e-13

File: toddlerbot/robot_descriptions/toddlerbot_legs/toddlerbot_legs_isaac.urdf (robot description, URDF)
Before this commit: robot toddlerbot_legs, 37 links, 36 joints
Links:
- link body_link: mass 0.45859597582513078606 -> 1.0086534506317459403
Joints:
- joint left_hip_yaw: origin xyz=-0.0093999999999960781594 0.033999999999999308553 0.2850000000000000866 rpy=9.5014891068789895479e-14 -1.3383908635459135619e-14 -4.8061927846509854508e-15 -> xyz=-0.0093999999999961926511 0.033999999999999301614 0.28500000000000003109 rpy=9.5014891068790173158e-14 -1.7824800733959379972e-14 -7.7962407392327512346e-15
- joint right_hip_yaw: origin xyz=-0.0093999999999962672442 -0.034000000000000779599 0.28499999999999980904 rpy=9.1462148145193586205e-14 -1.3383908635439859014e-14 -2.1556636800468298824e-13 -> xyz=-0.009399999999996381736 -0.034000000000000807354 0.28499999999999969802 rpy=9.1462148145194911492e-14 -1.7824800733940560906e-14 -2.1356041234847096424e-13
