Commit message: Add gain and fix the joint direction

File: toddlerbot/robot_descriptions/assemblies/sysID_XC430/sysID_XC430.urdf (robot description, URDF)
Before this commit: robot sysID_XC430, 2 links, 1 joints
Links:
- link arm_430: mass 0.37449999999999999956 -> 0.37449999999999994404
Joints:
- joint joint_0: origin xyz=0.054999999999999715783 0.032699857927858969053 0.0055693959459660099393 rpy=5.1209490560719009338e-16 1.5707963267948958919 0 -> xyz=0.054999999999999681088 0.032699857927858962114 0.0055693959459660142761 rpy=1.57079632679489678 -5.5511151231258061214e-17 -1.5707963267948972241

File: toddlerbot/robot_descriptions/sysID_XC430/sysID_XC430.urdf (robot description, URDF)
Before this commit: robot sysID_XC430, 2 links, 1 joints
Links:
- link arm_430: mass 0.37449999999999999956 -> 0.37449999999999994404
Joints:
- joint joint_0: origin xyz=0.054999999999999715783 0.032699857927858969053 0.0055693959459660099393 rpy=5.1209490560719009338e-16 1.5707963267948958919 0 -> xyz=0.054999999999999681088 0.032699857927858962114 0.0055693959459660142761 rpy=1.57079632679489678 -5.5511151231258061214e-17 -1.5707963267948972241
