Commit message: Sysid the parameters

File: toddlerbot/robot_descriptions/assemblies/sysID_2XL430/sysID_2XL430.urdf (robot description, URDF)
Before this commit: robot sysID_2XL430, 2 links, 1 joints
Links:
- link 2xl430: mass 0.11906239148352866508 -> 0.1190623914835286512
- link arm_430: mass 0.094500000000000014544 -> 0.094500000000000042299
Joints:
- joint joint_0: origin xyz=0.096000000152447931279 0.032699858643998887253 0.0062193960984140176859 rpy=-1.5707963267948950037 2.9918979570903574849e-15 -1.5707963267948910069 -> xyz=0.057999999847552184684 0.032699858643998928887 0.0046193957935183882491 rpy=1.5707963267948972241 -5.7592819402422363305e-16 -1.5707963267948974462

File: toddlerbot/robot_descriptions/sysID_2XL430/sysID_2XL430.urdf (robot description, URDF)
Before this commit: robot sysID_2XL430, 2 links, 1 joints
Links:
- link 2xl430: mass 0.11906239148352866508 -> 0.1190623914835286512
- link arm_430: mass 0.094500000000000014544 -> 0.094500000000000042299
Joints:
- joint joint_0: origin xyz=0.096000000152447931279 0.032699858643998887253 0.0062193960984140176859 rpy=-1.5707963267948950037 2.9918979570903574849e-15 -1.5707963267948910069 -> xyz=0.057999999847552184684 0.032699858643998928887 0.0046193957935183882491 rpy=1.5707963267948972241 -5.7592819402422363305e-16 -1.5707963267948974462
