Commit message: Add knee constraints

File: toddlerbot/robot_descriptions/assemblies/left_leg_XM430/left_leg_XM430.urdf (robot description, URDF)
Before this commit: robot left_leg_XM430, 12 links, 11 joints
Links:
- added link bearing_683, mass 0.00048694686130641793437; collision mesh filename=package:///meshes/left_bearing_683_collision.stl; visual mesh filename=package:///meshes/left_bearing_683_visual.stl
- added link bearing_683_2, mass 0.00048694686130641793437; collision mesh filename=package:///meshes/left_bearing_683_2_collision.stl; visual mesh filename=package:///meshes/left_bearing_683_2_visual.stl
- added link knee_rod, mass 0.0013369468613064179954; collision mesh filename=package:///meshes/left_knee_rod_collision.stl; visual mesh filename=package:///meshes/left_knee_rod_visual.stl
- added link knee_rod_2, mass 0.0013369468613064179954; collision mesh filename=package:///meshes/left_knee_rod_2_collision.stl; visual mesh filename=package:///meshes/left_knee_rod_2_visual.stl
- added link xm430_plate, mass 0.0026999999999999997093; collision mesh filename=package:///meshes/left_xm430_plate_collision.stl; visual mesh filename=package:///meshes/left_xm430_plate_visual.stl
- link ank_motor_rod_short: mass 0.0017000000000000001221 -> 0.0017000000000000005558
- link ank_roll_link: mass 0.024800000000000002598 -> 0.024799999999999995659
- link ank_rr_link: mass 0.0014499999999999999001 -> 0.0014500000000000003338
- link ank_rr_link_2: mass 0.0014499999999999999001 -> 0.0014500000000000003338
- link hip_yaw_link: mass 0.01799999999999999864 -> 0.017999999999999991701
- link left_calf_link: mass 0.079607494529051442411 -> 0.079607494529051470167
- link left_hip_pitch_link_xm430: mass 0.035548688791081778371 -> 0.029200901345856091623
Joints:
- removed joint left_ank_L_rev_1
- removed joint left_ank_L_rev_2
- removed joint left_ank_S_rev_1
- removed joint left_ank_S_rev_2
- removed joint left_knee
- added joint left_ank_long_rev_1: type revolute, parent ank_roll_link, child ank_rr_link, origin xyz=-0.018000000000000009048 0.016000000000000014211 -0.020599999999999993316 rpy=-6.6713492090580732284e-15 1.1685759706219267798e-15 3.1233695685467375291, axis 0 0 1, limit lower=-1.570796326794896558 upper=1.570796326794896558 effort=1 velocity=20
- added joint left_ank_long_rev_2: type revolute, parent ank_rr_link, child ank_motor_rod_long, origin xyz=-8.7083118494035716139e-16 0.0099999999999995092814 -1.0408340855860842566e-16 rpy=-1.5707963267948947816 1.3320366994106509484 -1.570796326794906328, axis 0 0 1, limit lower=-1.570796326794896558 upper=1.570796326794896558 effort=1 velocity=20
- added joint left_ank_small_rev_1: type revolute, parent ank_roll_link, child ank_rr_link_2, origin xyz=0.01799999999999999864 0.016000000000000014211 -0.020600000000000007194 rpy=-2.3610930013721657667e-14 1.8265926123726939121e-15 0.026118548507372812278, axis 0 0 1, limit lower=-1.570796326794896558 upper=1.570796326794896558 effort=1 velocity=20
- added joint left_ank_small_rev_2: type revolute, parent ank_rr_link_2, child ank_motor_rod_short, origin xyz=9.0899510141184691747e-16 -0.0099999999999995647926 -1.0755285551056203985e-16 rpy=-1.570796326794896558 -1.2119133862909823307 -1.5707963267948985564, axis 0 0 1, limit lower=-1.570796326794896558 upper=1.570796326794896558 effort=1 velocity=20
- added joint left_knee_act: type revolute, parent left_hip_pitch_link_xm430, child xm430_plate, origin xyz=-0.00014999999999896470931 -0.061499999999999964417 -0.030400000000000516887 rpy=2.3599861887888032906e-15 -6.5336749892428132544e-16 1.5707963267949343056, axis 0 0 1, limit lower=0 upper=1.9198621771937625091 effort=1 velocity=20
- added joint left_knee_back_rev_1: type revolute, parent xm430_plate, child knee_rod_2, origin xyz=-0.013858192987669298857 -0.0057402514854763692087 -0.0050000000000000061756 rpy=9.6510604012704973759e-16 9.5675773494330421551e-15 -3.1374563631279994702, axis 0 0 1, limit lower=-6.283185307179586232 upper=6.283185307179586232 effort=1 velocity=20
- added joint left_knee_back_rev_2: type revolute, parent left_calf_link, child bearing_683_2, origin xyz=0.0057402514854763397184 -0.013858192987669382124 -0.026199999999999508404 rpy=-6.0044740500748964117e-15 -1.2959392046781909549e-14 1.5749326172567148507, axis 0 0 1, limit lower=-6.283185307179586232 upper=6.283185307179586232 effort=1 velocity=20
- added joint left_knee_front_rev_1: type revolute, parent xm430_plate, child knee_rod, origin xyz=0.013858192987669243346 0.0057402514854761515009 -0.0049999999999995308614 rpy=2.700462081678478798e-15 1.0789304203485744068e-14 -3.135795592727541159, axis 0 0 1, limit lower=-6.283185307179586232 upper=6.283185307179586232 effort=1 velocity=20
- added joint left_knee_front_rev_2: type revolute, parent left_calf_link, child bearing_683, origin xyz=-0.0057402514854764550775 0.013858192987669104568 -0.026199999999999393913 rpy=-1.5337469739246175927e-15 -1.4481776095066082806e-14 1.5765933876571727179, axis 0 0 1, limit lower=-6.283185307179586232 upper=6.283185307179586232 effort=1 velocity=20
- added joint left_knee_pitch: type revolute, parent left_hip_pitch_link_xm430, child left_calf_link, origin xyz=1.7789635663640724108e-15 -0.095999999999999974243 -0.0092000000000004491379 rpy=-2.7292527217646126502e-15 1.3010425524809599738e-16 1.3434393505081787056e-14, axis 0 0 1, limit lower=0 upper=1.9198621771937625091 effort=1 velocity=20
- joint left_ank_act_1: origin xyz=0.013499999999996521727 -0.044499999999990991206 0.004000000000004368117 rpy=-4.1933768254600954213e-13 -2.2608993309587937077e-13 -0.21173394130242484401 -> xyz=0.013499999999998390024 -0.044499999999992517763 0.0040000000000047931242 rpy=-4.6624689386713196717e-13 -1.8602011869043692927e-13 -0.21173394130248007761
- joint left_ank_act_2: origin xyz=0.013499999999999821171 -0.064499999999989482413 -0.024800000000000977513 rpy=-3.141592653589404982 8.5681358223374411603e-14 -0.22995607267358961212 -> xyz=0.013500000000005686271 -0.064499999999986984411 -0.024800000000000939349 rpy=-3.1415926535893090588 1.5796958800869922317e-14 -0.22995607267388284978
- joint left_ank_pitch: origin xyz=1.7782265719353869385e-16 -0.099999999999999367173 -0.01040000000000083219 rpy=-1.1833532294864106881e-14 4.9479686682726630759e-20 -3.141592653589793116 -> xyz=1.3606094101523029521e-15 -0.099999999999999422684 -0.010399999999999753192 rpy=-2.7292527261128833795e-15 8.7089742034479944265e-27 -3.1415926535897842342
- joint left_ank_roll: origin xyz=0.0014999999999999969955 -5.5511151231257827021e-17 -1.116728237660069567e-17 rpy=5.4670424773813653591e-26 1.570796326794896558 0 -> xyz=0.001500000000001442237 -2.7755575615628913511e-17 5.1608023410310011059e-16 rpy=2.1179511264814085754e-16 1.570796326794896336 0
- joint left_hip_pitch: origin xyz=-0.024000000716151929925 -0.01900000015243963683 -0.019000000152454777497 rpy=1.5707963267952702591 1.5707963267945455055 0 -> xyz=-0.024000000716151263791 -0.019000000152441041956 -0.019000000152457022229 rpy=1.5707963267952340658 1.5707963267945734831 0
- joint left_hip_roll: origin xyz=0.018999999999999999528 -2.8647205520269057584e-18 -0.026000000000000002276 rpy=3.141592653589793116 -1.570796326794896558 0 -> xyz=0.018999999999999999528 -4.8230661142633672945e-18 -0.026000000000000002276 rpy=-3.141592653589793116 -1.570796326794896558 0

File: toddlerbot/robot_descriptions/assemblies/right_leg_XM430/right_leg_XM430.urdf (robot description, URDF)
Before this commit: robot right_leg_XM430, 12 links, 11 joints
Links:
- added link bearing_683, mass 0.00048694686130641793437; collision mesh filename=package:///meshes/right_bearing_683_collision.stl; visual mesh filename=package:///meshes/right_bearing_683_visual.stl
- added link bearing_683_2, mass 0.00048694686130641793437; collision mesh filename=package:///meshes/right_bearing_683_2_collision.stl; visual mesh filename=package:///meshes/right_bearing_683_2_visual.stl
- added link knee_rod, mass 0.0013369468613064179954; collision mesh filename=package:///meshes/right_knee_rod_collision.stl; visual mesh filename=package:///meshes/right_knee_rod_visual.stl
- added link knee_rod_2, mass 0.0013369468613064179954; collision mesh filename=package:///meshes/right_knee_rod_2_collision.stl; visual mesh filename=package:///meshes/right_knee_rod_2_visual.stl
- added link xm430_plate, mass 0.0026999999999999997093; collision mesh filename=package:///meshes/right_xm430_plate_collision.stl; visual mesh filename=package:///meshes/right_xm430_plate_visual.stl
- link ank_motor_rod_short: mass 0.0017000000000000001221 -> 0.0017000000000000005558
- link ank_roll_link: mass 0.024800000000000009537 -> 0.024800000000000006067
- link ank_rr_link: mass 0.0014499999999999999001 -> 0.0014500000000000003338
- link ank_rr_link_2: mass 0.0014499999999999999001 -> 0.0014500000000000003338
- link hip_yaw_link: mass 0.01799999999999999864 -> 0.017999999999999991701
- link right_calf_link: mass 0.079607494529051442411 -> 0.079607494529051470167
- link right_hip_pitch_link_xm430: mass 0.035548688791081764493 -> 0.029200901345856091623
Joints:
- removed joint right_knee
- added joint right_knee_act: type revolute, parent right_hip_pitch_link_xm430, child xm430_plate, origin xyz=0.00015000000000002473377 -0.061500000000000235034 -0.030399999999999871569 rpy=8.8262730457708764429e-15 -1.5870629741237974938e-14 3.1415926535897829019, axis 0 0 1, limit lower=-1.9198621771937625091 upper=0 effort=1 velocity=20
- added joint right_knee_back_rev_1: type revolute, parent xm430_plate, child knee_rod_2, origin xyz=0.0057402514854763518615 0.013858192987669284979 -0.004999999999999997502 rpy=1.5753282257193089183e-14 1.0921500977742974577e-14 1.5650006493638364269, axis 0 0 1, limit lower=-6.283185307179586232 upper=6.283185307179586232 effort=1 velocity=20
- added joint right_knee_back_rev_2: type revolute, parent right_calf_link, child bearing_683_2, origin xyz=0.0057402514854763301774 0.013858192987669354368 -0.026199999999999879635 rpy=-2.3762645872631018006e-14 4.5147572622556449325e-15 3.1357969761587378699, axis 0 0 1, limit lower=-6.283185307179586232 upper=6.283185307179586232 effort=1 velocity=20
- added joint right_knee_front_rev_1: type revolute, parent xm430_plate, child knee_rod, origin xyz=-0.0057402514854763501267 -0.013858192987669298857 -0.004999999999999997502 rpy=1.3724907179645707302e-14 8.5838369743180810428e-15 1.5650043890091744903, axis 0 0 1, limit lower=-6.283185307179586232 upper=6.283185307179586232 effort=1 velocity=20
- added joint right_knee_front_rev_2: type revolute, parent right_calf_link, child bearing_683, origin xyz=-0.0057402514854760396112 -0.013858192987670631124 -0.026200000000000334133 rpy=-2.6211415108180604669e-14 2.1401571334997732958e-15 3.1358007158040726026, axis 0 0 1, limit lower=-6.283185307179586232 upper=6.283185307179586232 effort=1 velocity=20
- added joint right_knee_pitch: type revolute, parent right_hip_pitch_link_xm430, child right_calf_link, origin xyz=-1.0147615000199594353e-17 -0.095999999999999974243 -0.0091999999999999963751 rpy=-2.6534330288551032658e-14 1.1031692555244897755e-16 3.1415926535897837901, axis 0 0 1, limit lower=-1.9198621771937625091 upper=0 effort=1 velocity=20
- joint right_ank_L_rev_1: origin xyz=0.017999999999999981293 0.015999999999999847677 -0.020600000000000014133 rpy=6.2884229534673233247e-16 3.939086273962429945e-15 0.018223085042996144817 -> xyz=0.018000000000000074968 0.0159999999999997089 -0.020600000000000378425 rpy=-5.2246648675592445302e-15 7.3924679944672393986e-16 0.018223085042994146415
- joint right_ank_L_rev_2: origin xyz=-6.9388939039072283776e-18 -0.0099999999999996203037 3.1225022567582527699e-17 rpy=-1.5707963267948887864 -1.3320366994106427327 -1.5707963267948827912 -> xyz=0 -0.010000000000000619504 3.2265856653168611956e-16 rpy=-1.5707963267948976682 -1.3320366994106360714 -1.5707963267948898967
- joint right_ank_S_rev_1: origin xyz=-0.018000000000000026396 0.016000000000000735856 -0.02059999999999996903 rpy=-4.338977813478965687e-16 1.6392354569195739132e-16 3.1154741050825114357 -> xyz=-0.01799999999999993619 0.015999999999999042766 -0.020600000000000055767 rpy=-1.7258701733812934599e-15 2.598884774487275976e-15 3.1154741050825038862
- joint right_ank_S_rev_2: origin xyz=-2.7755575615628913511e-16 0.010000000000000563993 -1.561251128379126385e-16 rpy=-1.5707963267949354158 1.2119133862908570975 -1.5707963267949336394 -> xyz=-6.9388939039072283776e-18 0.010000000000000008882 0 rpy=-1.570796326794896558 1.2119133862908271215 -1.5707963267949023312
- joint right_ank_act_1: origin xyz=0.013499999999995838246 0.044500000000006201262 0.0040000000000029352354 rpy=-2.9762431821176080221e-13 -7.5970722241046912715e-14 0.21173394130155420712 -> xyz=0.013499999999995892022 0.044500000000006756373 0.0040000000000032995273 rpy=-2.8438542481158199641e-13 -8.7103248833400898994e-14 0.21173394130149567061
- joint right_ank_act_2: origin xyz=0.013500000000004725234 0.064500000000008106404 -0.024800000000001404254 rpy=-3.1415926535894733718 -2.3305959971649736532e-13 0.22995607267265857909 -> xyz=0.013500000000004461556 0.064500000000007967627 -0.02480000000000005117 rpy=-3.1415926535894955762 -2.1645240671651661488e-13 0.22995607267264547846
- joint right_ank_pitch: origin xyz=-4.0265291502142843319e-17 0.10000000000000000555 -0.010399999999999947481 rpy=-5.6239133145192868052e-16 -1.1344214119702528777e-16 3.141592653589793116 -> xyz=-1.4869836122455719424e-16 0.10000000000000000555 -0.010399999999997862343 rpy=-2.681188604470794026e-14 -2.1107204178545346346e-15 -3.1415926535897873428
- joint right_ank_roll: origin xyz=0.0014999999999999924418 2.7755575615628913511e-17 -1.3877787807814456755e-17 rpy=3.141592653589793116 -1.570796326794896336 0 -> xyz=0.0015000000000003571674 -1.4710455076283324161e-15 -7.6869934029222264371e-17 rpy=3.1415926535897922278 -1.5707963267948936714 0
- joint right_hip_pitch: origin xyz=-0.024000000716142638746 -0.019000000152444462831 -0.019000000152450562119 rpy=1.5707963267951012831 1.5707963267947298025 0 -> xyz=-0.024000000716142645685 -0.01900000015244446977 -0.019000000152450565588 rpy=1.5707963267950877384 1.5707963267947149255 0
- joint right_hip_roll: origin xyz=-0.018999999999999999528 3.3500438890367473614e-18 -0.026000000000000002276 rpy=1.737531809691582777e-30 -1.570796326794896558 0 -> xyz=-0.019000000000000509537 -6.4654958575016212571e-17 -0.026000000000000463712 rpy=-1.3163472222772945962e-16 -1.5707963267948941155 0
