Commit message: Update ankle IK

File: toddlerbot/robot_descriptions/assemblies/left_leg_XM430/left_leg_XM430.urdf (robot description, URDF)
Before this commit: robot left_leg_XM430, 17 links, 16 joints
Links:
- added link left_sole_link, mass 0.013899999999999999162; collision mesh filename=package:///meshes/left_sole_link_collision.stl; visual mesh filename=package:///meshes/left_sole_link_visual.stl
- link ank_motor_rod_long: mass 0.0021712857268636710437 -> 0.0021712857268636714773
- link ank_roll_link: mass 0.024799999999999995659 -> 0.010900000000000006906
- link ank_rr_link: mass 0.0014500000000000003338 -> 0.0014499999999999999001
- link ank_rr_link_2: mass 0.0014500000000000003338 -> 0.0014499999999999999001
- link hip_yaw_link: mass 0.017999999999999991701 -> 0.017999999999999995171
- link left_hip_pitch_link_xm430: mass 0.029200901345856091623 -> 0.029200901345856088154
- link xm430_plate: mass 0.0026999999999999997093 -> 0.0027000000000000001429
Joints:
- removed joint left_ank_small_rev_1
- removed joint left_ank_small_rev_2
- added joint left_ank_short_rev_1: type revolute, parent ank_roll_link, child ank_rr_link_2, origin xyz=0.017999999999999995171 0.015999999999999930944 -0.020600000000000003725 rpy=-1.0311645834080153765e-16 5.6225127493299344711e-16 0.026118548507380327101, axis 0 0 1, limit lower=-1.570796326794896558 upper=1.570796326794896558 effort=1 velocity=20
- added joint left_ank_short_rev_2: type revolute, parent ank_rr_link_2, child ank_motor_rod_short, origin xyz=-3.4694469519536141888e-18 -0.010000000000000008882 6.9388939039072283776e-18 rpy=-1.570796326794896558 -1.2119133862910269617 -1.5707963267948883423, axis 0 0 1, limit lower=-1.570796326794896558 upper=1.570796326794896558 effort=1 velocity=20
- added joint left_sole: type fixed, parent ank_roll_link, child left_sole_link, origin xyz=-9.2157184661267876891e-18 0.024999999999999994449 -0.022600000000000002032 rpy=1.570796326794896558 1.570796326794896336 0, axis 0 0 1, limit effort=1 velocity=20
- joint left_ank_act_1: origin xyz=0.013499999999998390024 -0.044499999999992517763 0.0040000000000047931242 rpy=-4.6624689386713196717e-13 -1.8602011869043692927e-13 -0.21173394130248007761 -> xyz=0.013499999999997966751 -0.044499999999993017363 0.0040000000000045363852 rpy=-4.512918339157919121e-13 -1.8247036451598847972e-13 -0.21173394130250977607
- joint left_ank_act_2: origin xyz=0.013500000000005686271 -0.064499999999986984411 -0.024800000000000939349 rpy=-3.1415926535893090588 1.5796958800869922317e-14 -0.22995607267388284978 -> xyz=0.013500000000004746051 -0.064499999999987706056 -0.024800000000001584666 rpy=-3.1415926535893468063 1.0027652560385185679e-14 -0.22995607267388484818
- joint left_ank_long_rev_1: origin xyz=-0.018000000000000009048 0.016000000000000014211 -0.020599999999999993316 rpy=-6.6713492090580732284e-15 1.1685759706219267798e-15 3.1233695685467375291 -> xyz=-0.018000000000000009048 0.015999999999999986455 -0.020600000000000000255 rpy=2.8727848934883667062e-16 -5.525634831039645443e-16 3.123369568546756625
- joint left_ank_long_rev_2: origin xyz=-8.7083118494035716139e-16 0.0099999999999995092814 -1.0408340855860842566e-16 rpy=-1.5707963267948947816 1.3320366994106509484 -1.570796326794906328 -> xyz=0 0.0099999999999998978595 0 rpy=-1.570796326794896558 1.3320366994106831449 -1.5707963267948692465
- joint left_ank_pitch: origin xyz=1.3606094101523029521e-15 -0.099999999999999422684 -0.010399999999999753192 rpy=-2.7292527261128833795e-15 8.7089742034479944265e-27 -3.1415926535897842342 -> xyz=1.883621368080212499e-17 -0.10000000000000011657 -0.010400000000000679534 rpy=-2.2204498262023812517e-16 1.8329922217212873636e-25 3.1415926535897735761
- joint left_ank_roll: origin xyz=0.001500000000001442237 -2.7755575615628913511e-17 5.1608023410310011059e-16 rpy=2.1179511264814085754e-16 1.570796326794896336 0 -> xyz=0.0014999999999999985133 0 1.4961989980299961189e-17 rpy=-8.1315126453654400003e-20 1.5707963267948643615 0
- joint left_hip_pitch: origin xyz=-0.024000000716151263791 -0.019000000152441041956 -0.019000000152457022229 rpy=1.5707963267952340658 1.5707963267945734831 0 -> xyz=-0.024000000716151277669 -0.019000000152441035017 -0.019000000152457018759 rpy=1.5707963267952340658 1.5707963267945346253 0
- joint left_hip_roll: origin xyz=0.018999999999999999528 -4.8230661142633672945e-18 -0.026000000000000002276 rpy=-3.141592653589793116 -1.570796326794896558 0 -> xyz=0.018999999999999996059 -3.3500438890367315688e-18 -0.026000000000000002276 rpy=-3.141592653589793116 -1.5707963267948934494 0
- joint left_knee_act: origin xyz=-0.00014999999999896470931 -0.061499999999999964417 -0.030400000000000516887 rpy=2.3599861887888032906e-15 -6.5336749892428132544e-16 1.5707963267949343056 -> xyz=-0.00015000000000000730522 -0.061500000000000019929 -0.030400000000000135247 rpy=-1.3229322588422224447e-16 -9.4099897484365535516e-16 1.570796326794896558
- joint left_knee_back_rev_1: origin xyz=-0.013858192987669298857 -0.0057402514854763692087 -0.0050000000000000061756 rpy=9.6510604012704973759e-16 9.5675773494330421551e-15 -3.1374563631279994702 -> xyz=-0.013858192987669326612 -0.0057402514854763449226 -0.0049999999999999992367 rpy=-9.8678816935430688804e-17 1.9053378273586200235e-14 -3.1384682709221709551
- joint left_knee_back_rev_2: origin xyz=0.0057402514854763397184 -0.013858192987669382124 -0.026199999999999508404 rpy=-6.0044740500748964117e-15 -1.2959392046781909549e-14 1.5749326172567148507 -> xyz=0.0057402514854763683413 -0.013858192987669298857 -0.026199999999999869227 rpy=-3.4182534048236850093e-16 -2.9781674294251979449e-14 1.5739207094625164984
- joint left_knee_front_rev_1: origin xyz=0.013858192987669243346 0.0057402514854761515009 -0.0049999999999995308614 rpy=2.700462081678478798e-15 1.0789304203485744068e-14 -3.135795592727541159 -> xyz=0.013858192987669298857 0.0057402514854763466573 -0.0050000000000000027062 rpy=-8.6224438144716539469e-15 8.3081819011448317203e-15 -3.138681925343421053
- joint left_knee_front_rev_2: origin xyz=-0.0057402514854764550775 0.013858192987669104568 -0.026199999999999393913 rpy=-1.5337469739246175927e-15 -1.4481776095066082806e-14 1.5765933876571727179 -> xyz=-0.0057402514854763518615 0.013858192987669382124 -0.026199999999999619427 rpy=-2.0062355525798721356e-14 -1.903658682771083387e-14 1.5737070550412661785
- joint left_knee_pitch: origin xyz=1.7789635663640724108e-15 -0.095999999999999974243 -0.0092000000000004491379 rpy=-2.7292527217646126502e-15 1.3010425524809599738e-16 1.3434393505081787056e-14 -> xyz=2.2117522176442097808e-17 -0.095999999999999974243 -0.0091999999999999824973 rpy=-9.7888408496123132916e-15 3.4506032502141251583e-16 2.567762240649299705e-15

File: toddlerbot/robot_descriptions/assemblies/right_leg_XM430/right_leg_XM430.urdf (robot description, URDF)
Before this commit: robot right_leg_XM430, 17 links, 16 joints
Links:
- added link right_sole_link, mass 0.013900000000000004366; collision mesh filename=package:///meshes/right_sole_link_collision.stl; visual mesh filename=package:///meshes/right_sole_link_visual.stl
- link ank_motor_rod_long: mass 0.0021712857268636710437 -> 0.0021712857268636714773
- link ank_roll_link: mass 0.024800000000000006067 -> 0.010900000000000006906
- link ank_rr_link: mass 0.0014500000000000003338 -> 0.0014499999999999999001
- link ank_rr_link_2: mass 0.0014500000000000003338 -> 0.0014499999999999999001
- link hip_yaw_link: mass 0.017999999999999991701 -> 0.017999999999999995171
- link right_calf_link: mass 0.079607494529051470167 -> 0.079607494529051442411
- link right_hip_pitch_link_xm430: mass 0.029200901345856091623 -> 0.029200901345856088154
- link xm430_plate: mass 0.0026999999999999997093 -> 0.0027000000000000001429
Joints:
- removed joint right_ank_L_rev_1
- removed joint right_ank_L_rev_2
- removed joint right_ank_S_rev_1
- removed joint right_ank_S_rev_2
- added joint right_ank_long_rev_1: type revolute, parent ank_roll_link, child ank_rr_link, origin xyz=0.017999999999999988232 0.016000000000000014211 -0.020600000000000014133 rpy=-6.5592393894058373872e-17 4.425192650031777037e-16 0.01822308504299342824, axis 0 0 1, limit lower=-1.570796326794896558 upper=1.570796326794896558 effort=1 velocity=20
- added joint right_ank_long_rev_2: type revolute, parent ank_rr_link, child ank_motor_rod_long, origin xyz=3.4694469519536141888e-18 -0.0099999999999998423483 1.0408340855860842566e-17 rpy=-1.570796326794896558 -1.3320366994106278558 -1.5707963267948821251, axis 0 0 1, limit lower=-1.570796326794896558 upper=1.570796326794896558 effort=1 velocity=20
- added joint right_ank_short_rev_1: type revolute, parent ank_roll_link, child ank_rr_link_2, origin xyz=-0.018000000000000015987 0.016000000000000069722 -0.020599999999999996786 rpy=-5.1243183935211302546e-15 2.3393195508611717606e-14 3.115474105082493228, axis 0 0 1, limit lower=-1.570796326794896558 upper=1.570796326794896558 effort=1 velocity=20
- added joint right_ank_short_rev_2: type revolute, parent ank_rr_link_2, child ank_motor_rod_short, origin xyz=3.4694469519536141888e-18 0.010000000000000008882 -6.9388939039072283776e-18 rpy=-1.570796326794896558 1.211913386290874195 -1.5707963267949693886, axis 0 0 1, limit lower=-1.570796326794896558 upper=1.570796326794896558 effort=1 velocity=20
- added joint right_sole: type fixed, parent ank_roll_link, child right_sole_link, origin xyz=-8.9988780316296868023e-18 0.025000000000000022204 -0.022600000000000002032 rpy=1.5707963267948985564 1.5707963267948945596 0, axis 0 0 1, limit effort=1 velocity=20
- joint right_ank_act_1: origin xyz=0.013499999999995892022 0.044500000000006756373 0.0040000000000032995273 rpy=-2.8438542481158199641e-13 -8.7103248833400898994e-14 0.21173394130149567061 -> xyz=0.013499999999996532135 0.044500000000006922907 0.0040000000000042501558 rpy=-3.1437427131281823257e-13 -4.4003633570199104585e-14 0.21173394130151781956
- joint right_ank_act_2: origin xyz=0.013500000000004461556 0.064500000000007967627 -0.02480000000000005117 rpy=-3.1415926535894955762 -2.1645240671651661488e-13 0.22995607267264547846 -> xyz=0.013500000000004223899 0.06450000000000813416 -0.024800000000001803241 rpy=-3.1415926535895222216 -2.1045472835494036236e-13 0.22995607267266512941
- joint right_ank_pitch: origin xyz=-1.4869836122455719424e-16 0.10000000000000000555 -0.010399999999997862343 rpy=-2.681188604470794026e-14 -2.1107204178545346346e-15 -3.1415926535897873428 -> xyz=2.5458137454050591327e-17 0.10000000000000003331 -0.010400000000000018605 rpy=1.5825612599836936462e-15 -6.6613381503165742443e-16 -3.1415926535897873428
- joint right_ank_roll: origin xyz=0.0015000000000003571674 -1.4710455076283324161e-15 -7.6869934029222264371e-17 rpy=3.1415926535897922278 -1.5707963267948936714 0 -> xyz=0.0014999999999999998144 2.7755575615628913511e-17 -1.4419888894057208972e-17 rpy=-3.141592653589793116 -1.5707963267948947816 0
- joint right_hip_pitch: origin xyz=-0.024000000716142645685 -0.01900000015244446977 -0.019000000152450565588 rpy=1.5707963267950877384 1.5707963267947149255 0 -> xyz=-0.024000000716143048141 -0.019000000152443574652 -0.019000000152453549312 rpy=1.5707963267951119413 1.5707963267946947195 0
- joint right_hip_roll: origin xyz=-0.019000000000000509537 -6.4654958575016212571e-17 -0.026000000000000463712 rpy=-1.3163472222772945962e-16 -1.5707963267948941155 0 -> xyz=-0.018999999999999999528 3.350043889036771243e-18 -0.026000000000000002276 rpy=2.5210948034330457424e-32 -1.5707963267948741315 0
- joint right_knee_act: origin xyz=0.00015000000000002473377 -0.061500000000000235034 -0.030399999999999871569 rpy=8.8262730457708764429e-15 -1.5870629741237974938e-14 3.1415926535897829019 -> xyz=0.00014999999999999350875 -0.06150000000000001299 -0.030400000000000010347 rpy=1.3560136669320073081e-26 -9.9920072221372949076e-16 3.1415926535897598093
- joint right_knee_back_rev_1: origin xyz=0.0057402514854763518615 0.013858192987669284979 -0.004999999999999997502 rpy=1.5753282257193089183e-14 1.0921500977742974577e-14 1.5650006493638364269 -> xyz=0.0057402514854763509941 0.013858192987669298857 -0.0050000000000000009714 rpy=4.9254694032746774356e-16 3.0156850660129127871e-15 1.5650006493638755067
- joint right_knee_back_rev_2: origin xyz=0.0057402514854763301774 0.013858192987669354368 -0.026199999999999879635 rpy=-2.3762645872631018006e-14 4.5147572622556449325e-15 3.1357969761587378699 -> xyz=0.0057402514854763726782 0.013858192987669298857 -0.026200000000000001066 rpy=-1.8771482682971376925e-15 -9.8530873122510239724e-18 3.1357969761587902724
- joint right_knee_front_rev_1: origin xyz=-0.0057402514854763501267 -0.013858192987669298857 -0.004999999999999997502 rpy=1.3724907179645707302e-14 8.5838369743180810428e-15 1.5650043890091744903 -> xyz=-0.005740251485476348392 -0.013858192987669284979 -0.0050000000000000044409 rpy=-1.2384470314426580757e-14 -1.7414957345394515419e-15 1.5650043890091922538
- joint right_knee_front_rev_2: origin xyz=-0.0057402514854760396112 -0.013858192987670631124 -0.026200000000000334133 rpy=-2.6211415108180604669e-14 2.1401571334997732958e-15 3.1358007158040726026 -> xyz=-0.0057402514854763431879 -0.013858192987669298857 -0.026199999999999994127 rpy=-5.4477346283033895825e-15 1.0965747154702311575e-14 3.1358007158040965834
- joint right_knee_pitch: origin xyz=-1.0147615000199594353e-17 -0.095999999999999974243 -0.0091999999999999963751 rpy=-2.6534330288551032658e-14 1.1031692555244897755e-16 3.1415926535897837901 -> xyz=-3.0242154156037831921e-17 -0.096000000000000015876 -0.0091999999999999963751 rpy=1.9802508686334247224e-15 -1.2115308756231608563e-14 3.1415926535897615857
