Commit message: Fix the ankle IK

File: toddlerbot/robot_descriptions/toddlerbot/toddlerbot.urdf (robot description, URDF)
Before this commit: robot toddlerbot, 77 links, 76 joints
Links:
- link ank_motor_rod_short: mass 0.001700000000000000339 -> 0.0017000000000000001221
- link ank_motor_rod_short_2: mass 0.001700000000000000339 -> 0.0017000000000000001221
- link ank_roll_link: mass 0.010900000000000003436 -> 0.010900000000000005171
- link ank_roll_link_2: mass 0.010900000000000003436 -> 0.010900000000000005171
- link ank_rr_link: mass 0.0014499999999999996832 -> 0.0014499999999999999001
- link ank_rr_link_2: mass 0.0014499999999999996832 -> 0.0014499999999999999001
- link ank_rr_link_3: mass 0.0014499999999999996832 -> 0.0014499999999999999001
- link ank_rr_link_4: mass 0.0014499999999999996832 -> 0.0014499999999999999001
- link hip_yaw_link: mass 0.017999999999999995171 -> 0.017999999999999988232
- link hip_yaw_link_2: mass 0.017999999999999995171 -> 0.017999999999999988232
- link neck_pitch_link: mass 0.11211553874797880459 -> 0.11211553874797881847
- link neck_yaw_link: mass 0.0085168305947458285143 -> 0.0085168305947458250449
- link right_hip_pitch_link_xm430: mass 0.11480090135030567022 -> 0.1148009013503056841
- link right_sole_link: mass 0.013900000000000007835 -> 0.013900000000000000897
- link spiral_bevel_1m_14t_30deg: mass 0.00067997563436136246491 -> 0.00067997563436136235649
- link spiral_bevel_1m_14t_30deg_2: mass 0.00067997563436136246491 -> 0.00067997563436136235649
- link spur_gear_(13_teeth): mass 0.00081469437497230876716 -> 0.00081469437497230855032
- link spur_gear_19_teeth: mass 0.0010993711450650535313 -> 0.0010993711450650533144
- link spur_gear_19_teeth_2: mass 0.0010993711450650535313 -> 0.0010993711450650533144
- link spur_gear_21_teeth: mass 0.001006304652831797701 -> 0.0010063046528317972673
- link spur_gear_21_teeth_2: mass 0.001006304652831797701 -> 0.0010063046528317972673
- link torso: mass 0.58490521749923596317 -> 0.5849052174992360742
- link xm430_plate: mass 0.0026999999999999992756 -> 0.0026999999999999997093
- link xm430_plate_2: mass 0.0026999999999999992756 -> 0.0026999999999999997093
Joints:
- joint left_ank_act_1: origin xyz=0.013499999999998150632 -0.044499999999994099831 0.004000000000003878925 rpy=-4.199339249962906148e-13 -1.7566169631614281426e-13 -0.21173394130241762756 -> xyz=0.013499999999998665845 -0.044499999999995792921 0.0040000000000033272829 rpy=-4.1712942586566064875e-13 -1.3694125076526491156e-13 -0.21173394130239187039
- joint left_ank_act_2: origin xyz=0.013500000000004789419 -0.064499999999987761568 -0.024800000000002139777 rpy=-3.1415926535893099469 1.5472440156112037689e-14 -0.22995607267390710815 -> xyz=0.013500000000004905645 -0.064499999999988205657 -0.024800000000003801642 rpy=-3.1415926535893086147 1.5803801662501837498e-14 -0.22995607267385878569
- joint left_ank_long_rev_1: origin xyz=-0.018000000000002184392 0.015999999999998931743 -0.020599999999999191874 rpy=5.6928860135513275759e-16 -8.1605439123400921334e-16 3.1233695685467459668 -> xyz=-0.018000000000000005579 0.016000000000000041966 -0.020599999999999996786 rpy=2.5433593855225719214e-15 -2.6604907481913981572e-15 3.123369568546706887
- joint left_ank_long_rev_2: origin xyz=-2.1579960041151480254e-15 0.0099999999999990651922 -8.08381139805192106e-16 rpy=-1.5707963267948954478 1.3320366994106502823 -1.5707963267948126251 -> xyz=-6.9388939039072283776e-18 0.010000000000000008882 0 rpy=-1.570796326794896558 1.3320366994106418446 -1.5707963267948841235
- joint left_ank_pitch: origin xyz=-5.8754783795495723237e-17 -0.10000000000000036637 -0.01040000000000218007 rpy=-6.6613494777492792143e-16 5.5008909826911396159e-25 3.141592653589793116 -> xyz=-5.02528144577274134e-17 -0.10000000000000103251 -0.010400000000005618292 rpy=-1.9984048432388552166e-15 1.6503134118918274764e-24 3.1415926535897926719
- joint left_ank_roll: origin xyz=0.0014999999999999241371 -2.7755575615628913511e-17 1.5796825653113799603e-16 rpy=2.1953071957139364813e-17 1.5707963267948659158 0 -> xyz=0.0014999999999999601326 -3.3306690738754696213e-16 -2.7549577202856667668e-16 rpy=3.7524749012299854346e-16 1.5707963267948723551 0
- joint left_ank_short_rev_1: origin xyz=0.017999999999999995171 0.015999999999999986455 -0.020600000000000000255 rpy=-3.244504776895705127e-16 1.1087098867936222379e-15 0.026118548507359652666 -> xyz=0.01799999999999999864 0.015999999999999986455 -0.020600000000000003725 rpy=-9.884525357415052455e-16 2.7480857223716701119e-15 0.026118548507321499158
- joint left_ank_short_rev_2: origin xyz=-3.4694469519536141888e-18 -0.010000000000000064393 -6.9388939039072283776e-18 rpy=-1.570796326794896558 -1.2119133862910156374 -1.570796326794871467 -> xyz=3.4694469519536141888e-18 -0.010000000000000064393 -3.4694469519536141888e-18 rpy=-1.570796326794896558 -1.2119133862909994281 -1.5707963267948890085
- joint left_hip_pitch: origin xyz=-0.024000000716151263791 -0.019000000152441045426 -0.019000000152457018759 rpy=1.5707963267952340658 1.5707963267945517227 0 -> xyz=-0.024000000716151263791 -0.019000000152441052365 -0.019000000152457018759 rpy=1.5707963267952342878 1.5707963267945523889 0
- joint left_hip_roll: origin xyz=0.018999999999999194616 -8.636160306239192055e-16 -0.026000000000000224321 rpy=-3.141592653589793116 -1.5707963267948843455 0 -> xyz=0.018999999999999999528 -3.3500438890369418804e-18 -0.026000000000000002276 rpy=-3.141592653589793116 -1.5707963267948679142 0
- joint left_hip_yaw_drive: origin xyz=-0.036999999999999241829 0.037100000000004858258 -0.039500000000001048162 rpy=1.5707963267947455677 -6.8514345590022702401e-13 -2.4160785457991476196e-13 -> xyz=-0.0369999999999981663 0.037100000000004268452 -0.039500000000001450617 rpy=1.5707963267947455677 -6.8515340787203273188e-13 -2.5801190558218208173e-13
- joint left_hip_yaw_driven: origin xyz=-0.036999999999999977351 0.041100000000000032341 -0.019499999999999986094 rpy=1.5707963267948990005 -1.5707963267948927832 0 -> xyz=-0.03699999999999998429 0.041100000000000011524 -0.019499999999999999972 rpy=1.5707963267948956698 -1.5707963267948861219 0
- joint left_knee_act: origin xyz=-0.00015000000000003010057 -0.061500000000000082379 -0.030400000000000440559 rpy=-3.9687967765302122778e-16 -3.2670861344266613268e-15 1.570796326794896558 -> xyz=-0.00014999999999999462006 -0.061500000000000019929 -0.030400000000000017286 rpy=-1.4293624205725000014e-15 -9.8302390852442860967e-15 1.5707963267948961139
- joint left_knee_back_rev_1: origin xyz=-0.013858192987669298857 -0.0057402514854763440552 -0.0050000000000000009714 rpy=-2.9668697207277861891e-16 -3.5495245422933824495e-15 -3.1384682709222704311 -> xyz=-0.013858192987669298857 -0.0057402514854763457899 -0.004999999999999997502 rpy=-8.90060916222688594e-16 -9.8269699236230981438e-15 -3.1384682709223161723
- joint left_knee_back_rev_2: origin xyz=0.0057402514854763839539 -0.01385819298766921559 -0.026199999999999640243 rpy=-3.4995571909695562261e-16 -2.90815686857019016e-14 1.5739207094624192429 -> xyz=0.0057402514854764186483 -0.013858192987669104568 -0.026199999999998932476 rpy=6.9110111902347492695e-16 -8.195589825460743709e-14 1.5739207094623721694
- joint left_knee_front_rev_1: origin xyz=0.013858192987669312735 0.0057402514854763440552 -0.0050000000000000009714 rpy=-8.8273423888544989682e-15 5.9762404835944504039e-15 -3.1386819253434037336 -> xyz=0.013858192987669284979 0.0057402514854763449226 -0.0050000000000000044409 rpy=-2.6482027166570673961e-14 1.7928721450783686478e-14 -3.1386819253434268262
- joint left_knee_front_rev_2: origin xyz=-0.0057402514854763735455 0.013858192987669520901 -0.026199999999998880434 rpy=-2.0198851465398702307e-14 -3.8607515872534395329e-14 1.5737070550412859404 -> xyz=-0.0057402514854764646185 0.013858192987669826213 -0.026199999999996635702 rpy=4.271508439620268736e-16 -1.1008548509280322482e-13 1.5737070550412617376
- joint left_knee_pitch: origin xyz=1.9837028473669800546e-17 -0.096000000000000015876 -0.0091999999999999738237 rpy=-2.9366522548798717986e-14 3.5724636926721053889e-16 4.1927868643308625526e-16 -> xyz=2.2567659777873647925e-17 -0.096000000000000001998 -0.0091999999999999321904 rpy=-8.2328001363584503113e-14 -1.0561188185116160038e-15 1.3586247681681341312e-15
- joint left_leg_fixed: origin xyz=-4.336808689942017736e-19 0 -0.004999999999999997502 rpy=1.3877787807813717198e-16 1.6653345369377375223e-16 1.373730595408674402e-16 -> xyz=-4.336808689942017736e-19 0 -0.004999999999999997502 rpy=3.9256239966020548641e-16 6.0371007920787862203e-16 5.9674487573614440696e-16
- joint left_sho_pitch: origin xyz=-0.0029999999999997528644 0.062000000000000436706 0.10523651076281793915 rpy=-1.5707963267948983344 -2.9907641379514081331e-14 -1.2153003607487542119e-15 -> xyz=-0.0029999999999997528644 0.062000000000000436706 0.10523651076281793915 rpy=-1.5707963267948983344 6.3108872417680944433e-30 -1.215300360748803713e-15
- joint left_sole: origin xyz=-9.1072982488782372457e-18 0.024999999999999994449 -0.022600000000000002032 rpy=1.570796326794896558 1.570796326794896336 0 -> xyz=-9.1072982488782372457e-18 0.024999999999999994449 -0.022600000000000005501 rpy=1.570796326794896558 1.570796326794896336 0
- joint right_ank_long_rev_1: origin xyz=0.017999999999999995171 0.015999999999999986455 -0.020600000000000007194 rpy=-2.0731393629286849282e-16 7.494126450902431242e-16 0.018223085043010137096 -> xyz=0.01800000000000012354 0.015999999999999792166 -0.020600000000000121686 rpy=-6.0785451271832051227e-15 6.1863719170134657294e-15 0.018223085043009137896
- joint right_ank_pitch: origin xyz=4.3837881646777831769e-17 0.10000000000000000555 -0.010399999999999944011 rpy=2.2204460560390508438e-16 3.5527136779803609004e-15 3.1415926535897873428 -> xyz=1.2797197023165297585e-16 0.10000000000000003331 -0.010400000000000304834 rpy=1.0436096434816955048e-14 1.5765166945884729896e-14 -3.1415926535897877869
- joint right_ank_roll: origin xyz=0.0015000000000000004649 0 -9.7578195523695399061e-19 rpy=-3.141592653589793116 -1.5707963267948956698 0 -> xyz=0.0014999999999999933092 -2.7755575615628913511e-17 1.5634195327240973938e-16 rpy=3.1415926535897877869 -1.5707963267948930053 0
- joint right_ank_short_rev_1: origin xyz=-0.018000000000000009048 0.015999999999999986455 -0.020599999999999996786 rpy=1.2085562754084012184e-16 -4.4422865000044981723e-16 3.115474105082512768 -> xyz=-0.017999999999999880679 0.015999999999999847677 -0.020599999999999920458 rpy=6.2273204751553159641e-15 -5.6155890983045670953e-15 3.1154741050825118798
- joint right_hip_pitch: origin xyz=-0.024000000716143048141 -0.019000000152443574652 -0.019000000152453545843 rpy=1.5707963267951119413 1.5707963267947440134 0 -> xyz=-0.024000000716143055079 -0.019000000152443571183 -0.019000000152453538904 rpy=1.5707963267951119413 1.5707963267947451236 0
- joint right_hip_roll: origin xyz=-0.019000000000000096673 2.0909656639487276466e-16 -0.025999999999999905131 rpy=-2.4415165121040963179e-28 -1.5707963267948938935 0 -> xyz=-0.018999999999999992589 1.141437663717389789e-17 -0.025999999999999988398 rpy=-2.6923160331957161178e-28 -1.5707963267948961139 0
- joint right_hip_yaw_drive: origin xyz=0.037000000000000345113 0.037100000000003956202 -0.039500000000000284883 rpy=1.5707963267948685804 -4.0596895443104855274e-13 -3.0450824182461770003e-13 -> xyz=0.037000000000000601852 0.037100000000004115797 -0.039499999999999833855 rpy=1.5707963267948861219 -4.0933607639229270295e-13 -3.6944432958726287967e-13
- joint right_hip_yaw_driven: origin xyz=0.036999999999999991229 0.041100000000000004585 -0.019499999999999982625 rpy=1.5707963267949123232 -1.5707963267948839015 0 -> xyz=0.036999999999999998168 0.041100000000000011524 -0.01950000000000001385 rpy=1.5707963267949343056 -1.5707963267948712449 0
- joint right_knee_act: origin xyz=0.00014999999999998383225 -0.061500000000000006051 -0.030400000000000024225 rpy=-3.3306690735930707292e-16 -2.9976021666231129079e-15 3.1415926535897913396 -> xyz=0.00014999999999997578205 -0.061499999999999985234 -0.030400000000000010347 rpy=-6.661338147321435048e-16 -5.9952043331935243853e-15 -3.1415926535897913396
- joint right_knee_back_rev_1: origin xyz=0.0057402514854763509941 0.013858192987669284979 -0.0050000000000000009714 rpy=1.4780745018405688374e-15 -6.0371120429764004227e-16 1.5650006493639538885 -> xyz=0.005740251485476348392 0.013858192987669160079 -0.0049999999999999489297 rpy=4.4930411149395298006e-15 -3.5910940522596879248e-15 1.5650006493639521121
- joint right_knee_front_rev_1: origin xyz=-0.0057402514854763475247 -0.013858192987669298857 -0.0050000000000000009714 rpy=-7.6843565403024876539e-16 -7.2468500696722411095e-16 1.5650043890089964105 -> xyz=-0.0057402514854763535962 -0.013858192987669201712 -0.0050000000000000009714 rpy=2.2465197872961639694e-15 -3.7120791298133282167e-15 1.5650043890089946341
- joint right_knee_pitch: origin xyz=1.1564389868401171602e-17 -0.096000000000000029754 -0.0092000000000000067835 rpy=-6.0024085179096384259e-15 1.3010426071629226535e-16 3.1415926535897913396 -> xyz=8.4950131805016210509e-17 -0.095999999999999904854 -0.0091999999999998940264 rpy=-3.3306690739599518911e-15 1.3010426078690428966e-16 -3.141592653589793116
- joint right_leg_fixed: origin xyz=1.7347234759768070944e-18 0 -0.0050000000000000044409 rpy=-1.5390466678866437645e-14 2.775557561557233123e-17 3.0000653983610458155e-17 -> xyz=4.336808689942017736e-19 -6.9388939039072283776e-18 -0.0050000000000000044409 rpy=-4.6198149465961399771e-14 1.8953383221571858275e-31 2.6475889041157274137e-29
- joint right_sho_pitch: origin xyz=-0.0030000000000001275646 -0.061999999999999985678 0.10523651076281731465 rpy=-1.570796326794896558 2.7165362863923079035e-14 3.1415926535897922278 -> xyz=-0.0030000000000001275646 -0.061999999999999985678 0.10523651076281731465 rpy=-1.570796326794896558 -9.4663308626521416649e-30 3.1415926535897922278
- joint right_sole: origin xyz=-9.2157184661267876891e-18 0.024999999999999938938 -0.022599999999999998562 rpy=1.5707963267949021091 1.5707963267948905628 0 -> xyz=-8.9988780316296868023e-18 0.024999999999999966693 -0.022599999999999998562 rpy=1.5707963267949132113 1.5707963267948785724 0
- joint waist_act_1: origin xyz=4.6183233744605796308e-18 0.019599999999999964673 -0.012749999999999978365 rpy=-1.570796326794896336 1.1669078612757080027 -3.1415926535897904515 -> xyz=-6.2837407918937052528e-16 0.01959999999999966977 -0.012749999999999159575 rpy=1.570796326794896558 1.570796326794493103 0
- joint waist_act_2: origin xyz=9.335172205065111088e-18 0.01959999999999997855 -0.032750000000000001332 rpy=-1.5707963267948990005 0.94250838602002218192 3.1415926535897860106 -> xyz=1.7857132216672699403e-18 0.019600000000000002837 -0.03275000000000001521 rpy=1.5707963267948883423 1.3463968515392001901 -8.4737581302220905773e-15
- joint waist_roll: origin xyz=9.4639684746659082843e-19 -0.022707865260692291359 0.012999999999999997669 rpy=1.5707963267948985564 -4.8988590961582989196e-15 1.01240703429886086e-14 -> xyz=4.3613235720115761641e-19 -0.022707865260692444015 0.013000000000000013281 rpy=1.570796326794896558 -2.3897582906932224823e-15 2.1266135278953062992e-16
- joint waist_yaw: origin xyz=0 2.168404344971008868e-19 1.7347234759768070944e-18 rpy=-3.1415926535897926719 3.3306690738754839194e-16 -1.5056527786227653642 -> xyz=-7.6501305290577192864e-16 -3.9884543972351746136e-15 -7.771561172376095783e-16 rpy=-3.1415926535897922278 -2.0665189604238262613e-16 -1.5707963267945077579

Commit message: Update the sole mass

File: toddlerbot/robot_descriptions/assemblies/left_leg_XM430/left_leg_XM430.urdf (robot description, URDF)
Before this commit: robot left_leg_XM430, 18 links, 17 joints
Links:
- link ank_roll_link: mass 0.010899999999999999967 -> 0.012900000000000000008
- link hip_yaw_link: mass 0.017999999999999995171 -> 0.017999999999999991701
- link left_hip_pitch_link_xm430: mass 0.1148009013503056841 -> 0.11480090135030567022
- link left_sole_link: mass 0.013899999999999997427 -> 0.02300000000000000655
- link xm430_plate: mass 0.0026999999999999997093 -> 0.0027000000000000001429
Joints:
- joint left_sole: origin xyz=-9.1072982488782372457e-18 0.024999999999999994449 -0.022600000000000002032 rpy=1.570796326794896558 1.570796326794896336 0 -> xyz=8.123926878433884724e-16 0.024999999999999994449 -0.022599999999999929173 rpy=1.570796326794896558 1.570796326794896336 0

File: toddlerbot/robot_descriptions/assemblies/right_leg_XM430/right_leg_XM430.urdf (robot description, URDF)
Before this commit: robot right_leg_XM430, 18 links, 17 joints
Links:
- link ank_roll_link: mass 0.010899999999999999967 -> 0.012900000000000000008
- link hip_yaw_link: mass 0.017999999999999995171 -> 0.017999999999999991701
- link right_hip_pitch_link_xm430: mass 0.11480090135030567022 -> 0.1148009013503056841
- link right_sole_link: mass 0.013900000000000007835 -> 0.02300000000000001002
- link xm430_plate: mass 0.0026999999999999997093 -> 0.0027000000000000001429
Joints:
- joint right_sole: origin xyz=-8.8904578143811363589e-18 0.024999999999999966693 -0.022599999999999995093 rpy=1.570796326794896558 1.570796326794896336 0 -> xyz=-8.0230960763927328117e-18 0.024999999999999966693 -0.022599999999999995093 rpy=1.570796326794896558 1.570796326794896336 0

File: toddlerbot/robot_descriptions/toddlerbot/toddlerbot.urdf (robot description, URDF)
Before this commit: robot toddlerbot, 77 links, 76 joints
Links:
- link ank_roll_link: mass 0.010899999999999999967 -> 0.012900000000000000008
- link ank_roll_link_2: mass 0.010899999999999999967 -> 0.012900000000000000008
- link hip_yaw_link: mass 0.017999999999999995171 -> 0.017999999999999991701
- link hip_yaw_link_2: mass 0.017999999999999995171 -> 0.017999999999999991701
- link left_hip_pitch_link_xm430: mass 0.1148009013503056841 -> 0.11480090135030567022
- link left_sole_link: mass 0.013899999999999997427 -> 0.02300000000000000655
- link right_hip_pitch_link_xm430: mass 0.11480090135030567022 -> 0.1148009013503056841
- link right_sole_link: mass 0.013900000000000007835 -> 0.02300000000000001002
- link xm430_plate: mass 0.0026999999999999997093 -> 0.0027000000000000001429
- link xm430_plate_2: mass 0.0026999999999999997093 -> 0.0027000000000000001429
Joints:
- joint left_sole: origin xyz=-9.1072982488782372457e-18 0.024999999999999994449 -0.022600000000000002032 rpy=1.570796326794896558 1.570796326794896336 0 -> xyz=8.123926878433884724e-16 0.024999999999999994449 -0.022599999999999929173 rpy=1.570796326794896558 1.570796326794896336 0
- joint right_sole: origin xyz=-8.8904578143811363589e-18 0.024999999999999966693 -0.022599999999999995093 rpy=1.570796326794896558 1.570796326794896336 0 -> xyz=-8.0230960763927328117e-18 0.024999999999999966693 -0.022599999999999995093 rpy=1.570796326794896558 1.570796326794896336 0

Commit message: Update the hip roll joint limit

File: toddlerbot/robot_descriptions/assemblies/left_leg_XM430/left_leg_XM430.urdf (robot description, URDF)
Before this commit: robot left_leg_XM430, 17 links, 16 joints
Links:
- link ank_pitch_link: mass 0.0042238381753791605713 -> 0.0042238381753791614387
- link ank_rr_link: mass 0.0014500000000000001169 -> 0.0014499999999999996832
- link ank_rr_link_2: mass 0.0014500000000000001169 -> 0.0014499999999999996832
- link hip_roll_link: mass 0.11059999999836236939 -> 0.11059999999836234164
- link hip_yaw_link: mass 0.017999999999999995171 -> 0.018000000000000009048
- link xm430_plate: mass 0.0026999999999999992756 -> 0.0026999999999999997093
Joints:
- joint left_hip_roll: limit lower=-0.785398163397448279 upper=1.570796326794896558 effort=1 velocity=20 -> lower=-0.785398163397448279 upper=0.785398163397448279 effort=1 velocity=20

File: toddlerbot/robot_descriptions/assemblies/right_leg_XM430/right_leg_XM430.urdf (robot description, URDF)
Before this commit: robot right_leg_XM430, 17 links, 16 joints
Links:
- link ank_pitch_link: mass 0.0042238381753791605713 -> 0.0042238381753791614387
- link ank_rr_link: mass 0.0014500000000000001169 -> 0.0014499999999999996832
- link ank_rr_link_2: mass 0.0014500000000000001169 -> 0.0014499999999999996832
- link hip_roll_link: mass 0.11059999999836236939 -> 0.11059999999836234164
- link hip_yaw_link: mass 0.017999999999999995171 -> 0.018000000000000009048
- link right_calf_link: mass 0.086799999986183581924 -> 0.086799999986183568046
- link xm430_plate: mass 0.0026999999999999992756 -> 0.0026999999999999997093
Joints:
- joint right_hip_roll: limit lower=-0.785398163397448279 upper=1.570796326794896558 effort=1 velocity=20 -> lower=-0.785398163397448279 upper=0.785398163397448279 effort=1 velocity=20

File: toddlerbot/robot_descriptions/toddlerbot/toddlerbot.urdf (robot description, URDF)
Before this commit: robot toddlerbot, 75 links, 74 joints
Links:
- link ank_pitch_link: mass 0.0042238381753791605713 -> 0.0042238381753791614387
- link ank_pitch_link_2: mass 0.0042238381753791605713 -> 0.0042238381753791614387
- link ank_rr_link: mass 0.0014500000000000001169 -> 0.0014499999999999996832
- link ank_rr_link_2: mass 0.0014500000000000001169 -> 0.0014499999999999996832
- link ank_rr_link_3: mass 0.0014500000000000001169 -> 0.0014499999999999996832
- link ank_rr_link_4: mass 0.0014500000000000001169 -> 0.0014499999999999996832
- link hip_roll_link: mass 0.11059999999836236939 -> 0.11059999999836234164
- link hip_roll_link_2: mass 0.11059999999836236939 -> 0.11059999999836234164
- link hip_yaw_link: mass 0.017999999999999995171 -> 0.018000000000000009048
- link hip_yaw_link_2: mass 0.017999999999999995171 -> 0.018000000000000009048
- link right_calf_link: mass 0.086799999986183581924 -> 0.086799999986183568046
- link xm430_plate: mass 0.0026999999999999992756 -> 0.0026999999999999997093
- link xm430_plate_2: mass 0.0026999999999999992756 -> 0.0026999999999999997093
Joints:
- joint left_hip_roll: limit lower=-0.785398163397448279 upper=1.570796326794896558 effort=1 velocity=20 -> lower=-0.785398163397448279 upper=0.785398163397448279 effort=1 velocity=20
- joint right_hip_roll: limit lower=-0.785398163397448279 upper=1.570796326794896558 effort=1 velocity=20 -> lower=-0.785398163397448279 upper=0.785398163397448279 effort=1 velocity=20
