Commit message: Update the toddlerbot xml

File: toddlerbot/robot_descriptions/assemblies/left_leg_XM430/left_leg_XM430.urdf (robot description, URDF)
Before this commit: robot left_leg_XM430, 17 links, 16 joints
Links:
- link ank_motor_rod_short: mass 0.0017000000000000005558 -> 0.0017000000000000001221
- link ank_roll_link: mass 0.019499999999999989564 -> 0.027200000000000008893
- link ank_rr_link: mass 0.0014499999999999996832 -> 0.0014499999999999999001
- link ank_rr_link_2: mass 0.0014499999999999996832 -> 0.0014499999999999999001
- link hip_yaw_link: mass 0.018000000000000009048 -> 0.017999999999999988232
- link left_hip_pitch_link_xm430: mass 0.1148009013503056841 -> 0.11480090135030569798
- link xm430_plate: mass 0.0026999999999999997093 -> 0.0026999999999999992756
Joints:
- joint left_ank_long_rev_1: origin xyz=-0.018000000000000015987 0.01599999999999926481 -0.020600000000001391504 rpy=-2.876394309884160705e-16 1.6317439732762683578e-16 3.1233695685467286474 -> xyz=-0.018000000000000064559 0.015999999999999292566 -0.020600000000001391504 rpy=-2.876394309884160705e-16 1.6317439732762683578e-16 3.1233695685467286474
- joint left_ank_roll: origin xyz=0.0015000000000000002481 2.7755575615628913511e-17 3.2742905609062233907e-17 rpy=9.9573127520767875392e-16 1.570796326794891673 0 -> xyz=0.0014999999999999995975 0 -1.5395670849294162963e-17 rpy=9.9573127520767875392e-16 1.570796326794891673 0
- joint left_ank_short_rev_1: origin xyz=0.018000000000000002109 0.015999999999999986455 -0.020600000000000010664 rpy=4.2172831995673088897e-16 -4.4678623027074358005e-17 0.026118548507422217203 -> xyz=0.017999999999999953537 0.016000000000000014211 -0.020600000000000010664 rpy=4.2172831995673088897e-16 -4.4678623027074358005e-17 0.026118548507422217203

File: toddlerbot/robot_descriptions/assemblies/right_leg_XM430/right_leg_XM430.urdf (robot description, URDF)
Before this commit: robot right_leg_XM430, 17 links, 16 joints
Links:
- link ank_motor_rod_short: mass 0.0017000000000000005558 -> 0.0017000000000000001221
- link ank_roll_link: mass 0.019499999999999989564 -> 0.027200000000000008893
- link ank_rr_link: mass 0.0014499999999999996832 -> 0.0014499999999999999001
- link ank_rr_link_2: mass 0.0014499999999999996832 -> 0.0014499999999999999001
- link hip_yaw_link: mass 0.018000000000000009048 -> 0.017999999999999988232
- link right_calf_link: mass 0.086799999986183568046 -> 0.086799999986183554168
- link right_hip_pitch_link_xm430: mass 0.1148009013503056841 -> 0.11480090135030567022
- link xm430_plate: mass 0.0026999999999999997093 -> 0.0026999999999999992756
Joints:
- joint right_ank_long_rev_1: origin xyz=0.017999999999999995171 0.016000000000000014211 -0.020600000000000007194 rpy=2.4036779374278231896e-16 5.7386734097817399387e-16 0.018223085043007757056 -> xyz=0.01799999999999999864 0.015999999999999764411 -0.020600000000000132094 rpy=-7.8386807614170502355e-15 7.211088289180617976e-16 0.018223085043007757056
- joint right_ank_roll: origin xyz=0.0015000000000000002481 2.7755575615628913511e-17 1.2143064331837649661e-17 rpy=-8.0803901893659494053e-15 1.5707963267948927832 0 -> xyz=0.001499999999999998947 8.3266726846886740532e-17 1.3660947373317355868e-17 rpy=6.1391486757704172424e-30 1.5707963267948927832 0
- joint right_ank_short_rev_1: origin xyz=-0.018000000000000012518 0.016000000000000014211 -0.020599999999999993316 rpy=1.6033225897674528336e-14 -1.3300018467937457486e-14 3.1154741050824821258 -> xyz=-0.018000000000000009048 0.015999999999999764411 -0.020600000000000118217 rpy=2.411086010918130345e-14 -1.3088994399411267302e-14 3.1154741050824821258

File: toddlerbot/robot_descriptions/assemblies/toddlerbot/toddlerbot.urdf (robot description, URDF)
Before this commit: robot toddlerbot, 17 links, 16 joints
Links:
- link neck_pitch_link: mass 0.11211553874797881847 -> 0.11211553874797880459
- link neck_yaw_link: mass 0.0085168305947458267796 -> 0.0085168305947458250449
- link spiral_bevel_1m_14t_30deg: mass 0.00067997563436136246491 -> 0.00067997563436136257333
- link spiral_bevel_1m_14t_30deg_2: mass 0.00067997563436136246491 -> 0.00067997563436136257333
- link spur_1m_20t: mass 0.0015534950290892286448 -> 0.0015534950290892282111
- link spur_gear_(13_teeth): mass 0.00081469437497230865874 -> 0.00081469437497230876716
- link spur_gear_19_teeth: mass 0.0010993711450650533144 -> 0.0010993711450650535313
- link spur_gear_19_teeth_2: mass 0.0010993711450650533144 -> 0.0010993711450650535313
- link spur_gear_21_teeth: mass 0.0010063046528317972673 -> 0.0010063046528317974842
- link spur_gear_21_teeth_2: mass 0.0010063046528317972673 -> 0.0010063046528317974842
- link torso: mass 0.58475267652546314423 -> 0.59420757418972613983
- link waist_link: mass 0.16631953490612458313 -> 0.1663195349061246664
Joints:
- joint left_hip_yaw_drive: origin xyz=-0.036999999999998194056 0.037100000000006128076 -0.039500000000001291023 rpy=-1.5707963267949545116 -4.7906511943294847217e-13 -3.592506663906207747e-13 -> xyz=-0.03699999999999847855 0.037100000000005933787 -0.039500000000000194678 rpy=-1.5707963267949540676 -4.7732588435988597417e-13 -3.5949390257278751872e-13
- joint left_hip_yaw_driven: origin xyz=-0.037000000000000012046 0.041099999999999997646 -0.0194999999999999514 rpy=-1.5707963267948990005 -1.570796326794896558 0 -> xyz=-0.037000000000000005107 0.04110000000000003928 -0.019500000000000024258 rpy=-1.5707963267948961139 -1.5707963267948883423 0
- joint left_leg_fixed: origin xyz=0 0 0.004999999999999997502 rpy=3.1415926535897873428 -0 -1.6681280046507162628e-30 -> xyz=0 0 0.0050000000000000044409 rpy=3.141592653589793116 -2.7755575615625073977e-17 -3.33066907387546617e-16
- joint left_sho_pitch: origin xyz=-0.0030000000000065664245 0.062000000000004926171 0.10423651076282140771 rpy=-1.5707963267949054398 -3.6755753074147447628e-14 3.6857314245917344439e-14 -> xyz=-0.0030000000000002949654 0.062000000000001082023 0.10423651076281743866 rpy=-1.5707963267949081043 -4.127643409825574977e-14 3.4723733359249779961e-14
- joint neck_pitch_drive: origin xyz=-1.4224732503009818174e-16 0.015649999999999136824 -0.0087999999999959568897 rpy=-2.4492935983152098954e-16 -2.1427228763620856097e-15 -1.570796326794896558 -> xyz=-8.3266726846886740532e-17 0.015649999999999109068 -0.0087999999999961303621 rpy=-6.1232340018137966949e-17 -1.865637580072612815e-26 -1.570796326794896558
- joint neck_pitch_driven: origin xyz=3.7500001368040436489e-10 -0.0051500000614753682626 0.027499999999999830136 rpy=1.57079632679489678 1.7322096859329345721e-15 -3.1415926535897922278 -> xyz=3.7500136329526867485e-10 -0.0051500000614755217856 0.027499999999999982792 rpy=1.570796326794896558 8.6610484296647231505e-16 3.141592653589793116
- joint neck_yaw_drive: origin xyz=-0.0050000000000041591036 2.1706564040395755645e-15 0.12148651076282282468 rpy=-4.7086950490309927255e-15 -3.2377166610426843676e-14 2.947288666540578667e-14 -> xyz=-0.0049999999999993625932 3.342147474086756384e-17 0.12148651076281766215 rpy=7.9879995913373272052e-15 8.0038275409654909883e-15 -5.4161669716995088817e-15
- joint neck_yaw_driven: origin xyz=0.015999999999998446021 3.2990787509752002888e-15 0.12248651076282082717 rpy=2.3463681399312212716e-14 3.1845915227826135867e-14 3.141592653589793116 -> xyz=0.016000000000001415867 8.8819348604294950814e-19 0.12248651076281755201 rpy=-9.9708248341699279089e-16 -4.1376224834062942084e-15 3.1415926535897922278
- joint right_hip_yaw_drive: origin xyz=0.037000000000001746769 0.037100000000003664768 -0.039500000000000978773 rpy=-1.5707963267949545116 -4.7905720692590075245e-13 -3.5747430955122047375e-13 -> xyz=0.037000000000001344314 0.037100000000003394152 -0.039499999999999368949 rpy=-1.5707963267949540676 -4.7918343317333855547e-13 -3.3767433293974656194e-13
- joint right_hip_yaw_driven: origin xyz=0.036999999999999991229 0.041100000000000011524 -0.0194999999999999514 rpy=-1.5707963267949003328 -1.5707963267948956698 0 -> xyz=0.036999999999999991229 0.041099999999999997646 -0.019500000000000003442 rpy=-1.5707963267948961139 -1.5707963267948950037 0
- joint right_leg_fixed: origin xyz=0 0 0.0050000000000000044409 rpy=-3.141592653589793116 -0 -9.3397966250929058941e-32 -> xyz=4.336808689942017736e-19 0 0.0050000000000000044409 rpy=-3.141592653589793116 2.7755575615631236952e-17 -4.1633363423443401081e-17
- joint right_sho_pitch: origin xyz=-0.0030000000000019676726 -0.062000000000000089762 0.10423651076282176853 rpy=-1.5707963267948885644 3.4812325502379109658e-14 -3.1415926535897562566 -> xyz=-0.0029999999999986998872 -0.06200000000000097794 0.10423651076281731376 rpy=-1.5707963267948885644 3.4812325502379109658e-14 -3.1415926535897562566
- joint waist_act_1: origin xyz=5.380496587145115132e-16 0.019600000000000075695 -0.012750000000000080713 rpy=1.5707963267949007768 1.5707963267948907848 0 -> xyz=-5.1956727612250319334e-16 0.019600000000000002837 -0.012749999999999961017 rpy=1.570796326794896336 1.5707963267948870101 0
- joint waist_act_2: origin xyz=-2.6785082652000791162e-16 0.019599999999999902223 -0.032749999999999612754 rpy=1.5707963267948958919 1.3463968515392310543 -4.6125152814992733786e-14 -> xyz=2.5285386378767095671e-17 0.019599999999999995898 -0.032749999999999987454 rpy=1.5707963267948974462 1.3463968515392308323 3.4406882288644243018e-15
- joint waist_roll: origin xyz=-0.022707865260691548898 -1.3479418671744790767e-17 -0.014000000000000234479 rpy=-1.5707963267949187625 -1.0371626905663003511e-14 1.5707963267948794606 -> xyz=-0.022707865260692197684 -2.2800061759205613016e-17 -0.01399999999999972447 rpy=-1.570796326794896558 -1.4470091796846119987e-16 1.5707963267948970021
- joint waist_yaw: origin xyz=0 -9.8607613152626475676e-32 0 rpy=1.6626925279001758682e-14 4.9579962395338894532e-14 -3.1415926535897900074 -> xyz=0 6.1629758220391547298e-33 -2.4651903288156618919e-30 rpy=1.3285483818409156951e-16 -3.8508827433200160488e-15 3.1415926535897922278

File: toddlerbot/robot_descriptions/toddlerbot/toddlerbot.urdf (robot description, URDF)
Before this commit: robot toddlerbot, 75 links, 74 joints
Links:
- link ank_motor_rod_short: mass 0.0017000000000000005558 -> 0.0017000000000000001221
- link ank_motor_rod_short_2: mass 0.0017000000000000005558 -> 0.0017000000000000001221
- link ank_roll_link: mass 0.019499999999999989564 -> 0.027200000000000008893; geometry collision box size=0.041999999433755875 0.04500000271946192 0.12000000476837158; visual mesh filename=../assemblies/left_leg_XM430/meshes/left_ank_roll_link_visu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
- link ank_roll_link_2: mass 0.019499999999999989564 -> 0.027200000000000008893; geometry collision box size=0.041999999433755875 0.04500000271946192 0.12000000476837158; visual mesh filename=../assemblies/right_leg_XM430/meshes/right_ank_roll_link_vi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
- link ank_rr_link: mass 0.0014499999999999996832 -> 0.0014499999999999999001
- link ank_rr_link_2: mass 0.0014499999999999996832 -> 0.0014499999999999999001
- link ank_rr_link_3: mass 0.0014499999999999996832 -> 0.0014499999999999999001
- link ank_rr_link_4: mass 0.0014499999999999996832 -> 0.0014499999999999999001
- link hip_yaw_link: mass 0.018000000000000009048 -> 0.017999999999999988232
- link hip_yaw_link_2: mass 0.018000000000000009048 -> 0.017999999999999988232
- link left_hip_pitch_link_xm430: mass 0.1148009013503056841 -> 0.11480090135030569798
- link neck_pitch_link: mass 0.11211553874797881847 -> 0.11211553874797880459
- link neck_yaw_link: mass 0.0085168305947458267796 -> 0.0085168305947458250449
- link right_calf_link: mass 0.086799999986183568046 -> 0.086799999986183554168
- link right_hip_pitch_link_xm430: mass 0.1148009013503056841 -> 0.11480090135030567022
- link spiral_bevel_1m_14t_30deg: mass 0.00067997563436136246491 -> 0.00067997563436136257333
- link spiral_bevel_1m_14t_30deg_2: mass 0.00067997563436136246491 -> 0.00067997563436136257333
- link spur_1m_20t: mass 0.0015534950290892286448 -> 0.0015534950290892282111
- link spur_gear_(13_teeth): mass 0.00081469437497230865874 -> 0.00081469437497230876716
- link spur_gear_19_teeth: mass 0.0010993711450650533144 -> 0.0010993711450650535313
- link spur_gear_19_teeth_2: mass 0.0010993711450650533144 -> 0.0010993711450650535313
- link spur_gear_21_teeth: mass 0.0010063046528317972673 -> 0.0010063046528317974842
- link spur_gear_21_teeth_2: mass 0.0010063046528317972673 -> 0.0010063046528317974842
- link torso: mass 0.58475267652546314423 -> 0.59420757418972613983
- link waist_link: mass 0.16631953490612458313 -> 0.1663195349061246664
- link xm430_plate: mass 0.0026999999999999997093 -> 0.0026999999999999992756
- link xm430_plate_2: mass 0.0026999999999999997093 -> 0.0026999999999999992756
Joints:
- joint left_ank_long_rev_1: origin xyz=-0.018000000000000015987 0.01599999999999926481 -0.020600000000001391504 rpy=-2.876394309884160705e-16 1.6317439732762683578e-16 3.1233695685467286474 -> xyz=-0.018000000000000064559 0.015999999999999292566 -0.020600000000001391504 rpy=-2.876394309884160705e-16 1.6317439732762683578e-16 3.1233695685467286474
- joint left_ank_roll: origin xyz=0.0015000000000000002481 2.7755575615628913511e-17 3.2742905609062233907e-17 rpy=9.9573127520767875392e-16 1.570796326794891673 0 -> xyz=0.0014999999999999995975 0 -1.5395670849294162963e-17 rpy=9.9573127520767875392e-16 1.570796326794891673 0
- joint left_ank_short_rev_1: origin xyz=0.018000000000000002109 0.015999999999999986455 -0.020600000000000010664 rpy=4.2172831995673088897e-16 -4.4678623027074358005e-17 0.026118548507422217203 -> xyz=0.017999999999999953537 0.016000000000000014211 -0.020600000000000010664 rpy=4.2172831995673088897e-16 -4.4678623027074358005e-17 0.026118548507422217203
- joint left_hip_yaw_drive: origin xyz=-0.036999999999998194056 0.037100000000006128076 -0.039500000000001291023 rpy=-1.5707963267949545116 -4.7906511943294847217e-13 -3.592506663906207747e-13 -> xyz=-0.03699999999999847855 0.037100000000005933787 -0.039500000000000194678 rpy=-1.5707963267949540676 -4.7732588435988597417e-13 -3.5949390257278751872e-13
- joint left_hip_yaw_driven: origin xyz=-0.037000000000000012046 0.041099999999999997646 -0.0194999999999999514 rpy=-1.5707963267948990005 -1.570796326794896558 0 -> xyz=-0.037000000000000005107 0.04110000000000003928 -0.019500000000000024258 rpy=-1.5707963267948961139 -1.5707963267948883423 0
- joint left_leg_fixed: origin xyz=0 0 0.004999999999999997502 rpy=3.1415926535897873428 -0 -1.6681280046507162628e-30 -> xyz=0 0 0.0050000000000000044409 rpy=3.141592653589793116 -2.7755575615625073977e-17 -3.33066907387546617e-16
- joint left_sho_pitch: origin xyz=-0.0030000000000065664245 0.062000000000004926171 0.10423651076282140771 rpy=-1.5707963267949054398 -3.6755753074147447628e-14 3.6857314245917344439e-14 -> xyz=-0.0030000000000002949654 0.062000000000001082023 0.10423651076281743866 rpy=-1.5707963267949081043 -4.127643409825574977e-14 3.4723733359249779961e-14
- joint neck_pitch_drive: origin xyz=-1.4224732503009818174e-16 0.015649999999999136824 -0.0087999999999959568897 rpy=-2.4492935983152098954e-16 -2.1427228763620856097e-15 -1.570796326794896558 -> xyz=-8.3266726846886740532e-17 0.015649999999999109068 -0.0087999999999961303621 rpy=-6.1232340018137966949e-17 -1.865637580072612815e-26 -1.570796326794896558
- joint neck_pitch_driven: origin xyz=3.7500001368040436489e-10 -0.0051500000614753682626 0.027499999999999830136 rpy=1.57079632679489678 1.7322096859329345721e-15 -3.1415926535897922278 -> xyz=3.7500136329526867485e-10 -0.0051500000614755217856 0.027499999999999982792 rpy=1.570796326794896558 8.6610484296647231505e-16 3.141592653589793116
- joint neck_yaw_drive: origin xyz=-0.0050000000000041591036 2.1706564040395755645e-15 0.12148651076282282468 rpy=-4.7086950490309927255e-15 -3.2377166610426843676e-14 2.947288666540578667e-14 -> xyz=-0.0049999999999993625932 3.342147474086756384e-17 0.12148651076281766215 rpy=7.9879995913373272052e-15 8.0038275409654909883e-15 -5.4161669716995088817e-15
- joint neck_yaw_driven: origin xyz=0.015999999999998446021 3.2990787509752002888e-15 0.12248651076282082717 rpy=2.3463681399312212716e-14 3.1845915227826135867e-14 3.141592653589793116 -> xyz=0.016000000000001415867 8.8819348604294950814e-19 0.12248651076281755201 rpy=-9.9708248341699279089e-16 -4.1376224834062942084e-15 3.1415926535897922278
- joint right_ank_long_rev_1: origin xyz=0.017999999999999995171 0.016000000000000014211 -0.020600000000000007194 rpy=2.4036779374278231896e-16 5.7386734097817399387e-16 0.018223085043007757056 -> xyz=0.01799999999999999864 0.015999999999999764411 -0.020600000000000132094 rpy=-7.8386807614170502355e-15 7.211088289180617976e-16 0.018223085043007757056
- joint right_ank_roll: origin xyz=0.0015000000000000002481 2.7755575615628913511e-17 1.2143064331837649661e-17 rpy=-8.0803901893659494053e-15 1.5707963267948927832 0 -> xyz=0.001499999999999998947 8.3266726846886740532e-17 1.3660947373317355868e-17 rpy=6.1391486757704172424e-30 1.5707963267948927832 0
- joint right_ank_short_rev_1: origin xyz=-0.018000000000000012518 0.016000000000000014211 -0.020599999999999993316 rpy=1.6033225897674528336e-14 -1.3300018467937457486e-14 3.1154741050824821258 -> xyz=-0.018000000000000009048 0.015999999999999764411 -0.020600000000000118217 rpy=2.411086010918130345e-14 -1.3088994399411267302e-14 3.1154741050824821258
- joint right_hip_yaw_drive: origin xyz=0.037000000000001746769 0.037100000000003664768 -0.039500000000000978773 rpy=-1.5707963267949545116 -4.7905720692590075245e-13 -3.5747430955122047375e-13 -> xyz=0.037000000000001344314 0.037100000000003394152 -0.039499999999999368949 rpy=-1.5707963267949540676 -4.7918343317333855547e-13 -3.3767433293974656194e-13
- joint right_hip_yaw_driven: origin xyz=0.036999999999999991229 0.041100000000000011524 -0.0194999999999999514 rpy=-1.5707963267949003328 -1.5707963267948956698 0 -> xyz=0.036999999999999991229 0.041099999999999997646 -0.019500000000000003442 rpy=-1.5707963267948961139 -1.5707963267948950037 0
- joint right_leg_fixed: origin xyz=0 0 0.0050000000000000044409 rpy=-3.141592653589793116 -0 -9.3397966250929058941e-32 -> xyz=4.336808689942017736e-19 0 0.0050000000000000044409 rpy=-3.141592653589793116 2.7755575615631236952e-17 -4.1633363423443401081e-17
- joint right_sho_pitch: origin xyz=-0.0030000000000019676726 -0.062000000000000089762 0.10423651076282176853 rpy=-1.5707963267948885644 3.4812325502379109658e-14 -3.1415926535897562566 -> xyz=-0.0029999999999986998872 -0.06200000000000097794 0.10423651076281731376 rpy=-1.5707963267948885644 3.4812325502379109658e-14 -3.1415926535897562566
- joint waist_act_1: origin xyz=5.380496587145115132e-16 0.019600000000000075695 -0.012750000000000080713 rpy=1.5707963267949007768 1.5707963267948907848 0 -> xyz=-5.1956727612250319334e-16 0.019600000000000002837 -0.012749999999999961017 rpy=1.570796326794896336 1.5707963267948870101 0
- joint waist_act_2: origin xyz=-2.6785082652000791162e-16 0.019599999999999902223 -0.032749999999999612754 rpy=1.5707963267948958919 1.3463968515392310543 -4.6125152814992733786e-14 -> xyz=2.5285386378767095671e-17 0.019599999999999995898 -0.032749999999999987454 rpy=1.5707963267948974462 1.3463968515392308323 3.4406882288644243018e-15
- joint waist_roll: origin xyz=-0.022707865260691548898 -1.3479418671744790767e-17 -0.014000000000000234479 rpy=-1.5707963267949187625 -1.0371626905663003511e-14 1.5707963267948794606 -> xyz=-0.022707865260692197684 -2.2800061759205613016e-17 -0.01399999999999972447 rpy=-1.570796326794896558 -1.4470091796846119987e-16 1.5707963267948970021
- joint waist_yaw: origin xyz=0 -9.8607613152626475676e-32 0 rpy=1.6626925279001758682e-14 4.9579962395338894532e-14 -3.1415926535897900074 -> xyz=0 6.1629758220391547298e-33 -2.4651903288156618919e-30 rpy=1.3285483818409156951e-16 -3.8508827433200160488e-15 3.1415926535897922278
