Commit message: Update the sysID results

File: toddlerbot/robot_descriptions/assemblies/sysID_XC330/sysID_XC330.urdf (robot description, URDF)
Before this commit: robot sysID_XC330, 2 links, 1 joints
Links:
- link xc330: mass 0.0337537472645257422 -> 0.033753747264525735261
Joints:
- joint joint_0: limit lower=-1.3962634015954635824 upper=1.3962634015954635824 effort=1 velocity=20 -> lower=-1.570796326794896558 upper=1.570796326794896558 effort=1 velocity=20; origin xyz=0.089400000000000034994 0.021949857927858897055 0.0034193959459662111658 rpy=1.5707963267948978903 -1.6653345369377634068e-16 1.5707963267948961139 -> xyz=0.089400000000000048872 0.021949857927858893586 0.0034193959459662037932 rpy=1.57079632679489678 -2.5673907444456749928e-16 1.5707963267948961139

File: toddlerbot/robot_descriptions/sysID_XC330/sysID_XC330.urdf (robot description, URDF)
Before this commit: robot sysID_XC330, 2 links, 1 joints
Links:
- link xc330: mass 0.0337537472645257422 -> 0.033753747264525735261
Joints:
- joint joint_0: limit lower=-1.3962634015954635824 upper=1.3962634015954635824 effort=1 velocity=20 -> lower=-1.570796326794896558 upper=1.570796326794896558 effort=1 velocity=20; origin xyz=0.089400000000000034994 0.021949857927858897055 0.0034193959459662111658 rpy=1.5707963267948978903 -1.6653345369377634068e-16 1.5707963267948961139 -> xyz=0.089400000000000048872 0.021949857927858893586 0.0034193959459662037932 rpy=1.57079632679489678 -2.5673907444456749928e-16 1.5707963267948961139

Commit message: Add sysID for XC330

File: toddlerbot/robot_descriptions/assemblies/sysID_XC330/sysID_XC330.urdf (robot description, URDF)
Before this commit: robot sysID_XC330, 2 links, 1 joints
Links:
- link xc330: mass 0.033753747264525735261 -> 0.037349999993091763384
Joints:
- joint joint_0: origin xyz=0.089400000000000048872 0.021949857927858893586 0.0034193959459662037932 rpy=1.57079632679489678 -2.5673907444456749928e-16 1.5707963267948961139 -> xyz=0.089400000000000034994 0.021949857927858890116 0.0034193959459662072627 rpy=1.57079632679489678 -2.3592239273285399858e-16 1.5707963267948961139

File: toddlerbot/robot_descriptions/sysID_XC330/sysID_XC330.urdf (robot description, URDF)
Before this commit: robot sysID_XC330, 2 links, 1 joints
Links:
- link xc330: mass 0.033753747264525735261 -> 0.037349999993091763384
Joints:
- joint joint_0: origin xyz=0.089400000000000048872 0.021949857927858893586 0.0034193959459662037932 rpy=1.57079632679489678 -2.5673907444456749928e-16 1.5707963267948961139 -> xyz=0.089400000000000034994 0.021949857927858890116 0.0034193959459662072627 rpy=1.57079632679489678 -2.3592239273285399858e-16 1.5707963267948961139

Commit message: Update the load

File: toddlerbot/robot_descriptions/assemblies/sysID_XC330/sysID_XC330.urdf (robot description, URDF)
Before this commit: robot sysID_XC330, 2 links, 1 joints
Links:
- link arm_330: mass 0.094500000000000014544 -> 0.23449999999999995848

File: toddlerbot/robot_descriptions/sysID_XC330/sysID_XC330.urdf (robot description, URDF)
Before this commit: robot sysID_XC330, 2 links, 1 joints
Links:
- link arm_330: mass 0.094500000000000014544 -> 0.23449999999999995848
