Commit message: updated new toddlerbot_arms definition, improved baud in add_configs

File: toddlerbot/robot_descriptions/assemblies/toddlerbot_arms/toddlerbot_arms.urdf (robot description, URDF)
Before this commit: robot toddlerbot_arms, 3 links, 2 joints
Links:
- link left_arm_hand: mass 0.0085999999999999965361 -> 0.0085999999999999948014
- link right_arm_hand: mass 0.0085999999999999965361 -> 0.0085999999999999948014
- link torso: mass 0.58475267652546303321 -> 0.60023307803583569875
Joints:
- joint left_sho_pitch: limit lower=-1.570796326794896558 upper=1.570796326794896558 effort=1 velocity=20 -> lower=-3.141592653589793116 upper=1.570796326794896558 effort=1 velocity=20; origin xyz=-0.0030000000000004519579 0.062000000000001033451 0.10423651076281725825 rpy=-1.5707963267949092145 -3.6755753074147447628e-14 3.6857314245917344439e-14 -> xyz=-0.0030000000000002949654 0.062000000000001082023 0.10423651076281742478 rpy=-1.5707963267949081043 -4.0958527081001641839e-14 3.5234047634505718213e-14
- joint right_sho_pitch: limit lower=-1.570796326794896558 upper=1.570796326794896558 effort=1 velocity=20 -> lower=-1.570796326794896558 upper=3.141592653589793116 effort=1 velocity=20

File: toddlerbot/robot_descriptions/toddlerbot_arms/toddlerbot_arms.urdf (robot description, URDF)
Before this commit: robot toddlerbot_arms, 29 links, 28 joints
Links:
- link torso: mass 0.58475267652546303321 -> 0.60023307803583569875
Joints:
- joint left_sho_pitch: limit lower=-1.570796326794896558 upper=1.570796326794896558 effort=1 velocity=20 -> lower=-3.141592653589793116 upper=1.570796326794896558 effort=1 velocity=20; origin xyz=-0.0030000000000004519579 0.062000000000001033451 0.10423651076281725825 rpy=-1.5707963267949092145 -3.6755753074147447628e-14 3.6857314245917344439e-14 -> xyz=-0.0030000000000002949654 0.062000000000001082023 0.10423651076281742478 rpy=-1.5707963267949081043 -4.0958527081001641839e-14 3.5234047634505718213e-14
- joint right_sho_pitch: limit lower=-1.570796326794896558 upper=1.570796326794896558 effort=1 velocity=20 -> lower=-1.570796326794896558 upper=3.141592653589793116 effort=1 velocity=20
