Commit message: Update wrist roll axes

File: toddlerbot/robot_descriptions/assemblies/left_arm_gripper/left_arm_gripper.urdf (robot description, URDF)
Before this commit: robot left_arm_gripper, 19 links, 18 joints
Links:
- link gripper_connector: mass 0.009999999999999995004 -> 0.0099999999999999984734
- link left_rail_guide: mass 0.032142035224833366558 -> 0.032142035224833380436
- link rail: mass 0.011899999999999995651 -> 0.011900000000000000855
- link rail_2: mass 0.011899999999999995651 -> 0.011900000000000000855
- link sho_yaw_link: mass 0.01450000000000000247 -> 0.014500000000000007674
- link spur_1m_24t_driven: mass 0.0026999999999999988419 -> 0.0027000000000000001429
- link spur_1m_24t_driven_2: mass 0.0026999999999999988419 -> 0.0027000000000000001429
- link spur_1m_24t_driven_3: mass 0.0026999999999999988419 -> 0.0027000000000000001429
- link spur_gear_(14_teeth): mass 0.0012999999999999997235 -> 0.0012999999999999999403
- link wrist_bearing_plate: mass 0.0049000367468305539714 -> 0.0049000367468305548388
Joints:
- joint left_elbow_roll: origin xyz=0 -0.018999999999999999528 -0.058999999999999996891 rpy=1.570796326794896558 -3.6926048046507072339e-14 -1.4375687432866819107e-15 -> xyz=0 -0.018999999999999996059 -0.058999999999999983014 rpy=1.570796326794896558 5.5516872419979014276e-14 -4.4351709097753281525e-15
- joint left_elbow_yaw_drive: origin xyz=-0.024000000716140737489 -0.019000000152457868774 -0.019000000152442970969 rpy=1.5707963267946287722 -5.6813306574568390567e-14 9.3319541222405133527e-14 -> xyz=-0.02400000071614073055 -0.019000000152457841018 -0.019000000152442970969 rpy=1.5707963267946287722 -5.6790261222308772362e-14 9.8859639154170636391e-14
- joint left_elbow_yaw_driven: origin xyz=-3.5806480697120335321e-10 -0.027000000152458680791 -0.018999999999996700084 rpy=1.5707963267946756236 9.4368957093097095842e-15 -7.876460240842920118e-14 -> xyz=-3.5806481391009725712e-10 -0.027000000152458666913 -0.018999999999996696615 rpy=1.5707963267946756236 9.436895709310436914e-15 -7.5767000241948220497e-14
- joint left_elbow_yaw_fixed: origin xyz=3.4694469519536141888e-18 9.4663308626521416649e-30 0.0015999999999999903189 rpy=-3.1415926535897327199 -1.0860743139248627811e-15 -1.5707963267948983344 -> xyz=0 3.1554436208840472216e-30 0.0016000000000000041966 rpy=-3.1415926535897926719 -1.6686716652751508178e-29 -1.570796326794896558
- joint left_gripper_fixed: origin xyz=3.4694469519536141888e-18 0.037000000000000005107 0.03599999999999999728 rpy=1.5707963267948976682 1.570796326794896558 0 -> xyz=0 -0.037000000000000005107 -0.036000000000000004219 rpy=-1.57079632679489678 -1.570796326794896558 0
- joint left_gripper_motor: origin xyz=-0.021950000000000021577 0.022600000000000005501 0.023299999999999959632 rpy=-1.2800691559891638774e-14 -5.2435289262723915078e-30 8.0982650358454429916e-30 -> xyz=-0.021949999999999993822 0.022600000000000002032 0.023300000000000042899 rpy=-3.3306690738376151447e-16 -1.8578007987304439296e-17 1.8327083470280543311e-17
- joint left_gripper_pinion_1: origin xyz=-0.028872600000000105819 -0.014175000000000003569 -0.0053499999999986058707 rpy=3.1415926535897518157 1.5707963267948832353 0 -> xyz=-0.028872599999999620096 -0.014175000000000003569 -0.0053500000000002712053 rpy=3.141592653589793116 1.5707963267948952257 0
- joint left_gripper_pinion_2: origin xyz=0.062872600000001249709 0.014174999999999989692 -0.0053499999999986058707 rpy=-4.163336342340698169e-14 1.5707963267948832353 0 -> xyz=0.062872600000000888887 0.014174999999999993161 -0.0053500000000002434497 rpy=-1.1034025256268857111e-29 1.5707963267948952257 0
- joint left_gripper_rack: origin xyz=0.0079999999999986401433 -0.02250000000000004427 -0.020000000000001599831 rpy=-1.5014551190391114451e-15 -9.4941075965749556743e-16 -6.694912156253297952e-18 -> xyz=0.0079999999999986540211 -0.022500000000000068556 -0.020000000000001683098 rpy=-2.5268845972633189624e-15 -1.3993704652363439234e-15 1.9862277411454370245e-15
- joint left_sho_roll: origin xyz=-0.018999999999999930139 0.00099999999999997031368 0.026999999999999909489 rpy=3.1415926535897913396 1.5707963267947897545 0 -> xyz=-0.01899999999999992667 0.00099999999999997031368 0.026999999999999909489 rpy=3.1415926535897913396 1.5707963267948474861 0
- joint left_sho_yaw_drive: origin xyz=-0.024000000716139804208 -0.019000000152455391589 -0.019000000152449823126 rpy=1.570796326794926312 -3.985731521495478076e-14 1.5953258481899601487e-13 -> xyz=-0.024000000716139110318 -0.019000000152454975255 -0.019000000152449778024 rpy=1.5707963267949334174 -1.1191795890472901541e-13 1.4055336229792838361e-13
- joint left_sho_yaw_driven: origin xyz=-3.5806519207981502007e-10 -0.02700000015245392071 -0.019000000000003951228 rpy=1.570796326794921205 -4.6816437663822621511e-14 9.1955847476605894374e-14 -> xyz=-3.5806544534944251268e-10 -0.027000000152452456603 -0.01900000000000368755 rpy=1.5707963267949525132 -6.2878911843812520251e-14 1.1213824667586519115e-13
- joint left_sho_yaw_fixed: origin xyz=3.4694469519536141888e-18 3.9443045261050590271e-31 0.0016000000000000007272 rpy=3.1415926535897877869 6.3478650967004975275e-30 -3.9477588016902497579e-30 -> xyz=-3.4694469519536141888e-18 1.5777218104420236108e-30 0.0016000000000000041966 rpy=3.1415926535897771288 -2.9902758688536131143e-29 -1.1367870242563646532e-30
- joint left_wrist_pitch_drive: origin xyz=-1.5244435917471109994e-10 0.024000000358067929973 -0.0080000000000045659587 rpy=-5.3096416152614807834e-14 -6.1274079212673509226e-14 -1.5707963267947160357 -> xyz=-1.5244435917471112579e-10 0.024000000358067929973 -0.0080000000000045659587 rpy=-6.8143291540626782613e-14 -7.3946574628751046645e-14 -1.5707963267947160357
- joint left_wrist_pitch_driven: origin xyz=-2.7755575615628913511e-17 -3.1554436208840472216e-30 -0.0015999999999999987756 rpy=3.1872271311673666698e-15 -9.0981076131151630778e-15 -1.570796326794896558 -> xyz=-2.7755575615628913511e-17 -3.1554436208840472216e-30 -0.0015999999999999972577 rpy=1.8707257964927463223e-14 -2.230976160592272071e-14 -1.570796326794896558
- joint left_wrist_pitch_fixed: origin xyz=0.015500000000004770379 -6.3282712403633922804e-15 -0.045000000000001996736 rpy=-2.0039525594392854835e-14 -1.2819656091163158021e-13 -1.5707963267947810948 -> xyz=0.015500000000004772113 -6.3837823915946501074e-15 -0.045000000000001996736 rpy=-3.5027536426602388959e-14 -1.2834178164666087642e-13 -1.5707963267947810948
- joint left_wrist_roll: origin xyz=0.019000000000008614165 -3.5807912190932711383e-10 -0.02700000015245084678 rpy=3.1415926535897877869 1.5707963267947964159 0 -> xyz=0.019000000000008621104 -3.5807914966490272946e-10 -0.02700000015245084678 rpy=-5.342948306010493038e-15 1.5707963267948528152 0
- joint left_wrist_roll_fixed: origin xyz=3.1554436208840472216e-30 -0.025299999999999996103 -0.052000000000000032307 rpy=1.5707963267948923392 -1.5707963267948330532 0 -> xyz=3.1554436208840472216e-30 -0.025300000000000003042 -0.052000000000000032307 rpy=1.570796326794896558 -1.570796326794896558 0

File: toddlerbot/robot_descriptions/assemblies/left_arm_hand/left_arm_hand.urdf (robot description, URDF)
Before this commit: robot left_arm_hand, 14 links, 13 joints
Links:
- link elb_yaw_link: mass 0.017500000000000012074 -> 0.017500000000000001665
- link hand: mass 0.017000000000001444511 -> 0.017000000000001441042
- link sho_pitch_link: mass 0.0085999999999999948014 -> 0.0086000000000000017403
- link sho_yaw_link: mass 0.014500000000000011144 -> 0.014500000000000007674
- link wrist_bearing_plate: mass 0.0049000367468305539714 -> 0.0049000367468305548388
Joints:
- joint left_elbow_roll: origin xyz=1.1865508575681360526e-15 -0.018999999999999999528 -0.059000000000000024647 rpy=1.570796326794896558 -3.0035063655217005852e-13 -8.0812793815154920791e-14 -> xyz=3.4694469519536141888e-18 -0.018999999999999996059 -0.058999999999999983014 rpy=1.570796326794896336 -2.4424906541778151013e-14 3.0649833342774549336e-16
- joint left_elbow_yaw_drive: origin xyz=-0.024000000716141021984 -0.019000000152448556778 -0.019000000152448459634 rpy=1.5707963267949303088 5.3222446619528222415e-15 1.3540958880671982531e-14 -> xyz=-0.024000000716137528251 -0.0190000001524475437 -0.019000000152459547986 rpy=1.570796326795050879 -2.46739603138074785e-13 -6.062193916416980129e-14
- joint left_elbow_yaw_driven: origin xyz=-3.5806928949666527728e-10 -0.027000000152451103519 -0.019000000000003354483 rpy=1.5707963267948781283 1.57079632679478709 0 -> xyz=-3.5806395001780622067e-10 -0.027000000152452921509 -0.019000000000006608825 rpy=1.5707963267949589525 1.5707963267947417929 0
- joint left_elbow_yaw_fixed: origin xyz=2.6687419884145636134e-18 3.4694469519536141888e-18 0.0015999999999999903189 rpy=-3.141592653589793116 -7.7295713056774243222e-29 -3.8634032214012514384e-29 -> xyz=1.5777218104420236108e-30 0 0.0015999999999999903189 rpy=-3.141592653589793116 -1.5029469787693842406e-27 -1.0914409670812147614e-28
- joint left_sho_roll: origin xyz=-0.018999999999999999528 0.0010000000000000084776 0.027000000000001016243 rpy=-3.141592653589793116 1.5707963267945652674 0 -> xyz=-0.018999999999999999528 0.0010000000000000034903 0.027000000000000006634 rpy=-3.141592653589793116 1.570796326794896336 0
- joint left_sho_yaw_drive: origin xyz=-0.024000000716141008106 -0.019000000152450610691 -0.019000000152443286688 rpy=1.5707963267948328312 -1.2293716347296049066e-15 1.010090991001174754e-13 -> xyz=-0.024000000716141011575 -0.01900000015245061416 -0.019000000152443286688 rpy=1.5707963267948328312 -1.2486577482345307449e-15 8.257939689134084871e-14
- joint left_sho_yaw_driven: origin xyz=-3.5806878642685724401e-10 -0.027000000152450916169 -0.018999999999999881567 rpy=1.5707963267948492625 7.9618117061835143528e-14 1.0891287871571481832e-13 -> xyz=-3.5807090625894488767e-10 -0.027000000152451124336 -0.018999999999999364619 rpy=1.5707963267948492625 7.961811706183572413e-14 1.2023715356687380766e-13
- joint left_sho_yaw_fixed: origin xyz=-3.4694469519536141888e-18 3.9443045261050590271e-31 0.0016000000000000007272 rpy=3.1415926535897873428 -0 0 -> xyz=3.4694469519536141888e-18 3.9443045261050590271e-31 0.0016000000000000007272 rpy=3.1415926535897757965 -0 0
- joint left_wrist_pitch_drive: origin xyz=-1.5244060454932558359e-10 0.024000000358057327343 -0.0080000000000068800798 rpy=3.9435158482369467881e-14 -2.1741514499400786903e-13 -1.5707963267949176522 -> xyz=-1.5244060454932558359e-10 0.024000000358057327343 -0.0080000000000068835493 rpy=4.57965832526558921e-14 -2.10309717636365493e-13 -1.5707963267949176522
- joint left_wrist_pitch_driven: origin xyz=-2.7755575615628913511e-17 -2.6687419884003641171e-18 -0.0015999999999999992093 rpy=-1.2490008944217178404e-15 -8.8817841970011517436e-16 -1.570796326794896558 -> xyz=0 -1.5777218104420236108e-30 -0.0015999999999999953062 rpy=-2.8253475236412191385e-15 -3.552713678800508818e-15 -1.570796326794896558
- joint left_wrist_pitch_fixed: origin xyz=0.015500000000007823492 -1.8068879725774422695e-14 -0.044999999999998908928 rpy=5.4234394758357771884e-14 -2.8213542612434265448e-13 -1.570796326794906328 -> xyz=0.015500000000007821757 -1.8096635301390051609e-14 -0.044999999999998901989 rpy=8.1212814267639654023e-14 -2.8213542612434270497e-13 -1.570796326794906328
- joint left_wrist_roll: origin xyz=0.019000000000007042505 -3.5808098153289336096e-10 -0.027000000152448057344 rpy=-3.1415926535897193972 1.5707963267946853936 0 -> xyz=0.019000000000007045975 -3.5808098153289336096e-10 -0.027000000152448057344 rpy=-8.1915604995110887341e-29 1.5707963267945390662 0
- joint left_wrist_roll_fixed: origin xyz=-2.6687419884121970307e-18 -0.025299999999999999573 -0.052000000000000032307 rpy=1.5707963267948976682 -1.5707963267948956698 0 -> xyz=-7.8886090522101180541e-30 -0.025299999999999999573 -0.052000000000000032307 rpy=1.5707963267948985564 -1.5707963267948945596 0

File: toddlerbot/robot_descriptions/assemblies/right_arm_hand/right_arm_hand.urdf (robot description, URDF)
Before this commit: robot right_arm_hand, 14 links, 13 joints
Links:
- link elb_yaw_link: mass 0.017500000000000012074 -> 0.017500000000000001665
- link hand: mass 0.017000000000001444511 -> 0.017000000000001441042
- link sho_pitch_link: mass 0.0085999999999999948014 -> 0.0086000000000000017403
- link sho_yaw_link: mass 0.014500000000000011144 -> 0.014500000000000007674
- link wrist_bearing_plate: mass 0.0049000367468305539714 -> 0.0049000367468305548388

File: toddlerbot/robot_descriptions/assemblies/toddlerbot_arms/toddlerbot_arms.urdf (robot description, URDF)
Before this commit: robot toddlerbot_arms, 3 links, 2 joints
Links:
- link left_arm_hand: mass 0.0085999999999999948014 -> 0.0085999999999999965361
- link right_arm_hand: mass 0.0085999999999999948014 -> 0.0085999999999999965361
- link torso: mass 0.60023307803583569875 -> 0.60012685450989189384

File: toddlerbot/robot_descriptions/toddlerbot/toddlerbot.urdf (robot description, URDF)
Before this commit: robot toddlerbot, 85 links, 84 joints
Links:
- link gripper_connector: mass 0.009999999999999995004 -> 0.0099999999999999984734
- link left_rail_guide: mass 0.032142035224833366558 -> 0.032142035224833380436
- link rail: mass 0.011899999999999995651 -> 0.011900000000000000855
- link rail_2: mass 0.011899999999999995651 -> 0.011900000000000000855
- link sho_yaw_link: mass 0.01450000000000000247 -> 0.014500000000000007674
- link spur_1m_24t_driven: mass 0.0026999999999999988419 -> 0.0027000000000000001429
- link spur_1m_24t_driven_2: mass 0.0026999999999999988419 -> 0.0027000000000000001429
- link spur_1m_24t_driven_3: mass 0.0026999999999999988419 -> 0.0027000000000000001429
- link spur_gear_(14_teeth): mass 0.0012999999999999997235 -> 0.0012999999999999999403
- link wrist_bearing_plate: mass 0.0049000367468305539714 -> 0.0049000367468305548388
Joints:
- joint left_elbow_roll: origin xyz=0 -0.018999999999999999528 -0.058999999999999996891 rpy=1.570796326794896558 -3.6926048046507072339e-14 -1.4375687432866819107e-15 -> xyz=0 -0.018999999999999996059 -0.058999999999999983014 rpy=1.570796326794896558 5.5516872419979014276e-14 -4.4351709097753281525e-15
- joint left_elbow_yaw_drive: origin xyz=-0.024000000716140737489 -0.019000000152457868774 -0.019000000152442970969 rpy=1.5707963267946287722 -5.6813306574568390567e-14 9.3319541222405133527e-14 -> xyz=-0.02400000071614073055 -0.019000000152457841018 -0.019000000152442970969 rpy=1.5707963267946287722 -5.6790261222308772362e-14 9.8859639154170636391e-14
- joint left_elbow_yaw_driven: origin xyz=-3.5806480697120335321e-10 -0.027000000152458680791 -0.018999999999996700084 rpy=1.5707963267946756236 9.4368957093097095842e-15 -7.876460240842920118e-14 -> xyz=-3.5806481391009725712e-10 -0.027000000152458666913 -0.018999999999996696615 rpy=1.5707963267946756236 9.436895709310436914e-15 -7.5767000241948220497e-14
- joint left_elbow_yaw_fixed: origin xyz=3.4694469519536141888e-18 9.4663308626521416649e-30 0.0015999999999999903189 rpy=-3.1415926535897327199 -1.0860743139248627811e-15 -1.5707963267948983344 -> xyz=0 3.1554436208840472216e-30 0.0016000000000000041966 rpy=-3.1415926535897926719 -1.6686716652751508178e-29 -1.570796326794896558
- joint left_gripper_fixed: origin xyz=3.4694469519536141888e-18 0.037000000000000005107 0.03599999999999999728 rpy=1.5707963267948976682 1.570796326794896558 0 -> xyz=0 -0.037000000000000005107 -0.036000000000000004219 rpy=-1.57079632679489678 -1.570796326794896558 0
- joint left_gripper_motor: origin xyz=-0.021950000000000021577 0.022600000000000005501 0.023299999999999959632 rpy=-1.2800691559891638774e-14 -5.2435289262723915078e-30 8.0982650358454429916e-30 -> xyz=-0.021949999999999993822 0.022600000000000002032 0.023300000000000042899 rpy=-3.3306690738376151447e-16 -1.8578007987304439296e-17 1.8327083470280543311e-17
- joint left_gripper_pinion_1: origin xyz=-0.028872600000000105819 -0.014175000000000003569 -0.0053499999999986058707 rpy=3.1415926535897518157 1.5707963267948832353 0 -> xyz=-0.028872599999999620096 -0.014175000000000003569 -0.0053500000000002712053 rpy=3.141592653589793116 1.5707963267948952257 0
- joint left_gripper_pinion_2: origin xyz=0.062872600000001249709 0.014174999999999989692 -0.0053499999999986058707 rpy=-4.163336342340698169e-14 1.5707963267948832353 0 -> xyz=0.062872600000000888887 0.014174999999999993161 -0.0053500000000002434497 rpy=-1.1034025256268857111e-29 1.5707963267948952257 0
- joint left_gripper_rack: origin xyz=0.0079999999999986401433 -0.02250000000000004427 -0.020000000000001599831 rpy=-1.5014551190391114451e-15 -9.4941075965749556743e-16 -6.694912156253297952e-18 -> xyz=0.0079999999999986540211 -0.022500000000000068556 -0.020000000000001683098 rpy=-2.5268845972633189624e-15 -1.3993704652363439234e-15 1.9862277411454370245e-15
- joint left_sho_roll: origin xyz=-0.018999999999999930139 0.00099999999999997031368 0.026999999999999909489 rpy=3.1415926535897913396 1.5707963267947897545 0 -> xyz=-0.01899999999999992667 0.00099999999999997031368 0.026999999999999909489 rpy=3.1415926535897913396 1.5707963267948474861 0
- joint left_sho_yaw_drive: origin xyz=-0.024000000716139804208 -0.019000000152455391589 -0.019000000152449823126 rpy=1.570796326794926312 -3.985731521495478076e-14 1.5953258481899601487e-13 -> xyz=-0.024000000716139110318 -0.019000000152454975255 -0.019000000152449778024 rpy=1.5707963267949334174 -1.1191795890472901541e-13 1.4055336229792838361e-13
- joint left_sho_yaw_driven: origin xyz=-3.5806519207981502007e-10 -0.02700000015245392071 -0.019000000000003951228 rpy=1.570796326794921205 -4.6816437663822621511e-14 9.1955847476605894374e-14 -> xyz=-3.5806544534944251268e-10 -0.027000000152452456603 -0.01900000000000368755 rpy=1.5707963267949525132 -6.2878911843812520251e-14 1.1213824667586519115e-13
- joint left_sho_yaw_fixed: origin xyz=3.4694469519536141888e-18 3.9443045261050590271e-31 0.0016000000000000007272 rpy=3.1415926535897877869 6.3478650967004975275e-30 -3.9477588016902497579e-30 -> xyz=-3.4694469519536141888e-18 1.5777218104420236108e-30 0.0016000000000000041966 rpy=3.1415926535897771288 -2.9902758688536131143e-29 -1.1367870242563646532e-30
- joint left_wrist_pitch_drive: origin xyz=-1.5244435917471109994e-10 0.024000000358067929973 -0.0080000000000045659587 rpy=-5.3096416152614807834e-14 -6.1274079212673509226e-14 -1.5707963267947160357 -> xyz=-1.5244435917471112579e-10 0.024000000358067929973 -0.0080000000000045659587 rpy=-6.8143291540626782613e-14 -7.3946574628751046645e-14 -1.5707963267947160357
- joint left_wrist_pitch_driven: origin xyz=-2.7755575615628913511e-17 -3.1554436208840472216e-30 -0.0015999999999999987756 rpy=3.1872271311673666698e-15 -9.0981076131151630778e-15 -1.570796326794896558 -> xyz=-2.7755575615628913511e-17 -3.1554436208840472216e-30 -0.0015999999999999972577 rpy=1.8707257964927463223e-14 -2.230976160592272071e-14 -1.570796326794896558
- joint left_wrist_pitch_fixed: origin xyz=0.015500000000004770379 -6.3282712403633922804e-15 -0.045000000000001996736 rpy=-2.0039525594392854835e-14 -1.2819656091163158021e-13 -1.5707963267947810948 -> xyz=0.015500000000004772113 -6.3837823915946501074e-15 -0.045000000000001996736 rpy=-3.5027536426602388959e-14 -1.2834178164666087642e-13 -1.5707963267947810948
- joint left_wrist_roll: origin xyz=0.019000000000008614165 -3.5807912190932711383e-10 -0.02700000015245084678 rpy=3.1415926535897877869 1.5707963267947964159 0 -> xyz=0.019000000000008621104 -3.5807914966490272946e-10 -0.02700000015245084678 rpy=-5.342948306010493038e-15 1.5707963267948528152 0
- joint left_wrist_roll_fixed: origin xyz=3.1554436208840472216e-30 -0.025299999999999996103 -0.052000000000000032307 rpy=1.5707963267948923392 -1.5707963267948330532 0 -> xyz=3.1554436208840472216e-30 -0.025300000000000003042 -0.052000000000000032307 rpy=1.570796326794896558 -1.570796326794896558 0
