Commit message: Update wrist roll axes

File: toddlerbot/robot_descriptions/toddlerbot_arms/toddlerbot_arms.urdf (robot description, URDF)
Before this commit: robot toddlerbot_arms, 29 links, 28 joints
Links:
- link elb_yaw_link: mass 0.017500000000000012074 -> 0.017500000000000001665
- link elb_yaw_link_2: mass 0.017500000000000012074 -> 0.017500000000000001665
- link hand: mass 0.017000000000001444511 -> 0.017000000000001441042
- link hand_2: mass 0.017000000000001444511 -> 0.017000000000001441042
- link sho_pitch_link: mass 0.0085999999999999948014 -> 0.0086000000000000017403
- link sho_pitch_link_2: mass 0.0085999999999999948014 -> 0.0086000000000000017403
- link sho_yaw_link: mass 0.014500000000000011144 -> 0.014500000000000007674
- link sho_yaw_link_2: mass 0.014500000000000011144 -> 0.014500000000000007674
- link torso: mass 0.60023307803583569875 -> 0.60012685450989189384
- link wrist_bearing_plate: mass 0.0049000367468305539714 -> 0.0049000367468305548388
- link wrist_bearing_plate_2: mass 0.0049000367468305539714 -> 0.0049000367468305548388
Joints:
- joint left_elbow_roll: origin xyz=1.1865508575681360526e-15 -0.018999999999999999528 -0.059000000000000024647 rpy=1.570796326794896558 -3.0035063655217005852e-13 -8.0812793815154920791e-14 -> xyz=3.4694469519536141888e-18 -0.018999999999999996059 -0.058999999999999983014 rpy=1.570796326794896336 -2.4424906541778151013e-14 3.0649833342774549336e-16
- joint left_elbow_yaw_drive: origin xyz=-0.024000000716141021984 -0.019000000152448556778 -0.019000000152448459634 rpy=1.5707963267949303088 5.3222446619528222415e-15 1.3540958880671982531e-14 -> xyz=-0.024000000716137528251 -0.0190000001524475437 -0.019000000152459547986 rpy=1.570796326795050879 -2.46739603138074785e-13 -6.062193916416980129e-14
- joint left_elbow_yaw_driven: origin xyz=-3.5806928949666527728e-10 -0.027000000152451103519 -0.019000000000003354483 rpy=1.5707963267948781283 1.57079632679478709 0 -> xyz=-3.5806395001780622067e-10 -0.027000000152452921509 -0.019000000000006608825 rpy=1.5707963267949589525 1.5707963267947417929 0
- joint left_elbow_yaw_fixed: origin xyz=2.6687419884145636134e-18 3.4694469519536141888e-18 0.0015999999999999903189 rpy=-3.141592653589793116 -7.7295713056774243222e-29 -3.8634032214012514384e-29 -> xyz=1.5777218104420236108e-30 0 0.0015999999999999903189 rpy=-3.141592653589793116 -1.5029469787693842406e-27 -1.0914409670812147614e-28
- joint left_sho_roll: origin xyz=-0.018999999999999999528 0.0010000000000000084776 0.027000000000001016243 rpy=-3.141592653589793116 1.5707963267945652674 0 -> xyz=-0.018999999999999999528 0.0010000000000000034903 0.027000000000000006634 rpy=-3.141592653589793116 1.570796326794896336 0
- joint left_sho_yaw_drive: origin xyz=-0.024000000716141008106 -0.019000000152450610691 -0.019000000152443286688 rpy=1.5707963267948328312 -1.2293716347296049066e-15 1.010090991001174754e-13 -> xyz=-0.024000000716141011575 -0.01900000015245061416 -0.019000000152443286688 rpy=1.5707963267948328312 -1.2486577482345307449e-15 8.257939689134084871e-14
- joint left_sho_yaw_driven: origin xyz=-3.5806878642685724401e-10 -0.027000000152450916169 -0.018999999999999881567 rpy=1.5707963267948492625 7.9618117061835143528e-14 1.0891287871571481832e-13 -> xyz=-3.5807090625894488767e-10 -0.027000000152451124336 -0.018999999999999364619 rpy=1.5707963267948492625 7.961811706183572413e-14 1.2023715356687380766e-13
- joint left_sho_yaw_fixed: origin xyz=-3.4694469519536141888e-18 3.9443045261050590271e-31 0.0016000000000000007272 rpy=3.1415926535897873428 -0 0 -> xyz=3.4694469519536141888e-18 3.9443045261050590271e-31 0.0016000000000000007272 rpy=3.1415926535897757965 -0 0
- joint left_wrist_pitch_drive: origin xyz=-1.5244060454932558359e-10 0.024000000358057327343 -0.0080000000000068800798 rpy=3.9435158482369467881e-14 -2.1741514499400786903e-13 -1.5707963267949176522 -> xyz=-1.5244060454932558359e-10 0.024000000358057327343 -0.0080000000000068835493 rpy=4.57965832526558921e-14 -2.10309717636365493e-13 -1.5707963267949176522
- joint left_wrist_pitch_driven: origin xyz=-2.7755575615628913511e-17 -2.6687419884003641171e-18 -0.0015999999999999992093 rpy=-1.2490008944217178404e-15 -8.8817841970011517436e-16 -1.570796326794896558 -> xyz=0 -1.5777218104420236108e-30 -0.0015999999999999953062 rpy=-2.8253475236412191385e-15 -3.552713678800508818e-15 -1.570796326794896558
- joint left_wrist_pitch_fixed: origin xyz=0.015500000000007823492 -1.8068879725774422695e-14 -0.044999999999998908928 rpy=5.4234394758357771884e-14 -2.8213542612434265448e-13 -1.570796326794906328 -> xyz=0.015500000000007821757 -1.8096635301390051609e-14 -0.044999999999998901989 rpy=8.1212814267639654023e-14 -2.8213542612434270497e-13 -1.570796326794906328
- joint left_wrist_roll: origin xyz=0.019000000000007042505 -3.5808098153289336096e-10 -0.027000000152448057344 rpy=-3.1415926535897193972 1.5707963267946853936 0 -> xyz=0.019000000000007045975 -3.5808098153289336096e-10 -0.027000000152448057344 rpy=-8.1915604995110887341e-29 1.5707963267945390662 0
- joint left_wrist_roll_fixed: origin xyz=-2.6687419884121970307e-18 -0.025299999999999999573 -0.052000000000000032307 rpy=1.5707963267948976682 -1.5707963267948956698 0 -> xyz=-7.8886090522101180541e-30 -0.025299999999999999573 -0.052000000000000032307 rpy=1.5707963267948985564 -1.5707963267948945596 0

Commit message: Update the gripper pinions

File: toddlerbot/robot_descriptions/assemblies/left_arm_gripper/left_arm_gripper.urdf (robot description, URDF)
Before this commit: robot left_arm_gripper, 19 links, 18 joints
Links:
- link gripper_connector: mass 0.0099999999999999984734 -> 0.0099999999999999915345
- link left_rail_guide: mass 0.032142035224833380436 -> 0.032142035224833366558
- link sho_pitch_link: mass 0.0086000000000000017403 -> 0.0086000000000000000056
- link sho_yaw_link: mass 0.014500000000000007674 -> 0.014500000000000016348
- link spur_1m_24t_driven: mass 0.0027000000000000001429 -> 0.0026999999999999997093
- link spur_1m_24t_driven_2: mass 0.0027000000000000001429 -> 0.0026999999999999997093
- link spur_1m_24t_driven_3: mass 0.0027000000000000001429 -> 0.0026999999999999997093
Joints:
- removed joint left_gripper_pinion_1
- removed joint left_gripper_pinion_2
- added joint left_gripper_pinion: type prismatic, parent left_rail_guide, child rail, origin xyz=-0.028872599999999620096 -0.014175000000000003569 -0.0053500000000002712053 rpy=3.141592653589793116 1.5707963267948952257 0, axis 0 0 1, limit lower=-0.036872599999999998432 upper=0 effort=1 velocity=20
- added joint left_gripper_pinion_mirror: type prismatic, parent left_rail_guide, child rail_2, origin xyz=0.062872600000000888887 0.014174999999999993161 -0.0053500000000002434497 rpy=-1.1034025256268857111e-29 1.5707963267948952257 0, axis 0 0 1, limit lower=-0.036872599999999998432 upper=0 effort=1 velocity=20

File: toddlerbot/robot_descriptions/assemblies/right_arm_gripper/right_arm_gripper.urdf (robot description, URDF)
Before this commit: robot right_arm_gripper, 19 links, 18 joints
Links:
- link gripper_connector: mass 0.009999999999999995004 -> 0.0099999999999999915345
- link rail: mass 0.011899999999999995651 -> 0.011900000000000000855
- link rail_2: mass 0.011899999999999995651 -> 0.011900000000000000855
- link right_rail_guide: mass 0.030111386261699936429 -> 0.030111386261699946837
- link sho_pitch_link: mass 0.0086000000000000017403 -> 0.0086000000000000000056
- link sho_yaw_link: mass 0.01450000000000000247 -> 0.014500000000000016348
- link spur_1m_24t_driven: mass 0.0026999999999999988419 -> 0.0026999999999999997093
- link spur_1m_24t_driven_2: mass 0.0026999999999999988419 -> 0.0026999999999999997093
- link spur_1m_24t_driven_3: mass 0.0026999999999999988419 -> 0.0026999999999999997093
- link spur_gear_(14_teeth): mass 0.0012999999999999997235 -> 0.0012999999999999999403
- link wrist_bearing_plate: mass 0.0049000367468305539714 -> 0.0049000367468305548388
Joints:
- removed joint right_gripper_pinion_1
- removed joint right_gripper_pinion_2
- added joint right_gripper_pinion: type prismatic, parent right_rail_guide, child rail, origin xyz=-0.028872600000001191756 -0.014174999999999993161 -0.005350000000001076117 rpy=-3.141592653589793116 1.5707963267948954478 0, axis 0 0 1, limit lower=-0.036872599999999998432 upper=0 effort=1 velocity=20
- added joint right_gripper_pinion_mirror: type prismatic, parent right_rail_guide, child rail_2, origin xyz=0.062872599999998834974 0.01417499999999999663 -0.0053500000000010206058 rpy=9.1593399531549520226e-16 1.5707963267948945596 0, axis 0 0 1, limit lower=-0.036872599999999998432 upper=0 effort=1 velocity=20
