Commit message: Update the name of the robot

File: toddlerbot/robot_descriptions/toddlerbot/toddlerbot.urdf (robot description, URDF)
Before this commit: robot base_legs, 37 links, 36 joints
Links:
- added link elb_link, mass 0.012147845014428806237; collision mesh filename=collisions/left_elb_link_collision.stl; visual mesh filename=../assemblies/left_OP3_arm/meshes/left_elb_link_visual.stl
- added link elb_link_2, mass 0.012147845014428806237; collision mesh filename=collisions/right_elb_link_collision.stl; visual mesh filename=../assemblies/right_OP3_arm/meshes/right_elb_link_visual.stl
- added link head_link, mass 0.075015538754886992856; collision mesh filename=collisions/head_link_collision.stl; visual mesh filename=../assemblies/4R_body/meshes/head_link_visual.stl
- added link neck_link, mass 0.018378317023500286703; collision mesh filename=collisions/neck_link_collision.stl; visual mesh filename=../assemblies/4R_body/meshes/neck_link_visual.stl
- added link sho_pitch_link, mass 0.0053168741776095261239; visual mesh filename=../assemblies/left_OP3_arm/meshes/left_sho_pitch_link_visua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
- added link sho_pitch_link_2, mass 0.0053168741776095261239; visual mesh filename=../assemblies/right_OP3_arm/meshes/right_sho_pitch_link_vis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
- added link sho_roll_link, mass 0.14104718485994710564; collision mesh filename=collisions/left_sho_roll_link_collision.stl; visual mesh filename=../assemblies/left_OP3_arm/meshes/left_sho_roll_link_visual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
- added link sho_roll_link_2, mass 0.14104718485994710564; collision mesh filename=collisions/right_sho_roll_link_collision.stl; visual mesh filename=../assemblies/right_OP3_arm/meshes/right_sho_roll_link_visu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
- link body_link: mass 0.1326329205818372603 -> 1.3010345634555100514; geometry collision mesh filename=collisions/body_link_collision.stl; visual mesh filename=../assemblies/4R_body/meshes/body_link_visual.stl
Joints:
- added joint head: type fixed, parent neck_link, child head_link, origin xyz=0 -6.505213034913026604e-19 -0.039999999999999980016 rpy=-3.6199375412562401434e-16 -2.4218742848029192401e-16 -5.5511151231257722251e-17, axis 0 0 1, limit effort=1 velocity=20
- added joint left_elb: type revolute, parent sho_roll_link, child elb_link, origin xyz=-0.089499999999999663158 -3.2265856653168611956e-16 5.9049987122250513494e-15 rpy=3.1415926535897367167 2.2793048768987009608e-14 -1.5707963267948858999, axis 0 0 1, limit lower=-1.570796326794896558 upper=1.570796326794896558 effort=1 velocity=20
- added joint left_sho_pitch: type revolute, parent body_link, child sho_pitch_link, origin xyz=-0.00090000000000018190449 0.058000000000000113964 0.42079999999999984084 rpy=-1.570796326794871911 3.5360603334311235812e-14 -3.1415926535897371608, axis 0 0 1, limit lower=-1.570796326794896558 upper=1.570796326794896558 effort=1 velocity=20
- added joint left_sho_roll: type revolute, parent sho_pitch_link, child sho_roll_link, origin xyz=-0.018999999999999999528 0.0089999999999999646255 -0.027499999999999986261 rpy=-6.3254956828146051492e-14 -1.5707963267948947816 0, axis 0 0 1, limit lower=-1.570796326794896558 upper=1.570796326794896558 effort=1 velocity=20
- added joint neck: type fixed, parent body_link, child neck_link, origin xyz=-0.00089999999999998414602 -4.4507968385753129991e-18 0.44079999999999996962 rpy=-3.141592653589793116 8.5053965662326763145e-17 1.57079632679489678, axis 0 0 1, limit effort=1 velocity=20
- added joint right_elb: type revolute, parent sho_roll_link_2, child elb_link_2, origin xyz=-0.08949999999999827538 -7.2650219173908681114e-15 1.0956513474269513608e-14 rpy=-3.1415926535897145122 9.187667647645342109e-14 1.5707963267949796027, axis 0 0 1, limit lower=-1.570796326794896558 upper=1.570796326794896558 effort=1 velocity=20
- added joint right_sho_pitch: type revolute, parent body_link, child sho_pitch_link_2, origin xyz=-0.00090000000000000062589 -0.057999999999999982125 0.42079999999999995186 rpy=-1.5707963267948972241 1.3877787807856806753e-15 6.3545304591998415249e-17, axis 0 0 1, limit lower=-1.570796326794896558 upper=1.570796326794896558 effort=1 velocity=20
- added joint right_sho_roll: type revolute, parent sho_pitch_link_2, child sho_roll_link_2, origin xyz=0.018999999999999954425 0.0089999999999999576866 -0.027499999999999899525 rpy=-3.1415926535896976368 -1.5707963267948958919 0, axis 0 0 1, limit lower=-1.570796326794896558 upper=1.570796326794896558 effort=1 velocity=20
- joint left_hip_yaw: origin xyz=-0.0063999999999966045855 0.033999999999999447331 0.28550000000000008704 rpy=1.2173498077257119742e-16 -2.7439672175516685782e-14 -9.8815480994853422476e-14 -> xyz=-0.006400000000000070563 0.033999999999999967748 0.28550000000000003153 rpy=-1.0062408617649953783e-14 -1.7373496713084857328e-15 -1.0702550091647256269e-13
- joint right_hip_yaw: origin xyz=-0.006399999999996792803 -0.034000000000000661637 0.28549999999999997602 rpy=1.2173498094410956825e-16 -2.7428229798067236768e-14 -5.0714987764877150767e-13 -> xyz=-0.0064000000000002613826 -0.033999999999999974687 0.28549999999999997602 rpy=-2.4175737836120826254e-16 2.1811947592303793928e-16 -1.3443908046660001512e-14

File: toddlerbot/robot_descriptions/toddlerbot_legs/toddlerbot_legs.urdf (robot description, URDF)
Before this commit: robot base, 45 links, 44 joints
Links:
- removed link elb_link
- removed link elb_link_2
- removed link head_link
- removed link neck_link
- removed link sho_pitch_link
- removed link sho_pitch_link_2
- removed link sho_roll_link
- removed link sho_roll_link_2
- link body_link: mass 1.3010345634555100514 -> 0.1326329205818372603; geometry collision mesh filename=collisions/body_link_collision.stl; visual mesh filename=../assemblies/no_body/meshes/body_link_visual.stl
Joints:
- removed joint head
- removed joint left_elb
- removed joint left_sho_pitch
- removed joint left_sho_roll
- removed joint neck
- removed joint right_elb
- removed joint right_sho_pitch
- removed joint right_sho_roll
- joint left_hip_yaw: origin xyz=-0.006400000000000070563 0.033999999999999967748 0.28550000000000003153 rpy=-1.0062408617649953783e-14 -1.7373496713084857328e-15 -1.0702550091647256269e-13 -> xyz=-0.0063999999999966045855 0.033999999999999447331 0.28550000000000008704 rpy=1.2173498077257119742e-16 -2.7439672175516685782e-14 -9.8815480994853422476e-14
- joint right_hip_yaw: origin xyz=-0.0064000000000002613826 -0.033999999999999974687 0.28549999999999997602 rpy=-2.4175737836120826254e-16 2.1811947592303793928e-16 -1.3443908046660001512e-14 -> xyz=-0.006399999999996792803 -0.034000000000000661637 0.28549999999999997602 rpy=1.2173498094410956825e-16 -2.7428229798067236768e-14 -5.0714987764877150767e-13

Commit message: Update the config

File: toddlerbot/robot_descriptions/toddlerbot/toddlerbot.urdf (robot description, URDF)
Before this commit: robot toddlerbot, 85 links, 84 joints
Links:
- link 2xl430_gears: geometry collision mesh filename=../assemblies/left_arm/meshes/left_2xl430_gears_collision.s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; visual mesh filename=../assemblies/left_arm/meshes/left_2xl430_gears_visual.stl
- link 2xl430_gears_2: geometry collision mesh filename=../assemblies/left_arm/meshes/left_2xl430_gears_2_collision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; visual mesh filename=../assemblies/left_arm/meshes/left_2xl430_gears_2_visual.stl
- link 2xl430_gears_3: geometry collision mesh filename=../assemblies/left_arm/meshes/left_2xl430_gears_3_collision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; visual mesh filename=../assemblies/left_arm/meshes/left_2xl430_gears_3_visual.stl
- link 2xl430_gears_4: geometry collision mesh filename=../assemblies/right_arm/meshes/right_2xl430_gears_collision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; visual mesh filename=../assemblies/right_arm/meshes/right_2xl430_gears_visual.stl
- link 2xl430_gears_5: geometry collision mesh filename=../assemblies/right_arm/meshes/right_2xl430_gears_2_collisi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; visual mesh filename=../assemblies/right_arm/meshes/right_2xl430_gears_2_visual.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
- link 2xl430_gears_6: geometry collision mesh filename=../assemblies/right_arm/meshes/right_2xl430_gears_3_collisi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; visual mesh filename=../assemblies/right_arm/meshes/right_2xl430_gears_3_visual.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
- link ank_motor_arm: geometry collision mesh filename=../assemblies/left_leg/meshes/left_ank_motor_arm_collision.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; visual mesh filename=../assemblies/left_leg/meshes/left_ank_motor_arm_visual.stl
- link ank_motor_arm_2: geometry collision mesh filename=../assemblies/left_leg/meshes/left_ank_motor_arm_2_collisio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; visual mesh filename=../assemblies/left_leg/meshes/left_ank_motor_arm_2_visual.s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
- link ank_motor_arm_3: geometry collision mesh filename=../assemblies/right_leg/meshes/right_ank_motor_arm_collisio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; visual mesh filename=../assemblies/right_leg/meshes/right_ank_motor_arm_visual.s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
- link ank_motor_arm_4: geometry collision mesh filename=../assemblies/right_leg/meshes/right_ank_motor_arm_2_collis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; visual mesh filename=../assemblies/right_leg/meshes/right_ank_motor_arm_2_visual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
- link ank_motor_rod_long: geometry collision mesh filename=../assemblies/left_leg/meshes/left_ank_motor_rod_long_colli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; visual mesh filename=../assemblies/left_leg/meshes/left_ank_motor_rod_long_visua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
- link ank_motor_rod_long_2: geometry collision mesh filename=../assemblies/right_leg/meshes/right_ank_motor_rod_long_col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; visual mesh filename=../assemblies/right_leg/meshes/right_ank_motor_rod_long_vis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
- link ank_motor_rod_short: geometry collision mesh filename=../assemblies/left_leg/meshes/left_ank_motor_rod_short_coll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; visual mesh filename=../assemblies/left_leg/meshes/left_ank_motor_rod_short_visu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
- link ank_motor_rod_short_2: geometry collision mesh filename=../assemblies/right_leg/meshes/right_ank_motor_rod_short_co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; visual mesh filename=../assemblies/right_leg/meshes/right_ank_motor_rod_short_vi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
- link ank_pitch_link: geometry collision mesh filename=../assemblies/left_leg/meshes/left_ank_pitch_link_collision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; visual mesh filename=../assemblies/left_leg/meshes/left_ank_pitch_link_visual.stl
- link ank_pitch_link_2: geometry collision mesh filename=../assemblies/right_leg/meshes/right_ank_pitch_link_collisi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; visual mesh filename=../assemblies/right_leg/meshes/right_ank_pitch_link_visual.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
- link ank_roll_link: geometry collision mesh filename=../assemblies/left_leg/meshes/left_ank_roll_link_collision.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; visual mesh filename=../assemblies/left_leg/meshes/left_ank_roll_link_visual.stl
- link ank_roll_link_2: geometry collision mesh filename=../assemblies/right_leg/meshes/right_ank_roll_link_collisio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; visual mesh filename=../assemblies/right_leg/meshes/right_ank_roll_link_visual.s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
- link ank_rr_link: geometry collision mesh filename=../assemblies/left_leg/meshes/left_ank_rr_link_collision.stl; visual mesh filename=../assemblies/left_leg/meshes/left_ank_rr_link_visual.stl
- link ank_rr_link_2: geometry collision mesh filename=../assemblies/left_leg/meshes/left_ank_rr_link_2_collision.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; visual mesh filename=../assemblies/left_leg/meshes/left_ank_rr_link_2_visual.stl
- link ank_rr_link_3: geometry collision mesh filename=../assemblies/right_leg/meshes/right_ank_rr_link_collision.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; visual mesh filename=../assemblies/right_leg/meshes/right_ank_rr_link_visual.stl
- link ank_rr_link_4: geometry collision mesh filename=../assemblies/right_leg/meshes/right_ank_rr_link_2_collisio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; visual mesh filename=../assemblies/right_leg/meshes/right_ank_rr_link_2_visual.s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
- link ball_joint_ball: geometry collision mesh filename=../assemblies/left_leg/meshes/left_ball_joint_ball_collisio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; visual mesh filename=../assemblies/left_leg/meshes/left_ball_joint_ball_visual.s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
- link ball_joint_ball_2: geometry collision mesh filename=../assemblies/left_leg/meshes/left_ball_joint_ball_2_collis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; visual mesh filename=../assemblies/left_leg/meshes/left_ball_joint_ball_2_visual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
- link ball_joint_ball_3: geometry collision mesh filename=../assemblies/right_leg/meshes/right_ball_joint_ball_collis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; visual mesh filename=../assemblies/right_leg/meshes/right_ball_joint_ball_visual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
- link ball_joint_ball_4: geometry collision mesh filename=../assemblies/right_leg/meshes/right_ball_joint_ball_2_coll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; visual mesh filename=../assemblies/right_leg/meshes/right_ball_joint_ball_2_visu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
- link ball_joint_container: geometry collision mesh filename=../assemblies/left_leg/meshes/left_ball_joint_container_col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; visual mesh filename=../assemblies/left_leg/meshes/left_ball_joint_container_vis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
- link ball_joint_container_2: geometry collision mesh filename=../assemblies/left_leg/meshes/left_ball_joint_container_2_c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; visual mesh filename=../assemblies/left_leg/meshes/left_ball_joint_container_2_v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
- link ball_joint_container_3: geometry collision mesh filename=../assemblies/right_leg/meshes/right_ball_joint_container_c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; visual mesh filename=../assemblies/right_leg/meshes/right_ball_joint_container_v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
- link ball_joint_container_4: geometry collision mesh filename=../assemblies/right_leg/meshes/right_ball_joint_container_2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; visual mesh filename=../assemblies/right_leg/meshes/right_ball_joint_container_2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
- link elb_yaw_link: geometry collision mesh filename=../assemblies/left_arm/meshes/left_elb_yaw_link_collision.s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; visual mesh filename=../assemblies/left_arm/meshes/left_elb_yaw_link_visual.stl
- link elb_yaw_link_2: geometry collision mesh filename=../assemblies/right_arm/meshes/right_elb_yaw_link_collision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; visual mesh filename=../assemblies/right_arm/meshes/right_elb_yaw_link_visual.stl
- link gripper: geometry collision mesh filename=../assemblies/left_arm/meshes/left_gripper_collision.stl; visual mesh filename=../assemblies/left_arm/meshes/left_gripper_visual.stl
- link gripper_2: geometry collision mesh filename=../assemblies/right_arm/meshes/right_gripper_collision.stl; visual mesh filename=../assemblies/right_arm/meshes/right_gripper_visual.stl
- link gripper_connector: geometry collision mesh filename=../assemblies/left_arm/meshes/left_gripper_connector_collis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; visual mesh filename=../assemblies/left_arm/meshes/left_gripper_connector_visual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
- link gripper_connector_2: geometry collision mesh filename=../assemblies/right_arm/meshes/right_gripper_connector_coll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; visual mesh filename=../assemblies/right_arm/meshes/right_gripper_connector_visu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
- link hip_roll_link: geometry collision mesh filename=../assemblies/left_leg/meshes/left_hip_roll_link_collision.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; visual mesh filename=../assemblies/left_leg/meshes/left_hip_roll_link_visual.stl
- link hip_roll_link_2: geometry collision mesh filename=../assemblies/right_leg/meshes/right_hip_roll_link_collisio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; visual mesh filename=../assemblies/right_leg/meshes/right_hip_roll_link_visual.s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
- link hip_yaw_link: geometry collision mesh filename=../assemblies/left_leg/meshes/left_hip_yaw_link_collision.s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; visual mesh filename=../assemblies/left_leg/meshes/left_hip_yaw_link_visual.stl
- link hip_yaw_link_2: geometry collision mesh filename=../assemblies/right_leg/meshes/right_hip_yaw_link_collision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; visual mesh filename=../assemblies/right_leg/meshes/right_hip_yaw_link_visual.stl
- link left_calf_link: geometry collision mesh filename=../assemblies/left_leg/meshes/left_calf_link_collision.stl; visual mesh filename=../assemblies/left_leg/meshes/left_calf_link_visual.stl
- link left_hip_pitch_link: geometry collision mesh filename=../assemblies/left_leg/meshes/left_hip_pitch_link_collision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; visual mesh filename=../assemblies/left_leg/meshes/left_hip_pitch_link_visual.stl
- link neck_pitch_link: geometry collision mesh filename=../assemblies/toddlerbot/meshes/neck_pitch_link_collision.s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; visual mesh filename=../assemblies/toddlerbot/meshes/neck_pitch_link_visual.stl
- link neck_yaw_link: geometry collision mesh filename=../assemblies/toddlerbot/meshes/neck_yaw_link_collision.stl; visual mesh filename=../assemblies/toddlerbot/meshes/neck_yaw_link_visual.stl
- link right_calf_link: geometry collision mesh filename=../assemblies/right_leg/meshes/right_calf_link_collision.stl; visual mesh filename=../assemblies/right_leg/meshes/right_calf_link_visual.stl
- link right_hip_pitch_link: geometry collision mesh filename=../assemblies/right_leg/meshes/right_hip_pitch_link_collisi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; visual mesh filename=../assemblies/right_leg/meshes/right_hip_pitch_link_visual.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
- link sho_pitch_link: geometry collision mesh filename=../assemblies/left_arm/meshes/left_sho_pitch_link_collision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; visual mesh filename=../assemblies/left_arm/meshes/left_sho_pitch_link_visual.stl
- link sho_pitch_link_2: geometry collision mesh filename=../assemblies/right_arm/meshes/right_sho_pitch_link_collisi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; visual mesh filename=../assemblies/right_arm/meshes/right_sho_pitch_link_visual.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
- link sho_yaw_link: geometry collision mesh filename=../assemblies/left_arm/meshes/left_sho_yaw_link_collision.s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; visual mesh filename=../assemblies/left_arm/meshes/left_sho_yaw_link_visual.stl
- link sho_yaw_link_2: geometry collision mesh filename=../assemblies/right_arm/meshes/right_sho_yaw_link_collision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; visual mesh filename=../assemblies/right_arm/meshes/right_sho_yaw_link_visual.stl
- link spiral_bevel_1m_14t_30deg: geometry collision mesh filename=../assemblies/toddlerbot/meshes/spiral_bevel_1m_14t_30deg_c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; visual mesh filename=../assemblies/toddlerbot/meshes/spiral_bevel_1m_14t_30deg_v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
- link spiral_bevel_1m_14t_30deg_2: geometry collision mesh filename=../assemblies/toddlerbot/meshes/spiral_bevel_1m_14t_30deg_2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; visual mesh filename=../assemblies/toddlerbot/meshes/spiral_bevel_1m_14t_30deg_2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
- link spur_1m_20t: geometry collision mesh filename=../assemblies/toddlerbot/meshes/spur_1m_20t_collision.stl; visual mesh filename=../assemblies/toddlerbot/meshes/spur_1m_20t_visual.stl
- link spur_1m_24t_drive: geometry collision mesh filename=../assemblies/left_arm/meshes/left_spur_1m_24t_drive_collis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; visual mesh filename=../assemblies/left_arm/meshes/left_spur_1m_24t_drive_visual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
- link spur_1m_24t_drive_2: geometry collision mesh filename=../assemblies/left_arm/meshes/left_spur_1m_24t_drive_2_coll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; visual mesh filename=../assemblies/left_arm/meshes/left_spur_1m_24t_drive_2_visu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
- link spur_1m_24t_drive_3: geometry collision mesh filename=../assemblies/left_arm/meshes/left_spur_1m_24t_drive_3_coll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; visual mesh filename=../assemblies/left_arm/meshes/left_spur_1m_24t_drive_3_visu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
- link spur_1m_24t_drive_4: geometry collision mesh filename=../assemblies/right_arm/meshes/right_spur_1m_24t_drive_coll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; visual mesh filename=../assemblies/right_arm/meshes/right_spur_1m_24t_drive_visu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
- link spur_1m_24t_drive_5: geometry collision mesh filename=../assemblies/right_arm/meshes/right_spur_1m_24t_drive_2_co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; visual mesh filename=../assemblies/right_arm/meshes/right_spur_1m_24t_drive_2_vi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
- link spur_1m_24t_drive_6: geometry collision mesh filename=../assemblies/right_arm/meshes/right_spur_1m_24t_drive_3_co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; visual mesh filename=../assemblies/right_arm/meshes/right_spur_1m_24t_drive_3_vi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
- link spur_1m_24t_driven: geometry collision mesh filename=../assemblies/left_arm/meshes/left_spur_1m_24t_driven_colli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; visual mesh filename=../assemblies/left_arm/meshes/left_spur_1m_24t_driven_visua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
- link spur_1m_24t_driven_2: geometry collision mesh filename=../assemblies/left_arm/meshes/left_spur_1m_24t_driven_2_col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; visual mesh filename=../assemblies/left_arm/meshes/left_spur_1m_24t_driven_2_vis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
- link spur_1m_24t_driven_3: geometry collision mesh filename=../assemblies/left_arm/meshes/left_spur_1m_24t_driven_3_col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; visual mesh filename=../assemblies/left_arm/meshes/left_spur_1m_24t_driven_3_vis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
- link spur_1m_24t_driven_4: geometry collision mesh filename=../assemblies/right_arm/meshes/right_spur_1m_24t_driven_col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; visual mesh filename=../assemblies/right_arm/meshes/right_spur_1m_24t_driven_vis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
- link spur_1m_24t_driven_5: geometry collision mesh filename=../assemblies/right_arm/meshes/right_spur_1m_24t_driven_2_c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; visual mesh filename=../assemblies/right_arm/meshes/right_spur_1m_24t_driven_2_v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
- link spur_1m_24t_driven_6: geometry collision mesh filename=../assemblies/right_arm/meshes/right_spur_1m_24t_driven_3_c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; visual mesh filename=../assemblies/right_arm/meshes/right_spur_1m_24t_driven_3_v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
- link spur_gear_(13_teeth): geometry collision mesh filename=../assemblies/toddlerbot/meshes/spur_gear_(13_teeth)_collis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; visual mesh filename=../assemblies/toddlerbot/meshes/spur_gear_(13_teeth)_visual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
- link spur_gear_19_teeth: geometry collision mesh filename=../assemblies/toddlerbot/meshes/spur_gear_19_teeth_collisio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; visual mesh filename=../assemblies/toddlerbot/meshes/spur_gear_19_teeth_visual.s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
- link spur_gear_19_teeth_2: geometry collision mesh filename=../assemblies/toddlerbot/meshes/spur_gear_19_teeth_2_collis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; visual mesh filename=../assemblies/toddlerbot/meshes/spur_gear_19_teeth_2_visual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
- link spur_gear_21_teeth: geometry collision mesh filename=../assemblies/toddlerbot/meshes/spur_gear_21_teeth_collisio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; visual mesh filename=../assemblies/toddlerbot/meshes/spur_gear_21_teeth_visual.s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
- link spur_gear_21_teeth_2: geometry collision mesh filename=../assemblies/toddlerbot/meshes/spur_gear_21_teeth_2_collis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; visual mesh filename=../assemblies/toddlerbot/meshes/spur_gear_21_teeth_2_visual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
- link torso: geometry collision mesh filename=../assemblies/toddlerbot/meshes/torso_collision.stl; visual mesh filename=../assemblies/toddlerbot/meshes/torso_visual.stl
- link waist_gears: geometry collision mesh filename=../assemblies/toddlerbot/meshes/waist_gears_collision.stl; visual mesh filename=../assemblies/toddlerbot/meshes/waist_gears_visual.stl
- link waist_link: geometry collision mesh filename=../assemblies/toddlerbot/meshes/waist_link_collision.stl; visual mesh filename=../assemblies/toddlerbot/meshes/waist_link_visual.stl
- link wrist_bearing_plate: geometry collision mesh filename=../assemblies/left_arm/meshes/left_wrist_bearing_plate_coll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; visual mesh filename=../assemblies/left_arm/meshes/left_wrist_bearing_plate_visu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
- link wrist_bearing_plate_2: geometry collision mesh filename=../assemblies/right_arm/meshes/right_wrist_bearing_plate_co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; visual mesh filename=../assemblies/right_arm/meshes/right_wrist_bearing_plate_vi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
- link xc430: geometry collision mesh filename=../assemblies/left_arm/meshes/left_xc430_collision.stl; visual mesh filename=../assemblies/left_arm/meshes/left_xc430_visual.stl
- link xc430_2: geometry collision mesh filename=../assemblies/right_arm/meshes/right_xc430_collision.stl; visual mesh filename=../assemblies/right_arm/meshes/right_xc430_visual.stl
