Commit message: Update the MJCF

File: toddlerbot/robot_descriptions/toddlerbot/toddlerbot.urdf (robot description, URDF)
Before this commit: robot toddlerbot, 85 links, 84 joints
Links:
- link 2xl430_gears: geometry visual mesh filename=../assemblies/left_arm/meshes/left_2xl430_gears_visual.stl
- link 2xl430_gears_2: geometry visual mesh filename=../assemblies/left_arm/meshes/left_2xl430_gears_2_visual.stl
- link 2xl430_gears_3: geometry visual mesh filename=../assemblies/left_arm/meshes/left_2xl430_gears_3_visual.stl
- link 2xl430_gears_4: geometry visual mesh filename=../assemblies/right_arm/meshes/right_2xl430_gears_visual.stl
- link 2xl430_gears_5: geometry visual mesh filename=../assemblies/right_arm/meshes/right_2xl430_gears_2_visual.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
- link 2xl430_gears_6: geometry visual mesh filename=../assemblies/right_arm/meshes/right_2xl430_gears_3_visual.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
- link ank_motor_arm: geometry visual mesh filename=../assemblies/left_leg/meshes/left_ank_motor_arm_visual.stl
- link ank_motor_arm_2: geometry visual mesh filename=../assemblies/left_leg/meshes/left_ank_motor_arm_2_visual.s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
- link ank_motor_arm_3: geometry visual mesh filename=../assemblies/right_leg/meshes/right_ank_motor_arm_visual.s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
- link ank_motor_arm_4: geometry visual mesh filename=../assemblies/right_leg/meshes/right_ank_motor_arm_2_visual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
- link ank_motor_rod_long: geometry visual mesh filename=../assemblies/left_leg/meshes/left_ank_motor_rod_long_visua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
- link ank_motor_rod_long_2: geometry visual mesh filename=../assemblies/right_leg/meshes/right_ank_motor_rod_long_vis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
- link ank_motor_rod_short: geometry visual mesh filename=../assemblies/left_leg/meshes/left_ank_motor_rod_short_visu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
- link ank_motor_rod_short_2: geometry visual mesh filename=../assemblies/right_leg/meshes/right_ank_motor_rod_short_vi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
- link ank_pitch_link: geometry visual mesh filename=../assemblies/left_leg/meshes/left_ank_pitch_link_visual.stl
- link ank_pitch_link_2: geometry visual mesh filename=../assemblies/right_leg/meshes/right_ank_pitch_link_visual.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
- link ank_roll_link: geometry visual mesh filename=../assemblies/left_leg/meshes/left_ank_roll_link_visual.stl
- link ank_roll_link_2: geometry visual mesh filename=../assemblies/right_leg/meshes/right_ank_roll_link_visual.s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
- link ank_rr_link: geometry visual mesh filename=../assemblies/left_leg/meshes/left_ank_rr_link_visual.stl
- link ank_rr_link_2: geometry visual mesh filename=../assemblies/left_leg/meshes/left_ank_rr_link_2_visual.stl
- link ank_rr_link_3: geometry visual mesh filename=../assemblies/right_leg/meshes/right_ank_rr_link_visual.stl
- link ank_rr_link_4: geometry visual mesh filename=../assemblies/right_leg/meshes/right_ank_rr_link_2_visual.s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
- link ball_joint_ball: geometry visual mesh filename=../assemblies/left_leg/meshes/left_ball_joint_ball_visual.s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
- link ball_joint_ball_2: geometry visual mesh filename=../assemblies/left_leg/meshes/left_ball_joint_ball_2_visual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
- link ball_joint_ball_3: geometry visual mesh filename=../assemblies/right_leg/meshes/right_ball_joint_ball_visual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
- link ball_joint_ball_4: geometry visual mesh filename=../assemblies/right_leg/meshes/right_ball_joint_ball_2_visu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
- link ball_joint_container: geometry visual mesh filename=../assemblies/left_leg/meshes/left_ball_joint_container_vis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
- link ball_joint_container_2: geometry visual mesh filename=../assemblies/left_leg/meshes/left_ball_joint_container_2_v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
- link ball_joint_container_3: geometry visual mesh filename=../assemblies/right_leg/meshes/right_ball_joint_container_v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
- link ball_joint_container_4: geometry visual mesh filename=../assemblies/right_leg/meshes/right_ball_joint_container_2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
- link elb_yaw_link: geometry visual mesh filename=../assemblies/left_arm/meshes/left_elb_yaw_link_visual.stl
- link elb_yaw_link_2: geometry visual mesh filename=../assemblies/right_arm/meshes/right_elb_yaw_link_visual.stl
- link gripper: geometry visual mesh filename=../assemblies/left_arm/meshes/left_gripper_visual.stl
- link gripper_2: geometry visual mesh filename=../assemblies/right_arm/meshes/right_gripper_visual.stl
- link gripper_connector: geometry visual mesh filename=../assemblies/left_arm/meshes/left_gripper_connector_visual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
- link gripper_connector_2: geometry visual mesh filename=../assemblies/right_arm/meshes/right_gripper_connector_visu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
- link hip_roll_link: geometry visual mesh filename=../assemblies/left_leg/meshes/left_hip_roll_link_visual.stl
- link hip_roll_link_2: geometry visual mesh filename=../assemblies/right_leg/meshes/right_hip_roll_link_visual.s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
- link hip_yaw_link: geometry visual mesh filename=../assemblies/left_leg/meshes/left_hip_yaw_link_visual.stl
- link hip_yaw_link_2: geometry visual mesh filename=../assemblies/right_leg/meshes/right_hip_yaw_link_visual.stl
- link left_calf_link: geometry visual mesh filename=../assemblies/left_leg/meshes/left_calf_link_visual.stl
- link left_hip_pitch_link: geometry visual mesh filename=../assemblies/left_leg/meshes/left_hip_pitch_link_visual.stl
- link neck_pitch_link: geometry visual mesh filename=../assemblies/toddlerbot/meshes/neck_pitch_link_visual.stl
- link neck_yaw_link: geometry visual mesh filename=../assemblies/toddlerbot/meshes/neck_yaw_link_visual.stl
- link right_calf_link: geometry visual mesh filename=../assemblies/right_leg/meshes/right_calf_link_visual.stl
- link right_hip_pitch_link: geometry visual mesh filename=../assemblies/right_leg/meshes/right_hip_pitch_link_visual.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
- link sho_pitch_link: geometry visual mesh filename=../assemblies/left_arm/meshes/left_sho_pitch_link_visual.stl
- link sho_pitch_link_2: geometry visual mesh filename=../assemblies/right_arm/meshes/right_sho_pitch_link_visual.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
- link sho_yaw_link: geometry visual mesh filename=../assemblies/left_arm/meshes/left_sho_yaw_link_visual.stl
- link sho_yaw_link_2: geometry visual mesh filename=../assemblies/right_arm/meshes/right_sho_yaw_link_visual.stl
- link spiral_bevel_1m_14t_30deg: geometry visual mesh filename=../assemblies/toddlerbot/meshes/spiral_bevel_1m_14t_30deg_v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
- link spiral_bevel_1m_14t_30deg_2: geometry visual mesh filename=../assemblies/toddlerbot/meshes/spiral_bevel_1m_14t_30deg_2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
- link spur_1m_20t: geometry visual mesh filename=../assemblies/toddlerbot/meshes/spur_1m_20t_visual.stl
- link spur_1m_24t_drive: geometry visual mesh filename=../assemblies/left_arm/meshes/left_spur_1m_24t_drive_visual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
- link spur_1m_24t_drive_2: geometry visual mesh filename=../assemblies/left_arm/meshes/left_spur_1m_24t_drive_2_visu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
- link spur_1m_24t_drive_3: geometry visual mesh filename=../assemblies/left_arm/meshes/left_spur_1m_24t_drive_3_visu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
- link spur_1m_24t_drive_4: geometry visual mesh filename=../assemblies/right_arm/meshes/right_spur_1m_24t_drive_visu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
- link spur_1m_24t_drive_5: geometry visual mesh filename=../assemblies/right_arm/meshes/right_spur_1m_24t_drive_2_vi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
- link spur_1m_24t_drive_6: geometry visual mesh filename=../assemblies/right_arm/meshes/right_spur_1m_24t_drive_3_vi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
- link spur_1m_24t_driven: geometry visual mesh filename=../assemblies/left_arm/meshes/left_spur_1m_24t_driven_visua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
- link spur_1m_24t_driven_2: geometry visual mesh filename=../assemblies/left_arm/meshes/left_spur_1m_24t_driven_2_vis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
- link spur_1m_24t_driven_3: geometry visual mesh filename=../assemblies/left_arm/meshes/left_spur_1m_24t_driven_3_vis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
- link spur_1m_24t_driven_4: geometry visual mesh filename=../assemblies/right_arm/meshes/right_spur_1m_24t_driven_vis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
- link spur_1m_24t_driven_5: geometry visual mesh filename=../assemblies/right_arm/meshes/right_spur_1m_24t_driven_2_v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
- link spur_1m_24t_driven_6: geometry visual mesh filename=../assemblies/right_arm/meshes/right_spur_1m_24t_driven_3_v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
- link spur_gear_(13_teeth): geometry visual mesh filename=../assemblies/toddlerbot/meshes/spur_gear_(13_teeth)_visual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
- link spur_gear_19_teeth: geometry visual mesh filename=../assemblies/toddlerbot/meshes/spur_gear_19_teeth_visual.s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
- link spur_gear_19_teeth_2: geometry visual mesh filename=../assemblies/toddlerbot/meshes/spur_gear_19_teeth_2_visual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
- link spur_gear_21_teeth: geometry visual mesh filename=../assemblies/toddlerbot/meshes/spur_gear_21_teeth_visual.s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
- link spur_gear_21_teeth_2: geometry visual mesh filename=../assemblies/toddlerbot/meshes/spur_gear_21_teeth_2_visual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
- link torso: geometry visual mesh filename=../assemblies/toddlerbot/meshes/torso_visual.stl
- link waist_gears: geometry visual mesh filename=../assemblies/toddlerbot/meshes/waist_gears_visual.stl
- link waist_link: geometry visual mesh filename=../assemblies/toddlerbot/meshes/waist_link_visual.stl
- link wrist_bearing_plate: geometry visual mesh filename=../assemblies/left_arm/meshes/left_wrist_bearing_plate_visu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
- link wrist_bearing_plate_2: geometry visual mesh filename=../assemblies/right_arm/meshes/right_wrist_bearing_plate_vi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
- link xc430: geometry visual mesh filename=../assemblies/left_arm/meshes/left_xc430_visual.stl
- link xc430_2: geometry visual mesh filename=../assemblies/right_arm/meshes/right_xc430_visual.stl

Commit message: Fix the ankle constraints

File: toddlerbot/robot_descriptions/toddlerbot/toddlerbot.urdf (robot description, URDF)
Before this commit: robot toddlerbot, 67 links, 66 joints
Links:
- link ank_motor_rod_short_2: mass 0.0017000000000000005558 -> 0.0017000000000000001221
- link ank_rr_link_3: mass 0.0014499999999999999001 -> 0.0014500000000000001169
- link ank_rr_link_4: mass 0.0014499999999999999001 -> 0.0014500000000000001169
- link hip_roll_link: mass 0.10699970659110667748 -> 0.10699970659110669136
- link hip_roll_link_2: mass 0.10699970659110667748 -> 0.10699970659110669136
- link hip_yaw_link: mass 0.017999999999999991701 -> 0.017999999999999984762
- link hip_yaw_link_2: mass 0.01799999999999999864 -> 0.017999999999999984762
- link left_calf_link: mass 0.079607494529051470167 -> 0.079607494529051442411
- link left_hip_pitch_link_xm430: mass 0.035548688791081778371 -> 0.035548688791081757554
- link right_calf_link: mass 0.079607494529051456289 -> 0.079607494529051442411
Joints:
- joint right_ank_L_rev_1: origin xyz=0.017999999999999981293 0.015999999999999847677 -0.020600000000000014133 rpy=6.2884229534673233247e-16 3.939086273962429945e-15 0.018223085042996144817 -> xyz=0.017999999999999981293 0.015999999999999847677 -0.020600000000000010664 rpy=6.2884229534673233247e-16 3.9390862739624346782e-15 0.018223085042996144817
- joint right_ank_L_rev_2: origin xyz=-6.9388939039072283776e-18 -0.0099999999999996203037 3.1225022567582527699e-17 rpy=-1.5707963267948887864 -1.3320366994106427327 -1.5707963267948827912 -> xyz=-6.9388939039072283776e-18 -0.0099999999999996203037 2.7755575615628913511e-17 rpy=-1.5707963267948887864 -1.3320366994106427327 -1.5707963267948827912
- joint right_ank_S_rev_1: origin xyz=-0.018000000000000026396 0.016000000000000735856 -0.02059999999999996903 rpy=-4.338977813478965687e-16 1.6392354569195739132e-16 3.1154741050825114357 -> xyz=-0.018000000000000026396 0.016000000000000735856 -0.02059999999999996903 rpy=-4.338977813478965687e-16 1.6392354569195936347e-16 3.1154741050825114357
- joint right_ank_S_rev_2: origin xyz=-2.7755575615628913511e-16 0.010000000000000563993 -1.561251128379126385e-16 rpy=-1.5707963267949354158 1.2119133862908570975 -1.5707963267949336394 -> xyz=-2.7408630920433552092e-16 0.010000000000000508482 -1.561251128379126385e-16 rpy=-1.5707963267949354158 1.2119133862908570975 -1.5707963267949336394
- joint right_ank_act_1: origin xyz=0.013499999999995838246 0.044500000000006201262 0.0040000000000029352354 rpy=-2.9762431821176080221e-13 -7.5970722241046912715e-14 0.21173394130155420712 -> xyz=0.013499999999995845185 0.044500000000006201262 0.0040000000000029352354 rpy=-2.976243182117608527e-13 -7.5970722241046887472e-14 0.21173394130155420712
- joint right_ank_act_2: origin xyz=0.013500000000004725234 0.064500000000008106404 -0.024800000000001404254 rpy=-3.1415926535894733718 -2.3305959971649736532e-13 0.22995607267265857909 -> xyz=0.013500000000004732173 0.064500000000008106404 -0.024800000000001404254 rpy=-3.1415926535894733718 -2.3305959971649736532e-13 0.22995607267265857909
- joint right_ank_pitch: origin xyz=-4.0265291502142843319e-17 0.10000000000000000555 -0.010399999999999947481 rpy=-5.6239133145192868052e-16 -1.1344214119702528777e-16 3.141592653589793116 -> xyz=-3.3506429374353506934e-17 0.10000000000000000555 -0.01039999999999995442 rpy=-5.6239133145187819342e-16 -1.1344214119703426107e-16 3.141592653589793116
- joint right_ank_roll: origin xyz=0.0014999999999999924418 2.7755575615628913511e-17 -1.3877787807814456755e-17 rpy=3.141592653589793116 -1.570796326794896336 0 -> xyz=0.0014999999999999924418 2.7755575615628913511e-17 -6.9388939039072283776e-18 rpy=3.141592653589793116 -1.570796326794896336 0
- joint right_knee: origin xyz=-2.9922268808255885729e-17 -0.096000000000000029754 -0.0091999999999999235167 rpy=1.2825226684517786044e-14 1.3611434254495038701e-14 -3.1415926535897926719 -> xyz=3.9466670230816398047e-17 -0.096000000000000029754 -0.0091999999999999235167 rpy=1.282522668451654911e-14 1.4584655840118584511e-16 -3.1415926535897926719

Commit message: Update the collisions

File: toddlerbot/robot_descriptions/toddlerbot/toddlerbot.urdf (robot description, URDF)
Before this commit: robot toddlerbot, 79 links, 78 joints
Links:
- link 2xl430_gears: geometry collision mesh filename=collisions/left_2xl430_gears_collision.stl; visual mesh filename=../assemblies/left_arm_hand/meshes/left_2xl430_gears_visual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
- link 2xl430_gears_2: geometry collision mesh filename=collisions/left_2xl430_gears_2_collision.stl; visual mesh filename=../assemblies/left_arm_hand/meshes/left_2xl430_gears_2_visu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
- link 2xl430_gears_3: geometry collision mesh filename=collisions/left_2xl430_gears_3_collision.stl; visual mesh filename=../assemblies/left_arm_hand/meshes/left_2xl430_gears_3_visu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
- link 2xl430_gears_4: geometry collision mesh filename=collisions/right_2xl430_gears_collision.stl; visual mesh filename=../assemblies/right_arm_hand/meshes/right_2xl430_gears_visu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
- link 2xl430_gears_5: geometry collision mesh filename=collisions/right_2xl430_gears_2_collision.stl; visual mesh filename=../assemblies/right_arm_hand/meshes/right_2xl430_gears_2_vi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
- link 2xl430_gears_6: geometry collision mesh filename=collisions/right_2xl430_gears_3_collision.stl; visual mesh filename=../assemblies/right_arm_hand/meshes/right_2xl430_gears_3_vi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
- link hand: geometry collision mesh filename=../assemblies/left_arm_hand/meshes/left_hand_collision.stl; visual mesh filename=../assemblies/left_arm_hand/meshes/left_hand_visual.stl
- link hand_2: geometry collision mesh filename=../assemblies/right_arm_hand/meshes/right_hand_collision.stl; visual mesh filename=../assemblies/right_arm_hand/meshes/right_hand_visual.stl
- link hip_roll_link: geometry collision mesh filename=collisions/left_hip_roll_link_collision.stl; visual mesh filename=../assemblies/left_leg_XM430/meshes/left_hip_roll_link_visu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
- link hip_roll_link_2: geometry collision mesh filename=collisions/right_hip_roll_link_collision.stl; visual mesh filename=../assemblies/right_leg_XM430/meshes/right_hip_roll_link_vi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
- link left_calf_link: geometry collision mesh filename=collisions/left_calf_link_collision.stl; visual mesh filename=../assemblies/left_leg_XM430/meshes/left_calf_link_visual.s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
- link left_hip_pitch_link_xm430: geometry collision mesh filename=collisions/left_hip_pitch_link_xm430_collision.stl; visual mesh filename=../assemblies/left_leg_XM430/meshes/left_hip_pitch_link_xm4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
- link left_sole_link: geometry collision mesh filename=../assemblies/left_leg_XM430/meshes/left_sole_link_collisio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; visual mesh filename=../assemblies/left_leg_XM430/meshes/left_sole_link_visual.s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
- link neck_pitch_link: geometry collision mesh filename=collisions/neck_pitch_link_collision.stl; visual mesh filename=../assemblies/toddlerbot/meshes/neck_pitch_link_visual.stl
- link right_calf_link: geometry collision mesh filename=collisions/right_calf_link_collision.stl; visual mesh filename=../assemblies/right_leg_XM430/meshes/right_calf_link_visual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
- link right_hip_pitch_link_xm430: geometry collision mesh filename=collisions/right_hip_pitch_link_xm430_collision.stl; visual mesh filename=../assemblies/right_leg_XM430/meshes/right_hip_pitch_link_x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
- link right_sole_link: geometry collision mesh filename=../assemblies/right_leg_XM430/meshes/right_sole_link_collis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; visual mesh filename=../assemblies/right_leg_XM430/meshes/right_sole_link_visual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
- link torso: geometry collision mesh filename=collisions/torso_collision.stl; visual mesh filename=../assemblies/toddlerbot/meshes/torso_visual.stl
- link waist_link: geometry collision mesh filename=collisions/waist_link_collision.stl; visual mesh filename=../assemblies/toddlerbot/meshes/waist_link_visual.stl

Commit message: Update the standing test

File: toddlerbot/robot_descriptions/toddlerbot/toddlerbot.urdf (robot description, URDF)
Before this commit: robot toddlerbot, 77 links, 76 joints
Links:
- link left_sole_link: geometry collision mesh filename=collisions/left_sole_link_collision.stl; visual mesh filename=../assemblies/left_leg_XM430/meshes/left_sole_link_visual.s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
- link right_sole_link: geometry collision mesh filename=collisions/right_sole_link_collision.stl; visual mesh filename=../assemblies/right_leg_XM430/meshes/right_sole_link_visual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

Commit message: Use collision primitives

File: toddlerbot/robot_descriptions/toddlerbot/toddlerbot.urdf (robot description, URDF)
Before this commit: robot toddlerbot, 75 links, 74 joints
Links:
- link 2xl430_gears: geometry collision sphere radius=0.031146449113064925; visual mesh filename=../assemblies/left_arm_hand/meshes/left_2xl430_gears_visual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
- link 2xl430_gears_2: geometry collision sphere radius=0.031146338948323835; visual mesh filename=../assemblies/left_arm_hand/meshes/left_2xl430_gears_2_visu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
- link 2xl430_gears_4: geometry collision sphere radius=0.031146449113064925; visual mesh filename=../assemblies/right_arm_hand/meshes/right_2xl430_gears_visu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
- link 2xl430_gears_5: geometry collision sphere radius=0.03114710642898145; visual mesh filename=../assemblies/right_arm_hand/meshes/right_2xl430_gears_2_vi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
- link ank_roll_link: geometry collision box size=0.041999999433755875 0.04500000039115548 0.12000000104308128; visual mesh filename=../assemblies/left_leg_XM430/meshes/left_ank_roll_link_visu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
- link ank_roll_link_2: geometry collision box size=0.041999999433755875 0.04500000039115548 0.12000000104308128; visual mesh filename=../assemblies/right_leg_XM430/meshes/right_ank_roll_link_vi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
- link hand: geometry collision box size=0.020999999716877937 0.09677662048488855 0.04629777139052749; visual mesh filename=../assemblies/left_arm_hand/meshes/left_hand_visual.stl
- link hand_2: geometry collision box size=0.020999999716877937 0.09677662048488855 0.04629777115769684; visual mesh filename=../assemblies/right_arm_hand/meshes/right_hand_visual.stl
- link hip_roll_link: geometry collision box size=0.04650000110268593 0.04089999943971634 0.04090000095311552; visual mesh filename=../assemblies/left_leg_XM430/meshes/left_hip_roll_link_visu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
- link hip_roll_link_2: geometry collision box size=0.04650000110268593 0.04089999943971634 0.04090000095311552; visual mesh filename=../assemblies/right_leg_XM430/meshes/right_hip_roll_link_vi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
- link left_calf_link: geometry visual mesh filename=../assemblies/left_leg_XM430/meshes/left_calf_link_visual.s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
- link left_hip_pitch_link_xm430: geometry collision box size=0.03999999910593033 0.1190000013448298 0.049600002355873585; visual mesh filename=../assemblies/left_leg_XM430/meshes/left_hip_pitch_link_xm4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
- link neck_pitch_link: geometry visual mesh filename=../assemblies/toddlerbot/meshes/neck_pitch_link_visual.stl
- link right_calf_link: geometry visual mesh filename=../assemblies/right_leg_XM430/meshes/right_calf_link_visual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
- link right_hip_pitch_link_xm430: geometry collision box size=0.03999999910593033 0.1190000013448298 0.049599998630583286; visual mesh filename=../assemblies/right_leg_XM430/meshes/right_hip_pitch_link_x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
- link torso: geometry collision box size=0.13100000098347664 0.12759999930858612 0.12457482283934951; visual mesh filename=../assemblies/toddlerbot/meshes/torso_visual.stl
- link waist_link: geometry collision box size=0.10000000149011612 0.024500000523403287 0.06900000385940075; visual mesh filename=../assemblies/toddlerbot/meshes/waist_link_visual.stl

Commit message: Remove more collision bodies

File: toddlerbot/robot_descriptions/toddlerbot/toddlerbot.urdf (robot description, URDF)
Before this commit: robot toddlerbot, 75 links, 74 joints
Links:
- link 2xl430_gears: geometry visual mesh filename=../assemblies/left_arm_hand/meshes/left_2xl430_gears_visual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
- link 2xl430_gears_2: geometry visual mesh filename=../assemblies/left_arm_hand/meshes/left_2xl430_gears_2_visu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
- link 2xl430_gears_4: geometry visual mesh filename=../assemblies/right_arm_hand/meshes/right_2xl430_gears_visu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
- link 2xl430_gears_5: geometry visual mesh filename=../assemblies/right_arm_hand/meshes/right_2xl430_gears_2_vi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
- link hand: geometry visual mesh filename=../assemblies/left_arm_hand/meshes/left_hand_visual.stl
- link hand_2: geometry visual mesh filename=../assemblies/right_arm_hand/meshes/right_hand_visual.stl
- link hip_roll_link: geometry visual mesh filename=../assemblies/left_leg_XM430/meshes/left_hip_roll_link_visu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
- link hip_roll_link_2: geometry visual mesh filename=../assemblies/right_leg_XM430/meshes/right_hip_roll_link_vi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
- link left_hip_pitch_link_xm430: geometry visual mesh filename=../assemblies/left_leg_XM430/meshes/left_hip_pitch_link_xm4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
- link right_hip_pitch_link_xm430: geometry visual mesh filename=../assemblies/right_leg_XM430/meshes/right_hip_pitch_link_x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
- link torso: geometry visual mesh filename=../assemblies/toddlerbot/meshes/torso_visual.stl
- link waist_link: geometry visual mesh filename=../assemblies/toddlerbot/meshes/waist_link_visual.stl

Commit message: Update the box size

File: toddlerbot/robot_descriptions/toddlerbot/toddlerbot.urdf (robot description, URDF)
Before this commit: robot toddlerbot, 75 links, 74 joints
Links:
- link ank_roll_link: geometry collision box size=0.035699999518692495 0.04500000039115548 0.12000000104308128; visual mesh filename=../assemblies/left_leg_XM430/meshes/left_ank_roll_link_visu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
- link ank_roll_link_2: geometry collision box size=0.035699999518692495 0.04500000039115548 0.12000000104308128; visual mesh filename=../assemblies/right_leg_XM430/meshes/right_ank_roll_link_vi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
