Commit message: add collision for torso, adjust z and pitch on GUI

File: toddlerbot/robot_descriptions/toddlerbot/toddlerbot.urdf (robot description, URDF)
Before this commit: robot toddlerbot, 75 links, 74 joints
Links:
- link hand: geometry collision box size=0.020999999716877937 0.09677662048488855 0.04629777139052749; visual mesh filename=../assemblies/left_arm_hand/meshes/left_hand_visual.stl
- link hand_2: geometry collision box size=0.020999999716877937 0.09677662048488855 0.04629777115769684; visual mesh filename=../assemblies/right_arm_hand/meshes/right_hand_visual.stl
- link left_hip_pitch_link_xm430: geometry collision box size=0.03999999910593033 0.1190000013448298 0.049600002355873585; visual mesh filename=../assemblies/left_leg_XM430/meshes/left_hip_pitch_link_xm4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
- link right_hip_pitch_link_xm430: geometry collision box size=0.03999999910593033 0.1190000013448298 0.049599998630583286; visual mesh filename=../assemblies/right_leg_XM430/meshes/right_hip_pitch_link_x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
- link torso: geometry collision box size=0.13100000098347664 0.10207999944686891 0.1245468775741756; visual mesh filename=../assemblies/toddlerbot/meshes/torso_visual.stl

Commit message: synced toddlerbot from main branch

File: toddlerbot/robot_descriptions/toddlerbot/toddlerbot.urdf (robot description, URDF)
Before this commit: robot toddlerbot, 75 links, 74 joints
Links:
- link ank_motor_rod_short: mass 0.0017000000000000005558 -> 0.0017000000000000001221
- link ank_motor_rod_short_2: mass 0.0017000000000000005558 -> 0.0017000000000000001221
- link ank_roll_link: mass 0.019499999999999989564 -> 0.027200000000000008893; geometry collision box size=0.041999999433755875 0.04500000271946192 0.12000000476837158; visual mesh filename=../assemblies/left_leg_XM430/meshes/left_ank_roll_link_visu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
- link ank_roll_link_2: mass 0.019499999999999989564 -> 0.027200000000000008893; geometry collision box size=0.041999999433755875 0.04500000271946192 0.12000000476837158; visual mesh filename=../assemblies/right_leg_XM430/meshes/right_ank_roll_link_vi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
- link ank_rr_link: mass 0.0014499999999999996832 -> 0.0014499999999999999001
- link ank_rr_link_2: mass 0.0014499999999999996832 -> 0.0014499999999999999001
- link ank_rr_link_3: mass 0.0014499999999999996832 -> 0.0014499999999999999001
- link ank_rr_link_4: mass 0.0014499999999999996832 -> 0.0014499999999999999001
- link hip_yaw_link: mass 0.018000000000000009048 -> 0.017999999999999988232
- link hip_yaw_link_2: mass 0.018000000000000009048 -> 0.017999999999999988232
- link left_hip_pitch_link_xm430: mass 0.1148009013503056841 -> 0.11480090135030569798
- link right_calf_link: mass 0.086799999986183568046 -> 0.086799999986183554168
- link right_hip_pitch_link_xm430: mass 0.1148009013503056841 -> 0.11480090135030567022
- link spiral_bevel_1m_14t_30deg: mass 0.00067997563436136246491 -> 0.00073261524436595492574
- link spiral_bevel_1m_14t_30deg_2: mass 0.00067997563436136246491 -> 0.00073261524436595492574
- link spur_gear_19_teeth: mass 0.0010993711450650533144 -> 0.0011084409433758843876
- link spur_gear_19_teeth_2: mass 0.0010993711450650533144 -> 0.0011084409433758843876
- link spur_gear_21_teeth: mass 0.0010063046528317972673 -> 0.0010185686142775147826
- link spur_gear_21_teeth_2: mass 0.0010063046528317972673 -> 0.0010185686142775147826
- link torso: mass 0.58475267652546314423 -> 0.60012685450989189384
- link waist_gears: mass 0.025809950030454158199 -> 0.025874065810895640477
- link waist_link: mass 0.16631953490612458313 -> 0.16631953490612461088
- link xm430_plate: mass 0.0026999999999999997093 -> 0.0026999999999999992756
- link xm430_plate_2: mass 0.0026999999999999997093 -> 0.0026999999999999992756
Joints:
- joint left_ank_long_rev_1: origin xyz=-0.018000000000000015987 0.01599999999999926481 -0.020600000000001391504 rpy=-2.876394309884160705e-16 1.6317439732762683578e-16 3.1233695685467286474 -> xyz=-0.018000000000000064559 0.015999999999999292566 -0.020600000000001391504 rpy=-2.876394309884160705e-16 1.6317439732762683578e-16 3.1233695685467286474
- joint left_ank_roll: origin xyz=0.0015000000000000002481 2.7755575615628913511e-17 3.2742905609062233907e-17 rpy=9.9573127520767875392e-16 1.570796326794891673 0 -> xyz=0.0014999999999999995975 0 -1.5395670849294162963e-17 rpy=9.9573127520767875392e-16 1.570796326794891673 0
- joint left_ank_short_rev_1: origin xyz=0.018000000000000002109 0.015999999999999986455 -0.020600000000000010664 rpy=4.2172831995673088897e-16 -4.4678623027074358005e-17 0.026118548507422217203 -> xyz=0.017999999999999953537 0.016000000000000014211 -0.020600000000000010664 rpy=4.2172831995673088897e-16 -4.4678623027074358005e-17 0.026118548507422217203
- joint left_hip_yaw_drive: limit lower=-1.4211966766239538806 upper=1.4211966766239538806 effort=1 velocity=20 -> lower=-1.7361433085627806516 upper=1.7361433085627806516 effort=1 velocity=20; origin xyz=-0.036999999999998194056 0.037100000000006128076 -0.039500000000001291023 rpy=-1.5707963267949545116 -4.7906511943294847217e-13 -3.592506663906207747e-13 -> xyz=-0.036999999999998457734 0.037100000000005961542 -0.03950000000000024325 rpy=-1.5707963267949545116 -4.8003070743589248247e-13 -3.5749181392930616155e-13
- joint left_hip_yaw_driven: origin xyz=-0.037000000000000012046 0.041099999999999997646 -0.0194999999999999514 rpy=-1.5707963267948990005 -1.570796326794896558 0 -> xyz=-0.036999999999999998168 0.041100000000000011524 -0.019500000000000027728 rpy=-1.5707963267948947816 -1.570796326794896558 0
- joint left_leg_fixed: origin xyz=0 0 0.004999999999999997502 rpy=3.1415926535897873428 -0 -1.6681280046507162628e-30 -> xyz=0 0 0.004999999999999997502 rpy=3.1415926535897926719 -1.9428902930939016723e-16 -7.6327832942984196016e-16
- joint left_sho_pitch: limit lower=-1.570796326794896558 upper=1.570796326794896558 effort=1 velocity=20 -> lower=-3.141592653589793116 upper=1.570796326794896558 effort=1 velocity=20; origin xyz=-0.0030000000000065664245 0.062000000000004926171 0.10423651076282140771 rpy=-1.5707963267949054398 -3.6755753074147447628e-14 3.6857314245917344439e-14 -> xyz=-0.0030000000000002949654 0.062000000000001082023 0.10423651076281743866 rpy=-1.5707963267949081043 -4.127643409825574977e-14 3.4723733359249779961e-14
- joint neck_pitch_drive: limit lower=-1.4279966607226330932 upper=1.4279966607226330932 effort=1 velocity=20 -> lower=-2.174948760177549012 upper=2.174948760177549012 effort=1 velocity=20; origin xyz=-1.4224732503009818174e-16 0.015649999999999136824 -0.0087999999999959568897 rpy=-2.4492935983152098954e-16 -2.1427228763620856097e-15 -1.570796326794896558 -> xyz=-6.9735883734267645195e-16 0.015649999999999053557 -0.0087999999999970532349 rpy=-1.1409718301987536487e-15 4.409645192886135633e-16 -1.5707963267948976682
- joint neck_pitch_driven: origin xyz=3.7500001368040436489e-10 -0.0051500000614753682626 0.027499999999999830136 rpy=1.57079632679489678 1.7322096859329345721e-15 -3.1415926535897922278 -> xyz=3.7499979510524639181e-10 -0.0051500000614751947903 0.027499999999999941158 rpy=1.5707963267948978903 -2.0825786444073518345e-16 3.141592653589793116
- joint neck_yaw_drive: limit lower=-2.2689280275926284602 upper=2.2689280275926284602 effort=1 velocity=20 -> lower=-2.8797932657906435416 upper=2.8797932657906435416 effort=1 velocity=20; origin xyz=-0.0050000000000041591036 2.1706564040395755645e-15 0.12148651076282282468 rpy=-4.7086950490309927255e-15 -3.2377166610426843676e-14 2.947288666540578667e-14 -> xyz=-0.004999999999999517851 2.6555840535020396321e-18 0.121486510762817565 rpy=1.1318451824181020002e-14 2.6985403517595457696e-15 -5.3863140912757267331e-15
- joint neck_yaw_driven: limit lower=-3.141592653589793116 upper=3.141592653589793116 effort=1 velocity=20 -> lower=-2.6179938779914944114 upper=2.6179938779914944114 effort=1 velocity=20; origin xyz=0.015999999999998446021 3.2990787509752002888e-15 0.12248651076282082717 rpy=2.3463681399312212716e-14 3.1845915227826135867e-14 3.141592653589793116 -> xyz=0.016000000000001235456 2.2310681558151314601e-17 0.12248651076281746874 rpy=-4.8668742840765556337e-16 -4.0649010562893427138e-15 3.141592653589793116
- joint right_ank_long_rev_1: origin xyz=0.017999999999999995171 0.016000000000000014211 -0.020600000000000007194 rpy=2.4036779374278231896e-16 5.7386734097817399387e-16 0.018223085043007757056 -> xyz=0.01799999999999999864 0.015999999999999764411 -0.020600000000000132094 rpy=-7.8386807614170502355e-15 7.211088289180617976e-16 0.018223085043007757056
- joint right_ank_roll: origin xyz=0.0015000000000000002481 2.7755575615628913511e-17 1.2143064331837649661e-17 rpy=-8.0803901893659494053e-15 1.5707963267948927832 0 -> xyz=0.001499999999999998947 8.3266726846886740532e-17 1.3660947373317355868e-17 rpy=6.1391486757704172424e-30 1.5707963267948927832 0
- joint right_ank_short_rev_1: origin xyz=-0.018000000000000012518 0.016000000000000014211 -0.020599999999999993316 rpy=1.6033225897674528336e-14 -1.3300018467937457486e-14 3.1154741050824821258 -> xyz=-0.018000000000000009048 0.015999999999999764411 -0.020600000000000118217 rpy=2.411086010918130345e-14 -1.3088994399411267302e-14 3.1154741050824821258
- joint right_hip_yaw_drive: limit lower=-1.4211966766239538806 upper=1.4211966766239538806 effort=1 velocity=20 -> lower=-1.7361433085627806516 upper=1.7361433085627806516 effort=1 velocity=20; origin xyz=0.037000000000001746769 0.037100000000003664768 -0.039500000000000978773 rpy=-1.5707963267949545116 -4.7905720692590075245e-13 -3.5747430955122047375e-13 -> xyz=0.037000000000001719014 0.03710000000000327619 -0.0394999999999998061 rpy=-1.5707963267949545116 -4.8002361403961149694e-13 -3.5216274341110541015e-13
- joint right_hip_yaw_driven: origin xyz=0.036999999999999991229 0.041100000000000011524 -0.0194999999999999514 rpy=-1.5707963267949003328 -1.5707963267948956698 0 -> xyz=0.036999999999999991229 0.041100000000000011524 -0.019500000000000017319 rpy=-1.570796326794896558 -1.5707963267948961139 0
- joint right_leg_fixed: origin xyz=0 0 0.0050000000000000044409 rpy=-3.141592653589793116 -0 -9.3397966250929058941e-32 -> xyz=0 -6.9388939039072283776e-18 0.0050000000000000044409 rpy=-3.1415926535897926719 1.8281169925220331315e-17 -3.5772536718062127375e-16
- joint right_sho_pitch: limit lower=-1.570796326794896558 upper=1.570796326794896558 effort=1 velocity=20 -> lower=-1.570796326794896558 upper=3.141592653589793116 effort=1 velocity=20; origin xyz=-0.0030000000000019676726 -0.062000000000000089762 0.10423651076282176853 rpy=-1.5707963267948885644 3.4812325502379109658e-14 -3.1415926535897562566 -> xyz=-0.0029999999999986998872 -0.06200000000000097794 0.10423651076281731376 rpy=-1.5707963267948885644 3.4812325502379109658e-14 -3.1415926535897562566
- joint waist_act_1: limit lower=-2.7825534678416246059 upper=2.7825534678416246059 effort=1 velocity=20 -> lower=-4.6774823953448034786 upper=4.6774823953448034786 effort=1 velocity=20; origin xyz=5.380496587145115132e-16 0.019600000000000075695 -0.012750000000000080713 rpy=1.5707963267949007768 1.5707963267948907848 0 -> xyz=5.7457652915638341522e-17 0.019599999999999964673 -0.012750000000000025202 rpy=1.5707963267948954478 1.570796326794896336 0
- joint waist_act_2: limit lower=-2.7825534678416246059 upper=2.7825534678416246059 effort=1 velocity=20 -> lower=-4.6774823953448034786 upper=4.6774823953448034786 effort=1 velocity=20; origin xyz=-2.6785082652000791162e-16 0.019599999999999902223 -0.032749999999999612754 rpy=1.5707963267948958919 1.3463968515392310543 -4.6125152814992733786e-14 -> xyz=4.2745485696894321379e-17 0.019600000000000013245 -0.032749999999999994393 rpy=1.5707963267948956698 1.3463968515392303882 6.7698458176426589005e-15
- joint waist_roll: origin xyz=-0.022707865260691548898 -1.3479418671744790767e-17 -0.014000000000000234479 rpy=-1.5707963267949187625 -1.0371626905663003511e-14 1.5707963267948794606 -> xyz=-0.022707865260692617487 -2.4393502827093082036e-16 -0.013999999999999814676 rpy=-1.5707963267948974462 1.8675461532229772614e-15 1.5707963267948952257
- joint waist_yaw: origin xyz=0 -9.8607613152626475676e-32 0 rpy=1.6626925279001758682e-14 4.9579962395338894532e-14 -3.1415926535897900074 -> xyz=0 -3.1104917983741196655e-18 -7.5188305028877687703e-30 rpy=-1.4111145075746007461e-16 -4.1376224834060906822e-15 3.1415926535897922278
