Commit message: Add the gripper to the URDF

File: toddlerbot/robot_descriptions/toddlerbot/toddlerbot.urdf (robot description, URDF)
Before this commit: robot toddlerbot, 75 links, 74 joints
Links:
- removed link hand
- removed link hand_2
- added link gripper_connector, mass 0.0099999999999999967387; visual mesh filename=../assemblies/left_arm_gripper/meshes/left_gripper_connecto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
- added link gripper_connector_2, mass 0.0099999999999999967387; visual mesh filename=../assemblies/right_arm_gripper/meshes/right_gripper_connec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
- added link left_rail_guide, mass 0.032142035224833366558; visual mesh filename=../assemblies/left_arm_gripper/meshes/left_rail_guide_visua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
- added link rail, mass 0.01189999999999999912; visual mesh filename=../assemblies/left_arm_gripper/meshes/left_rail_visual.stl
- added link rail_2, mass 0.01189999999999999912; visual mesh filename=../assemblies/left_arm_gripper/meshes/left_rail_2_visual.stl
- added link rail_3, mass 0.01189999999999999912; visual mesh filename=../assemblies/right_arm_gripper/meshes/right_rail_visual.stl
- added link rail_4, mass 0.01189999999999999912; visual mesh filename=../assemblies/right_arm_gripper/meshes/right_rail_2_visual.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
- added link right_rail_guide, mass 0.030111386261699939898; visual mesh filename=../assemblies/right_arm_gripper/meshes/right_rail_guide_vis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
- added link spur_gear_(14_teeth), mass 0.0013000000000000001572; visual mesh filename=../assemblies/left_arm_gripper/meshes/left_spur_gear_(14_te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
- added link spur_gear_(14_teeth)_2, mass 0.0013000000000000001572; visual mesh filename=../assemblies/right_arm_gripper/meshes/right_spur_gear_(14_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
- added link xc330, mass 0.026599999993091760775; visual mesh filename=../assemblies/left_arm_gripper/meshes/left_xc330_visual.stl
- added link xc330_2, mass 0.026599999993091760775; visual mesh filename=../assemblies/right_arm_gripper/meshes/right_xc330_visual.s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
- link 2xl430_gears: mass 0.11800003674524907338 -> 0.11800003674524908726; geometry visual mesh filename=../assemblies/left_arm_gripper/meshes/left_2xl430_gears_vis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
- link 2xl430_gears_2: mass 0.11800003674524907338 -> 0.11800003674524908726; geometry visual mesh filename=../assemblies/left_arm_gripper/meshes/left_2xl430_gears_2_v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
- link 2xl430_gears_3: mass 0.11800003674524907338 -> 0.11800003674524908726; geometry visual mesh filename=../assemblies/left_arm_gripper/meshes/left_2xl430_gears_3_v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
- link 2xl430_gears_4: mass 0.11800003674524907338 -> 0.11800003674524908726; geometry visual mesh filename=../assemblies/right_arm_gripper/meshes/right_2xl430_gears_v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
- link 2xl430_gears_5: mass 0.11800003674524907338 -> 0.11800003674524908726; geometry visual mesh filename=../assemblies/right_arm_gripper/meshes/right_2xl430_gears_2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
- link 2xl430_gears_6: mass 0.11800003674524907338 -> 0.11800003674524908726; geometry visual mesh filename=../assemblies/right_arm_gripper/meshes/right_2xl430_gears_3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
- link elb_yaw_link: mass 0.017500000000000001665 -> 0.017500000000000012074; geometry visual mesh filename=../assemblies/left_arm_gripper/meshes/left_elb_yaw_link_vis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
- link elb_yaw_link_2: mass 0.017500000000000001665 -> 0.017500000000000012074; geometry visual mesh filename=../assemblies/right_arm_gripper/meshes/right_elb_yaw_link_v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
- link sho_pitch_link: mass 0.0086000000000000000056 -> 0.0085999999999999948014; geometry visual mesh filename=../assemblies/left_arm_gripper/meshes/left_sho_pitch_link_v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
- link sho_pitch_link_2: mass 0.0086000000000000000056 -> 0.0085999999999999948014; geometry visual mesh filename=../assemblies/right_arm_gripper/meshes/right_sho_pitch_link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
- link sho_yaw_link: mass 0.014500000000000019817 -> 0.014500000000000009409; geometry visual mesh filename=../assemblies/left_arm_gripper/meshes/left_sho_yaw_link_vis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
- link sho_yaw_link_2: mass 0.014500000000000019817 -> 0.014500000000000009409; geometry visual mesh filename=../assemblies/right_arm_gripper/meshes/right_sho_yaw_link_v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
- link spur_1m_24t_drive: geometry visual mesh filename=../assemblies/left_arm_gripper/meshes/left_spur_1m_24t_driv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
- link spur_1m_24t_drive_2: geometry visual mesh filename=../assemblies/left_arm_gripper/meshes/left_spur_1m_24t_driv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
- link spur_1m_24t_drive_3: geometry visual mesh filename=../assemblies/left_arm_gripper/meshes/left_spur_1m_24t_driv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
- link spur_1m_24t_drive_4: geometry visual mesh filename=../assemblies/right_arm_gripper/meshes/right_spur_1m_24t_dr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
- link spur_1m_24t_drive_5: geometry visual mesh filename=../assemblies/right_arm_gripper/meshes/right_spur_1m_24t_dr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
- link spur_1m_24t_drive_6: geometry visual mesh filename=../assemblies/right_arm_gripper/meshes/right_spur_1m_24t_dr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
- link spur_1m_24t_driven: mass 0.0027000000000000001429 -> 0.0026999999999999997093; geometry visual mesh filename=../assemblies/left_arm_gripper/meshes/left_spur_1m_24t_driv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
- link spur_1m_24t_driven_2: mass 0.0027000000000000001429 -> 0.0026999999999999997093; geometry visual mesh filename=../assemblies/left_arm_gripper/meshes/left_spur_1m_24t_driv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
- link spur_1m_24t_driven_3: mass 0.0027000000000000001429 -> 0.0026999999999999997093; geometry visual mesh filename=../assemblies/left_arm_gripper/meshes/left_spur_1m_24t_driv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
- link spur_1m_24t_driven_4: mass 0.0027000000000000001429 -> 0.0026999999999999997093; geometry visual mesh filename=../assemblies/right_arm_gripper/meshes/right_spur_1m_24t_dr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
- link spur_1m_24t_driven_5: mass 0.0027000000000000001429 -> 0.0026999999999999997093; geometry visual mesh filename=../assemblies/right_arm_gripper/meshes/right_spur_1m_24t_dr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
- link spur_1m_24t_driven_6: mass 0.0027000000000000001429 -> 0.0026999999999999997093; geometry visual mesh filename=../assemblies/right_arm_gripper/meshes/right_spur_1m_24t_dr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
- link wrist_bearing_plate: mass 0.0049000367468305539714 -> 0.0049000367468305548388; geometry visual mesh filename=../assemblies/left_arm_gripper/meshes/left_wrist_bearing_pl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
- link wrist_bearing_plate_2: mass 0.0049000367468305539714 -> 0.0049000367468305548388; geometry visual mesh filename=../assemblies/right_arm_gripper/meshes/right_wrist_bearing_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
Joints:
- removed joint left_wrist_pitch
- removed joint left_wrist_roll_drive
- removed joint left_wrist_roll_driven
- removed joint right_wrist_pitch
- removed joint right_wrist_roll_drive
- removed joint right_wrist_roll_driven
- added joint left_gripper_fixed: type fixed, parent gripper_connector, child left_rail_guide, origin xyz=3.4694469519536141888e-18 0.037000000000000005107 0.036000000000000004219 rpy=1.5707963267948954478 1.570796326794896558 0, axis 0 0 1, limit effort=1 velocity=20
- added joint left_gripper_motor: type fixed, parent left_rail_guide, child xc330, origin xyz=-0.021950000000000007699 0.022600000000000002032 0.023299999999999987388 rpy=7.2164496600760899834e-16 -8.5692192681739838362e-31 9.3430423746336819555e-31, axis 0 0 1, limit effort=1 velocity=20
- added joint left_gripper_pinion_1: type prismatic, parent left_rail_guide, child rail, origin xyz=-0.028872599999999967041 -0.014174999999999993161 -0.0053500000000000214051 rpy=3.141592653589793116 1.5707963267948954478 0, axis 0 0 1, limit lower=-0.036872599999999998432 upper=0 effort=1 velocity=20
- added joint left_gripper_pinion_2: type prismatic, parent left_rail_guide, child rail_2, origin xyz=0.062872600000000083975 0.014174999999999993161 -0.0053499999999999936495 rpy=-1.1102230241485031157e-16 1.5707963267948956698 0, axis 0 0 1, limit lower=-0.036872599999999998432 upper=0 effort=1 velocity=20
- added joint left_gripper_rack: type revolute, parent xc330, child spur_gear_(14_teeth), origin xyz=0.0079999999999998683275 -0.022500000000001255107 -0.020000000000000905942 rpy=6.855915668332168754e-16 -2.3037346225485797513e-16 -3.7700408238277826924e-17, axis 0 0 1, limit lower=0 upper=5.2359877559829888227 effort=1 velocity=20
- added joint left_wrist_pitch_drive: type revolute, parent 2xl430_gears_3, child spur_1m_24t_drive_3, origin xyz=-1.5244182510102145428e-10 0.024000000358063572348 -0.0080000000000052026022 rpy=3.8158623046065463386e-14 2.7687786355305660007e-15 -1.5707963267948872321, axis 0 0 1, limit lower=-1.570796326794896558 upper=1.570796326794896558 effort=1 velocity=20
- added joint left_wrist_pitch_driven: type revolute, parent spur_1m_24t_driven_3, child 2xl430_gears_3, origin xyz=-2.7755575615628913511e-17 0 -0.0015999999999999972577 rpy=2.4980018055243628788e-16 -1.6081226490223879062e-16 -1.570796326794896558, axis 0 0 1, limit lower=-1.570796326794896558 upper=1.570796326794896558 effort=1 velocity=20
- added joint left_wrist_roll: type revolute, parent 2xl430_gears_3, child gripper_connector, origin xyz=0.019000000000008565593 -3.5807690146327786351e-10 -0.027000000152451481689 rpy=3.1415926535897225058 1.5707963267948779063 0, axis 0 0 1, limit lower=-1.570796326794896558 upper=1.570796326794896558 effort=1 velocity=20
- added joint right_gripper_fixed: type fixed, parent gripper_connector_2, child right_rail_guide, origin xyz=3.4694469519536141888e-18 0.037000000000000005107 -0.001999999999999991368 rpy=1.5707963267949094366 1.5707963267948832353 0, axis 0 0 1, limit effort=1 velocity=20
- added joint right_gripper_motor: type fixed, parent right_rail_guide, child xc330_2, origin xyz=-0.0059500000000000038969 -0.022599999999999981215 0.023300000000000042899 rpy=-1.4352268952473380085e-25 1.0940480200944162675e-30 3.141592653589793116, axis 0 0 1, limit effort=1 velocity=20
- added joint right_gripper_pinion_1: type prismatic, parent right_rail_guide, child rail_3, origin xyz=-0.028872599999999963571 -0.014174999999999993161 -0.0053499999999999381384 rpy=3.141592653589793116 1.5707963267948958919 0, axis 0 0 1, limit lower=-0.036872599999999998432 upper=0 effort=1 velocity=20
- added joint right_gripper_pinion_2: type prismatic, parent right_rail_guide, child rail_4, origin xyz=0.062872600000000000708 0.0141750000000000001 -0.0053499999999999381384 rpy=-1.1235956670197897365e-25 1.5707963267948958919 0, axis 0 0 1, limit lower=-0.036872599999999998432 upper=0 effort=1 velocity=20
- added joint right_gripper_rack: type revolute, parent xc330_2, child spur_gear_(14_teeth)_2, origin xyz=0.0079999999999993375022 -0.022499999999995499295 -0.019999999999999656941 rpy=3.9513898910780635647e-26 -6.1232339957375240819e-17 -4.4058789844277850015e-17, axis 0 0 1, limit lower=0 upper=5.2359877559829888227 effort=1 velocity=20
- added joint right_wrist_pitch_drive: type revolute, parent 2xl430_gears_6, child spur_1m_24t_drive_6, origin xyz=-1.5244730108012700873e-10 0.024000000358075063156 -0.0080000000000021147945 rpy=-2.3760361364596328788e-14 9.1171344708605480535e-14 -1.5707963267948272801, axis 0 0 1, limit lower=-1.3962634015954635824 upper=1.9198621771937625091 effort=1 velocity=20
- added joint right_wrist_pitch_driven: type revolute, parent spur_1m_24t_driven_6, child 2xl430_gears_6, origin xyz=2.7755575615628913511e-17 -6.3108872417680944433e-30 -0.0015999999999999966072 rpy=-1.5154544286135535634e-14 1.7943243846840832321e-15 1.570796326794896558, axis 0 0 1, limit lower=-1.9198621771937625091 upper=1.3962634015954635824 effort=1 velocity=20
- added joint right_wrist_roll: type revolute, parent 2xl430_gears_6, child gripper_connector_2, origin xyz=0.019000000000003156725 -3.5806391185388974918e-10 -0.027000000152454312757 rpy=-3.141592653589708739 -1.5707963267948066299 0, axis 0 0 1, limit lower=-1.3962634015954635824 upper=1.9198621771937625091 effort=1 velocity=20
- joint left_elbow_roll: origin xyz=2.185751579730776939e-16 -0.018999999999999329925 -0.058999999999999733213 rpy=1.570796326794896558 -1.3443939455351824662e-14 1.2212453270787430779e-15 -> xyz=0 -0.019000000000000002998 -0.058999999999999989952 rpy=1.570796326794896558 -5.9921797729386389252e-15 -1.6081226496441365173e-16
- joint left_elbow_yaw_drive: origin xyz=-0.024000000716141011575 -0.019000000152448556778 -0.019000000152448452695 rpy=1.5707963267949249797 5.3833632274240703492e-15 -6.2781152873576405876e-14 -> xyz=-0.024000000716136535989 -0.019000000152454787905 -0.019000000152441284818 rpy=1.5707963267946079 -2.8216931162767297778e-14 6.7112934369983557895e-14
- joint left_elbow_yaw_driven: origin xyz=-3.5806929990500613314e-10 -0.027000000152451131274 -0.019000000000003351014 rpy=1.5707963267949591746 1.5707963267948683583 0 -> xyz=-3.5806391879278365309e-10 -0.027000000152454087243 -0.01899999999999553088 rpy=1.5707963267946445374 -1.957357187373244284e-14 -5.6726675369617376296e-14
- joint left_elbow_yaw_fixed: origin xyz=7.8886090522101180541e-31 3.4694469519536141888e-18 0.0015999999999999625633 rpy=3.141592653589793116 6.123233994422830684e-17 -1.57079632679489678 -> xyz=0 6.3108872417680944433e-30 0.0015999999999999903189 rpy=3.1415926535897926719 3.0894028578356351099e-29 -1.570796326794896558
- joint left_sho_roll: origin xyz=-0.018999999999999947486 0.0010000000000000076102 0.027000000000000003164 rpy=-3.141592653589793116 1.570796326794896558 0 -> xyz=-0.018999999999999937078 0.00099999999999997031368 0.02699999999999990602 rpy=3.1415926535897913396 1.5707963267948676922 0
- joint left_sho_yaw_drive: origin xyz=-0.024000000716141278723 -0.019000000152448490859 -0.0190000001524472939 rpy=1.570796326794886566 -1.7772407460995643501e-15 2.9721983312145830671e-14 -> xyz=-0.024000000716142340373 -0.019000000152452619501 -0.019000000152446860219 rpy=1.5707963267949109909 9.9706267968386760623e-14 1.1369019472068143296e-13
- joint left_sho_yaw_driven: origin xyz=-3.5807098258677783065e-10 -0.027000000152450111257 -0.019000000000003021416 rpy=1.5707963267949009989 2.5840015203544507292e-14 -4.9507333169721578628e-15 -> xyz=-3.5806818968198150799e-10 -0.027000000152451984758 -0.01900000000000318795 rpy=1.5707963267948918951 5.5868781814391237904e-14 7.1004483613505400622e-14
- joint left_sho_yaw_fixed: origin xyz=1.7347234759768070944e-17 -1.6375789611241112762e-17 0.0015999999999999972577 rpy=-3.1415926535897926719 2.775557561593911827e-16 4.4408920984097454411e-16 -> xyz=0 0 0.0016000000000000007272 rpy=-3.141592653589793116 4.050196108650232498e-16 6.2450045046961790355e-17
- joint left_wrist_pitch_fixed: origin xyz=0.015500000000005269979 -1.7125190154843039636e-14 -0.04500000000000015099 rpy=-4.057865155005087888e-14 -2.9093394360302217044e-13 -1.5707963267949061059 -> xyz=0.01550000000000705154 -7.0499162063697440317e-15 -0.045000000000003488598 rpy=2.3314683517158803644e-14 -2.7339241981393896051e-14 -1.5707963267949085484
- joint left_wrist_roll_fixed: origin xyz=-3.4694469519536141888e-18 -0.025300000000000003042 -0.051999999999999976796 rpy=1.570796326794896558 -1.570796326794896558 0 -> xyz=-6.3108872417680944433e-30 -0.025299999999999996103 -0.051999999999999976796 rpy=1.570796326794896558 -1.5707963267948958919 0
- joint right_elbow_roll: origin xyz=-2.2898349882893853646e-16 -0.019000000000000173001 -0.058999999999999837297 rpy=1.57079632679489678 -1.1224323958578838097e-14 -5.9062164171655744588e-15 -> xyz=-5.2041704279304212832e-17 -0.018999999999999964834 -0.059000000000000114853 rpy=1.5707963267948974462 5.0352015639126703846e-15 2.5592341453658362349e-15
- joint right_elbow_yaw_drive: origin xyz=-0.024000000716145233892 -0.019000000152448695556 -0.019000000152448716373 rpy=1.5707963267950251218 -1.5597582698688193762e-15 -8.7866473173388565758e-14 -> xyz=-0.024000000716145945129 -0.019000000152452470314 -0.019000000152448241059 rpy=1.5707963267948983344 1.6899208920332882627e-13 -6.1373298874875490715e-14
- joint right_elbow_yaw_driven: limit lower=-1.570796326794896558 upper=1.570796326794896558 effort=1 velocity=20 -> lower=-2.6179938779914944114 upper=2.6179938779914944114 effort=1 velocity=20; origin xyz=-3.5807111442576200488e-10 -0.027000000152451464341 -0.019000000000003632039 rpy=1.570796326794921427 1.0192981807050532901e-13 -4.32129208184743122e-14 -> xyz=-3.5806995563048005238e-10 -0.0270000001524559885 -0.01900000000000036729 rpy=1.5707963267948485964 8.4311697099246135987e-14 3.6920636757530582299e-14
- joint right_elbow_yaw_fixed: origin xyz=-3.4694469519536141888e-18 -1.5777218104420236108e-30 0.0015999999999999764411 rpy=-3.1415926535897891192 -8.3149610451184695905e-31 2.7073084493379207714e-30 -> xyz=0 3.1554436208840472216e-30 0.0016000000000000180744 rpy=-3.1415926535897873428 3.3907091715322312159e-31 -1.570796326794896558
- joint right_sho_roll: origin xyz=-0.01899999999999998565 0.0010000000000000112965 0.027000000000000013572 rpy=3.141592653589793116 1.570796326794896558 0 -> xyz=-0.01899999999999992667 0.0010000000000000069597 0.026999999999999999695 rpy=3.1415926535897922278 1.5707963267948588104 0
- joint right_sho_yaw_drive: origin xyz=-0.024000000716138513573 -0.019000000152446919199 -0.019000000152449438018 rpy=1.5707963267949425212 -7.4825707768639476445e-14 5.2729872485629252068e-14 -> xyz=-0.024000000716137483148 -0.019000000152449965374 -0.019000000152444667528 rpy=1.570796326794722475 -4.3999245160326114002e-14 5.9488666369146786408e-14
- joint right_sho_yaw_driven: origin xyz=-3.5806675333094339919e-10 -0.027000000152447987956 -0.019000000000004509809 rpy=1.5707963267949396347 -3.4289578266172945506e-14 -6.6930782579143983011e-15 -> xyz=-3.5806750273148502117e-10 -0.027000000152448928176 -0.018999999999998070516 rpy=1.5707963267947655517 -4.3564811365927410262e-14 2.9648675946254039113e-14
- joint right_sho_yaw_fixed: origin xyz=3.4694469519536141888e-18 0 0.0016000000000000076661 rpy=-3.1415926535897917837 7.3983136435179850071e-16 1.4710455076273652726e-15 -> xyz=5.2041704279304212832e-17 3.787910703300854279e-17 0.0015999999999998966438 rpy=3.141592653589793116 1.6554645777787879748e-29 8.3603448337486833053e-32
- joint right_wrist_pitch_fixed: origin xyz=0.015500000000003956793 4.5519144009631418157e-15 -0.045000000000003870237 rpy=-3.552713678787178252e-15 1.2051470932306258524e-13 -1.570796326794896558 -> xyz=0.01550000000000218911 9.9364960703951510368e-15 -0.045000000000006000478 rpy=-1.2645101217445535558e-15 1.2057022047428705255e-13 -1.5707963267947835373
- joint right_wrist_roll_fixed: origin xyz=3.4694469519536141888e-18 -0.025299999999999996103 -0.051999999999999990674 rpy=1.5707963267949205388 1.570796326794896558 0 -> xyz=0 -0.025299999999999999573 -0.051999999999999990674 rpy=1.570796326794896558 1.570796326794896558 0

Commit message: Update the gripper pinions

File: toddlerbot/robot_descriptions/toddlerbot/toddlerbot.urdf (robot description, URDF)
Before this commit: robot toddlerbot, 85 links, 84 joints
Links:
- link gripper_connector: mass 0.0099999999999999984734 -> 0.0099999999999999915345
- link gripper_connector_2: mass 0.009999999999999995004 -> 0.0099999999999999915345
- link left_rail_guide: mass 0.032142035224833380436 -> 0.032142035224833366558
- link rail_3: mass 0.011899999999999995651 -> 0.011900000000000000855
- link rail_4: mass 0.011899999999999995651 -> 0.011900000000000000855
- link right_rail_guide: mass 0.030111386261699936429 -> 0.030111386261699946837
- link sho_pitch_link: mass 0.0086000000000000017403 -> 0.0086000000000000000056
- link sho_pitch_link_2: mass 0.0086000000000000017403 -> 0.0086000000000000000056
- link sho_yaw_link: mass 0.014500000000000007674 -> 0.014500000000000016348
- link sho_yaw_link_2: mass 0.01450000000000000247 -> 0.014500000000000016348
- link spur_1m_24t_driven: mass 0.0027000000000000001429 -> 0.0026999999999999997093
- link spur_1m_24t_driven_2: mass 0.0027000000000000001429 -> 0.0026999999999999997093
- link spur_1m_24t_driven_3: mass 0.0027000000000000001429 -> 0.0026999999999999997093
- link spur_1m_24t_driven_4: mass 0.0026999999999999988419 -> 0.0026999999999999997093
- link spur_1m_24t_driven_5: mass 0.0026999999999999988419 -> 0.0026999999999999997093
- link spur_1m_24t_driven_6: mass 0.0026999999999999988419 -> 0.0026999999999999997093
- link spur_gear_(14_teeth)_2: mass 0.0012999999999999997235 -> 0.0012999999999999999403
- link wrist_bearing_plate_2: mass 0.0049000367468305539714 -> 0.0049000367468305548388
Joints:
- removed joint left_gripper_pinion_1
- removed joint left_gripper_pinion_2
- removed joint right_gripper_pinion_1
- removed joint right_gripper_pinion_2
- added joint left_gripper_pinion: type prismatic, parent left_rail_guide, child rail, origin xyz=-0.028872599999999620096 -0.014175000000000003569 -0.0053500000000002712053 rpy=3.141592653589793116 1.5707963267948952257 0, axis 0 0 1, limit lower=-0.036872599999999998432 upper=0 effort=1 velocity=20
- added joint left_gripper_pinion_mirror: type prismatic, parent left_rail_guide, child rail_2, origin xyz=0.062872600000000888887 0.014174999999999993161 -0.0053500000000002434497 rpy=-1.1034025256268857111e-29 1.5707963267948952257 0, axis 0 0 1, limit lower=-0.036872599999999998432 upper=0 effort=1 velocity=20
- added joint right_gripper_pinion: type prismatic, parent right_rail_guide, child rail_3, origin xyz=-0.028872600000001191756 -0.014174999999999993161 -0.005350000000001076117 rpy=-3.141592653589793116 1.5707963267948954478 0, axis 0 0 1, limit lower=-0.036872599999999998432 upper=0 effort=1 velocity=20
- added joint right_gripper_pinion_mirror: type prismatic, parent right_rail_guide, child rail_4, origin xyz=0.062872599999998834974 0.01417499999999999663 -0.0053500000000010206058 rpy=9.1593399531549520226e-16 1.5707963267948945596 0, axis 0 0 1, limit lower=-0.036872599999999998432 upper=0 effort=1 velocity=20
