Commit message: Fix toddlerbot_OP3 and pass the stand_open test

File: toddlerbot/robot_descriptions/toddlerbot_OP3/toddlerbot_OP3.urdf (robot description, URDF)
Before this commit: robot toddlerbot_OP3, 73 links, 72 joints
Links:
- link ank_roll_link: mass 0.042600000000000005917 -> 0.042600000000000012856; geometry collision box size=0.04900000058114529 0.041999999433755875 0.12000000104308128; visual mesh filename=../assemblies/left_leg_OP3/meshes/left_ank_roll_link_visual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
- link ank_roll_link_2: mass 0.042600000000000005917 -> 0.042600000000000012856; geometry collision box size=0.04900000058114529 0.041999999433755875 0.12000000104308128; visual mesh filename=../assemblies/right_leg_OP3/meshes/right_ank_roll_link_visu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
- link left_calf_link: mass 0.030999999999999999778 -> 0.031000000000000003247
- link right_calf_link: mass 0.03099999999999998937 -> 0.0309999999999999859
Joints:
- joint right_knee_front_rev_1: origin xyz=-0.0057402514854764941088 -0.013858192987669354368 -0.004999999999999997502 rpy=2.2689194189171478947e-15 -6.1057528575718748365e-15 1.5678717655286378285 -> xyz=-0.0057402514854764941088 -0.013858192987669354368 -0.004999999999999997502 rpy=2.2689194189169072921e-15 -9.1667614776401742833e-15 1.5678717655286389387
