Commit message: Fix toddlerbot_OP3 and pass the stand_open test

File: toddlerbot/robot_descriptions/assemblies/left_leg_OP3/left_leg_OP3.urdf (robot description, URDF)
Before this commit: robot left_leg_OP3, 11 links, 10 joints
Links:
- link ank_roll_link: mass 0.042600000000000005917 -> 0.042600000000000012856
- link left_calf_link: mass 0.030999999999999999778 -> 0.031000000000000003247

File: toddlerbot/robot_descriptions/assemblies/right_leg_OP3/right_leg_OP3.urdf (robot description, URDF)
Before this commit: robot right_leg_OP3, 11 links, 10 joints
Links:
- link ank_roll_link: mass 0.042600000000000005917 -> 0.042600000000000012856
- link right_calf_link: mass 0.03099999999999998937 -> 0.0309999999999999859
Joints:
- joint right_knee_front_rev_1: origin xyz=-0.0057402514854764941088 -0.013858192987669354368 -0.004999999999999997502 rpy=2.2689194189171478947e-15 -6.1057528575718748365e-15 1.5678717655286378285 -> xyz=-0.0057402514854764941088 -0.013858192987669354368 -0.004999999999999997502 rpy=2.2689194189169072921e-15 -9.1667614776401742833e-15 1.5678717655286389387

Commit message: Fix toddlerbot_OP3 RL training

File: toddlerbot/robot_descriptions/assemblies/left_leg_OP3/left_leg_OP3.urdf (robot description, URDF)
Before this commit: robot left_leg_OP3, 11 links, 10 joints
Links:
- link ank_pitch_link: mass 0.15976376693924945749 -> 0.15976376693924948524
- link ank_roll_link: mass 0.042600000000000012856 -> 0.042599999999999998979
- link bearing_683: mass 0.00048694686130641804279 -> 0.00048694686130641793437
- link bearing_683_2: mass 0.00048694686130641804279 -> 0.00048694686130641793437
- link hip_roll_link: mass 0.11059999999836231388 -> 0.11059999999836234164
- link hip_yaw_link: mass 0.017999999999999991701 -> 0.01799999999999999864
- link knee_rod: mass 0.0031629468613064179276 -> 0.0031629468613064183613
- link knee_rod_2: mass 0.0031629468613064179276 -> 0.0031629468613064183613
- link left_calf_link: mass 0.031000000000000003247 -> 0.030999999999999999778
- link left_hip_pitch_link_xm430: mass 0.11480090135030571186 -> 0.1148009013503056841
Joints:
- joint left_ank_pitch: origin xyz=0.00049999999999989310807 -0.099999999999999977796 -0.029400000000000373751 rpy=-3.141592653589793116 5.1278425949876957843e-15 -1.5707963267948956698 -> xyz=0.00050000000000004402902 -0.099999999999997202238 -0.029400000000001407646 rpy=-2.1321242293024632049e-15 1.8823484437772641304e-14 -1.5707963267948981123
- joint left_ank_roll: origin xyz=-4.9960036108132044319e-16 -0.022750000000003208628 -0.019000000000006171674 rpy=-1.5707963267948434893 -1.0354577980633209865e-13 -3.141592653589788231 -> xyz=-7.771561172376095783e-16 0.022750000000003930273 0.019000000000007229856 rpy=1.5707963267949729413 8.7734350778775080161e-14 3.1415926535897842342
- joint left_hip_pitch: origin xyz=-0.02400000071615559713 -0.019000000152441166856 -0.019000000152458167146 rpy=1.5707963267953672926 1.5707963267945022068 0 -> xyz=-0.024000000716156176528 -0.019000000152439990714 -0.019000000152458156738 rpy=1.5707963267953688469 1.5707963267944595742 0
- joint left_hip_roll: origin xyz=0.019000000000000002998 -3.3408590380431292134e-18 -0.025999999999999998807 rpy=3.141592653589793116 -1.5707963267948943376 0 -> xyz=0.018999999999999434008 3.7043493321931432202e-16 -0.026000000000000141054 rpy=-3.141592653589793116 -1.5707963267948932273 0
- joint left_knee_act: origin xyz=-0.00014999999999966212236 -0.061500000000000276668 -0.030400000000000156064 rpy=-1.2184487414508649095e-14 1.1572329706963895349e-14 1.5707963267948876762 -> xyz=-0.00015000000000014844124 -0.06150000000000001299 -0.030399999999999711975 rpy=-1.0766672541727743252e-14 1.3282815320613851332e-14 1.5707963267949027752
- joint left_knee_back_rev_1: origin xyz=-0.013858192987669284979 -0.0057402514854763379837 -0.0050000000000000321965 rpy=-1.7902130110758088672e-15 1.2957208404619350222e-14 -3.1386940726547267744 -> xyz=-0.013858192987669284979 -0.0057402514854763466573 -0.0050000000000000027062 rpy=-1.7626513399117519762e-14 2.0655748330454469805e-14 -3.1386940726547454261
- joint left_knee_back_rev_2: origin xyz=0.0057402514854762824725 -0.013858192987669576413 -0.026200000000000028821 rpy=-6.5544379830050492951e-15 -5.7215737298236230488e-15 1.5736949077299540178 -> xyz=0.0057402514854756501658 -0.013858192987669437635 -0.026199999999999720041 rpy=4.9560921740722585935e-15 -2.1168138603303528903e-14 1.5736949077299444699
- joint left_knee_front_rev_1: origin xyz=0.013858192987669298857 0.0057402514854763683413 -0.004999999999999966277 rpy=6.8152281266059555871e-15 1.7362503496778251608e-15 -3.1357955927274376862 -> xyz=0.013858192987669312735 0.0057402514854763449226 -0.0049999999999999992367 rpy=2.3955576787343955856e-15 2.4557124758423299065e-14 -3.1357955927274510088
- joint left_knee_front_rev_2: origin xyz=-0.005740251485476489772 0.01385819298766921559 -0.026199999999999820655 rpy=-8.9608725300154706869e-15 4.6129922847757146423e-15 1.5765933876572442163 -> xyz=-0.0057402514854767707972 0.013858192987668854768 -0.026199999999999168399 rpy=9.6260126850146175027e-15 -2.5081324750790058604e-14 1.5765933876572388872
- joint left_knee_pitch: origin xyz=1.549471946950906618e-16 -0.095999999999999932609 -0.009200000000000154235 rpy=-4.3715031594638534075e-15 -1.6535574677587582148e-16 3.720971275579667282e-17 -> xyz=2.6591951153791853136e-17 -0.096000000000000029754 -0.0091999999999999634154 rpy=-1.3783391157486681965e-14 -1.4843341659320182562e-14 4.5251917072955735634e-15

File: toddlerbot/robot_descriptions/assemblies/right_leg_OP3/right_leg_OP3.urdf (robot description, URDF)
Before this commit: robot right_leg_OP3, 11 links, 10 joints
Links:
- link ank_pitch_link: mass 0.15976376693924945749 -> 0.15976376693924948524
- link ank_roll_link: mass 0.042600000000000012856 -> 0.042599999999999998979
- link bearing_683: mass 0.00048694686130641804279 -> 0.00048694686130641793437
- link bearing_683_2: mass 0.00048694686130641804279 -> 0.00048694686130641793437
- link hip_roll_link: mass 0.11059999999836231388 -> 0.11059999999836234164
- link hip_yaw_link: mass 0.017999999999999991701 -> 0.01799999999999999864
- link knee_rod: mass 0.0031629468613064179276 -> 0.0031629468613064183613
- link knee_rod_2: mass 0.0031629468613064179276 -> 0.0031629468613064183613
- link right_calf_link: mass 0.0309999999999999859 -> 0.03099999999999998937
- link right_hip_pitch_link_xm430: mass 0.11480090135030571186 -> 0.11480090135030567022
Joints:
- joint right_ank_pitch: origin xyz=0.00050000000000010062437 0.099999999999999977796 0.0086000000000000208222 rpy=-7.4480623481441756806e-16 -2.1451753131548428425e-15 1.5707963267948934494 -> xyz=0.00049999999999975335441 0.099999999999999561462 0.0086000000000000676598 rpy=3.1415926535897877869 -1.4928027344634987948e-14 1.5707963267948785724
- joint right_ank_roll: origin xyz=-2.498001805406602216e-16 -0.022750000000001085326 -0.019000000000002174871 rpy=-1.5707963267948694686 1.175774048742249633e-14 -3.1415926535897815697 -> xyz=-2.2204460492503130808e-16 0.02275000000000106104 0.019000000000002178341 rpy=1.5707963267949220931 -3.6775852931107809278e-14 3.1415926535897313876
- joint right_hip_pitch: origin xyz=-0.02400000071614311753 -0.019000000152445541829 -0.019000000152453264818 rpy=1.5707963267950966202 1.5707963267947309127 0 -> xyz=-0.024000000716143346513 -0.019000000152445729179 -0.019000000152453181551 rpy=1.5707963267950966202 1.5707963267947326891 0
- joint right_hip_roll: origin xyz=-0.018999999999999968303 3.4814450885713959653e-18 -0.025999999999999967581 rpy=7.693748353958839089e-20 -1.5707963267948961139 0 -> xyz=-0.018999999999999916261 3.1092928099478391072e-16 -0.025999999999999925948 rpy=3.0774993384580180772e-19 -1.5707963267948932273 0
- joint right_knee_act: origin xyz=0.00014999999999998502487 -0.061499999999999561962 -0.030400000000000208106 rpy=-1.3157660724820988502e-14 2.289083756447533756e-16 3.1415926535897464866 -> xyz=0.00014999999999996659343 -0.061499999999998652966 -0.030399999999999018085 rpy=-3.9472982174462490613e-14 8.7088539502980777788e-16 3.141592653589793116
- joint right_knee_back_rev_1: origin xyz=0.0057402514854763501267 0.013858192987669271101 -0.0050000000000000148492 rpy=-3.1552336572096932e-15 -3.3270436898146921635e-14 1.5677951037379203036 -> xyz=0.0057402514854763535962 0.013858192987669271101 -0.0050000000000000061756 rpy=-1.919569185352210123e-15 -1.6455897748865722783e-15 1.5677951037378847765
- joint right_knee_back_rev_2: origin xyz=0.0057402514854764602817 0.01385819298766871599 -0.026199999999999792899 rpy=-2.1293173172291718105e-14 4.8029314978609855261e-14 3.1385914305327689 -> xyz=0.005740251485476185328 0.013858192987669409879 -0.026200000000000056577 rpy=-6.2585939741374333299e-15 -1.0479387378889103051e-16 3.1385914305327817786
- joint right_knee_front_rev_1: origin xyz=-0.0057402514854764941088 -0.013858192987669354368 -0.004999999999999997502 rpy=2.2689194189169072921e-15 -9.1667614776401742833e-15 1.5678717655286389387 -> xyz=-0.0057402514854763501267 -0.013858192987669284979 -0.0049999999999999957673 rpy=-5.0313204613631514412e-15 -1.1212819345950018642e-16 1.5678717655286047439
- joint right_knee_front_rev_2: origin xyz=-0.0057402514854764750268 -0.013858192987669187834 -0.026200000000000837203 rpy=2.6700561543117312309e-15 -7.7788101235701736907e-15 3.1386680923234866469 -> xyz=-0.0057402514854764195157 -0.013858192987669049057 -0.026200000000000209233 rpy=-4.792276793618950313e-15 -7.4425542615262678023e-15 3.1386680923234981933
- joint right_knee_pitch: origin xyz=5.842070865544391856e-17 -0.095999999999999585665 -0.0092000000000001299488 rpy=-1.390597706429142792e-15 -1.7669519698394562425e-15 -3.1415926535897917837 -> xyz=-1.4425300025281195314e-16 -0.095999999999999197087 -0.009200000000000072703 rpy=-4.4507648457556451305e-14 -3.3964226209539856629e-15 3.1415926535897926719

File: toddlerbot/robot_descriptions/toddlerbot_OP3/toddlerbot_OP3.urdf (robot description, URDF)
Before this commit: robot toddlerbot_OP3, 73 links, 72 joints
Links:
- link ank_pitch_link: mass 0.15976376693924945749 -> 0.15976376693924948524
- link ank_pitch_link_2: mass 0.15976376693924945749 -> 0.15976376693924948524
- link ank_roll_link: mass 0.042600000000000012856 -> 0.042599999999999998979
- link ank_roll_link_2: mass 0.042600000000000012856 -> 0.042599999999999998979
- link bearing_683: mass 0.00048694686130641804279 -> 0.00048694686130641793437
- link bearing_683_2: mass 0.00048694686130641804279 -> 0.00048694686130641793437
- link bearing_683_3: mass 0.00048694686130641804279 -> 0.00048694686130641793437
- link bearing_683_4: mass 0.00048694686130641804279 -> 0.00048694686130641793437
- link hip_roll_link: mass 0.11059999999836231388 -> 0.11059999999836234164
- link hip_roll_link_2: mass 0.11059999999836231388 -> 0.11059999999836234164
- link hip_yaw_link: mass 0.017999999999999991701 -> 0.01799999999999999864
- link hip_yaw_link_2: mass 0.017999999999999991701 -> 0.01799999999999999864
- link knee_rod: mass 0.0031629468613064179276 -> 0.0031629468613064183613
- link knee_rod_2: mass 0.0031629468613064179276 -> 0.0031629468613064183613
- link knee_rod_3: mass 0.0031629468613064179276 -> 0.0031629468613064183613
- link knee_rod_4: mass 0.0031629468613064179276 -> 0.0031629468613064183613
- link left_calf_link: mass 0.031000000000000003247 -> 0.030999999999999999778
- link left_hip_pitch_link_xm430: mass 0.11480090135030571186 -> 0.1148009013503056841
- link right_calf_link: mass 0.0309999999999999859 -> 0.03099999999999998937
- link right_hip_pitch_link_xm430: mass 0.11480090135030571186 -> 0.11480090135030567022
Joints:
- joint left_ank_pitch: origin xyz=0.00049999999999989310807 -0.099999999999999977796 -0.029400000000000373751 rpy=-3.141592653589793116 5.1278425949876957843e-15 -1.5707963267948956698 -> xyz=0.00050000000000004402902 -0.099999999999997202238 -0.029400000000001407646 rpy=-2.1321242293024632049e-15 1.8823484437772641304e-14 -1.5707963267948981123
- joint left_ank_roll: origin xyz=-4.9960036108132044319e-16 -0.022750000000003208628 -0.019000000000006171674 rpy=-1.5707963267948434893 -1.0354577980633209865e-13 -3.141592653589788231 -> xyz=-7.771561172376095783e-16 0.022750000000003930273 0.019000000000007229856 rpy=1.5707963267949729413 8.7734350778775080161e-14 3.1415926535897842342
- joint left_hip_pitch: origin xyz=-0.02400000071615559713 -0.019000000152441166856 -0.019000000152458167146 rpy=1.5707963267953672926 1.5707963267945022068 0 -> xyz=-0.024000000716156176528 -0.019000000152439990714 -0.019000000152458156738 rpy=1.5707963267953688469 1.5707963267944595742 0
- joint left_hip_roll: origin xyz=0.019000000000000002998 -3.3408590380431292134e-18 -0.025999999999999998807 rpy=3.141592653589793116 -1.5707963267948943376 0 -> xyz=0.018999999999999434008 3.7043493321931432202e-16 -0.026000000000000141054 rpy=-3.141592653589793116 -1.5707963267948932273 0
- joint left_knee_act: origin xyz=-0.00014999999999966212236 -0.061500000000000276668 -0.030400000000000156064 rpy=-1.2184487414508649095e-14 1.1572329706963895349e-14 1.5707963267948876762 -> xyz=-0.00015000000000014844124 -0.06150000000000001299 -0.030399999999999711975 rpy=-1.0766672541727743252e-14 1.3282815320613851332e-14 1.5707963267949027752
- joint left_knee_back_rev_1: origin xyz=-0.013858192987669284979 -0.0057402514854763379837 -0.0050000000000000321965 rpy=-1.7902130110758088672e-15 1.2957208404619350222e-14 -3.1386940726547267744 -> xyz=-0.013858192987669284979 -0.0057402514854763466573 -0.0050000000000000027062 rpy=-1.7626513399117519762e-14 2.0655748330454469805e-14 -3.1386940726547454261
- joint left_knee_back_rev_2: origin xyz=0.0057402514854762824725 -0.013858192987669576413 -0.026200000000000028821 rpy=-6.5544379830050492951e-15 -5.7215737298236230488e-15 1.5736949077299540178 -> xyz=0.0057402514854756501658 -0.013858192987669437635 -0.026199999999999720041 rpy=4.9560921740722585935e-15 -2.1168138603303528903e-14 1.5736949077299444699
- joint left_knee_front_rev_1: origin xyz=0.013858192987669298857 0.0057402514854763683413 -0.004999999999999966277 rpy=6.8152281266059555871e-15 1.7362503496778251608e-15 -3.1357955927274376862 -> xyz=0.013858192987669312735 0.0057402514854763449226 -0.0049999999999999992367 rpy=2.3955576787343955856e-15 2.4557124758423299065e-14 -3.1357955927274510088
- joint left_knee_front_rev_2: origin xyz=-0.005740251485476489772 0.01385819298766921559 -0.026199999999999820655 rpy=-8.9608725300154706869e-15 4.6129922847757146423e-15 1.5765933876572442163 -> xyz=-0.0057402514854767707972 0.013858192987668854768 -0.026199999999999168399 rpy=9.6260126850146175027e-15 -2.5081324750790058604e-14 1.5765933876572388872
- joint left_knee_pitch: origin xyz=1.549471946950906618e-16 -0.095999999999999932609 -0.009200000000000154235 rpy=-4.3715031594638534075e-15 -1.6535574677587582148e-16 3.720971275579667282e-17 -> xyz=2.6591951153791853136e-17 -0.096000000000000029754 -0.0091999999999999634154 rpy=-1.3783391157486681965e-14 -1.4843341659320182562e-14 4.5251917072955735634e-15
- joint right_ank_pitch: origin xyz=0.00050000000000010062437 0.099999999999999977796 0.0086000000000000208222 rpy=-7.4480623481441756806e-16 -2.1451753131548428425e-15 1.5707963267948934494 -> xyz=0.00049999999999975335441 0.099999999999999561462 0.0086000000000000676598 rpy=3.1415926535897877869 -1.4928027344634987948e-14 1.5707963267948785724
- joint right_ank_roll: origin xyz=-2.498001805406602216e-16 -0.022750000000001085326 -0.019000000000002174871 rpy=-1.5707963267948694686 1.175774048742249633e-14 -3.1415926535897815697 -> xyz=-2.2204460492503130808e-16 0.02275000000000106104 0.019000000000002178341 rpy=1.5707963267949220931 -3.6775852931107809278e-14 3.1415926535897313876
- joint right_hip_pitch: origin xyz=-0.02400000071614311753 -0.019000000152445541829 -0.019000000152453264818 rpy=1.5707963267950966202 1.5707963267947309127 0 -> xyz=-0.024000000716143346513 -0.019000000152445729179 -0.019000000152453181551 rpy=1.5707963267950966202 1.5707963267947326891 0
- joint right_hip_roll: origin xyz=-0.018999999999999968303 3.4814450885713959653e-18 -0.025999999999999967581 rpy=7.693748353958839089e-20 -1.5707963267948961139 0 -> xyz=-0.018999999999999916261 3.1092928099478391072e-16 -0.025999999999999925948 rpy=3.0774993384580180772e-19 -1.5707963267948932273 0
- joint right_knee_act: origin xyz=0.00014999999999998502487 -0.061499999999999561962 -0.030400000000000208106 rpy=-1.3157660724820988502e-14 2.289083756447533756e-16 3.1415926535897464866 -> xyz=0.00014999999999996659343 -0.061499999999998652966 -0.030399999999999018085 rpy=-3.9472982174462490613e-14 8.7088539502980777788e-16 3.141592653589793116
- joint right_knee_back_rev_1: origin xyz=0.0057402514854763501267 0.013858192987669271101 -0.0050000000000000148492 rpy=-3.1552336572096932e-15 -3.3270436898146921635e-14 1.5677951037379203036 -> xyz=0.0057402514854763535962 0.013858192987669271101 -0.0050000000000000061756 rpy=-1.919569185352210123e-15 -1.6455897748865722783e-15 1.5677951037378847765
- joint right_knee_back_rev_2: origin xyz=0.0057402514854764602817 0.01385819298766871599 -0.026199999999999792899 rpy=-2.1293173172291718105e-14 4.8029314978609855261e-14 3.1385914305327689 -> xyz=0.005740251485476185328 0.013858192987669409879 -0.026200000000000056577 rpy=-6.2585939741374333299e-15 -1.0479387378889103051e-16 3.1385914305327817786
- joint right_knee_front_rev_1: origin xyz=-0.0057402514854764941088 -0.013858192987669354368 -0.004999999999999997502 rpy=2.2689194189169072921e-15 -9.1667614776401742833e-15 1.5678717655286389387 -> xyz=-0.0057402514854763501267 -0.013858192987669284979 -0.0049999999999999957673 rpy=-5.0313204613631514412e-15 -1.1212819345950018642e-16 1.5678717655286047439
- joint right_knee_front_rev_2: origin xyz=-0.0057402514854764750268 -0.013858192987669187834 -0.026200000000000837203 rpy=2.6700561543117312309e-15 -7.7788101235701736907e-15 3.1386680923234866469 -> xyz=-0.0057402514854764195157 -0.013858192987669049057 -0.026200000000000209233 rpy=-4.792276793618950313e-15 -7.4425542615262678023e-15 3.1386680923234981933
- joint right_knee_pitch: origin xyz=5.842070865544391856e-17 -0.095999999999999585665 -0.0092000000000001299488 rpy=-1.390597706429142792e-15 -1.7669519698394562425e-15 -3.1415926535897917837 -> xyz=-1.4425300025281195314e-16 -0.095999999999999197087 -0.009200000000000072703 rpy=-4.4507648457556451305e-14 -3.3964226209539856629e-15 3.1415926535897926719
