Commit message: Add the teleop squat policy

File: toddlerbot/robot_descriptions/assemblies/left_leg_OP3/left_leg_OP3.urdf (robot description, URDF)
Before this commit: robot left_leg_OP3, 11 links, 10 joints
Links:
- link ank_roll_link: mass 0.042599999999999998979 -> 0.042600000000000005917
- link bearing_683: mass 0.00048694686130641793437 -> 0.00048694686130641804279
- link bearing_683_2: mass 0.00048694686130641793437 -> 0.00048694686130641804279
- link knee_rod: mass 0.0031629468613064183613 -> 0.0031629468613064179276
- link knee_rod_2: mass 0.0031629468613064183613 -> 0.0031629468613064179276
- link left_calf_link: mass 0.030999999999999999778 -> 0.030999999999999992839
- link left_hip_pitch_link_xm430: mass 0.1148009013503056841 -> 0.11480090135030569798
- link xm430_plate: mass 0.0026999999999999997093 -> 0.0026999999999999992756
Joints:
- joint left_ank_pitch: limit lower=-0.785398163397448279 upper=1.8325957145940461324 effort=1 velocity=20 -> lower=-1.7453292519943295336 upper=0.785398163397448279 effort=1 velocity=20; origin xyz=0.00050000000000004402902 -0.099999999999997202238 -0.029400000000001407646 rpy=-2.1321242293024632049e-15 1.8823484437772641304e-14 -1.5707963267948981123 -> xyz=0.00050000000000001020191 -0.099999999999999866773 -0.029399999999999901906 rpy=1.3838214396829414281e-15 2.3817753328472465846e-15 -1.5707963267948936714
- joint left_ank_roll: origin xyz=-7.771561172376095783e-16 0.022750000000003930273 0.019000000000007229856 rpy=1.5707963267949729413 8.7734350778775080161e-14 3.1415926535897842342 -> xyz=-1.3877787807814456755e-15 0.022750000000004225176 0.019000000000006383311 rpy=1.5707963267949556219 8.2263916424954431126e-14 3.1415926535897686911
- joint left_hip_pitch: origin xyz=-0.024000000716156176528 -0.019000000152439990714 -0.019000000152458156738 rpy=1.5707963267953688469 1.5707963267944595742 0 -> xyz=-0.024000000716156173058 -0.019000000152439983775 -0.019000000152458156738 rpy=1.5707963267953681807 1.570796326794433817 0
- joint left_hip_roll: origin xyz=0.018999999999999434008 3.7043493321931432202e-16 -0.026000000000000141054 rpy=-3.141592653589793116 -1.5707963267948932273 0 -> xyz=0.018999999999999999528 -3.3408590380433372139e-18 -0.026000000000000002276 rpy=3.141592653589793116 -1.5707963267948821251 0
- joint left_knee_act: limit lower=0 upper=1.9198621771937625091 effort=1 velocity=20 -> lower=0 upper=2.0943951023931952626 effort=1 velocity=20; origin xyz=-0.00015000000000014844124 -0.06150000000000001299 -0.030399999999999711975 rpy=-1.0766672541727743252e-14 1.3282815320613851332e-14 1.5707963267949027752 -> xyz=-0.00014999999999968871242 -0.061500000000000318301 -0.030400000000000086675 rpy=-1.0593309150913038177e-14 1.0308748735206783672e-14 1.5707963267949243136
- joint left_knee_back_rev_1: origin xyz=-0.013858192987669284979 -0.0057402514854763466573 -0.0050000000000000027062 rpy=-1.7626513399117519762e-14 2.0655748330454469805e-14 -3.1386940726547454261 -> xyz=-0.013858192987669326612 -0.0057402514854763431879 -0.004999999999999997502 rpy=-4.4795806497323614513e-17 1.2898425949264794231e-14 -3.1386940726547587488
- joint left_knee_back_rev_2: origin xyz=0.0057402514854756501658 -0.013858192987669437635 -0.026199999999999720041 rpy=4.9560921740722585935e-15 -2.1168138603303528903e-14 1.5736949077299444699 -> xyz=0.0057402514854763535962 -0.013858192987669326612 -0.026199999999999907391 rpy=4.2802438278248956281e-17 2.6960450327599089653e-16 1.5736949077299307032
- joint left_knee_front_rev_1: origin xyz=0.013858192987669312735 0.0057402514854763449226 -0.0049999999999999992367 rpy=2.3955576787343955856e-15 2.4557124758423299065e-14 -3.1357955927274510088 -> xyz=0.013858192987669507024 0.0057402514854762061447 -0.0050000000000007330248 rpy=7.2820716485250802911e-15 3.800162938454114633e-14 -3.1357955927274758778
- joint left_knee_front_rev_2: origin xyz=-0.0057402514854767707972 0.013858192987668854768 -0.026199999999999168399 rpy=9.6260126850146175027e-15 -2.5081324750790058604e-14 1.5765933876572388872 -> xyz=-0.0057402514854763509941 0.013858192987669243346 -0.026199999999999896982 rpy=3.0668764952338581412e-14 -2.4824741237762853711e-14 1.5765933876572135741
- joint left_knee_pitch: limit lower=0 upper=1.9198621771937625091 effort=1 velocity=20 -> lower=0 upper=2.0943951023931952626 effort=1 velocity=20; origin xyz=2.6591951153791853136e-17 -0.096000000000000029754 -0.0091999999999999634154 rpy=-1.3783391157486681965e-14 -1.4843341659320182562e-14 4.5251917072955735634e-15 -> xyz=3.2091917465512721632e-17 -0.09600000000000005751 -0.0091999999999999877015 rpy=2.8679386715174528955e-15 -1.3560834537223585781e-14 2.8113261283774143445e-14

File: toddlerbot/robot_descriptions/toddlerbot_OP3/toddlerbot_OP3.urdf (robot description, URDF)
Before this commit: robot toddlerbot_OP3, 63 links, 62 joints
Links:
- link ank_roll_link: mass 0.042599999999999998979 -> 0.042600000000000005917
- link ank_roll_link_2: mass 0.042599999999999998979 -> 0.042600000000000005917
- link bearing_683: mass 0.00048694686130641793437 -> 0.00048694686130641804279
- link bearing_683_2: mass 0.00048694686130641793437 -> 0.00048694686130641804279
- link bearing_683_3: mass 0.00048694686130641793437 -> 0.00048694686130641804279
- link bearing_683_4: mass 0.00048694686130641793437 -> 0.00048694686130641804279
- link knee_rod: mass 0.0031629468613064183613 -> 0.0031629468613064179276
- link knee_rod_2: mass 0.0031629468613064183613 -> 0.0031629468613064179276
- link knee_rod_3: mass 0.0031629468613064183613 -> 0.0031629468613064179276
- link knee_rod_4: mass 0.0031629468613064183613 -> 0.0031629468613064179276
- link left_calf_link: mass 0.030999999999999999778 -> 0.030999999999999992839
- link left_hip_pitch_link_xm430: mass 0.1148009013503056841 -> 0.11480090135030569798
- link right_calf_link: mass 0.03099999999999998937 -> 0.030999999999999982431
- link right_hip_pitch_link_xm430: mass 0.11480090135030567022 -> 0.1148009013503056841
- link xm430_plate: mass 0.0026999999999999997093 -> 0.0026999999999999992756
- link xm430_plate_2: mass 0.0026999999999999997093 -> 0.0026999999999999992756
Joints:
- joint left_ank_pitch: limit lower=-0.785398163397448279 upper=1.8325957145940461324 effort=1 velocity=20 -> lower=-1.7453292519943295336 upper=0.785398163397448279 effort=1 velocity=20; origin xyz=0.00050000000000004402902 -0.099999999999997202238 -0.029400000000001407646 rpy=-2.1321242293024632049e-15 1.8823484437772641304e-14 -1.5707963267948981123 -> xyz=0.00050000000000001020191 -0.099999999999999866773 -0.029399999999999901906 rpy=1.3838214396829414281e-15 2.3817753328472465846e-15 -1.5707963267948936714
- joint left_ank_roll: origin xyz=-7.771561172376095783e-16 0.022750000000003930273 0.019000000000007229856 rpy=1.5707963267949729413 8.7734350778775080161e-14 3.1415926535897842342 -> xyz=-1.3877787807814456755e-15 0.022750000000004225176 0.019000000000006383311 rpy=1.5707963267949556219 8.2263916424954431126e-14 3.1415926535897686911
- joint left_hip_pitch: origin xyz=-0.024000000716156176528 -0.019000000152439990714 -0.019000000152458156738 rpy=1.5707963267953688469 1.5707963267944595742 0 -> xyz=-0.024000000716156173058 -0.019000000152439983775 -0.019000000152458156738 rpy=1.5707963267953681807 1.570796326794433817 0
- joint left_hip_roll: origin xyz=0.018999999999999434008 3.7043493321931432202e-16 -0.026000000000000141054 rpy=-3.141592653589793116 -1.5707963267948932273 0 -> xyz=0.018999999999999999528 -3.3408590380433372139e-18 -0.026000000000000002276 rpy=3.141592653589793116 -1.5707963267948821251 0
- joint left_knee_act: limit lower=0 upper=1.9198621771937625091 effort=1 velocity=20 -> lower=0 upper=2.0943951023931952626 effort=1 velocity=20; origin xyz=-0.00015000000000014844124 -0.06150000000000001299 -0.030399999999999711975 rpy=-1.0766672541727743252e-14 1.3282815320613851332e-14 1.5707963267949027752 -> xyz=-0.00014999999999968871242 -0.061500000000000318301 -0.030400000000000086675 rpy=-1.0593309150913038177e-14 1.0308748735206783672e-14 1.5707963267949243136
- joint left_knee_back_rev_1: origin xyz=-0.013858192987669284979 -0.0057402514854763466573 -0.0050000000000000027062 rpy=-1.7626513399117519762e-14 2.0655748330454469805e-14 -3.1386940726547454261 -> xyz=-0.013858192987669326612 -0.0057402514854763431879 -0.004999999999999997502 rpy=-4.4795806497323614513e-17 1.2898425949264794231e-14 -3.1386940726547587488
- joint left_knee_back_rev_2: origin xyz=0.0057402514854756501658 -0.013858192987669437635 -0.026199999999999720041 rpy=4.9560921740722585935e-15 -2.1168138603303528903e-14 1.5736949077299444699 -> xyz=0.0057402514854763535962 -0.013858192987669326612 -0.026199999999999907391 rpy=4.2802438278248956281e-17 2.6960450327599089653e-16 1.5736949077299307032
- joint left_knee_front_rev_1: origin xyz=0.013858192987669312735 0.0057402514854763449226 -0.0049999999999999992367 rpy=2.3955576787343955856e-15 2.4557124758423299065e-14 -3.1357955927274510088 -> xyz=0.013858192987669507024 0.0057402514854762061447 -0.0050000000000007330248 rpy=7.2820716485250802911e-15 3.800162938454114633e-14 -3.1357955927274758778
- joint left_knee_front_rev_2: origin xyz=-0.0057402514854767707972 0.013858192987668854768 -0.026199999999999168399 rpy=9.6260126850146175027e-15 -2.5081324750790058604e-14 1.5765933876572388872 -> xyz=-0.0057402514854763509941 0.013858192987669243346 -0.026199999999999896982 rpy=3.0668764952338581412e-14 -2.4824741237762853711e-14 1.5765933876572135741
- joint left_knee_pitch: limit lower=0 upper=1.9198621771937625091 effort=1 velocity=20 -> lower=0 upper=2.0943951023931952626 effort=1 velocity=20; origin xyz=2.6591951153791853136e-17 -0.096000000000000029754 -0.0091999999999999634154 rpy=-1.3783391157486681965e-14 -1.4843341659320182562e-14 4.5251917072955735634e-15 -> xyz=3.2091917465512721632e-17 -0.09600000000000005751 -0.0091999999999999877015 rpy=2.8679386715174528955e-15 -1.3560834537223585781e-14 2.8113261283774143445e-14
- joint right_ank_pitch: limit lower=-0.785398163397448279 upper=1.8325957145940461324 effort=1 velocity=20 -> lower=-1.7453292519943295336 upper=0.785398163397448279 effort=1 velocity=20; origin xyz=0.00049999999999975335441 0.099999999999999561462 0.0086000000000000676598 rpy=3.1415926535897877869 -1.4928027344634987948e-14 1.5707963267948785724 -> xyz=0.00050000000000040452624 0.10000000000000006106 0.0086000000000003035822 rpy=3.141592653589793116 -9.7384055572523312245e-16 1.5707963267948936714
- joint right_ank_roll: origin xyz=-2.2204460492503130808e-16 0.02275000000000106104 0.019000000000002178341 rpy=1.5707963267949220931 -3.6775852931107809278e-14 3.1415926535897313876 -> xyz=1.9151347174783950322e-15 0.022749999999999825917 0.019000000000001193018 rpy=1.5707963267949667241 3.4534200721523706957e-14 3.1415926535897917837
- joint right_hip_pitch: origin xyz=-0.024000000716143346513 -0.019000000152445729179 -0.019000000152453181551 rpy=1.5707963267950966202 1.5707963267947326891 0 -> xyz=-0.024000000716147704138 -0.019000000152441253592 -0.01900000015245582527 rpy=1.570796326795185216 1.5707963267947977481 0
- joint right_hip_roll: origin xyz=-0.018999999999999916261 3.1092928099478391072e-16 -0.025999999999999925948 rpy=3.0774993384580180772e-19 -1.5707963267948932273 0 -> xyz=-0.018999999999999999528 -1.7604701631262654893e-16 -0.025999999999999919009 rpy=-2.8481848693987683332e-20 -1.5707963267948954478 0
- joint right_knee_act: limit lower=-1.9198621771937625091 upper=0 effort=1 velocity=20 -> lower=-2.0943951023931952626 upper=0 effort=1 velocity=20; origin xyz=0.00014999999999996659343 -0.061499999999998652966 -0.030399999999999018085 rpy=-3.9472982174462490613e-14 8.7088539502980777788e-16 3.141592653589793116 -> xyz=0.00015000000000000958205 -0.061499999999999971356 -0.030399999999999996469 rpy=1.8480226030005917304e-16 2.0301725913858999669e-15 3.1415926535897922278
- joint right_knee_back_rev_1: origin xyz=0.0057402514854763535962 0.013858192987669271101 -0.0050000000000000061756 rpy=-1.919569185352210123e-15 -1.6455897748865722783e-15 1.5677951037378847765 -> xyz=0.0057402514854763666066 0.01385819298766934049 -0.005000000000000016584 rpy=-5.9721322899995738745e-15 2.1763425120495147882e-14 1.5651031369169621232
- joint right_knee_back_rev_2: origin xyz=0.005740251485476185328 0.013858192987669409879 -0.026200000000000056577 rpy=-6.2585939741374333299e-15 -1.0479387378889103051e-16 3.1385914305327817786 -> xyz=0.0057402514854763960969 0.013858192987669354368 -0.026200000000000014944 rpy=2.0307557008913139329e-14 -1.7771544142448121049e-15 3.1358994637118597915
- joint right_knee_front_rev_1: origin xyz=-0.0057402514854763501267 -0.013858192987669284979 -0.0049999999999999957673 rpy=-5.0313204613631514412e-15 -1.1212819345950018642e-16 1.5678717655286047439 -> xyz=-0.0057402514854763735455 -0.013858192987669271101 -0.0049999999999999992367 rpy=3.7594106814525390121e-15 -6.9096598398549006487e-16 1.5651666422844430215
- joint right_knee_front_rev_2: origin xyz=-0.0057402514854764195157 -0.013858192987669049057 -0.026200000000000209233 rpy=-4.792276793618950313e-15 -7.4425542615262678023e-15 3.1386680923234981933 -> xyz=-0.0057402514854764195157 -0.013858192987669160079 -0.026200000000000063516 rpy=-5.1439183405559488125e-16 -2.9685331931264604348e-15 3.1359629690793391354
- joint right_knee_pitch: limit lower=-1.9198621771937625091 upper=0 effort=1 velocity=20 -> lower=-2.0943951023931952626 upper=0 effort=1 velocity=20; origin xyz=-1.4425300025281195314e-16 -0.095999999999999197087 -0.009200000000000072703 rpy=-4.4507648457556451305e-14 -3.3964226209539856629e-15 3.1415926535897926719 -> xyz=6.6012271456357184538e-18 -0.095999999999999877098 -0.009199999999999972089 rpy=-9.138977281102487298e-16 5.7742659530791861042e-17 3.141592653589793116
