Commit message: Fix the waist kinematics

File: toddlerbot/robot_descriptions/assemblies/left_arm_hand/left_arm_hand.urdf (robot description, URDF)
Before this commit: robot left_arm_hand, 15 links, 14 joints
Links:
- link elb_yaw_link: mass 0.017499999999999998196 -> 0.017500000000000001665
- link hand: mass 0.017000000000001441042 -> 0.017000000000000004691
- link sho_pitch_link: mass 0.0085999999999999930667 -> 0.008600000000000003475
- link sho_yaw_link: mass 0.01450000000000000247 -> 0.014499999999999986858
- link spur_1m_24t_driven: mass 0.0027000000000000001429 -> 0.0026999999999999997093
- link spur_1m_24t_driven_2: mass 0.0027000000000000001429 -> 0.0026999999999999997093
- link spur_1m_24t_driven_3: mass 0.0027000000000000001429 -> 0.0026999999999999997093
- link wrist_bearing_plate: mass 0.0049000367468305548388 -> 0.0049000367468305539714

File: toddlerbot/robot_descriptions/assemblies/left_leg_XM430/left_leg_XM430.urdf (robot description, URDF)
Before this commit: robot left_leg_XM430, 12 links, 11 joints
Links:
- link ank_rr_link: mass 0.0014500000000000001169 -> 0.0014499999999999999001
- link ank_rr_link_2: mass 0.0014500000000000001169 -> 0.0014499999999999999001
- link hip_roll_link: mass 0.10699970659110667748 -> 0.10699970659110669136
- link hip_yaw_link: mass 0.017999999999999991701 -> 0.01799999999999999864
- link left_calf_link: mass 0.079607494529051470167 -> 0.079607494529051442411

File: toddlerbot/robot_descriptions/assemblies/right_arm_hand/right_arm_hand.urdf (robot description, URDF)
Before this commit: robot right_arm_hand, 15 links, 14 joints
Links:
- link elb_yaw_link: mass 0.017499999999999998196 -> 0.017500000000000001665
- link hand: mass 0.017000000000001441042 -> 0.017000000000000004691
- link sho_pitch_link: mass 0.0085999999999999930667 -> 0.008600000000000003475
- link sho_yaw_link: mass 0.01450000000000000247 -> 0.014499999999999986858
- link spur_1m_24t_driven: mass 0.0027000000000000001429 -> 0.0026999999999999997093
- link spur_1m_24t_driven_2: mass 0.0027000000000000001429 -> 0.0026999999999999997093
- link spur_1m_24t_driven_3: mass 0.0027000000000000001429 -> 0.0026999999999999997093
- link wrist_bearing_plate: mass 0.0049000367468305548388 -> 0.0049000367468305539714

File: toddlerbot/robot_descriptions/assemblies/right_leg_XM430/right_leg_XM430.urdf (robot description, URDF)
Before this commit: robot right_leg_XM430, 12 links, 11 joints
Links:
- link ank_motor_rod_short: mass 0.0017000000000000005558 -> 0.0017000000000000001221
- link ank_roll_link: mass 0.024800000000000016476 -> 0.024800000000000009537
- link hip_roll_link: mass 0.10699970659110667748 -> 0.10699970659110669136
- link right_calf_link: mass 0.079607494529051456289 -> 0.079607494529051442411

File: toddlerbot/robot_descriptions/assemblies/toddlerbot/toddlerbot.urdf (robot description, URDF)
Before this commit: robot toddlerbot, 17 links, 16 joints
Links:
- link left_arm_hand: mass 0.47285924835363390972 -> 0.47285924835363246643
- link left_leg_xm430: mass 0.28007018314906156897 -> 0.28007018314906162448
- link neck_pitch_link: mass 0.10851928601941274177 -> 0.10851928601941271402
- link neck_yaw_link: mass 0.0085168305947458267796 -> 0.0085168305947458250449
- link right_arm_hand: mass 0.47285924835363390972 -> 0.47285924835363246643
- link spiral_bevel_1m_14t_30deg: mass 0.00067997563436136246491 -> 0.00067997563436136235649
- link spiral_bevel_1m_14t_30deg_2: mass 0.00067997563436136246491 -> 0.00067997563436136235649
- link spur_1m_20t: mass 0.0015534950290892282111 -> 0.0015534950290892286448
- link torso: mass 0.38210896478124972697 -> 0.38210896478125000453
- link waist_link: mass 0.15193452399186060942 -> 0.15193452399186058166
Joints:
- joint left_hip_yaw_driven: origin xyz=-0.037000000000000005107 -0.041100000000000080913 0.019500000000000003442 rpy=-1.5707963267948841235 1.5707963267948932273 0 -> xyz=-0.037000000000000005107 -0.041100000000000108669 0.019500000000000006911 rpy=-1.5707963267948841235 1.5707963267948932273 0
- joint left_leg_fixed: origin xyz=-4.336808689942017736e-19 -1.3877787807814456755e-17 -0.004999999999999997502 rpy=-1.0439449364097525548e-14 -1.9757585399875400437e-31 5.7250078249404190712e-30 -> xyz=3.0357660829594124152e-18 -1.3877787807814456755e-17 -0.0049999999999999697464 rpy=-1.0439449364097525548e-14 1.9685459861175557675e-31 1.834678230847674038e-29
- joint neck_pitch_driven: origin xyz=3.7500079430596855445e-10 0.0051500000614755261225 -0.02749999999999992728 rpy=1.57079632679489678 4.0384474451367016523e-16 -3.141592653589793116 -> xyz=3.7500073185592341929e-10 0.0051500000614755261225 -0.027499999999999941158 rpy=1.57079632679489678 -1.7934420258902467287e-15 -3.1415926535897922278
- joint neck_yaw_driven: origin xyz=0.016000000000001915468 1.4752314067929373936e-17 0.12348651076281796923 rpy=-3.141592653589793116 -2.1972867704039169433e-15 -3.1415926535897926719 -> xyz=0.016000000000001915468 1.4752314067929367773e-17 0.12348651076281796923 rpy=-3.141592653589793116 -0 -3.1415926535897922278
- joint right_hip_yaw_drive: origin xyz=0.037000000000000358991 -0.037100000000003852119 0.039500000000000069778 rpy=-1.5707963267949709429 3.0776023904592405576e-13 2.7738547283800353153e-13 -> xyz=0.037000000000000358991 -0.037100000000003852119 0.039500000000000062839 rpy=-1.5707963267949709429 3.0764921674346154011e-13 2.7727445053553844104e-13
- joint waist_act_1: limit lower=-6.283185307179586232 upper=6.283185307179586232 effort=1 velocity=20 -> lower=-2.7925268031909271649 upper=2.7925268031909271649 effort=1 velocity=20; origin xyz=3.5815341505539062119e-17 -0.019600000000000016714 0.012750000000000042549 rpy=-1.570796326794896336 -1.5707963267948215069 0 -> xyz=4.8392086706372466624e-17 -0.019600000000000009776 0.012750000000000042549 rpy=-1.5707963267948961139 -1.5707963267948215069 0
- joint waist_act_2: limit lower=-6.283185307179586232 upper=6.283185307179586232 effort=1 velocity=20 -> lower=-2.7925268031909271649 upper=2.7925268031909271649 effort=1 velocity=20; origin xyz=-6.3212258568462825292e-16 -0.019600000000000079164 0.032750000000000834 rpy=-1.5707963267948976682 -1.3463968515393018865 1.5503953316521244903e-14 -> xyz=-6.321225856846266752e-16 -0.019600000000000079164 0.032750000000000834 rpy=-1.5707963267948976682 -1.3463968515393018865 1.5503953316521244903e-14
- joint waist_roll: origin xyz=-6.2255683189587157383e-20 0.022707865260692461362 -0.013000000000000004607 rpy=1.5707963267948952257 1.2017992026080351615e-15 4.2181022606678868535e-16 -> xyz=-6.2255683191263486807e-20 0.022707865260692461362 -0.013000000000000004607 rpy=1.5707963267948952257 1.2017992026080351615e-15 4.2181022606678868535e-16
- joint waist_yaw: origin xyz=-1.7347234759768070944e-18 -9.8607613152626475676e-32 0 rpy=2.0946901476030943553e-15 7.1861600448343401911e-16 -1.5707963267948228392 -> xyz=-1.7347234759768070944e-18 -1.9721522630525295135e-31 0 rpy=2.0946901476030943553e-15 7.1861600448343401911e-16 -1.5707963267948228392

File: toddlerbot/robot_descriptions/toddlerbot/toddlerbot.urdf (robot description, URDF)
Before this commit: robot toddlerbot, 67 links, 66 joints
Links:
- link ank_roll_link_2: mass 0.024800000000000016476 -> 0.024800000000000009537
- link ank_rr_link: mass 0.0014500000000000001169 -> 0.0014499999999999999001
- link ank_rr_link_2: mass 0.0014500000000000001169 -> 0.0014499999999999999001
- link ank_rr_link_3: mass 0.0014500000000000001169 -> 0.0014499999999999999001
- link ank_rr_link_4: mass 0.0014500000000000001169 -> 0.0014499999999999999001
- link elb_yaw_link: mass 0.017499999999999998196 -> 0.017500000000000001665
- link elb_yaw_link_2: mass 0.017499999999999998196 -> 0.017500000000000001665
- link hand: mass 0.017000000000001441042 -> 0.017000000000000004691
- link hand_2: mass 0.017000000000001441042 -> 0.017000000000000004691
- link hip_yaw_link: mass 0.017999999999999984762 -> 0.01799999999999999864
- link hip_yaw_link_2: mass 0.017999999999999984762 -> 0.01799999999999999864
- link left_hip_pitch_link_xm430: mass 0.035548688791081757554 -> 0.035548688791081778371
- link neck_pitch_link: mass 0.10851928601941274177 -> 0.10851928601941271402
- link neck_yaw_link: mass 0.0085168305947458267796 -> 0.0085168305947458250449
- link sho_pitch_link: mass 0.0085999999999999930667 -> 0.008600000000000003475
- link sho_pitch_link_2: mass 0.0085999999999999930667 -> 0.008600000000000003475
- link sho_yaw_link: mass 0.01450000000000000247 -> 0.014499999999999986858
- link sho_yaw_link_2: mass 0.01450000000000000247 -> 0.014499999999999986858
- link spiral_bevel_1m_14t_30deg: mass 0.00067997563436136246491 -> 0.00067997563436136235649
- link spiral_bevel_1m_14t_30deg_2: mass 0.00067997563436136246491 -> 0.00067997563436136235649
- link spur_1m_20t: mass 0.0015534950290892282111 -> 0.0015534950290892286448
- link spur_1m_24t_driven: mass 0.0027000000000000001429 -> 0.0026999999999999997093
- link spur_1m_24t_driven_2: mass 0.0027000000000000001429 -> 0.0026999999999999997093
- link spur_1m_24t_driven_3: mass 0.0027000000000000001429 -> 0.0026999999999999997093
- link spur_1m_24t_driven_4: mass 0.0027000000000000001429 -> 0.0026999999999999997093
- link spur_1m_24t_driven_5: mass 0.0027000000000000001429 -> 0.0026999999999999997093
- link spur_1m_24t_driven_6: mass 0.0027000000000000001429 -> 0.0026999999999999997093
- link torso: mass 0.38210896478124972697 -> 0.38210896478125000453
- link waist_link: mass 0.15193452399186060942 -> 0.15193452399186058166
- link wrist_bearing_plate: mass 0.0049000367468305548388 -> 0.0049000367468305539714
- link wrist_bearing_plate_2: mass 0.0049000367468305548388 -> 0.0049000367468305539714
Joints:
- joint left_hip_yaw_driven: origin xyz=-0.037000000000000005107 -0.041100000000000080913 0.019500000000000003442 rpy=-1.5707963267948841235 1.5707963267948932273 0 -> xyz=-0.037000000000000005107 -0.041100000000000108669 0.019500000000000006911 rpy=-1.5707963267948841235 1.5707963267948932273 0
- joint left_leg_fixed: origin xyz=-4.336808689942017736e-19 -1.3877787807814456755e-17 -0.004999999999999997502 rpy=-1.0439449364097525548e-14 -1.9757585399875400437e-31 5.7250078249404190712e-30 -> xyz=3.0357660829594124152e-18 -1.3877787807814456755e-17 -0.0049999999999999697464 rpy=-1.0439449364097525548e-14 1.9685459861175557675e-31 1.834678230847674038e-29
- joint neck_pitch_driven: origin xyz=3.7500079430596855445e-10 0.0051500000614755261225 -0.02749999999999992728 rpy=1.57079632679489678 4.0384474451367016523e-16 -3.141592653589793116 -> xyz=3.7500073185592341929e-10 0.0051500000614755261225 -0.027499999999999941158 rpy=1.57079632679489678 -1.7934420258902467287e-15 -3.1415926535897922278
- joint neck_yaw_driven: origin xyz=0.016000000000001915468 1.4752314067929373936e-17 0.12348651076281796923 rpy=-3.141592653589793116 -2.1972867704039169433e-15 -3.1415926535897926719 -> xyz=0.016000000000001915468 1.4752314067929367773e-17 0.12348651076281796923 rpy=-3.141592653589793116 -0 -3.1415926535897922278
- joint right_ank_L_rev_1: origin xyz=0.017999999999999981293 0.015999999999999847677 -0.020600000000000010664 rpy=6.2884229534673233247e-16 3.9390862739624346782e-15 0.018223085042996144817 -> xyz=0.017999999999999981293 0.015999999999999847677 -0.020600000000000014133 rpy=6.2884229534673233247e-16 3.939086273962429945e-15 0.018223085042996144817
- joint right_ank_L_rev_2: origin xyz=-6.9388939039072283776e-18 -0.0099999999999996203037 2.7755575615628913511e-17 rpy=-1.5707963267948887864 -1.3320366994106427327 -1.5707963267948827912 -> xyz=-6.9388939039072283776e-18 -0.0099999999999996203037 3.1225022567582527699e-17 rpy=-1.5707963267948887864 -1.3320366994106427327 -1.5707963267948827912
- joint right_ank_S_rev_1: origin xyz=-0.018000000000000026396 0.016000000000000735856 -0.02059999999999996903 rpy=-4.338977813478965687e-16 1.6392354569195936347e-16 3.1154741050825114357 -> xyz=-0.018000000000000026396 0.016000000000000735856 -0.02059999999999996903 rpy=-4.338977813478965687e-16 1.6392354569195739132e-16 3.1154741050825114357
- joint right_ank_S_rev_2: origin xyz=-2.7408630920433552092e-16 0.010000000000000508482 -1.561251128379126385e-16 rpy=-1.5707963267949354158 1.2119133862908570975 -1.5707963267949336394 -> xyz=-2.7755575615628913511e-16 0.010000000000000563993 -1.561251128379126385e-16 rpy=-1.5707963267949354158 1.2119133862908570975 -1.5707963267949336394
- joint right_ank_act_1: origin xyz=0.013499999999995845185 0.044500000000006201262 0.0040000000000029352354 rpy=-2.976243182117608527e-13 -7.5970722241046887472e-14 0.21173394130155420712 -> xyz=0.013499999999995838246 0.044500000000006201262 0.0040000000000029352354 rpy=-2.9762431821176080221e-13 -7.5970722241046912715e-14 0.21173394130155420712
- joint right_ank_act_2: origin xyz=0.013500000000004732173 0.064500000000008106404 -0.024800000000001404254 rpy=-3.1415926535894733718 -2.3305959971649736532e-13 0.22995607267265857909 -> xyz=0.013500000000004725234 0.064500000000008106404 -0.024800000000001404254 rpy=-3.1415926535894733718 -2.3305959971649736532e-13 0.22995607267265857909
- joint right_ank_pitch: origin xyz=-3.3506429374353506934e-17 0.10000000000000000555 -0.01039999999999995442 rpy=-5.6239133145187819342e-16 -1.1344214119703426107e-16 3.141592653589793116 -> xyz=-4.0265291502142843319e-17 0.10000000000000000555 -0.010399999999999947481 rpy=-5.6239133145192868052e-16 -1.1344214119702528777e-16 3.141592653589793116
- joint right_ank_roll: origin xyz=0.0014999999999999924418 2.7755575615628913511e-17 -6.9388939039072283776e-18 rpy=3.141592653589793116 -1.570796326794896336 0 -> xyz=0.0014999999999999924418 2.7755575615628913511e-17 -1.3877787807814456755e-17 rpy=3.141592653589793116 -1.570796326794896336 0
- joint right_hip_yaw_drive: origin xyz=0.037000000000000358991 -0.037100000000003852119 0.039500000000000069778 rpy=-1.5707963267949709429 3.0776023904592405576e-13 2.7738547283800353153e-13 -> xyz=0.037000000000000358991 -0.037100000000003852119 0.039500000000000062839 rpy=-1.5707963267949709429 3.0764921674346154011e-13 2.7727445053553844104e-13
- joint right_knee: origin xyz=3.9466670230816398047e-17 -0.096000000000000029754 -0.0091999999999999235167 rpy=1.282522668451654911e-14 1.4584655840118584511e-16 -3.1415926535897926719 -> xyz=-2.9922268808255885729e-17 -0.096000000000000029754 -0.0091999999999999235167 rpy=1.2825226684517786044e-14 1.3611434254495038701e-14 -3.1415926535897926719
- joint waist_act_1: limit lower=-6.283185307179586232 upper=6.283185307179586232 effort=1 velocity=20 -> lower=-2.7925268031909271649 upper=2.7925268031909271649 effort=1 velocity=20; origin xyz=3.5815341505539062119e-17 -0.019600000000000016714 0.012750000000000042549 rpy=-1.570796326794896336 -1.5707963267948215069 0 -> xyz=4.8392086706372466624e-17 -0.019600000000000009776 0.012750000000000042549 rpy=-1.5707963267948961139 -1.5707963267948215069 0
- joint waist_act_2: limit lower=-6.283185307179586232 upper=6.283185307179586232 effort=1 velocity=20 -> lower=-2.7925268031909271649 upper=2.7925268031909271649 effort=1 velocity=20; origin xyz=-6.3212258568462825292e-16 -0.019600000000000079164 0.032750000000000834 rpy=-1.5707963267948976682 -1.3463968515393018865 1.5503953316521244903e-14 -> xyz=-6.321225856846266752e-16 -0.019600000000000079164 0.032750000000000834 rpy=-1.5707963267948976682 -1.3463968515393018865 1.5503953316521244903e-14
- joint waist_roll: origin xyz=-6.2255683189587157383e-20 0.022707865260692461362 -0.013000000000000004607 rpy=1.5707963267948952257 1.2017992026080351615e-15 4.2181022606678868535e-16 -> xyz=-6.2255683191263486807e-20 0.022707865260692461362 -0.013000000000000004607 rpy=1.5707963267948952257 1.2017992026080351615e-15 4.2181022606678868535e-16
- joint waist_yaw: origin xyz=-1.7347234759768070944e-18 -9.8607613152626475676e-32 0 rpy=2.0946901476030943553e-15 7.1861600448343401911e-16 -1.5707963267948228392 -> xyz=-1.7347234759768070944e-18 -1.9721522630525295135e-31 0 rpy=2.0946901476030943553e-15 7.1861600448343401911e-16 -1.5707963267948228392
