Commit message: Update the robot fk and ik

File: toddlerbot/robot_descriptions/toddlerbot/toddlerbot.urdf (robot description, URDF)
Before this commit: robot toddlerbot, 77 links, 76 joints
Links:
- link elb_yaw_link: mass 0.017500000000000001665 -> 0.017499999999999998196
- link elb_yaw_link_2: mass 0.017500000000000001665 -> 0.017499999999999998196
- link sho_pitch_link: mass 0.0085999999999999930667 -> 0.0085999999999999982708
- link sho_pitch_link_2: mass 0.0085999999999999930667 -> 0.0085999999999999982708
- link sho_yaw_link: mass 0.014500000000000007674 -> 0.014500000000000012879
- link sho_yaw_link_2: mass 0.014500000000000007674 -> 0.014500000000000012879
- link spur_1m_24t_driven: mass 0.0026999999999999997093 -> 0.0026999999999999992756
- link spur_1m_24t_driven_2: mass 0.0026999999999999997093 -> 0.0026999999999999992756
- link spur_1m_24t_driven_3: mass 0.0026999999999999997093 -> 0.0026999999999999992756
- link spur_1m_24t_driven_4: mass 0.0026999999999999997093 -> 0.0026999999999999992756
- link spur_1m_24t_driven_5: mass 0.0026999999999999997093 -> 0.0026999999999999992756
- link spur_1m_24t_driven_6: mass 0.0026999999999999997093 -> 0.0026999999999999992756
- link spur_gear_(13_teeth): mass 0.00081469437497230865874 -> 0.00081469437497230876716
- link spur_gear_21_teeth: mass 0.0010063046528317974842 -> 0.001006304652831797701
- link spur_gear_21_teeth_2: mass 0.0010063046528317974842 -> 0.001006304652831797701
- link torso: mass 0.58490521749923585215 -> 0.58490521749923596317
- link waist_gears: mass 0.02331580566917982808 -> 0.023315805669179824611
- link waist_link: mass 0.1663195349061246664 -> 0.16631953490612461088
Joints:
- joint left_elbow_yaw_driven: origin xyz=-3.5806829723483701855e-10 -0.027000000152447967139 -0.019000000000002889577 rpy=1.5707963267948912289 1.5707963267948952257 0 -> xyz=-3.5806832845985958613e-10 -0.027000000152447967139 -0.019000000000002903455 rpy=1.5707963267948912289 1.5707963267948950037 0
- joint left_elbow_yaw_fixed: origin xyz=1.5777218104420236108e-30 0 0.0015999999999999903189 rpy=3.141592653589793116 -0 -1.570796326794896558 -> xyz=-1.498879432863449632e-17 3.1225022567582527699e-17 0.0015999999999999903189 rpy=3.141592653589793116 6.1232339945831272199e-17 -1.57079632679489678
- joint left_hip_yaw_drive: origin xyz=-0.036999999999999207134 -0.037100000000004823564 0.039500000000000437539 rpy=-1.5707963267950579844 5.7109166702824404977e-13 2.6938840543896956895e-13 -> xyz=-0.036999999999999241829 0.037100000000004858258 -0.039500000000001048162 rpy=1.5707963267947455677 -6.8514345590022702401e-13 -2.4160785457991476196e-13
- joint left_hip_yaw_driven: origin xyz=-0.036999999999999998168 -0.041100000000000067035 0.019500000000000006911 rpy=-1.5707963267948841235 1.5707963267948956698 0 -> xyz=-0.036999999999999977351 0.041100000000000032341 -0.019499999999999986094 rpy=1.5707963267948990005 -1.5707963267948927832 0
- joint left_leg_fixed: origin xyz=-4.336808689942017736e-19 6.9388939039072283776e-18 -0.0050000000000000044409 rpy=-1.0439449364097535015e-14 3.7110850528220658615e-31 -4.3084061976207498209e-30 -> xyz=-4.336808689942017736e-19 0 -0.004999999999999997502 rpy=1.3877787807813717198e-16 1.6653345369377375223e-16 1.373730595408674402e-16
- joint left_sho_pitch: origin xyz=-0.0029999999999997389866 0.062000000000000464462 0.10523651076281793915 rpy=-1.5707963267948983344 -3.4972025276127318207e-15 -2.4598039012687864683e-16 -> xyz=-0.0029999999999997528644 0.062000000000000436706 0.10523651076281793915 rpy=-1.5707963267948983344 -2.9907641379514081331e-14 -1.2153003607487542119e-15
- joint left_sho_roll: limit lower=-1.570796326794896558 upper=1.570796326794896558 effort=1 velocity=20 -> lower=-1.570796326794896558 upper=0 effort=1 velocity=20
- joint left_sho_yaw_driven: origin xyz=-3.5807099299511868651e-10 -0.027000000152450111257 -0.019000000000003024886 rpy=1.5707963267949034414 2.5500465800399188824e-14 -4.889500977014397436e-15 -> xyz=-3.5807099299511868651e-10 -0.027000000152450111257 -0.019000000000003024886 rpy=1.5707963267949034414 2.5500465800399195135e-14 -4.8895009770147760892e-15
- joint left_sho_yaw_fixed: origin xyz=-6.9388939039072283776e-18 -3.9443045261050590271e-31 0.0015999999999999972577 rpy=-3.141592653589793116 -2.947294251859628371e-29 -3.8176863193325490556e-30 -> xyz=-6.9388939039072283776e-18 -3.9443045261050590271e-31 0.0015999999999999972577 rpy=-3.141592653589793116 3.4918029198749163057e-28 2.4932009224355828724e-30
- joint left_wrist_pitch_drive: origin xyz=-1.5244092446686785536e-10 0.024000000358059436767 -0.0080000000000068592632 rpy=7.9382516163035126435e-16 -8.221371570986757145e-15 -1.5707963267949174302 -> xyz=-1.5244092793631480731e-10 0.024000000358059436767 -0.0080000000000068592632 rpy=7.9382516163034810891e-16 -8.2213715709867981657e-15 -1.5707963267949174302
- joint neck_pitch_driven: origin xyz=3.7500073185592341929e-10 0.0051500000614755261225 -0.027499999999999941158 rpy=1.57079632679489678 -1.7934420258902467287e-15 -3.1415926535897922278 -> xyz=3.7500078736707465055e-10 0.0051500000614755261225 -0.027499999999999941158 rpy=1.570796326794896558 7.3154045537456631165e-17 -3.141592653589793116
- joint neck_yaw_driven: origin xyz=0.016000000000001915468 1.4752314067929367773e-17 0.12348651076281796923 rpy=-3.141592653589793116 -0 -3.1415926535897922278 -> xyz=0.016000000000001915468 1.75992996990887874e-17 0.12348651076281796923 rpy=3.141592653589793116 -1.8665960714277032613e-15 -3.141592653589793116
- joint right_elbow_roll: origin xyz=0 -0.018999999999999950956 -0.058999999999999955258 rpy=1.570796326794896558 -2.9936014833487158253e-15 -1.8179902027461223811e-15 -> xyz=1.3634926521177703762e-15 -0.018999999999998080924 -0.058999999999999955258 rpy=1.570796326794896558 4.7458355760175941122e-14 -1.8179902027463432622e-15
- joint right_elbow_yaw_drive: origin xyz=-0.024000000716145237362 -0.019000000152448695556 -0.019000000152448712903 rpy=1.5707963267950246777 1.6760397103577610108e-15 -7.8984688976387225082e-14 -> xyz=-0.024000000716145213076 -0.019000000152448681678 -0.019000000152448712903 rpy=1.5707963267950251218 7.4561439664805901366e-16 -7.8480721140448757714e-14
- joint right_elbow_yaw_driven: origin xyz=-3.5807088544226317595e-10 -0.027000000152451505975 -0.01900000000000293468 rpy=1.570796326794921427 8.4749116765166275158e-14 -2.9577354942701689238e-14 -> xyz=-3.5807097564788392674e-10 -0.027000000152451450464 -0.019000000000002660594 rpy=1.570796326794921427 8.594260651656727047e-14 -2.9577354942701670305e-14
- joint right_elbow_yaw_fixed: origin xyz=-3.4694469519536141888e-18 -2.3665827156630354162e-30 0.0015999999999999903189 rpy=-3.1415926535897917837 7.2632216806324781157e-16 -1.1934897514010108924e-15 -> xyz=0 -7.8886090522101180541e-31 0.0015999999999999903189 rpy=-3.1415926535897917837 -3.113586376513707077e-30 -9.3975474487378148241e-30
- joint right_hip_yaw_drive: origin xyz=0.037000000000000352052 -0.037100000000003852119 0.039500000000000062839 rpy=-1.5707963267949709429 3.0763843997160748787e-13 2.7733309074151655565e-13 -> xyz=0.037000000000000345113 0.037100000000003956202 -0.039500000000000284883 rpy=1.5707963267948685804 -4.0596895443104855274e-13 -3.0450824182461770003e-13
- joint right_hip_yaw_driven: origin xyz=0.036999999999999991229 -0.041099999999999997646 0.019500000000000006911 rpy=-1.5707963267948983344 1.5707963267948956698 0 -> xyz=0.036999999999999991229 0.041100000000000004585 -0.019499999999999982625 rpy=1.5707963267949123232 -1.5707963267948839015 0
- joint right_leg_fixed: origin xyz=0 -6.9388939039072283776e-18 -0.004999999999999997502 rpy=1.60982722631807463e-15 -3.5340660733628542786e-32 -3.0121122483794329866e-31 -> xyz=1.7347234759768070944e-18 0 -0.0050000000000000044409 rpy=-1.5390466678866437645e-14 2.775557561557233123e-17 3.0000653983610458155e-17
- joint right_sho_pitch: origin xyz=-0.0030000000000001136868 -0.061999999999999992617 0.10523651076281731465 rpy=-1.570796326794896558 -3.3306690742370509197e-16 3.141592653589793116 -> xyz=-0.0030000000000001275646 -0.061999999999999985678 0.10523651076281731465 rpy=-1.570796326794896558 2.7165362863923079035e-14 3.1415926535897922278
- joint right_sho_roll: limit lower=-1.570796326794896558 upper=1.570796326794896558 effort=1 velocity=20 -> lower=-1.570796326794896558 upper=0 effort=1 velocity=20
- joint right_sho_yaw_driven: origin xyz=-3.5806683312822329412e-10 -0.027000000152447932444 -0.019000000000004180212 rpy=1.570796326794941189 -3.7231669281427893777e-14 -1.380172419158038954e-15 -> xyz=-3.5806542800220775291e-10 -0.027000000152447953261 -0.019000000000004266948 rpy=1.5707963267949396347 -3.5760623773800501683e-14 -2.120003783509950459e-15
- joint right_sho_yaw_fixed: origin xyz=-5.898059818321144121e-17 1.201620916072157247e-16 0.0015999999999999972577 rpy=-3.141592653589793116 -5.4212913233780230364e-29 2.371286511247144379e-30 -> xyz=-1.4641066137244251877e-15 2.0460946366117099189e-16 0.0015999999999999764411 rpy=-3.1415926535897917837 7.3983136435191466048e-16 1.4710455076273571868e-15
- joint right_wrist_pitch_drive: origin xyz=-1.5244520229495961416e-10 0.0240000003580740362 -0.0080000000000021095903 rpy=-2.1390725319343247708e-14 -2.6312285683659644689e-14 -1.5707963267949076602 -> xyz=-1.5244519882551266221e-10 0.0240000003580740362 -0.0080000000000021130597 rpy=-2.1390725319341436483e-14 -2.6312285683659641534e-14 -1.5707963267949076602
- joint right_wrist_pitch_driven: origin xyz=0 0 -0.0016000000000000007272 rpy=2.5486097626493842382e-14 -1.8651746813702645656e-14 1.570796326794896558 -> xyz=0 -3.4694469519536141888e-18 -0.0015999999999999937883 rpy=2.5695941831520308968e-14 -1.8435423390073007778e-14 1.570796326794896336
- joint right_wrist_pitch_fixed: origin xyz=3.4694469519536141888e-18 -0.025299999999999999573 -0.052000000000000004552 rpy=1.5707963267949045516 1.570796326794896558 0 -> xyz=0 -0.025300000000000003042 -0.052000000000000032307 rpy=1.5707963267949045516 1.570796326794896558 0
- joint right_wrist_roll: origin xyz=0.019000000000002986722 -3.580650775880656056e-10 -0.027000000152453820096 rpy=-3.1415926535897797933 -1.5707963267947695485 0 -> xyz=0.019000000000002986722 -3.5806504983248998997e-10 -0.027000000152453823565 rpy=-3.1415926535897797933 -1.5707963267947699926 0
- joint right_wrist_roll_fixed: origin xyz=0.015500000000002378195 7.6882944455292090424e-15 -0.045000000000006055989 rpy=-4.8017145823115539524e-14 1.2051470932306250951e-13 -1.570796326794896558 -> xyz=0.015500000000002378195 7.7160500211448379559e-15 -0.045000000000006055989 rpy=-4.8017145823115337576e-14 1.2051470932306253475e-13 -1.570796326794896558
- joint waist_act_1: origin xyz=-4.3158571269690260163e-16 -0.019600000000000134676 0.012750000000000493577 rpy=-1.5707963267948961139 -1.5707963267948088504 0 -> xyz=4.6183233744605796308e-18 0.019599999999999964673 -0.012749999999999978365 rpy=-1.570796326794896336 1.1669078612757080027 -3.1415926535897904515
- joint waist_act_2: origin xyz=-5.8109383000701193055e-16 -0.019600000000000120798 0.03275000000000045236 rpy=-1.5707963267948927832 -1.3463968515393145431 1.0161280646543158659e-14 -> xyz=9.335172205065111088e-18 0.01959999999999997855 -0.032750000000000001332 rpy=-1.5707963267948990005 0.94250838602002218192 3.1415926535897860106
- joint waist_roll: origin xyz=-1.2306064131348466017e-19 0.022707865260692457893 -0.013000000000000011546 rpy=1.5707963267948952257 -4.14087346736882539e-15 4.2181022606674638269e-16 -> xyz=9.4639684746659082843e-19 -0.022707865260692291359 0.012999999999999997669 rpy=1.5707963267948985564 -4.8988590961582989196e-15 1.01240703429886086e-14
- joint waist_yaw: origin xyz=0 -3.9443045261050590271e-31 0 rpy=2.0946901476026454934e-15 7.1861600448342810266e-16 -1.5707963267948101826 -> xyz=0 2.168404344971008868e-19 1.7347234759768070944e-18 rpy=-3.1415926535897926719 3.3306690738754839194e-16 -1.5056527786227653642

Commit message: Update the robot description

File: toddlerbot/robot_descriptions/assemblies/left_arm_hand/left_arm_hand.urdf (robot description, URDF)
Before this commit: robot left_arm_hand, 14 links, 13 joints
Links:
- link elb_yaw_link: mass 0.017500000000000005135 -> 0.017500000000000001665
- link hand: mass 0.01700000000000000816 -> 0.017000000000001441042
- link sho_pitch_link: mass 0.0085999999999999948014 -> 0.0086000000000000000056
- link sho_yaw_link: mass 0.014500000000000014613 -> 0.014500000000000019817
- link wrist_bearing_plate: mass 0.0049000367468305548388 -> 0.0049000367468305539714

File: toddlerbot/robot_descriptions/assemblies/left_leg_XM430/left_leg_XM430.urdf (robot description, URDF)
Before this commit: robot left_leg_XM430, 18 links, 17 joints
Links:
- removed link left_sole_link
- link ank_motor_arm: mass 0.0020595846677894939954 -> 0.0021359401157891211472
- link ank_motor_arm_2: mass 0.0020595846677894939954 -> 0.0021359401157891211472
- link ank_pitch_link: mass 0.0042238381753791614387 -> 0.0042238381753791605713
- link ank_roll_link: mass 0.012900000000000000008 -> 0.019499999999999989564
- link ank_rr_link: mass 0.0014499999999999999001 -> 0.0014500000000000001169
- link ank_rr_link_2: mass 0.0014499999999999999001 -> 0.0014500000000000001169
- link hip_roll_link: mass 0.11059999999836234164 -> 0.11059999999836236939
- link hip_yaw_link: mass 0.017999999999999991701 -> 0.017999999999999995171
- link left_hip_pitch_link_xm430: mass 0.11480090135030567022 -> 0.1148009013503056841
- link xm430_plate: mass 0.0027000000000000001429 -> 0.0026999999999999992756
Joints:
- removed joint left_sole

File: toddlerbot/robot_descriptions/assemblies/right_arm_hand/right_arm_hand.urdf (robot description, URDF)
Before this commit: robot right_arm_hand, 14 links, 13 joints
Links:
- link elb_yaw_link: mass 0.017500000000000005135 -> 0.017500000000000001665
- link hand: mass 0.01700000000000000816 -> 0.017000000000001441042
- link sho_pitch_link: mass 0.0085999999999999948014 -> 0.0086000000000000000056
- link sho_yaw_link: mass 0.014500000000000014613 -> 0.014500000000000019817
- link wrist_bearing_plate: mass 0.0049000367468305548388 -> 0.0049000367468305539714

File: toddlerbot/robot_descriptions/assemblies/right_leg_XM430/right_leg_XM430.urdf (robot description, URDF)
Before this commit: robot right_leg_XM430, 18 links, 17 joints
Links:
- removed link right_sole_link
- link ank_motor_arm: mass 0.0020595846677894939954 -> 0.0021359401157891211472
- link ank_motor_arm_2: mass 0.0020595846677894939954 -> 0.0021359401157891211472
- link ank_pitch_link: mass 0.0042238381753791614387 -> 0.0042238381753791605713
- link ank_roll_link: mass 0.012900000000000000008 -> 0.019499999999999989564
- link ank_rr_link: mass 0.0014499999999999999001 -> 0.0014500000000000001169
- link ank_rr_link_2: mass 0.0014499999999999999001 -> 0.0014500000000000001169
- link hip_roll_link: mass 0.11059999999836234164 -> 0.11059999999836236939
- link hip_yaw_link: mass 0.017999999999999991701 -> 0.017999999999999995171
- link right_calf_link: mass 0.086799999986183568046 -> 0.086799999986183581924
- link xm430_plate: mass 0.0027000000000000001429 -> 0.0026999999999999992756
Joints:
- removed joint right_sole

File: toddlerbot/robot_descriptions/assemblies/toddlerbot/toddlerbot.urdf (robot description, URDF)
Before this commit: robot toddlerbot, 17 links, 16 joints
Links:
- link left_arm_hand: mass 0.0085999999999999965361 -> 0.0085999999999999930667
- link neck_pitch_link: mass 0.11211553874797881847 -> 0.11211553874797880459
- link right_arm_hand: mass 0.0085999999999999965361 -> 0.0085999999999999930667
- link spiral_bevel_1m_14t_30deg: mass 0.00067997563436136246491 -> 0.00067997563436136257333
- link spiral_bevel_1m_14t_30deg_2: mass 0.00067997563436136246491 -> 0.00067997563436136257333
- link spur_1m_20t: mass 0.0015534950290892282111 -> 0.0015534950290892286448
- link spur_gear_(13_teeth): mass 0.00081469437497230876716 -> 0.00081469437497230865874
- link waist_link: mass 0.16631953490612463864 -> 0.16631953490612461088
Joints:
- joint right_hip_yaw_drive: origin xyz=0.037000000000001108391 0.037100000000003796607 -0.039500000000000472233 rpy=-1.5707963267950055819 -5.5860638843048369188e-13 -3.8568016358434373564e-13 -> xyz=0.037000000000001094513 0.037100000000003796607 -0.039500000000000465294 rpy=-1.5707963267950058039 -5.5821781037186488709e-13 -3.8561893124432213586e-13

File: toddlerbot/robot_descriptions/toddlerbot/toddlerbot.urdf (robot description, URDF)
Before this commit: robot toddlerbot, 77 links, 76 joints
Links:
- removed link left_sole_link
- removed link right_sole_link
- link ank_motor_arm: mass 0.0020595846677894939954 -> 0.0021359401157891211472
- link ank_motor_arm_2: mass 0.0020595846677894939954 -> 0.0021359401157891211472
- link ank_motor_arm_3: mass 0.0020595846677894939954 -> 0.0021359401157891211472
- link ank_motor_arm_4: mass 0.0020595846677894939954 -> 0.0021359401157891211472
- link ank_pitch_link: mass 0.0042238381753791614387 -> 0.0042238381753791605713
- link ank_pitch_link_2: mass 0.0042238381753791614387 -> 0.0042238381753791605713
- link ank_roll_link: mass 0.012900000000000000008 -> 0.019499999999999989564; geometry collision mesh filename=collisions/left_ank_roll_link_collision.stl; visual mesh filename=../assemblies/left_leg_XM430/meshes/left_ank_roll_link_visu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
- link ank_roll_link_2: mass 0.012900000000000000008 -> 0.019499999999999989564; geometry collision mesh filename=collisions/right_ank_roll_link_collision.stl; visual mesh filename=../assemblies/right_leg_XM430/meshes/right_ank_roll_link_vi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
- link ank_rr_link: mass 0.0014499999999999999001 -> 0.0014500000000000001169
- link ank_rr_link_2: mass 0.0014499999999999999001 -> 0.0014500000000000001169
- link ank_rr_link_3: mass 0.0014499999999999999001 -> 0.0014500000000000001169
- link ank_rr_link_4: mass 0.0014499999999999999001 -> 0.0014500000000000001169
- link elb_yaw_link: mass 0.017500000000000005135 -> 0.017500000000000001665
- link elb_yaw_link_2: mass 0.017500000000000005135 -> 0.017500000000000001665
- link hand: mass 0.01700000000000000816 -> 0.017000000000001441042
- link hand_2: mass 0.01700000000000000816 -> 0.017000000000001441042
- link hip_roll_link: mass 0.11059999999836234164 -> 0.11059999999836236939
- link hip_roll_link_2: mass 0.11059999999836234164 -> 0.11059999999836236939
- link hip_yaw_link: mass 0.017999999999999991701 -> 0.017999999999999995171
- link hip_yaw_link_2: mass 0.017999999999999991701 -> 0.017999999999999995171
- link left_hip_pitch_link_xm430: mass 0.11480090135030567022 -> 0.1148009013503056841
- link neck_pitch_link: mass 0.11211553874797881847 -> 0.11211553874797880459
- link right_calf_link: mass 0.086799999986183568046 -> 0.086799999986183581924
- link sho_pitch_link: mass 0.0085999999999999948014 -> 0.0086000000000000000056
- link sho_pitch_link_2: mass 0.0085999999999999948014 -> 0.0086000000000000000056
- link sho_yaw_link: mass 0.014500000000000014613 -> 0.014500000000000019817
- link sho_yaw_link_2: mass 0.014500000000000014613 -> 0.014500000000000019817
- link spiral_bevel_1m_14t_30deg: mass 0.00067997563436136246491 -> 0.00067997563436136257333
- link spiral_bevel_1m_14t_30deg_2: mass 0.00067997563436136246491 -> 0.00067997563436136257333
- link spur_1m_20t: mass 0.0015534950290892282111 -> 0.0015534950290892286448
- link spur_gear_(13_teeth): mass 0.00081469437497230876716 -> 0.00081469437497230865874
- link waist_link: mass 0.16631953490612463864 -> 0.16631953490612461088
- link wrist_bearing_plate: mass 0.0049000367468305548388 -> 0.0049000367468305539714
- link wrist_bearing_plate_2: mass 0.0049000367468305548388 -> 0.0049000367468305539714
- link xm430_plate: mass 0.0027000000000000001429 -> 0.0026999999999999992756
- link xm430_plate_2: mass 0.0027000000000000001429 -> 0.0026999999999999992756
Joints:
- removed joint left_sole
- removed joint right_sole
- joint right_hip_yaw_drive: origin xyz=0.037000000000001108391 0.037100000000003796607 -0.039500000000000472233 rpy=-1.5707963267950055819 -5.5860638843048369188e-13 -3.8568016358434373564e-13 -> xyz=0.037000000000001094513 0.037100000000003796607 -0.039500000000000465294 rpy=-1.5707963267950058039 -5.5821781037186488709e-13 -3.8561893124432213586e-13
