Commit message: Update toddlerbot arms

File: toddlerbot/robot_descriptions/assemblies/left_arm_hand/left_arm_hand.urdf (robot description, URDF)
Before this commit: robot left_arm_hand, 14 links, 13 joints
Links:
- link 2xl430_gears: mass 0.11800003674524910113 -> 0.11800003674524907338
- link 2xl430_gears_2: mass 0.11800003674524910113 -> 0.11800003674524907338
- link 2xl430_gears_3: mass 0.11800003674524910113 -> 0.11800003674524907338
- link elb_yaw_link: mass 0.017500000000000001665 -> 0.017499999999999998196
- link sho_pitch_link: mass 0.0086000000000000017403 -> 0.0085999999999999930667
- link sho_yaw_link: mass 0.014500000000000007674 -> 0.014500000000000011144
- link spur_1m_24t_driven: mass 0.0027000000000000001429 -> 0.0026999999999999997093
- link spur_1m_24t_driven_2: mass 0.0027000000000000001429 -> 0.0026999999999999997093
- link spur_1m_24t_driven_3: mass 0.0027000000000000001429 -> 0.0026999999999999997093
- link wrist_bearing_plate: mass 0.0049000367468305548388 -> 0.0049000367468305539714

File: toddlerbot/robot_descriptions/assemblies/right_arm_hand/right_arm_hand.urdf (robot description, URDF)
Before this commit: robot right_arm_hand, 14 links, 13 joints
Links:
- link 2xl430_gears: mass 0.11800003674524910113 -> 0.11800003674524907338
- link 2xl430_gears_2: mass 0.11800003674524910113 -> 0.11800003674524907338
- link 2xl430_gears_3: mass 0.11800003674524910113 -> 0.11800003674524907338
- link elb_yaw_link: mass 0.017500000000000001665 -> 0.017499999999999998196
- link sho_pitch_link: mass 0.0086000000000000017403 -> 0.0085999999999999930667
- link sho_yaw_link: mass 0.014500000000000007674 -> 0.014500000000000011144
- link spur_1m_24t_driven: mass 0.0027000000000000001429 -> 0.0026999999999999997093
- link spur_1m_24t_driven_2: mass 0.0027000000000000001429 -> 0.0026999999999999997093
- link spur_1m_24t_driven_3: mass 0.0027000000000000001429 -> 0.0026999999999999997093
- link wrist_bearing_plate: mass 0.0049000367468305548388 -> 0.0049000367468305539714

File: toddlerbot/robot_descriptions/assemblies/toddlerbot_arms/toddlerbot_arms.urdf (robot description, URDF)
Before this commit: robot toddlerbot_arms, 3 links, 2 joints
Links:
- link left_arm_hand: mass 0.0085999999999999965361 -> 0.0085999999999999948014
- link right_arm_hand: mass 0.0085999999999999965361 -> 0.0085999999999999948014
- link torso: mass 0.60012685450989189384 -> 0.66652685450988358173

File: toddlerbot/robot_descriptions/toddlerbot_arms/toddlerbot_arms.urdf (robot description, URDF)
Before this commit: robot toddlerbot_arms, 29 links, 28 joints
Links:
- link 2xl430_gears: mass 0.11800003674524910113 -> 0.11800003674524907338
- link 2xl430_gears_2: mass 0.11800003674524910113 -> 0.11800003674524907338
- link 2xl430_gears_3: mass 0.11800003674524910113 -> 0.11800003674524907338
- link 2xl430_gears_4: mass 0.11800003674524910113 -> 0.11800003674524907338
- link 2xl430_gears_5: mass 0.11800003674524910113 -> 0.11800003674524907338
- link 2xl430_gears_6: mass 0.11800003674524910113 -> 0.11800003674524907338
- link elb_yaw_link: mass 0.017500000000000001665 -> 0.017499999999999998196
- link elb_yaw_link_2: mass 0.017500000000000001665 -> 0.017499999999999998196
- link sho_pitch_link: mass 0.0086000000000000017403 -> 0.0085999999999999930667
- link sho_pitch_link_2: mass 0.0086000000000000017403 -> 0.0085999999999999930667
- link sho_yaw_link: mass 0.014500000000000007674 -> 0.014500000000000011144
- link sho_yaw_link_2: mass 0.014500000000000007674 -> 0.014500000000000011144
- link spur_1m_24t_driven: mass 0.0027000000000000001429 -> 0.0026999999999999997093
- link spur_1m_24t_driven_2: mass 0.0027000000000000001429 -> 0.0026999999999999997093
- link spur_1m_24t_driven_3: mass 0.0027000000000000001429 -> 0.0026999999999999997093
- link spur_1m_24t_driven_4: mass 0.0027000000000000001429 -> 0.0026999999999999997093
- link spur_1m_24t_driven_5: mass 0.0027000000000000001429 -> 0.0026999999999999997093
- link spur_1m_24t_driven_6: mass 0.0027000000000000001429 -> 0.0026999999999999997093
- link torso: mass 0.60012685450989189384 -> 0.66652685450988358173
- link wrist_bearing_plate: mass 0.0049000367468305548388 -> 0.0049000367468305539714
- link wrist_bearing_plate_2: mass 0.0049000367468305548388 -> 0.0049000367468305539714
