Commit message: Fix left_wrist_roll direction

File: toddlerbot/robot_descriptions/assemblies/left_arm_umi/left_arm_umi.urdf (robot description, URDF)
Before this commit: robot left_arm_umi, 14 links, 13 joints
Links:
- link elb_yaw_link: mass 0.017499999999999998196 -> 0.017500000000000008604
- link hand: mass 0.03949999999999999345 -> 0.039499999999999979572
- link sho_pitch_link: mass 0.0085999999999999948014 -> 0.0086000000000000017403
- link sho_yaw_link: mass 0.01450000000000000594 -> 0.014500000000000016348
- link spur_1m_24t_drive: mass 0.0032000000000000001533 -> 0.003199999999999999286
- link spur_1m_24t_drive_2: mass 0.0032000000000000001533 -> 0.003199999999999999286
- link spur_1m_24t_drive_3: mass 0.0032000000000000001533 -> 0.003199999999999999286
- link spur_1m_24t_driven: mass 0.0027000000000000001429 -> 0.0026999999999999997093
- link spur_1m_24t_driven_2: mass 0.0027000000000000001429 -> 0.0026999999999999997093
- link spur_1m_24t_driven_3: mass 0.0027000000000000001429 -> 0.0026999999999999997093
- link wrist_bearing_plate: mass 0.0049000367468305557062 -> 0.0049000367468305565735
Joints:
- joint left_elbow_roll: origin xyz=1.17614251671227521e-15 -0.019000000000000002998 -0.05900000000000006628 rpy=1.5707963267948954478 -1.8257447566372568016e-14 -1.7593846109850829682e-16 -> xyz=2.0816681711721685133e-16 -0.019000000000000002998 -0.059000000000000059341 rpy=1.570796326794896558 -8.2694607970959069176e-16 -2.2204460490005989148e-16
- joint left_elbow_yaw_drive: origin xyz=-0.024000000716137517842 -0.0190000001524475437 -0.019000000152459544517 rpy=1.5707963267950562081 -2.4622204840090993627e-13 -1.7925499053412602242e-13 -> xyz=-0.024000000716137528251 -0.019000000152447529822 -0.019000000152459547986 rpy=1.570796326795050879 -2.4708842848455862195e-13 -6.0621939164177121919e-14
- joint left_elbow_yaw_driven: origin xyz=-3.5806394307891231676e-10 -0.027000000152452990898 -0.0190000000000065776 rpy=1.5707963267949589525 1.5707963267946882802 0 -> xyz=-3.5806398471227574021e-10 -0.027000000152453157432 -0.0190000000000067025 rpy=1.5707963267949571762 1.5707963267947377961 0
- joint left_elbow_yaw_fixed: origin xyz=1.5777218104420236108e-30 0 0.0015999999999999764411 rpy=-3.141592653589793116 -4.4866451871279772575e-27 -3.2816870322621037337e-28 -> xyz=1.5777218104420236108e-30 0 0.0015999999999999903189 rpy=-3.141592653589793116 6.8585119145426910438e-26 -7.6666465467942038555e-26
- joint left_sho_roll: origin xyz=-0.018999999999999999528 0.00099999999999999546717 0.027000000000000006634 rpy=-3.141592653589793116 1.5707963267948956698 0 -> xyz=-0.018999999999999999528 0.00099999999999997161472 0.026999999999999999695 rpy=-3.141592653589793116 1.5707963267948936714 0
- joint left_sho_yaw_drive: origin xyz=-0.024000000716140966472 -0.019000000152450589874 -0.019000000152443286688 rpy=1.5707963267948328312 -1.3331515362498170811e-15 8.2000365474799924889e-14 -> xyz=-0.024000000716141004636 -0.019000000152450596813 -0.019000000152443286688 rpy=1.5707963267948328312 -1.2258104172924911424e-15 7.6362147953450801566e-14
- joint left_sho_yaw_driven: origin xyz=-3.5807029563628134383e-10 -0.027000000152450926577 -0.018999999999999878098 rpy=1.5707963267948492625 7.9618117061828289905e-14 1.0047518372857611155e-13 -> xyz=-3.5807162096501699011e-10 -0.027000000152450989027 -0.01899999999999986075 rpy=1.5707963267948492625 8.0395273179087848749e-14 9.4924068605497912938e-14
- joint left_sho_yaw_fixed: origin xyz=-3.4694469519536141888e-18 0 0.0015999999999999972577 rpy=-3.1415926535897926719 -0 0 -> xyz=0 7.8886090522101180541e-31 0.0015999999999999868494 rpy=-3.1415926535897917837 7.7715611727616959238e-16 7.7715611725338728944e-16
- joint left_wrist_pitch_drive: origin xyz=-1.5244060454932555774e-10 0.024000000358057271832 -0.0080000000000068835493 rpy=3.6254446097225608906e-14 -2.2096785867264433738e-13 -1.5707963267949176522 -> xyz=-1.524411552671568168e-10 0.024000000358058659611 -0.0080000000000068835493 rpy=9.3688120281041050571e-15 -2.4754138690627644039e-13 -1.570796326794971387
- joint left_wrist_pitch_driven: origin xyz=-2.7755575615628913511e-17 -1.5777218104420236108e-30 -0.0015999999999999979083 rpy=-8.9315741575089004617e-15 -8.8817841970012507457e-15 -1.570796326794896558 -> xyz=2.7755575615628913511e-17 -1.5777218104420236108e-30 -0.0015999999999999974746 rpy=-2.6917187154893159429e-14 -2.6645352591003750659e-14 -1.570796326794896558
- joint left_wrist_pitch_fixed: origin xyz=0.015500000000007816553 -1.8068879725774422695e-14 -0.044999999999998901989 rpy=4.0745185003716278612e-14 -2.8213542612434270497e-13 -1.570796326794906328 -> xyz=0.015500000000007499099 -1.7430501486614957685e-14 -0.044999999999998915867 rpy=4.0578651550042264519e-14 -2.8213542612434331081e-13 -1.570796326794906328
- joint left_wrist_roll: origin xyz=0.019000000000007049444 -3.5808095377731774533e-10 -0.027000000152448057344 rpy=-7.3828629579122985512e-14 -1.5707963267945765917 0 -> xyz=0.019000000000007889051 -3.5808161991113252043e-10 -0.027000000152448057344 rpy=3.141592653589793116 -1.5707963267945475039 0
- joint left_wrist_roll_fixed: origin xyz=0 -0.025299999999999999573 -0.051999999999999962919 rpy=1.5707963267949056618 -1.5707963267948876762 0 -> xyz=0 -0.025300000000000003042 -0.05200000000000001843 rpy=1.5707963267949236474 -1.5707963267948696906 0

File: toddlerbot/robot_descriptions/toddlerbot_OP3/toddlerbot_OP3.urdf (robot description, URDF)
Before this commit: robot toddlerbot_OP3, 63 links, 62 joints
Links:
- link elb_yaw_link: mass 0.017499999999999998196 -> 0.017500000000000008604
- link hand: mass 0.03949999999999999345 -> 0.039499999999999979572
- link sho_pitch_link: mass 0.0085999999999999948014 -> 0.0086000000000000017403
- link sho_yaw_link: mass 0.01450000000000000594 -> 0.014500000000000016348
- link spur_1m_24t_drive: mass 0.0032000000000000001533 -> 0.003199999999999999286
- link spur_1m_24t_drive_2: mass 0.0032000000000000001533 -> 0.003199999999999999286
- link spur_1m_24t_drive_3: mass 0.0032000000000000001533 -> 0.003199999999999999286
- link spur_1m_24t_driven: mass 0.0027000000000000001429 -> 0.0026999999999999997093
- link spur_1m_24t_driven_2: mass 0.0027000000000000001429 -> 0.0026999999999999997093
- link spur_1m_24t_driven_3: mass 0.0027000000000000001429 -> 0.0026999999999999997093
- link wrist_bearing_plate: mass 0.0049000367468305557062 -> 0.0049000367468305565735
Joints:
- joint left_elbow_roll: origin xyz=1.17614251671227521e-15 -0.019000000000000002998 -0.05900000000000006628 rpy=1.5707963267948954478 -1.8257447566372568016e-14 -1.7593846109850829682e-16 -> xyz=2.0816681711721685133e-16 -0.019000000000000002998 -0.059000000000000059341 rpy=1.570796326794896558 -8.2694607970959069176e-16 -2.2204460490005989148e-16
- joint left_elbow_yaw_drive: origin xyz=-0.024000000716137517842 -0.0190000001524475437 -0.019000000152459544517 rpy=1.5707963267950562081 -2.4622204840090993627e-13 -1.7925499053412602242e-13 -> xyz=-0.024000000716137528251 -0.019000000152447529822 -0.019000000152459547986 rpy=1.570796326795050879 -2.4708842848455862195e-13 -6.0621939164177121919e-14
- joint left_elbow_yaw_driven: origin xyz=-3.5806394307891231676e-10 -0.027000000152452990898 -0.0190000000000065776 rpy=1.5707963267949589525 1.5707963267946882802 0 -> xyz=-3.5806398471227574021e-10 -0.027000000152453157432 -0.0190000000000067025 rpy=1.5707963267949571762 1.5707963267947377961 0
- joint left_elbow_yaw_fixed: origin xyz=1.5777218104420236108e-30 0 0.0015999999999999764411 rpy=-3.141592653589793116 -4.4866451871279772575e-27 -3.2816870322621037337e-28 -> xyz=1.5777218104420236108e-30 0 0.0015999999999999903189 rpy=-3.141592653589793116 6.8585119145426910438e-26 -7.6666465467942038555e-26
- joint left_sho_roll: origin xyz=-0.018999999999999999528 0.00099999999999999546717 0.027000000000000006634 rpy=-3.141592653589793116 1.5707963267948956698 0 -> xyz=-0.018999999999999999528 0.00099999999999997161472 0.026999999999999999695 rpy=-3.141592653589793116 1.5707963267948936714 0
- joint left_sho_yaw_drive: origin xyz=-0.024000000716140966472 -0.019000000152450589874 -0.019000000152443286688 rpy=1.5707963267948328312 -1.3331515362498170811e-15 8.2000365474799924889e-14 -> xyz=-0.024000000716141004636 -0.019000000152450596813 -0.019000000152443286688 rpy=1.5707963267948328312 -1.2258104172924911424e-15 7.6362147953450801566e-14
- joint left_sho_yaw_driven: origin xyz=-3.5807029563628134383e-10 -0.027000000152450926577 -0.018999999999999878098 rpy=1.5707963267948492625 7.9618117061828289905e-14 1.0047518372857611155e-13 -> xyz=-3.5807162096501699011e-10 -0.027000000152450989027 -0.01899999999999986075 rpy=1.5707963267948492625 8.0395273179087848749e-14 9.4924068605497912938e-14
- joint left_sho_yaw_fixed: origin xyz=-3.4694469519536141888e-18 0 0.0015999999999999972577 rpy=-3.1415926535897926719 -0 0 -> xyz=0 7.8886090522101180541e-31 0.0015999999999999868494 rpy=-3.1415926535897917837 7.7715611727616959238e-16 7.7715611725338728944e-16
- joint left_wrist_pitch_drive: origin xyz=-1.5244060454932555774e-10 0.024000000358057271832 -0.0080000000000068835493 rpy=3.6254446097225608906e-14 -2.2096785867264433738e-13 -1.5707963267949176522 -> xyz=-1.524411552671568168e-10 0.024000000358058659611 -0.0080000000000068835493 rpy=9.3688120281041050571e-15 -2.4754138690627644039e-13 -1.570796326794971387
- joint left_wrist_pitch_driven: origin xyz=-2.7755575615628913511e-17 -1.5777218104420236108e-30 -0.0015999999999999979083 rpy=-8.9315741575089004617e-15 -8.8817841970012507457e-15 -1.570796326794896558 -> xyz=2.7755575615628913511e-17 -1.5777218104420236108e-30 -0.0015999999999999974746 rpy=-2.6917187154893159429e-14 -2.6645352591003750659e-14 -1.570796326794896558
- joint left_wrist_pitch_fixed: origin xyz=0.015500000000007816553 -1.8068879725774422695e-14 -0.044999999999998901989 rpy=4.0745185003716278612e-14 -2.8213542612434270497e-13 -1.570796326794906328 -> xyz=0.015500000000007499099 -1.7430501486614957685e-14 -0.044999999999998915867 rpy=4.0578651550042264519e-14 -2.8213542612434331081e-13 -1.570796326794906328
- joint left_wrist_roll: origin xyz=0.019000000000007049444 -3.5808095377731774533e-10 -0.027000000152448057344 rpy=-7.3828629579122985512e-14 -1.5707963267945765917 0 -> xyz=0.019000000000007889051 -3.5808161991113252043e-10 -0.027000000152448057344 rpy=3.141592653589793116 -1.5707963267945475039 0
- joint left_wrist_roll_fixed: origin xyz=0 -0.025299999999999999573 -0.051999999999999962919 rpy=1.5707963267949056618 -1.5707963267948876762 0 -> xyz=0 -0.025300000000000003042 -0.05200000000000001843 rpy=1.5707963267949236474 -1.5707963267948696906 0
