Commit message: Update the mujoco env

File: toddlerbot/robot_descriptions/assemblies/toddlerbot/toddlerbot.urdf (robot description, URDF)
Before this commit: robot toddlerbot, 17 links, 16 joints
Links:
- removed link spiral_bevel_1m_14t_30deg
- removed link spiral_bevel_1m_14t_30deg_2
- link left_arm_hand: mass 0.0085999999999999930667 -> 0.0085999999999999965361
- link neck_pitch_link: mass 0.11211553874797880459 -> 0.11211553874797881847
- link right_arm_hand: mass 0.0085999999999999930667 -> 0.0085999999999999965361
- link torso: mass 0.58490521749923585215 -> 0.58475267652546303321
- link waist_gears: mass 0.023315805669179824611 -> 0.025809950030454161668
- link waist_link: mass 0.16631953490612461088 -> 0.16767948617484731977
Joints:
- removed joint waist_act_1
- removed joint waist_act_2
- joint left_hip_yaw_drive: origin xyz=-0.036999999999998325895 0.03710000000000578807 -0.0395000000000009302 rpy=-1.5707963267950055819 -5.5860808452836958954e-13 -3.9012105568284431132e-13 -> xyz=-0.036999999999998312017 0.037100000000006030931 -0.0395000000000006804 rpy=-1.5707963267949798247 -4.6304776107371661452e-13 -3.868919074001414487e-13
- joint left_hip_yaw_driven: origin xyz=-0.03699999999999998429 0.041100000000000004585 -0.019499999999999979156 rpy=-1.5707963267948983344 -1.570796326794896558 0 -> xyz=-0.037000000000000005107 0.041099999999999997646 -0.019499999999999979156 rpy=-1.5707963267948923392 -1.5707963267948932273 0
- joint left_leg_fixed: origin xyz=-7.3725747729014301513e-18 -6.9388939039072283776e-18 0.004999999999999997502 rpy=-3.141592653589793116 1.9721522630525295135e-31 -1.1102230246249028723e-16 -> xyz=-4.336808689942017736e-19 0 0.004999999999999997502 rpy=3.1415926535897851224 -1.1045608006607374766e-30 -4.2552910532817472121e-31
- joint left_sho_pitch: origin xyz=-0.0029999999999997528644 0.062000000000000436706 0.10523651076281793915 rpy=-1.5707963267948983344 8.0214786879603172751e-16 1.532501625198463655e-15 -> xyz=-0.0030000000000067082381 0.062000000000004690248 0.10423651076282114403 rpy=-1.5707963267949092145 -3.6755753074147472872e-14 3.4347079465292731775e-14
- joint neck_pitch_drive: origin xyz=-1.1692036228083679816e-15 0.01565000000000066338 -0.0087999999999981218246 rpy=1.2246467991513517459e-16 -6.1232339957502284403e-17 -1.5707963267949054398 -> xyz=-1.7971735211119721498e-15 0.015649999999999192335 -0.008799999999996657718 rpy=-9.1684649781985877855e-16 7.2823649231784177849e-17 -1.5707963267948912289
- joint neck_pitch_driven: origin xyz=3.7499999980261655708e-10 -0.0051500000614753986203 0.027500000000000010547 rpy=1.570796326794896558 8.661048429666698261e-16 3.1415926535897926719 -> xyz=3.7499998592482874926e-10 -0.0051500000614754029571 0.027499999999999941158 rpy=1.570796326794896336 8.6610484296623782615e-16 3.1415926535897926719
- joint neck_yaw_drive: origin xyz=-0.0049999999999990590166 -1.7787571338323640394e-16 0.12248651076281813488 rpy=1.900955487881492792e-15 1.6770488781412432481e-15 9.8514697225632145493e-16 -> xyz=-0.0050000000000043915566 2.1780059937422389857e-15 0.12148651076282247774 rpy=-4.6722658561527960149e-15 -3.0241828739332580702e-14 3.0478935990547233347e-14
- joint neck_yaw_driven: origin xyz=0.016000000000001790568 1.3355656282555062267e-17 0.12348651076281798311 rpy=5.2022234352156643924e-17 -1.693050922709124266e-15 -3.1415926535897926719 -> xyz=0.015999999999998633371 3.2287696509065600056e-15 0.12248651076282091044 rpy=2.3436576345318096491e-14 3.3282183470283369239e-14 -3.1415926535897926719
- joint right_hip_yaw_drive: origin xyz=0.037000000000001094513 0.037100000000003796607 -0.039500000000000465294 rpy=-1.5707963267950058039 -5.5821781037186488709e-13 -3.8561893124432213586e-13 -> xyz=0.037000000000001607992 0.037100000000003560685 -0.039500000000000486111 rpy=-1.5707963267949798247 -4.6304330256338374643e-13 -3.8689190740014134773e-13
- joint right_hip_yaw_driven: origin xyz=0.036999999999999998168 0.041100000000000011524 -0.019499999999999979156 rpy=-1.5707963267949129893 -1.570796326794896558 0 -> xyz=0.037000000000000005107 0.041099999999999997646 -0.019499999999999986094 rpy=-1.5707963267949132113 -1.5707963267948950037 0
- joint right_leg_fixed: origin xyz=6.9388939039072283776e-18 0 0.004999999999999997502 rpy=-3.1415926535897784611 1.8262365126862931582e-15 -3.6959871191238926143e-16 -> xyz=0 0 0.004999999999999997502 rpy=-3.1415926535897797933 -7.5781949123851955204e-18 -3.340101530512157196e-16
- joint right_sho_pitch: origin xyz=-0.0030000000000001275646 -0.061999999999999985678 0.10523651076281731465 rpy=-1.570796326794896558 -6.5632891966464542239e-16 -3.1415926535897917837 -> xyz=-0.0030000000000024208691 -0.061999999999999777511 0.10423651076282194894 rpy=-1.5707963267948847896 2.9071281258321823756e-14 -3.1415926535897589211
- joint waist_roll: origin xyz=-5.6460850897507995335e-16 -0.022707865260693318316 0.012999999999999227451 rpy=1.57079632679489678 9.8097267041675110992e-15 1.1042194747589474972e-14 -> xyz=-0.022707865260692145642 -3.2904492237211951884e-18 -0.014000000000000064476 rpy=-1.5707963267949034414 -6.2265052416776424318e-15 1.5707963267948885644
- joint waist_yaw: origin xyz=3.7643499428696713949e-16 3.9043635660773690095e-17 -3.1571967262777889118e-16 rpy=3.1415926535897917837 -1.9359568790009725236e-16 -1.57079632679489678 -> xyz=0 -4.3140830754274083108e-32 0 rpy=9.7872132923950749268e-15 4.0244775309734053704e-14 -3.1415926535897926719

File: toddlerbot/robot_descriptions/toddlerbot/toddlerbot.urdf (robot description, URDF)
Before this commit: robot toddlerbot, 75 links, 74 joints
Links:
- removed link spiral_bevel_1m_14t_30deg
- removed link spiral_bevel_1m_14t_30deg_2
- link neck_pitch_link: mass 0.11211553874797880459 -> 0.11211553874797881847
- link torso: mass 0.58490521749923585215 -> 0.58475267652546303321
- link waist_gears: mass 0.023315805669179824611 -> 0.025809950030454161668
- link waist_link: mass 0.16631953490612461088 -> 0.16767948617484731977
Joints:
- removed joint waist_act_1
- removed joint waist_act_2
- joint left_hip_yaw_drive: origin xyz=-0.036999999999998325895 0.03710000000000578807 -0.0395000000000009302 rpy=-1.5707963267950055819 -5.5860808452836958954e-13 -3.9012105568284431132e-13 -> xyz=-0.036999999999998312017 0.037100000000006030931 -0.0395000000000006804 rpy=-1.5707963267949798247 -4.6304776107371661452e-13 -3.868919074001414487e-13
- joint left_hip_yaw_driven: origin xyz=-0.03699999999999998429 0.041100000000000004585 -0.019499999999999979156 rpy=-1.5707963267948983344 -1.570796326794896558 0 -> xyz=-0.037000000000000005107 0.041099999999999997646 -0.019499999999999979156 rpy=-1.5707963267948923392 -1.5707963267948932273 0
- joint left_leg_fixed: origin xyz=-7.3725747729014301513e-18 -6.9388939039072283776e-18 0.004999999999999997502 rpy=-3.141592653589793116 1.9721522630525295135e-31 -1.1102230246249028723e-16 -> xyz=-4.336808689942017736e-19 0 0.004999999999999997502 rpy=3.1415926535897851224 -1.1045608006607374766e-30 -4.2552910532817472121e-31
- joint left_sho_pitch: origin xyz=-0.0029999999999997528644 0.062000000000000436706 0.10523651076281793915 rpy=-1.5707963267948983344 8.0214786879603172751e-16 1.532501625198463655e-15 -> xyz=-0.0030000000000067082381 0.062000000000004690248 0.10423651076282114403 rpy=-1.5707963267949092145 -3.6755753074147472872e-14 3.4347079465292731775e-14
- joint neck_pitch_drive: origin xyz=-1.1692036228083679816e-15 0.01565000000000066338 -0.0087999999999981218246 rpy=1.2246467991513517459e-16 -6.1232339957502284403e-17 -1.5707963267949054398 -> xyz=-1.7971735211119721498e-15 0.015649999999999192335 -0.008799999999996657718 rpy=-9.1684649781985877855e-16 7.2823649231784177849e-17 -1.5707963267948912289
- joint neck_pitch_driven: origin xyz=3.7499999980261655708e-10 -0.0051500000614753986203 0.027500000000000010547 rpy=1.570796326794896558 8.661048429666698261e-16 3.1415926535897926719 -> xyz=3.7499998592482874926e-10 -0.0051500000614754029571 0.027499999999999941158 rpy=1.570796326794896336 8.6610484296623782615e-16 3.1415926535897926719
- joint neck_yaw_drive: origin xyz=-0.0049999999999990590166 -1.7787571338323640394e-16 0.12248651076281813488 rpy=1.900955487881492792e-15 1.6770488781412432481e-15 9.8514697225632145493e-16 -> xyz=-0.0050000000000043915566 2.1780059937422389857e-15 0.12148651076282247774 rpy=-4.6722658561527960149e-15 -3.0241828739332580702e-14 3.0478935990547233347e-14
- joint neck_yaw_driven: origin xyz=0.016000000000001790568 1.3355656282555062267e-17 0.12348651076281798311 rpy=5.2022234352156643924e-17 -1.693050922709124266e-15 -3.1415926535897926719 -> xyz=0.015999999999998633371 3.2287696509065600056e-15 0.12248651076282091044 rpy=2.3436576345318096491e-14 3.3282183470283369239e-14 -3.1415926535897926719
- joint right_hip_yaw_drive: origin xyz=0.037000000000001094513 0.037100000000003796607 -0.039500000000000465294 rpy=-1.5707963267950058039 -5.5821781037186488709e-13 -3.8561893124432213586e-13 -> xyz=0.037000000000001607992 0.037100000000003560685 -0.039500000000000486111 rpy=-1.5707963267949798247 -4.6304330256338374643e-13 -3.8689190740014134773e-13
- joint right_hip_yaw_driven: origin xyz=0.036999999999999998168 0.041100000000000011524 -0.019499999999999979156 rpy=-1.5707963267949129893 -1.570796326794896558 0 -> xyz=0.037000000000000005107 0.041099999999999997646 -0.019499999999999986094 rpy=-1.5707963267949132113 -1.5707963267948950037 0
- joint right_leg_fixed: origin xyz=6.9388939039072283776e-18 0 0.004999999999999997502 rpy=-3.1415926535897784611 1.8262365126862931582e-15 -3.6959871191238926143e-16 -> xyz=0 0 0.004999999999999997502 rpy=-3.1415926535897797933 -7.5781949123851955204e-18 -3.340101530512157196e-16
- joint right_sho_pitch: origin xyz=-0.0030000000000001275646 -0.061999999999999985678 0.10523651076281731465 rpy=-1.570796326794896558 -6.5632891966464542239e-16 -3.1415926535897917837 -> xyz=-0.0030000000000024208691 -0.061999999999999777511 0.10423651076282194894 rpy=-1.5707963267948847896 2.9071281258321823756e-14 -3.1415926535897589211
- joint waist_roll: origin xyz=-5.6460850897507995335e-16 -0.022707865260693318316 0.012999999999999227451 rpy=1.57079632679489678 9.8097267041675110992e-15 1.1042194747589474972e-14 -> xyz=-0.022707865260692145642 -3.2904492237211951884e-18 -0.014000000000000064476 rpy=-1.5707963267949034414 -6.2265052416776424318e-15 1.5707963267948885644
- joint waist_yaw: origin xyz=3.7643499428696713949e-16 3.9043635660773690095e-17 -3.1571967262777889118e-16 rpy=3.1415926535897917837 -1.9359568790009725236e-16 -1.57079632679489678 -> xyz=0 -4.3140830754274083108e-32 0 rpy=9.7872132923950749268e-15 4.0244775309734053704e-14 -3.1415926535897926719
