Commit message: Update the collisions

File: toddlerbot/robot_descriptions/assemblies/toddlerbot/toddlerbot.urdf (robot description, URDF)
Before this commit: robot toddlerbot, 15 links, 14 joints
Links:
- added link spiral_bevel_1m_14t_30deg, mass 0.00067997563436136246491; collision mesh filename=package:///meshes/spiral_bevel_1m_14t_30deg_collision.stl; visual mesh filename=package:///meshes/spiral_bevel_1m_14t_30deg_visual.stl
- added link spiral_bevel_1m_14t_30deg_2, mass 0.00067997563436136246491; collision mesh filename=package:///meshes/spiral_bevel_1m_14t_30deg_2_collision.stl; visual mesh filename=package:///meshes/spiral_bevel_1m_14t_30deg_2_visual.stl
- link neck_yaw_link: mass 0.0085168305947458285143 -> 0.0085168305947458267796
- link spur_gear_19_teeth: mass 0.0010993711450650535313 -> 0.0010993711450650533144
- link spur_gear_19_teeth_2: mass 0.0010993711450650535313 -> 0.0010993711450650533144
- link spur_gear_21_teeth: mass 0.0010063046528317974842 -> 0.0010063046528317972673
- link spur_gear_21_teeth_2: mass 0.0010063046528317974842 -> 0.0010063046528317972673
- link torso: mass 0.58475267652546303321 -> 0.58475267652546314423
- link waist_gears: mass 0.025809950030454161668 -> 0.025809950030454158199
- link waist_link: mass 0.16767948617484731977 -> 0.16631953490612458313
Joints:
- added joint waist_act_1: type revolute, parent waist_link, child spiral_bevel_1m_14t_30deg, origin xyz=5.380496587145115132e-16 0.019600000000000075695 -0.012750000000000080713 rpy=1.5707963267949007768 1.5707963267948907848 0, axis 0 0 1, limit lower=-2.7825534678416246059 upper=2.7825534678416246059 effort=1 velocity=20
- added joint waist_act_2: type revolute, parent waist_link, child spiral_bevel_1m_14t_30deg_2, origin xyz=-2.6785082652000791162e-16 0.019599999999999902223 -0.032749999999999612754 rpy=1.5707963267948958919 1.3463968515392310543 -4.6125152814992733786e-14, axis 0 0 1, limit lower=-2.7825534678416246059 upper=2.7825534678416246059 effort=1 velocity=20
- joint left_hip_yaw_drive: origin xyz=-0.036999999999998312017 0.037100000000006030931 -0.0395000000000006804 rpy=-1.5707963267949798247 -4.6304776107371661452e-13 -3.868919074001414487e-13 -> xyz=-0.036999999999998194056 0.037100000000006128076 -0.039500000000001291023 rpy=-1.5707963267949545116 -4.7906511943294847217e-13 -3.592506663906207747e-13
- joint left_hip_yaw_driven: origin xyz=-0.037000000000000005107 0.041099999999999997646 -0.019499999999999979156 rpy=-1.5707963267948923392 -1.5707963267948932273 0 -> xyz=-0.037000000000000012046 0.041099999999999997646 -0.0194999999999999514 rpy=-1.5707963267948990005 -1.570796326794896558 0
- joint left_leg_fixed: origin xyz=-4.336808689942017736e-19 0 0.004999999999999997502 rpy=3.1415926535897851224 -1.1045608006607374766e-30 -4.2552910532817472121e-31 -> xyz=0 0 0.004999999999999997502 rpy=3.1415926535897873428 -0 -1.6681280046507162628e-30
- joint left_sho_pitch: origin xyz=-0.0030000000000067082381 0.062000000000004690248 0.10423651076282114403 rpy=-1.5707963267949092145 -3.6755753074147472872e-14 3.4347079465292731775e-14 -> xyz=-0.0030000000000065664245 0.062000000000004926171 0.10423651076282140771 rpy=-1.5707963267949054398 -3.6755753074147447628e-14 3.6857314245917344439e-14
- joint neck_pitch_drive: origin xyz=-1.7971735211119721498e-15 0.015649999999999192335 -0.008799999999996657718 rpy=-9.1684649781985877855e-16 7.2823649231784177849e-17 -1.5707963267948912289 -> xyz=-1.4224732503009818174e-16 0.015649999999999136824 -0.0087999999999959568897 rpy=-2.4492935983152098954e-16 -2.1427228763620856097e-15 -1.570796326794896558
- joint neck_pitch_driven: origin xyz=3.7499998592482874926e-10 -0.0051500000614754029571 0.027499999999999941158 rpy=1.570796326794896336 8.6610484296623782615e-16 3.1415926535897926719 -> xyz=3.7500001368040436489e-10 -0.0051500000614753682626 0.027499999999999830136 rpy=1.57079632679489678 1.7322096859329345721e-15 -3.1415926535897922278
- joint neck_yaw_drive: origin xyz=-0.0050000000000043915566 2.1780059937422389857e-15 0.12148651076282247774 rpy=-4.6722658561527960149e-15 -3.0241828739332580702e-14 3.0478935990547233347e-14 -> xyz=-0.0050000000000041591036 2.1706564040395755645e-15 0.12148651076282282468 rpy=-4.7086950490309927255e-15 -3.2377166610426843676e-14 2.947288666540578667e-14
- joint neck_yaw_driven: origin xyz=0.015999999999998633371 3.2287696509065600056e-15 0.12248651076282091044 rpy=2.3436576345318096491e-14 3.3282183470283369239e-14 -3.1415926535897926719 -> xyz=0.015999999999998446021 3.2990787509752002888e-15 0.12248651076282082717 rpy=2.3463681399312212716e-14 3.1845915227826135867e-14 3.141592653589793116
- joint right_hip_yaw_drive: origin xyz=0.037000000000001607992 0.037100000000003560685 -0.039500000000000486111 rpy=-1.5707963267949798247 -4.6304330256338374643e-13 -3.8689190740014134773e-13 -> xyz=0.037000000000001746769 0.037100000000003664768 -0.039500000000000978773 rpy=-1.5707963267949545116 -4.7905720692590075245e-13 -3.5747430955122047375e-13
- joint right_hip_yaw_driven: origin xyz=0.037000000000000005107 0.041099999999999997646 -0.019499999999999986094 rpy=-1.5707963267949132113 -1.5707963267948950037 0 -> xyz=0.036999999999999991229 0.041100000000000011524 -0.0194999999999999514 rpy=-1.5707963267949003328 -1.5707963267948956698 0
- joint right_leg_fixed: origin xyz=0 0 0.004999999999999997502 rpy=-3.1415926535897797933 -7.5781949123851955204e-18 -3.340101530512157196e-16 -> xyz=0 0 0.0050000000000000044409 rpy=-3.141592653589793116 -0 -9.3397966250929058941e-32
- joint right_sho_pitch: origin xyz=-0.0030000000000024208691 -0.061999999999999777511 0.10423651076282194894 rpy=-1.5707963267948847896 2.9071281258321823756e-14 -3.1415926535897589211 -> xyz=-0.0030000000000019676726 -0.062000000000000089762 0.10423651076282176853 rpy=-1.5707963267948885644 3.4812325502379109658e-14 -3.1415926535897562566
- joint waist_roll: origin xyz=-0.022707865260692145642 -3.2904492237211951884e-18 -0.014000000000000064476 rpy=-1.5707963267949034414 -6.2265052416776424318e-15 1.5707963267948885644 -> xyz=-0.022707865260691548898 -1.3479418671744790767e-17 -0.014000000000000234479 rpy=-1.5707963267949187625 -1.0371626905663003511e-14 1.5707963267948794606
- joint waist_yaw: origin xyz=0 -4.3140830754274083108e-32 0 rpy=9.7872132923950749268e-15 4.0244775309734053704e-14 -3.1415926535897926719 -> xyz=0 -9.8607613152626475676e-32 0 rpy=1.6626925279001758682e-14 4.9579962395338894532e-14 -3.1415926535897900074

File: toddlerbot/robot_descriptions/toddlerbot/toddlerbot.urdf (robot description, URDF)
Before this commit: robot toddlerbot, 73 links, 72 joints
Links:
- added link spiral_bevel_1m_14t_30deg, mass 0.00067997563436136246491; visual mesh filename=../assemblies/toddlerbot/meshes/spiral_bevel_1m_14t_30deg_v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
- added link spiral_bevel_1m_14t_30deg_2, mass 0.00067997563436136246491; visual mesh filename=../assemblies/toddlerbot/meshes/spiral_bevel_1m_14t_30deg_2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
- link 2xl430_gears_3: geometry visual mesh filename=../assemblies/left_arm_hand/meshes/left_2xl430_gears_3_visu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
- link 2xl430_gears_6: geometry visual mesh filename=../assemblies/right_arm_hand/meshes/right_2xl430_gears_3_vi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
- link hand: geometry collision mesh filename=collisions/left_hand_collision.stl; visual mesh filename=../assemblies/left_arm_hand/meshes/left_hand_visual.stl
- link hand_2: geometry collision mesh filename=collisions/right_hand_collision.stl; visual mesh filename=../assemblies/right_arm_hand/meshes/right_hand_visual.stl
- link neck_yaw_link: mass 0.0085168305947458285143 -> 0.0085168305947458267796
- link spur_gear_19_teeth: mass 0.0010993711450650535313 -> 0.0010993711450650533144
- link spur_gear_19_teeth_2: mass 0.0010993711450650535313 -> 0.0010993711450650533144
- link spur_gear_21_teeth: mass 0.0010063046528317974842 -> 0.0010063046528317972673
- link spur_gear_21_teeth_2: mass 0.0010063046528317974842 -> 0.0010063046528317972673
- link torso: mass 0.58475267652546303321 -> 0.58475267652546314423
- link waist_gears: mass 0.025809950030454161668 -> 0.025809950030454158199
- link waist_link: mass 0.16767948617484731977 -> 0.16631953490612458313
Joints:
- added joint waist_act_1: type revolute, parent waist_link, child spiral_bevel_1m_14t_30deg, origin xyz=5.380496587145115132e-16 0.019600000000000075695 -0.012750000000000080713 rpy=1.5707963267949007768 1.5707963267948907848 0, axis 0 0 1, limit lower=-2.7825534678416246059 upper=2.7825534678416246059 effort=1 velocity=20
- added joint waist_act_2: type revolute, parent waist_link, child spiral_bevel_1m_14t_30deg_2, origin xyz=-2.6785082652000791162e-16 0.019599999999999902223 -0.032749999999999612754 rpy=1.5707963267948958919 1.3463968515392310543 -4.6125152814992733786e-14, axis 0 0 1, limit lower=-2.7825534678416246059 upper=2.7825534678416246059 effort=1 velocity=20
- joint left_hip_yaw_drive: origin xyz=-0.036999999999998312017 0.037100000000006030931 -0.0395000000000006804 rpy=-1.5707963267949798247 -4.6304776107371661452e-13 -3.868919074001414487e-13 -> xyz=-0.036999999999998194056 0.037100000000006128076 -0.039500000000001291023 rpy=-1.5707963267949545116 -4.7906511943294847217e-13 -3.592506663906207747e-13
- joint left_hip_yaw_driven: origin xyz=-0.037000000000000005107 0.041099999999999997646 -0.019499999999999979156 rpy=-1.5707963267948923392 -1.5707963267948932273 0 -> xyz=-0.037000000000000012046 0.041099999999999997646 -0.0194999999999999514 rpy=-1.5707963267948990005 -1.570796326794896558 0
- joint left_leg_fixed: origin xyz=-4.336808689942017736e-19 0 0.004999999999999997502 rpy=3.1415926535897851224 -1.1045608006607374766e-30 -4.2552910532817472121e-31 -> xyz=0 0 0.004999999999999997502 rpy=3.1415926535897873428 -0 -1.6681280046507162628e-30
- joint left_sho_pitch: origin xyz=-0.0030000000000067082381 0.062000000000004690248 0.10423651076282114403 rpy=-1.5707963267949092145 -3.6755753074147472872e-14 3.4347079465292731775e-14 -> xyz=-0.0030000000000065664245 0.062000000000004926171 0.10423651076282140771 rpy=-1.5707963267949054398 -3.6755753074147447628e-14 3.6857314245917344439e-14
- joint neck_pitch_drive: origin xyz=-1.7971735211119721498e-15 0.015649999999999192335 -0.008799999999996657718 rpy=-9.1684649781985877855e-16 7.2823649231784177849e-17 -1.5707963267948912289 -> xyz=-1.4224732503009818174e-16 0.015649999999999136824 -0.0087999999999959568897 rpy=-2.4492935983152098954e-16 -2.1427228763620856097e-15 -1.570796326794896558
- joint neck_pitch_driven: origin xyz=3.7499998592482874926e-10 -0.0051500000614754029571 0.027499999999999941158 rpy=1.570796326794896336 8.6610484296623782615e-16 3.1415926535897926719 -> xyz=3.7500001368040436489e-10 -0.0051500000614753682626 0.027499999999999830136 rpy=1.57079632679489678 1.7322096859329345721e-15 -3.1415926535897922278
- joint neck_yaw_drive: origin xyz=-0.0050000000000043915566 2.1780059937422389857e-15 0.12148651076282247774 rpy=-4.6722658561527960149e-15 -3.0241828739332580702e-14 3.0478935990547233347e-14 -> xyz=-0.0050000000000041591036 2.1706564040395755645e-15 0.12148651076282282468 rpy=-4.7086950490309927255e-15 -3.2377166610426843676e-14 2.947288666540578667e-14
- joint neck_yaw_driven: origin xyz=0.015999999999998633371 3.2287696509065600056e-15 0.12248651076282091044 rpy=2.3436576345318096491e-14 3.3282183470283369239e-14 -3.1415926535897926719 -> xyz=0.015999999999998446021 3.2990787509752002888e-15 0.12248651076282082717 rpy=2.3463681399312212716e-14 3.1845915227826135867e-14 3.141592653589793116
- joint right_hip_yaw_drive: origin xyz=0.037000000000001607992 0.037100000000003560685 -0.039500000000000486111 rpy=-1.5707963267949798247 -4.6304330256338374643e-13 -3.8689190740014134773e-13 -> xyz=0.037000000000001746769 0.037100000000003664768 -0.039500000000000978773 rpy=-1.5707963267949545116 -4.7905720692590075245e-13 -3.5747430955122047375e-13
- joint right_hip_yaw_driven: origin xyz=0.037000000000000005107 0.041099999999999997646 -0.019499999999999986094 rpy=-1.5707963267949132113 -1.5707963267948950037 0 -> xyz=0.036999999999999991229 0.041100000000000011524 -0.0194999999999999514 rpy=-1.5707963267949003328 -1.5707963267948956698 0
- joint right_leg_fixed: origin xyz=0 0 0.004999999999999997502 rpy=-3.1415926535897797933 -7.5781949123851955204e-18 -3.340101530512157196e-16 -> xyz=0 0 0.0050000000000000044409 rpy=-3.141592653589793116 -0 -9.3397966250929058941e-32
- joint right_sho_pitch: origin xyz=-0.0030000000000024208691 -0.061999999999999777511 0.10423651076282194894 rpy=-1.5707963267948847896 2.9071281258321823756e-14 -3.1415926535897589211 -> xyz=-0.0030000000000019676726 -0.062000000000000089762 0.10423651076282176853 rpy=-1.5707963267948885644 3.4812325502379109658e-14 -3.1415926535897562566
- joint waist_roll: origin xyz=-0.022707865260692145642 -3.2904492237211951884e-18 -0.014000000000000064476 rpy=-1.5707963267949034414 -6.2265052416776424318e-15 1.5707963267948885644 -> xyz=-0.022707865260691548898 -1.3479418671744790767e-17 -0.014000000000000234479 rpy=-1.5707963267949187625 -1.0371626905663003511e-14 1.5707963267948794606
- joint waist_yaw: origin xyz=0 -4.3140830754274083108e-32 0 rpy=9.7872132923950749268e-15 4.0244775309734053704e-14 -3.1415926535897926719 -> xyz=0 -9.8607613152626475676e-32 0 rpy=1.6626925279001758682e-14 4.9579962395338894532e-14 -3.1415926535897900074

Commit message: Fix the waist yaw

File: toddlerbot/robot_descriptions/assemblies/toddlerbot/toddlerbot.urdf (robot description, URDF)
Before this commit: robot toddlerbot, 17 links, 16 joints
Links:
- link neck_yaw_link: mass 0.0085168305947458250449 -> 0.0085168305947458285143
- link spiral_bevel_1m_14t_30deg: mass 0.00067997563436136257333 -> 0.00067997563436136246491
- link spiral_bevel_1m_14t_30deg_2: mass 0.00067997563436136257333 -> 0.00067997563436136246491
- link spur_1m_20t: mass 0.0015534950290892282111 -> 0.0015534950290892286448
- link spur_gear_21_teeth: mass 0.0010063046528317974842 -> 0.0010063046528317972673
- link spur_gear_21_teeth_2: mass 0.0010063046528317974842 -> 0.0010063046528317972673
- link torso: mass 0.59420757418972613983 -> 0.59420757418972602881
- link waist_gears: mass 0.025809950030454158199 -> 0.025809950030454161668
- link waist_link: mass 0.1663195349061246664 -> 0.16631953490612461088
Joints:
- joint left_hip_yaw_driven: origin xyz=-0.037000000000000005107 0.04110000000000003928 -0.019500000000000024258 rpy=-1.5707963267948961139 -1.5707963267948883423 0 -> xyz=-0.036999999999999998168 0.04110000000000003928 -0.019500000000000027728 rpy=-1.5707963267948961139 -1.5707963267948883423 0
- joint left_leg_fixed: origin xyz=0 0 0.0050000000000000044409 rpy=3.141592653589793116 -2.7755575615625073977e-17 -3.33066907387546617e-16 -> xyz=4.7704895589362195096e-18 -6.9388939039072283776e-18 0.0050000000000000113798 rpy=3.141592653589793116 -2.7755575615623496255e-17 -3.3306690738754706073e-16
- joint neck_pitch_driven: origin xyz=3.7500136329526867485e-10 -0.0051500000614755217856 0.027499999999999982792 rpy=1.570796326794896558 8.6610484296647231505e-16 3.141592653589793116 -> xyz=3.7500132513135220336e-10 -0.0051500000614755217856 0.027499999999999982792 rpy=1.570796326794896558 2.1758709533710261129e-15 3.141592653589793116
- joint neck_yaw_driven: origin xyz=0.016000000000001415867 8.8819348604294950814e-19 0.12248651076281755201 rpy=-9.9708248341699279089e-16 -4.1376224834062942084e-15 3.1415926535897922278 -> xyz=0.016000000000001415867 8.8819348604293101922e-19 0.12248651076281755201 rpy=-9.9708248341698016912e-16 -2.8278563730017396217e-15 3.1415926535897922278
- joint right_hip_yaw_driven: origin xyz=0.036999999999999991229 0.041099999999999997646 -0.019500000000000003442 rpy=-1.5707963267948961139 -1.5707963267948950037 0 -> xyz=0.036999999999999991229 0.041099999999999997646 -0.019499999999999999972 rpy=-1.5707963267948961139 -1.5707963267948952257 0
- joint right_leg_fixed: origin xyz=4.336808689942017736e-19 0 0.0050000000000000044409 rpy=-3.141592653589793116 2.7755575615631236952e-17 -4.1633363423443401081e-17 -> xyz=-4.7704895589362195096e-18 0 0.0050000000000000044409 rpy=-3.141592653589793116 -8.3266726846891486023e-17 -4.1633363423432264583e-17
- joint waist_act_1: limit lower=-2.7825534678416246059 upper=2.7825534678416246059 effort=1 velocity=20 -> lower=-4.6774823953448034786 upper=4.6774823953448034786 effort=1 velocity=20
- joint waist_act_2: limit lower=-2.7825534678416246059 upper=2.7825534678416246059 effort=1 velocity=20 -> lower=-4.6774823953448034786 upper=4.6774823953448034786 effort=1 velocity=20
