Commit message: Update the joint limits

File: toddlerbot/robot_descriptions/assemblies/toddlerbot/toddlerbot.urdf (robot description, URDF)
Before this commit: robot toddlerbot, 17 links, 16 joints
Links:
- link neck_pitch_link: mass 0.11211553874797880459 -> 0.11211553874797881847
- link neck_yaw_link: mass 0.0085168305947458285143 -> 0.0085168305947458267796
- link spiral_bevel_1m_14t_30deg: mass 0.00067997563436136246491 -> 0.00073261524436595492574
- link spiral_bevel_1m_14t_30deg_2: mass 0.00067997563436136246491 -> 0.00073261524436595492574
- link spur_gear_(13_teeth): mass 0.00081469437497230876716 -> 0.00081469437497230865874
- link spur_gear_19_teeth: mass 0.0010993711450650535313 -> 0.0011084409433758843876
- link spur_gear_19_teeth_2: mass 0.0010993711450650535313 -> 0.0011084409433758843876
- link spur_gear_21_teeth: mass 0.0010063046528317972673 -> 0.0010185686142775147826
- link spur_gear_21_teeth_2: mass 0.0010063046528317972673 -> 0.0010185686142775147826
- link torso: mass 0.59420757418972602881 -> 0.60012685450989189384
- link waist_gears: mass 0.025809950030454161668 -> 0.025874065810895640477
Joints:
- joint left_hip_yaw_drive: limit lower=-1.4211966766239538806 upper=1.4211966766239538806 effort=1 velocity=20 -> lower=-1.7361433085627806516 upper=1.7361433085627806516 effort=1 velocity=20; origin xyz=-0.03699999999999847855 0.037100000000005933787 -0.039500000000000194678 rpy=-1.5707963267949540676 -4.7732588435988597417e-13 -3.5949390257278751872e-13 -> xyz=-0.036999999999998457734 0.037100000000005961542 -0.03950000000000024325 rpy=-1.5707963267949545116 -4.8003070743589248247e-13 -3.5749181392930616155e-13
- joint left_hip_yaw_driven: origin xyz=-0.036999999999999998168 0.04110000000000003928 -0.019500000000000027728 rpy=-1.5707963267948961139 -1.5707963267948883423 0 -> xyz=-0.036999999999999998168 0.041100000000000011524 -0.019500000000000027728 rpy=-1.5707963267948947816 -1.570796326794896558 0
- joint left_leg_fixed: origin xyz=4.7704895589362195096e-18 -6.9388939039072283776e-18 0.0050000000000000113798 rpy=3.141592653589793116 -2.7755575615623496255e-17 -3.3306690738754706073e-16 -> xyz=0 0 0.004999999999999997502 rpy=3.1415926535897926719 -1.9428902930939016723e-16 -7.6327832942984196016e-16
- joint left_sho_pitch: limit lower=-1.570796326794896558 upper=1.570796326794896558 effort=1 velocity=20 -> lower=-3.141592653589793116 upper=1.570796326794896558 effort=1 velocity=20
- joint neck_pitch_drive: limit lower=-1.4279966607226330932 upper=1.4279966607226330932 effort=1 velocity=20 -> lower=-2.174948760177549012 upper=2.174948760177549012 effort=1 velocity=20; origin xyz=-8.3266726846886740532e-17 0.015649999999999109068 -0.0087999999999961303621 rpy=-6.1232340018137966949e-17 -1.865637580072612815e-26 -1.570796326794896558 -> xyz=-6.9735883734267645195e-16 0.015649999999999053557 -0.0087999999999970532349 rpy=-1.1409718301987536487e-15 4.409645192886135633e-16 -1.5707963267948976682
- joint neck_pitch_driven: origin xyz=3.7500132513135220336e-10 -0.0051500000614755217856 0.027499999999999982792 rpy=1.570796326794896558 2.1758709533710261129e-15 3.141592653589793116 -> xyz=3.7499979510524639181e-10 -0.0051500000614751947903 0.027499999999999941158 rpy=1.5707963267948978903 -2.0825786444073518345e-16 3.141592653589793116
- joint neck_yaw_drive: limit lower=-2.2689280275926284602 upper=2.2689280275926284602 effort=1 velocity=20 -> lower=-2.8797932657906435416 upper=2.8797932657906435416 effort=1 velocity=20; origin xyz=-0.0049999999999993625932 3.342147474086756384e-17 0.12148651076281766215 rpy=7.9879995913373272052e-15 8.0038275409654909883e-15 -5.4161669716995088817e-15 -> xyz=-0.004999999999999517851 2.6555840535020396321e-18 0.121486510762817565 rpy=1.1318451824181020002e-14 2.6985403517595457696e-15 -5.3863140912757267331e-15
- joint neck_yaw_driven: limit lower=-3.141592653589793116 upper=3.141592653589793116 effort=1 velocity=20 -> lower=-2.6179938779914944114 upper=2.6179938779914944114 effort=1 velocity=20; origin xyz=0.016000000000001415867 8.8819348604293101922e-19 0.12248651076281755201 rpy=-9.9708248341698016912e-16 -2.8278563730017396217e-15 3.1415926535897922278 -> xyz=0.016000000000001235456 2.2310681558151314601e-17 0.12248651076281746874 rpy=-4.8668742840765556337e-16 -4.0649010562893427138e-15 3.141592653589793116
- joint right_hip_yaw_drive: limit lower=-1.4211966766239538806 upper=1.4211966766239538806 effort=1 velocity=20 -> lower=-1.7361433085627806516 upper=1.7361433085627806516 effort=1 velocity=20; origin xyz=0.037000000000001344314 0.037100000000003394152 -0.039499999999999368949 rpy=-1.5707963267949540676 -4.7918343317333855547e-13 -3.3767433293974656194e-13 -> xyz=0.037000000000001719014 0.03710000000000327619 -0.0394999999999998061 rpy=-1.5707963267949545116 -4.8002361403961149694e-13 -3.5216274341110541015e-13
- joint right_hip_yaw_driven: origin xyz=0.036999999999999991229 0.041099999999999997646 -0.019499999999999999972 rpy=-1.5707963267948961139 -1.5707963267948952257 0 -> xyz=0.036999999999999991229 0.041100000000000011524 -0.019500000000000017319 rpy=-1.570796326794896558 -1.5707963267948961139 0
- joint right_leg_fixed: origin xyz=-4.7704895589362195096e-18 0 0.0050000000000000044409 rpy=-3.141592653589793116 -8.3266726846891486023e-17 -4.1633363423432264583e-17 -> xyz=0 -6.9388939039072283776e-18 0.0050000000000000044409 rpy=-3.1415926535897926719 1.8281169925220331315e-17 -3.5772536718062127375e-16
- joint right_sho_pitch: limit lower=-1.570796326794896558 upper=1.570796326794896558 effort=1 velocity=20 -> lower=-1.570796326794896558 upper=3.141592653589793116 effort=1 velocity=20
- joint waist_act_1: origin xyz=-5.1956727612250319334e-16 0.019600000000000002837 -0.012749999999999961017 rpy=1.570796326794896336 1.5707963267948870101 0 -> xyz=5.7457652915638341522e-17 0.019599999999999964673 -0.012750000000000025202 rpy=1.5707963267948954478 1.570796326794896336 0
- joint waist_act_2: origin xyz=2.5285386378767095671e-17 0.019599999999999995898 -0.032749999999999987454 rpy=1.5707963267948974462 1.3463968515392308323 3.4406882288644243018e-15 -> xyz=4.2745485696894321379e-17 0.019600000000000013245 -0.032749999999999994393 rpy=1.5707963267948956698 1.3463968515392303882 6.7698458176426589005e-15
- joint waist_roll: origin xyz=-0.022707865260692197684 -2.2800061759205613016e-17 -0.01399999999999972447 rpy=-1.570796326794896558 -1.4470091796846119987e-16 1.5707963267948970021 -> xyz=-0.022707865260692617487 -2.4393502827093082036e-16 -0.013999999999999814676 rpy=-1.5707963267948974462 1.8675461532229772614e-15 1.5707963267948952257
- joint waist_yaw: origin xyz=0 6.1629758220391547298e-33 -2.4651903288156618919e-30 rpy=1.3285483818409156951e-16 -3.8508827433200160488e-15 3.1415926535897922278 -> xyz=0 -3.1104917983741196655e-18 -7.5188305028877687703e-30 rpy=-1.4111145075746007461e-16 -4.1376224834060906822e-15 3.1415926535897922278

File: toddlerbot/robot_descriptions/toddlerbot/toddlerbot.urdf (robot description, URDF)
Before this commit: robot toddlerbot, 75 links, 74 joints
Links:
- link neck_pitch_link: mass 0.11211553874797880459 -> 0.11211553874797881847
- link neck_yaw_link: mass 0.0085168305947458285143 -> 0.0085168305947458267796
- link spiral_bevel_1m_14t_30deg: mass 0.00067997563436136246491 -> 0.00073261524436595492574
- link spiral_bevel_1m_14t_30deg_2: mass 0.00067997563436136246491 -> 0.00073261524436595492574
- link spur_gear_(13_teeth): mass 0.00081469437497230876716 -> 0.00081469437497230865874
- link spur_gear_19_teeth: mass 0.0010993711450650535313 -> 0.0011084409433758843876
- link spur_gear_19_teeth_2: mass 0.0010993711450650535313 -> 0.0011084409433758843876
- link spur_gear_21_teeth: mass 0.0010063046528317972673 -> 0.0010185686142775147826
- link spur_gear_21_teeth_2: mass 0.0010063046528317972673 -> 0.0010185686142775147826
- link torso: mass 0.59420757418972602881 -> 0.60012685450989189384
- link waist_gears: mass 0.025809950030454161668 -> 0.025874065810895640477
Joints:
- joint left_hip_yaw_drive: limit lower=-1.4211966766239538806 upper=1.4211966766239538806 effort=1 velocity=20 -> lower=-1.7361433085627806516 upper=1.7361433085627806516 effort=1 velocity=20; origin xyz=-0.03699999999999847855 0.037100000000005933787 -0.039500000000000194678 rpy=-1.5707963267949540676 -4.7732588435988597417e-13 -3.5949390257278751872e-13 -> xyz=-0.036999999999998457734 0.037100000000005961542 -0.03950000000000024325 rpy=-1.5707963267949545116 -4.8003070743589248247e-13 -3.5749181392930616155e-13
- joint left_hip_yaw_driven: origin xyz=-0.036999999999999998168 0.04110000000000003928 -0.019500000000000027728 rpy=-1.5707963267948961139 -1.5707963267948883423 0 -> xyz=-0.036999999999999998168 0.041100000000000011524 -0.019500000000000027728 rpy=-1.5707963267948947816 -1.570796326794896558 0
- joint left_leg_fixed: origin xyz=4.7704895589362195096e-18 -6.9388939039072283776e-18 0.0050000000000000113798 rpy=3.141592653589793116 -2.7755575615623496255e-17 -3.3306690738754706073e-16 -> xyz=0 0 0.004999999999999997502 rpy=3.1415926535897926719 -1.9428902930939016723e-16 -7.6327832942984196016e-16
- joint left_sho_pitch: limit lower=-1.570796326794896558 upper=1.570796326794896558 effort=1 velocity=20 -> lower=-3.141592653589793116 upper=1.570796326794896558 effort=1 velocity=20
- joint neck_pitch_drive: limit lower=-1.4279966607226330932 upper=1.4279966607226330932 effort=1 velocity=20 -> lower=-2.174948760177549012 upper=2.174948760177549012 effort=1 velocity=20; origin xyz=-8.3266726846886740532e-17 0.015649999999999109068 -0.0087999999999961303621 rpy=-6.1232340018137966949e-17 -1.865637580072612815e-26 -1.570796326794896558 -> xyz=-6.9735883734267645195e-16 0.015649999999999053557 -0.0087999999999970532349 rpy=-1.1409718301987536487e-15 4.409645192886135633e-16 -1.5707963267948976682
- joint neck_pitch_driven: origin xyz=3.7500132513135220336e-10 -0.0051500000614755217856 0.027499999999999982792 rpy=1.570796326794896558 2.1758709533710261129e-15 3.141592653589793116 -> xyz=3.7499979510524639181e-10 -0.0051500000614751947903 0.027499999999999941158 rpy=1.5707963267948978903 -2.0825786444073518345e-16 3.141592653589793116
- joint neck_yaw_drive: limit lower=-2.2689280275926284602 upper=2.2689280275926284602 effort=1 velocity=20 -> lower=-2.8797932657906435416 upper=2.8797932657906435416 effort=1 velocity=20; origin xyz=-0.0049999999999993625932 3.342147474086756384e-17 0.12148651076281766215 rpy=7.9879995913373272052e-15 8.0038275409654909883e-15 -5.4161669716995088817e-15 -> xyz=-0.004999999999999517851 2.6555840535020396321e-18 0.121486510762817565 rpy=1.1318451824181020002e-14 2.6985403517595457696e-15 -5.3863140912757267331e-15
- joint neck_yaw_driven: limit lower=-3.141592653589793116 upper=3.141592653589793116 effort=1 velocity=20 -> lower=-2.6179938779914944114 upper=2.6179938779914944114 effort=1 velocity=20; origin xyz=0.016000000000001415867 8.8819348604293101922e-19 0.12248651076281755201 rpy=-9.9708248341698016912e-16 -2.8278563730017396217e-15 3.1415926535897922278 -> xyz=0.016000000000001235456 2.2310681558151314601e-17 0.12248651076281746874 rpy=-4.8668742840765556337e-16 -4.0649010562893427138e-15 3.141592653589793116
- joint right_hip_yaw_drive: limit lower=-1.4211966766239538806 upper=1.4211966766239538806 effort=1 velocity=20 -> lower=-1.7361433085627806516 upper=1.7361433085627806516 effort=1 velocity=20; origin xyz=0.037000000000001344314 0.037100000000003394152 -0.039499999999999368949 rpy=-1.5707963267949540676 -4.7918343317333855547e-13 -3.3767433293974656194e-13 -> xyz=0.037000000000001719014 0.03710000000000327619 -0.0394999999999998061 rpy=-1.5707963267949545116 -4.8002361403961149694e-13 -3.5216274341110541015e-13
- joint right_hip_yaw_driven: origin xyz=0.036999999999999991229 0.041099999999999997646 -0.019499999999999999972 rpy=-1.5707963267948961139 -1.5707963267948952257 0 -> xyz=0.036999999999999991229 0.041100000000000011524 -0.019500000000000017319 rpy=-1.570796326794896558 -1.5707963267948961139 0
- joint right_leg_fixed: origin xyz=-4.7704895589362195096e-18 0 0.0050000000000000044409 rpy=-3.141592653589793116 -8.3266726846891486023e-17 -4.1633363423432264583e-17 -> xyz=0 -6.9388939039072283776e-18 0.0050000000000000044409 rpy=-3.1415926535897926719 1.8281169925220331315e-17 -3.5772536718062127375e-16
- joint right_sho_pitch: limit lower=-1.570796326794896558 upper=1.570796326794896558 effort=1 velocity=20 -> lower=-1.570796326794896558 upper=3.141592653589793116 effort=1 velocity=20
- joint waist_act_1: origin xyz=-5.1956727612250319334e-16 0.019600000000000002837 -0.012749999999999961017 rpy=1.570796326794896336 1.5707963267948870101 0 -> xyz=5.7457652915638341522e-17 0.019599999999999964673 -0.012750000000000025202 rpy=1.5707963267948954478 1.570796326794896336 0
- joint waist_act_2: origin xyz=2.5285386378767095671e-17 0.019599999999999995898 -0.032749999999999987454 rpy=1.5707963267948974462 1.3463968515392308323 3.4406882288644243018e-15 -> xyz=4.2745485696894321379e-17 0.019600000000000013245 -0.032749999999999994393 rpy=1.5707963267948956698 1.3463968515392303882 6.7698458176426589005e-15
- joint waist_roll: origin xyz=-0.022707865260692197684 -2.2800061759205613016e-17 -0.01399999999999972447 rpy=-1.570796326794896558 -1.4470091796846119987e-16 1.5707963267948970021 -> xyz=-0.022707865260692617487 -2.4393502827093082036e-16 -0.013999999999999814676 rpy=-1.5707963267948974462 1.8675461532229772614e-15 1.5707963267948952257
- joint waist_yaw: origin xyz=0 6.1629758220391547298e-33 -2.4651903288156618919e-30 rpy=1.3285483818409156951e-16 -3.8508827433200160488e-15 3.1415926535897922278 -> xyz=0 -3.1104917983741196655e-18 -7.5188305028877687703e-30 rpy=-1.4111145075746007461e-16 -4.1376224834060906822e-15 3.1415926535897922278
