Commit message: Update the toddlerbot MJCF

File: toddlerbot/robot_descriptions/assemblies/toddlerbot/toddlerbot.urdf (robot description, URDF)
Before this commit: robot toddlerbot, 17 links, 16 joints
Links:
- link left_arm_hand: mass 0.0085999999999999965361 -> 0.0085999999999999948014
- link left_leg_xm430: mass 0.017999999999999995171 -> 0.01799999999999999864
- link neck_pitch_link: mass 0.11211553874797881847 -> 0.074299999993091794814
- link right_arm_hand: mass 0.0085999999999999965361 -> 0.0085999999999999948014
- link right_leg_xm430: mass 0.017999999999999995171 -> 0.01799999999999999864
- link spiral_bevel_1m_14t_30deg: mass 0.00073261524436595492574 -> 0.00073261524436595481732
- link spiral_bevel_1m_14t_30deg_2: mass 0.00073261524436595492574 -> 0.00073261524436595481732
- link spur_gear_(13_teeth): mass 0.00081469437497230865874 -> 0.00081469437497230876716
- link spur_gear_21_teeth: mass 0.0010185686142775147826 -> 0.0010185686142775145658
- link spur_gear_21_teeth_2: mass 0.0010185686142775147826 -> 0.0010185686142775145658
- link torso: mass 0.60012685450989189384 -> 0.6001268545098842333
- link waist_gears: mass 0.025874065810895640477 -> 0.026337180140419171048
- link waist_link: mass 0.16631953490612461088 -> 0.17011953490612463646

File: toddlerbot/robot_descriptions/toddlerbot_OP3/toddlerbot_OP3.urdf (robot description, URDF)
Before this commit: robot toddlerbot_OP3, 73 links, 72 joints
Links:
- removed link gripper_connector
- removed link gripper_connector_2
- removed link left_rail_guide
- removed link rail
- removed link rail_2
- removed link rail_3
- removed link rail_4
- removed link right_rail_guide
- removed link spur_gear_(14_teeth)
- removed link spur_gear_(14_teeth)_2
- removed link xc330
- removed link xc330_2
- added link hand, mass 0.03949999999999999345; visual mesh filename=../assemblies/left_arm_umi/meshes/left_hand_visual.stl
- added link hand_2, mass 0.039500000000000000389; visual mesh filename=../assemblies/right_arm_umi/meshes/right_hand_visual.stl
- link 2xl430_gears: mass 0.11800003674524910113 -> 0.11800003674524907338; geometry visual mesh filename=../assemblies/left_arm_umi/meshes/left_2xl430_gears_visual.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
- link 2xl430_gears_2: mass 0.11800003674524910113 -> 0.11800003674524907338; geometry visual mesh filename=../assemblies/left_arm_umi/meshes/left_2xl430_gears_2_visua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
- link 2xl430_gears_3: mass 0.11800003674524910113 -> 0.11800003674524907338; geometry visual mesh filename=../assemblies/left_arm_umi/meshes/left_2xl430_gears_3_visua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
- link 2xl430_gears_4: mass 0.11800003674524910113 -> 0.11800003674524907338; geometry visual mesh filename=../assemblies/right_arm_umi/meshes/right_2xl430_gears_visua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
- link 2xl430_gears_5: mass 0.11800003674524910113 -> 0.11800003674524907338; geometry visual mesh filename=../assemblies/right_arm_umi/meshes/right_2xl430_gears_2_vis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
- link 2xl430_gears_6: mass 0.11800003674524910113 -> 0.11800003674524907338; geometry visual mesh filename=../assemblies/right_arm_umi/meshes/right_2xl430_gears_3_vis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
- link elb_yaw_link: mass 0.017500000000000001665 -> 0.017499999999999998196; geometry visual mesh filename=../assemblies/left_arm_umi/meshes/left_elb_yaw_link_visual.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
- link elb_yaw_link_2: mass 0.017500000000000001665 -> 0.017499999999999998196; geometry visual mesh filename=../assemblies/right_arm_umi/meshes/right_elb_yaw_link_visua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
- link neck_pitch_link: mass 0.11211553874797881847 -> 0.074299999993091794814
- link sho_pitch_link: mass 0.0086000000000000000056 -> 0.0085999999999999948014; geometry visual mesh filename=../assemblies/left_arm_umi/meshes/left_sho_pitch_link_visua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
- link sho_pitch_link_2: mass 0.0086000000000000000056 -> 0.0085999999999999948014; geometry visual mesh filename=../assemblies/right_arm_umi/meshes/right_sho_pitch_link_vis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
- link sho_yaw_link: mass 0.014500000000000016348 -> 0.01450000000000000594; geometry visual mesh filename=../assemblies/left_arm_umi/meshes/left_sho_yaw_link_visual.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
- link sho_yaw_link_2: mass 0.014500000000000016348 -> 0.01450000000000000594; geometry visual mesh filename=../assemblies/right_arm_umi/meshes/right_sho_yaw_link_visua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
- link spiral_bevel_1m_14t_30deg: mass 0.00073261524436595492574 -> 0.00073261524436595481732
- link spiral_bevel_1m_14t_30deg_2: mass 0.00073261524436595492574 -> 0.00073261524436595481732
- link spur_1m_24t_drive: geometry visual mesh filename=../assemblies/left_arm_umi/meshes/left_spur_1m_24t_drive_vi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
- link spur_1m_24t_drive_2: geometry visual mesh filename=../assemblies/left_arm_umi/meshes/left_spur_1m_24t_drive_2_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
- link spur_1m_24t_drive_3: geometry visual mesh filename=../assemblies/left_arm_umi/meshes/left_spur_1m_24t_drive_3_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
- link spur_1m_24t_drive_4: geometry visual mesh filename=../assemblies/right_arm_umi/meshes/right_spur_1m_24t_drive_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
- link spur_1m_24t_drive_5: geometry visual mesh filename=../assemblies/right_arm_umi/meshes/right_spur_1m_24t_drive_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
- link spur_1m_24t_drive_6: geometry visual mesh filename=../assemblies/right_arm_umi/meshes/right_spur_1m_24t_drive_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
- link spur_1m_24t_driven: mass 0.0026999999999999997093 -> 0.0027000000000000001429; geometry visual mesh filename=../assemblies/left_arm_umi/meshes/left_spur_1m_24t_driven_v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
- link spur_1m_24t_driven_2: mass 0.0026999999999999997093 -> 0.0027000000000000001429; geometry visual mesh filename=../assemblies/left_arm_umi/meshes/left_spur_1m_24t_driven_2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
- link spur_1m_24t_driven_3: mass 0.0026999999999999997093 -> 0.0027000000000000001429; geometry visual mesh filename=../assemblies/left_arm_umi/meshes/left_spur_1m_24t_driven_3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
- link spur_1m_24t_driven_4: mass 0.0026999999999999997093 -> 0.0027000000000000001429; geometry visual mesh filename=../assemblies/right_arm_umi/meshes/right_spur_1m_24t_driven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
- link spur_1m_24t_driven_5: mass 0.0026999999999999997093 -> 0.0027000000000000001429; geometry visual mesh filename=../assemblies/right_arm_umi/meshes/right_spur_1m_24t_driven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
- link spur_1m_24t_driven_6: mass 0.0026999999999999997093 -> 0.0027000000000000001429; geometry visual mesh filename=../assemblies/right_arm_umi/meshes/right_spur_1m_24t_driven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
- link spur_gear_(13_teeth): mass 0.00081469437497230865874 -> 0.00081469437497230876716
- link spur_gear_21_teeth: mass 0.0010185686142775147826 -> 0.0010185686142775145658
- link spur_gear_21_teeth_2: mass 0.0010185686142775147826 -> 0.0010185686142775145658
- link torso: mass 0.60012685450989189384 -> 0.6001268545098842333
- link waist_gears: mass 0.025874065810895640477 -> 0.026337180140419171048
- link waist_link: mass 0.16631953490612461088 -> 0.17011953490612463646
- link wrist_bearing_plate: mass 0.0049000367468305548388 -> 0.0049000367468305557062; geometry visual mesh filename=../assemblies/left_arm_umi/meshes/left_wrist_bearing_plate_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
- link wrist_bearing_plate_2: mass 0.0049000367468305548388 -> 0.0049000367468305557062; geometry visual mesh filename=../assemblies/right_arm_umi/meshes/right_wrist_bearing_plat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
Joints:
- removed joint left_gripper_fixed
- removed joint left_gripper_motor
- removed joint left_gripper_pinion
- removed joint left_gripper_pinion_mirror
- removed joint left_gripper_rack
- removed joint right_gripper_fixed
- removed joint right_gripper_motor
- removed joint right_gripper_pinion
- removed joint right_gripper_pinion_mirror
- removed joint right_gripper_rack
- joint left_elbow_roll: origin xyz=0 -0.018999999999999996059 -0.058999999999999983014 rpy=1.570796326794896558 5.5516872419979014276e-14 -4.4351709097753281525e-15 -> xyz=1.17614251671227521e-15 -0.019000000000000002998 -0.05900000000000006628 rpy=1.5707963267948954478 -1.8257447566372568016e-14 -1.7593846109850829682e-16
- joint left_elbow_yaw_drive: origin xyz=-0.02400000071614073055 -0.019000000152457841018 -0.019000000152442970969 rpy=1.5707963267946287722 -5.6790261222308772362e-14 9.8859639154170636391e-14 -> xyz=-0.024000000716137517842 -0.0190000001524475437 -0.019000000152459544517 rpy=1.5707963267950562081 -2.4622204840090993627e-13 -1.7925499053412602242e-13
- joint left_elbow_yaw_driven: origin xyz=-3.5806481391009725712e-10 -0.027000000152458666913 -0.018999999999996696615 rpy=1.5707963267946756236 9.436895709310436914e-15 -7.5767000241948220497e-14 -> xyz=-3.5806394307891231676e-10 -0.027000000152452990898 -0.0190000000000065776 rpy=1.5707963267949589525 1.5707963267946882802 0
- joint left_elbow_yaw_fixed: origin xyz=0 3.1554436208840472216e-30 0.0016000000000000041966 rpy=-3.1415926535897926719 -1.6686716652751508178e-29 -1.570796326794896558 -> xyz=1.5777218104420236108e-30 0 0.0015999999999999764411 rpy=-3.141592653589793116 -4.4866451871279772575e-27 -3.2816870322621037337e-28
- joint left_sho_roll: origin xyz=-0.01899999999999992667 0.00099999999999997031368 0.026999999999999909489 rpy=3.1415926535897913396 1.5707963267948474861 0 -> xyz=-0.018999999999999999528 0.00099999999999999546717 0.027000000000000006634 rpy=-3.141592653589793116 1.5707963267948956698 0
- joint left_sho_yaw_drive: origin xyz=-0.024000000716139110318 -0.019000000152454975255 -0.019000000152449778024 rpy=1.5707963267949334174 -1.1191795890472901541e-13 1.4055336229792838361e-13 -> xyz=-0.024000000716140966472 -0.019000000152450589874 -0.019000000152443286688 rpy=1.5707963267948328312 -1.3331515362498170811e-15 8.2000365474799924889e-14
- joint left_sho_yaw_driven: origin xyz=-3.5806544534944251268e-10 -0.027000000152452456603 -0.01900000000000368755 rpy=1.5707963267949525132 -6.2878911843812520251e-14 1.1213824667586519115e-13 -> xyz=-3.5807029563628134383e-10 -0.027000000152450926577 -0.018999999999999878098 rpy=1.5707963267948492625 7.9618117061828289905e-14 1.0047518372857611155e-13
- joint left_sho_yaw_fixed: origin xyz=-3.4694469519536141888e-18 1.5777218104420236108e-30 0.0016000000000000041966 rpy=3.1415926535897771288 -2.9902758688536131143e-29 -1.1367870242563646532e-30 -> xyz=-3.4694469519536141888e-18 0 0.0015999999999999972577 rpy=-3.1415926535897926719 -0 0
- joint left_wrist_pitch_drive: origin xyz=-1.5244435917471112579e-10 0.024000000358067929973 -0.0080000000000045659587 rpy=-6.8143291540626782613e-14 -7.3946574628751046645e-14 -1.5707963267947160357 -> xyz=-1.5244060454932555774e-10 0.024000000358057271832 -0.0080000000000068835493 rpy=3.6254446097225608906e-14 -2.2096785867264433738e-13 -1.5707963267949176522
- joint left_wrist_pitch_driven: origin xyz=-2.7755575615628913511e-17 -3.1554436208840472216e-30 -0.0015999999999999972577 rpy=1.8707257964927463223e-14 -2.230976160592272071e-14 -1.570796326794896558 -> xyz=-2.7755575615628913511e-17 -1.5777218104420236108e-30 -0.0015999999999999979083 rpy=-8.9315741575089004617e-15 -8.8817841970012507457e-15 -1.570796326794896558
- joint left_wrist_pitch_fixed: origin xyz=0.015500000000004772113 -6.3837823915946501074e-15 -0.045000000000001996736 rpy=-3.5027536426602388959e-14 -1.2834178164666087642e-13 -1.5707963267947810948 -> xyz=0.015500000000007816553 -1.8068879725774422695e-14 -0.044999999999998901989 rpy=4.0745185003716278612e-14 -2.8213542612434270497e-13 -1.570796326794906328
- joint left_wrist_roll: child gripper_connector -> hand; origin xyz=0.019000000000008621104 -3.5807914966490272946e-10 -0.02700000015245084678 rpy=-5.342948306010493038e-15 1.5707963267948528152 0 -> xyz=0.019000000000007049444 -3.5808095377731774533e-10 -0.027000000152448057344 rpy=-7.3828629579122985512e-14 -1.5707963267945765917 0
- joint left_wrist_roll_fixed: origin xyz=3.1554436208840472216e-30 -0.025300000000000003042 -0.052000000000000032307 rpy=1.570796326794896558 -1.570796326794896558 0 -> xyz=0 -0.025299999999999999573 -0.051999999999999962919 rpy=1.5707963267949056618 -1.5707963267948876762 0
- joint right_elbow_roll: origin xyz=-3.4694469519536141888e-18 -0.018999999999999999528 -0.059000000000000010769 rpy=1.570796326794896558 5.4458140093899203203e-15 -1.8535314627675585241e-14 -> xyz=-1.7347234759768070944e-17 -0.019000000000000159123 -0.059000000000000135669 rpy=1.5707963267948952257 -4.3465231414242792334e-14 -2.6978419498660684154e-14
- joint right_elbow_yaw_drive: origin xyz=-0.02400000071614593472 -0.019000000152452525826 -0.019000000152448241059 rpy=1.5707963267948983344 1.6898711261348466559e-13 -7.2725329301663980295e-14 -> xyz=-0.024000000716147166374 -0.019000000152450874369 -0.019000000152450291502 rpy=1.5707963267949573982 3.0456550330441217593e-14 -3.9968028886506279166e-14
- joint right_elbow_yaw_driven: origin xyz=-3.5806997991660871605e-10 -0.027000000152456016256 -0.01900000000000036729 rpy=1.5707963267948485964 8.4311697099245782578e-14 3.098094357577576486e-14 -> xyz=-3.5807123932585227521e-10 -0.027000000152452963142 -0.019000000000002556511 rpy=1.5707963267949576203 3.0519690799675378401e-14 -4.0239863453830675462e-14
- joint right_elbow_yaw_fixed: origin xyz=0 7.8886090522101180541e-30 0.0015999999999999764411 rpy=3.141592653589793116 -4.1526642731421539574e-29 -1.570796326794896558 -> xyz=0 7.8886090522101180541e-31 0.0015999999999999903189 rpy=3.141592653589793116 5.5511151240344703462e-17 -1.57079632679489678
- joint right_sho_roll: origin xyz=-0.019000000000000002998 0.0010000000000000076102 0.027000000000000003164 rpy=3.141592653589793116 1.5707963267948827912 0 -> xyz=-0.0190000000000000481 0.0010000000000000234396 0.026999999999999982347 rpy=3.141592653589793116 1.5707963267948952257 0
- joint right_sho_yaw_drive: origin xyz=-0.02400000071613753172 -0.019000000152449930679 -0.01900000015244478202 rpy=1.5707963267947220309 -4.4297106944168913575e-14 6.810646137204639124e-14 -> xyz=-0.024000000716138260304 -0.019000000152445337132 -0.019000000152448428409 rpy=1.5707963267949289765 -7.4062049324254792929e-14 1.9645226351351914911e-14
- joint right_sho_yaw_driven: origin xyz=-3.5806749579259111727e-10 -0.027000000152448931645 -0.018999999999998073985 rpy=1.5707963267947655517 -4.3564811365923459647e-14 5.9791231064775441371e-14 -> xyz=-3.5806844642105595256e-10 -0.02700000015244657936 -0.019000000000003233053 rpy=1.5707963267949260899 -2.2055090607973039157e-14 7.6050277186033683693e-15
- joint right_sho_yaw_fixed: origin xyz=0 1.1832913578315177081e-30 0.0015999999999999937883 rpy=3.141592653589793116 -1.9721522629860631248e-30 4.8102873877572434203e-28 -> xyz=-3.4694469519536141888e-18 3.9443045261050590271e-31 0.0016000000000000041966 rpy=3.141592653589793116 -5.0487097934144755546e-29 -1.8301573001127473886e-28
- joint right_wrist_pitch_drive: origin xyz=-1.5244750094239886385e-10 0.0240000003580740362 -0.0080000000000028936853 rpy=-2.6466654378983997098e-14 5.3007428237114777825e-14 -1.5707963267948148456 -> xyz=-1.524431251168157451e-10 0.024000000358071760242 -0.0080000000000008727324 rpy=1.2483159056318501391e-14 7.3485321852726251993e-14 -1.5707963267948599206
- joint right_wrist_pitch_driven: origin xyz=-2.7755575615628913511e-17 6.3108872417680944433e-30 -0.0015999999999999992093 rpy=5.5511151231243844462e-16 1.2547220914404902092e-15 1.570796326794896558 -> xyz=2.7755575615628913511e-17 7.0997481469891062487e-30 -0.0015999999999999970409 rpy=-3.8285686988021856593e-16 -1.2621774483536197294e-29 1.570796326794896558
- joint right_wrist_pitch_fixed: origin xyz=0.015500000000002131864 9.6866958898544908152e-15 -0.045000000000006430689 rpy=-2.6645352590932944871e-15 1.1984857550828037264e-13 -1.5707963267947835373 -> xyz=0.015500000000003956793 4.5519144009631418157e-15 -0.045000000000003724521 rpy=-3.0531133177156822825e-15 1.2051470932306205513e-13 -1.570796326794896558
- joint right_wrist_roll: child gripper_connector_2 -> hand_2; origin xyz=0.019000000000002677941 -3.5806407838734344296e-10 -0.027000000152454406432 rpy=-3.1415926535897558125 -1.570796326794831721 0 -> xyz=0.019000000000002757738 -3.5806788090120278412e-10 -0.02700000015244990309 rpy=-1.9648186021258132771e-29 1.570796326794851927 0
- joint right_wrist_roll_fixed: origin xyz=1.5777218104420236108e-30 -0.025299999999999999573 -0.052000000000000004552 rpy=1.5707963267948974462 1.570796326794896558 0 -> xyz=-7.8886090522101180541e-31 -0.025299999999999999573 -0.051999999999999976796 rpy=1.570796326794896558 1.570796326794896558 0

Commit message: Update the mass

File: toddlerbot/robot_descriptions/assemblies/toddlerbot/toddlerbot.urdf (robot description, URDF)
Before this commit: robot toddlerbot, 17 links, 16 joints
Links:
- link spur_1m_20t: mass 0.0015534950290892286448 -> 0.0015534950290892282111
- link spur_gear_(13_teeth): mass 0.00081469437497230876716 -> 0.00081469437497230865874
- link torso: mass 0.6001268545098842333 -> 0.66652685450988358173
- link waist_gears: mass 0.026337180140419171048 -> 0.026337180140419174518
- link waist_link: mass 0.17011953490612463646 -> 0.17011953490612458095

File: toddlerbot/robot_descriptions/toddlerbot_OP3/toddlerbot_OP3.urdf (robot description, URDF)
Before this commit: robot toddlerbot_OP3, 63 links, 62 joints
Links:
- link spur_1m_20t: mass 0.0015534950290892286448 -> 0.0015534950290892282111
- link spur_gear_(13_teeth): mass 0.00081469437497230876716 -> 0.00081469437497230865874
- link torso: mass 0.6001268545098842333 -> 0.66652685450988358173
- link waist_gears: mass 0.026337180140419171048 -> 0.026337180140419174518
- link waist_link: mass 0.17011953490612463646 -> 0.17011953490612458095
