Commit message: Update the MJCF

File: toddlerbot/robot_descriptions/assemblies/toddlerbot/toddlerbot.urdf (robot description, URDF)
Before this commit: robot toddlerbot, 17 links, 16 joints
Links:
- removed link spur_gear_(13_teeth)
- added link spur_gear_13_teeth, mass 0.00091877519177533870359; collision mesh filename=package:///meshes/spur_gear_13_teeth_collision.stl; visual mesh filename=package:///meshes/spur_gear_13_teeth_visual.stl
- link left_arm_hand: mass 0.0085999999999999948014 -> 0.0085999999999999930667
- link neck_pitch_link: mass 0.074299999993091794814 -> 0.07429999999309182257
- link right_arm_hand: mass 0.0085999999999999948014 -> 0.0085999999999999930667
- link spur_1m_20t: mass 0.0015534950290892282111 -> 0.0015778025963745999881
- link spur_gear_19_teeth: mass 0.0011084409433758843876 -> 0.0010324984452316546789
- link spur_gear_19_teeth_2: mass 0.0011084409433758843876 -> 0.0010324984452316546789
- link spur_gear_21_teeth: mass 0.0010185686142775145658 -> 0.0010254193609188259288
- link spur_gear_21_teeth_2: mass 0.0010185686142775145658 -> 0.0010254193609188259288
- link torso: mass 0.66652685450988358173 -> 1.071065963101194507
- link waist_gears: mass 0.026337180140419174518 -> 0.026337180140419177987
- link waist_link: mass 0.17011953490612458095 -> 0.17011953490612460871
Joints:
- joint left_hip_yaw_drive: origin xyz=-0.036999999999998457734 0.037100000000005961542 -0.03950000000000024325 rpy=-1.5707963267949545116 -4.8003070743589248247e-13 -3.5749181392930616155e-13 -> xyz=-0.036999999999999783062 0.031099999999999981826 -0.039200000000000179146 rpy=1.570796326794896558 -7.8039718066171778704e-18 -3.1415926535897740202
- joint left_hip_yaw_driven: origin xyz=-0.036999999999999998168 0.041100000000000011524 -0.019500000000000027728 rpy=-1.5707963267948947816 -1.570796326794896558 0 -> xyz=-0.036999999999999991229 0.041100000000000011524 -0.019500000000000006911 rpy=-1.5707963267948903408 -1.5707963267948950037 0
- joint left_leg_fixed: origin xyz=0 0 0.004999999999999997502 rpy=3.1415926535897926719 -1.9428902930939016723e-16 -7.6327832942984196016e-16 -> xyz=4.336808689942017736e-19 6.9388939039072283776e-18 0.004999999999999997502 rpy=3.1415926535897873428 4.1823223096112866159e-31 9.0864025441047529406e-31
- joint left_sho_pitch: origin xyz=-0.0030000000000002949654 0.062000000000001082023 0.10423651076281743866 rpy=-1.5707963267949081043 -4.127643409825574977e-14 3.4723733359249779961e-14 -> xyz=-0.0035000000000004693156 0.067000000000001086464 0.104236510762817286 rpy=-1.5707963267949081043 -4.127643409825574977e-14 3.4723733359249779961e-14
- joint neck_pitch_drive: child spur_gear_(13_teeth) -> spur_gear_13_teeth; origin xyz=-6.9735883734267645195e-16 0.015649999999999053557 -0.0087999999999970532349 rpy=-1.1409718301987536487e-15 4.409645192886135633e-16 -1.5707963267948976682 -> xyz=2.2030988144905450099e-15 0.015649999999998998046 -0.0087999999999980177412 rpy=-2.2204460492487858954e-16 -6.1232339955881360132e-17 -1.5707963267948970021
- joint neck_pitch_driven: origin xyz=3.7499979510524639181e-10 -0.0051500000614751947903 0.027499999999999941158 rpy=1.5707963267948978903 -2.0825786444073518345e-16 3.141592653589793116 -> xyz=3.7500001714985131684e-10 -0.0051500000614753864772 0.027499999999999982792 rpy=1.5707963267948976682 -2.0825786444061155416e-16 3.141592653589793116
- joint neck_yaw_driven: origin xyz=0.016000000000001235456 2.2310681558151314601e-17 0.12248651076281746874 rpy=-4.8668742840765556337e-16 -4.0649010562893427138e-15 3.141592653589793116 -> xyz=0.016000000000000298706 -1.0553952915478177074e-17 0.12248651076281746874 rpy=3.1251798320819254749e-16 -4.2234156679321592005e-15 3.1415926535897926719
- joint right_hip_yaw_drive: origin xyz=0.037000000000001719014 0.03710000000000327619 -0.0394999999999998061 rpy=-1.5707963267949545116 -4.8002361403961149694e-13 -3.5216274341110541015e-13 -> xyz=0.03699999999999992184 0.031100000000000113665 -0.03920000000000027629 rpy=1.5707963267948945596 3.4666037472893071652e-15 -3.1415926535897917837
- joint right_hip_yaw_driven: origin xyz=0.036999999999999991229 0.041100000000000011524 -0.019500000000000017319 rpy=-1.570796326794896558 -1.5707963267948961139 0 -> xyz=0.037000000000000005107 0.041099999999999997646 -0.019500000000000003442 rpy=-1.5707963267948943376 -1.5707963267948945596 0
- joint right_leg_fixed: origin xyz=0 -6.9388939039072283776e-18 0.0050000000000000044409 rpy=-3.1415926535897926719 1.8281169925220331315e-17 -3.5772536718062127375e-16 -> xyz=-4.336808689942017736e-19 6.9388939039072283776e-18 0.004999999999999997502 rpy=3.1415926535897904515 8.3266726857062000968e-16 -7.4940054151664101128e-16
- joint right_sho_pitch: origin xyz=-0.0029999999999986998872 -0.06200000000000097794 0.10423651076281731376 rpy=-1.5707963267948885644 3.4812325502379109658e-14 -3.1415926535897562566 -> xyz=-0.003499999999998689923 -0.067000000000001030953 0.10423651076281729988 rpy=-1.5707963267948885644 3.4812325502379109658e-14 -3.1415926535897562566
- joint waist_act_1: origin xyz=5.7457652915638341522e-17 0.019599999999999964673 -0.012750000000000025202 rpy=1.5707963267948954478 1.570796326794896336 0 -> xyz=1.414969124206259699e-16 0.019599999999999985489 -0.01275000000000047623 rpy=1.5707963267948943376 1.5707963267948952257 0
- joint waist_act_2: origin xyz=4.2745485696894321379e-17 0.019600000000000013245 -0.032749999999999994393 rpy=1.5707963267948956698 1.3463968515392303882 6.7698458176426589005e-15 -> xyz=1.5688834189823429471e-16 0.01960000000000029774 -0.032750000000000542566 rpy=1.5707963267948947816 1.3463968515392290559 2.1929231817633944674e-14
- joint waist_roll: origin xyz=-0.022707865260692617487 -2.4393502827093082036e-16 -0.013999999999999814676 rpy=-1.5707963267948974462 1.8675461532229772614e-15 1.5707963267948952257 -> xyz=-0.022707865260693019943 -1.1379796490832543078e-16 -0.013999999999999696715 rpy=-1.570796326794896558 5.9153252221758794299e-15 1.5707963267948923392
- joint waist_yaw: origin xyz=0 -3.1104917983741196655e-18 -7.5188305028877687703e-30 rpy=-1.4111145075746007461e-16 -4.1376224834060906822e-15 3.1415926535897922278 -> xyz=0 3.3155877990083308985e-18 -2.2531839605375149692e-29 rpy=1.5032209321489623492e-16 -4.1376224834056962518e-15 3.1415926535897917837

File: toddlerbot/robot_descriptions/toddlerbot_OP3/toddlerbot_OP3.urdf (robot description, URDF)
Before this commit: robot toddlerbot_OP3, 63 links, 62 joints
Links:
- removed link spur_gear_(13_teeth)
- added link spur_gear_13_teeth, mass 0.00091877519177533870359; visual mesh filename=../assemblies/toddlerbot/meshes/spur_gear_13_teeth_visual.s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
- link neck_pitch_link: mass 0.074299999993091794814 -> 0.07429999999309182257
- link spur_1m_20t: mass 0.0015534950290892282111 -> 0.0015778025963745999881
- link spur_gear_19_teeth: mass 0.0011084409433758843876 -> 0.0010324984452316546789
- link spur_gear_19_teeth_2: mass 0.0011084409433758843876 -> 0.0010324984452316546789
- link spur_gear_21_teeth: mass 0.0010185686142775145658 -> 0.0010254193609188259288
- link spur_gear_21_teeth_2: mass 0.0010185686142775145658 -> 0.0010254193609188259288
- link torso: mass 0.66652685450988358173 -> 1.071065963101194507
- link waist_gears: mass 0.026337180140419174518 -> 0.026337180140419177987
- link waist_link: mass 0.17011953490612458095 -> 0.17011953490612460871
Joints:
- joint left_hip_yaw_drive: origin xyz=-0.036999999999998457734 0.037100000000005961542 -0.03950000000000024325 rpy=-1.5707963267949545116 -4.8003070743589248247e-13 -3.5749181392930616155e-13 -> xyz=-0.036999999999999783062 0.031099999999999981826 -0.039200000000000179146 rpy=1.570796326794896558 -7.8039718066171778704e-18 -3.1415926535897740202
- joint left_hip_yaw_driven: origin xyz=-0.036999999999999998168 0.041100000000000011524 -0.019500000000000027728 rpy=-1.5707963267948947816 -1.570796326794896558 0 -> xyz=-0.036999999999999991229 0.041100000000000011524 -0.019500000000000006911 rpy=-1.5707963267948903408 -1.5707963267948950037 0
- joint left_leg_fixed: origin xyz=0 0 0.004999999999999997502 rpy=3.1415926535897926719 -1.9428902930939016723e-16 -7.6327832942984196016e-16 -> xyz=4.336808689942017736e-19 6.9388939039072283776e-18 0.004999999999999997502 rpy=3.1415926535897873428 4.1823223096112866159e-31 9.0864025441047529406e-31
- joint left_sho_pitch: origin xyz=-0.0030000000000002949654 0.062000000000001082023 0.10423651076281743866 rpy=-1.5707963267949081043 -4.127643409825574977e-14 3.4723733359249779961e-14 -> xyz=-0.0035000000000004693156 0.067000000000001086464 0.104236510762817286 rpy=-1.5707963267949081043 -4.127643409825574977e-14 3.4723733359249779961e-14
- joint neck_pitch_drive: child spur_gear_(13_teeth) -> spur_gear_13_teeth; origin xyz=-6.9735883734267645195e-16 0.015649999999999053557 -0.0087999999999970532349 rpy=-1.1409718301987536487e-15 4.409645192886135633e-16 -1.5707963267948976682 -> xyz=2.2030988144905450099e-15 0.015649999999998998046 -0.0087999999999980177412 rpy=-2.2204460492487858954e-16 -6.1232339955881360132e-17 -1.5707963267948970021
- joint neck_pitch_driven: origin xyz=3.7499979510524639181e-10 -0.0051500000614751947903 0.027499999999999941158 rpy=1.5707963267948978903 -2.0825786444073518345e-16 3.141592653589793116 -> xyz=3.7500001714985131684e-10 -0.0051500000614753864772 0.027499999999999982792 rpy=1.5707963267948976682 -2.0825786444061155416e-16 3.141592653589793116
- joint neck_yaw_driven: origin xyz=0.016000000000001235456 2.2310681558151314601e-17 0.12248651076281746874 rpy=-4.8668742840765556337e-16 -4.0649010562893427138e-15 3.141592653589793116 -> xyz=0.016000000000000298706 -1.0553952915478177074e-17 0.12248651076281746874 rpy=3.1251798320819254749e-16 -4.2234156679321592005e-15 3.1415926535897926719
- joint right_hip_yaw_drive: origin xyz=0.037000000000001719014 0.03710000000000327619 -0.0394999999999998061 rpy=-1.5707963267949545116 -4.8002361403961149694e-13 -3.5216274341110541015e-13 -> xyz=0.03699999999999992184 0.031100000000000113665 -0.03920000000000027629 rpy=1.5707963267948945596 3.4666037472893071652e-15 -3.1415926535897917837
- joint right_hip_yaw_driven: origin xyz=0.036999999999999991229 0.041100000000000011524 -0.019500000000000017319 rpy=-1.570796326794896558 -1.5707963267948961139 0 -> xyz=0.037000000000000005107 0.041099999999999997646 -0.019500000000000003442 rpy=-1.5707963267948943376 -1.5707963267948945596 0
- joint right_leg_fixed: origin xyz=0 -6.9388939039072283776e-18 0.0050000000000000044409 rpy=-3.1415926535897926719 1.8281169925220331315e-17 -3.5772536718062127375e-16 -> xyz=-4.336808689942017736e-19 6.9388939039072283776e-18 0.004999999999999997502 rpy=3.1415926535897904515 8.3266726857062000968e-16 -7.4940054151664101128e-16
- joint right_sho_pitch: origin xyz=-0.0029999999999986998872 -0.06200000000000097794 0.10423651076281731376 rpy=-1.5707963267948885644 3.4812325502379109658e-14 -3.1415926535897562566 -> xyz=-0.003499999999998689923 -0.067000000000001030953 0.10423651076281729988 rpy=-1.5707963267948885644 3.4812325502379109658e-14 -3.1415926535897562566
- joint waist_act_1: origin xyz=5.7457652915638341522e-17 0.019599999999999964673 -0.012750000000000025202 rpy=1.5707963267948954478 1.570796326794896336 0 -> xyz=1.414969124206259699e-16 0.019599999999999985489 -0.01275000000000047623 rpy=1.5707963267948943376 1.5707963267948952257 0
- joint waist_act_2: origin xyz=4.2745485696894321379e-17 0.019600000000000013245 -0.032749999999999994393 rpy=1.5707963267948956698 1.3463968515392303882 6.7698458176426589005e-15 -> xyz=1.5688834189823429471e-16 0.01960000000000029774 -0.032750000000000542566 rpy=1.5707963267948947816 1.3463968515392290559 2.1929231817633944674e-14
- joint waist_roll: origin xyz=-0.022707865260692617487 -2.4393502827093082036e-16 -0.013999999999999814676 rpy=-1.5707963267948974462 1.8675461532229772614e-15 1.5707963267948952257 -> xyz=-0.022707865260693019943 -1.1379796490832543078e-16 -0.013999999999999696715 rpy=-1.570796326794896558 5.9153252221758794299e-15 1.5707963267948923392
- joint waist_yaw: origin xyz=0 -3.1104917983741196655e-18 -7.5188305028877687703e-30 rpy=-1.4111145075746007461e-16 -4.1376224834060906822e-15 3.1415926535897922278 -> xyz=0 3.3155877990083308985e-18 -2.2531839605375149692e-29 rpy=1.5032209321489623492e-16 -4.1376224834056962518e-15 3.1415926535897917837
