Commit message: Update the MJCF

File: toddlerbot/descriptions/assemblies/left_leg_OP3/left_leg_OP3.urdf (robot description, URDF)
Before this commit: robot left_leg_OP3, 11 links, 10 joints
Links:
- link ank_roll_link: mass 0.042600000000000005917 -> 0.042599999999999998979
- link bearing_683: mass 0.00048694686130641804279 -> 0.00048694686130641793437
- link bearing_683_2: mass 0.00048694686130641804279 -> 0.00048694686130641793437
- link hip_yaw_link: mass 0.01799999999999999864 -> 0.017999999999999991701
- link knee_rod: mass 0.0031629468613064179276 -> 0.0031629468613064183613
- link knee_rod_2: mass 0.0031629468613064179276 -> 0.0031629468613064183613
- link left_calf_link: mass 0.030999999999999992839 -> 0.031000000000000006717
- link xm430_plate: mass 0.0026999999999999992756 -> 0.0026999999999999988419
Joints:
- removed joint left_knee_pitch
- added joint left_knee: type revolute, parent left_hip_pitch_link_xm430, child left_calf_link, origin xyz=3.2091917465512721632e-17 -0.09600000000000005751 -0.0091999999999999877015 rpy=2.8679386715174528955e-15 -1.3560834537223585781e-14 2.8113261283774143445e-14, axis 0 0 1, limit lower=0 upper=2.0943951023931952626 effort=1 velocity=20
- joint left_knee_act: origin xyz=-0.00014999999999968871242 -0.061500000000000318301 -0.030400000000000086675 rpy=-1.0593309150913038177e-14 1.0308748735206783672e-14 1.5707963267949243136 -> xyz=-0.00014999999999969307633 -0.061500000000000415445 -0.030400000000000086675 rpy=-1.3551714611180039898e-14 9.6309787132097184291e-17 1.5707963267949209829
- joint left_knee_back_rev_1: origin xyz=-0.013858192987669326612 -0.0057402514854763431879 -0.004999999999999997502 rpy=-4.4795806497323614513e-17 1.2898425949264794231e-14 -3.1386940726547587488 -> xyz=-0.013858192987669507024 -0.0057402514854763657393 -0.0049999999999999992367 rpy=-4.5070697379485943445e-17 2.6946050681063704762e-15 -3.1386940726547556402
- joint left_knee_front_rev_1: origin xyz=0.013858192987669507024 0.0057402514854762061447 -0.0050000000000007330248 rpy=7.2820716485250802911e-15 3.800162938454114633e-14 -3.1357955927274758778 -> xyz=0.013858192987669312735 0.0057402514854763414531 -0.0049999999999999992367 rpy=2.7406072773284573378e-15 2.7806511995613255269e-14 -3.1357955927274727692

File: toddlerbot/descriptions/assemblies/right_leg_OP3/right_leg_OP3.urdf (robot description, URDF)
Before this commit: robot right_leg_OP3, 11 links, 10 joints
Links:
- link ank_roll_link: mass 0.042600000000000005917 -> 0.042599999999999998979
- link bearing_683: mass 0.00048694686130641804279 -> 0.00048694686130641793437
- link bearing_683_2: mass 0.00048694686130641804279 -> 0.00048694686130641793437
- link hip_yaw_link: mass 0.01799999999999999864 -> 0.017999999999999991701
- link knee_rod: mass 0.0031629468613064179276 -> 0.0031629468613064183613
- link knee_rod_2: mass 0.0031629468613064179276 -> 0.0031629468613064183613
- link right_calf_link: mass 0.030999999999999982431 -> 0.03099999999999998937
- link right_hip_pitch_link_xm430: mass 0.1148009013503056841 -> 0.11480090135030569798
- link xm430_plate: mass 0.0026999999999999992756 -> 0.0026999999999999988419
Joints:
- removed joint right_knee_pitch
- added joint right_knee: type revolute, parent right_hip_pitch_link_xm430, child right_calf_link, origin xyz=6.6012271456357184538e-18 -0.095999999999999877098 -0.009199999999999972089 rpy=-9.138977281102487298e-16 5.7742659530791861042e-17 3.141592653589793116, axis 0 0 1, limit lower=-2.0943951023931952626 upper=0 effort=1 velocity=20

File: toddlerbot/descriptions/assemblies/toddlerbot/toddlerbot.urdf (robot description, URDF)
Before this commit: robot toddlerbot, 17 links, 16 joints
Links:
- removed link neck_pitch_link
- removed link neck_yaw_link
- removed link spur_gear_13_teeth
- added link bearing_683, mass 0.00048694686130641793437; collision mesh filename=package:///meshes/bearing_683_collision.stl; visual mesh filename=package:///meshes/bearing_683_visual.stl
- added link bearing_683_2, mass 0.00048694686130641793437; collision mesh filename=package:///meshes/bearing_683_2_collision.stl; visual mesh filename=package:///meshes/bearing_683_2_visual.stl
- added link head, mass 0.12772101760550844118; collision mesh filename=package:///meshes/head_collision.stl; visual mesh filename=package:///meshes/head_visual.stl
- added link motor_plate, mass 0.0016999999999999996884; collision mesh filename=package:///meshes/motor_plate_collision.stl; visual mesh filename=package:///meshes/motor_plate_visual.stl
- added link neck_rod, mass 0.0031629468613064183613; collision mesh filename=package:///meshes/neck_rod_collision.stl; visual mesh filename=package:///meshes/neck_rod_visual.stl
- added link neck_rod_2, mass 0.0031629468613064183613; collision mesh filename=package:///meshes/neck_rod_2_collision.stl; visual mesh filename=package:///meshes/neck_rod_2_visual.stl
- added link neck_yaw_link_v2, mass 0.0067298837334394089049; collision mesh filename=package:///meshes/neck_yaw_link_v2_collision.stl; visual mesh filename=package:///meshes/neck_yaw_link_v2_visual.stl
- link left_arm_hand: mass 0.0085999999999999930667 -> 0.0085999999999999895972
- link left_leg_xm430: mass 0.01799999999999999864 -> 0.017999999999999991701
- link right_arm_hand: mass 0.0085999999999999930667 -> 0.0085999999999999895972
- link right_leg_xm430: mass 0.01799999999999999864 -> 0.017999999999999991701
- link spur_1m_20t: mass 0.0015778025963745999881 -> 0.0015778025963745997712
- link spur_gear_19_teeth: mass 0.0010324984452316546789 -> 0.0010324984452316548957
- link spur_gear_19_teeth_2: mass 0.0010324984452316546789 -> 0.0010324984452316548957
- link torso: mass 1.071065963101194507 -> 1.1229659631011945642
- link waist_gears: mass 0.026337180140419177987 -> 0.026337180140419174518
- link waist_link: mass 0.17011953490612460871 -> 0.1701195349061245532
Joints:
- removed joint neck_pitch_drive
- removed joint neck_pitch_driven
- added joint neck_pitch: type revolute, parent neck_yaw_link_v2, child head, origin xyz=-1.0061396160665481148e-16 0.0040000000000000607986 0.019400000000000028333 rpy=-1.570796326790486086 1.567169222346451507 3.1415926535866449676, axis 0 0 1, limit lower=-1.3962634015954635824 upper=0.61086523819801530344 effort=1 velocity=20
- added joint neck_pitch_act: type revolute, parent head, child motor_plate, origin xyz=-0.032615697718559516494 -0.026999999999999642342 0.0024999999999980927236 rpy=-3.1415926535897824579 -3.0391096960732561898e-13 -3.1415926535894773686, axis 0 0 1, limit lower=-1.3962634015954635824 upper=0.61086523819801530344 effort=1 velocity=20
- added joint neck_pitch_back_rev_1: type revolute, parent neck_yaw_link_v2, child neck_rod_2, origin xyz=0.007244443697168208296 -0.0040000000000001215139 0.021341142838269100412 rpy=1.570796326794926312 -0.88149812103389046936 3.1415926535897855665, axis 0 0 1, limit lower=-6.283185307179586232 upper=6.283185307179586232 effort=1 velocity=20
- added joint neck_pitch_back_rev_2: type revolute, parent motor_plate, child bearing_683_2, origin xyz=0.0019411428382689055461 0.0072444436971680157417 -0.0055000000000000014155 rpy=-2.6894721862809934635e-13 -1.70427982545233833e-13 0.87787101658577615382, axis 0 0 1, limit lower=-6.283185307179586232 upper=6.283185307179586232 effort=1 velocity=20
- added joint neck_pitch_front_rev_1: type revolute, parent neck_yaw_link_v2, child neck_rod, origin xyz=-0.0072444436971683887072 -0.0040000000000001223813 0.01745885716173128932 rpy=1.5707963267944309305 -0.8843930473262051617 -3.1415926535893787808, axis 0 0 1, limit lower=-6.283185307179586232 upper=6.283185307179586232 effort=1 velocity=20
- added joint neck_pitch_front_rev_2: type revolute, parent motor_plate, child bearing_683, origin xyz=-0.0019411428382688777905 -0.0072444436971680140069 -0.0055000000000000014155 rpy=-6.4149072816529488098e-15 7.6581010280206250727e-15 0.88076594287809084616, axis 0 0 1, limit lower=-6.283185307179586232 upper=6.283185307179586232 effort=1 velocity=20
- joint left_hip_yaw_drive: origin xyz=-0.036999999999999783062 0.031099999999999981826 -0.039200000000000179146 rpy=1.570796326794896558 -7.8039718066171778704e-18 -3.1415926535897740202 -> xyz=-0.03700000000000004674 0.03110000000000001652 -0.039199999999999998734 rpy=1.570796326794896558 -6.0440960687789003209e-17 3.141592653589793116
- joint left_hip_yaw_driven: origin xyz=-0.036999999999999991229 0.041100000000000011524 -0.019500000000000006911 rpy=-1.5707963267948903408 -1.5707963267948950037 0 -> xyz=-0.037000000000000012046 0.04109999999999997683 -0.019500000000000017319 rpy=-1.5707963267949192065 -1.5707963267948790165 0
- joint left_leg_fixed: origin xyz=4.336808689942017736e-19 6.9388939039072283776e-18 0.004999999999999997502 rpy=3.1415926535897873428 4.1823223096112866159e-31 9.0864025441047529406e-31 -> xyz=2.168404344971008868e-18 -1.3877787807814456755e-17 0.0049999999999999905631 rpy=-3.1415926535897704674 -7.7860248023657121854e-31 -1.137084089218072634e-30
- joint neck_yaw_drive: origin xyz=-0.004999999999999517851 2.6555840535020396321e-18 0.121486510762817565 rpy=1.1318451824181020002e-14 2.6985403517595457696e-15 -5.3863140912757267331e-15 -> xyz=-0.0049999999999995221878 3.1860588521011854095e-18 0.12148651076281755112 rpy=1.1607298201443905188e-14 1.6509758832059179101e-15 -5.3832337592600790636e-15
- joint neck_yaw_driven: child neck_yaw_link -> neck_yaw_link_v2; origin xyz=0.016000000000000298706 -1.0553952915478177074e-17 0.12248651076281746874 rpy=3.1251798320819254749e-16 -4.2234156679321592005e-15 3.1415926535897926719 -> xyz=0.016000000000000621364 3.9122381713629107253e-19 0.12248651076281739936 rpy=1.5470695466536949876e-14 -3.0902695541116811913e-15 -8.6007558735577539147e-16
- joint right_hip_yaw_drive: origin xyz=0.03699999999999992184 0.031100000000000113665 -0.03920000000000027629 rpy=1.5707963267948945596 3.4666037472893071652e-15 -3.1415926535897917837 -> xyz=0.036999999999999942657 0.031100000000000009581 -0.039200000000000005673 rpy=1.57079632679489678 3.044498544160610484e-18 3.141592653589793116
- joint right_hip_yaw_driven: origin xyz=0.037000000000000005107 0.041099999999999997646 -0.019500000000000003442 rpy=-1.5707963267948943376 -1.5707963267948945596 0 -> xyz=0.03699999999999998429 0.041099999999999969891 -0.019500000000000017319 rpy=-1.570796326794896558 -1.570796326794896558 0
- joint right_leg_fixed: origin xyz=-4.336808689942017736e-19 6.9388939039072283776e-18 0.004999999999999997502 rpy=3.1415926535897904515 8.3266726857062000968e-16 -7.4940054151664101128e-16 -> xyz=-4.336808689942017736e-19 -6.9388939039072283776e-18 0.0050000000000000113798 rpy=-3.141592653589793116 9.3906761299382808154e-30 1.9103766403509957361e-30
- joint waist_act_1: origin xyz=1.414969124206259699e-16 0.019599999999999985489 -0.01275000000000047623 rpy=1.5707963267948943376 1.5707963267948952257 0 -> xyz=-2.3414432044644055064e-17 0.019600000000000124267 -0.01275000000000019347 rpy=1.5707963267948936714 1.5707963267948950037 0
- joint waist_act_2: origin xyz=1.5688834189823429471e-16 0.01960000000000029774 -0.032750000000000542566 rpy=1.5707963267948947816 1.3463968515392290559 2.1929231817633944674e-14 -> xyz=-1.4470390030684367241e-17 0.019600000000000561418 -0.032750000000000556444 rpy=1.5707963267948972241 1.3463968515392352732 -2.5409194566005071493e-16
- joint waist_roll: origin xyz=-0.022707865260693019943 -1.1379796490832543078e-16 -0.013999999999999696715 rpy=-1.570796326794896558 5.9153252221758794299e-15 1.5707963267948923392 -> xyz=-0.022707865260692055437 -1.3063957582126781116e-17 -0.013999999999999981209 rpy=-1.5707963267948956698 -5.9937357430034153564e-14 1.5707963267948785724
- joint waist_yaw: origin xyz=0 3.3155877990083308985e-18 -2.2531839605375149692e-29 rpy=1.5032209321489623492e-16 -4.1376224834056962518e-15 3.1415926535897917837 -> xyz=0 3.6977854932234928379e-32 -2.4651903288156618919e-32 rpy=-3.0322117681687121616e-16 -4.1243331367303576527e-15 3.1415926535897904515
