Commit message: Update the ankle pitch to use XM430

File: toddlerbot/descriptions/assemblies/left_leg_OP3/left_leg_OP3.urdf (robot description, URDF)
Before this commit: robot left_leg_OP3, 11 links, 10 joints
Links:
- link ank_pitch_link: mass 0.15976376693924948524 -> 0.17676376695067905209
- link ank_roll_link: mass 0.042599999999999998979 -> 0.042600000000000005917
- link hip_yaw_link: mass 0.017999999999999991701 -> 0.017999999999999995171
- link knee_rod: mass 0.0031629468613064183613 -> 0.0031629468613064174939
- link knee_rod_2: mass 0.0031629468613064183613 -> 0.0031629468613064174939
- link left_calf_link: mass 0.031000000000000006717 -> 0.030999999999999996309
- link left_hip_pitch_link_xm430: mass 0.11480090135030569798 -> 0.11480090135030573961
- link xm430_plate: mass 0.0026999999999999988419 -> 0.0026999999999999992756
Joints:
- joint left_ank_pitch: origin xyz=0.00050000000000001020191 -0.099999999999999866773 -0.029399999999999901906 rpy=1.3838214396829414281e-15 2.3817753328472465846e-15 -1.5707963267948936714 -> xyz=0.00050000000000032288582 -0.099999999999996785904 -0.029400000000000661715 rpy=-3.7313901977116486581e-15 1.1636199395949206391e-16 -5.2669342108558058169e-15
- joint left_ank_roll: origin xyz=-1.3877787807814456755e-15 0.022750000000004225176 0.019000000000006383311 rpy=1.5707963267949556219 8.2263916424954431126e-14 3.1415926535897686911 -> xyz=0.022749999999994167249 -8.3266726846886740532e-17 0.019000000000001897316 rpy=1.5707963267950513231 1.4301315653119179755e-13 1.5707963267948481523
- joint left_hip_pitch: origin xyz=-0.024000000716156173058 -0.019000000152439983775 -0.019000000152458156738 rpy=1.5707963267953681807 1.570796326794433817 0 -> xyz=-0.024000000716156828784 -0.019000000152440157247 -0.019000000152458548786 rpy=1.5707963267953657382 1.5707963267943103602 0
- joint left_hip_roll: origin xyz=0.018999999999999999528 -3.3408590380433372139e-18 -0.026000000000000002276 rpy=3.141592653589793116 -1.5707963267948821251 0 -> xyz=0.018999999999999905853 4.4904419342659082281e-16 -0.025999999999999946765 rpy=-3.141592653589793116 -1.5707963267948918951 0
- joint left_knee: origin xyz=3.2091917465512721632e-17 -0.09600000000000005751 -0.0091999999999999877015 rpy=2.8679386715174528955e-15 -1.3560834537223585781e-14 2.8113261283774143445e-14 -> xyz=2.990790261972040031e-17 -0.09600000000000055711 -0.0092000000000000276001 rpy=2.5205532109825094148e-15 5.7598642354355467767e-16 3.8634704751188379083e-16
- joint left_knee_act: origin xyz=-0.00014999999999969307633 -0.061500000000000415445 -0.030400000000000086675 rpy=-1.3551714611180039898e-14 9.6309787132097184291e-17 1.5707963267949209829 -> xyz=-0.00015000000000009954372 -0.06150000000000001299 -0.030399999999999812589 rpy=-1.8754556207585452854e-15 2.8209809769508020585e-14 1.5707963267948990005
- joint left_knee_back_rev_1: origin xyz=-0.013858192987669507024 -0.0057402514854763657393 -0.0049999999999999992367 rpy=-4.5070697379485943445e-17 2.6946050681063704762e-15 -3.1386940726547556402 -> xyz=-0.013858192987669298857 -0.0057402514854763449226 -0.004999999999999997502 rpy=-2.3102540588711712824e-15 2.7442875060730908856e-14 -3.1386940726547187808
- joint left_knee_back_rev_2: origin xyz=0.0057402514854763535962 -0.013858192987669326612 -0.026199999999999907391 rpy=4.2802438278248956281e-17 2.6960450327599089653e-16 1.5736949077299307032 -> xyz=0.0057402514854764195157 -0.013858192987669493146 -0.026199999999999154521 rpy=5.4450106890480900015e-16 3.294464518329961217e-15 1.5736949077299704491
- joint left_knee_front_rev_1: origin xyz=0.013858192987669312735 0.0057402514854763414531 -0.0049999999999999992367 rpy=2.7406072773284573378e-15 2.7806511995613255269e-14 -3.1357955927274727692 -> xyz=0.013858192987669298857 0.0057402514854763440552 -0.004999999999999997502 rpy=-2.1480523090933430766e-15 2.7897458296366629566e-14 -3.1357955927274452357
- joint left_knee_front_rev_2: origin xyz=-0.0057402514854763509941 0.013858192987669243346 -0.026199999999999896982 rpy=3.0668764952338581412e-14 -2.4824741237762853711e-14 1.5765933876572135741 -> xyz=-0.0057402514854763319122 0.013858192987668660479 -0.026199999999999112887 rpy=8.8484216442970563213e-16 3.3685549164292615233e-15 1.576593387657243106

File: toddlerbot/descriptions/assemblies/right_leg_OP3/right_leg_OP3.urdf (robot description, URDF)
Before this commit: robot right_leg_OP3, 11 links, 10 joints
Links:
- link ank_pitch_link: mass 0.15976376693924948524 -> 0.17676376695067905209
- link ank_roll_link: mass 0.042599999999999998979 -> 0.042600000000000005917
- link hip_yaw_link: mass 0.017999999999999991701 -> 0.017999999999999995171
- link knee_rod: mass 0.0031629468613064183613 -> 0.0031629468613064174939
- link knee_rod_2: mass 0.0031629468613064183613 -> 0.0031629468613064174939
- link right_calf_link: mass 0.03099999999999998937 -> 0.030999999999999992839
- link right_hip_pitch_link_xm430: mass 0.11480090135030569798 -> 0.11480090135030572573
- link xm430_plate: mass 0.0026999999999999988419 -> 0.0026999999999999992756
Joints:
- joint right_ank_pitch: origin xyz=0.00050000000000040452624 0.10000000000000006106 0.0086000000000003035822 rpy=3.141592653589793116 -9.7384055572523312245e-16 1.5707963267948936714 -> xyz=0.00050000000000016339968 0.099999999999997118971 0.0086000000000002446016 rpy=-3.1415926535897926719 3.5599385721621441668e-15 5.4262150328496371087e-15
- joint right_ank_roll: origin xyz=1.9151347174783950322e-15 0.022749999999999825917 0.019000000000001193018 rpy=1.5707963267949667241 3.4534200721523706957e-14 3.1415926535897917837 -> xyz=0.022749999999995992178 -1.249000902703301108e-15 0.018999999999999073186 rpy=1.5707963267948399366 2.9058912904735880454e-14 1.5707963267948754638

File: toddlerbot/descriptions/assemblies/toddlerbot/toddlerbot.urdf (robot description, URDF)
Before this commit: robot toddlerbot, 21 links, 20 joints
Links:
- link head: mass 0.12772101760550844118 -> 0.12772101760550846894
- link neck_rod: mass 0.0031629468613064183613 -> 0.0031629468613064179276
- link neck_rod_2: mass 0.0031629468613064183613 -> 0.0031629468613064179276
- link neck_yaw_link_v2: mass 0.0067298837334394089049 -> 0.0067298837334394080376
- link spiral_bevel_1m_14t_30deg: mass 0.00073261524436595481732 -> 0.00073261524436595492574
- link spiral_bevel_1m_14t_30deg_2: mass 0.00073261524436595481732 -> 0.00073261524436595492574
- link spur_gear_19_teeth: mass 0.0010324984452316548957 -> 0.0010324984452316546789
- link spur_gear_19_teeth_2: mass 0.0010324984452316548957 -> 0.0010324984452316546789
- link spur_gear_21_teeth: mass 0.0010254193609188259288 -> 0.0010254193609188257119
- link spur_gear_21_teeth_2: mass 0.0010254193609188259288 -> 0.0010254193609188257119
- link torso: mass 1.1229659631011945642 -> 1.1369659631011950207
- link waist_gears: mass 0.026337180140419174518 -> 0.026337180140419177987
- link waist_link: mass 0.1701195349061245532 -> 0.17011953490612458095

File: toddlerbot/descriptions/toddlerbot_OP3/toddlerbot_OP3.urdf (robot description, URDF)
Before this commit: robot toddlerbot_OP3, 67 links, 66 joints
Links:
- link ank_pitch_link: mass 0.15976376693924948524 -> 0.17676376695067905209
- link ank_pitch_link_2: mass 0.15976376693924948524 -> 0.17676376695067905209
- link ank_roll_link: mass 0.042599999999999998979 -> 0.042600000000000005917
- link ank_roll_link_2: mass 0.042599999999999998979 -> 0.042600000000000005917
- link head: mass 0.12772101760550844118 -> 0.12772101760550846894
- link hip_yaw_link: mass 0.017999999999999991701 -> 0.017999999999999995171
- link hip_yaw_link_2: mass 0.017999999999999991701 -> 0.017999999999999995171
- link knee_rod: mass 0.0031629468613064183613 -> 0.0031629468613064174939
- link knee_rod_2: mass 0.0031629468613064183613 -> 0.0031629468613064174939
- link knee_rod_3: mass 0.0031629468613064183613 -> 0.0031629468613064174939
- link knee_rod_4: mass 0.0031629468613064183613 -> 0.0031629468613064174939
- link left_calf_link: mass 0.031000000000000006717 -> 0.030999999999999996309
- link left_hip_pitch_link_xm430: mass 0.11480090135030569798 -> 0.11480090135030573961
- link neck_rod: mass 0.0031629468613064183613 -> 0.0031629468613064179276
- link neck_rod_2: mass 0.0031629468613064183613 -> 0.0031629468613064179276
- link neck_yaw_link_v2: mass 0.0067298837334394089049 -> 0.0067298837334394080376
- link right_calf_link: mass 0.03099999999999998937 -> 0.030999999999999992839
- link right_hip_pitch_link_xm430: mass 0.11480090135030569798 -> 0.11480090135030572573
- link spiral_bevel_1m_14t_30deg: mass 0.00073261524436595481732 -> 0.00073261524436595492574
- link spiral_bevel_1m_14t_30deg_2: mass 0.00073261524436595481732 -> 0.00073261524436595492574
- link spur_gear_19_teeth: mass 0.0010324984452316548957 -> 0.0010324984452316546789
- link spur_gear_19_teeth_2: mass 0.0010324984452316548957 -> 0.0010324984452316546789
- link spur_gear_21_teeth: mass 0.0010254193609188259288 -> 0.0010254193609188257119
- link spur_gear_21_teeth_2: mass 0.0010254193609188259288 -> 0.0010254193609188257119
- link torso: mass 1.1229659631011945642 -> 1.1369659631011950207
- link waist_gears: mass 0.026337180140419174518 -> 0.026337180140419177987
- link waist_link: mass 0.1701195349061245532 -> 0.17011953490612458095
- link xm430_plate: mass 0.0026999999999999988419 -> 0.0026999999999999992756
- link xm430_plate_2: mass 0.0026999999999999988419 -> 0.0026999999999999992756
Joints:
- joint left_ank_pitch: origin xyz=0.00050000000000001020191 -0.099999999999999866773 -0.029399999999999901906 rpy=1.3838214396829414281e-15 2.3817753328472465846e-15 -1.5707963267948936714 -> xyz=0.00050000000000032288582 -0.099999999999996785904 -0.029400000000000661715 rpy=-3.7313901977116486581e-15 1.1636199395949206391e-16 -5.2669342108558058169e-15
- joint left_ank_roll: origin xyz=-1.3877787807814456755e-15 0.022750000000004225176 0.019000000000006383311 rpy=1.5707963267949556219 8.2263916424954431126e-14 3.1415926535897686911 -> xyz=0.022749999999994167249 -8.3266726846886740532e-17 0.019000000000001897316 rpy=1.5707963267950513231 1.4301315653119179755e-13 1.5707963267948481523
- joint left_hip_pitch: origin xyz=-0.024000000716156173058 -0.019000000152439983775 -0.019000000152458156738 rpy=1.5707963267953681807 1.570796326794433817 0 -> xyz=-0.024000000716156828784 -0.019000000152440157247 -0.019000000152458548786 rpy=1.5707963267953657382 1.5707963267943103602 0
- joint left_hip_roll: origin xyz=0.018999999999999999528 -3.3408590380433372139e-18 -0.026000000000000002276 rpy=3.141592653589793116 -1.5707963267948821251 0 -> xyz=0.018999999999999905853 4.4904419342659082281e-16 -0.025999999999999946765 rpy=-3.141592653589793116 -1.5707963267948918951 0
- joint left_knee: origin xyz=3.2091917465512721632e-17 -0.09600000000000005751 -0.0091999999999999877015 rpy=2.8679386715174528955e-15 -1.3560834537223585781e-14 2.8113261283774143445e-14 -> xyz=2.990790261972040031e-17 -0.09600000000000055711 -0.0092000000000000276001 rpy=2.5205532109825094148e-15 5.7598642354355467767e-16 3.8634704751188379083e-16
- joint left_knee_act: origin xyz=-0.00014999999999969307633 -0.061500000000000415445 -0.030400000000000086675 rpy=-1.3551714611180039898e-14 9.6309787132097184291e-17 1.5707963267949209829 -> xyz=-0.00015000000000009954372 -0.06150000000000001299 -0.030399999999999812589 rpy=-1.8754556207585452854e-15 2.8209809769508020585e-14 1.5707963267948990005
- joint left_knee_back_rev_1: origin xyz=-0.013858192987669507024 -0.0057402514854763657393 -0.0049999999999999992367 rpy=-4.5070697379485943445e-17 2.6946050681063704762e-15 -3.1386940726547556402 -> xyz=-0.013858192987669298857 -0.0057402514854763449226 -0.004999999999999997502 rpy=-2.3102540588711712824e-15 2.7442875060730908856e-14 -3.1386940726547187808
- joint left_knee_back_rev_2: origin xyz=0.0057402514854763535962 -0.013858192987669326612 -0.026199999999999907391 rpy=4.2802438278248956281e-17 2.6960450327599089653e-16 1.5736949077299307032 -> xyz=0.0057402514854764195157 -0.013858192987669493146 -0.026199999999999154521 rpy=5.4450106890480900015e-16 3.294464518329961217e-15 1.5736949077299704491
- joint left_knee_front_rev_1: origin xyz=0.013858192987669312735 0.0057402514854763414531 -0.0049999999999999992367 rpy=2.7406072773284573378e-15 2.7806511995613255269e-14 -3.1357955927274727692 -> xyz=0.013858192987669298857 0.0057402514854763440552 -0.004999999999999997502 rpy=-2.1480523090933430766e-15 2.7897458296366629566e-14 -3.1357955927274452357
- joint left_knee_front_rev_2: origin xyz=-0.0057402514854763509941 0.013858192987669243346 -0.026199999999999896982 rpy=3.0668764952338581412e-14 -2.4824741237762853711e-14 1.5765933876572135741 -> xyz=-0.0057402514854763319122 0.013858192987668660479 -0.026199999999999112887 rpy=8.8484216442970563213e-16 3.3685549164292615233e-15 1.576593387657243106
- joint right_ank_pitch: origin xyz=0.00050000000000040452624 0.10000000000000006106 0.0086000000000003035822 rpy=3.141592653589793116 -9.7384055572523312245e-16 1.5707963267948936714 -> xyz=0.00050000000000016339968 0.099999999999997118971 0.0086000000000002446016 rpy=-3.1415926535897926719 3.5599385721621441668e-15 5.4262150328496371087e-15
- joint right_ank_roll: origin xyz=1.9151347174783950322e-15 0.022749999999999825917 0.019000000000001193018 rpy=1.5707963267949667241 3.4534200721523706957e-14 3.1415926535897917837 -> xyz=0.022749999999995992178 -1.249000902703301108e-15 0.018999999999999073186 rpy=1.5707963267948399366 2.9058912904735880454e-14 1.5707963267948754638
