Commit message: merge auto encoder

File: toddlerbot/descriptions/assemblies/toddlerbot/toddlerbot.urdf (robot description, URDF)
Before this commit: robot toddlerbot, 17 links, 16 joints
Links:
- link head: mass 0.13722101760550839411 -> 0.13722101760550836635
- link neck_rod: mass 0.0031629468613064174939 -> 0.0031629468613064179276
- link neck_rod_2: mass 0.0031629468613064174939 -> 0.0031629468613064179276
- link neck_yaw_link_v2: mass 0.0067298837334394097723 -> 0.0067298837334394080376
- link torso: mass 1.085065963101202513 -> 1.0850659631011949635

File: toddlerbot/descriptions/toddlerbot/toddlerbot.urdf (robot description, URDF)
Before this commit: robot toddlerbot, 67 links, 66 joints
Links:
- link left_hip_pitch_link: geometry collision capsule length=0.03288564731177622 radius=0.03603217800708148; visual mesh filename=../assemblies/left_leg_reorder/meshes/left_hip_pitch_link_v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
