Commit message: Update the knee joint limit

File: toddlerbot/descriptions/assemblies/left_leg_2xm/left_leg_2xm.urdf (robot description, URDF)
Before this commit: robot left_leg_2xm, 13 links, 12 joints
Links:
- link hip_yaw_link: mass 0.013199999999999994724 -> 0.013199999999999989519
- link knee_rod: mass 0.0031629468613064166266 -> 0.0031629468613064179276
- link knee_rod_2: mass 0.0031629468613064166266 -> 0.0031629468613064179276
- link left_calf_link: mass 0.030999999999999999778 -> 0.03099999999999998937
- link spur_gear_18_teeth: mass 0.0008039935629263021688 -> 0.0012000000000000001117
- link spur_gear_21_teeth: mass 0.0022000000000000001325 -> 0.0021999999999999996989
Joints:
- joint left_ank_pitch: origin xyz=1.5046216775048590637e-16 0.099999999999999783507 0.027749999999999604844 rpy=3.141592653589793116 -4.9446121195035926866e-18 1.1657341758499214505e-15 -> xyz=1.3731962615615156409e-15 0.099999999999997951639 0.02774999999999918851 rpy=3.141592653589793116 -4.9446121211182754037e-18 -2.0452759225209035521e-15
- joint left_ank_roll: origin xyz=0.022749999999983006038 -8.8540286213856234099e-15 0.019000000000000970973 rpy=-1.5707963267949500707 -9.3226942268794927216e-15 1.5707963267952123054 -> xyz=0.022749999999981843773 -7.882583474838611437e-15 0.01900000000000073852 rpy=-1.5707963267949500707 -9.3641111455497678285e-15 1.5707963267951978725
- joint left_hip_roll: origin xyz=-0.024000000716155295288 0.023000000152476038351 0.019000000152447446555 rpy=1.5707963267945725949 -1.5707963267948183983 0 -> xyz=-0.023749999999998987199 0.022750000000000013267 -0.019050000000000236883 rpy=1.5707963267948872321 -1.5707963267948945596 0
- joint left_hip_yaw_drive: origin xyz=-0.019199999999995876615 0.00020000000000328088667 0.0064999999999706473131 rpy=-3.1415926535897922278 -1.8640355840337264655e-15 3.1415926535897926719 -> xyz=-0.019199999999993382083 0.00020000000000426967905 -3.438915818776422384e-14 rpy=-3.1415926535896581129 -4.9090714472496588269e-13 4.6739125815344266384e-13
- joint left_hip_yaw_driven: origin xyz=6.7133798344526554386e-18 2.4286128663675299322e-17 -0.0050000000000001085243 rpy=-3.1415926535897922278 -4.1724555867713866127e-17 7.2164496631611534065e-16 -> xyz=-1.5720931501039814293e-18 -3.4694469519536141888e-18 -0.0050000000000000044409 rpy=-3.1415926535897904515 -2.6731719319053922034e-15 1.0531803182873569707e-15
- joint left_hip_yaw_fixed: origin xyz=-6.9388939039072283776e-18 0.028000000000000004052 0.023000000000000003081 rpy=1.570796326794896558 -1.5707963267948945596 0 -> xyz=0 0.027999999999999993644 0.02300000000000000655 rpy=1.570796326794896336 -1.5707963267948870101 0
- joint left_knee: limit lower=-2.0943951023931952626 upper=0 effort=1 velocity=20 -> lower=-1.570796326794896558 upper=0 effort=1 velocity=20; origin xyz=2.8177799257657431582e-18 -0.0087500000000000563438 0.085949999999999887601 rpy=1.5707963267948985564 1.8042036078715074883e-15 3.1415926535897926719 -> xyz=3.2303803729205604611e-16 -0.0087500000000000285882 0.085950000000000484346 rpy=1.5707963267948998887 9.1903399882501304125e-17 -3.1415926535897926719
- joint left_knee_act: limit lower=-2.0943951023931952626 upper=0 effort=1 velocity=20 -> lower=-1.570796326794896558 upper=0 effort=1 velocity=20; origin xyz=4.9996245779180309423e-17 0.012450000000000013139 0.044500000000000046463 rpy=-1.5707963267948956698 1.5707963267948954478 0 -> xyz=1.4647571350279164903e-16 0.012449999999999985384 0.044500000000000053402 rpy=-1.57079632679489678 1.5707963267948930053 0
- joint left_knee_back_rev_1: origin xyz=-0.013858192987669243346 0.0057402514854763518615 0.0049999999999999836242 rpy=-3.1415926535897926719 2.8925793879955221593e-16 3.1404544176206239392 -> xyz=-0.013858192987669118446 0.0057402514854763457899 0.0049999999999999888284 rpy=3.1415926535897873428 1.9452985330695691049e-16 -3.1404562276602714377
- joint left_knee_back_rev_2: origin xyz=0.0057402514854763128302 0.013858192987669548657 0.026199999999999803307 rpy=3.1415926535897926719 -1.0795076530726939777e-15 -1.5719345627640688434 -> xyz=0.0057402514854765652325 0.013858192987669493146 0.026199999999999244726 rpy=-3.1415926535897873428 -6.1642758581299746636e-16 -1.569659900865386204
- joint left_knee_front_rev_1: origin xyz=0.013858192987669326612 -0.0057402514854763405858 0.0049999999999999142353 rpy=-3.1415926535897926719 -7.0790895644363073118e-16 3.1403871344570966073 -> xyz=0.013858192987669049057 -0.0057402514854763527288 0.0049999999999999914305 rpy=-3.1415926535897908956 3.4964474193337374653e-15 -3.1404560691349008295
- joint left_knee_front_rev_2: origin xyz=-0.0057402514854764073726 -0.01385819298766896579 0.026199999999999803307 rpy=3.141592653589793116 1.9636585933148879161e-17 -1.5720018459275957312 -> xyz=-0.0057402514854763136976 -0.013858192987669076812 0.026199999999999178807 rpy=3.141592653589793116 -3.6846712218145297232e-15 -1.5696597423400153737

File: toddlerbot/descriptions/assemblies/right_leg_2xm/right_leg_2xm.urdf (robot description, URDF)
Before this commit: robot right_leg_2xm, 13 links, 12 joints
Links:
- link hip_yaw_link: mass 0.013199999999999994724 -> 0.013199999999999989519
- link knee_rod: mass 0.0031629468613064166266 -> 0.0031629468613064179276
- link knee_rod_2: mass 0.0031629468613064166266 -> 0.0031629468613064179276
- link right_calf_link: mass 0.030999999999999992839 -> 0.0309999999999999859
- link right_thigh_link: mass 0.14548965119785950417 -> 0.14548965119785953193
- link spur_gear_18_teeth: mass 0.0008039935629263021688 -> 0.0012000000000000001117
- link spur_gear_21_teeth: mass 0.0022000000000000001325 -> 0.0021999999999999996989
Joints:
- joint right_ank_pitch: origin xyz=6.3426567189575575897e-16 -0.099999999999999256151 0.027750000000000531186 rpy=3.141592653589793116 -5.3018417016982154559e-16 -3.1415926535897917837 -> xyz=3.5236570605778894105e-17 -0.09999999999999995004 0.027749999999999993422 rpy=-3.1415926535897917837 -7.8513249565814058339e-16 -3.1415926535897864547
- joint right_ank_roll: origin xyz=-0.022749999999990111466 -3.2474023470285828807e-15 0.018999999999999316047 rpy=1.5707963267948144015 7.8784525869511768317e-15 1.5707963267948383823 -> xyz=-0.022749999999990028199 -3.5249581031848720158e-15 0.018999999999999451356 rpy=1.5707963267948190644 2.082200812017336445e-14 1.5707963267948397146
- joint right_hip_roll: origin xyz=-0.024000000716140813817 -0.022999999847552448501 0.019000000152444362217 rpy=-1.5707963267949578423 1.5707963267948077402 0 -> xyz=-0.023750000000001200706 -0.022749999999999999389 -0.018950000000000081363 rpy=-1.570796326794896558 1.5707963267948952257 0
- joint right_hip_yaw_drive: origin xyz=0.01919999999999948137 0.00019999999999986001198 0.0059999999999661712824 rpy=3.141592653589793116 -1.7243077159172707227e-15 -3.1415926535897926719 -> xyz=0.019200000000000608941 0.00019999999999991205368 -3.986394547794702703e-14 rpy=-3.1415926535897487071 -3.3554531021644002431e-13 4.6155381424903106362e-13
- joint right_hip_yaw_driven: origin xyz=6.7130455500876074463e-18 0 -0.0050000000000000044409 rpy=3.141592653589793116 1.8902520345519600665e-15 6.1775836156745547935e-16 -> xyz=-5.1120132432691534063e-17 -1.1449174941446926823e-16 -0.0050000000000000044409 rpy=3.141592653589793116 1.1586097708402311315e-16 -1.9261630240694359833e-15
- joint right_hip_yaw_fixed: origin xyz=-1.0408340855860842566e-17 0.028000000000000000583 0.023000000000000003081 rpy=1.5707963267948950037 1.5707963267948956698 0 -> xyz=1.1449174941446926823e-16 0.027999999999999990175 0.022999999999999951039 rpy=1.57079632679489678 1.570796326794896336 0
- joint right_knee: limit lower=0 upper=2.0943951023931952626 effort=1 velocity=20 -> lower=0 upper=1.570796326794896558 effort=1 velocity=20; origin xyz=3.8673524714199294822e-17 -0.0087500000000000077716 0.085950000000000234546 rpy=-1.570796326794896558 5.5658335141783220556e-17 1.301042607000131838e-16 -> xyz=9.915028867379938049e-17 -0.0087500000000001326717 0.085950000000000637002 rpy=-1.57079632679489678 -1.8596235662471439105e-15 -1.7091941954032421329e-15
- joint right_knee_act: limit lower=0 upper=2.0943951023931952626 effort=1 velocity=20 -> lower=0 upper=1.570796326794896558 effort=1 velocity=20; origin xyz=-4.6665632433496683265e-17 0.012450000000000016609 0.044500000000000108913 rpy=-1.5707963267949018871 8.0755692215136540146e-16 -1.5223259817910595414e-15 -> xyz=-3.4965520062657517997e-17 0.012449999999999900382 0.044500000000000414224 rpy=-1.5707963267948978903 -1.8873791418627653299e-15 -1.8392984561052994525e-15
- joint right_knee_back_rev_1: origin xyz=-0.005740251485476348392 0.013858192987669312735 0.004999999999999997502 rpy=-3.1415926535897917837 -8.5513789195627690368e-15 -1.5719616139296870294 -> xyz=-0.005740251485476307626 0.013858192987669243346 0.0050000000000000209208 rpy=-3.1415926535897926719 -7.2263408907627713374e-17 -1.5696756685021302502
- joint right_knee_back_rev_2: origin xyz=-0.0057402514854763449226 0.013858192987669326612 0.026200000000000008005 rpy=3.141592653589793116 1.3394980314611144159e-14 1.5696310396601069748 -> xyz=-0.0057402514854763934948 0.013858192987669021301 0.026199999999999980249 rpy=3.1415926535897922278 -1.6769178092422380047e-15 1.5719169850876628658
- joint right_knee_front_rev_1: origin xyz=0.0057402514854764212504 -0.013858192987669271101 0.005000000000001107725 rpy=-3.1415926535897922278 1.4155199868557711964e-15 -1.5696230531921417928 -> xyz=0.0057402514854763813518 -0.013858192987669354368 0.0049999999999999922978 rpy=-3.141592653589793116 -2.2680076696535559301e-15 -1.5696821854497560178
- joint right_knee_front_rev_2: origin xyz=0.0057402514854765279359 -0.013858192987670742147 0.026200000000002138245 rpy=-3.1415926535897917837 3.3833886305441284356e-15 1.5719696003976522114 -> xyz=0.0057402514854763718108 -0.013858192987669770702 0.026200000000000028821 rpy=3.141592653589793116 4.7532333134949093273e-16 1.5719104681400370982

File: toddlerbot/descriptions/assemblies/toddlerbot_2xm/toddlerbot_2xm.urdf (robot description, URDF)
Before this commit: robot toddlerbot_2xm, 17 links, 16 joints
Links:
- link head: mass 0.13722101760550839411 -> 0.13722101760550831084
- link motor_plate: mass 0.0016999999999999999053 -> 0.0016999999999999996884
- link neck_rod: mass 0.003162946861306418795 -> 0.0031629468613064179276
- link neck_rod_2: mass 0.003162946861306418795 -> 0.0031629468613064179276
- link neck_yaw_link_v2: mass 0.0067298837334394106396 -> 0.0067298837334394071702
- link pelvis_link: mass 0.10819999998618362591 -> 0.10819999998618366754
- link spiral_bevel_1m_14t_30deg: mass 0.00073261524436595481732 -> 0.00073261524436595492574
- link spiral_bevel_1m_14t_30deg_2: mass 0.00073261524436595481732 -> 0.00073261524436595492574
- link spur_1m_20t: mass 0.0015778025963746002049 -> 0.0015778025963745997712
- link torso: mass 0.76506596310119379112 -> 0.76506596310120122961
- link waist_gears: mass 0.026337180140419174518 -> 0.026337180140419177987
Joints:
- joint left_hip_pitch: origin xyz=0.056000000000000015044 -0.048100000000000017741 -0.022750000000000002859 rpy=-1.570796326794896558 1.6987796761745309088e-13 1.5707963267948961139 -> xyz=0.018000000000000015987 -0.048100000000000003864 -0.022750000000000006328 rpy=-1.570796326794896558 1.6504994128029653493e-13 1.570796326794901443
- joint left_sho_pitch: origin xyz=-0.0035000000000004853618 0.067000000000001086464 0.104236510762817286 rpy=-1.5707963267949092145 -4.1272540940440295364e-14 3.4662501019292450252e-14 -> xyz=-0.003500000000000471484 0.067000000000001072586 0.10423651076281729988 rpy=-1.5707963267949092145 -4.1300296516055854858e-14 3.4824310043944882416e-14
- joint neck_pitch: origin xyz=5.9674487573602164048e-16 0.0039999999999998587033 0.019399999999999806288 rpy=-1.5707963267948521491 1.5425174793631615255 3.1415926535897376048 -> xyz=5.2041704279304212832e-17 0.0039999999999999775319 0.0194000000000001116 rpy=-1.5707963267949143216 1.5425174793626117431 -3.141592653589773132
- joint neck_pitch_act: origin xyz=-0.032615697718560265894 -0.026999999999999926836 0.0024999999999994306291 rpy=-3.1415926535897717997 -2.7362616902435156123e-13 -3.1097313972841367224 -> xyz=-0.032615697718561015295 -0.026999999999999690914 0.0024999999999997845126 rpy=-3.1415926535897686911 -2.172400990893164017e-13 -3.1097313972849995878
- joint neck_pitch_back_rev_1: origin xyz=0.0072444436971678752291 -0.0040000000000001284528 0.021341142838268850612 rpy=1.5707963267948570341 -0.90902509982357204699 -3.1415926535897757965 -> xyz=0.0072444436971680417625 -0.0040000000000000339104 0.021341142838269072657 rpy=1.5707963267948958919 -0.9090250998239748359 3.1415926535897904515
- joint neck_pitch_back_rev_2: origin xyz=0.0019411428382691275907 0.0072444436971684199322 -0.0055000000000000586614 rpy=-2.3236823215650819985e-13 -1.4353241018555422443e-13 0.9126075086974965167 -> xyz=0.0019411428382689610572 0.0072444436971680226806 -0.005499999999999985803 rpy=-1.8767779702219551721e-13 -1.1288623462566221499e-13 0.91260750869648277206
- joint neck_pitch_front_rev_1: origin xyz=-0.0072444436971683227877 -0.0039999999999998803873 0.017458857161730817475 rpy=1.5707963267944347052 -0.90616957752271976023 -3.1415926535894160843 -> xyz=-0.0072444436971680417625 -0.0040000000000000599312 0.017458857161731150542 rpy=1.5707963267945426189 -0.90616957752344262644 -3.1415926535894937999
- joint neck_pitch_front_rev_2: origin xyz=-0.0019411428382686279903 -0.0072444436971679376791 -0.0055000000000000369774 rpy=1.0105280306711553975e-15 1.7427548910439371813e-15 0.90975198639664878186 -> xyz=-0.0019411428382688222793 -0.0072444436971680035986 -0.0054999999999999805989 rpy=-5.1957590769503590071e-16 7.0973975406608356491e-16 0.90975198639595111771
- joint neck_yaw_driven: origin xyz=0.016000000000000631772 -2.5386894722087491882e-18 0.12248651076281739936 rpy=-1.3877787815156550368e-16 4.0151578034893139621e-15 -8.6007558735577509564e-16 -> xyz=0.016000000000000624834 3.2103613134323069307e-17 0.12248651076281735772 rpy=-1.2490009034196296056e-15 7.5678714822898148914e-15 -8.6007558735577479982e-16
- joint right_hip_pitch: origin xyz=-0.056000000000000001166 -0.048100000000000017741 -0.022750000000000002859 rpy=1.570796326794896558 1.7781396319001008764e-13 1.570796326794896558 -> xyz=-0.018000000000000012518 -0.048100000000000017741 -0.022750000000000002859 rpy=1.570796326794896558 1.5655006806055883195e-13 1.570796326794896336
- joint right_sho_pitch: origin xyz=-0.003499999999998689923 -0.067000000000001017075 0.10423651076281731376 rpy=-1.5707963267948872321 3.5848643389728309658e-14 -3.1415926535897553684 -> xyz=-0.003499999999998689923 -0.067000000000001017075 0.10423651076281729988 rpy=-1.5707963267948874542 3.1641356201815939038e-14 -3.1415926535897420457
- joint waist_act_1: origin xyz=3.9653392986298993667e-17 -0.019600000000000013245 -0.012749999999999992242 rpy=1.5707963267948961139 4.5753542983692753168e-16 3.1415926535897913396 -> xyz=3.7125771266094977152e-17 -0.019600000000000020184 -0.012750000000000000916 rpy=1.570796326794896558 2.7529416277864663811e-15 -3.1415926535897913396
- joint waist_act_2: origin xyz=-2.5609669340318885381e-17 -0.019600000000000027123 -0.032750000000000001332 rpy=-1.5707963267948972241 3.058520389072880007e-17 3.1415926535897900074 -> xyz=8.2006622604210144818e-18 -0.019599999999999999367 -0.032750000000000001332 rpy=-1.570796326794896558 -5.4984382998055662717e-16 -3.1415926535897922278
- joint waist_roll: origin xyz=-0.022707865260692457893 -1.1505205732191483283e-18 -0.014000000000000000291 rpy=1.5707963267948970021 -1.1431802952161779006e-14 -1.57079632679489678 -> xyz=-0.022707865260687083719 -1.1505205732202515009e-18 -0.014000000000000000291 rpy=1.5707963267948970021 -3.0586650082910413294e-14 -1.57079632679489678
